Commit message: Amazon Robot: Lift link actuation works

File: amazon_robot/amazon_robot_description/urdf/amazon_robot_xacro_generated.urdf (robot description, URDF)
Before this commit: robot amazon_robot2, 10 links, 9 joints
Joints:
- joint lift_joint: limit lower=-0.05 upper=0.24 effort=10000.0 velocity=0.5 -> lower=0.20 upper=0.30 effort=10000.0 velocity=5

Commit message: Amazon Robot: Lift + Actuation + Navigation working

File: amazon_robot/amazon_robot_description/urdf/amazon_robot_xacro_generated.urdf (robot description, URDF)
Before this commit: robot amazon_robot2, 10 links, 9 joints
Joints:
- removed joint scan_joint
- added joint lidar_joint: type fixed, parent base_link, child base_scan, origin xyz=-0.064 0 0.244 rpy=0 0 0
- joint lift_joint: axis 0 0 1 -> ; limit lower=0.20 upper=0.30 effort=10000.0 velocity=5 -> lower=0.20 upper=0.30 effort=190.0 velocity=5.89; origin xyz=0 0 0.16 rpy=0. 0. 0. -> (none)
- joint platform_joint: origin xyz=0.0 0 0.20 rpy=0. 0. 0. -> xyz=-0.02 0.0 0.30 rpy=0. 0. 0.

Commit message: Amazon Robot: Working logic, but gazebo issues

File: amazon_robot/amazon_robot_description/urdf/amazon_robot_xacro_generated.urdf (robot description, URDF)
Before this commit: robot amazon_robot2, 10 links, 9 joints
Joints:
- joint wheel_left_joint: origin xyz=0.0 0.288 0.023 rpy=-1.57 0 0 -> xyz=0.0 0.288 0.046 rpy=-1.57 0 0
- joint wheel_right_joint: origin xyz=0.0 -0.288 0.023 rpy=-1.57 0 0 -> xyz=0.0 -0.288 0.046 rpy=-1.57 0 0

Commit message: Amazon Robot: Added Depth Sensor

File: amazon_robot/amazon_robot_description/urdf/amazon_robot_xacro_generated.urdf (robot description, URDF)
Before this commit: robot amazon_robot2, 10 links, 9 joints
Links:
- added link camera_depth_frame
- added link camera_depth_optical_frame
- added link camera_rgb_frame
- added link camera_rgb_optical_frame
Joints:
- added joint camera_depth_joint: type fixed, parent camera_rgb_frame, child camera_depth_frame, origin xyz=0.005 0.028 0.013 rpy=0 0 0
- added joint camera_depth_optical_joint: type fixed, parent camera_depth_frame, child camera_depth_optical_frame, origin xyz=0 0 0 rpy=-1.57 0 -1.57
- added joint camera_joint: type fixed, parent base_link, child camera_rgb_frame, origin xyz=0.23 0 0.23 rpy=0 0 0
- added joint camera_rgb_joint: type fixed, parent base_link, child camera_rgb_frame, origin xyz=0.23 0 0.23 rpy=0 0 0
- added joint camera_rgb_optical_joint: type fixed, parent camera_rgb_frame, child camera_rgb_optical_frame, origin xyz=0 0 0 rpy=-1.57 0 -1.57

Commit message: Amazon Robot: Costmap Works, but FollowPath/ BT Navigator dies

File: amazon_robot/amazon_robot_description/urdf/amazon_robot_xacro_generated.urdf (robot description, URDF)
Before this commit: robot amazon_robot2, 14 links, 14 joints
Joints:
- joint lift_joint: limit lower=0.20 upper=0.30 effort=190.0 velocity=5.89 -> lower=0.20 upper=0.30 effort=20.0 velocity=5.00
