Commit message: CustomRobots is now a ros2 package
Signed-off-by: Blanca <b.soriar.2019@alumnos.urjc.es>

File: CustomRobots/turtlebot2/kobuki_description/urdf/kobuki.urdf.xacro (robot description, xacro)
@@ -4,9 +4,9 @@
   be incorporated by other urdf files (e.g. turtlebot).
   See kobuki_standalone.urdf.xacro for a standalone urdf to be tested with
-      kobuki_description/launch/view_model.launch
+      custom_robots/launch/view_model.launch
  -->
 <robot name="kobuki" xmlns:xacro="http://ros.org/wiki/xacro">
-  <xacro:include filename="$(find kobuki_description)/urdf/common_properties.urdf.xacro"/>
-  <xacro:include filename="$(find kobuki_description)/urdf/kobuki_gazebo.urdf.xacro"/>
+  <xacro:include filename="$(find custom_robots)/urdf/common_properties.urdf.xacro"/>
+  <xacro:include filename="$(find custom_robots)/urdf/kobuki_gazebo.urdf.xacro"/>
   <!-- Kobuki -->
   <xacro:macro name="kobuki">
@@ -30,5 +30,5 @@
         <geometry>
           <!-- new mesh -->
-          <mesh filename="package://kobuki_description/meshes/main_body.dae" />
+          <mesh filename="package://custom_robots/meshes/main_body.dae" />
         </geometry>
         <origin xyz="0.001 0 0.05199" rpy="0 0 0"/>
@@ -65,5 +65,5 @@
       <visual>
         <geometry>
-          <mesh filename="package://kobuki_description/meshes/wheel.dae"/>
+          <mesh filename="package://custom_robots/meshes/wheel.dae"/>
         </geometry>
         <origin xyz="0 0 0" rpy="0 0 0"/>
@@ -92,5 +92,5 @@
       <visual>
         <geometry>
-          <mesh filename="package://kobuki_description/meshes/wheel.dae"/>
+          <mesh filename="package://custom_robots/meshes/wheel.dae"/>
         </geometry>
         <origin xyz="0 0 0" rpy="0 0 0"/>

File: CustomRobots/turtlebot2/kobuki_description/urdf/kobuki_standalone.urdf.xacro (robot description, xacro)
@@ -6,5 +6,5 @@
        xmlns:xacro="http://ros.org/wiki/xacro">
   <!-- Defines the kobuki component tag. -->
-  <xacro:include filename="$(find kobuki_description)/urdf/kobuki.urdf.xacro" />
+  <xacro:include filename="$(find custom_robots)/urdf/kobuki.urdf.xacro" />
   <xacro:kobuki/>
 </robot>

File: CustomRobots/turtlebot2/turtlebot2/urdf/turtlebot2.urdf (robot description, URDF)
Before this commit: robot turtlebot2, 24 links, 23 joints
Links:
- link base_link: geometry collision cylinder length=0.10938 radius=0.178; visual mesh filename=package://custom_robots/meshes/main_body.dae
- link wheel_left_link: geometry collision cylinder length=0.0206 radius=0.035; visual mesh filename=package://custom_robots/meshes/wheel.dae
- link wheel_right_link: geometry collision cylinder length=0.0206 radius=0.035; visual mesh filename=package://custom_robots/meshes/wheel.dae

File: CustomRobots/turtlebot2/turtlebot2/urdf/turtlebot2.urdf.xacro (robot description, xacro)
@@ -1,9 +1,9 @@
 <?xml version="1.0" ?>
 <robot name="turtlebot2" xmlns:xacro="http://ros.org/wiki/xacro">
-  <xacro:include filename="$(find kobuki_description)/urdf/kobuki.urdf"/>
-  <xacro:include filename="$(find turtlebot2)/urdf/sensors/camera.urdf.xacro"/>
-  <xacro:include filename="$(find turtlebot2)/urdf/sensors/lidar.urdf.xacro"/>
-  <xacro:include filename="$(find turtlebot2)/urdf/structures.urdf.xacro"/>
-  <xacro:include filename="$(find turtlebot2)/urdf/colors.urdf.xacro"/>
+  <xacro:include filename="$(find custom_robots)/urdf/kobuki.urdf"/>
+  <xacro:include filename="$(find custom_robots)/urdf/sensors/camera.urdf.xacro"/>
+  <xacro:include filename="$(find custom_robots)/urdf/sensors/lidar.urdf.xacro"/>
+  <xacro:include filename="$(find custom_robots)/urdf/structures.urdf.xacro"/>
+  <xacro:include filename="$(find custom_robots)/urdf/colors.urdf.xacro"/>
   <xacro:cylinder_structure name="base_tick1" x="0.08" y="0.14" z="0.25" length="0.35" radius="0.005" parent="base_link"/>
   <xacro:cylinder_structure name="base_tick2" x="-0.09" y="0.12" z="0.25" length="0.35" radius="0.005" parent="base_link"/>
