Commit message: Fixing turtlebot paths

File: CustomRobots/turtlebot3/urdf/turtlebot3_waffle.urdf (robot description, URDF)
Before this commit: robot turtlebot3_waffle, 13 links, 12 joints
Links:
- link base_link: geometry collision box size=0.266 0.266 0.094; visual mesh filename=package://turtlebot3/models/turtlebot3_common/meshes/waffle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 scale=0.001 0.001 0.001
- link base_scan: geometry collision cylinder length=0.0315 radius=0.055; visual mesh filename=package://turtlebot3/models/turtlebot3_common/meshes/lds.dae scale=0.001 0.001 0.001
- link camera_link: geometry collision box size=0.012 0.132 0.020; visual mesh filename=package://turtlebot3/models/turtlebot3_common/meshes/r200.d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
- link wheel_left_link: geometry collision cylinder length=0.018 radius=0.033; visual mesh filename=package://turtlebot3/models/turtlebot3_common/meshes/tire.d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 scale=0.001 0.001 0.001
- link wheel_right_link: geometry collision cylinder length=0.018 radius=0.033; visual mesh filename=package://turtlebot3/models/turtlebot3_common/meshes/tire.d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 scale=0.001 0.001 0.001
