Commit message: Update f1redbull.urdf

File: CustomRobots/f1/models/f1_redBull/f1redbull.urdf (robot description, URDF)
Before this commit: robot f1_renault, 1 links, 0 joints
Links:
- link f1: geometry visual mesh filename=package://f1/models/f1_redBull/Redbull/Car.obj scale=0.2 0.2 0.2; visual sphere radius=.005
