Commit message: urdf edit

File: CustomRobots/ackermann_cars/models/lincoln/lincoln.urdf (robot description, URDF)
Before this commit: robot lincoln, 10 links, 9 joints
Links:
- link lidar_link: geometry visual cylinder length=0.18 radius=0.0508; visual sphere radius=0.5

File: CustomRobots/ackermann_logistic_robot/models/ackermann_logistic_robot/ackermannLogisticRobot.urdf (robot description, URDF)
Before this commit: robot ackermann_logistic_robot, 9 links, 8 joints
Links:
- link chassis_link: geometry visual mesh filename=package://ackermann_logistic_robot/models/ackermann_logisti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 scale=0.5 0.5 0.5; visual sphere radius=0.25

File: CustomRobots/drone_assets/models/typhoon_h480_dual_cam/typhoon.urdf (robot description, URDF)
Before this commit: robot typhoon_h480_dual_cam, 13 links, 13 joints
Links:
- link base_link: geometry visual mesh filename=package://drone_assets/models/typhoon_h480_dual_cam/meshes/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 scale=0.001 0.001 0.001; visual sphere radius=0.15

File: CustomRobots/f1/models/f1_astonMartin/f1Aston.urdf (robot description, URDF)
Before this commit: robot f1_renault, 1 links, 0 joints
Links:
- link f1: geometry visual mesh filename=package://f1/models/f1_astonMartin/AstonMartin/Car.obj scale=0.2 0.2 0.2; visual sphere radius=0.1

File: CustomRobots/f1/models/f1_redBull/f1redbull.urdf (robot description, URDF)
Before this commit: robot f1_RedBull, 1 links, 0 joints
Links:
- link f1: geometry visual mesh filename=package://f1/models/f1_redBull/Redbull/Car.obj scale=0.2 0.2 0.2; visual sphere radius=0.1

File: CustomRobots/f1/models/f1_renault/f1renault.urdf (robot description, URDF)
Before this commit: robot f1_renault, 1 links, 0 joints
Links:
- link f1: geometry visual mesh filename=package://f1/models/f1_renault/Renault/Car.obj scale=0.2 0.2 0.2; visual sphere radius=0.1

File: CustomRobots/taxi_navigator/models/prius/urdf/prius.urdf (robot description, URDF)
Before this commit: robot prius, 28 links, 27 joints
Links:
- link chassis: geometry collision box size=1.168381 1.654253 0.272347; collision box size=1.267845 1.116344 0.244286

File: CustomRobots/turtlebot3/urdf/turtlebot3_waffle.urdf (robot description, URDF)
Before this commit: robot turtlebot3_waffle, 13 links, 12 joints
Links:
- link base_link: geometry collision box size=0.266 0.266 0.094; visual mesh filename=package://turtlebot3/models/turtlebot3_common/meshes/waffle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 scale=0.001 0.001 0.001
