Commit message: changing urdf

File: CustomRobots/roverrobotics_description/urdf/rover_4wd.urdf (robot description, URDF)
Before this commit: robot rover_4wd, 6 links, 5 joints
Links:
- link chassis_link: geometry collision mesh filename=package://roverrobotics_description/meshes/flipper_chassis.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; collision mesh filename=package://roverrobotics_description/meshes/flipper_track.dae
- link fl_wheel_link: geometry collision mesh filename=package://roverrobotics_description/meshes/pro_tire.dae; visual mesh filename=package://roverrobotics_description/meshes/pro_tire.dae
- link fr_wheel_link: geometry collision mesh filename=package://roverrobotics_description/meshes/pro_tire.dae; visual mesh filename=package://roverrobotics_description/meshes/pro_tire.dae
- link rl_wheel_link: geometry collision mesh filename=package://roverrobotics_description/meshes/pro_tire.dae; visual mesh filename=package://roverrobotics_description/meshes/pro_tire.dae
- link rr_wheel_link: geometry collision mesh filename=package://roverrobotics_description/meshes/pro_tire.dae; visual mesh filename=package://roverrobotics_description/meshes/pro_tire.dae
