Commit message: added urdfs to robots, glbs to worlds

File: CustomRobots/Turtlebot2/turtlebot2_simulated/turtlebot2/urdf/turtlebot2.urdf (robot description, URDF)
Before this commit: robot turtlebot2, 24 links, 23 joints
Links:
- link base_link: geometry collision cylinder length=0.10938 radius=0.178; visual mesh filename=package://Turtlebot2/turtlebot2_simulated/kobuki_descriptio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
- link wheel_left_link: geometry collision cylinder length=0.0206 radius=0.035; visual mesh filename=package://Turtlebot2/turtlebot2_simulated/kobuki_descriptio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
- link wheel_right_link: geometry collision cylinder length=0.0206 radius=0.035; visual mesh filename=package://Turtlebot2/turtlebot2_simulated/kobuki_descriptio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

File: CustomRobots/amazon_robot/urdf/amazon_robot.urdf (robot description, URDF)
Before this commit: robot amazon_robot, 15 links, 14 joints
Links:
- link base_link: geometry collision box size=0.532 0.532 0.188; visual mesh filename=package://amazon_robot/meshes/bases/waffle_pi_base.stl scale=0.002 0.002 0.002

File: CustomRobots/taxi_navigator/models/prius/urdf/prius.urdf (robot description, URDF)
Before this commit: robot prius, 28 links, 27 joints
Links:
- link chassis: geometry collision box size=1.168381 1.654253 0.272347; collision box size=1.267845 1.116344 0.244286
- link front_left_wheel: geometry collision sphere radius=0.31265; visual mesh filename=package://taxi_navigator/models/prius/meshes/wheel.obj scale=0.01 0.01 0.01
- link front_right_wheel: geometry collision sphere radius=0.31265; visual mesh filename=package://taxi_navigator/models/prius/meshes/wheel.obj scale=0.01 0.01 0.01
- link rear_left_wheel: geometry collision sphere radius=0.31265; visual mesh filename=package://taxi_navigator/models/prius/meshes/wheel.obj scale=0.01 0.01 0.01
- link rear_right_wheel: geometry collision sphere radius=0.31265; visual mesh filename=package://taxi_navigator/models/prius/meshes/wheel.obj scale=0.01 0.01 0.01
- link steering_wheel: geometry visual mesh filename=package://taxi_navigator/models/prius/meshes/steering_wheel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 scale=0.01 0.01 0.01

Commit message: adjusted turtlebot2 camera angle

File: CustomRobots/Turtlebot2/turtlebot2_simulated/turtlebot2/urdf/turtlebot2.urdf (robot description, URDF)
Before this commit: robot turtlebot2, 24 links, 23 joints
Joints:
- joint camera_joint: origin xyz=0.13 0 0.32 rpy=0 0 0 -> xyz=0.13 0 0.32 rpy=0 -0.32 0
