Commit message: Update path

File: CustomRobots/f1/models/f1_renault_laser_no_cam_classic/f1renaultLaserNoCamClassic.urdf (robot description, URDF)
Before this commit: robot f1_renault, 2 links, 1 joints
Links:
- link f1: geometry visual mesh filename=package://f1/models/f1_renault_laser_no_cam_classic/Renault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 scale=0.2 0.2 0.2
- link laser_body: geometry visual mesh filename=package://f1/models/f1_renault_laser_no_cam_classic/meshes/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
