Commit message: Ready to test

File: CustomRobots/f1/models/monaco/monaco.urdf (robot description, URDF)
Before this commit: robot circuito, 1 links, 0 joints
Links:
- link link: geometry visual mesh filename=package://f1/models/monaco/meshes/monaco.dae scale=1 1 1; visual mesh filename=package://f1/models/monaco/meshes/monaco_track.dae scale=1 1 1
