Commit message: Fixing paths in robot urdf

File: CustomRobots/rover_4wd_description/urdf/accessories/rover_dev_payload.urdf (robot description, URDF)
Before this commit: robot rover_miti_payload, 1 links, 1 joints
Links:
- link payload_link: geometry collision mesh filename=file://$(find custom_robots)/rover_4wd_description/meshes/r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; visual mesh filename=file://$(find custom_robots)/rover_4wd_description/meshes/r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

File: CustomRobots/rover_4wd_description/urdf/accessories/rplidar_s2.urdf (robot description, URDF)
Before this commit: robot rplidar_s2, 1 links, 1 joints
Links:
- link lidar_link: geometry collision mesh filename=file://$(find custom_robots)/rover_4wd_description/meshes/r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; visual mesh filename=file://$(find custom_robots)/rover_4wd_description/meshes/r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

File: CustomRobots/rover_4wd_description/urdf/rover_4wd.urdf (robot description, URDF)
Before this commit: robot rover_4wd, 6 links, 5 joints
Links:
- link chassis_link: geometry collision mesh filename=file://$(find custom_robots)/rover_4wd_description/meshes/f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; collision mesh filename=file://$(find custom_robots)/rover_4wd_description/meshes/f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
- link fl_wheel_link: geometry collision mesh filename=file://$(find custom_robots)/rover_4wd_description/meshes/p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; visual mesh filename=file://$(find custom_robots)/rover_4wd_description/meshes/p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
- link fr_wheel_link: geometry collision mesh filename=file://$(find custom_robots)/rover_4wd_description/meshes/p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; visual mesh filename=file://$(find custom_robots)/rover_4wd_description/meshes/p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
- link rl_wheel_link: geometry collision mesh filename=file://$(find custom_robots)/rover_4wd_description/meshes/p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; visual mesh filename=file://$(find custom_robots)/rover_4wd_description/meshes/p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
- link rr_wheel_link: geometry collision mesh filename=file://$(find custom_robots)/rover_4wd_description/meshes/p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; visual mesh filename=file://$(find custom_robots)/rover_4wd_description/meshes/p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

Commit message: Removing rover_4wd_description from paths

File: CustomRobots/rover_4wd_description/urdf/accessories/rover_dev_payload.urdf (robot description, URDF)
Before this commit: robot rover_miti_payload, 1 links, 1 joints
Links:
- link payload_link: geometry collision mesh filename=file://$(find custom_robots)/meshes/rover_payload.dae; visual mesh filename=file://$(find custom_robots)/meshes/rover_payload.dae

File: CustomRobots/rover_4wd_description/urdf/accessories/rplidar_s2.urdf (robot description, URDF)
Before this commit: robot rplidar_s2, 1 links, 1 joints
Links:
- link lidar_link: geometry collision mesh filename=file://$(find custom_robots)/meshes/rplidar_s2.dae; visual mesh filename=file://$(find custom_robots)/meshes/rplidar_s2.dae

File: CustomRobots/rover_4wd_description/urdf/rover_4wd.urdf (robot description, URDF)
Before this commit: robot rover_4wd, 6 links, 5 joints
Links:
- link chassis_link: geometry collision mesh filename=file://$(find custom_robots)/meshes/flipper_chassis.dae; collision mesh filename=file://$(find custom_robots)/meshes/flipper_track.dae
- link fl_wheel_link: geometry collision mesh filename=file://$(find custom_robots)/meshes/pro_tire.dae; visual mesh filename=file://$(find custom_robots)/meshes/pro_tire.dae
- link fr_wheel_link: geometry collision mesh filename=file://$(find custom_robots)/meshes/pro_tire.dae; visual mesh filename=file://$(find custom_robots)/meshes/pro_tire.dae
- link rl_wheel_link: geometry collision mesh filename=file://$(find custom_robots)/meshes/pro_tire.dae; visual mesh filename=file://$(find custom_robots)/meshes/pro_tire.dae
- link rr_wheel_link: geometry collision mesh filename=file://$(find custom_robots)/meshes/pro_tire.dae; visual mesh filename=file://$(find custom_robots)/meshes/pro_tire.dae
