Commit message: changes gz classic ackerman robot, frame correction

File: CustomRobots/ackermann_logistic_robot/models/ackermann_logistic_robot/ackermannLogisticRobot.urdf (robot description, URDF)
Before this commit: robot ackermann_logistic_robot, 9 links, 8 joints
Joints:
- added joint base_to_chassis: type fixed, parent , child , origin xyz=0 0 0 rpy=0 0 1.5707963

Commit message: fix rotation on base link

File: CustomRobots/ackermann_logistic_robot/models/ackermann_logistic_robot/ackermannLogisticRobot.urdf (robot description, URDF)
Before this commit: robot ackermann_logistic_robot, 9 links, 9 joints
Joints:
- removed joint base_to_chassis
- joint chassis_link_joint: origin xyz=0.0 0.0 0.0 rpy=0 0 0 -> xyz=0.0 0.0 0.0 rpy=0 0 -1.5707963

Commit message: rotate link

File: CustomRobots/ackermann_logistic_robot/models/ackermann_logistic_robot/ackermannLogisticRobot.urdf (robot description, URDF)
Before this commit: robot ackermann_logistic_robot, 9 links, 8 joints
Joints:
- joint chassis_link_joint: child chassis_link -> ; origin xyz=0.0 0.0 0.0 rpy=0 0 -1.5707963 -> (none); parent base_link -> 
