Commit message: Fix robot model

File: Industrial/ur5_gripper_description/urdf/ur5_robotiq_2f85_with_cams.urdf.xacro (robot description, xacro)
@@ -1,51 +1,7 @@
-<?xml version="1.0" ?>
-<!--
-# ===================================== COPYRIGHT ===================================== #
-#                                                                                       #
-#  IFRA (Intelligent Flexible Robotics and Assembly) Group, CRANFIELD UNIVERSITY        #
-#  Created on behalf of the IFRA Group at Cranfield University, United Kingdom          #
-#  E-mail: IFRA@cranfield.ac.uk                                                         #
-#                                                                                       #
-#  Licensed under the Apache-2.0 License.                                               #
-#  You may not use this file except in compliance with the License.                     #
-#  You may obtain a copy of the License at: http://www.apache.org/licenses/LICENSE-2.0  #
-#                                                                                       #
-#  Unless required by applicable law or agreed to in writing, software distributed      #
-#  under the License is distributed on an "as-is" basis, without warranties or          #
-#  conditions of any kind, either express or implied. See the License for the specific  #
-#  language governing permissions and limitations under the License.                    #
-#                                                                                       #
-#  IFRA Group - Cranfield University                                                    #
-#  AUTHORS: Mikel Bueno Viso - Mikel.Bueno-Viso@cranfield.ac.uk                         #
-#           Dr. Seemal Asif  - s.asif@cranfield.ac.uk                                   #
-#           Prof. Phil Webb  - p.f.webb@cranfield.ac.uk                                 #
-#                                                                                       #
-#  Date: April, 2023.                                                                   #
-#                                                                                       #
-# ===================================== COPYRIGHT ===================================== #
-# ======= CITE OUR WORK ======= #
-# You can cite our work with the following statement:
-# IFRA-Cranfield (2023) ROS 2 Sim-to-Real Robot Control. URL: https://github.com/IFRA-Cranfield/ros2_SimRealRobotControl.
--->
+<?xml version="1.0"?>
 <robot name="ur5" xmlns:xacro="http://ros.org/wiki/xacro">
-  <!-- PASS ARGUMENTS: -->
-  <xacro:arg name="bringup" default="false"/>
-  <xacro:property name="bringup" value="$(arg bringup)"/>
   <xacro:arg name="hmi" default="false"/>
-  <xacro:property name="hmi" value="$(arg hmi)"/>
-  <xacro:arg name="robot_ip" default="0.0.0.0"/>
-  <xacro:property name="robot_ip" value="$(arg robot_ip)"/>
-  <xacro:arg name="EE" default="false"/>
-  <xacro:property name="EE" value="$(arg EE)"/>
-  <xacro:arg name="EE_name" default="none"/>
-  <xacro:property name="EE_name" value="$(arg EE_name)"/>
-  <!-- UR5 Control ARGUMENTS -->
-  <xacro:arg name="script_filename" default="none"/>
-  <xacro:property name="script_filename" value="$(arg script_filename)"/>
-  <xacro:arg name="input_recipe_filename" default="none"/>
-  <xacro:property name="input_recipe_filename" value="$(arg input_recipe_filename)"/>
-  <xacro:arg name="output_recipe_filename" default="none"/>
-  <xacro:property name="output_recipe_filename" value="$(arg output_recipe_filename)"/>
-  <!-- Include XACRO-MACRO file of the UR5: -->
+  <xacro:arg name="EE" default="true"/>
+  <xacro:arg name="EE_name" default="robotiq_2f85"/>
   <xacro:include filename="$(find ros2srrc_robots)/ur5/urdf/ur5_macro.urdf.xacro"/>
   <xacro:include filename="$(find ros2srrc_ur5_gazebo)/urdf/common_properties.xacro"/>
@@ -54,74 +10,52 @@
   <xacro:include filename="$(find ros2srrc_ur5_gazebo)/urdf/cam_on_base_params.xacro"/>
   <xacro:include filename="$(find ros2srrc_ur5_gazebo)/urdf/cam_on_base.xacro"/>
+  <xacro:include filename="$(find ros2srrc_endeffectors)/robotiq_2f85/urdf/robotiq_2f85_macro.urdf.xacro"/>
   <xacro:ur5
-    bringup="${bringup}"
-    robot_ip="${robot_ip}"
+    bringup="false"
+    robot_ip="0.0.0.0"
     EE="${EE}"
     EE_name="${EE_name}"
-    script_filename="${script_filename}"
-    input_recipe_filename="${input_recipe_filename}"
-    output_recipe_filename="${output_recipe_filename}"
+    script_filename="none"
+    input_recipe_filename="none"
+    output_recipe_filename="none"
   />
-  <!-- Include XACRO-MACRO file of the Robotiq 2f-85: -->
-  <xacro:include filename="$(find ros2srrc_endeffectors)/robotiq_2f85/urdf/robotiq_2f85_macro.urdf.xacro"/>
   <xacro:robotiq_2f85
-    bringup="${bringup}"
+    bringup="false"
     parent_link="tool0"
   />
-  <!-- Load ROS 2 Gazebo Plugin -->
-  <xacro:unless value="${bringup}">
-    <gazebo>
-        <plugin filename="gz_ros2_control-system" name="gz_ros2_control">
-            <robot_sim_type>gz_ros2_control/GazeboSimSystem</robot_sim_type>
-            <parameters>$(find ros2srrc_robots)/ur5/config/controller.yaml</parameters>
-            <parameters>$(find ros2srrc_endeffectors)/${EE_name}/config/controller.yaml</parameters>
-        </plugin>
-    </gazebo>
-  </xacro:unless>
-  <!-- World: LINK -->
   <link name="world"/>
-  <!-- Robot Stand: LINK -->
-  <link name='robot_stand'>
-    <inertial>
-      <origin xyz="0 0 0" rpy="0 0 0"/>
-      <mass value="100"/>
-      <inertia ixx="0.01"  ixy="0"  ixz="0" iyy="0.01" iyz="0" izz="0.01" />
-    </inertial>
-    <collision name='collision'>
-      <origin xyz="0 0 0" rpy=" 0 0 0"/>
+  <link name="robot_stand">
+    <visual>
       <geometry>
-        <box size = "0.2 0.2 1.0"/>
+        <box size="0.2 0.2 1.0"/>
+      </geometry>
+    </visual>
+    <collision>
+      <geometry>
+        <box size="0.2 0.2 1.0"/>
       </geometry>
     </collision>
-    <visual name='chassis_visual'>
-      <origin xyz="0 0 0" rpy=" 0 0 0"/>
-      <geometry>
-        <box size = "0.2 0.2 1.0"/>
-      </geometry>
-    </visual>
+    <inertial>
+      <mass value="100"/>
+      <inertia ixx="0.01" iyy="0.01" izz="0.01"
+               ixy="0" ixz="0" iyz="0"/>
+    </inertial>
   </link>
-  <!-- Robot Stand: FIXED JOINT -->
   <joint name="world_joint" type="fixed">
-    <parent link= "world" />
-    <child link = "robot_stand" />
-    <origin xyz="0.0 0.0 0.5" rpy="0.0 0.0 0.0" />
+    <parent link="world"/>
+    <child link="robot_stand"/>
+    <origin xyz="0 0 0.5"/>
   </joint>
-  <!-- Robot Stand: Robot+Stand JOINT -->
   <joint name="stand_joint" type="fixed">
-    <parent link= "robot_stand" />
-    <child link = "base_link" />
-    <origin xyz="0.0 0.0 0.52" rpy="0.0 0.0 0.0" />
+    <parent link="robot_stand"/>
+    <child link="base_link"/>
+    <origin xyz="0 0 0.52"/>
   </joint>
-  <!-- ros2srrc_HMI CAMERA -->
-  <xacro:if value="${hmi}">
-    <xacro:include filename="$(find ros2srrc_hmi)/urdf/hmicamera.urdf.xacro"/>
-    <xacro:HMI_camera
-      x="2.5"
-      y="1.50"
-      z="2.0"
-      roll="0.0"
-      pitch="0.35"
-      yaw="-2.6"
-    />
-  </xacro:if>
+  <gazebo>
+    <plugin filename="gz_ros2_control-system" name="gz_ros2_control">
+      <robot_sim_type>gz_ros2_control/GazeboSimSystem</robot_sim_type>
+      <parameters>$(find ros2srrc_robots)/ur5/config/controller.yaml</parameters>
+      <parameters>$(find ros2srrc_endeffectors)/${EE_name}/config/controller.yaml</parameters>
+    </plugin>
+  </gazebo>
 </robot>

Commit message: Fix robot model

File: Industrial/ur5_gripper_description/urdf/ur5_robotiq_2f85_with_cams.urdf.xacro (robot description, xacro)
@@ -4,4 +4,6 @@
   <xacro:arg name="EE" default="true"/>
   <xacro:arg name="EE_name" default="robotiq_2f85"/>
+  <xacro:property name="EE" value="$(arg EE)"/>
+  <xacro:property name="EE_name" value="$(arg EE_name)"/>
   <xacro:include filename="$(find ros2srrc_robots)/ur5/urdf/ur5_macro.urdf.xacro"/>
   <xacro:include filename="$(find ros2srrc_ur5_gazebo)/urdf/common_properties.xacro"/>
@@ -14,6 +16,6 @@
     bringup="false"
     robot_ip="0.0.0.0"
-    EE="${EE}"
-    EE_name="${EE_name}"
+    EE="$(arg EE)"
+    EE_name="$(arg EE_name)"
     script_filename="none"
     input_recipe_filename="none"
@@ -56,5 +58,5 @@
       <robot_sim_type>gz_ros2_control/GazeboSimSystem</robot_sim_type>
       <parameters>$(find ros2srrc_robots)/ur5/config/controller.yaml</parameters>
-      <parameters>$(find ros2srrc_endeffectors)/${EE_name}/config/controller.yaml</parameters>
+      <parameters>$(find ros2srrc_endeffectors)/$(arg EE_name)/config/controller.yaml</parameters>
     </plugin>
   </gazebo>

Commit message: Add meshes, fix renders and change arm position

File: Industrial/ur5_gripper_description/urdf/ur5_robotiq_2f85_with_cams.urdf.xacro (robot description, xacro)
@@ -1,30 +1,30 @@
 <?xml version="1.0"?>
-<robot name="ur5" xmlns:xacro="http://ros.org/wiki/xacro">
-  <xacro:arg name="hmi" default="false"/>
-  <xacro:arg name="EE" default="true"/>
-  <xacro:arg name="EE_name" default="robotiq_2f85"/>
-  <xacro:property name="EE" value="$(arg EE)"/>
-  <xacro:property name="EE_name" value="$(arg EE_name)"/>
-  <xacro:include filename="$(find ros2srrc_robots)/ur5/urdf/ur5_macro.urdf.xacro"/>
-  <xacro:include filename="$(find ros2srrc_ur5_gazebo)/urdf/common_properties.xacro"/>
-  <xacro:include filename="$(find ros2srrc_ur5_gazebo)/urdf/cam_on_hand_params.xacro"/>
-  <xacro:include filename="$(find ros2srrc_ur5_gazebo)/urdf/cam_on_hand.xacro"/>
-  <xacro:include filename="$(find ros2srrc_ur5_gazebo)/urdf/cam_on_base_params.xacro"/>
-  <xacro:include filename="$(find ros2srrc_ur5_gazebo)/urdf/cam_on_base.xacro"/>
-  <xacro:include filename="$(find ros2srrc_endeffectors)/robotiq_2f85/urdf/robotiq_2f85_macro.urdf.xacro"/>
-  <xacro:ur5
-    bringup="false"
-    robot_ip="0.0.0.0"
-    EE="$(arg EE)"
-    EE_name="$(arg EE_name)"
-    script_filename="none"
-    input_recipe_filename="none"
-    output_recipe_filename="none"
+<robot name="ur5" xmlns:xacro="http://www.ros.org/wiki/xacro">
+  <xacro:arg name="sim_gz" default="true"/>
+  <xacro:include filename="$(find ur5_gripper_description)/urdf/ur.urdf.xacro"/>
+  <xacro:include filename="$(find robotiq_description)/urdf/robotiq_85_gripper.urdf.xacro"/>
+  <xacro:include filename="$(find robotiq_description)/urdf/robotiq_85_gripper.ros2_control.xacro"/>
+  <xacro:ur
+    name="ur"
+    ur_type="ur5"
+    prefix=""
+    sim_gz="true"
+    use_fake_hardware="false"
   />
-  <xacro:robotiq_2f85
-    bringup="false"
-    parent_link="tool0"
-  />
-  <link name="world"/>
+  <link name="robotiq_coupler">
+    <visual>
+      <geometry>
+        <mesh filename="package://robotiq_description/meshes/robotiq_85_coupler.stl"/>
+      </geometry>
+    </visual>
+  </link>
+  <joint name="robotiq_coupler_joint" type="fixed">
+    <parent link="tool0"/>
+    <child link="robotiq_coupler"/>
+    <origin xyz="0 0 0.004" rpy="0 0 ${-pi/2}"/>
+  </joint>
+  <xacro:robotiq_85_gripper parent="robotiq_coupler">
+    <origin xyz="0 0 0.004" rpy="0 ${-pi/2} ${pi}"/>
+  </xacro:robotiq_85_gripper>
   <link name="robot_stand">
     <visual>
@@ -44,4 +44,5 @@
     </inertial>
   </link>
+  <link name="world"/>
   <joint name="world_joint" type="fixed">
     <parent link="world"/>
@@ -54,10 +55,69 @@
     <origin xyz="0 0 0.52"/>
   </joint>
-  <gazebo>
-    <plugin filename="gz_ros2_control-system" name="gz_ros2_control">
-      <robot_sim_type>gz_ros2_control/GazeboSimSystem</robot_sim_type>
-      <parameters>$(find ros2srrc_robots)/ur5/config/controller.yaml</parameters>
-      <parameters>$(find ros2srrc_endeffectors)/$(arg EE_name)/config/controller.yaml</parameters>
-    </plugin>
+  <link name="camera_base_link">
+    <visual>
+      <geometry>
+        <box size="0.05 0.05 0.05"/>
+      </geometry>
+      <material>
+        <ambient>0 0 0 1</ambient>
+      </material>
+    </visual>
+  </link>
+  <joint name="camera_base_joint" type="fixed">
+    <parent link="base_link"/>
+    <child link="camera_base_link"/>
+    <origin xyz="0.4 0 1.2" rpy="0 0 0"/>
+  </joint>
+  <gazebo reference="camera_base_link">
+    <sensor name="camera_base" type="camera">
+      <always_on>true</always_on>
+      <update_rate>30</update_rate>
+      <camera>
+        <horizontal_fov>1.047</horizontal_fov>
+        <image>
+          <width>640</width>
+          <height>480</height>
+          <format>R8G8B8</format>
+        </image>
+        <clip>
+          <near>0.1</near>
+          <far>100</far>
+        </clip>
+      </camera>
+    </sensor>
   </gazebo>
+  <link name="camera_hand_link">
+    <visual>
+      <geometry>
+        <box size="0.04 0.04 0.04"/>
+      </geometry>
+      <material>
+        <ambient>0 0 0 1</ambient>
+      </material>
+    </visual>
+  </link>
+  <joint name="camera_hand_joint" type="fixed">
+    <parent link="tool0"/>
+    <child link="camera_hand_link"/>
+    <origin xyz="0.05 0 0.1" rpy="0 0 0"/>
+  </joint>
+  <gazebo reference="camera_hand_link">
+    <sensor name="camera_hand" type="camera">
+      <always_on>true</always_on>
+      <update_rate>30</update_rate>
+      <camera>
+        <horizontal_fov>1.047</horizontal_fov>
+        <image>
+          <width>640</width>
+          <height>480</height>
+          <format>R8G8B8</format>
+        </image>
+      </camera>
+    </sensor>
+  </gazebo>
+  <xacro:robotiq_85_ros2_control
+    name="robotiq"
+    sim_gz="true"
+    use_fake_hardware="false"/>
 </robot>

Commit message: Fix xacro

File: Industrial/ur5_gripper_description/urdf/ur5_robotiq_2f85_with_cams.urdf.xacro (robot description, xacro)
@@ -1,30 +1,30 @@
 <?xml version="1.0"?>
-<robot name="ur5" xmlns:xacro="http://www.ros.org/wiki/xacro">
-  <xacro:arg name="sim_gz" default="true"/>
-  <xacro:include filename="$(find ur5_gripper_description)/urdf/ur.urdf.xacro"/>
-  <xacro:include filename="$(find robotiq_description)/urdf/robotiq_85_gripper.urdf.xacro"/>
-  <xacro:include filename="$(find robotiq_description)/urdf/robotiq_85_gripper.ros2_control.xacro"/>
-  <xacro:ur
-    name="ur"
-    ur_type="ur5"
-    prefix=""
-    sim_gz="true"
-    use_fake_hardware="false"
+<robot name="ur5" xmlns:xacro="http://ros.org/wiki/xacro">
+  <xacro:arg name="hmi" default="false"/>
+  <xacro:arg name="EE" default="true"/>
+  <xacro:arg name="EE_name" default="robotiq_2f85"/>
+  <xacro:property name="EE" value="$(arg EE)"/>
+  <xacro:property name="EE_name" value="$(arg EE_name)"/>
+  <xacro:include filename="$(find ros2srrc_robots)/ur5/urdf/ur5_macro.urdf.xacro"/>
+  <xacro:include filename="$(find ros2srrc_ur5_gazebo)/urdf/common_properties.xacro"/>
+  <xacro:include filename="$(find ros2srrc_ur5_gazebo)/urdf/cam_on_hand_params.xacro"/>
+  <xacro:include filename="$(find ros2srrc_ur5_gazebo)/urdf/cam_on_hand.xacro"/>
+  <xacro:include filename="$(find ros2srrc_ur5_gazebo)/urdf/cam_on_base_params.xacro"/>
+  <xacro:include filename="$(find ros2srrc_ur5_gazebo)/urdf/cam_on_base.xacro"/>
+  <xacro:include filename="$(find ros2srrc_endeffectors)/robotiq_2f85/urdf/robotiq_2f85_macro.urdf.xacro"/>
+  <xacro:ur5
+    bringup="false"
+    robot_ip="0.0.0.0"
+    EE="$(arg EE)"
+    EE_name="$(arg EE_name)"
+    script_filename="none"
+    input_recipe_filename="none"
+    output_recipe_filename="none"
   />
-  <link name="robotiq_coupler">
-    <visual>
-      <geometry>
-        <mesh filename="package://robotiq_description/meshes/robotiq_85_coupler.stl"/>
-      </geometry>
-    </visual>
-  </link>
-  <joint name="robotiq_coupler_joint" type="fixed">
-    <parent link="tool0"/>
-    <child link="robotiq_coupler"/>
-    <origin xyz="0 0 0.004" rpy="0 0 ${-pi/2}"/>
-  </joint>
-  <xacro:robotiq_85_gripper parent="robotiq_coupler">
-    <origin xyz="0 0 0.004" rpy="0 ${-pi/2} ${pi}"/>
-  </xacro:robotiq_85_gripper>
+  <xacro:robotiq_2f85
+    bringup="false"
+    parent_link="tool0"
+  />
+  <link name="world"/>
   <link name="robot_stand">
     <visual>
@@ -44,5 +44,4 @@
     </inertial>
   </link>
-  <link name="world"/>
   <joint name="world_joint" type="fixed">
     <parent link="world"/>
@@ -55,69 +54,10 @@
     <origin xyz="0 0 0.52"/>
   </joint>
-  <link name="camera_base_link">
-    <visual>
-      <geometry>
-        <box size="0.05 0.05 0.05"/>
-      </geometry>
-      <material>
-        <ambient>0 0 0 1</ambient>
-      </material>
-    </visual>
-  </link>
-  <joint name="camera_base_joint" type="fixed">
-    <parent link="base_link"/>
-    <child link="camera_base_link"/>
-    <origin xyz="0.4 0 1.2" rpy="0 0 0"/>
-  </joint>
-  <gazebo reference="camera_base_link">
-    <sensor name="camera_base" type="camera">
-      <always_on>true</always_on>
-      <update_rate>30</update_rate>
-      <camera>
-        <horizontal_fov>1.047</horizontal_fov>
-        <image>
-          <width>640</width>
-          <height>480</height>
-          <format>R8G8B8</format>
-        </image>
-        <clip>
-          <near>0.1</near>
-          <far>100</far>
-        </clip>
-      </camera>
-    </sensor>
+  <gazebo>
+    <plugin filename="gz_ros2_control-system" name="gz_ros2_control">
+      <robot_sim_type>gz_ros2_control/GazeboSimSystem</robot_sim_type>
+      <parameters>$(find ros2srrc_robots)/ur5/config/controller.yaml</parameters>
+      <parameters>$(find ros2srrc_endeffectors)/$(arg EE_name)/config/controller.yaml</parameters>
+    </plugin>
   </gazebo>
-  <link name="camera_hand_link">
-    <visual>
-      <geometry>
-        <box size="0.04 0.04 0.04"/>
-      </geometry>
-      <material>
-        <ambient>0 0 0 1</ambient>
-      </material>
-    </visual>
-  </link>
-  <joint name="camera_hand_joint" type="fixed">
-    <parent link="tool0"/>
-    <child link="camera_hand_link"/>
-    <origin xyz="0.05 0 0.1" rpy="0 0 0"/>
-  </joint>
-  <gazebo reference="camera_hand_link">
-    <sensor name="camera_hand" type="camera">
-      <always_on>true</always_on>
-      <update_rate>30</update_rate>
-      <camera>
-        <horizontal_fov>1.047</horizontal_fov>
-        <image>
-          <width>640</width>
-          <height>480</height>
-          <format>R8G8B8</format>
-        </image>
-      </camera>
-    </sensor>
-  </gazebo>
-  <xacro:robotiq_85_ros2_control
-    name="robotiq"
-    sim_gz="true"
-    use_fake_hardware="false"/>
 </robot>

Commit message: Fix xacro

File: Industrial/ur5_gripper_description/urdf/ur5_robotiq_2f85_with_cams.urdf.xacro (robot description, xacro)
@@ -1,63 +1,38 @@
 <?xml version="1.0"?>
-<robot name="ur5" xmlns:xacro="http://ros.org/wiki/xacro">
-  <xacro:arg name="hmi" default="false"/>
-  <xacro:arg name="EE" default="true"/>
-  <xacro:arg name="EE_name" default="robotiq_2f85"/>
-  <xacro:property name="EE" value="$(arg EE)"/>
-  <xacro:property name="EE_name" value="$(arg EE_name)"/>
-  <xacro:include filename="$(find ros2srrc_robots)/ur5/urdf/ur5_macro.urdf.xacro"/>
-  <xacro:include filename="$(find ros2srrc_ur5_gazebo)/urdf/common_properties.xacro"/>
-  <xacro:include filename="$(find ros2srrc_ur5_gazebo)/urdf/cam_on_hand_params.xacro"/>
-  <xacro:include filename="$(find ros2srrc_ur5_gazebo)/urdf/cam_on_hand.xacro"/>
-  <xacro:include filename="$(find ros2srrc_ur5_gazebo)/urdf/cam_on_base_params.xacro"/>
-  <xacro:include filename="$(find ros2srrc_ur5_gazebo)/urdf/cam_on_base.xacro"/>
-  <xacro:include filename="$(find ros2srrc_endeffectors)/robotiq_2f85/urdf/robotiq_2f85_macro.urdf.xacro"/>
-  <xacro:ur5
-    bringup="false"
-    robot_ip="0.0.0.0"
-    EE="$(arg EE)"
-    EE_name="$(arg EE_name)"
-    script_filename="none"
-    input_recipe_filename="none"
-    output_recipe_filename="none"
-  />
-  <xacro:robotiq_2f85
-    bringup="false"
-    parent_link="tool0"
-  />
-  <link name="world"/>
-  <link name="robot_stand">
+<robot name="ur5" xmlns:xacro="http://www.ros.org/wiki/xacro">
+  <xacro:include filename="$(find ur5_gripper_description)/urdf/ur5_robotiq85_gripper.urdf.xacro"/>
+  <link name="camera_base_link">
     <visual>
       <geometry>
-        <box size="0.2 0.2 1.0"/>
+        <box size="0.05 0.05 0.05"/>
       </geometry>
     </visual>
-    <collision>
+  </link>
+  <joint name="camera_base_joint" type="fixed">
+    <parent link="base_link"/>
+    <child link="camera_base_link"/>
+    <origin xyz="0.4 0 1.2"/>
+  </joint>
+  <gazebo reference="camera_base_link">
+    <sensor name="camera_base" type="camera">
+      <update_rate>30</update_rate>
+    </sensor>
+  </gazebo>
+  <link name="camera_hand_link">
+    <visual>
       <geometry>
-        <box size="0.2 0.2 1.0"/>
+        <box size="0.04 0.04 0.04"/>
       </geometry>
-    </collision>
-    <inertial>
-      <mass value="100"/>
-      <inertia ixx="0.01" iyy="0.01" izz="0.01"
-               ixy="0" ixz="0" iyz="0"/>
-    </inertial>
+    </visual>
   </link>
-  <joint name="world_joint" type="fixed">
-    <parent link="world"/>
-    <child link="robot_stand"/>
-    <origin xyz="0 0 0.5"/>
+  <joint name="camera_hand_joint" type="fixed">
+    <parent link="tool0"/>
+    <child link="camera_hand_link"/>
+    <origin xyz="0.05 0 0.1"/>
   </joint>
-  <joint name="stand_joint" type="fixed">
-    <parent link="robot_stand"/>
-    <child link="base_link"/>
-    <origin xyz="0 0 0.52"/>
-  </joint>
-  <gazebo>
-    <plugin filename="gz_ros2_control-system" name="gz_ros2_control">
-      <robot_sim_type>gz_ros2_control/GazeboSimSystem</robot_sim_type>
-      <parameters>$(find ros2srrc_robots)/ur5/config/controller.yaml</parameters>
-      <parameters>$(find ros2srrc_endeffectors)/$(arg EE_name)/config/controller.yaml</parameters>
-    </plugin>
+  <gazebo reference="camera_hand_link">
+    <sensor name="camera_hand" type="camera">
+      <update_rate>30</update_rate>
+    </sensor>
   </gazebo>
 </robot>
