Commit message: Fix xacro and launcher

File: Industrial/ros2_SimRealRobotControl_gz/packages/ur5/ros2srrc_ur5_gazebo/urdf/ur5_robotiq_2f85.urdf.xacro (robot description, xacro)
@@ -47,4 +47,6 @@
   <xacro:arg name="output_recipe_filename" default="none"/>
   <xacro:property name="output_recipe_filename" value="$(arg output_recipe_filename)"/>
+  <xacro:arg name="simulation_controllers" default=""/>
+  <xacro:property name="simulation_controllers" value="$(arg simulation_controllers)"/>
   <!-- Include XACRO-MACRO file of the UR5: -->
   <xacro:include filename="/home/ws/src/Industrial/ros2_SimRealRobotControl_gz/ros2srrc_robots/ur5/urdf/ur5_macro.urdf.xacro"/>
@@ -73,6 +75,5 @@
           </hardware>
         </ros2_control>
-        <parameters>/home/ws/src/Industrial/ros2_SimRealRobotControl_gz/ros2srrc_robots/ur5/config/controller.yaml</parameters>
-        <parameters>/home/ws/src/Industrial/ros2_SimRealRobotControl_gz/ros2srrc_endeffectors/${EE_name}/config/controller.yaml</parameters>
+        <parameters>${simulation_controllers}</parameters>
       </plugin>
       <plugin filename="libgz_mimic_joint.so" name="gz_mimic_joint">
