Commit message: Migrate cameras to harmonic

File: Industrial/ros2_SimRealRobotControl_gz/packages/ur5/ros2srrc_ur5_gazebo/urdf/ur5_robotiq_2f85_with_cams_gz.urdf.xacro (robot description, xacro)
@@ -1,130 +1,100 @@
-<?xml version="1.0" ?>
-<!--
-# ===================================== COPYRIGHT ===================================== #
-#                                                                                       #
-#  IFRA (Intelligent Flexible Robotics and Assembly) Group, CRANFIELD UNIVERSITY        #
-#  Created on behalf of the IFRA Group at Cranfield University, United Kingdom          #
-#  E-mail: IFRA@cranfield.ac.uk                                                         #
-#                                                                                       #
-#  Licensed under the Apache-2.0 License.                                               #
-#  You may not use this file except in compliance with the License.                     #
-#  You may obtain a copy of the License at: http://www.apache.org/licenses/LICENSE-2.0  #
-#                                                                                       #
-#  Unless required by applicable law or agreed to in writing, software distributed      #
-#  under the License is distributed on an "as-is" basis, without warranties or          #
-#  conditions of any kind, either express or implied. See the License for the specific  #
-#  language governing permissions and limitations under the License.                    #
-#                                                                                       #
-#  IFRA Group - Cranfield University                                                    #
-#  AUTHORS: Mikel Bueno Viso - Mikel.Bueno-Viso@cranfield.ac.uk                         #
-#           Dr. Seemal Asif  - s.asif@cranfield.ac.uk                                   #
-#           Prof. Phil Webb  - p.f.webb@cranfield.ac.uk                                 #
-#                                                                                       #
-#  Date: April, 2023.                                                                   #
-#                                                                                       #
-# ===================================== COPYRIGHT ===================================== #
-# ======= CITE OUR WORK ======= #
-# You can cite our work with the following statement:
-# IFRA-Cranfield (2023) ROS 2 Sim-to-Real Robot Control. URL: https://github.com/IFRA-Cranfield/ros2_SimRealRobotControl.
--->
-<robot name="ur5" xmlns:xacro="http://ros.org/wiki/xacro">
-  <!-- PASS ARGUMENTS: -->
-  <xacro:arg name="bringup" default="false"/>
-  <xacro:property name="bringup" value="$(arg bringup)"/>
-  <xacro:arg name="hmi" default="false"/>
-  <xacro:property name="hmi" value="$(arg hmi)"/>
-  <xacro:arg name="robot_ip" default="0.0.0.0"/>
-  <xacro:property name="robot_ip" value="$(arg robot_ip)"/>
-  <xacro:arg name="EE" default="false"/>
-  <xacro:property name="EE" value="$(arg EE)"/>
-  <xacro:arg name="EE_name" default="none"/>
-  <xacro:property name="EE_name" value="$(arg EE_name)"/>
-  <!-- UR5 Control ARGUMENTS -->
-  <xacro:arg name="script_filename" default="none"/>
-  <xacro:property name="script_filename" value="$(arg script_filename)"/>
-  <xacro:arg name="input_recipe_filename" default="none"/>
-  <xacro:property name="input_recipe_filename" value="$(arg input_recipe_filename)"/>
-  <xacro:arg name="output_recipe_filename" default="none"/>
-  <xacro:property name="output_recipe_filename" value="$(arg output_recipe_filename)"/>
+<?xml version="1.0"?>
+<robot name="ur5" xmlns:xacro="http://www.ros.org/wiki/xacro">
+  <!-- ================= ARGUMENTOS ================= -->
   <xacro:arg name="sim_gz" default="true"/>
-  <xacro:arg name="simulation_controllers" default="$(find ros2srrc_robots)/ur5/config/controller.yaml"/>
-  <!-- Include XACRO-MACRO file of the UR5: -->
-  <xacro:include filename="$(find ros2srrc_robots)/ur5/urdf/ur5_macro.urdf.xacro"/>
-  <xacro:include filename="$(find ros2srrc_ur5_gazebo)/urdf/common_properties.xacro"/>
-  <xacro:include filename="$(find ros2srrc_ur5_gazebo)/urdf/cam_on_hand_params.xacro"/>
-  <xacro:include filename="$(find ros2srrc_ur5_gazebo)/urdf/cam_on_hand_gz.xacro"/>
-  <xacro:include filename="$(find ros2srrc_ur5_gazebo)/urdf/cam_on_base_params.xacro"/>
-  <xacro:include filename="$(find ros2srrc_ur5_gazebo)/urdf/cam_on_base_gz.xacro"/>
-  <xacro:ur5
-    bringup="${bringup}"
-    robot_ip="${robot_ip}"
-    EE="${EE}"
-    EE_name="${EE_name}"
-    script_filename="${script_filename}"
-    input_recipe_filename="${input_recipe_filename}"
-    output_recipe_filename="${output_recipe_filename}"
+  <xacro:arg name="use_fake_hardware" default="false"/>
+  <!-- ================= UR5 OFICIAL (TEXTURAS OK) ================= -->
+  <xacro:include filename="$(find ur5_gripper_description)/urdf/ur.urdf.xacro"/>
+  <xacro:ur_robot
+    name="ur"
+    prefix=""
+    ur_type="ur5"
   />
-  <!-- Include XACRO-MACRO file of the Robotiq 2f-85: -->
-  <xacro:include filename="$(find ros2srrc_endeffectors)/robotiq_2f85/urdf/robotiq_2f85_macro.urdf.xacro"/>
-  <xacro:robotiq_2f85
-    bringup="${bringup}"
-    parent_link="tool0"
-  />
-  <!-- Load ROS 2 Gazebo Plugin -->
-  <xacro:if value="$(arg sim_gz)">
-    <gazebo>
-      <plugin filename="gz_ros2_control-system" name="gz_ros2_control::GazeboSimROS2ControlPlugin">
-        <parameters>$(arg simulation_controllers)</parameters>
-        <xacro:if value="${EE}">
-          <parameters>$(find ros2srrc_endeffectors)/${EE_name}/config/controller.yaml</parameters>
-        </xacro:if>
-      </plugin>
-    </gazebo>
-  </xacro:if>
-  <!-- World: LINK -->
-  <link name="world"/>
-  <!-- Robot Stand: LINK -->
-  <link name='robot_stand'>
-    <inertial>
-      <origin xyz="0 0 0" rpy="0 0 0"/>
-      <mass value="100"/>
-      <inertia ixx="0.01"  ixy="0"  ixz="0" iyy="0.01" iyz="0" izz="0.01" />
-    </inertial>
-    <collision name='collision'>
-      <origin xyz="0 0 0" rpy=" 0 0 0"/>
+  <!-- ================= GRIPPER ================= -->
+  <xacro:include filename="$(find robotiq_description)/urdf/robotiq_85_gripper.urdf.xacro"/>
+  <xacro:include filename="$(find robotiq_description)/urdf/robotiq_85_gripper.ros2_control.xacro"/>
+  <!-- Coupler -->
+  <link name="robotiq_coupler">
+    <visual>
       <geometry>
-        <box size = "0.2 0.2 1.0"/>
+        <mesh filename="package://robotiq_description/meshes/robotiq_85_coupler.stl"/>
+      </geometry>
+    </visual>
+    <collision>
+      <geometry>
+        <cylinder radius="0.04" length="0.015"/>
       </geometry>
     </collision>
-    <visual name='chassis_visual'>
-      <origin xyz="0 0 0" rpy=" 0 0 0"/>
+  </link>
+  <joint name="robotiq_coupler_joint" type="fixed">
+    <origin xyz="0 0 0.004" rpy="0 0 ${-pi/2.0}"/>
+    <parent link="tool0"/>
+    <child link="robotiq_coupler"/>
+  </joint>
+  <xacro:robotiq_85_gripper prefix="" parent="robotiq_coupler">
+    <origin xyz="0 0 0.004" rpy="0 ${-pi/2} ${pi}"/>
+  </xacro:robotiq_85_gripper>
+  <!-- ================= ROS2 CONTROL ================= -->
+  <xacro:include filename="$(find ur5_gripper_description)/urdf/ur.ros2_control.xacro"/>
+  <xacro:ur_ros2_control
+    name="ur"
+    prefix=""
+    sim_gz="true"
+    use_fake_hardware="${use_fake_hardware}"
+    script_filename=""
+    output_recipe_filename=""
+    input_recipe_filename=""
+    tf_prefix=""
+    hash_kinematics=""
+    robot_ip="0.0.0.0"
+  />
+  <xacro:robotiq_85_ros2_control
+    name="robotiq"
+    prefix=""
+    sim_gz="true"
+    use_fake_hardware="${use_fake_hardware}"
+  />
+  <!-- ================= STAND ================= -->
+  <link name="world"/>
+  <link name="robot_stand">
+    <inertial>
+      <origin xyz="0 0 0"/>
+      <mass value="100"/>
+      <inertia ixx="0.01" ixy="0" ixz="0" iyy="0.01" iyz="0" izz="0.01"/>
+    </inertial>
+    <visual>
       <geometry>
-        <box size = "0.2 0.2 1.0"/>
+        <box size="0.2 0.2 1.0"/>
       </geometry>
     </visual>
+    <collision>
+      <geometry>
+        <box size="0.2 0.2 1.0"/>
+      </geometry>
+    </collision>
   </link>
-  <!-- Robot Stand: FIXED JOINT -->
   <joint name="world_joint" type="fixed">
-    <parent link= "world" />
-    <child link = "robot_stand" />
-    <origin xyz="0.0 0.0 0.5" rpy="0.0 0.0 0.0" />
+    <parent link="world"/>
+    <child link="robot_stand"/>
+    <origin xyz="0 0 0.5"/>
   </joint>
-  <!-- Robot Stand: Robot+Stand JOINT -->
   <joint name="stand_joint" type="fixed">
-    <parent link= "robot_stand" />
-    <child link = "base_link" />
-    <origin xyz="0.0 0.0 0.52" rpy="0.0 0.0 0.0" />
+    <parent link="robot_stand"/>
+    <child link="base_link"/>
+    <origin xyz="0 0 0.52"/>
   </joint>
-  <!-- ros2srrc_HMI CAMERA -->
-  <xacro:if value="${hmi}">
-    <xacro:include filename="$(find ros2srrc_hmi)/urdf/hmicamera.urdf.xacro"/>
-    <xacro:HMI_camera
-      x="2.5"
-      y="1.50"
-      z="2.0"
-      roll="0.0"
-      pitch="0.35"
-      yaw="-2.6"
-    />
-  </xacro:if>
+  <!-- ================= CAMARAS (USANDO TUS MACROS) ================= -->
+  <!-- PARAMS -->
+  <xacro:include filename="$(find ros2srrc_ur5_gazebo)/urdf/cam_on_hand_params.xacro"/>
+  <xacro:include filename="$(find ros2srrc_ur5_gazebo)/urdf/cam_on_base_params.xacro"/>
+  <!-- GZ SENSORS -->
+  <xacro:include filename="$(find ros2srrc_ur5_gazebo)/urdf/cam_on_hand_gz.xacro"/>
+  <xacro:include filename="$(find ros2srrc_ur5_gazebo)/urdf/cam_on_base_gz.xacro"/>
+  <!-- INSTANCIACIÓN -->
+  <xacro:cam_on_hand_gz parent_link="wrist_3_link"/>
+  <xacro:cam_on_base_gz parent_link="base_link"/>
+  <!-- ================= GAZEBO CONTROL ================= -->
+  <gazebo>
+    <plugin filename="gz_ros2_control-system" name="gz_ros2_control::GazeboSimROS2ControlPlugin"/>
+  </gazebo>
 </robot>
