Commit message: Fix robot spawn in classic

File: Industrial/ros2_SimRealRobotControl_gz/packages/ur5/ros2srrc_ur5_gazebo/urdf/ur5_robotiq_2f85_with_cams.urdf.xacro (robot description, xacro)
@@ -40,4 +40,7 @@
   <xacro:arg name="EE_name" default="none"/>
   <xacro:property name="EE_name" value="$(arg EE_name)"/>
+  <!-- Argument to choose between classic and harmonic -->
+  <xacro:arg name="sim" default="classic"/>
+  <xacro:property name="sim" value="$(arg sim)"/>
   <!-- UR5 Control ARGUMENTS -->
   <xacro:arg name="script_filename" default="none"/>
@@ -59,4 +62,6 @@
     EE="${EE}"
     EE_name="${EE_name}"
+    sim_gazebo="${sim == 'classic'}"
+    sim_gz="${sim == 'gz'}"
     script_filename="${script_filename}"
     input_recipe_filename="${input_recipe_filename}"
@@ -69,15 +74,25 @@
     parent_link="tool0"
   />
-  <!-- Load ROS 2 Gazebo Plugin -->
+  <!-- Load ROS 2 Control Plugin (Classic vs GZ) -->
   <xacro:unless value="${bringup}">
-    <gazebo>
-      <plugin filename="libgazebo_ros2_control.so" name="gazebo_ros2_control">
-        <robot_sim_type>gazebo_ros2_control/GazeboSystem</robot_sim_type>
-        <!-- UR5 Controller -->
-        <parameters>$(find ros2srrc_robots)/ur5/config/controller.yaml</parameters>
-        <!-- End-Effector Controller (if needed) -->
-        <parameters>$(find ros2srrc_endeffectors)/${EE_name}/config/controller.yaml</parameters>
-      </plugin>
-    </gazebo>
+    <!-- Gazebo Classic -->
+    <xacro:if value="${sim == 'gz'}">
+      <gazebo>
+        <plugin filename="libgz_ros2_control-system.so" name="gz_ros2_control::GazeboSimROS2ControlPlugin">
+          <robot_sim_type>gz_ros2_control/GazeboSimSystem</robot_sim_type>
+          <parameters>$(find ros2srrc_robots)/ur5/config/controller.yaml</parameters>
+          <parameters>$(find ros2srrc_endeffectors)/${EE_name}/config/controller.yaml</parameters>
+        </plugin>
+      </gazebo>
+    </xacro:if>
+    <!-- Gazebo Harmonic / GZ -->
+    <xacro:if value="${sim == 'gz'}">
+      <gazebo>
+        <plugin filename="libgz_ros2_control-system.so" name="gz_ros2_control::GazeboSimROS2ControlPlugin">
+          <parameters>$(find ros2srrc_robots)/ur5/config/controller.yaml</parameters>
+          <parameters>$(find ros2srrc_endeffectors)/${EE_name}/config/controller.yaml</parameters>
+        </plugin>
+      </gazebo>
+    </xacro:if>
   </xacro:unless>
   <!-- World: LINK -->

File: Industrial/ur5_gripper_description/urdf/ur.ros2_control.xacro (robot description, xacro)
@@ -22,7 +22,9 @@
           <plugin>gazebo_ros2_control/GazeboSystem</plugin>
         </xacro:if>
-        <xacro:if value="${sim_gz}">
-          <plugin>gz_ros2_control/GazeboSimSystem</plugin>
-        </xacro:if>
+        <xacro:unless value="${sim_gazebo}">
+          <xacro:if value="${sim_gz}">
+            <plugin>gz_ros2_control/GazeboSimSystem</plugin>
+          </xacro:if>
+        </xacro:unless>
         <xacro:if value="${use_fake_hardware}">
           <plugin>mock_components/GenericSystem</plugin>

Commit message: Resart

File: Industrial/ros2_SimRealRobotControl_gz/packages/ur5/ros2srrc_ur5_gazebo/urdf/ur5_robotiq_2f85_with_cams.urdf.xacro (robot description, xacro)
@@ -40,7 +40,4 @@
   <xacro:arg name="EE_name" default="none"/>
   <xacro:property name="EE_name" value="$(arg EE_name)"/>
-  <!-- Argument to choose between classic and harmonic -->
-  <xacro:arg name="sim" default="classic"/>
-  <xacro:property name="sim" value="$(arg sim)"/>
   <!-- UR5 Control ARGUMENTS -->
   <xacro:arg name="script_filename" default="none"/>
@@ -62,6 +59,4 @@
     EE="${EE}"
     EE_name="${EE_name}"
-    sim_gazebo="${sim == 'classic'}"
-    sim_gz="${sim == 'gz'}"
     script_filename="${script_filename}"
     input_recipe_filename="${input_recipe_filename}"
@@ -74,25 +69,15 @@
     parent_link="tool0"
   />
-  <!-- Load ROS 2 Control Plugin (Classic vs GZ) -->
+  <!-- Load ROS 2 Gazebo Plugin -->
   <xacro:unless value="${bringup}">
-    <!-- Gazebo Classic -->
-    <xacro:if value="${sim == 'gz'}">
-      <gazebo>
-        <plugin filename="libgz_ros2_control-system.so" name="gz_ros2_control::GazeboSimROS2ControlPlugin">
-          <robot_sim_type>gz_ros2_control/GazeboSimSystem</robot_sim_type>
-          <parameters>$(find ros2srrc_robots)/ur5/config/controller.yaml</parameters>
-          <parameters>$(find ros2srrc_endeffectors)/${EE_name}/config/controller.yaml</parameters>
-        </plugin>
-      </gazebo>
-    </xacro:if>
-    <!-- Gazebo Harmonic / GZ -->
-    <xacro:if value="${sim == 'gz'}">
-      <gazebo>
-        <plugin filename="libgz_ros2_control-system.so" name="gz_ros2_control::GazeboSimROS2ControlPlugin">
-          <parameters>$(find ros2srrc_robots)/ur5/config/controller.yaml</parameters>
-          <parameters>$(find ros2srrc_endeffectors)/${EE_name}/config/controller.yaml</parameters>
-        </plugin>
-      </gazebo>
-    </xacro:if>
+    <gazebo>
+      <plugin filename="libgazebo_ros2_control.so" name="gazebo_ros2_control">
+        <robot_sim_type>gazebo_ros2_control/GazeboSystem</robot_sim_type>
+        <!-- UR5 Controller -->
+        <parameters>$(find ros2srrc_robots)/ur5/config/controller.yaml</parameters>
+        <!-- End-Effector Controller (if needed) -->
+        <parameters>$(find ros2srrc_endeffectors)/${EE_name}/config/controller.yaml</parameters>
+      </plugin>
+    </gazebo>
   </xacro:unless>
   <!-- World: LINK -->

File: Industrial/ros2_SimRealRobotControl_gz/ros2srrc_robots/ur5/urdf/ur5_macro.urdf.xacro (robot description, xacro)
@@ -58,5 +58,5 @@
   <xacro:include filename="$(find ros2srrc_robots)/ur5/urdf/ur5_common.xacro"/>
   <!-- XACRO-MACRO of UR5: -->
-  <xacro:macro name="ur5" params="bringup robot_ip EE EE_name script_filename input_recipe_filename output_recipe_filename sim">
+  <xacro:macro name="ur5" params="bringup robot_ip EE EE_name script_filename input_recipe_filename output_recipe_filename">
     <!-- LOAD UR5-Common: -->
     <xacro:ur5_common/>
@@ -68,30 +68,13 @@
     <!-- UR5 GAZEBO - ROS2_CONTROL: -->
     <xacro:include filename="$(find ros2srrc_robots)/ur5/urdf/ur5_ros2control.xacro" />
-    <xacro:if value="${sim == 'classic'}">
-      <xacro:ur5_ros2control
-        bringup="${bringup}"
-        robot_ip="${robot_ip}"
-        EE="${EE}"
-        EE_name="${EE_name}"
-        script_filename="${script_filename}"
-        input_recipe_filename="${input_recipe_filename}"
-        output_recipe_filename="${output_recipe_filename}"
-        sim_gazebo="true"
-        sim_gz="false"
-      />
-    </xacro:if>
-    <xacro:if value="${sim == 'gz'}">
-      <xacro:ur5_ros2control
-        bringup="${bringup}"
-        robot_ip="${robot_ip}"
-        EE="${EE}"
-        EE_name="${EE_name}"
-        script_filename="${script_filename}"
-        input_recipe_filename="${input_recipe_filename}"
-        output_recipe_filename="${output_recipe_filename}"
-        sim_gazebo="false"
-        sim_gz="true"
-      />
-    </xacro:if>
+    <xacro:ur5_ros2control
+      bringup="${bringup}"
+      robot_ip="${robot_ip}"
+      EE="${EE}"
+      EE_name="${EE_name}"
+      script_filename="${script_filename}"
+      input_recipe_filename="${input_recipe_filename}"
+      output_recipe_filename="${output_recipe_filename}"
+    />
     <!-- ***** UR5 ROBOT .urdf SERIAL CHAIN ***** -->
     <!-- Links: -->

File: Industrial/ros2_SimRealRobotControl_gz/ros2srrc_robots/ur5/urdf/ur5_ros2control.xacro (robot description, xacro)
@@ -98,9 +98,5 @@
   <xacro:arg name="tf_prefix" default=""/>
   <xacro:property name="tf_prefix" value="$(arg tf_prefix)"/>
-  <xacro:macro name="ur5_ros2control" params="
-    bringup robot_ip EE EE_name
-    script_filename input_recipe_filename output_recipe_filename
-    sim_gazebo:=false sim_gz:=false
-  ">
+  <xacro:macro name="ur5_ros2control" params="bringup robot_ip EE EE_name script_filename input_recipe_filename output_recipe_filename" >
     <!-- ROS2_CONTROL tag name: -->
     <!-- A. GAZEBO SIMULATION: -->

File: Industrial/ur5_gripper_description/urdf/ur.ros2_control.xacro (robot description, xacro)
@@ -22,9 +22,7 @@
           <plugin>gazebo_ros2_control/GazeboSystem</plugin>
         </xacro:if>
-        <xacro:unless value="${sim_gazebo}">
-          <xacro:if value="${sim_gz}">
-            <plugin>gz_ros2_control/GazeboSimSystem</plugin>
-          </xacro:if>
-        </xacro:unless>
+        <xacro:if value="${sim_gz}">
+          <plugin>gz_ros2_control/GazeboSimSystem</plugin>
+        </xacro:if>
         <xacro:if value="${use_fake_hardware}">
           <plugin>mock_components/GenericSystem</plugin>

Commit message: Fix ros2 control plugin

File: Industrial/ros2_SimRealRobotControl_gz/packages/ur5/ros2srrc_ur5_gazebo/urdf/ur5_robotiq_2f85_with_cams.urdf.xacro (robot description, xacro)
@@ -1,124 +1,130 @@
-<?xml version="1.0" ?>
-<!--
-# ===================================== COPYRIGHT ===================================== #
-#                                                                                       #
-#  IFRA (Intelligent Flexible Robotics and Assembly) Group, CRANFIELD UNIVERSITY        #
-#  Created on behalf of the IFRA Group at Cranfield University, United Kingdom          #
-#  E-mail: IFRA@cranfield.ac.uk                                                         #
-#                                                                                       #
-#  Licensed under the Apache-2.0 License.                                               #
-#  You may not use this file except in compliance with the License.                     #
-#  You may obtain a copy of the License at: http://www.apache.org/licenses/LICENSE-2.0  #
-#                                                                                       #
-#  Unless required by applicable law or agreed to in writing, software distributed      #
-#  under the License is distributed on an "as-is" basis, without warranties or          #
-#  conditions of any kind, either express or implied. See the License for the specific  #
-#  language governing permissions and limitations under the License.                    #
-#                                                                                       #
-#  IFRA Group - Cranfield University                                                    #
-#  AUTHORS: Mikel Bueno Viso - Mikel.Bueno-Viso@cranfield.ac.uk                         #
-#           Dr. Seemal Asif  - s.asif@cranfield.ac.uk                                   #
-#           Prof. Phil Webb  - p.f.webb@cranfield.ac.uk                                 #
-#                                                                                       #
-#  Date: April, 2023.                                                                   #
-#                                                                                       #
-# ===================================== COPYRIGHT ===================================== #
-# ======= CITE OUR WORK ======= #
-# You can cite our work with the following statement:
-# IFRA-Cranfield (2023) ROS 2 Sim-to-Real Robot Control. URL: https://github.com/IFRA-Cranfield/ros2_SimRealRobotControl.
--->
-<robot name="ur5" xmlns:xacro="http://ros.org/wiki/xacro">
-  <!-- PASS ARGUMENTS: -->
-  <xacro:arg name="bringup" default="false"/>
-  <xacro:property name="bringup" value="$(arg bringup)"/>
+<?xml version="1.0"?>
+<robot name="ur5" xmlns:xacro="http://www.ros.org/wiki/xacro">
+  <!-- ========================= -->
+  <!-- ARGUMENTS -->
+  <!-- ========================= -->
+  <xacro:arg name="name" default="ur"/>
+  <xacro:arg name="ur_type" default="ur5"/>
+  <xacro:arg name="prefix" default=""/>
+  <xacro:arg name="use_fake_hardware" default="false"/>
+  <xacro:arg name="fake_sensor_commands" default="false"/>
+  <xacro:arg name="sim_gazebo" default="false"/>
+  <xacro:arg name="sim_gz" default="true"/>
+  <xacro:arg name="simulation_controllers" default=""/>
   <xacro:arg name="hmi" default="false"/>
-  <xacro:property name="hmi" value="$(arg hmi)"/>
-  <xacro:arg name="robot_ip" default="0.0.0.0"/>
-  <xacro:property name="robot_ip" value="$(arg robot_ip)"/>
-  <xacro:arg name="EE" default="false"/>
-  <xacro:property name="EE" value="$(arg EE)"/>
-  <xacro:arg name="EE_name" default="none"/>
-  <xacro:property name="EE_name" value="$(arg EE_name)"/>
-  <!-- UR5 Control ARGUMENTS -->
-  <xacro:arg name="script_filename" default="none"/>
-  <xacro:property name="script_filename" value="$(arg script_filename)"/>
-  <xacro:arg name="input_recipe_filename" default="none"/>
-  <xacro:property name="input_recipe_filename" value="$(arg input_recipe_filename)"/>
-  <xacro:arg name="output_recipe_filename" default="none"/>
-  <xacro:property name="output_recipe_filename" value="$(arg output_recipe_filename)"/>
-  <!-- Include XACRO-MACRO file of the UR5: -->
-  <xacro:include filename="$(find ros2srrc_robots)/ur5/urdf/ur5_macro.urdf.xacro"/>
-  <xacro:include filename="$(find ros2srrc_ur5_gazebo)/urdf/common_properties.xacro"/>
+  <!-- ========================= -->
+  <!-- CORE -->
+  <!-- ========================= -->
+  <xacro:include filename="$(find ur5_gripper_description)/urdf/ur.urdf.xacro" />
+  <xacro:include filename="$(find robotiq_description)/urdf/robotiq_85_gripper.urdf.xacro" />
+  <xacro:include filename="$(find robotiq_description)/urdf/robotiq_85_gripper.ros2_control.xacro" />
+  <xacro:include filename="$(find ur5_gripper_description)/urdf/ur.ros2_control.xacro" />
+  <!-- ========================= -->
+  <!-- UR5 BASE -->
+  <!-- ========================= -->
+  <xacro:ur_robot
+    name="$(arg name)"
+    prefix="$(arg prefix)"
+    parent="world"
+    joint_limits_parameters_file="$(find ur5_gripper_description)/config/ur5/joint_limits.yaml"
+    kinematics_parameters_file="$(find ur5_gripper_description)/config/ur5/default_kinematics.yaml"
+    physical_parameters_file="$(find ur5_gripper_description)/config/ur5/physical_parameters.yaml"
+    visual_parameters_file="$(find ur5_gripper_description)/config/ur5/visual_parameters.yaml"
+    use_fake_hardware="$(arg use_fake_hardware)"
+    fake_sensor_commands="$(arg fake_sensor_commands)"
+    sim_gazebo="$(arg sim_gazebo)"
+    sim_gz="$(arg sim_gz)"
+    initial_positions="${load_yaml('$(find ur5_gripper_description)/config/initial_positions.yaml')}"
+    robot_ip="0.0.0.0"
+  >
+    <origin xyz="0 0 0" rpy="0 0 0"/>
+  </xacro:ur_robot>
+  <!-- ========================= -->
+  <!-- GRIPPER -->
+  <!-- ========================= -->
+  <!-- Coupler -->
+  <link name="robotiq_coupler">
+    <visual>
+      <geometry>
+        <mesh filename="package://robotiq_description/meshes/robotiq_85_coupler.stl"/>
+      </geometry>
+    </visual>
+    <collision>
+      <geometry>
+        <cylinder radius="0.04" length="0.015"/>
+      </geometry>
+    </collision>
+  </link>
+  <joint name="robotiq_coupler_joint" type="fixed">
+    <origin xyz="0 0 0.004" rpy="0 0 ${-pi/2.0}" />
+    <parent link="tool0"/>
+    <child link="robotiq_coupler"/>
+  </joint>
+  <xacro:robotiq_85_gripper prefix="" parent="robotiq_coupler">
+    <origin xyz="0 0 0.004" rpy="0 ${-pi/2} ${pi}"/>
+  </xacro:robotiq_85_gripper>
+  <!-- ros2_control -->
+  <xacro:robotiq_85_ros2_control
+    name="robotiq"
+    prefix=""
+    sim_gz="true"
+    use_fake_hardware="false"/>
+  <xacro:ur_ros2_control
+    name="ur"
+    prefix=""
+    sim_gz="true"
+    use_fake_hardware="false"
+    script_filename=""
+    output_recipe_filename=""
+    input_recipe_filename=""
+    tf_prefix=""
+    hash_kinematics=""
+    robot_ip="0.0.0.0"
+  />
+  <!-- ========================= -->
+  <!-- STAND -->
+  <!-- ========================= -->
+  <link name="robot_stand">
+    <inertial>
+      <origin xyz="0 0 0"/>
+      <mass value="100"/>
+      <inertia ixx="0.01" iyy="0.01" izz="0.01"/>
+    </inertial>
+    <visual>
+      <geometry>
+        <box size="0.2 0.2 1.0"/>
+      </geometry>
+    </visual>
+    <collision>
+      <geometry>
+        <box size="0.2 0.2 1.0"/>
+      </geometry>
+    </collision>
+  </link>
+  <joint name="world_to_stand" type="fixed">
+    <parent link="world"/>
+    <child link="robot_stand"/>
+    <origin xyz="0 0 0.5"/>
+  </joint>
+  <joint name="stand_to_robot" type="fixed">
+    <parent link="robot_stand"/>
+    <child link="base_link"/>
+    <origin xyz="0 0 0.52"/>
+  </joint>
+  <!-- ========================= -->
+  <!-- CAMERAS -->
+  <!-- ========================= -->
   <xacro:include filename="$(find ros2srrc_ur5_gazebo)/urdf/cam_on_hand_params.xacro"/>
   <xacro:include filename="$(find ros2srrc_ur5_gazebo)/urdf/cam_on_hand.xacro"/>
   <xacro:include filename="$(find ros2srrc_ur5_gazebo)/urdf/cam_on_base_params.xacro"/>
   <xacro:include filename="$(find ros2srrc_ur5_gazebo)/urdf/cam_on_base.xacro"/>
-  <xacro:ur5
-    bringup="${bringup}"
-    robot_ip="${robot_ip}"
-    EE="${EE}"
-    EE_name="${EE_name}"
-    script_filename="${script_filename}"
-    input_recipe_filename="${input_recipe_filename}"
-    output_recipe_filename="${output_recipe_filename}"
-  />
-  <!-- Include XACRO-MACRO file of the Robotiq 2f-85: -->
-  <xacro:include filename="$(find ros2srrc_endeffectors)/robotiq_2f85/urdf/robotiq_2f85_macro.urdf.xacro"/>
-  <xacro:robotiq_2f85
-    bringup="${bringup}"
-    parent_link="tool0"
-  />
-  <!-- Load ROS 2 Gazebo Plugin -->
-  <xacro:unless value="${bringup}">
-    <gazebo>
-      <plugin filename="libgazebo_ros2_control.so" name="gazebo_ros2_control">
-        <robot_sim_type>gazebo_ros2_control/GazeboSystem</robot_sim_type>
-        <!-- UR5 Controller -->
-        <parameters>$(find ros2srrc_robots)/ur5/config/controller.yaml</parameters>
-        <!-- End-Effector Controller (if needed) -->
-        <parameters>$(find ros2srrc_endeffectors)/${EE_name}/config/controller.yaml</parameters>
-      </plugin>
-    </gazebo>
-  </xacro:unless>
-  <!-- World: LINK -->
-  <link name="world"/>
-  <!-- Robot Stand: LINK -->
-  <link name='robot_stand'>
-    <inertial>
-      <origin xyz="0 0 0" rpy="0 0 0"/>
-      <mass value="100"/>
-      <inertia ixx="0.01"  ixy="0"  ixz="0" iyy="0.01" iyz="0" izz="0.01" />
-    </inertial>
-    <collision name='collision'>
-      <origin xyz="0 0 0" rpy=" 0 0 0"/>
-      <geometry>
-        <box size = "0.2 0.2 1.0"/>
-      </geometry>
-    </collision>
-    <visual name='chassis_visual'>
-      <origin xyz="0 0 0" rpy=" 0 0 0"/>
-      <geometry>
-        <box size = "0.2 0.2 1.0"/>
-      </geometry>
-    </visual>
-  </link>
-  <!-- Robot Stand: FIXED JOINT -->
-  <joint name="world_joint" type="fixed">
-    <parent link= "world" />
-    <child link = "robot_stand" />
-    <origin xyz="0.0 0.0 0.5" rpy="0.0 0.0 0.0" />
-  </joint>
-  <!-- Robot Stand: Robot+Stand JOINT -->
-  <joint name="stand_joint" type="fixed">
-    <parent link= "robot_stand" />
-    <child link = "base_link" />
-    <origin xyz="0.0 0.0 0.52" rpy="0.0 0.0 0.0" />
-  </joint>
-  <!-- ros2srrc_HMI CAMERA -->
-  <xacro:if value="${hmi}">
+  <!-- ========================= -->
+  <!-- HMI CAMERA -->
+  <!-- ========================= -->
+  <xacro:if value="$(arg hmi)">
     <xacro:include filename="$(find ros2srrc_hmi)/urdf/hmicamera.urdf.xacro"/>
     <xacro:HMI_camera
       x="2.5"
-      y="1.50"
+      y="1.5"
       z="2.0"
       roll="0.0"

File: Industrial/ur5_gripper_description/urdf/ur.urdf.xacro (robot description, xacro)
@@ -81,5 +81,5 @@
      <origin xyz="0 0 0" rpy="0 0 0" />
    </xacro:ur_robot>
-   <xacro:if value="$(arg sim_gazebo)">
+   <xacro:if value="$(arg sim_gazebo) and not $(arg sim_gz)">
     <!-- Gazebo plugins -->
     <!-- update the plugin  -->
