Commit message: Fix xacro

File: Industrial/ros2_SimRealRobotControl_gz/packages/ur5/ros2srrc_ur5_gazebo/urdf/ur5_robotiq_2f85_with_cams.urdf.xacro (robot description, xacro)
@@ -1,130 +1,115 @@
-<?xml version="1.0"?>
-<robot name="ur5" xmlns:xacro="http://www.ros.org/wiki/xacro">
-  <!-- ========================= -->
-  <!-- ARGUMENTS -->
-  <!-- ========================= -->
-  <xacro:arg name="name" default="ur"/>
-  <xacro:arg name="ur_type" default="ur5"/>
-  <xacro:arg name="prefix" default=""/>
-  <xacro:arg name="use_fake_hardware" default="false"/>
-  <xacro:arg name="fake_sensor_commands" default="false"/>
-  <xacro:arg name="sim_gazebo" default="false"/>
+<?xml version="1.0" ?>
+<!--
+# ===================================== COPYRIGHT ===================================== #
+#                                                                                       #
+#  IFRA (Intelligent Flexible Robotics and Assembly) Group, CRANFIELD UNIVERSITY        #
+#  Created on behalf of the IFRA Group at Cranfield University, United Kingdom          #
+#  E-mail: IFRA@cranfield.ac.uk                                                         #
+#                                                                                       #
+#  Licensed under the Apache-2.0 License.                                               #
+#  You may not use this file except in compliance with the License.                     #
+#  You may obtain a copy of the License at: http://www.apache.org/licenses/LICENSE-2.0  #
+#                                                                                       #
+#  Unless required by applicable law or agreed to in writing, software distributed      #
+#  under the License is distributed on an "as-is" basis, without warranties or          #
+#  conditions of any kind, either express or implied. See the License for the specific  #
+#  language governing permissions and limitations under the License.                    #
+#                                                                                       #
+#  IFRA Group - Cranfield University                                                    #
+#  AUTHORS: Mikel Bueno Viso - Mikel.Bueno-Viso@cranfield.ac.uk                         #
+#           Dr. Seemal Asif  - s.asif@cranfield.ac.uk                                   #
+#           Prof. Phil Webb  - p.f.webb@cranfield.ac.uk                                 #
+#                                                                                       #
+#  Date: April, 2023.                                                                   #
+#                                                                                       #
+# ===================================== COPYRIGHT ===================================== #
+# ======= CITE OUR WORK ======= #
+# You can cite our work with the following statement:
+# IFRA-Cranfield (2023) ROS 2 Sim-to-Real Robot Control. URL: https://github.com/IFRA-Cranfield/ros2_SimRealRobotControl.
+-->
+<robot name="ur5" xmlns:xacro="http://ros.org/wiki/xacro">
+  <!-- PASS ARGUMENTS: -->
+  <xacro:arg name="bringup" default="false"/>
+  <xacro:property name="bringup" value="$(arg bringup)"/>
+  <xacro:arg name="hmi" default="false"/>
+  <xacro:property name="hmi" value="$(arg hmi)"/>
+  <xacro:arg name="robot_ip" default="0.0.0.0"/>
+  <xacro:property name="robot_ip" value="$(arg robot_ip)"/>
+  <xacro:arg name="EE" default="false"/>
+  <xacro:property name="EE" value="$(arg EE)"/>
+  <xacro:arg name="EE_name" default="none"/>
+  <xacro:property name="EE_name" value="$(arg EE_name)"/>
   <xacro:arg name="sim_gz" default="true"/>
+  <xacro:property name="sim_gz" value="$(arg sim_gz)"/>
   <xacro:arg name="simulation_controllers" default=""/>
-  <xacro:arg name="hmi" default="false"/>
-  <!-- ========================= -->
-  <!-- CORE -->
-  <!-- ========================= -->
-  <xacro:include filename="$(find ur5_gripper_description)/urdf/ur.urdf.xacro" />
-  <xacro:include filename="$(find robotiq_description)/urdf/robotiq_85_gripper.urdf.xacro" />
-  <xacro:include filename="$(find robotiq_description)/urdf/robotiq_85_gripper.ros2_control.xacro" />
-  <xacro:include filename="$(find ur5_gripper_description)/urdf/ur.ros2_control.xacro" />
-  <!-- ========================= -->
-  <!-- UR5 BASE -->
-  <!-- ========================= -->
-  <xacro:ur_robot
-    name="$(arg name)"
-    prefix="$(arg prefix)"
-    parent="world"
-    joint_limits_parameters_file="$(find ur5_gripper_description)/config/ur5/joint_limits.yaml"
-    kinematics_parameters_file="$(find ur5_gripper_description)/config/ur5/default_kinematics.yaml"
-    physical_parameters_file="$(find ur5_gripper_description)/config/ur5/physical_parameters.yaml"
-    visual_parameters_file="$(find ur5_gripper_description)/config/ur5/visual_parameters.yaml"
-    use_fake_hardware="$(arg use_fake_hardware)"
-    fake_sensor_commands="$(arg fake_sensor_commands)"
-    sim_gazebo="$(arg sim_gazebo)"
-    sim_gz="$(arg sim_gz)"
-    initial_positions="${load_yaml('$(find ur5_gripper_description)/config/initial_positions.yaml')}"
-    robot_ip="0.0.0.0"
-  >
-    <origin xyz="0 0 0" rpy="0 0 0"/>
-  </xacro:ur_robot>
-  <!-- ========================= -->
-  <!-- GRIPPER -->
-  <!-- ========================= -->
-  <!-- Coupler -->
-  <link name="robotiq_coupler">
-    <visual>
-      <geometry>
-        <mesh filename="package://robotiq_description/meshes/robotiq_85_coupler.stl"/>
-      </geometry>
-    </visual>
-    <collision>
-      <geometry>
-        <cylinder radius="0.04" length="0.015"/>
-      </geometry>
-    </collision>
-  </link>
-  <joint name="robotiq_coupler_joint" type="fixed">
-    <origin xyz="0 0 0.004" rpy="0 0 ${-pi/2.0}" />
-    <parent link="tool0"/>
-    <child link="robotiq_coupler"/>
-  </joint>
-  <xacro:robotiq_85_gripper prefix="" parent="robotiq_coupler">
-    <origin xyz="0 0 0.004" rpy="0 ${-pi/2} ${pi}"/>
-  </xacro:robotiq_85_gripper>
-  <!-- ros2_control -->
-  <xacro:robotiq_85_ros2_control
-    name="robotiq"
-    prefix=""
-    sim_gz="true"
-    use_fake_hardware="false"/>
-  <xacro:ur_ros2_control
-    name="ur"
-    prefix=""
-    sim_gz="true"
-    use_fake_hardware="false"
-    script_filename=""
-    output_recipe_filename=""
-    input_recipe_filename=""
-    tf_prefix=""
-    hash_kinematics=""
-    robot_ip="0.0.0.0"
-  />
-  <!-- ========================= -->
-  <!-- STAND -->
-  <!-- ========================= -->
-  <link name="robot_stand">
-    <inertial>
-      <origin xyz="0 0 0"/>
-      <mass value="100"/>
-      <inertia ixx="0.01" iyy="0.01" izz="0.01"/>
-    </inertial>
-    <visual>
-      <geometry>
-        <box size="0.2 0.2 1.0"/>
-      </geometry>
-    </visual>
-    <collision>
-      <geometry>
-        <box size="0.2 0.2 1.0"/>
-      </geometry>
-    </collision>
-  </link>
-  <joint name="world_to_stand" type="fixed">
-    <parent link="world"/>
-    <child link="robot_stand"/>
-    <origin xyz="0 0 0.5"/>
-  </joint>
-  <joint name="stand_to_robot" type="fixed">
-    <parent link="robot_stand"/>
-    <child link="base_link"/>
-    <origin xyz="0 0 0.52"/>
-  </joint>
-  <!-- ========================= -->
-  <!-- CAMERAS -->
-  <!-- ========================= -->
+  <!-- UR5 Control ARGUMENTS -->
+  <xacro:arg name="script_filename" default="none"/>
+  <xacro:property name="script_filename" value="$(arg script_filename)"/>
+  <xacro:arg name="input_recipe_filename" default="none"/>
+  <xacro:property name="input_recipe_filename" value="$(arg input_recipe_filename)"/>
+  <xacro:arg name="output_recipe_filename" default="none"/>
+  <xacro:property name="output_recipe_filename" value="$(arg output_recipe_filename)"/>
+  <!-- Include XACRO-MACRO file of the UR5: -->
+  <xacro:include filename="$(find ros2srrc_robots)/ur5/urdf/ur5_macro.urdf.xacro"/>
+  <xacro:include filename="$(find ros2srrc_ur5_gazebo)/urdf/common_properties.xacro"/>
   <xacro:include filename="$(find ros2srrc_ur5_gazebo)/urdf/cam_on_hand_params.xacro"/>
   <xacro:include filename="$(find ros2srrc_ur5_gazebo)/urdf/cam_on_hand.xacro"/>
   <xacro:include filename="$(find ros2srrc_ur5_gazebo)/urdf/cam_on_base_params.xacro"/>
   <xacro:include filename="$(find ros2srrc_ur5_gazebo)/urdf/cam_on_base.xacro"/>
-  <!-- ========================= -->
-  <!-- HMI CAMERA -->
-  <!-- ========================= -->
-  <xacro:if value="$(arg hmi)">
+  <xacro:ur5
+    bringup="${bringup}"
+    robot_ip="${robot_ip}"
+    EE="${EE}"
+    EE_name="${EE_name}"
+    script_filename="${script_filename}"
+    input_recipe_filename="${input_recipe_filename}"
+    output_recipe_filename="${output_recipe_filename}"
+  />
+  <!-- Include XACRO-MACRO file of the Robotiq 2f-85: -->
+  <xacro:include filename="$(find ros2srrc_endeffectors)/robotiq_2f85/urdf/robotiq_2f85_macro.urdf.xacro"/>
+  <xacro:robotiq_2f85
+    bringup="${bringup}"
+    parent_link="tool0"
+  />
+  <!-- World: LINK -->
+  <link name="world"/>
+  <!-- Robot Stand: LINK -->
+  <link name='robot_stand'>
+    <inertial>
+      <origin xyz="0 0 0" rpy="0 0 0"/>
+      <mass value="100"/>
+      <inertia ixx="0.01"  ixy="0"  ixz="0" iyy="0.01" iyz="0" izz="0.01" />
+    </inertial>
+    <collision name='collision'>
+      <origin xyz="0 0 0" rpy=" 0 0 0"/>
+      <geometry>
+        <box size = "0.2 0.2 1.0"/>
+      </geometry>
+    </collision>
+    <visual name='chassis_visual'>
+      <origin xyz="0 0 0" rpy=" 0 0 0"/>
+      <geometry>
+        <box size = "0.2 0.2 1.0"/>
+      </geometry>
+    </visual>
+  </link>
+  <!-- Robot Stand: FIXED JOINT -->
+  <joint name="world_joint" type="fixed">
+    <parent link= "world" />
+    <child link = "robot_stand" />
+    <origin xyz="0.0 0.0 0.5" rpy="0.0 0.0 0.0" />
+  </joint>
+  <!-- Robot Stand: Robot+Stand JOINT -->
+  <joint name="stand_joint" type="fixed">
+    <parent link= "robot_stand" />
+    <child link = "base_link" />
+    <origin xyz="0.0 0.0 0.52" rpy="0.0 0.0 0.0" />
+  </joint>
+  <!-- ros2srrc_HMI CAMERA -->
+  <xacro:if value="${hmi}">
     <xacro:include filename="$(find ros2srrc_hmi)/urdf/hmicamera.urdf.xacro"/>
     <xacro:HMI_camera
       x="2.5"
-      y="1.5"
+      y="1.50"
       z="2.0"
       roll="0.0"
@@ -133,3 +118,11 @@
     />
   </xacro:if>
+  <xacro:if value="${sim_gz and not bringup}">
+    <gazebo>
+      <plugin filename="gz_ros2_control-system"
+              name="gz_ros2_control::GazeboSimROS2ControlPlugin">
+        <parameters>$(arg simulation_controllers)</parameters>
+      </plugin>
+    </gazebo>
+  </xacro:if>
 </robot>

File: Industrial/ur5_gripper_description/urdf/ur.urdf.xacro (robot description, xacro)
@@ -81,5 +81,5 @@
      <origin xyz="0 0 0" rpy="0 0 0" />
    </xacro:ur_robot>
-   <xacro:if value="$(arg sim_gazebo) and not $(arg sim_gz)">
+   <xacro:if value="$(arg sim_gazebo)">
     <!-- Gazebo plugins -->
     <!-- update the plugin  -->

Commit message: Fix srdf in urdf

File: Industrial/ros2_SimRealRobotControl_gz/packages/ur5/ros2srrc_ur5_gazebo/urdf/ur5_robotiq_2f85_with_cams.urdf.xacro (robot description, xacro)
@@ -67,9 +67,10 @@
   />
   <!-- Include XACRO-MACRO file of the Robotiq 2f-85: -->
-  <xacro:include filename="$(find ros2srrc_endeffectors)/robotiq_2f85/urdf/robotiq_2f85_macro.urdf.xacro"/>
-  <xacro:robotiq_2f85
-    bringup="${bringup}"
-    parent_link="tool0"
-  />
+  <xacro:include filename="$(find robotiq_description)/urdf/robotiq_85_gripper.urdf.xacro"/>
+  <xacro:robotiq_85_gripper
+    prefix=""
+    parent="tool0">
+    <origin xyz="0 0 0.004" rpy="0 ${-pi/2} ${pi}"/>
+  </xacro:robotiq_85_gripper>
   <!-- World: LINK -->
   <link name="world"/>

Commit message: Add cams on gz harmonic

File: Industrial/ros2_SimRealRobotControl_gz/packages/ur5/ros2srrc_ur5_gazebo/urdf/ur5_robotiq_2f85_with_cams.urdf.xacro (robot description, xacro)
@@ -54,7 +54,7 @@
   <xacro:include filename="$(find ros2srrc_ur5_gazebo)/urdf/common_properties.xacro"/>
   <xacro:include filename="$(find ros2srrc_ur5_gazebo)/urdf/cam_on_hand_params.xacro"/>
-  <xacro:include filename="$(find ros2srrc_ur5_gazebo)/urdf/cam_on_hand.xacro"/>
+  <xacro:include filename="$(find ros2srrc_ur5_gazebo)/urdf/cam_on_hand_gz.xacro"/>
   <xacro:include filename="$(find ros2srrc_ur5_gazebo)/urdf/cam_on_base_params.xacro"/>
-  <xacro:include filename="$(find ros2srrc_ur5_gazebo)/urdf/cam_on_base.xacro"/>
+  <xacro:include filename="$(find ros2srrc_ur5_gazebo)/urdf/cam_on_base_gz.xacro"/>
   <xacro:ur5
     bringup="${bringup}"
@@ -67,10 +67,9 @@
   />
   <!-- Include XACRO-MACRO file of the Robotiq 2f-85: -->
-  <xacro:include filename="$(find robotiq_description)/urdf/robotiq_85_gripper.urdf.xacro"/>
-  <xacro:robotiq_85_gripper
-    prefix=""
-    parent="tool0">
-    <origin xyz="0 0 0.004" rpy="0 ${-pi/2} ${pi}"/>
-  </xacro:robotiq_85_gripper>
+  <xacro:include filename="$(find ros2srrc_endeffectors)/robotiq_2f85/urdf/robotiq_2f85_macro.urdf.xacro"/>
+  <xacro:robotiq_2f85
+    bringup="${bringup}"
+    parent_link="tool0"
+  />
   <!-- World: LINK -->
   <link name="world"/>

Commit message: Fix collision

File: Industrial/ros2_SimRealRobotControl_gz/packages/ur5/ros2srrc_ur5_gazebo/urdf/ur5_robotiq_2f85_with_cams.urdf.xacro (robot description, xacro)
@@ -67,9 +67,10 @@
   />
   <!-- Include XACRO-MACRO file of the Robotiq 2f-85: -->
-  <xacro:include filename="$(find ros2srrc_endeffectors)/robotiq_2f85/urdf/robotiq_2f85_macro.urdf.xacro"/>
-  <xacro:robotiq_2f85
-    bringup="${bringup}"
-    parent_link="tool0"
-  />
+  <xacro:include filename="$(find tu_paquete)/urdf/robotiq_85_gripper.urdf.xacro"/>
+  <xacro:robotiq_85_gripper
+    prefix=""
+    parent="tool0">
+    <origin xyz="0 0 0" rpy="0 0 0"/>
+  </xacro:robotiq_85_gripper>
   <!-- World: LINK -->
   <link name="world"/>

File: Industrial/ros2_SimRealRobotControl_gz/ros2srrc_robots/ur5/urdf/ur5_macro.urdf.xacro (robot description, xacro)
@@ -93,5 +93,5 @@
         <origin xyz="0 0 0" rpy="0 0 ${pi}"/>
         <geometry>
-          <mesh filename="file://$(find ros2srrc_robots)/ur5/meshes/collision/base.stl"/>
+          <box size="0.3 0.3 0.2"/>
         </geometry>
       </collision>
@@ -113,5 +113,5 @@
         <origin xyz="0 0 0" rpy="0 0 ${pi}"/>
         <geometry>
-          <mesh filename="file://$(find ros2srrc_robots)/ur5/meshes/collision/shoulder.stl"/>
+          <box size="0.25 0.25 0.25"/>
         </geometry>
       </collision>
@@ -131,7 +131,7 @@
       </visual>
       <collision>
-        <origin xyz="0 0 ${shoulder_offset}" rpy="${pi/2} 0 ${-pi/2}"/>
-        <geometry>
-          <mesh filename="file://$(find ros2srrc_robots)/ur5/meshes/collision/upperarm.stl"/>
+        <origin xyz="0 0 0" rpy="0 0 0"/>
+        <geometry>
+          <cylinder radius="0.06" length="0.4"/>
         </geometry>
       </collision>
@@ -151,7 +151,7 @@
       </visual>
       <collision>
-        <origin xyz="0 0 ${elbow_offset}" rpy="${pi/2} 0 ${-pi/2}"/>
-        <geometry>
-          <mesh filename="file://$(find ros2srrc_robots)/ur5/meshes/collision/forearm.stl"/>
+        <origin xyz="0 0 0" rpy="0 0 0"/>
+        <geometry>
+          <cylinder radius="0.05" length="0.4"/>
         </geometry>
       </collision>
@@ -171,7 +171,7 @@
       </visual>
       <collision>
-        <origin xyz="0 0 ${wrist_1_visual_offset}" rpy="${pi/2} 0 0"/>
-        <geometry>
-          <mesh filename="file://$(find ros2srrc_robots)/ur5/meshes/collision/wrist1.stl"/>
+        <origin xyz="0 0 0" rpy="0 0 0"/>
+        <geometry>
+          <cylinder radius="0.05" length="0.1"/>
         </geometry>
       </collision>
@@ -191,7 +191,7 @@
       </visual>
       <collision>
-        <origin xyz="0 0 ${wrist_2_visual_offset}" rpy="0 0 0"/>
-        <geometry>
-          <mesh filename="file://$(find ros2srrc_robots)/ur5/meshes/collision/wrist2.stl"/>
+        <origin xyz="0 0 0" rpy="0 0 0"/>
+        <geometry>
+          <cylinder radius="0.04" length="0.1"/>
         </geometry>
       </collision>
@@ -211,7 +211,7 @@
       </visual>
       <collision>
-        <origin xyz="0 0 ${wrist_3_visual_offset}" rpy="${pi/2} 0 0"/>
-        <geometry>
-          <mesh filename="file://$(find ros2srrc_robots)/ur5/meshes/collision/wrist3.stl"/>
+        <origin xyz="0 0 0" rpy="0 0 0"/>
+        <geometry>
+          <cylinder radius="0.04" length="0.1"/>
         </geometry>
       </collision>

Commit message: Restart collision

File: Industrial/ros2_SimRealRobotControl_gz/packages/ur5/ros2srrc_ur5_gazebo/urdf/ur5_robotiq_2f85_with_cams.urdf.xacro (robot description, xacro)
@@ -67,10 +67,9 @@
   />
   <!-- Include XACRO-MACRO file of the Robotiq 2f-85: -->
-  <xacro:include filename="$(find tu_paquete)/urdf/robotiq_85_gripper.urdf.xacro"/>
-  <xacro:robotiq_85_gripper
-    prefix=""
-    parent="tool0">
-    <origin xyz="0 0 0" rpy="0 0 0"/>
-  </xacro:robotiq_85_gripper>
+  <xacro:include filename="$(find ros2srrc_endeffectors)/robotiq_2f85/urdf/robotiq_2f85_macro.urdf.xacro"/>
+  <xacro:robotiq_2f85
+    bringup="${bringup}"
+    parent_link="tool0"
+  />
   <!-- World: LINK -->
   <link name="world"/>

File: Industrial/ros2_SimRealRobotControl_gz/ros2srrc_robots/ur5/urdf/ur5_macro.urdf.xacro (robot description, xacro)
@@ -93,5 +93,5 @@
         <origin xyz="0 0 0" rpy="0 0 ${pi}"/>
         <geometry>
-          <box size="0.3 0.3 0.2"/>
+          <mesh filename="file://$(find ros2srrc_robots)/ur5/meshes/collision/base.stl"/>
         </geometry>
       </collision>
@@ -113,5 +113,5 @@
         <origin xyz="0 0 0" rpy="0 0 ${pi}"/>
         <geometry>
-          <box size="0.25 0.25 0.25"/>
+          <mesh filename="file://$(find ros2srrc_robots)/ur5/meshes/collision/shoulder.stl"/>
         </geometry>
       </collision>
@@ -131,7 +131,7 @@
       </visual>
       <collision>
-        <origin xyz="0 0 0" rpy="0 0 0"/>
-        <geometry>
-          <cylinder radius="0.06" length="0.4"/>
+        <origin xyz="0 0 ${shoulder_offset}" rpy="${pi/2} 0 ${-pi/2}"/>
+        <geometry>
+          <mesh filename="file://$(find ros2srrc_robots)/ur5/meshes/collision/upperarm.stl"/>
         </geometry>
       </collision>
@@ -151,7 +151,7 @@
       </visual>
       <collision>
-        <origin xyz="0 0 0" rpy="0 0 0"/>
-        <geometry>
-          <cylinder radius="0.05" length="0.4"/>
+        <origin xyz="0 0 ${elbow_offset}" rpy="${pi/2} 0 ${-pi/2}"/>
+        <geometry>
+          <mesh filename="file://$(find ros2srrc_robots)/ur5/meshes/collision/forearm.stl"/>
         </geometry>
       </collision>
@@ -171,7 +171,7 @@
       </visual>
       <collision>
-        <origin xyz="0 0 0" rpy="0 0 0"/>
-        <geometry>
-          <cylinder radius="0.05" length="0.1"/>
+        <origin xyz="0 0 ${wrist_1_visual_offset}" rpy="${pi/2} 0 0"/>
+        <geometry>
+          <mesh filename="file://$(find ros2srrc_robots)/ur5/meshes/collision/wrist1.stl"/>
         </geometry>
       </collision>
@@ -191,7 +191,7 @@
       </visual>
       <collision>
-        <origin xyz="0 0 0" rpy="0 0 0"/>
-        <geometry>
-          <cylinder radius="0.04" length="0.1"/>
+        <origin xyz="0 0 ${wrist_2_visual_offset}" rpy="0 0 0"/>
+        <geometry>
+          <mesh filename="file://$(find ros2srrc_robots)/ur5/meshes/collision/wrist2.stl"/>
         </geometry>
       </collision>
@@ -211,7 +211,7 @@
       </visual>
       <collision>
-        <origin xyz="0 0 0" rpy="0 0 0"/>
-        <geometry>
-          <cylinder radius="0.04" length="0.1"/>
+        <origin xyz="0 0 ${wrist_3_visual_offset}" rpy="${pi/2} 0 0"/>
+        <geometry>
+          <mesh filename="file://$(find ros2srrc_robots)/ur5/meshes/collision/wrist3.stl"/>
         </geometry>
       </collision>
