Commit message: Fix cam_on_base_params.xacro

File: Industrial/ros2_SimRealRobotControl_gz/packages/ur5/ros2srrc_ur5_gazebo/urdf/cam_on_base_params.xacro (robot description, xacro)
@@ -1,4 +1,5 @@
 <?xml version="1.0"?>
 <robot xmlns:xacro="http://ros.org/wiki/xacro">
+    <xacro:property name="pi" value="3.14159265359"/>
     <xacro:property name="cam_base_px" value="1.0" />
     <xacro:property name="cam_base_py" value="0.0" />

Commit message: Fix cam_on_base_params.xacro

File: Industrial/ros2_SimRealRobotControl_gz/packages/ur5/ros2srrc_ur5_gazebo/urdf/cam_on_base_params.xacro (robot description, xacro)
@@ -1,5 +1,4 @@
 <?xml version="1.0"?>
 <robot xmlns:xacro="http://ros.org/wiki/xacro">
-    <xacro:property name="pi" value="3.14159265359"/>
     <xacro:property name="cam_base_px" value="1.0" />
     <xacro:property name="cam_base_py" value="0.0" />

File: Industrial/ros2_SimRealRobotControl_gz/packages/ur5/ros2srrc_ur5_gazebo/urdf/cam_on_hand_gz.xacro (robot description, xacro)
@@ -1,5 +1,5 @@
 <?xml version="1.0"?>
 <robot xmlns:xacro="http://ros.org/wiki/xacro">
-  <link name="base_camera_link">
+  <link name="hand_camera_link">
     <inertial>
       <origin xyz="-0.00936 -0.00003 -0.00273" rpy="0 0 0"/>
@@ -23,22 +23,22 @@
     <material>Gazebo/Grey</material>
   </gazebo>
-  <joint name="base_camera_joint" type="fixed">
-    <parent link="base_link"/>
-    <child link="base_camera_link"/>
-    <origin xyz="${cam_base_px} ${cam_base_py} ${cam_base_pz}"
-            rpy="${cam_base_or} ${cam_base_op} ${cam_base_oy}"/>
+  <joint name="hand_camera_joint" type="fixed">
+    <parent link="tool0"/>
+    <child link="hand_camera_link"/>
+    <origin xyz="${cam_hand_px} ${cam_hand_py} ${cam_hand_pz}"
+            rpy="${cam_hand_or} ${cam_hand_op} ${cam_hand_oy}"/>
   </joint>
-  <link name="base_camera_optical_link"/>
-  <joint name="base_camera_optical_joint" type="fixed">
-    <parent link="base_camera_link"/>
-    <child link="base_camera_optical_link"/>
+  <link name="hand_camera_optical_link"/>
+  <joint name="hand_camera_optical_joint" type="fixed">
+    <parent link="hand_camera_link"/>
+    <child link="hand_camera_optical_link"/>
     <origin xyz="0 0 0" rpy="-1.57 0 -1.57"/>
   </joint>
-  <gazebo reference="base_camera_link">
-    <sensor name="base_camera" type="rgbd_camera">
+  <gazebo reference="hand_camera_link">
+    <sensor name="hand_camera" type="rgbd_camera">
       <always_on>true</always_on>
       <visualize>true</visualize>
       <update_rate>30</update_rate>
-      <topic>/base_camera</topic>
+      <topic>/hand_camera</topic>
       <camera>
         <horizontal_fov>1.047</horizontal_fov>

Commit message: Fix camera orientation

File: Industrial/ros2_SimRealRobotControl_gz/packages/ur5/ros2srrc_ur5_gazebo/urdf/cam_on_base_params.xacro (robot description, xacro)
@@ -5,6 +5,6 @@
     <xacro:property name="cam_base_pz" value="1.4" />
     <xacro:property name="cam_base_or" value="0.0" />
-    <xacro:property name="cam_base_op" value="${pi/4}" />
-    <xacro:property name="cam_base_oy" value="${pi}" />
+    <xacro:property name="cam_base_op" value="$0" />
+    <xacro:property name="cam_base_oy" value="$0" />
     <xacro:property name="parent_base" value="world" />
 </robot>

File: Industrial/ros2_SimRealRobotControl_gz/packages/ur5/ros2srrc_ur5_gazebo/urdf/cam_on_hand_gz.xacro (robot description, xacro)
@@ -11,10 +11,10 @@
     <visual>
       <geometry>
-        <mesh filename="file://$(find ros2srrc_ur5_gazebo)/meshes/kinetic.stl"/>
+        <mesh filename="file://$(find ros2srrc_ur5_gazebo)/meshes/kinetic.glb"/>
       </geometry>
     </visual>
     <collision>
       <geometry>
-        <mesh filename="file://$(find ros2srrc_ur5_gazebo)/meshes/kinetic.glb"/>
+        <mesh filename="file://$(find ros2srrc_ur5_gazebo)/meshes/kinetic.stl"/>
       </geometry>
     </collision>

File: Industrial/ros2_SimRealRobotControl_gz/packages/ur5/ros2srrc_ur5_gazebo/urdf/cam_on_hand_params.xacro (robot description, xacro)
@@ -5,6 +5,6 @@
     <xacro:property name="cam_hand_pz" value="0.03" />
     <xacro:property name="cam_hand_or" value="0" />
-    <xacro:property name="cam_hand_op" value="-1.57" />
-    <xacro:property name="cam_hand_oy" value="1.57" />
+    <xacro:property name="cam_hand_op" value="0" />
+    <xacro:property name="cam_hand_oy" value="0" />
     <xacro:property name="parent_hand" value="tool0" />
 </robot>
