Commit message: Fix camera pose

File: Industrial/ros2_SimRealRobotControl_gz/packages/ur5/ros2srrc_ur5_gazebo/urdf/cam_on_base_params_gz.xacro (robot description, xacro)
@@ -4,7 +4,7 @@
     <xacro:property name="cam_base_py" value="0.0" />
     <xacro:property name="cam_base_pz" value="1.4" />
-    <xacro:property name="cam_base_or" value="0.0" />
-    <xacro:property name="cam_base_op" value="${pi/4}" />
-    <xacro:property name="cam_base_oy" value="${pi}" />
+    <xacro:property name="cam_base_or" value="1.57" />
+    <xacro:property name="cam_base_op" value="0" />
+    <xacro:property name="cam_base_oy" value="3.14" />
     <xacro:property name="parent_base" value="world" />
 </robot>

File: Industrial/ros2_SimRealRobotControl_gz/packages/ur5/ros2srrc_ur5_gazebo/urdf/cam_on_hand_params_gz.xacro (robot description, xacro)
@@ -5,6 +5,6 @@
     <xacro:property name="cam_hand_pz" value="0.03" />
     <xacro:property name="cam_hand_or" value="0" />
-    <xacro:property name="cam_hand_op" value="-1.57" />
-    <xacro:property name="cam_hand_oy" value="1.57" />
+    <xacro:property name="cam_hand_op" value="1.57" />
+    <xacro:property name="cam_hand_oy" value="0" />
     <xacro:property name="parent_hand" value="tool0" />
 </robot>

File: Industrial/ros2_SimRealRobotControl_gz/packages/ur5/ros2srrc_ur5_gazebo/urdf/ur5_robotiq_2f85_with_cams.urdf.xacro (robot description, xacro)
@@ -10,9 +10,9 @@
   <xacro:include filename="$(find ros2srrc_ur5_gazebo)/urdf/common_properties.xacro"/>
   <!-- HAND CAMERA -->
-  <xacro:include filename="$(find ros2srrc_ur5_gazebo)/urdf/cam_on_hand_params.xacro"/>
+  <xacro:include filename="$(find ros2srrc_ur5_gazebo)/urdf/cam_on_hand_params_gz.xacro"/>
   <xacro:property name="parent_hand" value="tool0"/>
   <xacro:include filename="$(find ros2srrc_ur5_gazebo)/urdf/cam_on_hand_gz.xacro"/>
   <!-- BASE CAMERA -->
-  <xacro:include filename="$(find ros2srrc_ur5_gazebo)/urdf/cam_on_base_params.xacro"/>
+  <xacro:include filename="$(find ros2srrc_ur5_gazebo)/urdf/cam_on_base_params_gz.xacro"/>
   <xacro:property name="parent_base" value="base_link"/>
   <xacro:property name="cam_base_pz" value="0.5"/>

Commit message: Fix camera pose

File: Industrial/ros2_SimRealRobotControl_gz/packages/ur5/ros2srrc_ur5_gazebo/urdf/cam_on_base_params_gz.xacro (robot description, xacro)
@@ -5,5 +5,5 @@
     <xacro:property name="cam_base_pz" value="1.4" />
     <xacro:property name="cam_base_or" value="1.57" />
-    <xacro:property name="cam_base_op" value="0" />
+    <xacro:property name="cam_base_op" value="0.4" />
     <xacro:property name="cam_base_oy" value="3.14" />
     <xacro:property name="parent_base" value="world" />

File: Industrial/ros2_SimRealRobotControl_gz/packages/ur5/ros2srrc_ur5_gazebo/urdf/cam_on_hand_params_gz.xacro (robot description, xacro)
@@ -4,6 +4,6 @@
     <xacro:property name="cam_hand_py" value="-0.067" />
     <xacro:property name="cam_hand_pz" value="0.03" />
-    <xacro:property name="cam_hand_or" value="0" />
-    <xacro:property name="cam_hand_op" value="1.57" />
+    <xacro:property name="cam_hand_or" value="3.14" />
+    <xacro:property name="cam_hand_op" value="-1.57" />
     <xacro:property name="cam_hand_oy" value="0" />
     <xacro:property name="parent_hand" value="tool0" />
