Commit message: Migrate cameras to harmonic

File: Industrial/ros2_SimRealRobotControl_gz/packages/ur5/ros2srrc_ur5_gazebo/urdf/cam_on_base_gz.xacro (robot description, xacro)
@@ -11,5 +11,5 @@
         <visual>
             <geometry>
-                <mesh filename="file://$(find ros2srrc_ur5_gazebo)/meshes/kinetic.stl"/>
+                <mesh filename="package://ros2srrc_ur5_gazebo/meshes/kinetic.stl"/>
             </geometry>
             <material name="dark_grey"/>
@@ -17,5 +17,5 @@
         <collision>
             <geometry>
-                <mesh filename="file://$(find ros2srrc_ur5_gazebo)/meshes/kinetic.dae"/>
+                <mesh filename="package://ros2srrc_ur5_gazebo/meshes/kinetic.dae"/>
             </geometry>
         </collision>

File: Industrial/ros2_SimRealRobotControl_gz/packages/ur5/ros2srrc_ur5_gazebo/urdf/cam_on_hand_gz.xacro (robot description, xacro)
@@ -11,5 +11,5 @@
         <visual>
             <geometry>
-                <mesh filename="file://$(find ros2srrc_ur5_gazebo)/meshes/kinetic.stl"/>
+                <mesh filename="package://ros2srrc_ur5_gazebo/meshes/kinetic.stl"/>
             </geometry>
             <material name="dark_grey"/>
@@ -17,5 +17,5 @@
         <collision>
             <geometry>
-                <mesh filename="file://$(find ros2srrc_ur5_gazebo)/meshes/kinetic.dae"/>
+                <mesh filename="package://ros2srrc_ur5_gazebo/meshes/kinetic.dae"/>
             </geometry>
         </collision>

File: Industrial/ros2_SimRealRobotControl_gz/packages/ur5/ros2srrc_ur5_gazebo/urdf/ur5_robotiq_2f85_with_cams_gz.urdf.xacro (robot description, xacro)
@@ -1,100 +1,130 @@
-<?xml version="1.0"?>
-<robot name="ur5" xmlns:xacro="http://www.ros.org/wiki/xacro">
-  <!-- ================= ARGUMENTOS ================= -->
+<?xml version="1.0" ?>
+<!--
+# ===================================== COPYRIGHT ===================================== #
+#                                                                                       #
+#  IFRA (Intelligent Flexible Robotics and Assembly) Group, CRANFIELD UNIVERSITY        #
+#  Created on behalf of the IFRA Group at Cranfield University, United Kingdom          #
+#  E-mail: IFRA@cranfield.ac.uk                                                         #
+#                                                                                       #
+#  Licensed under the Apache-2.0 License.                                               #
+#  You may not use this file except in compliance with the License.                     #
+#  You may obtain a copy of the License at: http://www.apache.org/licenses/LICENSE-2.0  #
+#                                                                                       #
+#  Unless required by applicable law or agreed to in writing, software distributed      #
+#  under the License is distributed on an "as-is" basis, without warranties or          #
+#  conditions of any kind, either express or implied. See the License for the specific  #
+#  language governing permissions and limitations under the License.                    #
+#                                                                                       #
+#  IFRA Group - Cranfield University                                                    #
+#  AUTHORS: Mikel Bueno Viso - Mikel.Bueno-Viso@cranfield.ac.uk                         #
+#           Dr. Seemal Asif  - s.asif@cranfield.ac.uk                                   #
+#           Prof. Phil Webb  - p.f.webb@cranfield.ac.uk                                 #
+#                                                                                       #
+#  Date: April, 2023.                                                                   #
+#                                                                                       #
+# ===================================== COPYRIGHT ===================================== #
+# ======= CITE OUR WORK ======= #
+# You can cite our work with the following statement:
+# IFRA-Cranfield (2023) ROS 2 Sim-to-Real Robot Control. URL: https://github.com/IFRA-Cranfield/ros2_SimRealRobotControl.
+-->
+<robot name="ur5" xmlns:xacro="http://ros.org/wiki/xacro">
+  <!-- PASS ARGUMENTS: -->
+  <xacro:arg name="bringup" default="false"/>
+  <xacro:property name="bringup" value="$(arg bringup)"/>
+  <xacro:arg name="hmi" default="false"/>
+  <xacro:property name="hmi" value="$(arg hmi)"/>
+  <xacro:arg name="robot_ip" default="0.0.0.0"/>
+  <xacro:property name="robot_ip" value="$(arg robot_ip)"/>
+  <xacro:arg name="EE" default="false"/>
+  <xacro:property name="EE" value="$(arg EE)"/>
+  <xacro:arg name="EE_name" default="none"/>
+  <xacro:property name="EE_name" value="$(arg EE_name)"/>
+  <!-- UR5 Control ARGUMENTS -->
+  <xacro:arg name="script_filename" default="none"/>
+  <xacro:property name="script_filename" value="$(arg script_filename)"/>
+  <xacro:arg name="input_recipe_filename" default="none"/>
+  <xacro:property name="input_recipe_filename" value="$(arg input_recipe_filename)"/>
+  <xacro:arg name="output_recipe_filename" default="none"/>
+  <xacro:property name="output_recipe_filename" value="$(arg output_recipe_filename)"/>
   <xacro:arg name="sim_gz" default="true"/>
-  <xacro:arg name="use_fake_hardware" default="false"/>
-  <!-- ================= UR5 OFICIAL (TEXTURAS OK) ================= -->
-  <xacro:include filename="$(find ur5_gripper_description)/urdf/ur.urdf.xacro"/>
-  <xacro:ur_robot
-    name="ur"
-    prefix=""
-    ur_type="ur5"
+  <xacro:arg name="simulation_controllers" default="$(find ros2srrc_robots)/ur5/config/controller.yaml"/>
+  <!-- Include XACRO-MACRO file of the UR5: -->
+  <xacro:include filename="$(find ros2srrc_robots)/ur5/urdf/ur5_macro.urdf.xacro"/>
+  <xacro:include filename="$(find ros2srrc_ur5_gazebo)/urdf/common_properties.xacro"/>
+  <xacro:include filename="$(find ros2srrc_ur5_gazebo)/urdf/cam_on_hand_params.xacro"/>
+  <xacro:include filename="$(find ros2srrc_ur5_gazebo)/urdf/cam_on_hand_gz.xacro"/>
+  <xacro:include filename="$(find ros2srrc_ur5_gazebo)/urdf/cam_on_base_params.xacro"/>
+  <xacro:include filename="$(find ros2srrc_ur5_gazebo)/urdf/cam_on_base_gz.xacro"/>
+  <xacro:ur5
+    bringup="${bringup}"
+    robot_ip="${robot_ip}"
+    EE="${EE}"
+    EE_name="${EE_name}"
+    script_filename="${script_filename}"
+    input_recipe_filename="${input_recipe_filename}"
+    output_recipe_filename="${output_recipe_filename}"
   />
-  <!-- ================= GRIPPER ================= -->
-  <xacro:include filename="$(find robotiq_description)/urdf/robotiq_85_gripper.urdf.xacro"/>
-  <xacro:include filename="$(find robotiq_description)/urdf/robotiq_85_gripper.ros2_control.xacro"/>
-  <!-- Coupler -->
-  <link name="robotiq_coupler">
-    <visual>
+  <!-- Include XACRO-MACRO file of the Robotiq 2f-85: -->
+  <xacro:include filename="$(find ros2srrc_endeffectors)/robotiq_2f85/urdf/robotiq_2f85_macro.urdf.xacro"/>
+  <xacro:robotiq_2f85
+    bringup="${bringup}"
+    parent_link="tool0"
+  />
+  <!-- Load ROS 2 Gazebo Plugin -->
+  <xacro:if value="$(arg sim_gz)">
+    <gazebo>
+      <plugin filename="gz_ros2_control-system" name="gz_ros2_control::GazeboSimROS2ControlPlugin">
+        <parameters>$(arg simulation_controllers)</parameters>
+        <xacro:if value="${EE}">
+          <parameters>$(find ros2srrc_endeffectors)/${EE_name}/config/controller.yaml</parameters>
+        </xacro:if>
+      </plugin>
+    </gazebo>
+  </xacro:if>
+  <!-- World: LINK -->
+  <link name="world"/>
+  <!-- Robot Stand: LINK -->
+  <link name='robot_stand'>
+    <inertial>
+      <origin xyz="0 0 0" rpy="0 0 0"/>
+      <mass value="100"/>
+      <inertia ixx="0.01"  ixy="0"  ixz="0" iyy="0.01" iyz="0" izz="0.01" />
+    </inertial>
+    <collision name='collision'>
+      <origin xyz="0 0 0" rpy=" 0 0 0"/>
       <geometry>
-        <mesh filename="package://robotiq_description/meshes/robotiq_85_coupler.stl"/>
+        <box size = "0.2 0.2 1.0"/>
+      </geometry>
+    </collision>
+    <visual name='chassis_visual'>
+      <origin xyz="0 0 0" rpy=" 0 0 0"/>
+      <geometry>
+        <box size = "0.2 0.2 1.0"/>
       </geometry>
     </visual>
-    <collision>
-      <geometry>
-        <cylinder radius="0.04" length="0.015"/>
-      </geometry>
-    </collision>
   </link>
-  <joint name="robotiq_coupler_joint" type="fixed">
-    <origin xyz="0 0 0.004" rpy="0 0 ${-pi/2.0}"/>
-    <parent link="tool0"/>
-    <child link="robotiq_coupler"/>
+  <!-- Robot Stand: FIXED JOINT -->
+  <joint name="world_joint" type="fixed">
+    <parent link= "world" />
+    <child link = "robot_stand" />
+    <origin xyz="0.0 0.0 0.5" rpy="0.0 0.0 0.0" />
   </joint>
-  <xacro:robotiq_85_gripper prefix="" parent="robotiq_coupler">
-    <origin xyz="0 0 0.004" rpy="0 ${-pi/2} ${pi}"/>
-  </xacro:robotiq_85_gripper>
-  <!-- ================= ROS2 CONTROL ================= -->
-  <xacro:include filename="$(find ur5_gripper_description)/urdf/ur.ros2_control.xacro"/>
-  <xacro:ur_ros2_control
-    name="ur"
-    prefix=""
-    sim_gz="true"
-    use_fake_hardware="${use_fake_hardware}"
-    script_filename=""
-    output_recipe_filename=""
-    input_recipe_filename=""
-    tf_prefix=""
-    hash_kinematics=""
-    robot_ip="0.0.0.0"
-  />
-  <xacro:robotiq_85_ros2_control
-    name="robotiq"
-    prefix=""
-    sim_gz="true"
-    use_fake_hardware="${use_fake_hardware}"
-  />
-  <!-- ================= STAND ================= -->
-  <link name="world"/>
-  <link name="robot_stand">
-    <inertial>
-      <origin xyz="0 0 0"/>
-      <mass value="100"/>
-      <inertia ixx="0.01" ixy="0" ixz="0" iyy="0.01" iyz="0" izz="0.01"/>
-    </inertial>
-    <visual>
-      <geometry>
-        <box size="0.2 0.2 1.0"/>
-      </geometry>
-    </visual>
-    <collision>
-      <geometry>
-        <box size="0.2 0.2 1.0"/>
-      </geometry>
-    </collision>
-  </link>
-  <joint name="world_joint" type="fixed">
-    <parent link="world"/>
-    <child link="robot_stand"/>
-    <origin xyz="0 0 0.5"/>
+  <!-- Robot Stand: Robot+Stand JOINT -->
+  <joint name="stand_joint" type="fixed">
+    <parent link= "robot_stand" />
+    <child link = "base_link" />
+    <origin xyz="0.0 0.0 0.52" rpy="0.0 0.0 0.0" />
   </joint>
-  <joint name="stand_joint" type="fixed">
-    <parent link="robot_stand"/>
-    <child link="base_link"/>
-    <origin xyz="0 0 0.52"/>
-  </joint>
-  <!-- ================= CAMARAS (USANDO TUS MACROS) ================= -->
-  <!-- PARAMS -->
-  <xacro:include filename="$(find ros2srrc_ur5_gazebo)/urdf/cam_on_hand_params.xacro"/>
-  <xacro:include filename="$(find ros2srrc_ur5_gazebo)/urdf/cam_on_base_params.xacro"/>
-  <!-- GZ SENSORS -->
-  <xacro:include filename="$(find ros2srrc_ur5_gazebo)/urdf/cam_on_hand_gz.xacro"/>
-  <xacro:include filename="$(find ros2srrc_ur5_gazebo)/urdf/cam_on_base_gz.xacro"/>
-  <!-- INSTANCIACIÓN -->
-  <xacro:cam_on_hand_gz parent_link="wrist_3_link"/>
-  <xacro:cam_on_base_gz parent_link="base_link"/>
-  <!-- ================= GAZEBO CONTROL ================= -->
-  <gazebo>
-    <plugin filename="gz_ros2_control-system" name="gz_ros2_control::GazeboSimROS2ControlPlugin"/>
-  </gazebo>
+  <!-- ros2srrc_HMI CAMERA -->
+  <xacro:if value="${hmi}">
+    <xacro:include filename="$(find ros2srrc_hmi)/urdf/hmicamera.urdf.xacro"/>
+    <xacro:HMI_camera
+      x="2.5"
+      y="1.50"
+      z="2.0"
+      roll="0.0"
+      pitch="0.35"
+      yaw="-2.6"
+    />
+  </xacro:if>
 </robot>

Commit message: Fix cam xacros

File: Industrial/ros2_SimRealRobotControl_gz/packages/ur5/ros2srrc_ur5_gazebo/urdf/cam_on_base_gz.xacro (robot description, xacro)
@@ -21,5 +21,5 @@
   </link>
   <joint name="base_camera_joint" type="fixed">
-    <parent link="${parent_base}"/>
+    <parent link="base_link"/>
     <child link="base_camera_link"/>
     <origin xyz="${cam_base_px} ${cam_base_py} ${cam_base_pz}"
@@ -33,8 +33,8 @@
   </joint>
   <gazebo reference="base_camera_link">
-    <sensor name="base_camera" type="depth_camera">
+    <sensor name="base_camera" type="rgbd_camera">
       <always_on>true</always_on>
+      <visualize>true</visualize>
       <update_rate>30</update_rate>
-      <visualize>true</visualize>
       <topic>/base_camera</topic>
       <camera>

File: Industrial/ros2_SimRealRobotControl_gz/packages/ur5/ros2srrc_ur5_gazebo/urdf/cam_on_hand_gz.xacro (robot description, xacro)
@@ -21,5 +21,5 @@
   </link>
   <joint name="hand_camera_joint" type="fixed">
-    <parent link="${parent_hand}"/>
+    <parent link="tool0"/>
     <child link="hand_camera_link"/>
     <origin xyz="${cam_hand_px} ${cam_hand_py} ${cam_hand_pz}"
@@ -33,8 +33,8 @@
   </joint>
   <gazebo reference="hand_camera_link">
-    <sensor name="hand_camera" type="depth_camera">
+    <sensor name="hand_camera" type="rgbd_camera">
       <always_on>true</always_on>
+      <visualize>true</visualize>
       <update_rate>30</update_rate>
-      <visualize>true</visualize>
       <topic>/hand_camera</topic>
       <camera>

Commit message: Try to fix camera texture

File: Industrial/ros2_SimRealRobotControl_gz/packages/ur5/ros2srrc_ur5_gazebo/urdf/cam_on_base_gz.xacro (robot description, xacro)
@@ -11,6 +11,12 @@
     <visual>
       <geometry>
-        <mesh filename="file://$(find ros2srrc_ur5_gazebo)/meshes/kinetic.stl"/>
+        <box>
+          <size>0.05 0.05 0.05</size>
+        </box>
       </geometry>
+      <material>
+        <ambient>0.2 0.2 0.2 1</ambient>
+        <diffuse>0.2 0.2 0.2 1</diffuse>
+      </material>
     </visual>
     <collision>

File: Industrial/ros2_SimRealRobotControl_gz/packages/ur5/ros2srrc_ur5_gazebo/urdf/cam_on_hand_gz.xacro (robot description, xacro)
@@ -11,6 +11,12 @@
     <visual>
       <geometry>
-        <mesh filename="file://$(find ros2srrc_ur5_gazebo)/meshes/kinetic.stl"/>
+        <box>
+          <size>0.05 0.05 0.05</size>
+        </box>
       </geometry>
+      <material>
+        <ambient>0.2 0.2 0.2 1</ambient>
+        <diffuse>0.2 0.2 0.2 1</diffuse>
+      </material>
     </visual>
     <collision>

Commit message: Try to fix camera texture

File: Industrial/ros2_SimRealRobotControl_gz/packages/ur5/ros2srrc_ur5_gazebo/urdf/cam_on_base_gz.xacro (robot description, xacro)
@@ -1,5 +1,5 @@
 <?xml version="1.0"?>
 <robot xmlns:xacro="http://ros.org/wiki/xacro">
-  <link name="base_camera_link">
+  <link name="hand_camera_link">
     <inertial>
       <origin xyz="-0.00936 -0.00003 -0.00273" rpy="0 0 0"/>
@@ -11,12 +11,6 @@
     <visual>
       <geometry>
-        <box>
-          <size>0.05 0.05 0.05</size>
-        </box>
+        <mesh filename="file://$(find ros2srrc_ur5_gazebo)/meshes/kinetic.stl"/>
       </geometry>
-      <material>
-        <ambient>0.2 0.2 0.2 1</ambient>
-        <diffuse>0.2 0.2 0.2 1</diffuse>
-      </material>
     </visual>
     <collision>
@@ -26,22 +20,25 @@
     </collision>
   </link>
-  <joint name="base_camera_joint" type="fixed">
-    <parent link="base_link"/>
-    <child link="base_camera_link"/>
-    <origin xyz="${cam_base_px} ${cam_base_py} ${cam_base_pz}"
-            rpy="${cam_base_or} ${cam_base_op} ${cam_base_oy}"/>
+  <gazebo reference="hand_camera_link">
+    <material>Gazebo/Grey</material>
+  </gazebo>
+  <joint name="hand_camera_joint" type="fixed">
+    <parent link="tool0"/>
+    <child link="hand_camera_link"/>
+    <origin xyz="${cam_hand_px} ${cam_hand_py} ${cam_hand_pz}"
+            rpy="${cam_hand_or} ${cam_hand_op} ${cam_hand_oy}"/>
   </joint>
-  <link name="base_camera_optical_link"/>
-  <joint name="base_camera_optical_joint" type="fixed">
-    <parent link="base_camera_link"/>
-    <child link="base_camera_optical_link"/>
+  <link name="hand_camera_optical_link"/>
+  <joint name="hand_camera_optical_joint" type="fixed">
+    <parent link="hand_camera_link"/>
+    <child link="hand_camera_optical_link"/>
     <origin xyz="0 0 0" rpy="-1.57 0 -1.57"/>
   </joint>
-  <gazebo reference="base_camera_link">
-    <sensor name="base_camera" type="rgbd_camera">
+  <gazebo reference="hand_camera_link">
+    <sensor name="hand_camera" type="rgbd_camera">
       <always_on>true</always_on>
       <visualize>true</visualize>
       <update_rate>30</update_rate>
-      <topic>/base_camera</topic>
+      <topic>/hand_camera</topic>
       <camera>
         <horizontal_fov>1.047</horizontal_fov>

File: Industrial/ros2_SimRealRobotControl_gz/packages/ur5/ros2srrc_ur5_gazebo/urdf/cam_on_hand_gz.xacro (robot description, xacro)
@@ -1,5 +1,5 @@
 <?xml version="1.0"?>
 <robot xmlns:xacro="http://ros.org/wiki/xacro">
-  <link name="hand_camera_link">
+  <link name="base_camera_link">
     <inertial>
       <origin xyz="-0.00936 -0.00003 -0.00273" rpy="0 0 0"/>
@@ -11,12 +11,6 @@
     <visual>
       <geometry>
-        <box>
-          <size>0.05 0.05 0.05</size>
-        </box>
+        <mesh filename="file://$(find ros2srrc_ur5_gazebo)/meshes/kinetic.stl"/>
       </geometry>
-      <material>
-        <ambient>0.2 0.2 0.2 1</ambient>
-        <diffuse>0.2 0.2 0.2 1</diffuse>
-      </material>
     </visual>
     <collision>
@@ -26,22 +20,25 @@
     </collision>
   </link>
-  <joint name="hand_camera_joint" type="fixed">
-    <parent link="tool0"/>
-    <child link="hand_camera_link"/>
-    <origin xyz="${cam_hand_px} ${cam_hand_py} ${cam_hand_pz}"
-            rpy="${cam_hand_or} ${cam_hand_op} ${cam_hand_oy}"/>
+  <gazebo reference="hand_camera_link">
+    <material>Gazebo/Grey</material>
+  </gazebo>
+  <joint name="base_camera_joint" type="fixed">
+    <parent link="base_link"/>
+    <child link="base_camera_link"/>
+    <origin xyz="${cam_base_px} ${cam_base_py} ${cam_base_pz}"
+            rpy="${cam_base_or} ${cam_base_op} ${cam_base_oy}"/>
   </joint>
-  <link name="hand_camera_optical_link"/>
-  <joint name="hand_camera_optical_joint" type="fixed">
-    <parent link="hand_camera_link"/>
-    <child link="hand_camera_optical_link"/>
+  <link name="base_camera_optical_link"/>
+  <joint name="base_camera_optical_joint" type="fixed">
+    <parent link="base_camera_link"/>
+    <child link="base_camera_optical_link"/>
     <origin xyz="0 0 0" rpy="-1.57 0 -1.57"/>
   </joint>
-  <gazebo reference="hand_camera_link">
-    <sensor name="hand_camera" type="rgbd_camera">
+  <gazebo reference="base_camera_link">
+    <sensor name="base_camera" type="rgbd_camera">
       <always_on>true</always_on>
       <visualize>true</visualize>
       <update_rate>30</update_rate>
-      <topic>/hand_camera</topic>
+      <topic>/base_camera</topic>
       <camera>
         <horizontal_fov>1.047</horizontal_fov>

Commit message: Fix camera base xacro

File: Industrial/ros2_SimRealRobotControl_gz/packages/ur5/ros2srrc_ur5_gazebo/urdf/cam_on_base_gz.xacro (robot description, xacro)
@@ -1,5 +1,5 @@
 <?xml version="1.0"?>
 <robot xmlns:xacro="http://ros.org/wiki/xacro">
-  <link name="hand_camera_link">
+  <link name="base_camera_link">
     <inertial>
       <origin xyz="-0.00936 -0.00003 -0.00273" rpy="0 0 0"/>
@@ -20,25 +20,25 @@
     </collision>
   </link>
-  <gazebo reference="hand_camera_link">
+  <gazebo reference="base_camera_link">
     <material>Gazebo/Grey</material>
   </gazebo>
-  <joint name="hand_camera_joint" type="fixed">
-    <parent link="tool0"/>
-    <child link="hand_camera_link"/>
-    <origin xyz="${cam_hand_px} ${cam_hand_py} ${cam_hand_pz}"
-            rpy="${cam_hand_or} ${cam_hand_op} ${cam_hand_oy}"/>
+  <joint name="base_camera_joint" type="fixed">
+    <parent link="base_link"/>
+    <child link="base_camera_link"/>
+    <origin xyz="${cam_base_px} ${cam_base_py} ${cam_base_pz}"
+            rpy="${cam_base_or} ${cam_base_op} ${cam_base_oy}"/>
   </joint>
-  <link name="hand_camera_optical_link"/>
-  <joint name="hand_camera_optical_joint" type="fixed">
-    <parent link="hand_camera_link"/>
-    <child link="hand_camera_optical_link"/>
+  <link name="base_camera_optical_link"/>
+  <joint name="base_camera_optical_joint" type="fixed">
+    <parent link="base_camera_link"/>
+    <child link="base_camera_optical_link"/>
     <origin xyz="0 0 0" rpy="-1.57 0 -1.57"/>
   </joint>
-  <gazebo reference="hand_camera_link">
-    <sensor name="hand_camera" type="rgbd_camera">
+  <gazebo reference="base_camera_link">
+    <sensor name="base_camera" type="rgbd_camera">
       <always_on>true</always_on>
       <visualize>true</visualize>
       <update_rate>30</update_rate>
-      <topic>/hand_camera</topic>
+      <topic>/base_camera</topic>
       <camera>
         <horizontal_fov>1.047</horizontal_fov>

Commit message: Try new camera texture

File: Industrial/ros2_SimRealRobotControl_gz/packages/ur5/ros2srrc_ur5_gazebo/urdf/cam_on_base_gz.xacro (robot description, xacro)
@@ -11,5 +11,5 @@
     <visual>
       <geometry>
-        <mesh filename="file://$(find ros2srrc_ur5_gazebo)/meshes/kinetic.stl"/>
+        <mesh filename="file://$(find ros2srrc_ur5_gazebo)/meshes/kinetic.gbl"/>
       </geometry>
     </visual>

File: Industrial/ros2_SimRealRobotControl_gz/packages/ur5/ros2srrc_ur5_gazebo/urdf/cam_on_hand_gz.xacro (robot description, xacro)
@@ -16,5 +16,5 @@
     <collision>
       <geometry>
-        <mesh filename="file://$(find ros2srrc_ur5_gazebo)/meshes/kinetic.dae"/>
+        <mesh filename="file://$(find ros2srrc_ur5_gazebo)/meshes/kinetic.gbl"/>
       </geometry>
     </collision>

Commit message: Try new camera texture

File: Industrial/ros2_SimRealRobotControl_gz/packages/ur5/ros2srrc_ur5_gazebo/urdf/cam_on_base_gz.xacro (robot description, xacro)
@@ -16,11 +16,8 @@
     <collision>
       <geometry>
-        <mesh filename="file://$(find ros2srrc_ur5_gazebo)/meshes/kinetic.dae"/>
+        <mesh filename="file://$(find ros2srrc_ur5_gazebo)/meshes/kinetic.stl"/>
       </geometry>
     </collision>
   </link>
-  <gazebo reference="base_camera_link">
-    <material>Gazebo/Grey</material>
-  </gazebo>
   <joint name="base_camera_joint" type="fixed">
     <parent link="base_link"/>

File: Industrial/ros2_SimRealRobotControl_gz/packages/ur5/ros2srrc_ur5_gazebo/urdf/cam_on_hand_gz.xacro (robot description, xacro)
@@ -20,7 +20,4 @@
     </collision>
   </link>
-  <gazebo reference="hand_camera_link">
-    <material>Gazebo/Grey</material>
-  </gazebo>
   <joint name="hand_camera_joint" type="fixed">
     <parent link="tool0"/>

Commit message: Try new camera texture

File: Industrial/ros2_SimRealRobotControl_gz/packages/ur5/ros2srrc_ur5_gazebo/urdf/cam_on_base_gz.xacro (robot description, xacro)
@@ -11,5 +11,5 @@
     <visual>
       <geometry>
-        <mesh filename="file://$(find ros2srrc_ur5_gazebo)/meshes/kinetic.gbl"/>
+        <mesh filename="file://$(find ros2srrc_ur5_gazebo)/meshes/kinetic.glb"/>
       </geometry>
     </visual>

File: Industrial/ros2_SimRealRobotControl_gz/packages/ur5/ros2srrc_ur5_gazebo/urdf/cam_on_hand_gz.xacro (robot description, xacro)
@@ -16,5 +16,5 @@
     <collision>
       <geometry>
-        <mesh filename="file://$(find ros2srrc_ur5_gazebo)/meshes/kinetic.gbl"/>
+        <mesh filename="file://$(find ros2srrc_ur5_gazebo)/meshes/kinetic.glb"/>
       </geometry>
     </collision>
