Commit message: Final fix

File: Industrial/ros2_SimRealRobotControl_gz/packages/ur5/ros2srrc_ur5_gazebo/urdf/cam_on_base_gz.xacro (robot description, xacro)
@@ -5,7 +5,5 @@
       <origin xyz="-0.00936 -0.00003 -0.00273" rpy="0 0 0"/>
       <mass value="0.2197"/>
-      <inertia ixx="4.29247e-06" ixy="0" ixz="2.565e-08"
-               iyy="8.027e-08" iyz="0"
-               izz="4.27339e-06"/>
+      <inertia ixx="4.29247e-06" ixy="0" ixz="2.565e-08" iyy="8.027e-08" iyz="0" izz="4.27339e-06"/>
     </inertial>
     <visual>
@@ -23,6 +21,5 @@
     <parent link="base_link"/>
     <child link="base_camera_link"/>
-    <origin xyz="${cam_base_px} ${cam_base_py} ${cam_base_pz}"
-            rpy="${cam_base_or} ${cam_base_op} ${cam_base_oy}"/>
+    <origin xyz="${cam_base_px} ${cam_base_py} ${cam_base_pz}" rpy="${cam_base_or} ${cam_base_op} ${cam_base_oy}"/>
   </joint>
   <link name="base_camera_optical_link"/>
@@ -33,10 +30,11 @@
   </joint>
   <gazebo reference="base_camera_link">
-    <sensor name="base_camera" type="rgbd_camera">
+    <sensor name="base_camera" type="camera">
       <always_on>true</always_on>
       <visualize>true</visualize>
       <update_rate>30</update_rate>
-      <topic>/base_camera</topic>
-      <camera>
+      <topic>/base_camera/image</topic>
+      <camera name="base_camera">
+        <camera_info_topic>/base_camera/camera_info</camera_info_topic>
         <horizontal_fov>1.047</horizontal_fov>
         <image>

File: Industrial/ros2_SimRealRobotControl_gz/packages/ur5/ros2srrc_ur5_gazebo/urdf/cam_on_hand_gz.xacro (robot description, xacro)
@@ -5,7 +5,5 @@
       <origin xyz="-0.00936 -0.00003 -0.00273" rpy="0 0 0"/>
       <mass value="0.2197"/>
-      <inertia ixx="4.29247e-06" ixy="0" ixz="2.565e-08"
-               iyy="8.027e-08" iyz="0"
-               izz="4.27339e-06"/>
+      <inertia ixx="4.29247e-06" ixy="0" ixz="2.565e-08" iyy="8.027e-08" iyz="0" izz="4.27339e-06"/>
     </inertial>
     <visual>
@@ -23,6 +21,5 @@
     <parent link="tool0"/>
     <child link="hand_camera_link"/>
-    <origin xyz="${cam_hand_px} ${cam_hand_py} ${cam_hand_pz}"
-            rpy="${cam_hand_or} ${cam_hand_op} ${cam_hand_oy}"/>
+    <origin xyz="${cam_hand_px} ${cam_hand_py} ${cam_hand_pz}" rpy="${cam_hand_or} ${cam_hand_op} ${cam_hand_oy}"/>
   </joint>
   <link name="hand_camera_optical_link"/>
@@ -33,10 +30,11 @@
   </joint>
   <gazebo reference="hand_camera_link">
-    <sensor name="hand_camera" type="rgbd_camera">
+    <sensor name="hand_camera" type="camera">
       <always_on>true</always_on>
       <visualize>true</visualize>
       <update_rate>30</update_rate>
-      <topic>/hand_camera</topic>
-      <camera>
+      <topic>/hand_camera/image</topic>
+      <camera name="camera">
+        <camera_info_topic>/hand_camera/camera_info</camera_info_topic>
         <horizontal_fov>1.047</horizontal_fov>
         <image>

File: Industrial/ur5_gripper_description/urdf/ur5_robotiq85_gripper.urdf.xacro (robot description, xacro)
@@ -16,8 +16,9 @@
   <xacro:include filename="$(find ur5_gripper_description)/urdf/ur.ros2_control.xacro" />
   <xacro:if value="$(arg camera)">
-    <xacro:include filename="$(find ros2srrc_ur5_gazebo)/urdf/cam_on_hand_params.xacro"/>
-    <xacro:include filename="$(find ros2srrc_ur5_gazebo)/urdf/cam_on_hand.xacro"/>
-    <xacro:include filename="$(find ros2srrc_ur5_gazebo)/urdf/cam_on_base_params.xacro"/>
-    <xacro:include filename="$(find ros2srrc_ur5_gazebo)/urdf/cam_on_base.xacro"/>
+    <xacro:include filename="$(find ros2srrc_ur5_gazebo)/urdf/common_properties.xacro"/>
+    <xacro:include filename="$(find ros2srrc_ur5_gazebo)/urdf/cam_on_hand_params_gz.xacro"/>
+    <xacro:include filename="$(find ros2srrc_ur5_gazebo)/urdf/cam_on_hand_gz.xacro"/>
+    <xacro:include filename="$(find ros2srrc_ur5_gazebo)/urdf/cam_on_base_params_gz.xacro"/>
+    <xacro:include filename="$(find ros2srrc_ur5_gazebo)/urdf/cam_on_base_gz.xacro"/>
   </xacro:if>
   <!-- Coupler -->
