Commit message: Update urdf of circuits

File: Universes/montmelo_line.urdf (robot description, URDF)
Before this commit: robot f1_montmelo, 1 links, 0 joints
Links:
- link f1: geometry visual mesh filename=package://f1/models/f1_renault/Renault/Car.obj scale=0.2 0.2 0.2; visual mesh filename=package://f1/models/montmelo_line/meshes/montmelo.dae

File: Universes/montreal_line.urdf (robot description, URDF)
Before this commit: robot f1_monteral, 1 links, 0 joints
Links:
- link f1: geometry visual mesh filename=package://f1/models/f1_renault/Renault/Car.obj scale=0.2 0.2 0.2; visual mesh filename=package://f1/models/montreal_line/meshes/montreal.dae

File: Universes/nurburgring_line.urdf (robot description, URDF)
Before this commit: robot numburgring_line, 1 links, 0 joints
Links:
- link f1: geometry visual mesh filename=package://f1/models/f1_renault/Renault/Car.obj scale=0.2 0.2 0.2; visual mesh filename=package://f1/models/nurburgring_line/meshes/Circuito_Nurbur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

File: Universes/nurburgring_line_ackermann.urdf (robot description, URDF)
Before this commit: robot numburgring_line, 1 links, 0 joints
Links:
- link f1: geometry visual mesh filename=package://f1/models/f1_renault/Renault/Car.obj scale=0.2 0.2 0.2; visual mesh filename=package://f1/models/nurburgring_line/meshes/Circuito_Nurbur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

File: Universes/nurburgring_line_followingcam.urdf (robot description, URDF)
Before this commit: robot numburgring_line, 1 links, 0 joints
Links:
- link f1: geometry visual mesh filename=package://f1/models/f1_renault/Renault/Car.obj scale=0.2 0.2 0.2; visual mesh filename=package://f1/models/nurburgring_line/meshes/Circuito_Nurbur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

File: Universes/simple_circuit.urdf (robot description, URDF)
Before this commit: robot simple_circuit, 1 links, 0 joints
Links:
- link f1: geometry visual mesh filename=package://f1/models/f1_renault/Renault/Car.obj scale=0.2 0.2 0.2; visual mesh filename=package://f1/models/simple_circuit/meshes/simple_line.obj

File: Universes/simple_circuit_ackermann.urdf (robot description, URDF)
Before this commit: robot simple_circuit, 1 links, 0 joints
Links:
- link f1: geometry visual mesh filename=package://f1/models/f1_renault/Renault/Car.obj scale=0.2 0.2 0.2; visual mesh filename=package://f1/models/simple_circuit/meshes/simple_line.obj
