Commit message: Fix urdf mesh

File: Universes/simple_circuit.urdf (robot description, URDF)
Before this commit: robot simple_circuit, 1 links, 0 joints
Links:
- link f1: geometry visual mesh filename=package://f1/models/f1_renault/Renault/Car.obj scale=0.2 0.2 0.2; visual mesh filename=package://f1/models/simple_circuit/meshes/simple_line.dae

File: Universes/simple_circuit_ackermann.urdf (robot description, URDF)
Before this commit: robot simple_circuit, 1 links, 0 joints
Links:
- link f1: geometry visual mesh filename=package://f1/models/f1_renault/Renault/Car.obj scale=0.2 0.2 0.2; visual mesh filename=package://f1/models/simple_circuit/meshes/simple_line.dae

File: Universes/simple_circuit_obstacles.urdf (robot description, URDF)
Before this commit: robot simple_circuit, 13 links, 0 joints
Links:
- link f1: geometry visual mesh filename=package://f1/models/f1_renault/Renault/Car.obj scale=0.2 0.2 0.2; visual mesh filename=package://f1/models/simple_circuit/meshes/simple_line.dae
