Commit message: Fix broken urdfs

File: Universes/pallet_warehouse_with_robot.urdf (robot description, URDF)
Before this commit: robot pallet_warehouse_with_robot, 58 links, 14 joints
Links:
- link base_link: geometry collision box size=0.532 0.532 0.188; visual mesh filename=package://amazon_warehouse_harmonic/models/amazon_robot_har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 scale=0.002 0.002 0.002
- link base_scan: geometry collision cylinder length=0.0315 radius=0.055; visual mesh filename=package://amazon_warehouse_harmonic/models/amazon_robot_har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 scale=0.002 0.002 0.002
- link warehouse_walls: geometry visual mesh filename=package://amazon_warehouse_harmonic//models/warehouse_walls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
- link wheel_left_link: geometry collision cylinder length=0.020 radius=0.072; visual mesh filename=package://amazon_warehouse_harmonic/models/amazon_robot_har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 scale=0.002 0.002 0.002
- link wheel_right_link: geometry collision cylinder length=0.020 radius=0.072; visual mesh filename=package://amazon_warehouse_harmonic/models/amazon_robot_har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 scale=0.002 0.002 0.002
