Commit message: Clean couple of scenes in urdf

File: Universes/autopark_battery.urdf (robot description, URDF)
Before this commit: robot autopark_battery, 20 links, 1 joints
Links:
- removed link prius_autoparking
Joints:
- removed joint base_joint

File: Universes/autopark_line.urdf (robot description, URDF)
Before this commit: robot autopark_line, 16 links, 1 joints
Links:
- removed link prius_autoparking
Joints:
- removed joint base_joint

File: Universes/autopark_sideways.urdf (robot description, URDF)
Before this commit: robot autopark_sideways, 19 links, 1 joints
Links:
- removed link prius_autoparking
Joints:
- removed joint base_joint

File: Universes/basic_city.urdf (robot description, URDF)
Before this commit: robot cityLarge_harmonic, 1 links, 0 joints
Links:
- link city: geometry visual mesh filename=package://city_assets/models/large_basic_city/meshes/city.o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 scale=1 1 1
