Commit message: Change house

File: Universes/detailed_house.urdf (robot description, URDF)
Before this commit: robot global_nav, 1 links, 0 joints
Links:
- removed link Lake House
- added link grass_link; visual box size=15 15 0.01
- added link marker_visual_loc_link; visual mesh filename=package://marker_visual_loc/models/Lake House/meshes/house.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 scale=0.1 0.1 0.1
