Commit message: Clean more worlds

File: Universes/laser_map.urdf (robot description, URDF)
Before this commit: robot warehouse_world, 38 links, 37 joints
Links:
- removed link base_link
- removed link base_scan
- removed link camera_depth_frame
- removed link camera_depth_optical_frame
- removed link camera_link
- removed link camera_rgb_frame
- removed link camera_rgb_optical_frame
- removed link caster_back_left_link
- removed link caster_back_right_link
- removed link imu_link
- removed link wheel_left_link
- removed link wheel_right_link
Joints:
- removed joint base_footprint_robot
- removed joint camera_depth_joint
- removed joint camera_depth_optical_joint
- removed joint camera_joint
- removed joint camera_rgb_joint
- removed joint camera_rgb_optical_joint
- removed joint caster_back_left_joint
- removed joint caster_back_right_joint
- removed joint imu_joint
- removed joint scan_joint
- removed joint wheel_left_joint
- removed joint wheel_right_joint

File: Universes/rescue_people.urdf (robot description, URDF)
Before this commit: robot rescue_people, 8 links, 0 joints
Links:
- link ocean: geometry visual box size=150 150 0.01

File: Universes/small_house.urdf (robot description, URDF)
Before this commit: robot roomba_house, 32 links, 28 joints
Links:
- removed link RoCKIn
- removed link Wall_12
- removed link Wall_14
- removed link Wall_16
- removed link Wall_18
- removed link Wall_2
- removed link Wall_20
- removed link Wall_22
- removed link Wall_24
- removed link Wall_28
- removed link Wall_30
- removed link Wall_32
- removed link Wall_35
- removed link Wall_8
- link base: geometry visual mesh filename=package://roomba_robot/models/house_int2/meshes/model.dae
- link floor: geometry 
Joints:
- removed joint RoCKIn_joint
- removed joint Wall_12_joint
- removed joint Wall_14_joint
- removed joint Wall_16_joint
- removed joint Wall_18_joint
- removed joint Wall_20_joint
- removed joint Wall_22_joint
- removed joint Wall_24_joint
- removed joint Wall_28_joint
- removed joint Wall_2_joint
- removed joint Wall_30_joint
- removed joint Wall_32_joint
- removed joint Wall_35_joint
- removed joint Wall_8_joint

File: Universes/warehouse1.urdf (robot description, URDF)
Before this commit: robot small_warehouse, 30 links, 14 joints
Links:
- removed link base_footprint
- removed link base_link
- removed link base_scan
- removed link camera_depth_frame
- removed link camera_depth_optical_frame
- removed link camera_link
- removed link camera_rgb_frame
- removed link camera_rgb_optical_frame
- removed link caster_back_left_link
- removed link caster_back_right_link
- removed link imu_link
- removed link link_platform_mid
- removed link wheel_left_link
- removed link wheel_right_link
Joints:
- removed joint base_joint
- removed joint camera_depth_joint
- removed joint camera_depth_optical_joint
- removed joint camera_joint
- removed joint camera_rgb_joint
- removed joint camera_rgb_optical_joint
- removed joint caster_back_left_joint
- removed joint caster_back_right_joint
- removed joint imu_joint
- removed joint lift_joint
- removed joint platform_joint
- removed joint scan_joint
- removed joint wheel_left_joint
- removed joint wheel_right_joint

File: Universes/warehouse2.urdf (robot description, URDF)
Before this commit: robot pallet_warehouse_with_robot, 318 links, 266 joints
Links:
- removed link base_footprint
- removed link base_link
- removed link base_scan
- removed link camera_depth_frame
- removed link camera_depth_optical_frame
- removed link camera_link
- removed link camera_rgb_frame
- removed link camera_rgb_optical_frame
- removed link caster_back_left_link
- removed link caster_back_right_link
- removed link imu_link
- removed link link_platform_mid
- removed link wheel_left_link
- removed link wheel_right_link
Joints:
- removed joint base_joint
- removed joint camera_depth_joint
- removed joint camera_depth_optical_joint
- removed joint camera_joint
- removed joint camera_rgb_joint
- removed joint camera_rgb_optical_joint
- removed joint caster_back_left_joint
- removed joint caster_back_right_joint
- removed joint imu_joint
- removed joint lift_joint
- removed joint platform_joint
- removed joint scan_joint
- removed joint wheel_left_joint
- removed joint wheel_right_joint
