Commit message: Test without pose

File: CustomRobots/f1/urdf/f1.urdf (robot description, URDF)
Before this commit: robot f1, 1 links, 0 joints
Joints:
- added joint cam_f1_joint: type fixed, parent f1, child camera_link, origin xyz=0.45 0.04 0.1 rpy=0 0 0

Commit message: Test origin

File: CustomRobots/f1/urdf/f1.urdf (robot description, URDF)
Before this commit: robot f1, 1 links, 1 joints
Joints:
- removed joint cam_f1_joint
