Commit message: Test revolute limits

File: CustomRobots/f1/urdf/f1_ackermann_cam.urdf (robot description, URDF)
Before this commit: robot f1, 9 links, 8 joints
Joints:
- joint br_axle: limit (none) -> lower=-5 upper=5
- joint fl_axle: limit (none) -> lower=-5 upper=5
- joint fr_axle: limit (none) -> lower=-5 upper=5
- joint front_steering: limit (none) -> lower=-5 upper=5

Commit message: Check again

File: CustomRobots/f1/urdf/f1_ackermann_cam.urdf (robot description, URDF)
Before this commit: robot f1, 9 links, 8 joints
Joints:
- joint bl_axle: limit (none) -> lower=-5 upper=5

Commit message: Test again

File: CustomRobots/f1/urdf/f1_ackermann_cam.urdf (robot description, URDF)
Before this commit: robot f1, 9 links, 8 joints
Joints:
- joint bl_axle: limit lower=-5 upper=5 -> lower=-5 upper=5 effort=1000 velocity=100
- joint br_axle: limit lower=-5 upper=5 -> lower=-5 upper=5 effort=1000 velocity=100
- joint fl_axle: limit lower=-5 upper=5 -> lower=-5 upper=5 effort=1000 velocity=100
- joint fr_axle: limit lower=-5 upper=5 -> lower=-5 upper=5 effort=1000 velocity=100
- joint front_steering: limit lower=-5 upper=5 -> lower=-5 upper=5 effort=1000 velocity=100
- joint steering_joint: limit lower=-5 upper=5 -> lower=-5 upper=5 effort=1000 velocity=100

Commit message: Test again

File: CustomRobots/f1/urdf/f1_ackermann_cam.urdf (robot description, URDF)
Before this commit: robot f1, 9 links, 8 joints
Links:
- link chassis_link: geometry collision mesh filename=file:///home/ws/install/custom_robots/share/custom_robots/m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 scale=5 5 5; visual mesh filename=file:///home/ws/install/custom_robots/share/custom_robots/m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 scale=1 1 1

Commit message: Test scale

File: CustomRobots/f1/urdf/f1_ackermann_cam.urdf (robot description, URDF)
Before this commit: robot f1, 9 links, 8 joints
Links:
- link chassis_link: geometry collision mesh filename=file:///home/ws/install/custom_robots/share/custom_robots/m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 scale=5 5 5; visual mesh filename=file:///home/ws/install/custom_robots/share/custom_robots/m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 scale=5 5 5

Commit message: Change scale

File: CustomRobots/f1/urdf/f1_ackermann_cam.urdf (robot description, URDF)
Before this commit: robot f1, 9 links, 8 joints
Links:
- link bl_1: geometry collision cylinder length=0.22 radius=0.3425; visual mesh filename=file:///home/ws/install/custom_robots/share/custom_robots/m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 scale=0.02 0.02 0.02

Commit message: Add rotation

File: CustomRobots/f1/urdf/f1_ackermann_cam.urdf (robot description, URDF)
Before this commit: robot f1, 9 links, 8 joints
Joints:
- joint bl_axle: origin xyz=-0.775 -1.83364 0.324997 rpy=0 -0 0 -> xyz=-0.775 -1.83364 0.324997 rpy=-1.5708 0 0
- joint br_axle: origin xyz=0.775 -1.83364 0.324997 rpy=0 -0 0 -> xyz=0.775 -1.83364 0.324997 rpy=-1.5708 0 0

Commit message: Add scale

File: CustomRobots/f1/urdf/f1_ackermann_cam.urdf (robot description, URDF)
Before this commit: robot f1, 9 links, 8 joints
Links:
- link br_1: geometry collision cylinder length=0.22 radius=0.3425; visual mesh filename=file:///home/ws/install/custom_robots/share/custom_robots/m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 scale=0.02 0.02 0.02

Commit message: Change distances

File: CustomRobots/f1/urdf/f1_ackermann_cam.urdf (robot description, URDF)
Before this commit: robot f1, 9 links, 8 joints
Joints:
- joint bl_axle: origin xyz=-0.775 -1.83364 0.324997 rpy=-1.5708 0 0 -> xyz=-0.155 -0.366728 0.0649994 rpy=0 -1.5708 0

Commit message: Change wheel pose

File: CustomRobots/f1/urdf/f1_ackermann_cam.urdf (robot description, URDF)
Before this commit: robot f1, 9 links, 8 joints
Joints:
- joint bl_axle: origin xyz=-0.155 -0.366728 0.0649994 rpy=0 -1.5708 0 -> xyz=-0.155 -0.366728 0.0649994 rpy=0 0 -1.5708
- joint br_axle: origin xyz=0.775 -1.83364 0.324997 rpy=-1.5708 0 0 -> xyz=-0.155 -0.366728 0.0649994 rpy=0 0 -1.5708

Commit message: Fix urdf

File: CustomRobots/f1/urdf/f1_ackermann_cam.urdf (robot description, URDF)
Before this commit: robot f1, 8 links, 7 joints
Links:
- link bl_1: geometry collision cylinder length=0.0685 radius=0.066; visual mesh filename=file:///home/ws/install/custom_robots/share/custom_robots/m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 scale=0.02 0.02 0.02
- link br_1: geometry collision cylinder length=0.0685 radius=0.066; visual mesh filename=file:///home/ws/install/custom_robots/share/custom_robots/m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 scale=0.02 0.02 0.02
- link chassis_link: geometry collision mesh filename=file:///home/ws/install/custom_robots/share/custom_robots/m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 scale=1 1 1; visual mesh filename=file:///home/ws/install/custom_robots/share/custom_robots/m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 scale=1 1 1
- link fl_1: geometry collision cylinder length=0.0685 radius=0.066; visual mesh filename=file:///home/ws/install/custom_robots/share/custom_robots/m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 scale=0.02 0.02 0.02
- link fr_1: geometry collision cylinder length=0.0685 radius=0.066; visual mesh filename=file:///home/ws/install/custom_robots/share/custom_robots/m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 scale=0.02 0.02 0.02
- link front_steering_link: geometry 
Joints:
- joint bl_axle: origin xyz=-0.465 0.095 0 rpy=0 -1.5708 0 -> xyz=-0.155 -0.366728 0.0649994 rpy=0 0 0
- joint br_axle: origin xyz=-0.465 0.095 0 rpy=0 -1.5708 0 -> xyz=0.155 -0.366728 0.0649994 rpy=0 0 0
- joint cam_f1_left_to_base: origin xyz=0.09 0.04 0.1 rpy=0 0 0 -> xyz=0 0.0276 0.04 rpy=0 0 1.57
- joint chassis_link_joint: origin xyz=0.0 0.0 0.0 rpy=1.5708 0 0 -> xyz=0.0 0.0 0.0 rpy=0 0 -1.5708
- joint front_steering: origin xyz=0.0015 0.065 0 rpy=0 -1.5708 0 -> xyz=0 0.303472 0.0649994 rpy=0 0 0

Commit message: Move camera pose

File: CustomRobots/f1/urdf/f1_ackermann_cam.urdf (robot description, URDF)
Before this commit: robot f1, 8 links, 7 joints
Joints:
- joint cam_f1_left_to_base: origin xyz=0 0.0276 0.04 rpy=0 0 1.57 -> xyz=0.45 0.04 0.1 rpy=0 0 0
