Commit message: Update car models

File: CustomRobots/f1/urdf/f1_ackermann_laser.urdf (robot description, URDF)
Before this commit: robot f1, 9 links, 8 joints
Links:
- removed link steering_wheel
- link bl_1: geometry collision cylinder length=0.0685 radius=0.066; visual mesh filename=file:///home/ws/install/custom_robots/share/custom_robots/m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 scale=0.02 0.02 0.02
- link br_1: geometry collision cylinder length=0.0685 radius=0.066; visual mesh filename=file:///home/ws/install/custom_robots/share/custom_robots/m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 scale=0.02 0.02 0.02
- link chassis_link: geometry collision mesh filename=file:///home/ws/install/custom_robots/share/custom_robots/m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 scale=1 1 1; visual mesh filename=file:///home/ws/install/custom_robots/share/custom_robots/m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 scale=1 1 1
- link fl_1: geometry collision cylinder length=0.0685 radius=0.066; visual mesh filename=file:///home/ws/install/custom_robots/share/custom_robots/m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 scale=0.02 0.02 0.02
- link fr_1: geometry collision cylinder length=0.0685 radius=0.066; visual mesh filename=file:///home/ws/install/custom_robots/share/custom_robots/m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 scale=0.02 0.02 0.02
Joints:
- removed joint steering_joint
- joint bl_axle: axis -1 0 0 -> 1 0 0; limit (none) -> lower=-5 upper=5 effort=1000 velocity=100; origin xyz=-0.775 -1.83364 0.324997 rpy=0 -0 0 -> xyz=-0.155 -0.366728 0.0649994 rpy=0 0 0
- joint br_axle: limit (none) -> lower=-5 upper=5 effort=1000 velocity=100; origin xyz=0.775 -1.83364 0.324997 rpy=0 -0 0 -> xyz=0.155 -0.366728 0.0649994 rpy=0 0 0
- joint chassis_link_joint: origin xyz=0.0 0.0 0.0 rpy=0 0 0 -> xyz=0.0 0.0 0.0 rpy=0 0 -1.5708
- joint fl_axle: limit (none) -> lower=-5 upper=5 effort=1000 velocity=100; origin xyz=-0.05 0 0 rpy=0 -0 0 -> xyz=-0.165 0 0 rpy=0 -0 0
- joint fr_axle: limit (none) -> lower=-5 upper=5 effort=1000 velocity=100; origin xyz=0.825 0 0 rpy=0 -0 0 -> xyz=0.165 0 0 rpy=0 -0 0
- joint front_steering: limit (none) -> lower=-5 upper=5 effort=1000 velocity=100; origin xyz=0 1.51736 0.324997 rpy=0 -0 0 -> xyz=0 0.303472 0.0649994 rpy=0 0 0
