Commit message: Update urdf

File: CustomRobots/f1/models/f1/f1.urdf.xacro (robot description, xacro)
@@ -11,5 +11,5 @@
     <visual name="car">
       <geometry>
-        <mesh filename="package://f1/models/f1/meshes/Car.obj" scale="0.2 0.2 0.2"/>
+        <mesh filename="file://$(find custom_robots)/models/f1/meshes/Car.obj" scale="0.2 0.2 0.2"/>
       </geometry>
     </visual>

File: CustomRobots/f1/models/f1/f1_gz.urdf.xacro (robot description, xacro)
@@ -11,5 +11,5 @@
       </geometry>
     </visual>
-    <gazebo reference="camera_link">
+    <gz reference="camera_link">
       <sensor name="${name}" type="camera">
         <pose>${xyzrpy}</pose>
@@ -37,15 +37,15 @@
         </camera>
       </sensor>
-    </gazebo>
+    </gz>
   </xacro:macro>
   <xacro:macro name="f1_velocity" params="topic">
-    <gazebo>
+    <gz>
       <plugin filename="gz-sim-velocity-control-system" name="gz::sim::systems::VelocityControl">
         <topic>${topic}</topic>
       </plugin>
-    </gazebo>
+    </gz>
   </xacro:macro>
   <xacro:macro name="f1_odom" params="topic">
-    <gazebo>
+    <gz>
       <plugin filename="gz-sim-odometry-publisher-system" name="gz::sim::systems::OdometryPublisher">
         <odom_frame>odom</odom_frame>
@@ -55,5 +55,5 @@
         <dimensions>3</dimensions>
       </plugin>
-    </gazebo>
+    </gz>
   </xacro:macro>
 </robot>

File: CustomRobots/f1/urdf/f1.urdf (robot description, URDF)
Before this commit: robot f1, 1 links, 0 joints
Links:
- link f1: geometry visual mesh filename=file://$(find custom_robots)/models/f1/meshes/Car.obj scale=0.2 0.2 0.2

Commit message: Add collision

File: CustomRobots/f1/models/f1/f1.urdf.xacro (robot description, xacro)
@@ -9,4 +9,9 @@
       <inertia ixx="1" ixy="0.0" ixz="0.0" iyy="1" iyz="0.0" izz="1.0"/>
     </inertial>
+    <collision>
+      <geometry>
+        <mesh filename="file://$(find custom_robots)/models/f1/meshes/Car.obj" scale="0.2 0.2 0.2"/>
+      </geometry>
+    </collision>
     <visual name="car">
       <geometry>

File: CustomRobots/f1/urdf/f1.urdf (robot description, URDF)
Before this commit: robot f1, 1 links, 0 joints
Links:
- link f1: geometry collision mesh filename=file://$(find custom_robots)/models/f1/meshes/Car.obj scale=0.2 0.2 0.2; visual mesh filename=file://$(find custom_robots)/models/f1/meshes/Car.obj scale=0.2 0.2 0.2

Commit message: Update urdf

File: CustomRobots/f1/models/f1/f1.urdf.xacro (robot description, xacro)
@@ -3,5 +3,5 @@
   xmlns:xacro="http://ros.org/wiki/xacro">
   <xacro:include filename="$(find custom_robots)/models/f1/f1_gz.urdf.xacro"/>
-  <link name="f1">
+  <link name="base">
     <origin rpy="0 0 0" xyz="0 0 0"/>
     <inertial>
@@ -20,5 +20,5 @@
     </visual>
   </link>
-  <xacro:f1_camera xyzrpy="0.45 0.04 0.1 0 0 0" name="cam_f1_left"/>
+  <xacro:f1_camera xyz="0.45 0.04 0.1" rpy="0 0 0" name="cam_f1_left" parent="base"/>
   <xacro:f1_velocity topic="/F1ROS/cmd_vel"/>
   <xacro:f1_odom topic="/F1ROS/odom"/>

File: CustomRobots/f1/models/f1/f1_gz.urdf.xacro (robot description, xacro)
@@ -2,16 +2,19 @@
 <robot name="f1_gz"
   xmlns:xacro="http://ros.org/wiki/xacro">
-  <xacro:macro name="f1_camera" params="xyzrpy name">
-    <visual name='${name}_pose'>
-      <pose>${xyzrpy}</pose>
-      <geometry>
-        <sphere>
-          <radius>.005</radius>
-        </sphere>
-      </geometry>
-    </visual>
-    <gz reference="camera_link">
+  <xacro:macro name="f1_camera" params="xyz rpy name parent">
+    <link name="${name}_link">
+      <visual>
+        <geometry>
+          <sphere radius="0.005"/>
+        </geometry>
+      </visual>
+    </link>
+    <joint name="${name}_to_${parent}" type="fixed">
+      <parent link="${parent}"/>
+      <child link="${name}_link"/>
+      <origin xyz="${xyz}" rpy="${rpy}"/>
+    </joint>
+    <gazebo reference="${name}_link">
       <sensor name="${name}" type="camera">
-        <pose>${xyzrpy}</pose>
         <always_on>true</always_on>
         <visualize>true</visualize>
@@ -37,15 +40,15 @@
         </camera>
       </sensor>
-    </gz>
+    </gazebo>
   </xacro:macro>
   <xacro:macro name="f1_velocity" params="topic">
-    <gz>
+    <gazebo>
       <plugin filename="gz-sim-velocity-control-system" name="gz::sim::systems::VelocityControl">
         <topic>${topic}</topic>
       </plugin>
-    </gz>
+    </gazebo>
   </xacro:macro>
   <xacro:macro name="f1_odom" params="topic">
-    <gz>
+    <gazebo>
       <plugin filename="gz-sim-odometry-publisher-system" name="gz::sim::systems::OdometryPublisher">
         <odom_frame>odom</odom_frame>
@@ -55,5 +58,5 @@
         <dimensions>3</dimensions>
       </plugin>
-    </gz>
+    </gazebo>
   </xacro:macro>
 </robot>

File: CustomRobots/f1/urdf/f1.urdf (robot description, URDF)
Before this commit: robot f1, 1 links, 0 joints
Links:
- removed link f1
- added link base, mass 10; collision mesh filename=file://$(find custom_robots)/models/f1/meshes/Car.obj scale=0.2 0.2 0.2; visual mesh filename=file://$(find custom_robots)/models/f1/meshes/Car.obj scale=0.2 0.2 0.2
- added link camera_link; visual sphere radius=0.005
Joints:
- added joint lidar_to_base: type fixed, parent base, child camera_link, origin xyz=0.45 0.04 0.1 rpy=0 0 0

Commit message: Start with base ackermann

File: CustomRobots/f1/models/f1/f1.urdf.xacro (robot description, xacro)
@@ -22,5 +22,164 @@
     </link>
     <xacro:f1_velocity topic="/F1ROS/cmd_vel"/>
-    <xacro:f1_odom topic="/F1ROS/odom"/>
+    <xacro:f1_odom topic="/F1ROS/odom" freq="50"/>
+  </xacro:macro>
+  <xacro:macro name="ackermann">
+    <link name="base_link"/>
+    <joint name="chassis_link_joint" type="fixed">
+      <origin rpy="0 0 0" xyz="0.0 0.0 0.0"/>
+      <parent link="base_link"/>
+      <child link="chassis_link"/>
+    </joint>
+    <link name="chassis_link">
+      <inertial>
+        <origin rpy="0 -0 0" xyz="1e-06 0.07307 0.65096"/>
+        <mass value="1580"/>
+        <inertia ixx="1997.86" ixy="-3e-05" ixz="-1e-06" iyy="442.769" iyz="62.5206" izz="2238.05"/>
+      </inertial>
+      <visual>
+        <origin rpy="0 -0 1.5708" xyz="0 1.51 0"/>
+        <geometry>
+          <mesh filename="package://ackermann_cars/models/f1_renault_ackermann/Renault/chasis.dae" scale="5 5 5"/>
+        </geometry>
+      </visual>
+    </link>
+    <joint name="bl_axle" type="revolute">
+      <origin rpy="0 -0 0" xyz="-0.775 -1.83364 0.324997"/>
+      <parent link="chassis_link"/>
+      <child link="bl_1"/>
+      <axis xyz="-1 0 0"/>
+      <dynamics friction="12.031606150200002"/>
+    </joint>
+    <link name="bl_1">
+      <origin rpy="0 -0 0" xyz="0 0 0"/>
+      <inertial>
+        <origin rpy="0 -0 0" xyz="-0.0377 0 -0"/>
+        <mass value="24.5"/>
+        <inertia ixx="1.84514" ixy="0" ixz="0" iyy="1.04961" iyz="0" izz="1.04961"/>
+      </inertial>
+      <visual>
+        <origin rpy="0 -0 0" xyz="0.875 1.0136 0.1444"/>
+        <geometry>
+          <mesh filename="package://ackermann_cars/models/f1_renault_ackermann/Renault/back_left.dae" scale="0.1 0.1 0.1"/>
+        </geometry>
+      </visual>
+    </link>
+    <joint name="br_axle" type="revolute">
+      <origin rpy="0 -0 0" xyz="0.775 -1.83364 0.324997"/>
+      <parent link="chassis_link"/>
+      <child link="br_1"/>
+      <axis xyz="-1 0 0"/>
+      <dynamics friction="12.031606150200002"/>
+    </joint>
+    <link name="br_1">
+      <origin rpy="0 -0 0" xyz="0 0 0"/>
+      <inertial>
+        <origin rpy="0 -0 0" xyz="-0.0377 0 -0"/>
+        <mass value="24.5"/>
+        <inertia ixx="1.84514" ixy="0" ixz="0" iyy="1.04961" iyz="0" izz="1.04961"/>
+      </inertial>
+      <visual>
+        <origin rpy="0 -0 0" xyz="-0.875 1.0136 0.1444"/>
+        <geometry>
+          <mesh filename="package://ackermann_cars/models/f1_renault_ackermann/Renault/back_right.dae" scale="0.1 0.1 0.1"/>
+        </geometry>
+      </visual>
+    </link>
+    <joint name="l_steer" type="revolute">
+      <origin rpy="0 -0 0" xyz="-0.825 1.51736 0.324997"/>
+      <parent link="chassis_link"/>
+      <child link="l_steer_1"/>
+      <axis xyz="0 0 1"/>
+      <limit lower="-0.95" upper="0.95"/>
+      <dynamics friction="18.0474092253"/>
+    </joint>
+    <link name="l_steer_1">
+      <origin rpy="0 -0 0" xyz="0 0 0"/>
+      <inertial>
+        <origin rpy="0 -0 0" xyz="0.003381 0 0.02162"/>
+        <mass value="1"/>
+        <inertia ixx="1" ixy="0" ixz="0" iyy="1" iyz="0" izz="1"/>
+      </inertial>
+    </link>
+    <joint name="fl_axle" type="revolute">
+      <origin rpy="0 -0 0" xyz="-0.05 0 0"/>
+      <parent link="l_steer_1"/>
+      <child link="fl_1"/>
+      <axis xyz="-1 0 0"/>
+      <dynamics friction="12.031606150200002"/>
+    </joint>
+    <link name="fl_1">
+      <origin rpy="0 -0 0" xyz="0 0 0"/>
+      <inertial>
+        <origin rpy="0 -0 0" xyz="-0.0377 0 -0"/>
+        <mass value="24.5"/>
+        <inertia ixx="1.84514" ixy="0" ixz="0" iyy="1.04961" iyz="0" izz="1.04961"/>
+      </inertial>
+      <visual>
+        <origin rpy="0 -0 0" xyz="0.875 -1.5174 0.1444"/>
+        <geometry>
+          <mesh filename="package://ackermann_cars/models/f1_renault_ackermann/Renault/front_left.dae" scale="0.1 0.1 0.1"/>
+        </geometry>
+      </visual>
+    </link>
+    <joint name="r_steer" type="revolute">
+      <origin rpy="0 -0 0" xyz="0.825 1.51736 0.324997"/>
+      <parent link="chassis_link"/>
+      <child link="r_steer_1"/>
+      <axis xyz="0 0 1"/>
+      <limit lower="-0.95" upper="0.95"/>
+      <dynamics damping="0.01" friction="18.0474092253"/>
+    </joint>
+    <link name="r_steer_1">
+      <origin rpy="0 -0 0" xyz="0 0 0"/>
+      <inertial>
+        <origin rpy="0 -0 0" xyz="0.003381 0 0.02162"/>
+        <mass value="1"/>
+        <inertia ixx="1" ixy="0" ixz="0" iyy="1" iyz="0" izz="1"/>
+      </inertial>
+    </link>
+    <joint name="fr_axle" type="revolute">
+      <origin rpy="0 -0 0" xyz="0.05 0 0"/>
+      <parent link="r_steer_1"/>
+      <child link="fr_1"/>
+      <axis xyz="-1 0 0"/>
+      <dynamics friction="12.031606150200002"/>
+    </joint>
+    <link name="fr_1">
+      <origin rpy="0 -0 0" xyz="0 0 0"/>
+      <inertial>
+        <origin rpy="0 -0 0" xyz="-0.0377 0 -0"/>
+        <mass value="24.5"/>
+        <inertia ixx="1.84514" ixy="0" ixz="0" iyy="1.04961" iyz="0" izz="1.04961"/>
+      </inertial>
+      <visual>
+        <origin rpy="0 -0 0" xyz="-0.875 -1.5174 0.1444"/>
+        <geometry>
+          <mesh filename="package://ackermann_cars/models/f1_renault_ackermann/Renault/front_right.dae" scale="0.1 0.1 0.1"/>
+        </geometry>
+      </visual>
+    </link>
+    <joint name="steering_joint" type="revolute">
+      <origin rpy="0 0 0" xyz="-0.01 0.6 0.6"/>
+      <parent link="chassis_link"/>
+      <child link="steering_wheel"/>
+      <axis xyz="0.0 -1.0 0.0"/>
+      <limit lower="-100" upper="100"/>
+      <dynamics damping="10.0"/>
+    </joint>
+    <link name="steering_wheel">
+      <origin rpy="0 0 1.5708" xyz="0 0.87 -0.54"/>
+      <visual>
+        <origin rpy="0 0 0" xyz="0 0 0"/>
+        <geometry>
+          <mesh filename="package://ackermann_cars/models/f1_renault_ackermann/Renault/steering_wheel.dae" scale="4.7 4.7 4.7"/>
+        </geometry>
+      </visual>
+    </link>
+    <xacro:f1_ackermann_steering topic="/model/f1_renault_ackermann_harmonic"/>
+    <xacro:f1_joints/>
+    <xacro:f1_odom topic="/model/f1_renault_ackermann_harmonic/odom" freq="50"/>
+    <xacro:f1_pose freq="50"/>
+    <xacro:f1_steer_controller topic="/model/f1_renault_ackermann_harmonic/steering_wheel_cmd" joint="steering_joint"/>
   </xacro:macro>
 </robot>

File: CustomRobots/f1/models/f1/f1_gz.urdf.xacro (robot description, xacro)
@@ -87,10 +87,33 @@
     </gazebo>
   </xacro:macro>
-  <xacro:macro name="f1_odom" params="topic">
+  <xacro:macro name="f1_ackermann_steering" params="topic">
+    <gazebo>
+      <plugin filename="gz-sim-ackermann-steering-system" name="gz::sim::systems::AckermannSteering">
+        <left_joint>fl_axle</left_joint>
+        <left_joint>bl_axle</left_joint>
+        <right_joint>fr_axle</right_joint>
+        <right_joint>br_axle</right_joint>
+        <left_steering_joint>front_steering</left_steering_joint>
+        <right_steering_joint>front_steering</right_steering_joint>
+        <kingpin_width>1.65</kingpin_width>
+        <steering_limit>0.3</steering_limit>
+        <wheel_base>3.351</wheel_base>
+        <wheel_separation>1.65</wheel_separation>
+        <wheel_radius>0.3425</wheel_radius>
+        <sub_topic>${topic}/steer_angle</sub_topic>
+        <min_velocity>-50</min_velocity>
+        <max_velocity>50</max_velocity>
+        <min_acceleration>-50</min_acceleration>
+        <max_acceleration>50</max_acceleration>
+        <topic>${topic}/cmd_vel</topic>
+      </plugin>
+    </gazebo>
+  </xacro:macro>
+  <xacro:macro name="f1_odom" params="topic freq">
     <gazebo>
       <plugin filename="gz-sim-odometry-publisher-system" name="gz::sim::systems::OdometryPublisher">
         <odom_frame>odom</odom_frame>
-        <robot_base_frame>xf1</robot_base_frame>
-        <odom_publish_frequency>20.0</odom_publish_frequency>
+        <robot_base_frame>chassis_link</robot_base_frame>
+        <odom_publish_frequency>${freq}</odom_publish_frequency>
         <odom_topic>${topic}</odom_topic>
         <dimensions>3</dimensions>
@@ -98,3 +121,37 @@
     </gazebo>
   </xacro:macro>
+  <xacro:macro name="f1_pose" params="freq">
+    <gazebo>
+      <plugin filename="gz-sim-pose-publisher-system" name="gz::sim::systems::PosePublisher">
+        <publish_link_pose>true</publish_link_pose>
+        <publish_collision_pose>false</publish_collision_pose>
+        <publish_visual_pose>false</publish_visual_pose>
+        <publish_nested_model_pose>true</publish_nested_model_pose>
+        <update_frequency>${freq}</update_frequency>
+      </plugin>
+    </gazebo>
+  </xacro:macro>
+  <xacro:macro name="f1_joints">
+    <gazebo>
+      <plugin filename="gz-sim-joint-state-publisher-system" name="gz::sim::systems::JointStatePublisher">
+        <joint_name>fl_axle</joint_name>
+        <joint_name>fr_axle</joint_name>
+        <joint_name>bl_axle</joint_name>
+        <joint_name>br_axle</joint_name>
+        <joint_name>front_steering</joint_name>
+        <joint_name>steering_joint</joint_name>
+      </plugin>
+    </gazebo>
+  </xacro:macro>
+  <xacro:macro name="f1_steer_controller" params="topic joint">
+    <gazebo>
+      <plugin filename="gz-sim-joint-position-controller-system" name="gz::sim::systems::JointPositionController">
+        <joint_name>${joint}</joint_name>
+        <sub_topic>${topic}</sub_topic>
+        <p_gain>10</p_gain>
+        <i_gain>0.1</i_gain>
+        <d_gain>1</d_gain>
+      </plugin>
+    </gazebo>
+  </xacro:macro>
 </robot>

Commit message: Add ackermann urdf

File: CustomRobots/f1/models/f1/f1.urdf.xacro (robot description, xacro)
@@ -25,20 +25,26 @@
   </xacro:macro>
   <xacro:macro name="ackermann">
-    <link name="base_link"/>
+    <link name="base"/>
     <joint name="chassis_link_joint" type="fixed">
       <origin rpy="0 0 0" xyz="0.0 0.0 0.0"/>
-      <parent link="base_link"/>
+      <parent link="base"/>
       <child link="chassis_link"/>
     </joint>
     <link name="chassis_link">
       <inertial>
-        <origin rpy="0 -0 0" xyz="1e-06 0.07307 0.65096"/>
+        <origin rpy="0 0 0" xyz="0 0.07307 0.65096"/>
         <mass value="1580"/>
         <inertia ixx="1997.86" ixy="-3e-05" ixz="-1e-06" iyy="442.769" iyz="62.5206" izz="2238.05"/>
       </inertial>
+      <collision>
+        <origin rpy="0 1.51 0" xyz="1.5708 0 1.5708"/>
+        <geometry>
+          <mesh filename="file://$(find custom_robots)/models/f1/meshes/chasis.obj" scale="5 5 5"/>
+        </geometry>
+      </collision>
       <visual>
-        <origin rpy="0 -0 1.5708" xyz="0 1.51 0"/>
+        <origin rpy="0 1.51 0" xyz="1.5708 0 1.5708"/>
         <geometry>
-          <mesh filename="package://ackermann_cars/models/f1_renault_ackermann/Renault/chasis.dae" scale="5 5 5"/>
+          <mesh filename="file://$(find custom_robots)/models/f1/meshes/chasis.obj" scale="5 5 5"/>
         </geometry>
       </visual>
@@ -58,8 +64,14 @@
         <inertia ixx="1.84514" ixy="0" ixz="0" iyy="1.04961" iyz="0" izz="1.04961"/>
       </inertial>
+      <collision>
+        <origin rpy="0 1.5708 0" xyz="0 0 0"/>
+        <geometry>
+          <cylinder radius="0.3425" length="0.22"/>
+        </geometry>
+      </collision>
       <visual>
-        <origin rpy="0 -0 0" xyz="0.875 1.0136 0.1444"/>
+        <origin rpy="0 0 0" xyz="0.875  0.14 -1.0126"/>
         <geometry>
-          <mesh filename="package://ackermann_cars/models/f1_renault_ackermann/Renault/back_left.dae" scale="0.1 0.1 0.1"/>
+          <mesh filename="file://$(find custom_robots)/models/f1/meshes/back_left.obj" scale="0.1 0.1 0.1"/>
         </geometry>
       </visual>
@@ -79,30 +91,35 @@
         <inertia ixx="1.84514" ixy="0" ixz="0" iyy="1.04961" iyz="0" izz="1.04961"/>
       </inertial>
+      <collision>
+        <origin rpy="0 1.5708 0" xyz="0 0 0"/>
+        <geometry>
+          <cylinder radius="0.3425" length="0.22"/>
+        </geometry>
+      </collision>
       <visual>
-        <origin rpy="0 -0 0" xyz="-0.875 1.0136 0.1444"/>
+        <origin rpy="0 0 0" xyz="-0.875  0.14 -1.0126"/>
         <geometry>
-          <mesh filename="package://ackermann_cars/models/f1_renault_ackermann/Renault/back_right.dae" scale="0.1 0.1 0.1"/>
+          <mesh filename="file://$(find custom_robots)/models/f1/meshes/back_right.obj" scale="0.1 0.1 0.1"/>
         </geometry>
       </visual>
     </link>
-    <joint name="l_steer" type="revolute">
-      <origin rpy="0 -0 0" xyz="-0.825 1.51736 0.324997"/>
+    <joint name="front_steering" type="revolute">
+      <origin rpy="0 -0 0" xyz="0 1.51736 0.324997"/>
       <parent link="chassis_link"/>
-      <child link="l_steer_1"/>
+      <child link="front_steering_link"/>
       <axis xyz="0 0 1"/>
-      <limit lower="-0.95" upper="0.95"/>
-      <dynamics friction="18.0474092253"/>
+      <dynamics friction="0.5"/>
     </joint>
-    <link name="l_steer_1">
+    <link name="front_steering_link">
       <origin rpy="0 -0 0" xyz="0 0 0"/>
       <inertial>
-        <origin rpy="0 -0 0" xyz="0.003381 0 0.02162"/>
-        <mass value="1"/>
-        <inertia ixx="1" ixy="0" ixz="0" iyy="1" iyz="0" izz="1"/>
+        <origin rpy="0 0 0" xyz="0 0 0"/>
+        <mass value="2"/>
+        <inertia ixx="0.01" ixy="0" ixz="0" iyy="0.01" iyz="0" izz="0.01"/>
       </inertial>
     </link>
     <joint name="fl_axle" type="revolute">
       <origin rpy="0 -0 0" xyz="-0.05 0 0"/>
-      <parent link="l_steer_1"/>
+      <parent link="front_steering_link"/>
       <child link="fl_1"/>
       <axis xyz="-1 0 0"/>
@@ -116,30 +133,20 @@
         <inertia ixx="1.84514" ixy="0" ixz="0" iyy="1.04961" iyz="0" izz="1.04961"/>
       </inertial>
+      <collision>
+        <origin rpy="0 0 0" xyz="0.875 -1.5174 0.1444"/>
+        <geometry>
+          <mesh filename="file://$(find custom_robots)/models/f1/meshes/fl_1.stl" scale="0.001 0.001 0.001"/>
+        </geometry>
+      </collision>
       <visual>
-        <origin rpy="0 -0 0" xyz="0.875 -1.5174 0.1444"/>
+        <origin rpy="0 0 0" xyz="0.875  0.1444 -1.5174"/>
         <geometry>
-          <mesh filename="package://ackermann_cars/models/f1_renault_ackermann/Renault/front_left.dae" scale="0.1 0.1 0.1"/>
+          <mesh filename="file://$(find custom_robots)/models/f1/meshes/front_left.obj" scale="0.1 0.1 0.1"/>
         </geometry>
       </visual>
     </link>
-    <joint name="r_steer" type="revolute">
-      <origin rpy="0 -0 0" xyz="0.825 1.51736 0.324997"/>
-      <parent link="chassis_link"/>
-      <child link="r_steer_1"/>
-      <axis xyz="0 0 1"/>
-      <limit lower="-0.95" upper="0.95"/>
-      <dynamics damping="0.01" friction="18.0474092253"/>
-    </joint>
-    <link name="r_steer_1">
-      <origin rpy="0 -0 0" xyz="0 0 0"/>
-      <inertial>
-        <origin rpy="0 -0 0" xyz="0.003381 0 0.02162"/>
-        <mass value="1"/>
-        <inertia ixx="1" ixy="0" ixz="0" iyy="1" iyz="0" izz="1"/>
-      </inertial>
-    </link>
     <joint name="fr_axle" type="revolute">
-      <origin rpy="0 -0 0" xyz="0.05 0 0"/>
-      <parent link="r_steer_1"/>
+      <origin rpy="0 -0 0" xyz="0.825 0 0"/>
+      <parent link="front_steering_link"/>
       <child link="fr_1"/>
       <axis xyz="-1 0 0"/>
@@ -147,14 +154,20 @@
     </joint>
     <link name="fr_1">
-      <origin rpy="0 -0 0" xyz="0 0 0"/>
+      <origin rpy="0 0 0" xyz="0 0 0"/>
       <inertial>
-        <origin rpy="0 -0 0" xyz="-0.0377 0 -0"/>
+        <origin rpy="0 0 0" xyz="-0.0377 0 0"/>
         <mass value="24.5"/>
         <inertia ixx="1.84514" ixy="0" ixz="0" iyy="1.04961" iyz="0" izz="1.04961"/>
       </inertial>
+      <collision>
+        <origin rpy="0 0 0" xyz="-0.875 -1.5174 0.1444"/>
+        <geometry>
+          <mesh filename="file://$(find custom_robots)/models/f1/meshes/fr_1.stl" scale="0.001 0.001 0.001"/>
+        </geometry>
+      </collision>
       <visual>
-        <origin rpy="0 -0 0" xyz="-0.875 -1.5174 0.1444"/>
+        <origin rpy="0 0 0" xyz="-0.875  0.1444 -1.5174"/>
         <geometry>
-          <mesh filename="package://ackermann_cars/models/f1_renault_ackermann/Renault/front_right.dae" scale="0.1 0.1 0.1"/>
+          <mesh filename="file://$(find custom_robots)/models/f1/meshes/front_right.obj" scale="0.1 0.1 0.1"/>
         </geometry>
       </visual>
@@ -165,5 +178,5 @@
       <child link="steering_wheel"/>
       <axis xyz="0.0 -1.0 0.0"/>
-      <limit lower="-100" upper="100"/>
+      <limit lower="-5" upper="5"/>
       <dynamics damping="10.0"/>
     </joint>
@@ -173,5 +186,5 @@
         <origin rpy="0 0 0" xyz="0 0 0"/>
         <geometry>
-          <mesh filename="package://ackermann_cars/models/f1_renault_ackermann/Renault/steering_wheel.dae" scale="4.7 4.7 4.7"/>
+          <mesh filename="file://$(find custom_robots)/models/f1/meshes/steering_wheel.dae" scale="4.7 4.7 4.7"/>
         </geometry>
       </visual>
