Commit message: Update models

File: CustomRobots/f1/models/f1/f1.urdf.xacro (robot description, xacro)
@@ -55,4 +55,5 @@
       <child link="bl_1"/>
       <axis xyz="-1 0 0"/>
+      <limit lower="-5" upper="5"/>
       <dynamics friction="12.031606150200002"/>
     </joint>
@@ -82,4 +83,5 @@
       <child link="br_1"/>
       <axis xyz="-1 0 0"/>
+      <limit lower="-5" upper="5"/>
       <dynamics friction="12.031606150200002"/>
     </joint>
@@ -124,4 +126,5 @@
       <child link="fl_1"/>
       <axis xyz="-1 0 0"/>
+      <limit lower="-5" upper="5"/>
       <dynamics friction="12.031606150200002"/>
     </joint>
@@ -151,4 +154,5 @@
       <child link="fr_1"/>
       <axis xyz="-1 0 0"/>
+      <limit lower="-5" upper="5"/>
       <dynamics friction="12.031606150200002"/>
     </joint>

File: CustomRobots/f1/urdf/f1_ackermann_cam.urdf (robot description, URDF)
Before this commit: robot f1, 9 links, 8 joints
Links:
- removed link steering_wheel
- link bl_1: geometry collision cylinder length=0.05 radius=0.066; visual mesh filename=file:///home/ws/install/custom_robots/share/custom_robots/m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 scale=0.02 0.02 0.02
- link br_1: geometry collision cylinder length=0.05 radius=0.066; visual mesh filename=file:///home/ws/install/custom_robots/share/custom_robots/m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 scale=0.02 0.02 0.02
- link fl_1: geometry collision cylinder length=0.05 radius=0.066; visual mesh filename=file:///home/ws/install/custom_robots/share/custom_robots/m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 scale=0.02 0.02 0.02
- link fr_1: geometry collision cylinder length=0.05 radius=0.066; visual mesh filename=file:///home/ws/install/custom_robots/share/custom_robots/m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 scale=0.02 0.02 0.02
- link front_steering_link: geometry visual cylinder length=0.3 radius=0.01
Joints:
- removed joint steering_joint
- joint bl_axle: axis -1 0 0 -> 1 0 0; origin xyz=-0.155 -0.366728 0.0649994 rpy=0 0 -1.5708 -> xyz=-0.465 0.095 0 rpy=0 -1.5708 0
- joint br_axle: origin xyz=-0.155 -0.366728 0.0649994 rpy=0 0 -1.5708 -> xyz=-0.465 0.095 0 rpy=0 -1.5708 0
- joint cam_f1_left_to_base: origin xyz=0.45 0.04 0.1 rpy=0 0 0 -> xyz=0.09 0.04 0.1 rpy=0 0 0
- joint chassis_link_joint: origin xyz=0.0 0.0 0.0 rpy=0 0 0 -> xyz=0.0 0.0 0.0 rpy=1.5708 0 0
- joint fl_axle: origin xyz=-0.05 0 0 rpy=0 -0 0 -> xyz=-0.165 0 0 rpy=0 -0 0
- joint fr_axle: origin xyz=0.825 0 0 rpy=0 -0 0 -> xyz=0.165 0 0 rpy=0 -0 0
- joint front_steering: origin xyz=0 1.51736 0.324997 rpy=0 -0 0 -> xyz=0.0015 0.065 0 rpy=0 -1.5708 0

Commit message: Update xacro

File: CustomRobots/f1/models/f1/f1.urdf.xacro (robot description, xacro)
@@ -27,5 +27,5 @@
     <link name="base"/>
     <joint name="chassis_link_joint" type="fixed">
-      <origin rpy="0 0 0" xyz="0.0 0.0 0.0"/>
+      <origin rpy="0 0 -1.5708" xyz="0.0 0.0 0.0"/>
       <parent link="base"/>
       <child link="chassis_link"/>
@@ -33,27 +33,27 @@
     <link name="chassis_link">
       <inertial>
-        <origin rpy="0 0 0" xyz="0 0.07307 0.65096"/>
+        <origin rpy="0 0 0" xyz="0 0.014614 0.130192"/>
         <mass value="1580"/>
         <inertia ixx="1997.86" ixy="-3e-05" ixz="-1e-06" iyy="442.769" iyz="62.5206" izz="2238.05"/>
       </inertial>
       <collision>
-        <origin rpy="0 1.51 0" xyz="1.5708 0 1.5708"/>
-        <geometry>
-          <mesh filename="file://$(find custom_robots)/models/f1/meshes/chasis.obj" scale="5 5 5"/>
-        </geometry>
-      </collision>
-      <visual>
-        <origin rpy="0 1.51 0" xyz="1.5708 0 1.5708"/>
-        <geometry>
-          <mesh filename="file://$(find custom_robots)/models/f1/meshes/chasis.obj" scale="5 5 5"/>
+        <origin rpy="1.5708 0 1.5708" xyz="0 0.302 0"/>
+        <geometry>
+          <mesh filename="file:///home/ws/install/custom_robots/share/custom_robots/models/f1/meshes/chasis.obj" scale="1 1 1"/>
+        </geometry>
+      </collision>
+      <visual>
+        <origin rpy="1.5708 0 1.5708" xyz="0 0.302 0"/>
+        <geometry>
+          <mesh filename="file:///home/ws/install/custom_robots/share/custom_robots/models/f1/meshes/chasis.obj" scale="1 1 1"/>
         </geometry>
       </visual>
     </link>
     <joint name="bl_axle" type="revolute">
-      <origin rpy="0 -0 0" xyz="-0.775 -1.83364 0.324997"/>
+      <origin rpy="0 0 0" xyz="-0.155 -0.366728 0.0649994"/>
       <parent link="chassis_link"/>
       <child link="bl_1"/>
-      <axis xyz="-1 0 0"/>
-      <limit lower="-5" upper="5"/>
+      <axis xyz="1 0 0"/>
+      <limit lower="-5" upper="5" effort="1000" velocity="100"/>
       <dynamics friction="12.031606150200002"/>
     </joint>
@@ -68,24 +68,24 @@
         <origin rpy="0 1.5708 0" xyz="0 0 0"/>
         <geometry>
-          <cylinder radius="0.3425" length="0.22"/>
-        </geometry>
-      </collision>
-      <visual>
-        <origin rpy="0 0 0" xyz="0.875  0.14 -1.0126"/>
-        <geometry>
-          <mesh filename="file://$(find custom_robots)/models/f1/meshes/back_left.obj" scale="0.1 0.1 0.1"/>
+          <cylinder length="0.0685" radius="0.066"/>
+        </geometry>
+      </collision>
+      <visual>
+        <origin rpy="0 0 0" xyz="0.175 0.028 -0.20252"/>
+        <geometry>
+          <mesh filename="file:///home/ws/install/custom_robots/share/custom_robots/models/f1/meshes/back_left.obj" scale="0.02 0.02 0.02"/>
         </geometry>
       </visual>
     </link>
     <joint name="br_axle" type="revolute">
-      <origin rpy="0 -0 0" xyz="0.775 -1.83364 0.324997"/>
+      <origin rpy="0 0 0" xyz="0.155 -0.366728 0.0649994"/>
       <parent link="chassis_link"/>
       <child link="br_1"/>
       <axis xyz="-1 0 0"/>
-      <limit lower="-5" upper="5"/>
+      <limit lower="-5" upper="5" effort="1000" velocity="100"/>
       <dynamics friction="12.031606150200002"/>
     </joint>
     <link name="br_1">
-      <origin rpy="0 -0 0" xyz="0 0 0"/>
+      <origin rpy="0 0 0" xyz="0 0 0"/>
       <inertial>
         <origin rpy="0 -0 0" xyz="-0.0377 0 -0"/>
@@ -96,19 +96,20 @@
         <origin rpy="0 1.5708 0" xyz="0 0 0"/>
         <geometry>
-          <cylinder radius="0.3425" length="0.22"/>
-        </geometry>
-      </collision>
-      <visual>
-        <origin rpy="0 0 0" xyz="-0.875  0.14 -1.0126"/>
-        <geometry>
-          <mesh filename="file://$(find custom_robots)/models/f1/meshes/back_right.obj" scale="0.1 0.1 0.1"/>
+          <cylinder length="0.0685" radius="0.066"/>
+        </geometry>
+      </collision>
+      <visual>
+        <origin rpy="0 0 0" xyz="-0.175 0.028 -0.20252"/>
+        <geometry>
+          <mesh filename="file:///home/ws/install/custom_robots/share/custom_robots/models/f1/meshes/back_right.obj" scale="0.02 0.02 0.02"/>
         </geometry>
       </visual>
     </link>
     <joint name="front_steering" type="revolute">
-      <origin rpy="0 -0 0" xyz="0 1.51736 0.324997"/>
+      <origin rpy="0 0 0" xyz="0 0.303472 0.0649994"/>
       <parent link="chassis_link"/>
       <child link="front_steering_link"/>
       <axis xyz="0 0 1"/>
+      <limit lower="-5" upper="5" effort="1000" velocity="100"/>
       <dynamics friction="0.5"/>
     </joint>
@@ -122,9 +123,9 @@
     </link>
     <joint name="fl_axle" type="revolute">
-      <origin rpy="0 -0 0" xyz="-0.05 0 0"/>
+      <origin rpy="0 -0 0" xyz="-0.165 0 0"/>
       <parent link="front_steering_link"/>
       <child link="fl_1"/>
       <axis xyz="-1 0 0"/>
-      <limit lower="-5" upper="5"/>
+      <limit lower="-5" upper="5" effort="1000" velocity="100"/>
       <dynamics friction="12.031606150200002"/>
     </joint>
@@ -137,22 +138,22 @@
       </inertial>
       <collision>
-        <origin rpy="0 0 0" xyz="0.875 -1.5174 0.1444"/>
-        <geometry>
-          <mesh filename="file://$(find custom_robots)/models/f1/meshes/fl_1.stl" scale="0.001 0.001 0.001"/>
-        </geometry>
-      </collision>
-      <visual>
-        <origin rpy="0 0 0" xyz="0.875  0.1444 -1.5174"/>
-        <geometry>
-          <mesh filename="file://$(find custom_robots)/models/f1/meshes/front_left.obj" scale="0.1 0.1 0.1"/>
+        <origin rpy="0 1.5708 0" xyz="0 0 0"/>
+        <geometry>
+          <cylinder length="0.0685" radius="0.066"/>
+        </geometry>
+      </collision>
+      <visual>
+        <origin rpy="0 0 0" xyz="0.175 0.02888 0.30348"/>
+        <geometry>
+          <mesh filename="file:///home/ws/install/custom_robots/share/custom_robots/models/f1/meshes/front_left.obj" scale="0.02 0.02 0.02"/>
         </geometry>
       </visual>
     </link>
     <joint name="fr_axle" type="revolute">
-      <origin rpy="0 -0 0" xyz="0.825 0 0"/>
+      <origin rpy="0 -0 0" xyz="0.165 0 0"/>
       <parent link="front_steering_link"/>
       <child link="fr_1"/>
       <axis xyz="-1 0 0"/>
-      <limit lower="-5" upper="5"/>
+      <limit lower="-5" upper="5" effort="1000" velocity="100"/>
       <dynamics friction="12.031606150200002"/>
     </joint>
@@ -165,17 +166,17 @@
       </inertial>
       <collision>
-        <origin rpy="0 0 0" xyz="-0.875 -1.5174 0.1444"/>
-        <geometry>
-          <mesh filename="file://$(find custom_robots)/models/f1/meshes/fr_1.stl" scale="0.001 0.001 0.001"/>
-        </geometry>
-      </collision>
-      <visual>
-        <origin rpy="0 0 0" xyz="-0.875  0.1444 -1.5174"/>
-        <geometry>
-          <mesh filename="file://$(find custom_robots)/models/f1/meshes/front_right.obj" scale="0.1 0.1 0.1"/>
-        </geometry>
-      </visual>
-    </link>
-    <joint name="steering_joint" type="revolute">
+        <origin rpy="0 1.5708 0" xyz="0 0 0"/>
+        <geometry>
+          <cylinder length="0.0685" radius="0.066"/>
+        </geometry>
+      </collision>
+      <visual>
+        <origin rpy="0 0 0" xyz="-0.175 0.02888 0.30348"/>
+        <geometry>
+          <mesh filename="file:///home/ws/install/custom_robots/share/custom_robots/models/f1/meshes/front_right.obj" scale="0.02 0.02 0.02"/>
+        </geometry>
+      </visual>
+    </link>
+    <!-- <joint name="steering_joint" type="revolute">
       <origin rpy="0 0 0" xyz="-0.01 0.6 0.6"/>
       <parent link="chassis_link"/>
@@ -193,10 +194,9 @@
         </geometry>
       </visual>
-    </link>
-    <xacro:f1_ackermann_steering topic="/model/f1_renault_ackermann_harmonic"/>
+    </link> -->
+    <xacro:f1_ackermann_steering topic="/F1ROS/cmd_vel"/>
     <xacro:f1_joints/>
-    <xacro:f1_odom topic="/model/f1_renault_ackermann_harmonic/odom" freq="50"/>
-    <xacro:f1_pose freq="50"/>
-    <xacro:f1_steer_controller topic="/model/f1_renault_ackermann_harmonic/steering_wheel_cmd" joint="steering_joint"/>
+    <xacro:f1_odom topic="/F1ROS/odom" freq="50"/>
+    <!-- <xacro:f1_steer_controller topic="/model/f1_renault_ackermann_harmonic/steering_wheel_cmd" joint="steering_joint"/> -->
   </xacro:macro>
 </robot>

File: CustomRobots/f1/models/f1/f1_gz.urdf.xacro (robot description, xacro)
@@ -101,10 +101,10 @@
         <wheel_separation>1.65</wheel_separation>
         <wheel_radius>0.3425</wheel_radius>
-        <sub_topic>${topic}/steer_angle</sub_topic>
+        <!-- <sub_topic>${topic}/steer_angle</sub_topic> -->
         <min_velocity>-50</min_velocity>
         <max_velocity>50</max_velocity>
         <min_acceleration>-50</min_acceleration>
         <max_acceleration>50</max_acceleration>
-        <topic>${topic}/cmd_vel</topic>
+        <topic>${topic}</topic>
       </plugin>
     </gazebo>
@@ -121,15 +121,4 @@
     </gazebo>
   </xacro:macro>
-  <xacro:macro name="f1_pose" params="freq">
-    <gazebo>
-      <plugin filename="gz-sim-pose-publisher-system" name="gz::sim::systems::PosePublisher">
-        <publish_link_pose>true</publish_link_pose>
-        <publish_collision_pose>false</publish_collision_pose>
-        <publish_visual_pose>false</publish_visual_pose>
-        <publish_nested_model_pose>true</publish_nested_model_pose>
-        <update_frequency>${freq}</update_frequency>
-      </plugin>
-    </gazebo>
-  </xacro:macro>
   <xacro:macro name="f1_joints">
     <gazebo>
@@ -140,5 +129,5 @@
         <joint_name>br_axle</joint_name>
         <joint_name>front_steering</joint_name>
-        <joint_name>steering_joint</joint_name>
+        <!-- <joint_name>steering_joint</joint_name> -->
       </plugin>
     </gazebo>

Commit message: Fix wheel joints

File: CustomRobots/f1/models/f1/f1.urdf.xacro (robot description, xacro)
@@ -50,10 +50,10 @@
       </visual>
     </link>
-    <joint name="bl_axle" type="revolute">
+    <joint name="bl_axle" type="continuous">
       <origin rpy="0 0 0" xyz="-0.155 -0.366728 0.0649994"/>
       <parent link="chassis_link"/>
       <child link="bl_1"/>
       <axis xyz="1 0 0"/>
-      <limit lower="-5" upper="5" effort="1000" velocity="100"/>
+      <limit effort="1000" velocity="100"/>
       <dynamics friction="12.031606150200002"/>
     </joint>
@@ -78,10 +78,10 @@
       </visual>
     </link>
-    <joint name="br_axle" type="revolute">
+    <joint name="br_axle" type="continuous">
       <origin rpy="0 0 0" xyz="0.155 -0.366728 0.0649994"/>
       <parent link="chassis_link"/>
       <child link="br_1"/>
       <axis xyz="-1 0 0"/>
-      <limit lower="-5" upper="5" effort="1000" velocity="100"/>
+      <limit effort="1000" velocity="100"/>
       <dynamics friction="12.031606150200002"/>
     </joint>
@@ -122,10 +122,10 @@
       </inertial>
     </link>
-    <joint name="fl_axle" type="revolute">
+    <joint name="fl_axle" type="continuous">
       <origin rpy="0 -0 0" xyz="-0.165 0 0"/>
       <parent link="front_steering_link"/>
       <child link="fl_1"/>
       <axis xyz="-1 0 0"/>
-      <limit lower="-5" upper="5" effort="1000" velocity="100"/>
+      <limit effort="1000" velocity="100"/>
       <dynamics friction="12.031606150200002"/>
     </joint>
@@ -150,10 +150,10 @@
       </visual>
     </link>
-    <joint name="fr_axle" type="revolute">
+    <joint name="fr_axle" type="continuous">
       <origin rpy="0 -0 0" xyz="0.165 0 0"/>
       <parent link="front_steering_link"/>
       <child link="fr_1"/>
       <axis xyz="-1 0 0"/>
-      <limit lower="-5" upper="5" effort="1000" velocity="100"/>
+      <limit effort="1000" velocity="100"/>
       <dynamics friction="12.031606150200002"/>
     </joint>

File: CustomRobots/f1/urdf/f1_ackermann_cam.urdf (robot description, URDF)
Before this commit: robot f1, 8 links, 7 joints
Joints:
- joint bl_axle: limit lower=-5 upper=5 effort=1000 velocity=100 -> effort=1000 velocity=100; type revolute -> continuous
- joint br_axle: limit lower=-5 upper=5 effort=1000 velocity=100 -> effort=1000 velocity=100; type revolute -> continuous
- joint fl_axle: limit lower=-5 upper=5 effort=1000 velocity=100 -> effort=1000 velocity=100; type revolute -> continuous
- joint fr_axle: limit lower=-5 upper=5 effort=1000 velocity=100 -> effort=1000 velocity=100; type revolute -> continuous

File: CustomRobots/f1/urdf/f1_ackermann_laser.urdf (robot description, URDF)
Before this commit: robot f1, 8 links, 7 joints
Joints:
- joint bl_axle: limit lower=-5 upper=5 effort=1000 velocity=100 -> effort=1000 velocity=100; type revolute -> continuous
- joint br_axle: limit lower=-5 upper=5 effort=1000 velocity=100 -> effort=1000 velocity=100; type revolute -> continuous
- joint fl_axle: limit lower=-5 upper=5 effort=1000 velocity=100 -> effort=1000 velocity=100; type revolute -> continuous
- joint fr_axle: limit lower=-5 upper=5 effort=1000 velocity=100 -> effort=1000 velocity=100; type revolute -> continuous
