Commit message: Update f1 launcher

File: CustomRobots/f1/models/f1/f1.urdf.xacro (robot description, xacro)
@@ -2,201 +2,21 @@
 <robot name="f1"
   xmlns:xacro="http://ros.org/wiki/xacro">
+  <xacro:arg name="holonomic" default="true"/>
+  <xacro:arg name="ackermann" default="false"/>
+  <xacro:arg name="camera" default="true"/>
+  <xacro:arg name="laser" default="false"/>
   <xacro:include filename="$(find custom_robots)/models/f1/f1_gz.urdf.xacro"/>
-  <xacro:macro name="holonomic">
-    <link name="base">
-      <origin rpy="0 0 0" xyz="0 0 0"/>
-      <inertial>
-        <mass value="10"/>
-        <inertia ixx="1" ixy="0.0" ixz="0.0" iyy="1" iyz="0.0" izz="1.0"/>
-      </inertial>
-      <collision>
-        <geometry>
-          <mesh filename="file://$(find custom_robots)/models/f1/meshes/Car.obj" scale="0.2 0.2 0.2"/>
-        </geometry>
-      </collision>
-      <visual name="car">
-        <geometry>
-          <mesh filename="file://$(find custom_robots)/models/f1/meshes/Car.obj" scale="0.2 0.2 0.2"/>
-        </geometry>
-      </visual>
-    </link>
-    <xacro:f1_velocity topic="/F1ROS/cmd_vel"/>
-    <xacro:f1_odom topic="/F1ROS/odom" freq="50"/>
-  </xacro:macro>
-  <xacro:macro name="ackermann">
-    <link name="base"/>
-    <joint name="chassis_link_joint" type="fixed">
-      <origin rpy="0 0 -1.5708" xyz="0.0 0.0 0.0"/>
-      <parent link="base"/>
-      <child link="chassis_link"/>
-    </joint>
-    <link name="chassis_link">
-      <inertial>
-        <origin rpy="0 0 0" xyz="0 0.014614 0.130192"/>
-        <mass value="1580"/>
-        <inertia ixx="1997.86" ixy="-3e-05" ixz="-1e-06" iyy="442.769" iyz="62.5206" izz="2238.05"/>
-      </inertial>
-      <collision>
-        <origin rpy="1.5708 0 1.5708" xyz="0 0.302 0"/>
-        <geometry>
-          <mesh filename="file:///home/ws/install/custom_robots/share/custom_robots/models/f1/meshes/chasis.obj" scale="1 1 1"/>
-        </geometry>
-      </collision>
-      <visual>
-        <origin rpy="1.5708 0 1.5708" xyz="0 0.302 0"/>
-        <geometry>
-          <mesh filename="file:///home/ws/install/custom_robots/share/custom_robots/models/f1/meshes/chasis.obj" scale="1 1 1"/>
-        </geometry>
-      </visual>
-    </link>
-    <joint name="bl_axle" type="continuous">
-      <origin rpy="0 0 0" xyz="-0.155 -0.366728 0.0649994"/>
-      <parent link="chassis_link"/>
-      <child link="bl_1"/>
-      <axis xyz="1 0 0"/>
-      <limit effort="1000" velocity="100"/>
-      <dynamics friction="12.031606150200002"/>
-    </joint>
-    <link name="bl_1">
-      <origin rpy="0 -0 0" xyz="0 0 0"/>
-      <inertial>
-        <origin rpy="0 -0 0" xyz="-0.0377 0 -0"/>
-        <mass value="24.5"/>
-        <inertia ixx="1.84514" ixy="0" ixz="0" iyy="1.04961" iyz="0" izz="1.04961"/>
-      </inertial>
-      <collision>
-        <origin rpy="0 1.5708 0" xyz="0 0 0"/>
-        <geometry>
-          <cylinder length="0.0685" radius="0.066"/>
-        </geometry>
-      </collision>
-      <visual>
-        <origin rpy="0 0 0" xyz="0.175 0.028 -0.20252"/>
-        <geometry>
-          <mesh filename="file:///home/ws/install/custom_robots/share/custom_robots/models/f1/meshes/back_left.obj" scale="0.02 0.02 0.02"/>
-        </geometry>
-      </visual>
-    </link>
-    <joint name="br_axle" type="continuous">
-      <origin rpy="0 0 0" xyz="0.155 -0.366728 0.0649994"/>
-      <parent link="chassis_link"/>
-      <child link="br_1"/>
-      <axis xyz="-1 0 0"/>
-      <limit effort="1000" velocity="100"/>
-      <dynamics friction="12.031606150200002"/>
-    </joint>
-    <link name="br_1">
-      <origin rpy="0 0 0" xyz="0 0 0"/>
-      <inertial>
-        <origin rpy="0 -0 0" xyz="-0.0377 0 -0"/>
-        <mass value="24.5"/>
-        <inertia ixx="1.84514" ixy="0" ixz="0" iyy="1.04961" iyz="0" izz="1.04961"/>
-      </inertial>
-      <collision>
-        <origin rpy="0 1.5708 0" xyz="0 0 0"/>
-        <geometry>
-          <cylinder length="0.0685" radius="0.066"/>
-        </geometry>
-      </collision>
-      <visual>
-        <origin rpy="0 0 0" xyz="-0.175 0.028 -0.20252"/>
-        <geometry>
-          <mesh filename="file:///home/ws/install/custom_robots/share/custom_robots/models/f1/meshes/back_right.obj" scale="0.02 0.02 0.02"/>
-        </geometry>
-      </visual>
-    </link>
-    <joint name="front_steering" type="revolute">
-      <origin rpy="0 0 0" xyz="0 0.303472 0.0649994"/>
-      <parent link="chassis_link"/>
-      <child link="front_steering_link"/>
-      <axis xyz="0 0 1"/>
-      <limit lower="-5" upper="5" effort="1000" velocity="100"/>
-      <dynamics friction="0.5"/>
-    </joint>
-    <link name="front_steering_link">
-      <origin rpy="0 -0 0" xyz="0 0 0"/>
-      <inertial>
-        <origin rpy="0 0 0" xyz="0 0 0"/>
-        <mass value="2"/>
-        <inertia ixx="0.01" ixy="0" ixz="0" iyy="0.01" iyz="0" izz="0.01"/>
-      </inertial>
-    </link>
-    <joint name="fl_axle" type="continuous">
-      <origin rpy="0 -0 0" xyz="-0.165 0 0"/>
-      <parent link="front_steering_link"/>
-      <child link="fl_1"/>
-      <axis xyz="-1 0 0"/>
-      <limit effort="1000" velocity="100"/>
-      <dynamics friction="12.031606150200002"/>
-    </joint>
-    <link name="fl_1">
-      <origin rpy="0 -0 0" xyz="0 0 0"/>
-      <inertial>
-        <origin rpy="0 -0 0" xyz="-0.0377 0 -0"/>
-        <mass value="24.5"/>
-        <inertia ixx="1.84514" ixy="0" ixz="0" iyy="1.04961" iyz="0" izz="1.04961"/>
-      </inertial>
-      <collision>
-        <origin rpy="0 1.5708 0" xyz="0 0 0"/>
-        <geometry>
-          <cylinder length="0.0685" radius="0.066"/>
-        </geometry>
-      </collision>
-      <visual>
-        <origin rpy="0 0 0" xyz="0.175 0.02888 0.30348"/>
-        <geometry>
-          <mesh filename="file:///home/ws/install/custom_robots/share/custom_robots/models/f1/meshes/front_left.obj" scale="0.02 0.02 0.02"/>
-        </geometry>
-      </visual>
-    </link>
-    <joint name="fr_axle" type="continuous">
-      <origin rpy="0 -0 0" xyz="0.165 0 0"/>
-      <parent link="front_steering_link"/>
-      <child link="fr_1"/>
-      <axis xyz="-1 0 0"/>
-      <limit effort="1000" velocity="100"/>
-      <dynamics friction="12.031606150200002"/>
-    </joint>
-    <link name="fr_1">
-      <origin rpy="0 0 0" xyz="0 0 0"/>
-      <inertial>
-        <origin rpy="0 0 0" xyz="-0.0377 0 0"/>
-        <mass value="24.5"/>
-        <inertia ixx="1.84514" ixy="0" ixz="0" iyy="1.04961" iyz="0" izz="1.04961"/>
-      </inertial>
-      <collision>
-        <origin rpy="0 1.5708 0" xyz="0 0 0"/>
-        <geometry>
-          <cylinder length="0.0685" radius="0.066"/>
-        </geometry>
-      </collision>
-      <visual>
-        <origin rpy="0 0 0" xyz="-0.175 0.02888 0.30348"/>
-        <geometry>
-          <mesh filename="file:///home/ws/install/custom_robots/share/custom_robots/models/f1/meshes/front_right.obj" scale="0.02 0.02 0.02"/>
-        </geometry>
-      </visual>
-    </link>
-    <!-- <joint name="steering_joint" type="revolute">
-      <origin rpy="0 0 0" xyz="-0.01 0.6 0.6"/>
-      <parent link="chassis_link"/>
-      <child link="steering_wheel"/>
-      <axis xyz="0.0 -1.0 0.0"/>
-      <limit lower="-5" upper="5"/>
-      <dynamics damping="10.0"/>
-    </joint>
-    <link name="steering_wheel">
-      <origin rpy="0 0 1.5708" xyz="0 0.87 -0.54"/>
-      <visual>
-        <origin rpy="0 0 0" xyz="0 0 0"/>
-        <geometry>
-          <mesh filename="file://$(find custom_robots)/models/f1/meshes/steering_wheel.dae" scale="4.7 4.7 4.7"/>
-        </geometry>
-      </visual>
-    </link> -->
-    <xacro:f1_ackermann_steering topic="/F1ROS/cmd_vel"/>
-    <xacro:f1_joints/>
-    <xacro:f1_odom topic="/F1ROS/odom" freq="50"/>
-    <!-- <xacro:f1_steer_controller topic="/model/f1_renault_ackermann_harmonic/steering_wheel_cmd" joint="steering_joint"/> -->
-  </xacro:macro>
+  <xacro:include filename="$(find custom_robots)/models/f1/f1_common.urdf.xacro"/>
+  <xacro:if value="$(arg holonomic)">
+    <xacro:holonomic/>
+  </xacro:if>
+  <xacro:if value="$(arg ackermann)">
+    <xacro:ackermann/>
+  </xacro:if>
+  <xacro:if value="$(arg camera)">
+    <xacro:f1_camera xyz="0.45 0.04 0.1" rpy="0 0 0" name="cam_f1_left" parent="base"/>
+  </xacro:if>
+  <xacro:if value="$(arg laser)">
+    <xacro:f1_laser xyz="0.5 0 0.072" rpy="0 0 0" name="laser" parent="base"/>
+  </xacro:if>
 </robot>
