Commit message: Fix robot spawn in classic

File: Industrial/ros2_SimRealRobotControl_gz/ros2srrc_robots/ur5/urdf/ur5_ros2control.xacro (robot description, xacro)
@@ -98,5 +98,9 @@
   <xacro:arg name="tf_prefix" default=""/>
   <xacro:property name="tf_prefix" value="$(arg tf_prefix)"/>
-  <xacro:macro name="ur5_ros2control" params="bringup robot_ip EE EE_name script_filename input_recipe_filename output_recipe_filename" >
+  <xacro:macro name="ur5_ros2control" params="
+    bringup robot_ip EE EE_name
+    script_filename input_recipe_filename output_recipe_filename
+    sim_gazebo:=false sim_gz:=false
+  ">
     <!-- ROS2_CONTROL tag name: -->
     <!-- A. GAZEBO SIMULATION: -->

Commit message: Fix spawn robot in classic

File: Industrial/ros2_SimRealRobotControl_gz/ros2srrc_robots/ur5/urdf/ur5_ros2control.xacro (robot description, xacro)
@@ -98,4 +98,6 @@
   <xacro:arg name="tf_prefix" default=""/>
   <xacro:property name="tf_prefix" value="$(arg tf_prefix)"/>
+  <xacro:arg name="sim_gazebo_classic" default="true"/>
+  <xacro:property name="sim_gazebo_classic" value="$(arg sim_gazebo_classic)"/>
   <xacro:macro name="ur5_ros2control" params="bringup robot_ip EE EE_name script_filename input_recipe_filename output_recipe_filename" >
     <!-- ROS2_CONTROL tag name: -->
@@ -113,5 +115,10 @@
       <xacro:unless value="${bringup}">
         <hardware>
-          <plugin>gz_ros2_control/GazeboSimSystem</plugin>
+          <xacro:if value="${sim_gazebo_classic}">
+            <plugin>gazebo_ros2_control/GazeboSystem</plugin>
+          </xacro:if>
+          <xacro:unless value="${sim_gazebo_classic}">
+            <plugin>gz_ros2_control/GazeboSimSystem</plugin>
+          </xacro:unless>
         </hardware>
       </xacro:unless>
