Commit message: Fix robot spawn in classic

File: Industrial/ros2_SimRealRobotControl_gz/ros2srrc_robots/ur5/urdf/ur5_macro.urdf.xacro (robot description, xacro)
@@ -58,5 +58,5 @@
   <xacro:include filename="$(find ros2srrc_robots)/ur5/urdf/ur5_common.xacro"/>
   <!-- XACRO-MACRO of UR5: -->
-  <xacro:macro name="ur5" params="bringup robot_ip EE EE_name script_filename input_recipe_filename output_recipe_filename">
+  <xacro:macro name="ur5" params="bringup robot_ip EE EE_name script_filename input_recipe_filename output_recipe_filename sim">
     <!-- LOAD UR5-Common: -->
     <xacro:ur5_common/>
@@ -68,13 +68,30 @@
     <!-- UR5 GAZEBO - ROS2_CONTROL: -->
     <xacro:include filename="$(find ros2srrc_robots)/ur5/urdf/ur5_ros2control.xacro" />
-    <xacro:ur5_ros2control
-      bringup="${bringup}"
-      robot_ip="${robot_ip}"
-      EE="${EE}"
-      EE_name="${EE_name}"
-      script_filename="${script_filename}"
-      input_recipe_filename="${input_recipe_filename}"
-      output_recipe_filename="${output_recipe_filename}"
-    />
+    <xacro:if value="${sim == 'classic'}">
+      <xacro:ur5_ros2control
+        bringup="${bringup}"
+        robot_ip="${robot_ip}"
+        EE="${EE}"
+        EE_name="${EE_name}"
+        script_filename="${script_filename}"
+        input_recipe_filename="${input_recipe_filename}"
+        output_recipe_filename="${output_recipe_filename}"
+        sim_gazebo="true"
+        sim_gz="false"
+      />
+    </xacro:if>
+    <xacro:if value="${sim == 'gz'}">
+      <xacro:ur5_ros2control
+        bringup="${bringup}"
+        robot_ip="${robot_ip}"
+        EE="${EE}"
+        EE_name="${EE_name}"
+        script_filename="${script_filename}"
+        input_recipe_filename="${input_recipe_filename}"
+        output_recipe_filename="${output_recipe_filename}"
+        sim_gazebo="false"
+        sim_gz="true"
+      />
+    </xacro:if>
     <!-- ***** UR5 ROBOT .urdf SERIAL CHAIN ***** -->
     <!-- Links: -->

Commit message: Fix robot pose in harmonic

File: Industrial/ros2_SimRealRobotControl_gz/ros2srrc_robots/ur5/urdf/ur5_macro.urdf.xacro (robot description, xacro)
@@ -84,8 +84,9 @@
         <origin xyz="0 0 0" rpy="0 0 ${pi}"/>
         <geometry>
-          <mesh filename="file://$(find ros2srrc_robots)/ur5/meshes/visual/base.dae"/>
-        </geometry>
-        <material name="LightGrey">
-          <color rgba="0.7 0.7 0.7 1.0"/>
+          <mesh filename="package://ros2srrc_robots/ur5/meshes/visual/base.dae"/>
+        </geometry>
+        <material>
+          <ambient>0.7 0.7 0.7 1</ambient>
+          <diffuse>0.7 0.7 0.7 1</diffuse>
         </material>
       </visual>
@@ -93,5 +94,5 @@
         <origin xyz="0 0 0" rpy="0 0 ${pi}"/>
         <geometry>
-          <mesh filename="file://$(find ros2srrc_robots)/ur5/meshes/collision/base.stl"/>
+          <mesh filename="package://ros2srrc_robots/ur5/meshes/collision/base.stl"/>
         </geometry>
       </collision>
@@ -104,8 +105,9 @@
         <origin xyz="0 0 0" rpy="0 0 ${pi}"/>
         <geometry>
-          <mesh filename="file://$(find ros2srrc_robots)/ur5/meshes/visual/shoulder.dae"/>
-        </geometry>
-        <material name="LightGrey">
-          <color rgba="0.7 0.7 0.7 1.0"/>
+          <mesh filename="package://ros2srrc_robots/ur5/meshes/visual/shoulder.dae"/>
+        </geometry>
+        <material>
+          <ambient>0.7 0.7 0.7 1</ambient>
+          <diffuse>0.7 0.7 0.7 1</diffuse>
         </material>
       </visual>
@@ -113,5 +115,5 @@
         <origin xyz="0 0 0" rpy="0 0 ${pi}"/>
         <geometry>
-          <mesh filename="file://$(find ros2srrc_robots)/ur5/meshes/collision/shoulder.stl"/>
+          <mesh filename="package://ros2srrc_robots/ur5/meshes/collision/shoulder.stl"/>
         </geometry>
       </collision>
@@ -124,8 +126,9 @@
         <origin xyz="0 0 ${shoulder_offset}" rpy="${pi/2} 0 ${-pi/2}"/>
         <geometry>
-          <mesh filename="file://$(find ros2srrc_robots)/ur5/meshes/visual/upperarm.dae"/>
-        </geometry>
-        <material name="LightGrey">
-          <color rgba="0.7 0.7 0.7 1.0"/>
+          <mesh filename="package://ros2srrc_robots/ur5/meshes/visual/upperarm.dae"/>
+        </geometry>
+        <material>
+          <ambient>0.7 0.7 0.7 1</ambient>
+          <diffuse>0.7 0.7 0.7 1</diffuse>
         </material>
       </visual>
@@ -133,5 +136,5 @@
         <origin xyz="0 0 ${shoulder_offset}" rpy="${pi/2} 0 ${-pi/2}"/>
         <geometry>
-          <mesh filename="file://$(find ros2srrc_robots)/ur5/meshes/collision/upperarm.stl"/>
+          <mesh filename="package://ros2srrc_robots/ur5/meshes/collision/upperarm.stl"/>
         </geometry>
       </collision>
@@ -144,8 +147,9 @@
         <origin xyz="0 0 ${elbow_offset}" rpy="${pi/2} 0 ${-pi/2}"/>
         <geometry>
-          <mesh filename="file://$(find ros2srrc_robots)/ur5/meshes/visual/forearm.dae"/>
-        </geometry>
-        <material name="LightGrey">
-          <color rgba="0.7 0.7 0.7 1.0"/>
+          <mesh filename="package://ros2srrc_robots/ur5/meshes/visual/forearm.dae"/>
+        </geometry>
+        <material>
+          <ambient>0.7 0.7 0.7 1</ambient>
+          <diffuse>0.7 0.7 0.7 1</diffuse>
         </material>
       </visual>
@@ -153,5 +157,5 @@
         <origin xyz="0 0 ${elbow_offset}" rpy="${pi/2} 0 ${-pi/2}"/>
         <geometry>
-          <mesh filename="file://$(find ros2srrc_robots)/ur5/meshes/collision/forearm.stl"/>
+          <mesh filename="package://ros2srrc_robots/ur5/meshes/collision/forearm.stl"/>
         </geometry>
       </collision>
@@ -164,8 +168,9 @@
         <origin xyz="0 0 ${wrist_1_visual_offset}" rpy="${pi/2} 0 0"/>
         <geometry>
-          <mesh filename="file://$(find ros2srrc_robots)/ur5/meshes/visual/wrist1.dae"/>
-        </geometry>
-        <material name="LightGrey">
-          <color rgba="0.7 0.7 0.7 1.0"/>
+          <mesh filename="package://ros2srrc_robots/ur5/meshes/visual/wrist1.dae"/>
+        </geometry>
+        <material>
+          <ambient>0.7 0.7 0.7 1</ambient>
+          <diffuse>0.7 0.7 0.7 1</diffuse>
         </material>
       </visual>
@@ -173,5 +178,5 @@
         <origin xyz="0 0 ${wrist_1_visual_offset}" rpy="${pi/2} 0 0"/>
         <geometry>
-          <mesh filename="file://$(find ros2srrc_robots)/ur5/meshes/collision/wrist1.stl"/>
+          <mesh filename="package://ros2srrc_robots/ur5/meshes/collision/wrist1.stl"/>
         </geometry>
       </collision>
@@ -184,8 +189,9 @@
         <origin xyz="0 0 ${wrist_2_visual_offset}" rpy="0 0 0"/>
         <geometry>
-          <mesh filename="file://$(find ros2srrc_robots)/ur5/meshes/visual/wrist2.dae"/>
-        </geometry>
-        <material name="LightGrey">
-          <color rgba="0.7 0.7 0.7 1.0"/>
+          <mesh filename="package://ros2srrc_robots/ur5/meshes/visual/wrist2.dae"/>
+        </geometry>
+        <material>
+          <ambient>0.7 0.7 0.7 1</ambient>
+          <diffuse>0.7 0.7 0.7 1</diffuse>
         </material>
       </visual>
@@ -193,5 +199,5 @@
         <origin xyz="0 0 ${wrist_2_visual_offset}" rpy="0 0 0"/>
         <geometry>
-          <mesh filename="file://$(find ros2srrc_robots)/ur5/meshes/collision/wrist2.stl"/>
+          <mesh filename="package://ros2srrc_robots/ur5/meshes/collision/wrist2.stl"/>
         </geometry>
       </collision>
@@ -204,8 +210,9 @@
         <origin xyz="0 0 ${wrist_3_visual_offset}" rpy="${pi/2} 0 0"/>
         <geometry>
-          <mesh filename="file://$(find ros2srrc_robots)/ur5/meshes/visual/wrist3.dae"/>
-        </geometry>
-        <material name="LightGrey">
-          <color rgba="0.7 0.7 0.7 1.0"/>
+          <mesh filename="package://ros2srrc_robots/ur5/meshes/visual/wrist3.dae"/>
+        </geometry>
+        <material>
+          <ambient>0.7 0.7 0.7 1</ambient>
+          <diffuse>0.7 0.7 0.7 1</diffuse>
         </material>
       </visual>
@@ -213,5 +220,5 @@
         <origin xyz="0 0 ${wrist_3_visual_offset}" rpy="${pi/2} 0 0"/>
         <geometry>
-          <mesh filename="file://$(find ros2srrc_robots)/ur5/meshes/collision/wrist3.stl"/>
+          <mesh filename="package://ros2srrc_robots/ur5/meshes/collision/wrist3.stl"/>
         </geometry>
       </collision>

Commit message: Fix classic launcher

File: Industrial/ros2_SimRealRobotControl_gz/ros2srrc_robots/ur5/urdf/ur5_macro.urdf.xacro (robot description, xacro)
@@ -84,9 +84,8 @@
         <origin xyz="0 0 0" rpy="0 0 ${pi}"/>
         <geometry>
-          <mesh filename="package://ros2srrc_robots/ur5/meshes/visual/base.dae"/>
-        </geometry>
-        <material>
-          <ambient>0.7 0.7 0.7 1</ambient>
-          <diffuse>0.7 0.7 0.7 1</diffuse>
+          <mesh filename="file://$(find ros2srrc_robots)/ur5/meshes/visual/base.dae"/>
+        </geometry>
+        <material name="LightGrey">
+          <color rgba="0.7 0.7 0.7 1.0"/>
         </material>
       </visual>
@@ -94,5 +93,5 @@
         <origin xyz="0 0 0" rpy="0 0 ${pi}"/>
         <geometry>
-          <mesh filename="package://ros2srrc_robots/ur5/meshes/collision/base.stl"/>
+          <mesh filename="file://$(find ros2srrc_robots)/ur5/meshes/collision/base.stl"/>
         </geometry>
       </collision>
@@ -105,9 +104,8 @@
         <origin xyz="0 0 0" rpy="0 0 ${pi}"/>
         <geometry>
-          <mesh filename="package://ros2srrc_robots/ur5/meshes/visual/shoulder.dae"/>
-        </geometry>
-        <material>
-          <ambient>0.7 0.7 0.7 1</ambient>
-          <diffuse>0.7 0.7 0.7 1</diffuse>
+          <mesh filename="file://$(find ros2srrc_robots)/ur5/meshes/visual/shoulder.dae"/>
+        </geometry>
+        <material name="LightGrey">
+          <color rgba="0.7 0.7 0.7 1.0"/>
         </material>
       </visual>
@@ -115,5 +113,5 @@
         <origin xyz="0 0 0" rpy="0 0 ${pi}"/>
         <geometry>
-          <mesh filename="package://ros2srrc_robots/ur5/meshes/collision/shoulder.stl"/>
+          <mesh filename="file://$(find ros2srrc_robots)/ur5/meshes/collision/shoulder.stl"/>
         </geometry>
       </collision>
@@ -126,9 +124,8 @@
         <origin xyz="0 0 ${shoulder_offset}" rpy="${pi/2} 0 ${-pi/2}"/>
         <geometry>
-          <mesh filename="package://ros2srrc_robots/ur5/meshes/visual/upperarm.dae"/>
-        </geometry>
-        <material>
-          <ambient>0.7 0.7 0.7 1</ambient>
-          <diffuse>0.7 0.7 0.7 1</diffuse>
+          <mesh filename="file://$(find ros2srrc_robots)/ur5/meshes/visual/upperarm.dae"/>
+        </geometry>
+        <material name="LightGrey">
+          <color rgba="0.7 0.7 0.7 1.0"/>
         </material>
       </visual>
@@ -136,5 +133,5 @@
         <origin xyz="0 0 ${shoulder_offset}" rpy="${pi/2} 0 ${-pi/2}"/>
         <geometry>
-          <mesh filename="package://ros2srrc_robots/ur5/meshes/collision/upperarm.stl"/>
+          <mesh filename="file://$(find ros2srrc_robots)/ur5/meshes/collision/upperarm.stl"/>
         </geometry>
       </collision>
@@ -147,9 +144,8 @@
         <origin xyz="0 0 ${elbow_offset}" rpy="${pi/2} 0 ${-pi/2}"/>
         <geometry>
-          <mesh filename="package://ros2srrc_robots/ur5/meshes/visual/forearm.dae"/>
-        </geometry>
-        <material>
-          <ambient>0.7 0.7 0.7 1</ambient>
-          <diffuse>0.7 0.7 0.7 1</diffuse>
+          <mesh filename="file://$(find ros2srrc_robots)/ur5/meshes/visual/forearm.dae"/>
+        </geometry>
+        <material name="LightGrey">
+          <color rgba="0.7 0.7 0.7 1.0"/>
         </material>
       </visual>
@@ -157,5 +153,5 @@
         <origin xyz="0 0 ${elbow_offset}" rpy="${pi/2} 0 ${-pi/2}"/>
         <geometry>
-          <mesh filename="package://ros2srrc_robots/ur5/meshes/collision/forearm.stl"/>
+          <mesh filename="file://$(find ros2srrc_robots)/ur5/meshes/collision/forearm.stl"/>
         </geometry>
       </collision>
@@ -168,9 +164,8 @@
         <origin xyz="0 0 ${wrist_1_visual_offset}" rpy="${pi/2} 0 0"/>
         <geometry>
-          <mesh filename="package://ros2srrc_robots/ur5/meshes/visual/wrist1.dae"/>
-        </geometry>
-        <material>
-          <ambient>0.7 0.7 0.7 1</ambient>
-          <diffuse>0.7 0.7 0.7 1</diffuse>
+          <mesh filename="file://$(find ros2srrc_robots)/ur5/meshes/visual/wrist1.dae"/>
+        </geometry>
+        <material name="LightGrey">
+          <color rgba="0.7 0.7 0.7 1.0"/>
         </material>
       </visual>
@@ -178,5 +173,5 @@
         <origin xyz="0 0 ${wrist_1_visual_offset}" rpy="${pi/2} 0 0"/>
         <geometry>
-          <mesh filename="package://ros2srrc_robots/ur5/meshes/collision/wrist1.stl"/>
+          <mesh filename="file://$(find ros2srrc_robots)/ur5/meshes/collision/wrist1.stl"/>
         </geometry>
       </collision>
@@ -189,9 +184,8 @@
         <origin xyz="0 0 ${wrist_2_visual_offset}" rpy="0 0 0"/>
         <geometry>
-          <mesh filename="package://ros2srrc_robots/ur5/meshes/visual/wrist2.dae"/>
-        </geometry>
-        <material>
-          <ambient>0.7 0.7 0.7 1</ambient>
-          <diffuse>0.7 0.7 0.7 1</diffuse>
+          <mesh filename="file://$(find ros2srrc_robots)/ur5/meshes/visual/wrist2.dae"/>
+        </geometry>
+        <material name="LightGrey">
+          <color rgba="0.7 0.7 0.7 1.0"/>
         </material>
       </visual>
@@ -199,5 +193,5 @@
         <origin xyz="0 0 ${wrist_2_visual_offset}" rpy="0 0 0"/>
         <geometry>
-          <mesh filename="package://ros2srrc_robots/ur5/meshes/collision/wrist2.stl"/>
+          <mesh filename="file://$(find ros2srrc_robots)/ur5/meshes/collision/wrist2.stl"/>
         </geometry>
       </collision>
@@ -210,9 +204,8 @@
         <origin xyz="0 0 ${wrist_3_visual_offset}" rpy="${pi/2} 0 0"/>
         <geometry>
-          <mesh filename="package://ros2srrc_robots/ur5/meshes/visual/wrist3.dae"/>
-        </geometry>
-        <material>
-          <ambient>0.7 0.7 0.7 1</ambient>
-          <diffuse>0.7 0.7 0.7 1</diffuse>
+          <mesh filename="file://$(find ros2srrc_robots)/ur5/meshes/visual/wrist3.dae"/>
+        </geometry>
+        <material name="LightGrey">
+          <color rgba="0.7 0.7 0.7 1.0"/>
         </material>
       </visual>
@@ -220,5 +213,5 @@
         <origin xyz="0 0 ${wrist_3_visual_offset}" rpy="${pi/2} 0 0"/>
         <geometry>
-          <mesh filename="package://ros2srrc_robots/ur5/meshes/collision/wrist3.stl"/>
+          <mesh filename="file://$(find ros2srrc_robots)/ur5/meshes/collision/wrist3.stl"/>
         </geometry>
       </collision>
