Commit message: Fix typo

File: CustomRobots/autonomous_car/models/autonomous_car/autonomous_car_common.urdf.xacro (robot description, xacro)
@@ -141,5 +141,5 @@
         <origin rpy="0 0 0" xyz="0.13 0 0"/>
         <geometry>
-          <mesh filename="$(find custom_robots)/models/f1/meshes/front_left.obj" scale="0.02 0.02 0.02"/>
+          <mesh filename="$(find custom_robots)/models/autonomous_car/meshes/wheel.obj" scale="0.01 0.01 0.01"/>
         </geometry>
       </visual>
@@ -169,5 +169,5 @@
         <origin rpy="0 0 0" xyz="-0.13 0 0"/>
         <geometry>
-          <mesh filename="file://$(find custom_robots)/models/f1/meshes/front_left.obj" scale="0.02 0.02 0.02"/>
+          <mesh filename="$(find custom_robots)/models/autonomous_car/meshes/wheel.obj" scale="0.01 0.01 0.01"/>
         </geometry>
       </visual>

Commit message: Working autonomous car

File: CustomRobots/autonomous_car/models/autonomous_car/autonomous_car_common.urdf.xacro (robot description, xacro)
@@ -30,5 +30,5 @@
     </link>
     <joint name="bl_axle" type="continuous">
-      <origin rpy="0 0 0" xyz="-0.775 -1.63364 0.324997"/>
+      <origin rpy="0 0 0" xyz="-0.775 -1.52 0.324997"/>
       <parent link="chassis_link"/>
       <child link="bl_1"/>
@@ -58,5 +58,5 @@
     </link>
     <joint name="br_axle" type="continuous">
-      <origin rpy="0 0 0" xyz="0.775 -1.63364 0.324997"/>
+      <origin rpy="0 0 0" xyz="0.775 -1.52 0.324997"/>
       <parent link="chassis_link"/>
       <child link="br_1"/>
@@ -86,5 +86,5 @@
     </link>
     <joint name="l_steer" type="revolute">
-      <origin rpy="0 0 0" xyz="-0.825 1.51736 0.324997"/>
+      <origin rpy="0 0 0" xyz="-0.825 1.32 0.324997"/>
       <parent link="chassis_link"/>
       <child link="l_steer_1"/>
@@ -102,5 +102,5 @@
     </link>
     <joint name="r_steer" type="revolute">
-      <origin rpy="0 0 0" xyz="0.825 1.51736 0.324997"/>
+      <origin rpy="0 0 0" xyz="0.825 1.32 0.324997"/>
       <parent link="chassis_link"/>
       <child link="r_steer_1"/>

File: CustomRobots/autonomous_car/models/autonomous_car/autonomous_car_gz.urdf.xacro (robot description, xacro)
@@ -57,5 +57,5 @@
     </joint>
     <gazebo reference="${name}_link">
-      <sensor name="laser" type="gpu_lidar">
+      <sensor name="${name}" type="gpu_lidar">
         <always_on>1</always_on>
         <visualize>1</visualize>
