Commit message: Test holo taxi

File: CustomRobots/autonomous_car/models/autonomous_car/autonomous_car.urdf.xacro (robot description, xacro)
@@ -5,7 +5,8 @@
   <xacro:arg name="lidar" default="false"/>
   <xacro:arg name="laser" default="false"/>
+  <xacro:arg name="steering" default="ackermann"/>
   <xacro:include filename="$(find custom_robots)/models/autonomous_car/autonomous_car_gz.urdf.xacro"/>
   <xacro:include filename="$(find custom_robots)/models/autonomous_car/autonomous_car_common.urdf.xacro"/>
-  <xacro:autonomous_car/>
+  <xacro:autonomous_car steering="$(arg ackermann)"/>
   <xacro:if value="$(arg camera)">
     <xacro:camera xyz="0 0.2 1.45" rpy="0 0 1.5708" name="prius_autoparking" parent="base_link"/>

File: CustomRobots/autonomous_car/models/autonomous_car/autonomous_car_common.urdf.xacro (robot description, xacro)
@@ -3,5 +3,5 @@
   xmlns:xacro="http://ros.org/wiki/xacro">
   <xacro:include filename="$(find custom_robots)/models/autonomous_car/autonomous_car_gz.urdf.xacro"/>
-  <xacro:macro name="autonomous_car">
+  <xacro:macro name="autonomous_car" params="steering">
     <link name="base_link"/>
     <joint name="chassis_link_joint" type="fixed">
@@ -191,5 +191,10 @@
       <pose relative_to='steering_joint'>0 0.87 -0.54 0 0 1.5708</pose>
     </link> -->
-    <xacro:ackermann_steering topic="/prius_autoparking/cmd_vel"/>
+    <xacro:if value="${steering == 'holonomic'}">
+      <xacro:velocity topic="/cmd_vel"/>
+    </xacro:if>
+    <xacro:if value="${steering == 'ackermann'}">
+      <xacro:ackermann_steering topic="/prius_autoparking/cmd_vel"/>
+    </xacro:if>
     <xacro:joints/>
     <xacro:odom topic="/prius_autoparking/odom" freq="50"/>

File: CustomRobots/autonomous_car/models/autonomous_car/autonomous_car_gz.urdf.xacro (robot description, xacro)
@@ -192,4 +192,11 @@
     </gazebo>
   </xacro:macro>
+  <xacro:macro name="velocity" params="topic freq">
+    <gazebo>
+      <plugin filename="gz-sim-velocity-control-system" name="gz::sim::systems::VelocityControl">
+        <topic>${topic}</topic>
+      </plugin>
+    </gazebo>
+  </xacro:macro>
   <xacro:macro name="joints">
     <gazebo>

Commit message: Test argument

File: CustomRobots/autonomous_car/models/autonomous_car/autonomous_car.urdf.xacro (robot description, xacro)
@@ -6,7 +6,8 @@
   <xacro:arg name="laser" default="false"/>
   <xacro:arg name="steering" default="ackermann"/>
+  <xacro:property name="steering" value="$(arg steering)"/>
   <xacro:include filename="$(find custom_robots)/models/autonomous_car/autonomous_car_gz.urdf.xacro"/>
   <xacro:include filename="$(find custom_robots)/models/autonomous_car/autonomous_car_common.urdf.xacro"/>
-  <xacro:autonomous_car steering="$(arg ackermann)"/>
+  <xacro:autonomous_car steering="${ackermann}"/>
   <xacro:if value="$(arg camera)">
     <xacro:camera xyz="0 0.2 1.45" rpy="0 0 1.5708" name="prius_autoparking" parent="base_link"/>
