Commit message: Update autonomous car

File: CustomRobots/autonomous_car/models/autonomous_car/autonomous_car.urdf.xacro (robot description, xacro)
@@ -6,18 +6,20 @@
   <xacro:arg name="laser" default="false"/>
   <xacro:arg name="steering" default="ackermann"/>
+  <xacro:arg name="namespace" default="autonomous_car"/>
   <xacro:property name="steering" value="$(arg steering)"/>
+  <xacro:property name="namespace" value="$(arg namespace)"/>
   <xacro:include filename="$(find custom_robots)/models/autonomous_car/autonomous_car_gz.urdf.xacro"/>
   <xacro:include filename="$(find custom_robots)/models/autonomous_car/autonomous_car_common.urdf.xacro"/>
-  <xacro:autonomous_car steering="${steering}"/>
+  <xacro:autonomous_car steering="${steering}" namespace="${namespace}"/>
   <xacro:if value="$(arg camera)">
-    <xacro:camera xyz="0 0.2 1.45" rpy="0 0 0" name="prius_autoparking" parent="base_link"/>
+    <xacro:camera xyz="0 0.2 1.45" rpy="0 0 0" parent="base_link" name="camera" namespace="${namespace}"/>
   </xacro:if>
   <xacro:if value="$(arg lidar)">
-    <xacro:lidar xyz="-1.25 0 1.725" rpy="0 0 -1.578" name="lidar" parent="base_link" topic="/prius_autoparking/pc2"/>
+    <xacro:lidar xyz="-1.25 0 1.725" rpy="0 0 -1.578" name="lidar" parent="base_link" namespace="${namespace}"/>
   </xacro:if>
   <xacro:if value="$(arg laser)">
-    <xacro:laser xyz="-0.024 2.39 0.5" rpy="0 0 1.5708" name="laser_front" parent="chassis_link" topic="/prius_autoparking/scan_front"/>
-    <xacro:laser xyz="1.1 0 0.5" rpy="0 0 0" name="laser_side" parent="chassis_link" topic="/prius_autoparking/scan_side"/>
-    <xacro:laser xyz="-0.024 -2.6 0.5" rpy="0 0 -1.5708" name="laser_back" parent="chassis_link" topic="/prius_autoparking/scan_back"/>
+    <xacro:laser xyz="-0.024 2.39 0.5" rpy="0 0 1.5708" name="laser_front" parent="chassis_link" namespace="${namespace}"/>
+    <xacro:laser xyz="1.1 0 0.5" rpy="0 0 0" name="laser_side" parent="chassis_link" namespace="${namespace}"/>
+    <xacro:laser xyz="-0.024 -2.6 0.5" rpy="0 0 -1.5708" name="laser_back" parent="chassis_link" namespace="${namespace}"/>
   </xacro:if>
 </robot>

File: CustomRobots/autonomous_car/models/autonomous_car/autonomous_car_common.urdf.xacro (robot description, xacro)
@@ -3,5 +3,5 @@
   xmlns:xacro="http://ros.org/wiki/xacro">
   <xacro:include filename="$(find custom_robots)/models/autonomous_car/autonomous_car_gz.urdf.xacro"/>
-  <xacro:macro name="autonomous_car" params="steering">
+  <xacro:macro name="autonomous_car" params="steering namespace">
     <link name="base_link"/>
     <joint name="chassis_link_joint" type="fixed">
@@ -192,11 +192,11 @@
     </link> -->
     <xacro:if value="${steering == 'holonomic'}">
-      <xacro:velocity topic="/cmd_vel"/>
+      <xacro:velocity namespace="${namespace}"/>
     </xacro:if>
     <xacro:if value="${steering == 'ackermann'}">
-      <xacro:ackermann_steering topic="/prius_autoparking/cmd_vel"/>
+      <xacro:ackermann_steering namespace="${namespace}"/>
     </xacro:if>
     <xacro:joints/>
-    <xacro:odom topic="/prius_autoparking/odom" freq="50"/>
+    <xacro:odom namespace="${namespace}" freq="50"/>
     <!-- <xacro:f1_steer_controller topic="/model/prius_autoparking/steering_wheel_cmd" joint="steering_joint"/> -->
   </xacro:macro>

File: CustomRobots/autonomous_car/models/autonomous_car/autonomous_car_gz.urdf.xacro (robot description, xacro)
@@ -2,5 +2,5 @@
 <robot name="autonomous_car_gz"
   xmlns:xacro="http://ros.org/wiki/xacro">
-  <xacro:macro name="camera" params="xyz rpy name parent">
+  <xacro:macro name="camera" params="xyz rpy parent name namespace">
     <link name="${name}_link"></link>
     <joint name="${name}_to_${parent}" type="fixed">
@@ -14,7 +14,7 @@
         <visualize>false</visualize>
         <update_rate>20</update_rate>
-        <topic>/${name}/image_raw</topic>
+        <topic>/${namespace}/${name}/image_raw</topic>
         <camera name="camera">
-          <camera_info_topic>/${name}/camera_info</camera_info_topic>
+          <camera_info_topic>/${namespace}/${name}/camera_info</camera_info_topic>
           <horizontal_fov>2.094</horizontal_fov>
           <lens>
@@ -49,5 +49,5 @@
     </gazebo>
   </xacro:macro>
-  <xacro:macro name="laser" params="xyz rpy name parent topic">
+  <xacro:macro name="laser" params="xyz rpy name parent namespace">
     <link name="${name}_link"></link>
     <joint name="${name}_to_${parent}" type="fixed">
@@ -61,5 +61,5 @@
         <visualize>1</visualize>
         <update_rate>20</update_rate>
-        <topic>${topic}</topic>
+        <topic>/${namespace}/${name}/scan</topic>
         <gz_frame_id>base_scan</gz_frame_id>
         <lidar>
@@ -81,5 +81,5 @@
     </gazebo>
   </xacro:macro>
-  <xacro:macro name="lidar" params="xyz rpy name parent topic">
+  <xacro:macro name="lidar" params="xyz rpy name parent namespace">
     <material name="white">
       <color rgba="1.0 1.0 1.0 1.0"/>
@@ -128,5 +128,5 @@
         <visualize>1</visualize>
         <update_rate>20</update_rate>
-        <topic>${topic}</topic>
+        <topic>/${namespace}/${name}/pc2</topic>
         <gz_frame_id>base_scan</gz_frame_id>
         <lidar>
@@ -159,5 +159,5 @@
     </gazebo>
   </xacro:macro>
-  <xacro:macro name="ackermann_steering" params="topic">
+  <xacro:macro name="ackermann_steering" params="namespace">
     <gazebo>
       <plugin filename="gz-sim-ackermann-steering-system" name="gz::sim::systems::AckermannSteering">
@@ -177,9 +177,9 @@
         <min_acceleration>-50</min_acceleration>
         <max_acceleration>50</max_acceleration>
-        <topic>${topic}</topic>
-      </plugin>
-    </gazebo>
-  </xacro:macro>
-  <xacro:macro name="odom" params="topic freq">
+        <topic>/${namespace}/cmd_vel</topic>
+      </plugin>
+    </gazebo>
+  </xacro:macro>
+  <xacro:macro name="odom" params="namespace freq">
     <gazebo>
       <plugin filename="gz-sim-odometry-publisher-system" name="gz::sim::systems::OdometryPublisher">
@@ -187,5 +187,5 @@
         <robot_base_frame>chassis_link</robot_base_frame>
         <odom_publish_frequency>${freq}</odom_publish_frequency>
-        <odom_topic>${topic}</odom_topic>
+        <odom_topic>/${namespace}/odom</odom_topic>
         <dimensions>3</dimensions>
       </plugin>
@@ -195,5 +195,5 @@
     <gazebo>
       <plugin filename="gz-sim-velocity-control-system" name="gz::sim::systems::VelocityControl">
-        <topic>${topic}</topic>
+        <topic>/${namespace}/cmd_vel</topic>
       </plugin>
     </gazebo>
