Commit message: Fix final topic

File: CustomRobots/autonomous_car/models/autonomous_car/autonomous_car_gz.urdf.xacro (robot description, xacro)
@@ -192,5 +192,5 @@
     </gazebo>
   </xacro:macro>
-  <xacro:macro name="velocity" params="topic freq">
+  <xacro:macro name="velocity" params="topic">
     <gazebo>
       <plugin filename="gz-sim-velocity-control-system" name="gz::sim::systems::VelocityControl">
