Commit message: More tests

File: CustomRobots/vacuum_cleaner/models/vacuum_cleaner/vacuum_cleaner.urdf.xacro (robot description, xacro)
@@ -7,4 +7,7 @@
   <xacro:include filename="$(find custom_robots)/models/vacuum_cleaner/vacuum_cleaner_common.urdf.xacro"/>
   <xacro:vacuum_cleaner/>
+  <gazebo>
+    <plugin name="gz::sim::systems::Contact" filename="gz-sim-contact-system"></plugin>
+  </gazebo>
   <xacro:if value="$(arg camera)">
     <xacro:camera xyz="0 0 0" rpy="0 -1.57 0" name="camera" parent="base"/>

File: CustomRobots/vacuum_cleaner/models/vacuum_cleaner/vacuum_cleaner_common.urdf.xacro (robot description, xacro)
@@ -43,11 +43,11 @@
     </joint>
     <link name="center_bumper_link">
-      <collision>
+      <collision name="center_bumper_collision">
         <geometry>
           <mesh filename="$(find custom_robots)/models/vacuum_cleaner/meshes/center_bumper.dae"/>
         </geometry>
       </collision>
+      <xacro:bumper topic="/roombaROS/events/center_bumper" name="center_bumper"/>
     </link>
-    <xacro:bumper topic="/roombaROS/events/center_bumper" name="center_bumper"/>
     <joint name="left_bumper_joint" type="fixed">
       <origin rpy="0 0 0" xyz="-0.01 0 0.03"/>

File: CustomRobots/vacuum_cleaner/models/vacuum_cleaner/vacuum_cleaner_gz.urdf.xacro (robot description, xacro)
@@ -83,17 +83,10 @@
   </xacro:macro>
   <xacro:macro name="bumper" params="topic name">
-    <gazebo reference="${name}_link">
-      <mu1>0.1</mu1>
-      <mu2>0.1</mu2>
-      <maxVel>0.01</maxVel>
-      <minDepth>0.001</minDepth>
-      <maxContacts>10</maxContacts>
-      <material>Gazebo/DarkGrey</material>
-      <plugin name="gz::sim::systems::Contact" filename="gz-sim-contact-system"></plugin>
-      <sensor name='${name}_sensor' type='contact'>
+    <gazebo>
+      <sensor name='${name}' type='contact'>
         <always_on>true</always_on>
         <update_rate>20</update_rate>
         <contact>
-          <collision>${name}_link_collision</collision>
+          <collision>${name}_collision</collision>
           <topic>${topic}</topic>
         </contact>

Commit message: Clean xacro

File: CustomRobots/vacuum_cleaner/models/vacuum_cleaner/vacuum_cleaner.urdf.xacro (robot description, xacro)
@@ -7,7 +7,4 @@
   <xacro:include filename="$(find custom_robots)/models/vacuum_cleaner/vacuum_cleaner_common.urdf.xacro"/>
   <xacro:vacuum_cleaner/>
-  <gazebo>
-    <plugin name="gz::sim::systems::Contact" filename="gz-sim-contact-system"></plugin>
-  </gazebo>
   <xacro:if value="$(arg camera)">
     <xacro:camera xyz="0 0 0" rpy="0 -1.57 0" name="camera" parent="base"/>

File: CustomRobots/vacuum_cleaner/models/vacuum_cleaner/vacuum_cleaner_common.urdf.xacro (robot description, xacro)
@@ -3,4 +3,7 @@
   <xacro:include filename="$(find custom_robots)/models/vacuum_cleaner/vacuum_cleaner_gz.urdf.xacro"/>
   <xacro:macro name="vacuum_cleaner">
+    <gazebo>
+      <plugin name="gz::sim::systems::Contact" filename="gz-sim-contact-system"></plugin>
+    </gazebo>
     <link name="base">
       <inertial>
@@ -28,11 +31,10 @@
     </joint>
     <link name="right_bumper_link">
-      <collision>
-        <origin rpy="0 0 0" xyz="0 0 0"/>
+      <collision name="right_bumper_collision">
         <geometry>
           <mesh filename="$(find custom_robots)/models/vacuum_cleaner/meshes/right_bumper.dae"/>
         </geometry>
       </collision>
-      <!-- <xacro:bumper topic="/roombaROS/events/right_bumper" name="right_bumper_link"/> -->
+      <xacro:bumper topic="/roombaROS/events/right_bumper" name="right_bumper"/>
     </link>
     <joint name="center_bumper_joint" type="fixed">
@@ -47,16 +49,6 @@
         </geometry>
       </collision>
-      <!-- <xacro:bumper topic="/roombaROS/events/center_bumper" name="center_bumper"/> -->
+      <xacro:bumper topic="/roombaROS/events/center_bumper" name="center_bumper"/>
     </link>
-    <gazebo>
-      <sensor name="center_bumper" type="contact">
-        <always_on>true</always_on>
-        <update_rate>20.0</update_rate>
-        <contact>
-          <collision>center_bumper_collision</collision>
-          <topic>/roombaROS/events/center_bumper</topic>
-        </contact>
-      </sensor>
-    </gazebo>
     <joint name="left_bumper_joint" type="fixed">
       <origin rpy="0 0 0" xyz="-0.01 0 0.03"/>
@@ -65,11 +57,10 @@
     </joint>
     <link name="left_bumper_link">
-      <collision>
-        <origin rpy="0 0 0" xyz="0 0 0"/>
+      <collision name="left_bumper_collision">
         <geometry>
           <mesh filename="$(find custom_robots)/models/vacuum_cleaner/meshes/left_bumper.dae"/>
         </geometry>
       </collision>
-      <!-- <xacro:bumper topic="/roombaROS/events/left_bumper" name="left_bumper_link"/> -->
+      <xacro:bumper topic="/roombaROS/events/left_bumper" name="left_bumper"/>
     </link>
     <joint name="front_wheel_joint" type="fixed">

File: CustomRobots/vacuum_cleaner/models/vacuum_cleaner/vacuum_cleaner_gz.urdf.xacro (robot description, xacro)
@@ -92,12 +92,4 @@
         </contact>
       </sensor>
-      <sensor name="${name}" type="contact">
-        <always_on>true</always_on>
-        <update_rate>20.0</update_rate>
-        <contact>
-          <collision>center_bumper_collision</collision>
-          <topic>/roombaROS/events/center_bumper</topic>
-        </contact>
-      </sensor>
     </gazebo>
   </xacro:macro>
