Commit message: Update vacuum cleaner

File: CustomRobots/vacuum_cleaner/models/vacuum_cleaner/vacuum_cleaner.urdf.xacro (robot description, xacro)
@@ -4,12 +4,14 @@
   <xacro:arg name="camera" default="true"/>
   <xacro:arg name="laser" default="false"/>
+  <xacro:arg name="namespace" default="vacuum_cleaner"/>
+  <xacro:property name="namespace" value="$(arg namespace)"/>
   <xacro:include filename="$(find custom_robots)/models/vacuum_cleaner/vacuum_cleaner_gz.urdf.xacro"/>
   <xacro:include filename="$(find custom_robots)/models/vacuum_cleaner/vacuum_cleaner_common.urdf.xacro"/>
-  <xacro:vacuum_cleaner/>
+  <xacro:vacuum_cleaner namespace="${namespace}"/>
   <xacro:if value="$(arg camera)">
-    <xacro:camera xyz="0 0 0" rpy="0 -1.57 0" name="camera" parent="base"/>
+    <xacro:camera xyz="0 0 0" rpy="0 -1.57 0" name="camera" parent="base" namespace="${namespace}"/>
   </xacro:if>
   <xacro:if value="$(arg laser)">
-    <xacro:laser xyz="0.139 0 0.0752" rpy="0 0 0" name="laser" parent="base" topic="/roombaROS/laser/scan"/>
+    <xacro:laser xyz="0.139 0 0.0752" rpy="0 0 0" name="laser" parent="base" namespace="${namespace}"/>
   </xacro:if>
 </robot>

File: CustomRobots/vacuum_cleaner/models/vacuum_cleaner/vacuum_cleaner_common.urdf.xacro (robot description, xacro)
@@ -2,5 +2,5 @@
 <robot xmlns:xacro="http://ros.org/wiki/xacro">
   <xacro:include filename="$(find custom_robots)/models/vacuum_cleaner/vacuum_cleaner_gz.urdf.xacro"/>
-  <xacro:macro name="vacuum_cleaner">
+  <xacro:macro name="vacuum_cleaner" params="namespace">
     <gazebo>
       <plugin name="gz::sim::systems::Contact" filename="gz-sim-contact-system"></plugin>
@@ -37,5 +37,5 @@
       </collision>
     </link>
-    <xacro:bumper topic="/roombaROS/events/right_bumper" name="right_bumper"/>
+    <xacro:bumper topic="events/right_bumper" name="right_bumper" namespace="${namespace}"/>
     <joint name="center_bumper_joint" type="fixed">
       <origin rpy="0 0 0" xyz="-0.01 0 0.03"/>
@@ -50,5 +50,5 @@
       </collision>
     </link>
-    <xacro:bumper topic="/roombaROS/events/center_bumper" name="center_bumper"/>
+    <xacro:bumper topic="events/center_bumper" name="center_bumper" namespace="${namespace}"/>
     <joint name="left_bumper_joint" type="fixed">
       <origin rpy="0 0 0" xyz="-0.01 0 0.03"/>
@@ -63,5 +63,5 @@
       </collision>
     </link>
-    <xacro:bumper topic="/roombaROS/events/left_bumper" name="left_bumper"/>
+    <xacro:bumper topic="events/left_bumper" name="left_bumper" namespace="${namespace}"/>
     <joint name="front_wheel_joint" type="fixed">
       <origin rpy="0 1.570700 1.570700" xyz="0.13 0 0.017"/>
@@ -154,7 +154,7 @@
       </visual>
     </link>
-    <xacro:velocity topic="/roombaROS/cmd_vel"/>
-    <xacro:odom topic="/roombaROS/odom" freq="20"/>
-    <xacro:noise_odom topic="/odom_noisy"/>
+    <xacro:velocity namespace="${namespace}"/>
+    <xacro:odom freq="20" namespace="${namespace}"/>
+    <xacro:noise_odom namespace="${namespace}"/>
   </xacro:macro>
 </robot>

File: CustomRobots/vacuum_cleaner/models/vacuum_cleaner/vacuum_cleaner_gz.urdf.xacro (robot description, xacro)
@@ -2,5 +2,5 @@
 <robot name="vacuum_cleaner_gz"
   xmlns:xacro="http://ros.org/wiki/xacro">
-  <xacro:macro name="camera" params="xyz rpy name parent">
+  <xacro:macro name="camera" params="xyz rpy name parent namespace">
     <link name="${name}_link"></link>
     <joint name="${name}_to_${parent}" type="fixed">
@@ -14,7 +14,7 @@
         <visualize>false</visualize>
         <update_rate>20</update_rate>
-        <topic>/${name}/image_raw</topic>
+        <topic>/${namespace}/${name}/image_raw</topic>
         <camera name="camera">
-          <camera_info_topic>/${name}/camera_info</camera_info_topic>
+          <camera_info_topic>/${namespace}/${name}/camera_info</camera_info_topic>
           <horizontal_fov>1.089</horizontal_fov>
           <distortion>
@@ -44,5 +44,5 @@
     </gazebo>
   </xacro:macro>
-  <xacro:macro name="laser" params="xyz rpy name parent topic">
+  <xacro:macro name="laser" params="xyz rpy name parent namespace">
     <link name="${name}_link">
       <visual>
@@ -62,5 +62,5 @@
         <visualize>1</visualize>
         <update_rate>20</update_rate>
-        <topic>${topic}</topic>
+        <topic>/${namespace}/laser/scan</topic>
         <gz_frame_id>laser</gz_frame_id>
         <lidar>
@@ -82,5 +82,5 @@
     </gazebo>
   </xacro:macro>
-  <xacro:macro name="bumper" params="topic name">
+  <xacro:macro name="bumper" params="topic name namespace">
     <gazebo reference="${name}">
       <mu1>0.1</mu1>
@@ -96,17 +96,17 @@
         <contact>
           <collision>${name}_collision</collision>
-          <topic>${topic}</topic>
+          <topic>/${namespace}/${topic}</topic>
         </contact>
       </sensor>
     </gazebo>
   </xacro:macro>
-  <xacro:macro name="velocity" params="topic">
+  <xacro:macro name="velocity" params="namespace">
     <gazebo>
       <plugin filename="gz-sim-velocity-control-system" name="gz::sim::systems::VelocityControl">
-        <topic>${topic}</topic>
+        <topic>/${namespace}/cmd_vel</topic>
       </plugin>
     </gazebo>
   </xacro:macro>
-  <xacro:macro name="odom" params="topic freq">
+  <xacro:macro name="odom" params="freq namespace">
     <gazebo>
       <plugin filename="gz-sim-odometry-publisher-system" name="gz::sim::systems::OdometryPublisher">
@@ -114,13 +114,13 @@
         <robot_base_frame>base</robot_base_frame>
         <odom_publish_frequency>${freq}</odom_publish_frequency>
-        <odom_topic>${topic}</odom_topic>
+        <odom_topic>/${namespace}/odom</odom_topic>
         <dimensions>3</dimensions>
       </plugin>
     </gazebo>
   </xacro:macro>
-  <xacro:macro name="noise_odom" params="topic">
+  <xacro:macro name="noise_odom" params="topic namespace">
     <gazebo>
       <plugin filename="libNoisyOdometryPlugin.so" name="custom_plugins::NoisyOdometryPlugin">
-        <ros_topic>${topic}</ros_topic>
+        <ros_topic>/${namespace}/odom_noisy</ros_topic>
         <frame_id>odom</frame_id>
         <child_frame_id>base</child_frame_id>
