Commit message: Test

File: CustomRobots/vacuum_cleaner/models/vacuum_cleaner/vacuum_cleaner_common.urdf.xacro (robot description, xacro)
@@ -29,5 +29,5 @@
     </joint>
     <link name="right_bumper_link">
-      <collision>
+      <collision name="right_bumper">
         <origin rpy="0 0 0" xyz="0 0 0"/>
         <geometry>
@@ -43,5 +43,5 @@
     </joint>
     <link name="center_bumper_link">
-      <collision>
+      <collision name="center_bumper">
         <origin rpy="0 0 0" xyz="0 0 0"/>
         <geometry>
@@ -57,5 +57,5 @@
     </joint>
     <link name="left_bumper_link">
-      <collision>
+      <collision name="left_bumper">
         <origin rpy="0 0 0" xyz="0 0 0"/>
         <geometry>

File: CustomRobots/vacuum_cleaner/models/vacuum_cleaner/vacuum_cleaner_gz.urdf.xacro (robot description, xacro)
@@ -85,7 +85,15 @@
     <gazebo>
       <plugin name="gz::sim::systems::Contact" filename="gz-sim-contact-system"></plugin>
-      <sensor name='${name}' type='contact'>
+      <sensor name='${name}_sensor' type='contact'>
         <contact>
-          <collision>collision</collision>
+          <collision>${name}</collision>
+          <topic>${topic}</topic>
+        </contact>
+        <always_on>1</always_on>
+        <update_rate>20</update_rate>
+      </sensor>
+      <!-- <sensor name='${name}' type='contact'>
+        <contact>
+          <collision>${name}</collision>
         </contact>
       </sensor>
@@ -95,5 +103,5 @@
         <time>0.001</time>
         <enabled>true</enabled>
-      </plugin>
+      </plugin> -->
     </gazebo>
   </xacro:macro>

Commit message: Test again

File: CustomRobots/vacuum_cleaner/models/vacuum_cleaner/vacuum_cleaner_common.urdf.xacro (robot description, xacro)
@@ -29,5 +29,5 @@
     </joint>
     <link name="right_bumper_link">
-      <collision name="right_bumper">
+      <collision>
         <origin rpy="0 0 0" xyz="0 0 0"/>
         <geometry>
@@ -35,5 +35,5 @@
         </geometry>
       </collision>
-      <xacro:bumper topic="/roombaROS/events/right_bumper" name="right_bumper"/>
+      <xacro:bumper topic="/roombaROS/events/right_bumper" name="right_bumper_link"/>
     </link>
     <joint name="center_bumper_joint" type="fixed">
@@ -43,5 +43,5 @@
     </joint>
     <link name="center_bumper_link">
-      <collision name="center_bumper">
+      <collision>
         <origin rpy="0 0 0" xyz="0 0 0"/>
         <geometry>
@@ -49,5 +49,5 @@
         </geometry>
       </collision>
-      <xacro:bumper topic="/roombaROS/events/center_bumper" name="center_bumper"/>
+      <xacro:bumper topic="/roombaROS/events/center_bumper" name="center_bumper_link"/>
     </link>
     <joint name="left_bumper_joint" type="fixed">
@@ -57,5 +57,5 @@
     </joint>
     <link name="left_bumper_link">
-      <collision name="left_bumper">
+      <collision>
         <origin rpy="0 0 0" xyz="0 0 0"/>
         <geometry>
@@ -63,5 +63,5 @@
         </geometry>
       </collision>
-      <xacro:bumper topic="/roombaROS/events/left_bumper" name="left_bumper"/>
+      <xacro:bumper topic="/roombaROS/events/left_bumper" name="left_bumper_link"/>
     </link>
     <joint name="front_wheel_joint" type="fixed">

File: CustomRobots/vacuum_cleaner/models/vacuum_cleaner/vacuum_cleaner_gz.urdf.xacro (robot description, xacro)
@@ -87,8 +87,8 @@
       <sensor name='${name}_sensor' type='contact'>
         <contact>
-          <collision>${name}</collision>
+          <collision>${name}_collision</collision>
           <topic>${topic}</topic>
         </contact>
-        <always_on>1</always_on>
+        <always_on>true</always_on>
         <update_rate>20</update_rate>
       </sensor>

Commit message: TEst again

File: CustomRobots/vacuum_cleaner/models/vacuum_cleaner/vacuum_cleaner_common.urdf.xacro (robot description, xacro)
@@ -35,5 +35,5 @@
         </geometry>
       </collision>
-      <xacro:bumper topic="/roombaROS/events/right_bumper" name="right_bumper_link"/>
+      <!-- <xacro:bumper topic="/roombaROS/events/right_bumper" name="right_bumper_link"/> -->
     </link>
     <joint name="center_bumper_joint" type="fixed">
@@ -49,5 +49,5 @@
         </geometry>
       </collision>
-      <xacro:bumper topic="/roombaROS/events/center_bumper" name="center_bumper_link"/>
+      <xacro:bumper topic="/roombaROS/events/center_bumper" name="center_bumper"/>
     </link>
     <joint name="left_bumper_joint" type="fixed">
@@ -63,5 +63,5 @@
         </geometry>
       </collision>
-      <xacro:bumper topic="/roombaROS/events/left_bumper" name="left_bumper_link"/>
+      <!-- <xacro:bumper topic="/roombaROS/events/left_bumper" name="left_bumper_link"/> -->
     </link>
     <joint name="front_wheel_joint" type="fixed">

File: CustomRobots/vacuum_cleaner/models/vacuum_cleaner/vacuum_cleaner_gz.urdf.xacro (robot description, xacro)
@@ -87,5 +87,5 @@
       <sensor name='${name}_sensor' type='contact'>
         <contact>
-          <collision>${name}_collision</collision>
+          <collision>${name}_link_collision</collision>
           <topic>${topic}</topic>
         </contact>

Commit message: Update gz

File: CustomRobots/vacuum_cleaner/models/vacuum_cleaner/vacuum_cleaner_common.urdf.xacro (robot description, xacro)
@@ -44,5 +44,4 @@
     <link name="center_bumper_link">
       <collision>
-        <origin rpy="0 0 0" xyz="0 0 0"/>
         <geometry>
           <mesh filename="$(find custom_robots)/models/vacuum_cleaner/meshes/center_bumper.dae"/>

File: CustomRobots/vacuum_cleaner/models/vacuum_cleaner/vacuum_cleaner_gz.urdf.xacro (robot description, xacro)
@@ -83,25 +83,20 @@
   </xacro:macro>
   <xacro:macro name="bumper" params="topic name">
-    <gazebo>
+    <gazebo reference="${name}_link">
+      <mu1>0.1</mu1>
+      <mu2>0.1</mu2>
+      <maxVel>0.01</maxVel>
+      <minDepth>0.001</minDepth>
+      <maxContacts>10</maxContacts>
+      <material>Gazebo/DarkGrey</material>
       <plugin name="gz::sim::systems::Contact" filename="gz-sim-contact-system"></plugin>
       <sensor name='${name}_sensor' type='contact'>
+        <always_on>true</always_on>
+        <update_rate>20</update_rate>
         <contact>
           <collision>${name}_link_collision</collision>
           <topic>${topic}</topic>
         </contact>
-        <always_on>true</always_on>
-        <update_rate>20</update_rate>
       </sensor>
-      <!-- <sensor name='${name}' type='contact'>
-        <contact>
-          <collision>${name}</collision>
-        </contact>
-      </sensor>
-      <plugin filename="gz-sim-touchplugin-system" name="gz::sim::systems::TouchPlugin">
-        <target>house_int2_harmonic</target>
-        <namespace>${topic}</namespace>
-        <time>0.001</time>
-        <enabled>true</enabled>
-      </plugin> -->
     </gazebo>
   </xacro:macro>

Commit message: Fix pose

File: CustomRobots/vacuum_cleaner/models/vacuum_cleaner/vacuum_cleaner_common.urdf.xacro (robot description, xacro)
@@ -129,5 +129,5 @@
     </link>
     <joint name="right_wheel_joint" type="continuous">
-      <origin rpy="0 0 0" xyz="0 0.13 0.032"/>
+      <origin rpy="0 0 0" xyz="0 -0.13 0.032"/>
       <parent link="base"/>
       <child link="right_wheel_link"/>

Commit message: Test again

File: CustomRobots/vacuum_cleaner/models/vacuum_cleaner/vacuum_cleaner_common.urdf.xacro (robot description, xacro)
@@ -47,6 +47,16 @@
         </geometry>
       </collision>
-      <xacro:bumper topic="/roombaROS/events/center_bumper" name="center_bumper"/>
+      <!-- <xacro:bumper topic="/roombaROS/events/center_bumper" name="center_bumper"/> -->
     </link>
+    <gazebo>
+      <sensor name="center_bumper" type="contact">
+        <always_on>true</always_on>
+        <update_rate>20.0</update_rate>
+        <contact>
+          <collision>center_bumper_collision</collision>
+          <topic>/roombaROS/events/center_bumper</topic>
+        </contact>
+      </sensor>
+    </gazebo>
     <joint name="left_bumper_joint" type="fixed">
       <origin rpy="0 0 0" xyz="-0.01 0 0.03"/>

File: CustomRobots/vacuum_cleaner/models/vacuum_cleaner/vacuum_cleaner_gz.urdf.xacro (robot description, xacro)
@@ -92,4 +92,12 @@
         </contact>
       </sensor>
+      <sensor name="${name}" type="contact">
+        <always_on>true</always_on>
+        <update_rate>20.0</update_rate>
+        <contact>
+          <collision>center_bumper_collision</collision>
+          <topic>/roombaROS/events/center_bumper</topic>
+        </contact>
+      </sensor>
     </gazebo>
   </xacro:macro>

Commit message: Remove bumpers

File: CustomRobots/vacuum_cleaner/models/vacuum_cleaner/vacuum_cleaner_common.urdf.xacro (robot description, xacro)
@@ -28,40 +28,40 @@
       <origin rpy="0 0 0" xyz="-0.01 0 0.03"/>
       <parent link="base"/>
-      <child link="right_bumper_link"/>
+      <child link="right_bumper"/>
     </joint>
-    <link name="right_bumper_link">
-      <collision name="right_bumper_collision">
+    <link name="right_bumper">
+      <collision>
         <geometry>
           <mesh filename="$(find custom_robots)/models/vacuum_cleaner/meshes/right_bumper.dae"/>
         </geometry>
       </collision>
-      <xacro:bumper topic="/roombaROS/events/right_bumper" name="right_bumper"/>
     </link>
+    <xacro:bumper topic="/roombaROS/events/right_bumper" name="right_bumper"/>
     <joint name="center_bumper_joint" type="fixed">
-      <origin rpy="0 0 0" xyz="-0.01 0 0.03"/>
+      <origin rpy="0 0 0" xyz="0.01 0 0.03"/>
       <parent link="base"/>
-      <child link="center_bumper_link"/>
+      <child link="center_bumper"/>
     </joint>
-    <link name="center_bumper_link">
-      <collision name="center_bumper_collision">
+    <link name="center_bumper">
+      <collision>
         <geometry>
           <mesh filename="$(find custom_robots)/models/vacuum_cleaner/meshes/center_bumper.dae"/>
         </geometry>
       </collision>
-      <xacro:bumper topic="/roombaROS/events/center_bumper" name="center_bumper"/>
     </link>
+    <xacro:bumper topic="/roombaROS/events/center_bumper" name="center_bumper"/>
     <joint name="left_bumper_joint" type="fixed">
       <origin rpy="0 0 0" xyz="-0.01 0 0.03"/>
       <parent link="base"/>
-      <child link="left_bumper_link"/>
+      <child link="left_bumper"/>
     </joint>
-    <link name="left_bumper_link">
-      <collision name="left_bumper_collision">
+    <link name="left_bumper">
+      <collision>
         <geometry>
           <mesh filename="$(find custom_robots)/models/vacuum_cleaner/meshes/left_bumper.dae"/>
         </geometry>
       </collision>
-      <xacro:bumper topic="/roombaROS/events/left_bumper" name="left_bumper"/>
     </link>
+    <xacro:bumper topic="/roombaROS/events/left_bumper" name="left_bumper"/>
     <joint name="front_wheel_joint" type="fixed">
       <origin rpy="0 1.570700 1.570700" xyz="0.13 0 0.017"/>
@@ -156,5 +156,5 @@
     <xacro:velocity topic="/roombaROS/cmd_vel"/>
     <xacro:odom topic="/roombaROS/odom" freq="20"/>
-    <xacro:noise_odom topic="/odom_noisy" vel_topic="/roombaROS/cmd_vel"/>
+    <xacro:noise_odom topic="/odom_noisy"/>
   </xacro:macro>
 </robot>

Commit message: Apply suggestion from @javizqh

File: CustomRobots/vacuum_cleaner/models/vacuum_cleaner/vacuum_cleaner_common.urdf.xacro (robot description, xacro)
@@ -39,5 +39,5 @@
     <xacro:bumper topic="/roombaROS/events/right_bumper" name="right_bumper"/>
     <joint name="center_bumper_joint" type="fixed">
-      <origin rpy="0 0 0" xyz="0.01 0 0.03"/>
+      <origin rpy="0 0 0" xyz="-0.01 0 0.03"/>
       <parent link="base"/>
       <child link="center_bumper"/>
