Commit message: Fix param

File: CustomRobots/vacuum_cleaner/models/vacuum_cleaner/vacuum_cleaner_gz.urdf.xacro (robot description, xacro)
@@ -119,5 +119,5 @@
     </gazebo>
   </xacro:macro>
-  <xacro:macro name="noise_odom" params="topic namespace">
+  <xacro:macro name="noise_odom" params="namespace">
     <gazebo>
       <plugin filename="libNoisyOdometryPlugin.so" name="custom_plugins::NoisyOdometryPlugin">

Commit message: Test custom bumper

File: CustomRobots/vacuum_cleaner/models/vacuum_cleaner/vacuum_cleaner_gz.urdf.xacro (robot description, xacro)
@@ -5,7 +5,7 @@
     <link name="${name}_link"></link>
     <joint name="${name}_to_${parent}" type="fixed">
-      <parent link="${parent}"/>
-      <child link="${name}_link"/>
-      <origin xyz="${xyz}" rpy="${rpy}"/>
+      <parent link="${parent}" />
+      <child link="${name}_link" />
+      <origin xyz="${xyz}" rpy="${rpy}" />
     </joint>
     <gazebo reference="${name}_link">
@@ -48,12 +48,13 @@
       <visual>
         <geometry>
-          <mesh filename="file://$(find custom_robots)/models/f1/meshes/hokuyo.dae" scale="0.1 0.1 0.1"/>
+          <mesh filename="file://$(find custom_robots)/models/f1/meshes/hokuyo.dae"
+            scale="0.1 0.1 0.1" />
         </geometry>
       </visual>
     </link>
     <joint name="${name}_to_${parent}" type="fixed">
-      <parent link="${parent}"/>
-      <child link="${name}_link"/>
-      <origin xyz="${xyz}" rpy="${rpy}"/>
+      <parent link="${parent}" />
+      <child link="${name}_link" />
+      <origin xyz="${xyz}" rpy="${rpy}" />
     </joint>
     <gazebo reference="${name}_link">
@@ -90,5 +91,5 @@
       <maxContacts>10</maxContacts>
       <material>Gazebo/DarkGrey</material>
-      <sensor name='${name}_contact_sensor' type='contact'>
+      <plugin filename="libBumperPlugin.so" name="custom_plugins::BumperPlugin">
         <always_on>true</always_on>
         <update_rate>100</update_rate>
@@ -98,5 +99,7 @@
           <topic>/${namespace}/${topic}</topic>
         </contact>
-      </sensor>
+      </plugin>
+      <!-- <sensor name='${name}_contact_sensor' type='contact'>
+      </sensor> -->
     </gazebo>
   </xacro:macro>
