Commit message: Change meshes

File: CustomRobots/Turtlebot2/model/turtlebot2/kobuki.urdf.xacro (robot description, xacro)
@@ -31,5 +31,5 @@
         <geometry>
           <!-- new mesh -->
-          <mesh filename="package://custom_robots/meshes/main_body.dae" />
+          <mesh filename="$(find custom_robots)/model/turtlebot2/meshes/main_body.dae" />
         </geometry>
         <origin xyz="0.001 0 0.05199" rpy="0 0 0"/>
@@ -65,5 +65,5 @@
       <visual>
         <geometry>
-          <mesh filename="package://custom_robots/meshes/wheel.dae"/>
+          <mesh filename="$(find custom_robots)/model/turtlebot2/meshes/wheel.dae"/>
         </geometry>
         <origin xyz="0 0 0" rpy="0 0 0"/>
@@ -90,5 +90,5 @@
       <visual>
         <geometry>
-          <mesh filename="package://custom_robots/meshes/wheel.dae"/>
+          <mesh filename="$(find custom_robots)/model/turtlebot2/meshes/wheel.dae"/>
         </geometry>
         <origin xyz="0 0 0" rpy="0 0 0"/>

Commit message: Fix t2

File: CustomRobots/Turtlebot2/model/turtlebot2/kobuki.urdf.xacro (robot description, xacro)
@@ -9,5 +9,45 @@
   xmlns:xacro="http://ros.org/wiki/xacro">
   <xacro:include filename="$(find custom_robots)/model/turtlebot2/common_properties.urdf.xacro"/>
-  <xacro:include filename="$(find custom_robots)/model/turtlebot2/kobuki_gazebo.urdf.xacro"/>
+  <xacro:include filename="$(find custom_robots)/model/turtlebot2/turtlebot2_gz.urdf.xacro"/>
+  <!-- Poles -->
+  <xacro:macro name="pole" parameters="parent name xyz height type">
+    <link name="pole_${name}">
+      <visual>
+        <geometry>
+          <mesh filename="$(find custom_robots)/model/turtlebot2/meshes/stacks/hexagons/pole_${type}.dae"/>
+        </geometry>
+      </visual>
+      <collision>
+        <geometry>
+          <box size="0.012 0.012 ${height}"/>
+        </geometry>
+      </collision>
+    </link>
+    <joint name="pole_${name}_to_${parent}" type="fixed">
+      <origin xyz="${xyz}" rpy="0 0 0" />
+      <parent link="${parent}"/>
+      <child link="pole_${name}" />
+    </joint>
+  </xacro:macro>
+  <!-- Plates -->
+  <xacro:macro name="plate" parameters="parent xyz type">
+    <link name="plate_${type}">
+      <visual>
+        <geometry>
+          <mesh filename="$(find custom_robots)/model/turtlebot2/meshes/stacks/hexagons/plate_${type}.dae"/>
+        </geometry>
+      </visual>
+      <collision>
+        <geometry>
+          <box size="0.34 0.34 0.006"/>
+        </geometry>
+      </collision>
+    </link>
+    <joint name="pole_${type}_to_${parent}" type="fixed">
+      <origin xyz="${xyz}" rpy="0 0 0" />
+      <parent link="${parent}"/>
+      <child link="pole_${type}" />
+    </joint>
+  </xacro:macro>
   <!-- Kobuki -->
   <xacro:macro name="kobuki">
@@ -142,4 +182,24 @@
       </inertial>
     </link>
+    <!-- Platform -->
+    <xacro:pole parent="base_link" name="0" xyz="0.12 0.082 0.113" height="0.0492" type="bottom"/>
+    <xacro:pole parent="base_link" name="1" xyz="0.055 0.12 0.113" height="0.0492" type="bottom"/>
+    <xacro:pole parent="base_link" name="2" xyz="-0.055 0.12 0.113" height="0.0492" type="bottom"/>
+    <xacro:pole parent="base_link" name="3" xyz="0.12 -0.082 0.113" height="0.0492" type="bottom"/>
+    <xacro:pole parent="base_link" name="4" xyz="0.055 -0.12 0.113" height="0.0492" type="bottom"/>
+    <xacro:pole parent="base_link" name="5" xyz="-0.055 -0.12 0.113" height="0.0492" type="bottom"/>
+    <xacro:pole parent="base_link" name="0" xyz="-0.1024 0.098 0.2474" height="0.0936" type="sensor"/>
+    <xacro:pole parent="base_link" name="1" xyz="-0.1024 -0.098 0.2474" height="0.0936" type="sensor"/>
+    <xacro:pole parent="base_link" name="0" xyz="0.0381 0.1505 0.1742" height="0.0608" type="middle"/>
+    <xacro:pole parent="base_link" name="1" xyz="0.0381 -0.1505 0.1742" height="0.0608" type="middle"/>
+    <xacro:pole parent="base_link" name="2" xyz="-0.0381 0.1505 0.1742" height="0.0608" type="middle"/>
+    <xacro:pole parent="base_link" name="3" xyz="-0.0381 -0.1505 0.1742" height="0.0608" type="middle"/>
+    <xacro:pole parent="base_link" name="0" xyz="0.0381 0.1505 0.3022" height="0.2032" type="top"/>
+    <xacro:pole parent="base_link" name="1" xyz="0.0381 -0.1505 0.3022" height="0.2032" type="top"/>
+    <xacro:pole parent="base_link" name="2" xyz="-0.0381 0.1505 0.3022" height="0.2032" type="top"/>
+    <xacro:pole parent="base_link" name="3" xyz="-0.0381 -0.1505 0.3022" height="0.2032" type="top"/>
+    <xacro:plate parent="base_link" xyz="0.02364 0 0.1408" type="bottom"/>
+    <xacro:plate parent="base_link" xyz="-0.01364 0 0.1976" type="middle"/>
+    <xacro:plate parent="base_link" xyz="-0.01364 0 0.4068" type="top"/>
     <!-- Kobuki's sensors -->
     <joint name="gyro_joint" type="fixed">
@@ -193,5 +253,11 @@
     </link>
     <!-- Kobuki Gazebo simulation details -->
-    <xacro:kobuki_sim/>
+    <!-- <xacro:kobuki_sim/> -->
+    <xacro:camera xyz="-0.118 0 0.2812" rpy="0 0 0" name="depth_camera" parent="base_link"/>
+    <xacro:laser xyz="0 0 0.44" rpy="0 0 0" name="laser" parent="base_link" topic="scan"/>
+    <xacro:odom topic="odom" freq="20"/>
+    <xacro:velocity topic="cmd_vel"/>
+    <xacro:imu topic="imu"/>
+    <xacro:extra/>
   </xacro:macro>
 </robot>

Commit message: Fix typo

File: CustomRobots/Turtlebot2/model/turtlebot2/kobuki.urdf.xacro (robot description, xacro)
@@ -11,5 +11,5 @@
   <xacro:include filename="$(find custom_robots)/model/turtlebot2/turtlebot2_gz.urdf.xacro"/>
   <!-- Poles -->
-  <xacro:macro name="pole" parameters="parent name xyz height type">
+  <xacro:macro name="pole" params="parent name xyz height type">
     <link name="pole_${name}">
       <visual>
@@ -31,5 +31,5 @@
   </xacro:macro>
   <!-- Plates -->
-  <xacro:macro name="plate" parameters="parent xyz type">
+  <xacro:macro name="plate" params="parent xyz type">
     <link name="plate_${type}">
       <visual>

Commit message: Fix unique

File: CustomRobots/Turtlebot2/model/turtlebot2/kobuki.urdf.xacro (robot description, xacro)
@@ -12,5 +12,5 @@
   <!-- Poles -->
   <xacro:macro name="pole" params="parent name xyz height type">
-    <link name="pole_${name}">
+    <link name="pole_${type}_${name}">
       <visual>
         <geometry>
@@ -24,8 +24,8 @@
       </collision>
     </link>
-    <joint name="pole_${name}_to_${parent}" type="fixed">
+    <joint name="pole_${type}_${name}_to_${parent}" type="fixed">
       <origin xyz="${xyz}" rpy="0 0 0" />
       <parent link="${parent}"/>
-      <child link="pole_${name}" />
+      <child link="pole_${type}_${name}" />
     </joint>
   </xacro:macro>

Commit message: Fix typo

File: CustomRobots/Turtlebot2/model/turtlebot2/kobuki.urdf.xacro (robot description, xacro)
@@ -44,8 +44,8 @@
       </collision>
     </link>
-    <joint name="pole_${type}_to_${parent}" type="fixed">
+    <joint name="plate_${type}_to_${parent}" type="fixed">
       <origin xyz="${xyz}" rpy="0 0 0" />
       <parent link="${parent}"/>
-      <child link="pole_${type}" />
+      <child link="plate_${type}" />
     </joint>
   </xacro:macro>
