Commit message: Fix stereo pose

File: CustomRobots/Turtlebot2/model/turtlebot2/turtlebot2.urdf.xacro (robot description, xacro)
@@ -12,7 +12,7 @@
   </xacro:if>
   <xacro:if value="$(arg stereo)">
-    <xacro:fake_camera xyz="-0.118 0 0.2812" rpy="0 0 0" name="depth_camera" parent="base_link"/>
-    <xacro:stereo_camera xyz="-0.05 0.076 0.2424" rpy="-1.57 0 3.14" name="cam_turtlebot_left" parent="base_link"/>
-    <xacro:stereo_camera xyz="-0.05 -0.076 0.2424" rpy="-1.57 0 3.14" name="cam_turtlebot_right" parent="base_link"/>
+    <xacro:fake_camera xyz="-0.118 0 0.23" rpy="0 0 0" name="depth_camera" parent="base_link"/>
+    <xacro:stereo_camera xyz="-0.05 0.076 0.2424" rpy="0 0 0" name="cam_turtlebot_left" parent="base_link"/>
+    <xacro:stereo_camera xyz="-0.05 -0.076 0.2424" rpy="0 0 0" name="cam_turtlebot_right" parent="base_link"/>
   </xacro:if>
 </robot>

File: CustomRobots/Turtlebot2/model/turtlebot2/turtlebot2_gz.urdf.xacro (robot description, xacro)
@@ -63,5 +63,4 @@
     <gazebo reference="${name}_link">
       <sensor name="${name}" type="camera">
-        <origin xyz="0 0 0" rpy="-1.57 0 3.14"/>
         <always_on>true</always_on>
         <visualize>false</visualize>
