Commit message: Update turtlebot2

File: CustomRobots/Turtlebot2/model/turtlebot2/turtlebot2.urdf.xacro (robot description, xacro)
@@ -4,15 +4,17 @@
   <xacro:arg name="camera" default="true"/>
   <xacro:arg name="stereo" default="false"/>
+  <xacro:arg name="namespace" default="turtlebot2"/>
+  <xacro:property name="namespace" value="$(arg namespace)"/>
   <xacro:include filename="$(find custom_robots)/model/turtlebot2/turtlebot2_gz.urdf.xacro"/>
   <xacro:include filename="$(find custom_robots)/model/turtlebot2/turtlebot2_common.urdf.xacro"/>
-  <xacro:turtlebot2/>
+  <xacro:turtlebot2 namespace="${namespace}"/>
   <xacro:if value="$(arg camera)">
-    <xacro:camera xyz="-0.118 0 0.2812" rpy="0 0 0" name="depth_camera" parent="base_link"/>
-    <xacro:laser xyz="0 0 0.44" rpy="0 0 0" name="laser" parent="base_link" topic="scan"/>
+    <xacro:camera xyz="-0.118 0 0.2812" rpy="0 0 0" name="camera" parent="base_link" namespace="${namespace}"/>
+    <xacro:laser xyz="0 0 0.44" rpy="0 0 0" name="laser" parent="base_link" namespace="${namespace}"/>
   </xacro:if>
   <xacro:if value="$(arg stereo)">
     <xacro:fake_camera xyz="-0.118 0 0.23" rpy="0 0 0" name="depth_camera" parent="base_link"/>
-    <xacro:stereo_camera xyz="-0.05 0.076 0.2424" rpy="0 0 0" name="cam_turtlebot_left" parent="base_link"/>
-    <xacro:stereo_camera xyz="-0.05 -0.076 0.2424" rpy="0 0 0" name="cam_turtlebot_right" parent="base_link"/>
+    <xacro:stereo_camera xyz="-0.05 0.076 0.2424" rpy="0 0 0" name="camera_left" parent="base_link" namespace="${namespace}"/>
+    <xacro:stereo_camera xyz="-0.05 -0.076 0.2424" rpy="0 0 0" name="camera_right" parent="base_link" namespace="${namespace}"/>
   </xacro:if>
 </robot>

File: CustomRobots/Turtlebot2/model/turtlebot2/turtlebot2_common.urdf.xacro (robot description, xacro)
@@ -51,5 +51,5 @@
   </xacro:macro>
   <!-- Kobuki -->
-  <xacro:macro name="turtlebot2">
+  <xacro:macro name="turtlebot2" params="namespace">
     <link name="base_footprint"/>
     <!--
@@ -253,7 +253,7 @@
     </link>
     <!-- Kobuki Gazebo simulation details -->
-    <xacro:odom topic="odom" freq="20"/>
-    <xacro:velocity topic="cmd_vel"/>
-    <xacro:imu topic="imu"/>
+    <xacro:odom namespace="${namespace}" freq="20"/>
+    <xacro:velocity namespace="${namespace}"/>
+    <xacro:imu namespace="${namespace}"/>
     <xacro:extra/>
   </xacro:macro>

File: CustomRobots/Turtlebot2/model/turtlebot2/turtlebot2_gz.urdf.xacro (robot description, xacro)
@@ -2,5 +2,5 @@
 <robot name="vacuum_cleaner_gz"
   xmlns:xacro="http://ros.org/wiki/xacro">
-  <xacro:macro name="camera" params="xyz rpy name parent">
+  <xacro:macro name="camera" params="xyz rpy name parent namespace">
     <link name="${name}_link">
       <visual>
@@ -21,7 +21,7 @@
         <visualize>false</visualize>
         <update_rate>5</update_rate>
-        <topic>/${name}/image_raw</topic>
+        <topic>/${namespace}/${name}/image_raw</topic>
         <camera name="camera">
-          <camera_info_topic>/${name}/camera_info</camera_info_topic>
+          <camera_info_topic>/${namespace}/${name}/camera_info</camera_info_topic>
           <horizontal_fov>1.0472</horizontal_fov>
           <image>
@@ -53,5 +53,5 @@
     </joint>
   </xacro:macro>
-  <xacro:macro name="stereo_camera" params="xyz rpy name parent">
+  <xacro:macro name="stereo_camera" params="xyz rpy name parent namespace">
     <link name="${name}_link">
     </link>
@@ -66,7 +66,7 @@
         <visualize>false</visualize>
         <update_rate>5</update_rate>
-        <topic>/${name}/image_raw</topic>
+        <topic>/${namespace}/${name}/image_raw</topic>
         <camera name="camera">
-          <camera_info_topic>/${name}/camera_info</camera_info_topic>
+          <camera_info_topic>/${namespace}/${name}/camera_info</camera_info_topic>
           <horizontal_fov>1.570000</horizontal_fov>
           <image>
@@ -88,5 +88,5 @@
     </gazebo>
   </xacro:macro>
-  <xacro:macro name="laser" params="xyz rpy name parent topic">
+  <xacro:macro name="laser" params="xyz rpy name parent namespace">
     <link name="${name}_link">
       <visual>
@@ -106,5 +106,5 @@
         <visualize>1</visualize>
         <update_rate>5</update_rate>
-        <topic>${topic}</topic>
+        <topic>/${namespace}/${name}/scan</topic>
         <gz_frame_id>laser</gz_frame_id>
         <lidar>
@@ -126,5 +126,5 @@
     </gazebo>
   </xacro:macro>
-  <xacro:macro name="bumper" params="topic name">
+  <xacro:macro name="bumper" params="topic name namespace">
     <gz>
       <sensor name='${name}' type='contact'>
@@ -133,10 +133,10 @@
         <contact>
           <collision>${name}_collision</collision>
-          <topic>${topic}</topic>
+          <topic>/${namespace}/${topic}</topic>
         </contact>
       </sensor>
     </gz>
   </xacro:macro>
-  <xacro:macro name="imu" params="topic">
+  <xacro:macro name="imu" params="namespace">
     <gazebo>
       <plugin filename="gz-sim-imu-system" name="gz::sim::systems::Imu">
@@ -146,5 +146,5 @@
           <always_on>1</always_on>
           <update_rate>50</update_rate>
-          <topic>${topic}</topic>
+          <topic>/${namespace}/imu</topic>
           <imu>
             <noise>
@@ -202,5 +202,5 @@
     </gazebo>
   </xacro:macro>
-  <xacro:macro name="velocity" params="topic">
+  <xacro:macro name="velocity" params="namespace">
     <gazebo>
       <plugin filename="gz-sim-diff-drive-system" name="gz::sim::systems::DiffDrive">
@@ -210,9 +210,9 @@
         <wheel_separation>.230</wheel_separation>
         <wheel_diameter>0.070</wheel_diameter>
-        <topic>${topic}</topic>
+        <topic>/${namespace}/cmd_vel</topic>
       </plugin>
     </gazebo>
   </xacro:macro>
-  <xacro:macro name="odom" params="topic freq">
+  <xacro:macro name="odom" params="namespace freq">
     <gazebo>
       <plugin filename="gz-sim-odometry-publisher-system" name="gz::sim::systems::OdometryPublisher">
@@ -220,5 +220,5 @@
         <robot_base_frame>base_footprint</robot_base_frame>
         <odom_publish_frequency>${freq}</odom_publish_frequency>
-        <odom_topic>${topic}</odom_topic>
+        <odom_topic>/${namespace}/odom</odom_topic>
         <dimensions>3</dimensions>
       </plugin>
