Commit message: Fix typo

File: CustomRobots/logistic_holonomic_robot/models/logistic_holonomic_robot/logistic_holonomic_robot_common.urdf.xacro (robot description, xacro)
@@ -37,5 +37,5 @@
     <link name="left_wheel_link">
       <inertial>
-        <origin rpy="-1.57 0 0<" xyz="0.0 0.288 0.046"/>
+        <origin rpy="-1.57 0 0" xyz="0.0 0.288 0.046"/>
         <mass value="0.1"/>
         <inertia ixx="0.001" ixy="0" ixz="0" iyy="0.001" iyz="0" izz="0.001"/>

Commit message: Fix more typos

File: CustomRobots/logistic_holonomic_robot/models/logistic_holonomic_robot/logistic_holonomic_robot_common.urdf.xacro (robot description, xacro)
@@ -42,5 +42,5 @@
       </inertial>
       <collision>
-        <origin rpy="-1.57 0 0<" xyz="0.0 0.288 0.046"/>
+        <origin rpy="-1.57 0 0" xyz="0.0 0.288 0.046"/>
         <geometry>
           <cylinder radius="0.1" lenght="0.02"/>
@@ -84,10 +84,10 @@
     <link name="right_wheel_link">
       <inertial>
-        <origin rpy="-1.57 0 0<" xyz="0.0 -0.288 0.046"/>
-        <mass value="0.1"/>
-        <inertia ixx="0.001" ixy="0" ixz="0" iyy="0.001" iyz="0" izz="0.001"/>
-      </inertial>
-      <collision>
-        <origin rpy="-1.57 0 0<" xyz="0.0 -0.288 0.046"/>
+        <origin rpy="-1.57 0 0" xyz="0.0 -0.288 0.046"/>
+        <mass value="0.1"/>
+        <inertia ixx="0.001" ixy="0" ixz="0" iyy="0.001" iyz="0" izz="0.001"/>
+      </inertial>
+      <collision>
+        <origin rpy="-1.57 0 0" xyz="0.0 -0.288 0.046"/>
         <geometry>
           <cylinder radius="0.1" lenght="0.02"/>

Commit message: Test logistic

File: CustomRobots/logistic_holonomic_robot/models/logistic_holonomic_robot/logistic_holonomic_robot_common.urdf.xacro (robot description, xacro)
@@ -46,25 +46,27 @@
           <cylinder radius="0.1" lenght="0.02"/>
         </geometry>
-        <surface>
-          <friction>
-            <ode>
-              <mu>10.0</mu>
-              <mu2>10.0</mu2>
-              <fdir1>0 0 0</fdir1>
-              <slip1>0.0</slip1>
-              <slip2>0.0</slip2>
-            </ode>
-          </friction>
-          <contact>
-            <ode>
-              <soft_cfm>0.001</soft_cfm>
-              <soft_erp>0.5</soft_erp>
-              <kp>1e+5</kp>
-              <kd>1</kd>
-              <max_vel>0.01</max_vel>
-              <min_depth>0.001</min_depth>
-            </ode>
-          </contact>
-        </surface>
+        <gz>
+          <surface>
+            <friction>
+              <ode>
+                <mu>10.0</mu>
+                <mu2>10.0</mu2>
+                <fdir1>0 0 0</fdir1>
+                <slip1>0.0</slip1>
+                <slip2>0.0</slip2>
+              </ode>
+            </friction>
+            <contact>
+              <ode>
+                <soft_cfm>0.001</soft_cfm>
+                <soft_erp>0.5</soft_erp>
+                <kp>1e+5</kp>
+                <kd>1</kd>
+                <max_vel>0.01</max_vel>
+                <min_depth>0.001</min_depth>
+              </ode>
+            </contact>
+          </surface>
+        </gz>
       </collision>
       <visual>
@@ -93,25 +95,27 @@
           <cylinder radius="0.1" lenght="0.02"/>
         </geometry>
-        <surface>
-          <friction>
-            <ode>
-              <mu>10.0</mu>
-              <mu2>10.0</mu2>
-              <fdir1>0 0 0</fdir1>
-              <slip1>0.0</slip1>
-              <slip2>0.0</slip2>
-            </ode>
-          </friction>
-          <contact>
-            <ode>
-              <soft_cfm>0.001</soft_cfm>
-              <soft_erp>0.5</soft_erp>
-              <kp>1e+5</kp>
-              <kd>1</kd>
-              <max_vel>0.01</max_vel>
-              <min_depth>0.001</min_depth>
-            </ode>
-          </contact>
-        </surface>
+        <gz>
+          <surface>
+            <friction>
+              <ode>
+                <mu>10.0</mu>
+                <mu2>10.0</mu2>
+                <fdir1>0 0 0</fdir1>
+                <slip1>0.0</slip1>
+                <slip2>0.0</slip2>
+              </ode>
+            </friction>
+            <contact>
+              <ode>
+                <soft_cfm>0.001</soft_cfm>
+                <soft_erp>0.5</soft_erp>
+                <kp>1e+5</kp>
+                <kd>1</kd>
+                <max_vel>0.01</max_vel>
+                <min_depth>0.001</min_depth>
+              </ode>
+            </contact>
+          </surface>
+        </gz>
       </collision>
       <visual>
@@ -122,5 +126,5 @@
       </visual>
     </link>
-    <joint name="back_right_caster_joint" type="ball">
+    <joint name="back_right_caster_joint" type="fixed">
       <origin rpy="0 0 0" xyz="-0.29 -0.13 -0.0275"/>
       <parent link="base"/>
@@ -137,24 +141,26 @@
           <sphere radius="0.025"/>
         </geometry>
-        <surface>
-          <contact>
-            <ode>
-              <soft_cfm>0</soft_cfm>
-              <soft_erp>0.2</soft_erp>
-              <kp>1e+5</kp>
-              <kd>1</kd>
-              <max_vel>0.01</max_vel>
-              <min_depth>0.001</min_depth>
-            </ode>
-          </contact>
-        </surface>
-      </collision>
-      <visual>
-        <geometry>
-          <sphere radius="0.025"/>
-        </geometry>
-      </visual>
-    </link>
-    <joint name="back_left_caster_joint" type="ball">
+        <gz>
+          <surface>
+            <contact>
+              <ode>
+                <soft_cfm>0</soft_cfm>
+                <soft_erp>0.2</soft_erp>
+                <kp>1e+5</kp>
+                <kd>1</kd>
+                <max_vel>0.01</max_vel>
+                <min_depth>0.001</min_depth>
+              </ode>
+            </contact>
+          </surface>
+        </gz>
+      </collision>
+      <visual>
+        <geometry>
+          <sphere radius="0.025"/>
+        </geometry>
+      </visual>
+    </link>
+    <joint name="back_left_caster_joint" type="fixed">
       <origin rpy="0 0 0" xyz="-0.29  0.13 -0.0275"/>
       <parent link="base"/>
@@ -171,16 +177,18 @@
           <sphere radius="0.025"/>
         </geometry>
-        <surface>
-          <contact>
-            <ode>
-              <soft_cfm>0</soft_cfm>
-              <soft_erp>0.2</soft_erp>
-              <kp>1e+5</kp>
-              <kd>1</kd>
-              <max_vel>0.01</max_vel>
-              <min_depth>0.001</min_depth>
-            </ode>
-          </contact>
-        </surface>
+        <gz>
+          <surface>
+            <contact>
+              <ode>
+                <soft_cfm>0</soft_cfm>
+                <soft_erp>0.2</soft_erp>
+                <kp>1e+5</kp>
+                <kd>1</kd>
+                <max_vel>0.01</max_vel>
+                <min_depth>0.001</min_depth>
+              </ode>
+            </contact>
+          </surface>
+        </gz>
       </collision>
       <visual>
@@ -248,25 +256,27 @@
           <box size="0.55 0.55 0.04"/>
         </geometry>
-        <surface>
-          <friction>
-            <ode>
-              <mu>1000000</mu>
-              <mu2>100000</mu2>
-              <fdir1>0 0 0</fdir1>
-              <slip1>0.0</slip1>
-              <slip2>0.0</slip2>
-            </ode>
-          </friction>
-          <contact>
-            <ode>
-              <soft_cfm>0</soft_cfm>
-              <soft_erp>0.2</soft_erp>
-              <kp>1e+5</kp>
-              <kd>1</kd>
-              <max_vel>0.01</max_vel>
-              <min_depth>0.001</min_depth>
-            </ode>
-          </contact>
-        </surface>
+        <gz>
+          <surface>
+            <friction>
+              <ode>
+                <mu>1000000</mu>
+                <mu2>100000</mu2>
+                <fdir1>0 0 0</fdir1>
+                <slip1>0.0</slip1>
+                <slip2>0.0</slip2>
+              </ode>
+            </friction>
+            <contact>
+              <ode>
+                <soft_cfm>0</soft_cfm>
+                <soft_erp>0.2</soft_erp>
+                <kp>1e+5</kp>
+                <kd>1</kd>
+                <max_vel>0.01</max_vel>
+                <min_depth>0.001</min_depth>
+              </ode>
+            </contact>
+          </surface>
+        </gz>
       </collision>
       <visual>

Commit message: Fix jpint

File: CustomRobots/logistic_holonomic_robot/models/logistic_holonomic_robot/logistic_holonomic_robot_common.urdf.xacro (robot description, xacro)
@@ -44,5 +44,5 @@
         <origin rpy="-1.57 0 0" xyz="0.0 0.288 0.046"/>
         <geometry>
-          <cylinder radius="0.1" lenght="0.02"/>
+          <cylinder radius="0.1" length="0.02"/>
         </geometry>
         <gz>
@@ -93,5 +93,5 @@
         <origin rpy="-1.57 0 0" xyz="0.0 -0.288 0.046"/>
         <geometry>
-          <cylinder radius="0.1" lenght="0.02"/>
+          <cylinder radius="0.1" length="0.02"/>
         </geometry>
         <gz>
@@ -218,31 +218,20 @@
       <parent link="platform_link"/>
       <child link="platform_support_link"/>
-      <axis>
-        <xyz>0 0 1</xyz>
-        <limit>
-          <lower>0.01</lower>
-          <upper>0.13</upper>
-          <effort>20</effort>
-          <velocity>0.5</velocity>
-        </limit>
-        <dynamics>
-          <damping>1.0</damping>
-          <friction>0</friction>
-          <spring_reference>0</spring_reference>
-          <spring_stiffness>0</spring_stiffness>
-        </dynamics>
-        <use_parent_model_frame>0</use_parent_model_frame>
-      </axis>
-      <physics>
-        <provide_feedback>1</provide_feedback>
-        <ode>
-          <implicit_spring_damper>0</implicit_spring_damper>
-          <cfm_damping>0</cfm_damping>
-          <limit>
-            <cfm>0.0</cfm>
-            <erp>0.8</erp>
-          </limit>
-        </ode>
-      </physics>
+      <axis xyz="0 0 1"/>
+      <limit effort="20" velocity="0.5" lower="0.01" upper="0.13"/>
+      <dynamics damping="0.01" friction="0" spring_reference="0" spring_stiffness="0"/>
+      <gz>
+        <physics>
+          <provide_feedback>1</provide_feedback>
+          <ode>
+            <implicit_spring_damper>0</implicit_spring_damper>
+            <cfm_damping>0</cfm_damping>
+            <limit>
+              <cfm>0.0</cfm>
+              <erp>0.8</erp>
+            </limit>
+          </ode>
+        </physics>
+      </gz>
     </joint>
     <link name="platform_link">

Commit message: Fix joint

File: CustomRobots/logistic_holonomic_robot/models/logistic_holonomic_robot/logistic_holonomic_robot_common.urdf.xacro (robot description, xacro)
@@ -198,10 +198,10 @@
       </visual>
     </link>
-    <joint name="platform_support_link" type="fixed">
+    <joint name="platform_support_joint" type="fixed">
       <origin rpy="0 0 0" xyz="-0.02 0.0 0.2"/>
       <parent link="base"/>
       <child link="platform_support_link"/>
     </joint>
-    <link name="platform_support_joint">
+    <link name="platform_support_link">
       <inertial>
         <mass value="0.1"/>

Commit message: Fix joint

File: CustomRobots/logistic_holonomic_robot/models/logistic_holonomic_robot/logistic_holonomic_robot_common.urdf.xacro (robot description, xacro)
@@ -216,6 +216,6 @@
     <joint name="lift_joint" type="prismatic">
       <origin rpy="0 0 0" xyz="-0.02 0.0 0.2"/>
-      <parent link="platform_link"/>
-      <child link="platform_support_link"/>
+      <parent link="platform_support_link"/>
+      <child link="platform_link"/>
       <axis xyz="0 0 1"/>
       <limit effort="20" velocity="0.5" lower="0.01" upper="0.13"/>

Commit message: Fix meshes

File: CustomRobots/logistic_holonomic_robot/models/logistic_holonomic_robot/logistic_holonomic_robot_common.urdf.xacro (robot description, xacro)
@@ -6,10 +6,8 @@
     <link name="base">
       <inertial>
-        <origin rpy="0 0 0" xyz="0 0 0"/>
         <mass value="1.5"/>
         <inertia ixx="0.001" ixy="0" ixz="0" iyy="0.001" iyz="0" izz="0.001"/>
       </inertial>
       <collision>
-        <origin rpy="0 0 0" xyz="0 0 0.045"/>
         <geometry>
           <box size="0.532 0.532 0.188"/>
@@ -17,5 +15,4 @@
       </collision>
       <visual>
-        <origin rpy="0 0 0" xyz="0 0 -0.048"/>
         <geometry>
           <mesh filename="$(find custom_robots)/models/logistic_holonomic_robot/meshes/waffle_pi_base.dae" scale="0.002 0.002 0.002"/>
@@ -24,23 +21,21 @@
     </link>
     <joint name="base_to_base_footprint" type="fixed">
-      <origin rpy="0 0 0" xyz="-0.064 0 0.048"/>
+      <origin rpy="0 0 0" xyz="0 0 0.048"/>
       <parent link="base_footprint"/>
       <child link="base"/>
     </joint>
     <joint name="left_wheel_joint" type="continuous">
-      <origin rpy="-1.57 0 0" xyz="0.0 0.288 0.046"/>
+      <origin rpy="0 0 0" xyz="0.127 0.288 0.046"/>
       <parent link="base"/>
       <child link="left_wheel_link"/>
-      <axis xyz="0 1 0"/>
+      <axis xyz="0 0 1"/>
       <limit effort="1000" velocity="100"/>
     </joint>
     <link name="left_wheel_link">
       <inertial>
-        <origin rpy="-1.57 0 0" xyz="0.0 0.288 0.046"/>
-        <mass value="0.1"/>
-        <inertia ixx="0.001" ixy="0" ixz="0" iyy="0.001" iyz="0" izz="0.001"/>
-      </inertial>
-      <collision>
-        <origin rpy="-1.57 0 0" xyz="0.0 0.288 0.046"/>
+        <mass value="0.1"/>
+        <inertia ixx="0.001" ixy="0" ixz="0" iyy="0.001" iyz="0" izz="0.001"/>
+      </inertial>
+      <collision>
         <geometry>
           <cylinder radius="0.1" length="0.02"/>
@@ -71,5 +66,4 @@
       </collision>
       <visual>
-        <origin rpy="0 0 0" xyz="0.0 0.288 0.046"/>
         <geometry>
           <mesh filename="$(find custom_robots)/models/logistic_holonomic_robot/meshes/left_tire.dae" scale="0.003 0.003 0.003"/>
@@ -78,18 +72,16 @@
     </link>
     <joint name="right_wheel_joint" type="continuous">
-      <origin rpy="-1.57 0 0" xyz="0.0 -0.288 0.046"/>
+      <origin rpy="0 0 0" xyz="0.127 -0.288 0.046"/>
       <parent link="base"/>
       <child link="right_wheel_link"/>
-      <axis xyz="0 1 0"/>
+      <axis xyz="0 0 1"/>
       <limit effort="1000" velocity="100"/>
     </joint>
     <link name="right_wheel_link">
       <inertial>
-        <origin rpy="-1.57 0 0" xyz="0.0 -0.288 0.046"/>
-        <mass value="0.1"/>
-        <inertia ixx="0.001" ixy="0" ixz="0" iyy="0.001" iyz="0" izz="0.001"/>
-      </inertial>
-      <collision>
-        <origin rpy="-1.57 0 0" xyz="0.0 -0.288 0.046"/>
+        <mass value="0.1"/>
+        <inertia ixx="0.001" ixy="0" ixz="0" iyy="0.001" iyz="0" izz="0.001"/>
+      </inertial>
+      <collision>
         <geometry>
           <cylinder radius="0.1" length="0.02"/>
@@ -120,5 +112,4 @@
       </collision>
       <visual>
-        <origin rpy="0 0 0" xyz="0.0 -0.288 0.046"/>
         <geometry>
           <mesh filename="$(find custom_robots)/models/logistic_holonomic_robot/meshes/right_tire.dae" scale="0.003 0.003 0.003"/>
@@ -127,5 +118,5 @@
     </link>
     <joint name="back_right_caster_joint" type="fixed">
-      <origin rpy="0 0 0" xyz="-0.29 -0.13 -0.0275"/>
+      <origin rpy="0 0 0" xyz="-0.23 -0.13 -0.0275"/>
       <parent link="base"/>
       <child link="back_right_caster_link"/>
@@ -133,5 +124,4 @@
     <link name="back_right_caster_link">
       <inertial>
-        <origin rpy="0 0 0" xyz="0 0 0"/>
         <mass value="0.8"/>
         <inertia ixx="0.00001" ixy="0" ixz="0" iyy="0.00001" iyz="0" izz="0.00001"/>
@@ -163,5 +153,5 @@
     </link>
     <joint name="back_left_caster_joint" type="fixed">
-      <origin rpy="0 0 0" xyz="-0.29  0.13 -0.0275"/>
+      <origin rpy="0 0 0" xyz="-0.23  0.13 -0.0275"/>
       <parent link="base"/>
       <child link="back_left_caster_link"/>
@@ -169,5 +159,4 @@
     <link name="back_left_caster_link">
       <inertial>
-        <origin rpy="0 0 0" xyz="0 0 0"/>
         <mass value="0.8"/>
         <inertia ixx="0.00001" ixy="0" ixz="0" iyy="0.00001" iyz="0" izz="0.00001"/>
@@ -215,5 +204,5 @@
     </link>
     <joint name="lift_joint" type="prismatic">
-      <origin rpy="0 0 0" xyz="-0.02 0.0 0.2"/>
+      <origin rpy="0 0 0" xyz="0 0.0 0.09"/>
       <parent link="platform_support_link"/>
       <child link="platform_link"/>

Commit message: Fix wheels

File: CustomRobots/logistic_holonomic_robot/models/logistic_holonomic_robot/logistic_holonomic_robot_common.urdf.xacro (robot description, xacro)
@@ -10,4 +10,5 @@
       </inertial>
       <collision>
+        <origin rpy="0 0 0" xyz="0 0 0.07"/>
         <geometry>
           <box size="0.532 0.532 0.188"/>
@@ -26,5 +27,5 @@
     </joint>
     <joint name="left_wheel_joint" type="continuous">
-      <origin rpy="0 0 0" xyz="0.127 0.288 0.046"/>
+      <origin rpy="-1.57 0 0" xyz="0.127 0.288 0.046"/>
       <parent link="base"/>
       <child link="left_wheel_link"/>
@@ -66,4 +67,5 @@
       </collision>
       <visual>
+        <origin rpy="1.57 0 0" xyz="0 0 0"/>
         <geometry>
           <mesh filename="$(find custom_robots)/models/logistic_holonomic_robot/meshes/left_tire.dae" scale="0.003 0.003 0.003"/>
@@ -72,5 +74,5 @@
     </link>
     <joint name="right_wheel_joint" type="continuous">
-      <origin rpy="0 0 0" xyz="0.127 -0.288 0.046"/>
+      <origin rpy="-1.57 0 0" xyz="0.127 -0.288 0.046"/>
       <parent link="base"/>
       <child link="right_wheel_link"/>
@@ -112,4 +114,5 @@
       </collision>
       <visual>
+        <origin rpy="1.57 0 0" xyz="0 0 0"/>
         <geometry>
           <mesh filename="$(find custom_robots)/models/logistic_holonomic_robot/meshes/right_tire.dae" scale="0.003 0.003 0.003"/>
@@ -117,5 +120,5 @@
       </visual>
     </link>
-    <joint name="back_right_caster_joint" type="fixed">
+    <!-- <joint name="back_right_caster_joint" type="fixed">
       <origin rpy="0 0 0" xyz="-0.23 -0.13 -0.0275"/>
       <parent link="base"/>
@@ -186,5 +189,5 @@
         </geometry>
       </visual>
-    </link>
+    </link> -->
     <joint name="platform_support_joint" type="fixed">
       <origin rpy="0 0 0" xyz="-0.02 0.0 0.2"/>

Commit message: Fix spawn

File: CustomRobots/logistic_holonomic_robot/models/logistic_holonomic_robot/logistic_holonomic_robot_common.urdf.xacro (robot description, xacro)
@@ -27,5 +27,5 @@
     </joint>
     <joint name="left_wheel_joint" type="continuous">
-      <origin rpy="-1.57 0 0" xyz="0.127 0.288 0.046"/>
+      <origin rpy="-1.57 0 0" xyz="0 0.288 0.046"/>
       <parent link="base"/>
       <child link="left_wheel_link"/>
@@ -74,5 +74,5 @@
     </link>
     <joint name="right_wheel_joint" type="continuous">
-      <origin rpy="-1.57 0 0" xyz="0.127 -0.288 0.046"/>
+      <origin rpy="-1.57 0 0" xyz="0 -0.288 0.046"/>
       <parent link="base"/>
       <child link="right_wheel_link"/>

Commit message: Fix wheels pose

File: CustomRobots/logistic_holonomic_robot/models/logistic_holonomic_robot/logistic_holonomic_robot_common.urdf.xacro (robot description, xacro)
@@ -27,5 +27,5 @@
     </joint>
     <joint name="left_wheel_joint" type="continuous">
-      <origin rpy="-1.57 0 0" xyz="0 0.288 0.046"/>
+      <origin rpy="-1.57 0 0" xyz="0.05 0.288 0.046"/>
       <parent link="base"/>
       <child link="left_wheel_link"/>
@@ -74,5 +74,5 @@
     </link>
     <joint name="right_wheel_joint" type="continuous">
-      <origin rpy="-1.57 0 0" xyz="0 -0.288 0.046"/>
+      <origin rpy="-1.57 0 0" xyz="0.05 -0.288 0.046"/>
       <parent link="base"/>
       <child link="right_wheel_link"/>
@@ -120,9 +120,27 @@
       </visual>
     </link>
-    <!-- <joint name="back_right_caster_joint" type="fixed">
+    <joint name="back_right_caster_joint_roll" type="continuous">
       <origin rpy="0 0 0" xyz="-0.23 -0.13 -0.0275"/>
       <parent link="base"/>
       <child link="back_right_caster_link"/>
-    </joint>
+      <axis xyz="1 0 0"/>
+      <limit effort="1000" velocity="100"/>
+    </joint>
+    <!-- <link name="back_right_caster_roll_link"/>
+    <joint name="back_right_caster_joint_pitch" type="continuous">
+      <origin rpy="0 0 0" xyz="0 0 0"/>
+      <parent link="back_right_caster_roll_link"/>
+      <child link="back_right_caster_pitch_link"/>
+      <axis xyz="0 1 0"/>
+      <limit effort="1000" velocity="100"/>
+    </joint>
+    <link name="back_right_caster_pitch_link"/>
+    <joint name="back_right_caster_joint_yaw" type="continuous">
+      <origin rpy="0 0 0" xyz="0 0 0"/>
+      <parent link="back_right_caster_pitch_link"/>
+      <child link="back_right_caster_link"/>
+      <axis xyz="0 0 1"/>
+      <limit effort="1000" velocity="100"/>
+    </joint> -->
     <link name="back_right_caster_link">
       <inertial>
@@ -155,9 +173,27 @@
       </visual>
     </link>
-    <joint name="back_left_caster_joint" type="fixed">
+    <joint name="back_left_caster_joint_roll" type="continuous">
       <origin rpy="0 0 0" xyz="-0.23  0.13 -0.0275"/>
       <parent link="base"/>
       <child link="back_left_caster_link"/>
-    </joint>
+      <axis xyz="0 0 1"/>
+      <limit effort="1000" velocity="100"/>
+    </joint>
+    <!-- <link name="back_left_caster_roll_link"/>
+    <joint name="back_left_caster_joint_pitch" type="continuous">
+      <origin rpy="0 0 0" xyz="0 0 0"/>
+      <parent link="back_left_caster_roll_link"/>
+      <child link="back_left_caster_pitch_link"/>
+      <axis xyz="0 1 0"/>
+      <limit effort="1000" velocity="100"/>
+    </joint>
+    <link name="back_left_caster_pitch_link"/>
+    <joint name="back_left_caster_joint_yaw" type="continuous">
+      <origin rpy="0 0 0" xyz="0 0 0"/>
+      <parent link="back_left_caster_pitch_link"/>
+      <child link="back_left_caster_link"/>
+      <axis xyz="1 0 0"/>
+      <limit effort="1000" velocity="100"/>
+    </joint> -->
     <link name="back_left_caster_link">
       <inertial>
@@ -189,5 +225,5 @@
         </geometry>
       </visual>
-    </link> -->
+    </link>
     <joint name="platform_support_joint" type="fixed">
       <origin rpy="0 0 0" xyz="-0.02 0.0 0.2"/>
