Commit message: fix logistic_holomic_robot urdf and namespace

File: CustomRobots/logistic_holonomic_robot/models/logistic_holonomic_robot/logistic_holonomic_robot_common.urdf.xacro (robot description, xacro)
@@ -120,41 +120,14 @@
       </visual>
     </link>
-    <link name="back_right_caster_roll_link">
-      <inertial>
-        <mass value="0.0001"/>
-        <inertia ixx="1" ixy="0" ixz="0" iyy="1" iyz="0" izz="1"/>
-      </inertial>
-    </link>
-    <link name="back_right_caster_pitch_link">
-      <inertial>
-        <mass value="0.0001"/>
-        <inertia ixx="1" ixy="0" ixz="0" iyy="1" iyz="0" izz="1"/>
-      </inertial>
-    </link>
-    <joint name="back_right_caster_joint_roll" type="continuous">
+    <!-- Caster is a fixed sphere since the rotating joint chain made the physics unstable -->
+    <joint name="back_right_caster_joint" type="fixed">
       <origin rpy="0 0 0" xyz="-0.23 -0.13 -0.0175"/>
       <parent link="base"/>
-      <child link="back_right_caster_roll_link"/>
-      <axis xyz="1 0 0"/>
-      <limit effort="1000" velocity="100"/>
-    </joint>
-    <joint name="back_right_caster_joint_pitch" type="continuous">
-      <origin rpy="0 0 0" xyz="0 0 0"/>
-      <parent link="back_right_caster_roll_link"/>
-      <child link="back_right_caster_pitch_link"/>
-      <axis xyz="0 1 0"/>
-      <limit effort="1000" velocity="100"/>
-    </joint>
-    <joint name="back_right_caster_joint_yaw" type="continuous">
-      <origin rpy="0 0 0" xyz="0 0 0"/>
-      <parent link="back_right_caster_pitch_link"/>
       <child link="back_right_caster_link"/>
-      <axis xyz="0 0 1"/>
-      <limit effort="1000" velocity="100"/>
     </joint>
     <link name="back_right_caster_link">
       <inertial>
         <mass value="0.8"/>
-        <inertia ixx="0.00001" ixy="0" ixz="0" iyy="0.00001" iyz="0" izz="0.00001"/>
+        <inertia ixx="0.0002" ixy="0" ixz="0" iyy="0.0002" iyz="0" izz="0.0002"/>
       </inertial>
       <collision>
@@ -183,41 +156,13 @@
       </visual>
     </link>
-    <link name="back_left_caster_roll_link">
-      <inertial>
-        <mass value="0.0001"/>
-        <inertia ixx="1" ixy="0" ixz="0" iyy="1" iyz="0" izz="1"/>
-      </inertial>
-    </link>
-    <link name="back_left_caster_pitch_link">
-      <inertial>
-        <mass value="0.0001"/>
-        <inertia ixx="1" ixy="0" ixz="0" iyy="1" iyz="0" izz="1"/>
-      </inertial>
-    </link>
-    <joint name="back_left_caster_joint_roll" type="continuous">
-      <origin rpy="0 0 0" xyz="-0.23  0.13 -0.0175"/>
-      <parent link="base"/>
-      <child link="back_left_caster_roll_link"/>
-      <axis xyz="0 0 1"/>
-      <limit effort="1000" velocity="100"/>
-    </joint>
-    <joint name="back_left_caster_joint_pitch" type="continuous">
-      <origin rpy="0 0 0" xyz="0 0 0"/>
-      <parent link="back_left_caster_roll_link"/>
-      <child link="back_left_caster_pitch_link"/>
-      <axis xyz="0 1 0"/>
-      <limit effort="1000" velocity="100"/>
-    </joint>
-    <joint name="back_left_caster_joint_yaw" type="continuous">
-      <origin rpy="0 0 0" xyz="0 0 0"/>
-      <parent link="back_left_caster_pitch_link"/>
+    <joint name="back_left_caster_joint" type="fixed">
+      <origin rpy="0 0 0" xyz="-0.23 0.13 -0.0175"/>
+      <parent link="base"/>
       <child link="back_left_caster_link"/>
-      <axis xyz="1 0 0"/>
-      <limit effort="1000" velocity="100"/>
     </joint>
     <link name="back_left_caster_link">
       <inertial>
         <mass value="0.8"/>
-        <inertia ixx="0.00001" ixy="0" ixz="0" iyy="0.00001" iyz="0" izz="0.00001"/>
+        <inertia ixx="0.0002" ixy="0" ixz="0" iyy="0.0002" iyz="0" izz="0.0002"/>
       </inertial>
       <collision>

Commit message: reduce holomic wheel weight

File: CustomRobots/logistic_holonomic_robot/models/logistic_holonomic_robot/logistic_holonomic_robot_common.urdf.xacro (robot description, xacro)
@@ -128,6 +128,6 @@
     <link name="back_right_caster_link">
       <inertial>
-        <mass value="0.8"/>
-        <inertia ixx="0.0002" ixy="0" ixz="0" iyy="0.0002" iyz="0" izz="0.0002"/>
+        <mass value="0.01"/>
+        <inertia ixx="0.001" ixy="0" ixz="0" iyy="0.001" iyz="0" izz="0.001"/>
       </inertial>
       <collision>
@@ -163,6 +163,6 @@
     <link name="back_left_caster_link">
       <inertial>
-        <mass value="0.8"/>
-        <inertia ixx="0.0002" ixy="0" ixz="0" iyy="0.0002" iyz="0" izz="0.0002"/>
+        <mass value="0.01"/>
+        <inertia ixx="0.001" ixy="0" ixz="0" iyy="0.001" iyz="0" izz="0.001"/>
       </inertial>
       <collision>

Commit message: Working nav2 and rviz in warehouse1 with holo robot

File: CustomRobots/logistic_holonomic_robot/models/logistic_holonomic_robot/logistic_holonomic_robot_common.urdf.xacro (robot description, xacro)
@@ -268,4 +268,5 @@
       </visual>
     </link>
+    <xacro:laser xyz="0.5 0 0" rpy="0 0 0" name="laser" parent="base" namespace="${namespace}"/>
     <xacro:velocity namespace="${namespace}"/>
     <xacro:odom namespace="${namespace}" freq="50"/>

File: CustomRobots/logistic_holonomic_robot/models/logistic_holonomic_robot/logistic_holonomic_robot_gz.urdf.xacro (robot description, xacro)
@@ -1,4 +1,42 @@
 <?xml version="1.0"?>
 <robot xmlns:xacro="http://ros.org/wiki/xacro">
+ <xacro:macro name="laser" params="xyz rpy name parent namespace">
+    <link name="${name}_link">
+      <visual>
+        <geometry>
+          <mesh filename="file://$(find custom_robots)/models/f1/meshes/hokuyo.dae"/>
+        </geometry>
+      </visual>
+    </link>
+    <joint name="${name}_to_${parent}" type="fixed">
+      <parent link="${parent}"/>
+      <child link="${name}_link"/>
+      <origin xyz="${xyz}" rpy="${rpy}"/>
+    </joint>
+    <gazebo reference="${name}_link">
+      <sensor name="laser" type="gpu_lidar">
+        <always_on>1</always_on>
+        <visualize>1</visualize>
+        <update_rate>20</update_rate>
+        <topic>/${namespace}/laser/scan</topic>
+        <gz_frame_id>laser_link</gz_frame_id>
+        <lidar>
+          <scan>
+            <horizontal>
+              <samples>180</samples>
+              <resolution>1</resolution>
+              <min_angle>-1.570000</min_angle>
+              <max_angle>1.570000</max_angle>
+            </horizontal>
+          </scan>
+          <range>
+            <min>0.080000</min>
+            <max>10.000000</max>
+            <resolution>0.010000</resolution>
+          </range>
+        </lidar>
+      </sensor>
+    </gazebo>
+  </xacro:macro>
   <xacro:macro name="velocity" params="namespace">
     <gazebo>
@@ -19,4 +57,5 @@
         <odom_publish_frequency>${freq}</odom_publish_frequency>
         <odom_topic>/${namespace}/odom</odom_topic>
+        <tf_topic>/tf</tf_topic>
         <dimensions>3</dimensions>
       </plugin>
