Commit message: Change stack to use _mimic

File: Industrial/robotiq_description/urdf/robotiq_85_gripper.ros2_control.xacro (robot description, xacro)
@@ -31,5 +31,5 @@
       </joint>
       <!-- Mimic joints - need to be included for proper state publishing -->
-      <joint name="${prefix}robotiq_85_right_knuckle_joint">
+      <joint name="${prefix}robotiq_85_right_knuckle_joint_mimic">
         <param name="mimic">${prefix}robotiq_85_left_knuckle_joint</param>
         <param name="multiplier">1.0</param>
@@ -42,5 +42,5 @@
         <state_interface name="effort"/>
       </joint>
-      <joint name="${prefix}robotiq_85_left_inner_knuckle_joint">
+      <joint name="${prefix}robotiq_85_left_inner_knuckle_joint_mimic">
         <param name="mimic">${prefix}robotiq_85_left_knuckle_joint</param>
         <param name="multiplier">1.0</param>
@@ -52,5 +52,5 @@
         <state_interface name="velocity"/>
       </joint>
-      <joint name="${prefix}robotiq_85_right_inner_knuckle_joint">
+      <joint name="${prefix}robotiq_85_right_inner_knuckle_joint_mimic">
         <param name="mimic">${prefix}robotiq_85_left_knuckle_joint</param>
         <param name="multiplier">1.0</param>
@@ -62,5 +62,5 @@
         <state_interface name="velocity"/>
       </joint>
-      <joint name="${prefix}robotiq_85_left_finger_tip_joint">
+      <joint name="${prefix}robotiq_85_left_finger_tip_joint_mimic">
         <param name="mimic">${prefix}robotiq_85_left_knuckle_joint</param>
         <param name="multiplier">-1.0</param>
@@ -72,5 +72,5 @@
         <state_interface name="velocity"/>
       </joint>
-      <joint name="${prefix}robotiq_85_right_finger_tip_joint">
+      <joint name="${prefix}robotiq_85_right_finger_tip_joint_mimic">
         <param name="mimic">${prefix}robotiq_85_left_knuckle_joint</param>
         <param name="multiplier">-1.0</param>

Commit message: Change stack to use _mimic

File: Industrial/robotiq_description/urdf/robotiq_85_gripper.ros2_control.xacro (robot description, xacro)
@@ -31,5 +31,5 @@
       </joint>
       <!-- Mimic joints - need to be included for proper state publishing -->
-      <joint name="${prefix}robotiq_85_right_knuckle_joint_mimic">
+      <joint name="${prefix}robotiq_85_right_knuckle_joint">
         <param name="mimic">${prefix}robotiq_85_left_knuckle_joint</param>
         <param name="multiplier">1.0</param>
@@ -42,5 +42,5 @@
         <state_interface name="effort"/>
       </joint>
-      <joint name="${prefix}robotiq_85_left_inner_knuckle_joint_mimic">
+      <joint name="${prefix}robotiq_85_left_inner_knuckle_joint">
         <param name="mimic">${prefix}robotiq_85_left_knuckle_joint</param>
         <param name="multiplier">1.0</param>
@@ -52,5 +52,5 @@
         <state_interface name="velocity"/>
       </joint>
-      <joint name="${prefix}robotiq_85_right_inner_knuckle_joint_mimic">
+      <joint name="${prefix}robotiq_85_right_inner_knuckle_joint">
         <param name="mimic">${prefix}robotiq_85_left_knuckle_joint</param>
         <param name="multiplier">1.0</param>
@@ -62,5 +62,5 @@
         <state_interface name="velocity"/>
       </joint>
-      <joint name="${prefix}robotiq_85_left_finger_tip_joint_mimic">
+      <joint name="${prefix}robotiq_85_left_finger_tip_joint">
         <param name="mimic">${prefix}robotiq_85_left_knuckle_joint</param>
         <param name="multiplier">-1.0</param>
@@ -72,5 +72,5 @@
         <state_interface name="velocity"/>
       </joint>
-      <joint name="${prefix}robotiq_85_right_finger_tip_joint_mimic">
+      <joint name="${prefix}robotiq_85_right_finger_tip_joint">
         <param name="mimic">${prefix}robotiq_85_left_knuckle_joint</param>
         <param name="multiplier">-1.0</param>
