Commit message: Fix xacro and srdf

File: Industrial/robotiq_description/urdf/robotiq_85_gripper.urdf.xacro (robot description, xacro)
@@ -40,5 +40,5 @@
       <origin rpy="0.0 0.0 0.0" xyz="0.05490451627 -0.03060114443 0.0"/>
       <limit lower="-3.14" upper="3.14" velocity="100.0" effort="1000"/>
-      <mimic joint="${prefix}robotiq_85_left_knuckle_joint"/>
+      <mimic joint="${prefix}robotiq_85_left_knuckle_joint" multiplier="1.0"/>
     </joint>
     <link name="${prefix}robotiq_85_left_knuckle_link">
@@ -134,5 +134,5 @@
       <origin xyz="0.06142 0.0127 0" rpy="${pi} 0.0 0.0" />
       <limit lower="-3.14" upper="3.14" velocity="100.0" effort="0.1"/>
-      <mimic joint="${prefix}robotiq_85_left_knuckle_joint" offset="0"/>
+      <mimic joint="${prefix}robotiq_85_left_knuckle_joint" multiplier="1.0" offset="0"/>
     </joint>
     <joint name="${prefix}robotiq_85_right_inner_knuckle_joint" type="continuous">
@@ -142,5 +142,5 @@
       <origin xyz="0.06142 -0.0127 0" rpy="0 0 0"/>
       <limit lower="-3.14" upper="3.14" velocity="100.0" effort="0.1"/>
-      <mimic joint="${prefix}robotiq_85_left_knuckle_joint" offset="0"/>
+      <mimic joint="${prefix}robotiq_85_left_knuckle_joint" multiplier="1.0" offset="0"/>
     </joint>
     <link name="${prefix}robotiq_85_left_inner_knuckle_link">

File: Industrial/ros2_SimRealRobotControl_gz/ros2srrc_endeffectors/robotiq_2f85/urdf/robotiq_2f85_macro.urdf.xacro (robot description, xacro)
@@ -145,5 +145,6 @@
       <axis xyz="0 0 1"/>
       <origin rpy="0 0 0" xyz="0.05490451627 -0.03060114443 0.0"/>
-      <mimic joint="robotiq_85_left_knuckle_joint" multiplier="1"/>
+      <limit lower="-0.05" upper="0.80285" velocity="0.5" effort="1000"/>
+      <dynamics damping="1.0" friction="1.0"/>
     </joint>
     <!-- Robotiq: left_finger -->
@@ -224,5 +225,5 @@
       <axis xyz="0 0 1"/>
       <origin xyz="0.06142 0.0127 0" rpy="${pi} 0.0 0.0" />
-      <mimic joint="robotiq_85_left_knuckle_joint" multiplier="1"/>
+      <limit lower="-0.05" upper="0.80285" velocity="0.5" effort="1000"/>
       <dynamics damping="1.0" friction="1.0"/>
     </joint>
@@ -252,5 +253,5 @@
       <axis xyz="0 0 1"/>
       <origin xyz="0.06142 -0.0127 0" rpy="0 0 0"/>
-      <mimic joint="robotiq_85_left_knuckle_joint" multiplier="1"/>
+      <limit lower="-0.05" upper="0.80285" velocity="0.5" effort="1000"/>
       <dynamics damping="1.0" friction="1.0"/>
     </joint>
@@ -282,5 +283,5 @@
       <axis xyz="0 0 1"/>
       <origin xyz="0.04303959807 -0.03759940821 0.0" rpy="0.0 0.0 0.0"/>
-      <mimic joint="robotiq_85_left_knuckle_joint" multiplier="-1"/>
+      <limit lower="-0.80285" upper="0.05" velocity="0.5" effort="1000"/>
       <dynamics damping="1.0" friction="1.0"/>
     </joint>
@@ -312,5 +313,5 @@
       <axis xyz="0 0 1"/>
       <origin rpy="0.0 0.0 0.0" xyz="0.04303959807 -0.03759940821  0.0"/>
-      <mimic joint="robotiq_85_left_knuckle_joint" multiplier="-1"/>
+      <limit lower="-0.80285" upper="0.05" velocity="0.5" effort="1000"/>
       <dynamics damping="1.0" friction="1.0"/>
     </joint>

Commit message: Fix xacros

File: Industrial/robotiq_description/urdf/robotiq_85_gripper.urdf.xacro (robot description, xacro)
@@ -34,5 +34,5 @@
       <limit lower="0.0" upper="0.80285" velocity="0.5" effort="1000"/>
     </joint>
-    <joint name="${prefix}robotiq_85_right_knuckle_joint" type="continuous">
+    <joint name="${prefix}robotiq_85_right_knuckle_joint" type="fixed">
       <parent link="${prefix}robotiq_85_base_link"/>
       <child link="${prefix}robotiq_85_right_knuckle_link"/>
@@ -40,5 +40,4 @@
       <origin rpy="0.0 0.0 0.0" xyz="0.05490451627 -0.03060114443 0.0"/>
       <limit lower="-3.14" upper="3.14" velocity="100.0" effort="1000"/>
-      <mimic joint="${prefix}robotiq_85_left_knuckle_joint" multiplier="1.0"/>
     </joint>
     <link name="${prefix}robotiq_85_left_knuckle_link">
@@ -128,5 +127,5 @@
       </inertial>
     </link>
-    <joint name="${prefix}robotiq_85_left_inner_knuckle_joint" type="continuous">
+    <joint name="${prefix}robotiq_85_left_inner_knuckle_joint" type="fixed">
       <parent link="${prefix}robotiq_85_base_link"/>
       <child link="${prefix}robotiq_85_left_inner_knuckle_link"/>
@@ -134,7 +133,6 @@
       <origin xyz="0.06142 0.0127 0" rpy="${pi} 0.0 0.0" />
       <limit lower="-3.14" upper="3.14" velocity="100.0" effort="0.1"/>
-      <mimic joint="${prefix}robotiq_85_left_knuckle_joint" multiplier="1.0" offset="0"/>
-    </joint>
-    <joint name="${prefix}robotiq_85_right_inner_knuckle_joint" type="continuous">
+    </joint>
+    <joint name="${prefix}robotiq_85_right_inner_knuckle_joint" type="fixed">
       <parent link="${prefix}robotiq_85_base_link"/>
       <child link="${prefix}robotiq_85_right_inner_knuckle_link"/>
@@ -142,5 +140,4 @@
       <origin xyz="0.06142 -0.0127 0" rpy="0 0 0"/>
       <limit lower="-3.14" upper="3.14" velocity="100.0" effort="0.1"/>
-      <mimic joint="${prefix}robotiq_85_left_knuckle_joint" multiplier="1.0" offset="0"/>
     </joint>
     <link name="${prefix}robotiq_85_left_inner_knuckle_link">
@@ -182,5 +179,5 @@
       </inertial>
     </link>
-    <joint name="${prefix}robotiq_85_left_finger_tip_joint" type="continuous">
+    <joint name="${prefix}robotiq_85_left_finger_tip_joint" type="fixed">
       <parent link="${prefix}robotiq_85_left_inner_knuckle_link"/>
       <child link="${prefix}robotiq_85_left_finger_tip_link"/>
@@ -188,7 +185,6 @@
       <origin xyz="0.04303959807 -0.03759940821 0.0" rpy="0.0 0.0 0.0"/>
       <limit lower="-3.14" upper="3.14" velocity="100.0" effort="0.1"/>
-      <mimic joint="${prefix}robotiq_85_left_knuckle_joint" multiplier="-1"/>
-    </joint>
-    <joint name="${prefix}robotiq_85_right_finger_tip_joint" type="continuous">
+    </joint>
+    <joint name="${prefix}robotiq_85_right_finger_tip_joint" type="fixed">
       <parent link="${prefix}robotiq_85_right_inner_knuckle_link"/>
       <child link="${prefix}robotiq_85_right_finger_tip_link"/>
@@ -196,5 +192,4 @@
       <origin rpy="0.0 0.0 0.0" xyz="0.04303959807 -0.03759940821  0.0"/>
       <limit lower="-3.14" upper="3.14" velocity="100.0" effort="0.1"/>
-      <mimic joint="${prefix}robotiq_85_left_knuckle_joint" multiplier="-1"/>
     </joint>
     <link name="${prefix}robotiq_85_left_finger_tip_link">
@@ -250,36 +245,4 @@
       <minDepth>0.001</minDepth>
     </gazebo>
-    <gazebo>
-      <plugin filename="gz-sim-mimic-joint-system" name="gz::sim::systems::MimicJoint">
-        <joint>${prefix}robotiq_85_right_knuckle_joint</joint>
-        <mimic_joint>${prefix}robotiq_85_left_knuckle_joint</mimic_joint>
-        <multiplier>1.0</multiplier>
-        <offset>0.0</offset>
-      </plugin>
-      <plugin filename="gz-sim-mimic-joint-system" name="gz::sim::systems::MimicJoint">
-        <joint>${prefix}robotiq_85_left_inner_knuckle_joint</joint>
-        <mimic_joint>${prefix}robotiq_85_left_knuckle_joint</mimic_joint>
-        <multiplier>1.0</multiplier>
-        <offset>0.0</offset>
-      </plugin>
-      <plugin filename="gz-sim-mimic-joint-system" name="gz::sim::systems::MimicJoint">
-        <joint>${prefix}robotiq_85_right_inner_knuckle_joint</joint>
-        <mimic_joint>${prefix}robotiq_85_left_knuckle_joint</mimic_joint>
-        <multiplier>1.0</multiplier>
-        <offset>0.0</offset>
-      </plugin>
-      <plugin filename="gz-sim-mimic-joint-system" name="gz::sim::systems::MimicJoint">
-        <joint>${prefix}robotiq_85_left_finger_tip_joint</joint>
-        <mimic_joint>${prefix}robotiq_85_left_knuckle_joint</mimic_joint>
-        <multiplier>-1.0</multiplier>
-        <offset>0.0</offset>
-      </plugin>
-      <plugin filename="gz-sim-mimic-joint-system" name="gz::sim::systems::MimicJoint">
-        <joint>${prefix}robotiq_85_right_finger_tip_joint</joint>
-        <mimic_joint>${prefix}robotiq_85_left_knuckle_joint</mimic_joint>
-        <multiplier>-1.0</multiplier>
-        <offset>0.0</offset>
-      </plugin>
-    </gazebo>
     <xacro:robotiq_85_gripper_transmission prefix="${prefix}" />
   </xacro:macro>

File: Industrial/ros2_SimRealRobotControl_gz/packages/ur5/ros2srrc_ur5_gazebo/urdf/ur5_robotiq_2f85.urdf.xacro (robot description, xacro)
@@ -77,8 +77,8 @@
         <parameters>${simulation_controllers}</parameters>
       </plugin>
-      <plugin filename="libgz_mimic_joint.so" name="gz_mimic_joint">
+      <!--<plugin filename="libgz_mimic_joint.so" name="gz_mimic_joint::MimicJoint">
         <parent_joint>robotiq_85_left_knuckle_joint</parent_joint>
         <mimic_joint>robotiq_85_right_knuckle_joint</mimic_joint>
-      </plugin>
+      </plugin>-->
     </gazebo>
   </xacro:unless>

Commit message: Fix gripper visual issue

File: Industrial/robotiq_description/urdf/robotiq_85_gripper.urdf.xacro (robot description, xacro)
@@ -34,5 +34,5 @@
       <limit lower="0.0" upper="0.80285" velocity="0.5" effort="1000"/>
     </joint>
-    <joint name="${prefix}robotiq_85_right_knuckle_joint" type="fixed">
+    <joint name="${prefix}robotiq_85_right_knuckle_joint" type="continuous">
       <parent link="${prefix}robotiq_85_base_link"/>
       <child link="${prefix}robotiq_85_right_knuckle_link"/>
@@ -40,4 +40,5 @@
       <origin rpy="0.0 0.0 0.0" xyz="0.05490451627 -0.03060114443 0.0"/>
       <limit lower="-3.14" upper="3.14" velocity="100.0" effort="1000"/>
+      <mimic joint="${prefix}robotiq_85_left_knuckle_joint" multiplier="1.0"/>
     </joint>
     <link name="${prefix}robotiq_85_left_knuckle_link">
@@ -127,5 +128,5 @@
       </inertial>
     </link>
-    <joint name="${prefix}robotiq_85_left_inner_knuckle_joint" type="fixed">
+    <joint name="${prefix}robotiq_85_left_inner_knuckle_joint" type="continuous">
       <parent link="${prefix}robotiq_85_base_link"/>
       <child link="${prefix}robotiq_85_left_inner_knuckle_link"/>
@@ -133,6 +134,7 @@
       <origin xyz="0.06142 0.0127 0" rpy="${pi} 0.0 0.0" />
       <limit lower="-3.14" upper="3.14" velocity="100.0" effort="0.1"/>
-    </joint>
-    <joint name="${prefix}robotiq_85_right_inner_knuckle_joint" type="fixed">
+      <mimic joint="${prefix}robotiq_85_left_knuckle_joint" offset="0"/>
+    </joint>
+    <joint name="${prefix}robotiq_85_right_inner_knuckle_joint" type="continuous">
       <parent link="${prefix}robotiq_85_base_link"/>
       <child link="${prefix}robotiq_85_right_inner_knuckle_link"/>
@@ -140,4 +142,5 @@
       <origin xyz="0.06142 -0.0127 0" rpy="0 0 0"/>
       <limit lower="-3.14" upper="3.14" velocity="100.0" effort="0.1"/>
+      <mimic joint="${prefix}robotiq_85_left_knuckle_joint" offset="0"/>
     </joint>
     <link name="${prefix}robotiq_85_left_inner_knuckle_link">
@@ -179,5 +182,5 @@
       </inertial>
     </link>
-    <joint name="${prefix}robotiq_85_left_finger_tip_joint" type="fixed">
+    <joint name="${prefix}robotiq_85_left_finger_tip_joint" type="continuous">
       <parent link="${prefix}robotiq_85_left_inner_knuckle_link"/>
       <child link="${prefix}robotiq_85_left_finger_tip_link"/>
@@ -185,6 +188,7 @@
       <origin xyz="0.04303959807 -0.03759940821 0.0" rpy="0.0 0.0 0.0"/>
       <limit lower="-3.14" upper="3.14" velocity="100.0" effort="0.1"/>
-    </joint>
-    <joint name="${prefix}robotiq_85_right_finger_tip_joint" type="fixed">
+      <mimic joint="${prefix}robotiq_85_left_knuckle_joint" multiplier="-1"/>
+    </joint>
+    <joint name="${prefix}robotiq_85_right_finger_tip_joint" type="continuous">
       <parent link="${prefix}robotiq_85_right_inner_knuckle_link"/>
       <child link="${prefix}robotiq_85_right_finger_tip_link"/>
@@ -192,4 +196,5 @@
       <origin rpy="0.0 0.0 0.0" xyz="0.04303959807 -0.03759940821  0.0"/>
       <limit lower="-3.14" upper="3.14" velocity="100.0" effort="0.1"/>
+      <mimic joint="${prefix}robotiq_85_left_knuckle_joint" multiplier="-1"/>
     </joint>
     <link name="${prefix}robotiq_85_left_finger_tip_link">
@@ -245,4 +250,36 @@
       <minDepth>0.001</minDepth>
     </gazebo>
+    <gazebo>
+      <plugin filename="gz-sim-mimic-joint-system" name="gz::sim::systems::MimicJoint">
+        <joint>${prefix}robotiq_85_right_knuckle_joint</joint>
+        <mimic_joint>${prefix}robotiq_85_left_knuckle_joint</mimic_joint>
+        <multiplier>1.0</multiplier>
+        <offset>0.0</offset>
+      </plugin>
+      <plugin filename="gz-sim-mimic-joint-system" name="gz::sim::systems::MimicJoint">
+        <joint>${prefix}robotiq_85_left_inner_knuckle_joint</joint>
+        <mimic_joint>${prefix}robotiq_85_left_knuckle_joint</mimic_joint>
+        <multiplier>1.0</multiplier>
+        <offset>0.0</offset>
+      </plugin>
+      <plugin filename="gz-sim-mimic-joint-system" name="gz::sim::systems::MimicJoint">
+        <joint>${prefix}robotiq_85_right_inner_knuckle_joint</joint>
+        <mimic_joint>${prefix}robotiq_85_left_knuckle_joint</mimic_joint>
+        <multiplier>1.0</multiplier>
+        <offset>0.0</offset>
+      </plugin>
+      <plugin filename="gz-sim-mimic-joint-system" name="gz::sim::systems::MimicJoint">
+        <joint>${prefix}robotiq_85_left_finger_tip_joint</joint>
+        <mimic_joint>${prefix}robotiq_85_left_knuckle_joint</mimic_joint>
+        <multiplier>-1.0</multiplier>
+        <offset>0.0</offset>
+      </plugin>
+      <plugin filename="gz-sim-mimic-joint-system" name="gz::sim::systems::MimicJoint">
+        <joint>${prefix}robotiq_85_right_finger_tip_joint</joint>
+        <mimic_joint>${prefix}robotiq_85_left_knuckle_joint</mimic_joint>
+        <multiplier>-1.0</multiplier>
+        <offset>0.0</offset>
+      </plugin>
+    </gazebo>
     <xacro:robotiq_85_gripper_transmission prefix="${prefix}" />
   </xacro:macro>

File: Industrial/ur5_gripper_description/urdf/ur5_robotiq85_gripper.urdf.xacro (robot description, xacro)
@@ -46,5 +46,5 @@
     prefix=""
     sim_gz="true"
-    use_fake_hardware="true"
+    use_fake_hardware="false"
     script_filename=""
     output_recipe_filename=""

Commit message: Restart mimic joint

File: Industrial/robotiq_description/urdf/robotiq_85_gripper.urdf.xacro (robot description, xacro)
@@ -250,4 +250,36 @@
       <minDepth>0.001</minDepth>
     </gazebo>
+    <gazebo>
+      <plugin filename="gz-sim-mimic-joint-system" name="gz::sim::systems::MimicJoint">
+        <joint>${prefix}robotiq_85_right_knuckle_joint</joint>
+        <mimic_joint>${prefix}robotiq_85_left_knuckle_joint</mimic_joint>
+        <multiplier>1.0</multiplier>
+        <offset>0.0</offset>
+      </plugin>
+      <plugin filename="gz-sim-mimic-joint-system" name="gz::sim::systems::MimicJoint">
+        <joint>${prefix}robotiq_85_left_inner_knuckle_joint</joint>
+        <mimic_joint>${prefix}robotiq_85_left_knuckle_joint</mimic_joint>
+        <multiplier>1.0</multiplier>
+        <offset>0.0</offset>
+      </plugin>
+      <plugin filename="gz-sim-mimic-joint-system" name="gz::sim::systems::MimicJoint">
+        <joint>${prefix}robotiq_85_right_inner_knuckle_joint</joint>
+        <mimic_joint>${prefix}robotiq_85_left_knuckle_joint</mimic_joint>
+        <multiplier>1.0</multiplier>
+        <offset>0.0</offset>
+      </plugin>
+      <plugin filename="gz-sim-mimic-joint-system" name="gz::sim::systems::MimicJoint">
+        <joint>${prefix}robotiq_85_left_finger_tip_joint</joint>
+        <mimic_joint>${prefix}robotiq_85_left_knuckle_joint</mimic_joint>
+        <multiplier>-1.0</multiplier>
+        <offset>0.0</offset>
+      </plugin>
+      <plugin filename="gz-sim-mimic-joint-system" name="gz::sim::systems::MimicJoint">
+        <joint>${prefix}robotiq_85_right_finger_tip_joint</joint>
+        <mimic_joint>${prefix}robotiq_85_left_knuckle_joint</mimic_joint>
+        <multiplier>-1.0</multiplier>
+        <offset>0.0</offset>
+      </plugin>
+    </gazebo>
     <xacro:robotiq_85_gripper_transmission prefix="${prefix}" />
   </xacro:macro>

Commit message: Add collision sensor to the gripper tip and link attacher plugin

File: Industrial/robotiq_description/urdf/robotiq_85_gripper.urdf.xacro (robot description, xacro)
@@ -204,5 +204,5 @@
         </geometry>
       </visual>
-      <collision>
+      <collision name="collision">
         <geometry>
           <box size="0.02 0.02 0.02"/>
@@ -223,5 +223,5 @@
         </geometry>
       </visual>
-      <collision>
+      <collision name="collision">
         <geometry>
           <box size="0.02 0.02 0.02"/>
@@ -242,4 +242,11 @@
       <mu2>1.0</mu2>
       <minDepth>0.001</minDepth>
+      <sensor name="${prefix}left_finger_contact" type="contact">
+        <always_on>true</always_on>
+        <update_rate>100</update_rate>
+        <contact>
+          <collision>collision</collision>
+        </contact>
+      </sensor>
     </gazebo>
     <gazebo reference="${prefix}robotiq_85_right_finger_tip_link">
@@ -249,4 +256,11 @@
       <mu2>1.0</mu2>
       <minDepth>0.001</minDepth>
+      <sensor name="${prefix}right_finger_contact" type="contact">
+        <always_on>true</always_on>
+        <update_rate>100</update_rate>
+        <contact>
+          <collision>collision</collision>
+        </contact>
+      </sensor>
     </gazebo>
     <xacro:robotiq_85_gripper_transmission prefix="${prefix}" />

Commit message: Change collision names

File: Industrial/robotiq_description/urdf/robotiq_85_gripper.urdf.xacro (robot description, xacro)
@@ -204,5 +204,5 @@
         </geometry>
       </visual>
-      <collision name="collision">
+      <collision name="${prefix}left_finger_tip_collision">
         <geometry>
           <box size="0.02 0.02 0.02"/>
@@ -223,5 +223,5 @@
         </geometry>
       </visual>
-      <collision name="collision">
+      <collision name="${prefix}right_finger_tip_collision">
         <geometry>
           <box size="0.02 0.02 0.02"/>
@@ -246,5 +246,5 @@
         <update_rate>100</update_rate>
         <contact>
-          <collision>collision</collision>
+          <collision>${prefix}left_finger_tip_collision</collision>
         </contact>
       </sensor>
@@ -260,5 +260,5 @@
         <update_rate>100</update_rate>
         <contact>
-          <collision>collision</collision>
+          <collision>${prefix}right_finger_tip_collision</collision>
         </contact>
       </sensor>

Commit message: Add visual collision box

File: Industrial/robotiq_description/urdf/robotiq_85_gripper.urdf.xacro (robot description, xacro)
@@ -205,8 +205,18 @@
       </visual>
       <collision name="${prefix}left_finger_tip_collision">
-        <geometry>
-          <box size="0.02 0.02 0.02"/>
-        </geometry>
-      </collision>
+        <origin xyz="0 0 0" rpy="0 0 0"/>
+        <geometry>
+          <box size="0.02 0.02 0.02"/>
+        </geometry>
+      </collision>
+      <visual name="left_debug_collision">
+        <origin xyz="0 0 0" rpy="0 0 0"/>
+        <geometry>
+          <box size="0.02 0.02 0.02"/>
+        </geometry>
+        <material>
+          <color rgba="1 0 0 0.5"/>
+        </material>
+      </visual>
       <inertial>
         <mass value="0.019555" />
@@ -224,8 +234,18 @@
       </visual>
       <collision name="${prefix}right_finger_tip_collision">
-        <geometry>
-          <box size="0.02 0.02 0.02"/>
-        </geometry>
-      </collision>
+        <origin xyz="0 0 0" rpy="0 0 0"/>
+        <geometry>
+          <box size="0.02 0.02 0.02"/>
+        </geometry>
+      </collision>
+      <visual name="right_debug_collision">
+        <origin xyz="0 0 0" rpy="0 0 0"/>
+        <geometry>
+          <box size="0.02 0.02 0.02"/>
+        </geometry>
+        <material>
+          <color rgba="0 1 0 0.5"/>
+        </material>
+      </visual>
       <inertial>
         <mass value="0.019555" />
