Commit message: Change collision sensor

File: Industrial/robotiq_description/urdf/robotiq_85_gripper.urdf.xacro (robot description, xacro)
@@ -226,62 +226,50 @@
              izx = "0.000000" izy = "0.000000" izz = "0.000006" />
       </inertial>
-    </link>
-    <link name="${prefix}robotiq_85_right_finger_tip_link">
-      <visual>
-        <geometry>
-          <mesh filename="package://robotiq_description/meshes/visual/robotiq_85_finger_tip_link.dae"/>
-        </geometry>
-      </visual>
-      <collision name="${prefix}right_finger_tip_collision">
-        <origin xyz="0 0 0" rpy="0 0 0"/>
-        <geometry>
-          <box size="0.02 0.02 0.02"/>
-        </geometry>
-      </collision>
-      <visual name="right_debug_collision">
-        <origin xyz="0 0 0" rpy="0 0 0"/>
-        <geometry>
-          <box size="0.02 0.02 0.02"/>
-        </geometry>
-        <material>
-          <color rgba="0 1 0 0.5"/>
-        </material>
-      </visual>
-      <inertial>
-        <mass value="0.019555" />
-        <origin xyz="0.0 0.0 0.0" />
-        <inertia ixx = "0.000002" ixy = "0.000000" ixz = "0.000000"
-             iyx = "0.000000" iyy = "0.000005" iyz = "0.000000"
-             izx = "0.000000" izy = "0.000000" izz = "0.000006" />
-      </inertial>
-    </link>
-    <gazebo reference="${prefix}robotiq_85_left_finger_tip_link">
-      <kp>1000000.0</kp>
-      <kd>1.0</kd>
-      <mu1>1.0</mu1>
-      <mu2>1.0</mu2>
-      <minDepth>0.001</minDepth>
-      <sensor name="${prefix}left_finger_contact" type="contact">
+      <sensor name="left_finger_contact" type="contact">
         <always_on>true</always_on>
         <update_rate>100</update_rate>
+        <topic>/left_finger_contact</topic>
         <contact>
           <collision>${prefix}left_finger_tip_collision</collision>
         </contact>
       </sensor>
-    </gazebo>
-    <gazebo reference="${prefix}robotiq_85_right_finger_tip_link">
-      <kp>1000000.0</kp>
-      <kd>1.0</kd>
-      <mu1>1.0</mu1>
-      <mu2>1.0</mu2>
-      <minDepth>0.001</minDepth>
-      <sensor name="${prefix}right_finger_contact" type="contact">
+    </link>
+    <link name="${prefix}robotiq_85_right_finger_tip_link">
+      <visual>
+        <geometry>
+          <mesh filename="package://robotiq_description/meshes/visual/robotiq_85_finger_tip_link.dae"/>
+        </geometry>
+      </visual>
+      <collision name="${prefix}right_finger_tip_collision">
+        <origin xyz="0 0 0" rpy="0 0 0"/>
+        <geometry>
+          <box size="0.02 0.02 0.02"/>
+        </geometry>
+      </collision>
+      <visual name="right_debug_collision">
+        <origin xyz="0 0 0" rpy="0 0 0"/>
+        <geometry>
+          <box size="0.02 0.02 0.02"/>
+        </geometry>
+        <material>
+          <color rgba="0 1 0 0.5"/>
+        </material>
+      </visual>
+      <inertial>
+        <mass value="0.019555" />
+        <origin xyz="0.0 0.0 0.0" />
+        <inertia ixx = "0.000002" ixy = "0.000000" ixz = "0.000000"
+             iyx = "0.000000" iyy = "0.000005" iyz = "0.000000"
+             izx = "0.000000" izy = "0.000000" izz = "0.000006" />
+      </inertial>
+      <sensor name="right_finger_contact" type="contact">
         <always_on>true</always_on>
         <update_rate>100</update_rate>
+        <topic>/right_finger_contact</topic>
         <contact>
           <collision>${prefix}right_finger_tip_collision</collision>
         </contact>
       </sensor>
-    </gazebo>
+    </link>
     <xacro:robotiq_85_gripper_transmission prefix="${prefix}" />
   </xacro:macro>

Commit message: Change collision sensor

File: Industrial/robotiq_description/urdf/robotiq_85_gripper.urdf.xacro (robot description, xacro)
@@ -226,4 +226,35 @@
              izx = "0.000000" izy = "0.000000" izz = "0.000006" />
       </inertial>
+    </link>
+    <link name="${prefix}robotiq_85_right_finger_tip_link">
+      <visual>
+        <geometry>
+          <mesh filename="package://robotiq_description/meshes/visual/robotiq_85_finger_tip_link.dae"/>
+        </geometry>
+      </visual>
+      <collision name="${prefix}right_finger_tip_collision">
+        <origin xyz="0 0 0" rpy="0 0 0"/>
+        <geometry>
+          <box size="0.02 0.02 0.02"/>
+        </geometry>
+      </collision>
+      <visual name="right_debug_collision">
+        <origin xyz="0 0 0" rpy="0 0 0"/>
+        <geometry>
+          <box size="0.02 0.02 0.02"/>
+        </geometry>
+        <material>
+          <color rgba="0 1 0 0.5"/>
+        </material>
+      </visual>
+      <inertial>
+        <mass value="0.019555" />
+        <origin xyz="0.0 0.0 0.0" />
+        <inertia ixx = "0.000002" ixy = "0.000000" ixz = "0.000000"
+             iyx = "0.000000" iyy = "0.000005" iyz = "0.000000"
+             izx = "0.000000" izy = "0.000000" izz = "0.000006" />
+      </inertial>
+    </link>
+    <gazebo reference="${prefix}robotiq_85_left_finger_tip_link">
       <sensor name="left_finger_contact" type="contact">
         <always_on>true</always_on>
@@ -234,33 +265,6 @@
         </contact>
       </sensor>
-    </link>
-    <link name="${prefix}robotiq_85_right_finger_tip_link">
-      <visual>
-        <geometry>
-          <mesh filename="package://robotiq_description/meshes/visual/robotiq_85_finger_tip_link.dae"/>
-        </geometry>
-      </visual>
-      <collision name="${prefix}right_finger_tip_collision">
-        <origin xyz="0 0 0" rpy="0 0 0"/>
-        <geometry>
-          <box size="0.02 0.02 0.02"/>
-        </geometry>
-      </collision>
-      <visual name="right_debug_collision">
-        <origin xyz="0 0 0" rpy="0 0 0"/>
-        <geometry>
-          <box size="0.02 0.02 0.02"/>
-        </geometry>
-        <material>
-          <color rgba="0 1 0 0.5"/>
-        </material>
-      </visual>
-      <inertial>
-        <mass value="0.019555" />
-        <origin xyz="0.0 0.0 0.0" />
-        <inertia ixx = "0.000002" ixy = "0.000000" ixz = "0.000000"
-             iyx = "0.000000" iyy = "0.000005" iyz = "0.000000"
-             izx = "0.000000" izy = "0.000000" izz = "0.000006" />
-      </inertial>
+    </gazebo>
+    <gazebo reference="${prefix}robotiq_85_right_finger_tip_link">
       <sensor name="right_finger_contact" type="contact">
         <always_on>true</always_on>
@@ -271,5 +275,5 @@
         </contact>
       </sensor>
-    </link>
+    </gazebo>
     <xacro:robotiq_85_gripper_transmission prefix="${prefix}" />
   </xacro:macro>

Commit message: Add collision visual box

File: Industrial/robotiq_description/urdf/robotiq_85_gripper.urdf.xacro (robot description, xacro)
@@ -204,17 +204,17 @@
         </geometry>
       </visual>
-      <collision name="${prefix}left_finger_tip_collision">
-        <origin xyz="0 0 0" rpy="0 0 0"/>
-        <geometry>
-          <box size="0.02 0.02 0.02"/>
-        </geometry>
-      </collision>
-      <visual name="left_debug_collision">
-        <origin xyz="0 0 0" rpy="0 0 0"/>
-        <geometry>
-          <box size="0.02 0.02 0.02"/>
-        </geometry>
-        <material>
-          <color rgba="1 0 0 0.5"/>
+      <collision>
+        <origin xyz="0 0 0" rpy="0 0 0"/>
+        <geometry>
+          <box size="0.06 0.06 0.06"/>
+        </geometry>
+      </collision>
+      <visual>
+        <origin xyz="0 0 0" rpy="0 0 0"/>
+        <geometry>
+          <box size="0.06 0.06 0.06"/>
+        </geometry>
+        <material name="Red">
+          <color rgba="1 0 0 0.8"/>
         </material>
       </visual>
@@ -233,17 +233,17 @@
         </geometry>
       </visual>
-      <collision name="${prefix}right_finger_tip_collision">
-        <origin xyz="0 0 0" rpy="0 0 0"/>
-        <geometry>
-          <box size="0.02 0.02 0.02"/>
-        </geometry>
-      </collision>
-      <visual name="right_debug_collision">
-        <origin xyz="0 0 0" rpy="0 0 0"/>
-        <geometry>
-          <box size="0.02 0.02 0.02"/>
-        </geometry>
-        <material>
-          <color rgba="0 1 0 0.5"/>
+      <collision>
+        <origin xyz="0 0 0" rpy="0 0 0"/>
+        <geometry>
+          <box size="0.06 0.06 0.06"/>
+        </geometry>
+      </collision>
+      <visual>
+        <origin xyz="0 0 0" rpy="0 0 0"/>
+        <geometry>
+          <box size="0.06 0.06 0.06"/>
+        </geometry>
+        <material name="Green">
+          <color rgba="0 1 0 0.8"/>
         </material>
       </visual>
@@ -257,22 +257,16 @@
     </link>
     <gazebo reference="${prefix}robotiq_85_left_finger_tip_link">
-      <sensor name="left_finger_contact" type="contact">
-        <always_on>true</always_on>
-        <update_rate>100</update_rate>
-        <topic>/left_finger_contact</topic>
-        <contact>
-          <collision>${prefix}left_finger_tip_collision</collision>
-        </contact>
-      </sensor>
+      <kp>1000000.0</kp>
+      <kd>1.0</kd>
+      <mu1>1.0</mu1>
+      <mu2>1.0</mu2>
+      <minDepth>0.001</minDepth>
     </gazebo>
     <gazebo reference="${prefix}robotiq_85_right_finger_tip_link">
-      <sensor name="right_finger_contact" type="contact">
-        <always_on>true</always_on>
-        <update_rate>100</update_rate>
-        <topic>/right_finger_contact</topic>
-        <contact>
-          <collision>${prefix}right_finger_tip_collision</collision>
-        </contact>
-      </sensor>
+      <kp>1000000.0</kp>
+      <kd>1.0</kd>
+      <mu1>1.0</mu1>
+      <mu2>1.0</mu2>
+      <minDepth>0.001</minDepth>
     </gazebo>
     <xacro:robotiq_85_gripper_transmission prefix="${prefix}" />

Commit message: Fix visual collisio box

File: Industrial/robotiq_description/urdf/robotiq_85_gripper.urdf.xacro (robot description, xacro)
@@ -205,13 +205,13 @@
       </visual>
       <collision>
-        <origin xyz="0 0 0" rpy="0 0 0"/>
-        <geometry>
-          <box size="0.06 0.06 0.06"/>
-        </geometry>
-      </collision>
-      <visual>
-        <origin xyz="0 0 0" rpy="0 0 0"/>
-        <geometry>
-          <box size="0.06 0.06 0.06"/>
+        <origin xyz="0.04 0 0" rpy="0 0 0"/>
+        <geometry>
+          <box size="0.02 0.02 0.02"/>
+        </geometry>
+      </collision>
+      <visual>
+        <origin xyz="0.04 0 0" rpy="0 0 0"/>
+        <geometry>
+          <box size="0.02 0.02 0.02"/>
         </geometry>
         <material name="Red">
@@ -234,13 +234,13 @@
       </visual>
       <collision>
-        <origin xyz="0 0 0" rpy="0 0 0"/>
-        <geometry>
-          <box size="0.06 0.06 0.06"/>
-        </geometry>
-      </collision>
-      <visual>
-        <origin xyz="0 0 0" rpy="0 0 0"/>
-        <geometry>
-          <box size="0.06 0.06 0.06"/>
+        <origin xyz="0.04 0 0" rpy="0 0 0"/>
+        <geometry>
+          <box size="0.02 0.02 0.02"/>
+        </geometry>
+      </collision>
+      <visual>
+        <origin xyz="0.04 0 0" rpy="0 0 0"/>
+        <geometry>
+          <box size="0.02 0.02 0.02"/>
         </geometry>
         <material name="Green">

Commit message: Add contatc sensor to the fingers

File: Industrial/robotiq_description/urdf/robotiq_85_gripper.urdf.xacro (robot description, xacro)
@@ -204,12 +204,12 @@
         </geometry>
       </visual>
-      <collision>
-        <origin xyz="0.04 0 0" rpy="0 0 0"/>
-        <geometry>
-          <box size="0.02 0.02 0.02"/>
-        </geometry>
-      </collision>
-      <visual>
-        <origin xyz="0.04 0 0" rpy="0 0 0"/>
+      <collision name="robotiq_85_left_finger_tip_link_collision">
+        <origin xyz="0 0 0" rpy="0 0 0"/>
+        <geometry>
+          <box size="0.02 0.02 0.02"/>
+        </geometry>
+      </collision>
+      <visual>
+        <origin xyz="0 0 0" rpy="0 0 0"/>
         <geometry>
           <box size="0.02 0.02 0.02"/>
@@ -233,12 +233,12 @@
         </geometry>
       </visual>
-      <collision>
-        <origin xyz="0.04 0 0" rpy="0 0 0"/>
-        <geometry>
-          <box size="0.02 0.02 0.02"/>
-        </geometry>
-      </collision>
-      <visual>
-        <origin xyz="0.04 0 0" rpy="0 0 0"/>
+      <collision name="robotiq_85_right_finger_tip_link_collision">
+        <origin xyz="0 0 0" rpy="0 0 0"/>
+        <geometry>
+          <box size="0.02 0.02 0.02"/>
+        </geometry>
+      </collision>
+      <visual>
+        <origin xyz="0 0 0" rpy="0 0 0"/>
         <geometry>
           <box size="0.02 0.02 0.02"/>
@@ -262,4 +262,12 @@
       <mu2>1.0</mu2>
       <minDepth>0.001</minDepth>
+      <sensor name="left_finger_contact" type="contact">
+        <always_on>true</always_on>
+        <update_rate>100</update_rate>
+        <contact>
+          <collision>robotiq_85_left_finger_tip_link_collision</collision>
+        </contact>
+        <topic>/left_finger_contact</topic>
+      </sensor>
     </gazebo>
     <gazebo reference="${prefix}robotiq_85_right_finger_tip_link">
@@ -269,4 +277,12 @@
       <mu2>1.0</mu2>
       <minDepth>0.001</minDepth>
+      <sensor name="right_finger_contact" type="contact">
+        <always_on>true</always_on>
+        <update_rate>100</update_rate>
+        <contact>
+          <collision>robotiq_85_right_finger_tip_link_collision</collision>
+        </contact>
+        <topic>/right_finger_contact</topic>
+      </sensor>
     </gazebo>
     <xacro:robotiq_85_gripper_transmission prefix="${prefix}" />

Commit message: Add contatc sensor to the fingers

File: Industrial/robotiq_description/urdf/robotiq_85_gripper.urdf.xacro (robot description, xacro)
@@ -205,11 +205,11 @@
       </visual>
       <collision name="robotiq_85_left_finger_tip_link_collision">
-        <origin xyz="0 0 0" rpy="0 0 0"/>
-        <geometry>
-          <box size="0.02 0.02 0.02"/>
-        </geometry>
-      </collision>
-      <visual>
-        <origin xyz="0 0 0" rpy="0 0 0"/>
+        <origin xyz="0.03 0 0" rpy="0 0 0"/>
+        <geometry>
+          <box size="0.02 0.02 0.02"/>
+        </geometry>
+      </collision>
+      <visual>
+        <origin xyz="0.03 0 0" rpy="0 0 0"/>
         <geometry>
           <box size="0.02 0.02 0.02"/>
@@ -227,39 +227,5 @@
       </inertial>
     </link>
-    <link name="${prefix}robotiq_85_right_finger_tip_link">
-      <visual>
-        <geometry>
-          <mesh filename="package://robotiq_description/meshes/visual/robotiq_85_finger_tip_link.dae"/>
-        </geometry>
-      </visual>
-      <collision name="robotiq_85_right_finger_tip_link_collision">
-        <origin xyz="0 0 0" rpy="0 0 0"/>
-        <geometry>
-          <box size="0.02 0.02 0.02"/>
-        </geometry>
-      </collision>
-      <visual>
-        <origin xyz="0 0 0" rpy="0 0 0"/>
-        <geometry>
-          <box size="0.02 0.02 0.02"/>
-        </geometry>
-        <material name="Green">
-          <color rgba="0 1 0 0.8"/>
-        </material>
-      </visual>
-      <inertial>
-        <mass value="0.019555" />
-        <origin xyz="0.0 0.0 0.0" />
-        <inertia ixx = "0.000002" ixy = "0.000000" ixz = "0.000000"
-             iyx = "0.000000" iyy = "0.000005" iyz = "0.000000"
-             izx = "0.000000" izy = "0.000000" izz = "0.000006" />
-      </inertial>
-    </link>
     <gazebo reference="${prefix}robotiq_85_left_finger_tip_link">
-      <kp>1000000.0</kp>
-      <kd>1.0</kd>
-      <mu1>1.0</mu1>
-      <mu2>1.0</mu2>
-      <minDepth>0.001</minDepth>
       <sensor name="left_finger_contact" type="contact">
         <always_on>true</always_on>
@@ -271,10 +237,34 @@
       </sensor>
     </gazebo>
+    <link name="${prefix}robotiq_85_right_finger_tip_link">
+      <visual>
+        <geometry>
+          <mesh filename="package://robotiq_description/meshes/visual/robotiq_85_finger_tip_link.dae"/>
+        </geometry>
+      </visual>
+      <collision name="robotiq_85_right_finger_tip_link_collision">
+        <origin xyz="0.03 0 0" rpy="0 0 0"/>
+        <geometry>
+          <box size="0.02 0.02 0.02"/>
+        </geometry>
+      </collision>
+      <visual>
+        <origin xyz="0.03 0 0" rpy="0 0 0"/>
+        <geometry>
+          <box size="0.02 0.02 0.02"/>
+        </geometry>
+        <material name="Green">
+          <color rgba="0 1 0 0.8"/>
+        </material>
+      </visual>
+      <inertial>
+        <mass value="0.019555" />
+        <origin xyz="0.0 0.0 0.0" />
+        <inertia ixx = "0.000002" ixy = "0.000000" ixz = "0.000000"
+             iyx = "0.000000" iyy = "0.000005" iyz = "0.000000"
+             izx = "0.000000" izy = "0.000000" izz = "0.000006" />
+      </inertial>
+    </link>
     <gazebo reference="${prefix}robotiq_85_right_finger_tip_link">
-      <kp>1000000.0</kp>
-      <kd>1.0</kd>
-      <mu1>1.0</mu1>
-      <mu2>1.0</mu2>
-      <minDepth>0.001</minDepth>
       <sensor name="right_finger_contact" type="contact">
         <always_on>true</always_on>

Commit message: Fix xacro

File: Industrial/robotiq_description/urdf/robotiq_85_gripper.urdf.xacro (robot description, xacro)
@@ -204,28 +204,33 @@
         </geometry>
       </visual>
+      <inertial>
+        <mass value="0.019555" />
+        <origin xyz="0.0 0.0 0.0" />
+        <inertia ixx = "0.000002" ixy = "0.000000" ixz = "0.000000"
+             iyx = "0.000000" iyy = "0.000005" iyz = "0.000000"
+             izx = "0.000000" izy = "0.000000" izz = "0.000006" />
+      </inertial>
+    </link>
+    <gazebo reference="${prefix}robotiq_85_left_finger_tip_link">
       <collision name="robotiq_85_left_finger_tip_link_collision">
-        <origin xyz="0.03 0 0" rpy="0 0 0"/>
-        <geometry>
-          <box size="0.02 0.02 0.02"/>
-        </geometry>
-      </collision>
-      <visual>
-        <origin xyz="0.03 0 0" rpy="0 0 0"/>
-        <geometry>
-          <box size="0.02 0.02 0.02"/>
-        </geometry>
-        <material name="Red">
-          <color rgba="1 0 0 0.8"/>
+        <pose>0.05 0 0 0 0 0</pose>
+        <geometry>
+          <box>
+            <size>0.08 0.08 0.08</size>
+          </box>
+        </geometry>
+      </collision>
+      <visual name="debug_left_contact_visual">
+        <pose>0.05 0 0 0 0 0</pose>
+        <geometry>
+          <box>
+            <size>0.08 0.08 0.08</size>
+          </box>
+        </geometry>
+        <material>
+          <ambient>1 0 0 0.4</ambient>
+          <diffuse>1 0 0 0.4</diffuse>
         </material>
       </visual>
-      <inertial>
-        <mass value="0.019555" />
-        <origin xyz="0.0 0.0 0.0" />
-        <inertia ixx = "0.000002" ixy = "0.000000" ixz = "0.000000"
-             iyx = "0.000000" iyy = "0.000005" iyz = "0.000000"
-             izx = "0.000000" izy = "0.000000" izz = "0.000006" />
-      </inertial>
-    </link>
-    <gazebo reference="${prefix}robotiq_85_left_finger_tip_link">
       <sensor name="left_finger_contact" type="contact">
         <always_on>true</always_on>
@@ -234,5 +239,4 @@
           <collision>robotiq_85_left_finger_tip_link_collision</collision>
         </contact>
-        <topic>/left_finger_contact</topic>
       </sensor>
     </gazebo>
@@ -243,28 +247,33 @@
         </geometry>
       </visual>
+      <inertial>
+        <mass value="0.019555" />
+        <origin xyz="0.0 0.0 0.0" />
+        <inertia ixx = "0.000002" ixy = "0.000000" ixz = "0.000000"
+             iyx = "0.000000" iyy = "0.000005" iyz = "0.000000"
+             izx = "0.000000" izy = "0.000000" izz = "0.000006" />
+      </inertial>
+    </link>
+    <gazebo reference="${prefix}robotiq_85_right_finger_tip_link">
       <collision name="robotiq_85_right_finger_tip_link_collision">
-        <origin xyz="0.03 0 0" rpy="0 0 0"/>
-        <geometry>
-          <box size="0.02 0.02 0.02"/>
-        </geometry>
-      </collision>
-      <visual>
-        <origin xyz="0.03 0 0" rpy="0 0 0"/>
-        <geometry>
-          <box size="0.02 0.02 0.02"/>
-        </geometry>
-        <material name="Green">
-          <color rgba="0 1 0 0.8"/>
+              <pose>0.05 0 0 0 0 0</pose>
+        <geometry>
+          <box>
+            <size>0.08 0.08 0.08</size>
+          </box>
+        </geometry>
+      </collision>
+      <visual name="debug_left_contact_visual">
+        <pose>0.05 0 0 0 0 0</pose>
+        <geometry>
+          <box>
+            <size>0.08 0.08 0.08</size>
+          </box>
+        </geometry>
+        <material>
+          <ambient>1 0 0 0.4</ambient>
+          <diffuse>1 0 0 0.4</diffuse>
         </material>
       </visual>
-      <inertial>
-        <mass value="0.019555" />
-        <origin xyz="0.0 0.0 0.0" />
-        <inertia ixx = "0.000002" ixy = "0.000000" ixz = "0.000000"
-             iyx = "0.000000" iyy = "0.000005" iyz = "0.000000"
-             izx = "0.000000" izy = "0.000000" izz = "0.000006" />
-      </inertial>
-    </link>
-    <gazebo reference="${prefix}robotiq_85_right_finger_tip_link">
       <sensor name="right_finger_contact" type="contact">
         <always_on>true</always_on>
@@ -273,5 +282,4 @@
           <collision>robotiq_85_right_finger_tip_link_collision</collision>
         </contact>
-        <topic>/right_finger_contact</topic>
       </sensor>
     </gazebo>
