Commit message: Fix xacro

File: Industrial/robotiq_description/urdf/robotiq_85_gripper.urdf.xacro (robot description, xacro)
@@ -204,13 +204,4 @@
         </geometry>
       </visual>
-      <inertial>
-        <mass value="0.019555" />
-        <origin xyz="0.0 0.0 0.0" />
-        <inertia ixx = "0.000002" ixy = "0.000000" ixz = "0.000000"
-             iyx = "0.000000" iyy = "0.000005" iyz = "0.000000"
-             izx = "0.000000" izy = "0.000000" izz = "0.000006" />
-      </inertial>
-    </link>
-    <gazebo reference="${prefix}robotiq_85_left_finger_tip_link">
       <collision name="robotiq_85_left_finger_tip_link_collision">
         <pose>0.05 0 0 0 0 0</pose>
@@ -221,16 +212,13 @@
         </geometry>
       </collision>
-      <visual name="debug_left_contact_visual">
-        <pose>0.05 0 0 0 0 0</pose>
-        <geometry>
-          <box>
-            <size>0.08 0.08 0.08</size>
-          </box>
-        </geometry>
-        <material>
-          <ambient>1 0 0 0.4</ambient>
-          <diffuse>1 0 0 0.4</diffuse>
-        </material>
-      </visual>
+      <inertial>
+        <mass value="0.019555" />
+        <origin xyz="0.0 0.0 0.0" />
+        <inertia ixx = "0.000002" ixy = "0.000000" ixz = "0.000000"
+             iyx = "0.000000" iyy = "0.000005" iyz = "0.000000"
+             izx = "0.000000" izy = "0.000000" izz = "0.000006" />
+      </inertial>
+    </link>
+    <gazebo reference="${prefix}robotiq_85_left_finger_tip_link">
       <sensor name="left_finger_contact" type="contact">
         <always_on>true</always_on>
@@ -247,13 +235,4 @@
         </geometry>
       </visual>
-      <inertial>
-        <mass value="0.019555" />
-        <origin xyz="0.0 0.0 0.0" />
-        <inertia ixx = "0.000002" ixy = "0.000000" ixz = "0.000000"
-             iyx = "0.000000" iyy = "0.000005" iyz = "0.000000"
-             izx = "0.000000" izy = "0.000000" izz = "0.000006" />
-      </inertial>
-    </link>
-    <gazebo reference="${prefix}robotiq_85_right_finger_tip_link">
       <collision name="robotiq_85_right_finger_tip_link_collision">
               <pose>0.05 0 0 0 0 0</pose>
@@ -264,16 +243,13 @@
         </geometry>
       </collision>
-      <visual name="debug_left_contact_visual">
-        <pose>0.05 0 0 0 0 0</pose>
-        <geometry>
-          <box>
-            <size>0.08 0.08 0.08</size>
-          </box>
-        </geometry>
-        <material>
-          <ambient>1 0 0 0.4</ambient>
-          <diffuse>1 0 0 0.4</diffuse>
-        </material>
-      </visual>
+      <inertial>
+        <mass value="0.019555" />
+        <origin xyz="0.0 0.0 0.0" />
+        <inertia ixx = "0.000002" ixy = "0.000000" ixz = "0.000000"
+             iyx = "0.000000" iyy = "0.000005" iyz = "0.000000"
+             izx = "0.000000" izy = "0.000000" izz = "0.000006" />
+      </inertial>
+    </link>
+    <gazebo reference="${prefix}robotiq_85_right_finger_tip_link">
       <sensor name="right_finger_contact" type="contact">
         <always_on>true</always_on>

Commit message: Fix xacro

File: Industrial/robotiq_description/urdf/robotiq_85_gripper.urdf.xacro (robot description, xacro)
@@ -205,9 +205,7 @@
       </visual>
       <collision name="robotiq_85_left_finger_tip_link_collision">
-        <pose>0.05 0 0 0 0 0</pose>
-        <geometry>
-          <box>
-            <size>0.08 0.08 0.08</size>
-          </box>
+        <origin xyz="0.05 0 0" rpy="0 0 0"/>
+        <geometry>
+          <box size="0.08 0.08 0.08"/>
         </geometry>
       </collision>
@@ -236,9 +234,7 @@
       </visual>
       <collision name="robotiq_85_right_finger_tip_link_collision">
-              <pose>0.05 0 0 0 0 0</pose>
-        <geometry>
-          <box>
-            <size>0.08 0.08 0.08</size>
-          </box>
+        <origin xyz="0.05 0 0" rpy="0 0 0"/>
+        <geometry>
+          <box size="0.08 0.08 0.08"/>
         </geometry>
       </collision>

Commit message: Fix xacro

File: Industrial/robotiq_description/urdf/robotiq_85_gripper.urdf.xacro (robot description, xacro)
@@ -205,9 +205,23 @@
       </visual>
       <collision name="robotiq_85_left_finger_tip_link_collision">
-        <origin xyz="0.05 0 0" rpy="0 0 0"/>
-        <geometry>
-          <box size="0.08 0.08 0.08"/>
-        </geometry>
-      </collision>
+        <origin xyz="0.03 0 0" rpy="0 0 0"/>
+        <geometry>
+          <box size="0.02 0.02 0.02"/>
+        </geometry>
+        <surface>
+          <contact>
+            <collide_without_contact>false</collide_without_contact>
+          </contact>
+        </surface>
+      </collision>
+      <visual>
+        <origin xyz="0.03 0 0" rpy="0 0 0"/>
+        <geometry>
+          <box size="0.02 0.02 0.02"/>
+        </geometry>
+        <material name="red_debug">
+          <color rgba="1 0 0 0.5"/>
+        </material>
+      </visual>
       <inertial>
         <mass value="0.019555" />
@@ -234,9 +248,23 @@
       </visual>
       <collision name="robotiq_85_right_finger_tip_link_collision">
-        <origin xyz="0.05 0 0" rpy="0 0 0"/>
-        <geometry>
-          <box size="0.08 0.08 0.08"/>
-        </geometry>
-      </collision>
+        <origin xyz="0.03 0 0" rpy="0 0 0"/>
+        <geometry>
+          <box size="0.02 0.02 0.02"/>
+        </geometry>
+        <surface>
+          <contact>
+            <collide_without_contact>false</collide_without_contact>
+          </contact>
+        </surface>
+      </collision>
+      <visual>
+        <origin xyz="0.03 0 0" rpy="0 0 0"/>
+        <geometry>
+          <box size="0.02 0.02 0.02"/>
+        </geometry>
+        <material name="red_debug">
+          <color rgba="1 0 0 0.5"/>
+        </material>
+      </visual>
       <inertial>
         <mass value="0.019555" />

Commit message: Fix xacro

File: Industrial/robotiq_description/urdf/robotiq_85_gripper.urdf.xacro (robot description, xacro)
@@ -204,8 +204,19 @@
         </geometry>
       </visual>
+      <inertial>
+        <mass value="0.019555" />
+        <origin xyz="0.0 0.0 0.0" />
+        <inertia ixx = "0.000002" ixy = "0.000000" ixz = "0.000000"
+             iyx = "0.000000" iyy = "0.000005" iyz = "0.000000"
+             izx = "0.000000" izy = "0.000000" izz = "0.000006" />
+      </inertial>
+    </link>
+    <gazebo reference="${prefix}robotiq_85_left_finger_tip_link">
       <collision name="robotiq_85_left_finger_tip_link_collision">
-        <origin xyz="0.03 0 0" rpy="0 0 0"/>
-        <geometry>
-          <box size="0.02 0.02 0.02"/>
+        <pose>0.03 0 0 0 0 0</pose>
+        <geometry>
+          <box>
+            <size>0.02 0.02 0.02</size>
+          </box>
         </geometry>
         <surface>
@@ -215,27 +226,23 @@
         </surface>
       </collision>
-      <visual>
-        <origin xyz="0.03 0 0" rpy="0 0 0"/>
-        <geometry>
-          <box size="0.02 0.02 0.02"/>
-        </geometry>
-        <material name="red_debug">
-          <color rgba="1 0 0 0.5"/>
+      <visual name="left_contact_debug_visual">
+        <pose>0.03 0 0 0 0 0</pose>
+        <geometry>
+          <box>
+            <size>0.02 0.02 0.02</size>
+          </box>
+        </geometry>
+        <material>
+          <ambient>1 0 0 0.5</ambient>
+          <diffuse>1 0 0 0.5</diffuse>
         </material>
       </visual>
-      <inertial>
-        <mass value="0.019555" />
-        <origin xyz="0.0 0.0 0.0" />
-        <inertia ixx = "0.000002" ixy = "0.000000" ixz = "0.000000"
-             iyx = "0.000000" iyy = "0.000005" iyz = "0.000000"
-             izx = "0.000000" izy = "0.000000" izz = "0.000006" />
-      </inertial>
-    </link>
-    <gazebo reference="${prefix}robotiq_85_left_finger_tip_link">
       <sensor name="left_finger_contact" type="contact">
         <always_on>true</always_on>
         <update_rate>100</update_rate>
         <contact>
-          <collision>robotiq_85_left_finger_tip_link_collision</collision>
+          <collision>
+            robotiq_85_left_finger_tip_link_collision
+          </collision>
         </contact>
       </sensor>
@@ -247,8 +254,19 @@
         </geometry>
       </visual>
+      <inertial>
+        <mass value="0.019555" />
+        <origin xyz="0.0 0.0 0.0" />
+        <inertia ixx = "0.000002" ixy = "0.000000" ixz = "0.000000"
+             iyx = "0.000000" iyy = "0.000005" iyz = "0.000000"
+             izx = "0.000000" izy = "0.000000" izz = "0.000006" />
+      </inertial>
+    </link>
+    <gazebo reference="${prefix}robotiq_85_right_finger_tip_link">
       <collision name="robotiq_85_right_finger_tip_link_collision">
-        <origin xyz="0.03 0 0" rpy="0 0 0"/>
-        <geometry>
-          <box size="0.02 0.02 0.02"/>
+        <pose>0.03 0 0 0 0 0</pose>
+        <geometry>
+          <box>
+            <size>0.02 0.02 0.02</size>
+          </box>
         </geometry>
         <surface>
@@ -258,27 +276,23 @@
         </surface>
       </collision>
-      <visual>
-        <origin xyz="0.03 0 0" rpy="0 0 0"/>
-        <geometry>
-          <box size="0.02 0.02 0.02"/>
-        </geometry>
-        <material name="red_debug">
-          <color rgba="1 0 0 0.5"/>
+      <visual name="right_contact_debug_visual">
+        <pose>0.03 0 0 0 0 0</pose>
+        <geometry>
+          <box>
+            <size>0.02 0.02 0.02</size>
+          </box>
+        </geometry>
+        <material>
+          <ambient>1 0 0 0.5</ambient>
+          <diffuse>1 0 0 0.5</diffuse>
         </material>
       </visual>
-      <inertial>
-        <mass value="0.019555" />
-        <origin xyz="0.0 0.0 0.0" />
-        <inertia ixx = "0.000002" ixy = "0.000000" ixz = "0.000000"
-             iyx = "0.000000" iyy = "0.000005" iyz = "0.000000"
-             izx = "0.000000" izy = "0.000000" izz = "0.000006" />
-      </inertial>
-    </link>
-    <gazebo reference="${prefix}robotiq_85_right_finger_tip_link">
       <sensor name="right_finger_contact" type="contact">
         <always_on>true</always_on>
         <update_rate>100</update_rate>
         <contact>
-          <collision>robotiq_85_right_finger_tip_link_collision</collision>
+          <collision>
+            robotiq_85_right_finger_tip_link_collision
+          </collision>
         </contact>
       </sensor>

Commit message: Fix xacro

File: Industrial/robotiq_description/urdf/robotiq_85_gripper.urdf.xacro (robot description, xacro)
@@ -204,4 +204,10 @@
         </geometry>
       </visual>
+      <collision name="${prefix}robotiq_85_left_finger_tip_collision">
+        <origin xyz="0.03 0 0" rpy="0 0 0"/>
+        <geometry>
+          <box size="0.02 0.02 0.02"/>
+        </geometry>
+      </collision>
       <inertial>
         <mass value="0.019555" />
@@ -213,29 +219,4 @@
     </link>
     <gazebo reference="${prefix}robotiq_85_left_finger_tip_link">
-      <collision name="robotiq_85_left_finger_tip_link_collision">
-        <pose>0.03 0 0 0 0 0</pose>
-        <geometry>
-          <box>
-            <size>0.02 0.02 0.02</size>
-          </box>
-        </geometry>
-        <surface>
-          <contact>
-            <collide_without_contact>false</collide_without_contact>
-          </contact>
-        </surface>
-      </collision>
-      <visual name="left_contact_debug_visual">
-        <pose>0.03 0 0 0 0 0</pose>
-        <geometry>
-          <box>
-            <size>0.02 0.02 0.02</size>
-          </box>
-        </geometry>
-        <material>
-          <ambient>1 0 0 0.5</ambient>
-          <diffuse>1 0 0 0.5</diffuse>
-        </material>
-      </visual>
       <sensor name="left_finger_contact" type="contact">
         <always_on>true</always_on>
@@ -243,5 +224,5 @@
         <contact>
           <collision>
-            robotiq_85_left_finger_tip_link_collision
+            ${prefix}robotiq_85_left_finger_tip_collision
           </collision>
         </contact>
@@ -254,4 +235,10 @@
         </geometry>
       </visual>
+      <collision name="${prefix}robotiq_85_right_finger_tip_collision">
+        <origin xyz="0.03 0 0" rpy="0 0 0"/>
+        <geometry>
+          <box size="0.02 0.02 0.02"/>
+        </geometry>
+      </collision>
       <inertial>
         <mass value="0.019555" />
@@ -263,29 +250,4 @@
     </link>
     <gazebo reference="${prefix}robotiq_85_right_finger_tip_link">
-      <collision name="robotiq_85_right_finger_tip_link_collision">
-        <pose>0.03 0 0 0 0 0</pose>
-        <geometry>
-          <box>
-            <size>0.02 0.02 0.02</size>
-          </box>
-        </geometry>
-        <surface>
-          <contact>
-            <collide_without_contact>false</collide_without_contact>
-          </contact>
-        </surface>
-      </collision>
-      <visual name="right_contact_debug_visual">
-        <pose>0.03 0 0 0 0 0</pose>
-        <geometry>
-          <box>
-            <size>0.02 0.02 0.02</size>
-          </box>
-        </geometry>
-        <material>
-          <ambient>1 0 0 0.5</ambient>
-          <diffuse>1 0 0 0.5</diffuse>
-        </material>
-      </visual>
       <sensor name="right_finger_contact" type="contact">
         <always_on>true</always_on>
@@ -293,5 +255,5 @@
         <contact>
           <collision>
-            robotiq_85_right_finger_tip_link_collision
+            ${prefix}robotiq_85_right_finger_tip_collision
           </collision>
         </contact>

Commit message: Fix xacro

File: Industrial/robotiq_description/urdf/robotiq_85_gripper.urdf.xacro (robot description, xacro)
@@ -204,5 +204,5 @@
         </geometry>
       </visual>
-      <collision name="${prefix}robotiq_85_left_finger_tip_collision">
+      <collision>
         <origin xyz="0.03 0 0" rpy="0 0 0"/>
         <geometry>
@@ -224,5 +224,5 @@
         <contact>
           <collision>
-            ${prefix}robotiq_85_left_finger_tip_collision
+            robotiq_85_left_finger_tip_link_collision
           </collision>
         </contact>

Commit message: Fix xacro

File: Industrial/robotiq_description/urdf/robotiq_85_gripper.urdf.xacro (robot description, xacro)
@@ -235,5 +235,5 @@
         </geometry>
       </visual>
-      <collision name="${prefix}robotiq_85_right_finger_tip_collision">
+      <collision>
         <origin xyz="0.03 0 0" rpy="0 0 0"/>
         <geometry>
@@ -255,5 +255,5 @@
         <contact>
           <collision>
-            ${prefix}robotiq_85_right_finger_tip_collision
+            robotiq_85_right_finger_tip_link_collision
           </collision>
         </contact>
