Commit message: Test ball joints

File: CustomRobots/turtlebot3/models/turtlebot3/turtlebot3_common.urdf.xacro (robot description, xacro)
@@ -135,56 +135,4 @@
       </visual>
     </link>
-    <link name="caster_back_right_link">
-      <origin rpy="-1.57 0 0" xyz="-0.177 -0.064 -0.004"/>
-      <inertial>
-        <mass value="0.001"/>
-        <inertia ixx="0.00001" ixy="0" ixz="0" iyy="0.00001" iyz="0" izz="0.00001"/>
-      </inertial>
-      <collision>
-        <geometry>
-          <sphere radius="0.005"/>
-        </geometry>
-        <gazebo>
-          <surface>
-            <contact>
-              <ode>
-                <soft_cfm>0</soft_cfm>
-                <soft_erp>0.2</soft_erp>
-                <kp>1e+5</kp>
-                <kd>1</kd>
-                <max_vel>0.01</max_vel>
-                <min_depth>0.001</min_depth>
-              </ode>
-            </contact>
-          </surface>
-        </gazebo>
-      </collision>
-    </link>
-    <link name="caster_back_left_link">
-      <origin rpy="-1.57 0 0" xyz="-0.177 0.064 -0.004"/>
-      <inertial>
-        <mass value="0.001"/>
-        <inertia ixx="0.00001" ixy="0" ixz="0" iyy="0.00001" iyz="0" izz="0.00001"/>
-      </inertial>
-      <collision>
-        <geometry>
-          <sphere radius="0.005"/>
-        </geometry>
-        <gazebo>
-          <surface>
-            <contact>
-              <ode>
-                <soft_cfm>0</soft_cfm>
-                <soft_erp>0.2</soft_erp>
-                <kp>1e+5</kp>
-                <kd>1</kd>
-                <max_vel>0.01</max_vel>
-                <min_depth>0.001</min_depth>
-              </ode>
-            </contact>
-          </surface>
-        </gazebo>
-      </collision>
-    </link>
     <link name="camera_link"/>
     <joint name="base_to_base_link" type="fixed">
@@ -215,14 +163,40 @@
     </joint>
     <!-- Ball joints -->
-    <joint name="caster_back_right_joint" type="continuous">
+    <joint name="caster_back_left_joint" type="fixed">
+      <parent link="base_link"/>
+      <child link="caster_back_left_link"/>
+      <origin xyz="-0.177 0.064 -0.004" rpy="-1.57 0 0"/>
+    </joint>
+    <link name="caster_back_left_link">
+      <collision>
+        <origin xyz="0 0.001 0" rpy="0 0 0"/>
+        <geometry>
+          <box size="0.030 0.009 0.020"/>
+        </geometry>
+      </collision>
+      <inertial>
+        <origin xyz="0 0 0" />
+        <mass value="0.005" />
+        <inertia ixx="0.001" ixy="0.0" ixz="0.0" iyy="0.001" iyz="0.0" izz="0.001" />
+      </inertial>
+    </link>
+    <joint name="caster_back_right_joint" type="fixed">
       <parent link="base_link"/>
       <child link="caster_back_right_link"/>
-      <limit effort="20" velocity="100"/>
-    </joint>
-    <joint name="caster_back_left_joint" type="continuous">
-      <parent link="base_link"/>
-      <child link="caster_back_left_link"/>
-      <limit effort="20" velocity="100"/>
-    </joint>
+      <origin xyz="-0.177 -0.064 -0.004" rpy="-1.57 0 0"/>
+    </joint>
+    <link name="caster_back_right_link">
+      <collision>
+        <origin xyz="0 0.001 0" rpy="0 0 0"/>
+        <geometry>
+          <box size="0.030 0.009 0.020"/>
+        </geometry>
+      </collision>
+      <inertial>
+        <origin xyz="0 0 0" />
+        <mass value="0.005" />
+        <inertia ixx="0.001" ixy="0.0" ixz="0.0" iyy="0.001" iyz="0.0" izz="0.001" />
+      </inertial>
+    </link>
     <xacro:imu parent="imu_link" topic="turtlebot3/imu" xyz="-0.032 0 0.068" rpy="0 0 0"/>
     <xacro:lidar xyz="-0.064 0 0.121" rpy="0 0 0" name="lidar" parent="base_link" topic="turtlebot3/laser/scan"/>

Commit message: Fix import typos

File: CustomRobots/turtlebot3/models/turtlebot3/turtlebot3_common.urdf.xacro (robot description, xacro)
@@ -1,5 +1,5 @@
 <?xml version="1.0" ?>
 <robot xmlns:xacro="http://ros.org/wiki/xacro">
-  <xacro:include filename="$(find custom_robots)/models/turtlebo3/turtlebo3_gz.urdf.xacro"/>
+  <xacro:include filename="$(find custom_robots)/models/turtlebot3/turtlebot3_gz.urdf.xacro"/>
   <xacro:macro name="turtlebot3">
     <link name="base_footprint"></link>
@@ -18,5 +18,5 @@
         <origin rpy="0 0 0" xyz="-0.064  0 0"/>
         <geometry>
-          <mesh filename="$(find custom_robots)/model/urtlebot3/meshes/waffle_base.dae" scale="0.001 0.001 0.001"/>
+          <mesh filename="$(find custom_robots)/model/turtlebot3/meshes/waffle_base.dae" scale="0.001 0.001 0.001"/>
         </geometry>
         <gazebo>
@@ -72,5 +72,5 @@
         <origin rpy="0 0 0" xyz="0.0 0.144 0.023"/>
         <geometry>
-          <mesh filename="$(find custom_robots)/model/urtlebot3/meshes/tire.dae" scale="0.001 0.001 0.001"/>
+          <mesh filename="$(find custom_robots)/model/turtlebot3/meshes/tire.dae" scale="0.001 0.001 0.001"/>
         </geometry>
         <gazebo>
@@ -123,5 +123,5 @@
         <origin rpy="0 0 0" xyz="0.0 -0.144 0.023"/>
         <geometry>
-          <mesh filename="$(find custom_robots)/model/urtlebot3/meshes/tire.dae" scale="0.001 0.001 0.001"/>
+          <mesh filename="$(find custom_robots)/model/turtlebot3/meshes/tire.dae" scale="0.001 0.001 0.001"/>
         </geometry>
         <gazebo>
@@ -200,5 +200,5 @@
     </link>
     <xacro:imu parent="imu_link" topic="turtlebot3/imu" xyz="-0.032 0 0.068" rpy="0 0 0"/>
-    <xacro:lidar xyz="-0.064 0 0.121" rpy="0 0 0" name="lidar" parent="base_link" topic="turtlebot3/laser/scan"/>
+    <xacro:laser xyz="-0.064 0 0.121" rpy="0 0 0" name="lidar" parent="base_link" topic="turtlebot3/laser/scan"/>
     <xacro:velocity topic="turtlebot3/cmd_vel"/>
     <xacro:odom topic="/turtlebot3/odom" freq="50"/>

Commit message: Fix errors in turtlebot3

File: CustomRobots/turtlebot3/models/turtlebot3/turtlebot3_common.urdf.xacro (robot description, xacro)
@@ -3,4 +3,17 @@
   <xacro:include filename="$(find custom_robots)/models/turtlebot3/turtlebot3_gz.urdf.xacro"/>
   <xacro:macro name="turtlebot3">
+    <!-- Init colour -->
+    <material name="black">
+      <color rgba="0.0 0.0 0.0 1.0"/>
+    </material>
+    <material name="dark">
+      <color rgba="0.3 0.3 0.3 1.0"/>
+    </material>
+    <material name="light_black">
+      <color rgba="0.4 0.4 0.4 1.0"/>
+    </material>
+    <material name="white">
+      <color rgba="1.0 1.0 1.0 1.0"/>
+    </material>
     <link name="base_footprint"></link>
     <link name="base_link">
@@ -18,27 +31,15 @@
         <origin rpy="0 0 0" xyz="-0.064  0 0"/>
         <geometry>
-          <mesh filename="$(find custom_robots)/model/turtlebot3/meshes/waffle_base.dae" scale="0.001 0.001 0.001"/>
+          <mesh filename="file://$(find custom_robots)/models/turtlebot3/meshes/waffle_base.dae" scale="0.001 0.001 0.001"/>
         </geometry>
-        <gazebo>
-          <material>
-            <ambient>1 1 1 1</ambient>
-            <diffuse>1 1 1 1</diffuse>
-            <specular>0.2 0.2 0.2 1</specular>
-            <emissive>0 0 0 1</emissive>
-            <script>
-              <name>Gazebo/Grey</name>
-            </script>
-          </material>
-        </gazebo>
+        <material name="light_black"/>
       </visual>
     </link>
     <link name="wheel_left_link">
       <inertial>
-        <origin rpy="-1.57 0 0" xyz="0.0 0.144 0.023"/>
         <mass value="0.1"/>
         <inertia ixx="1.1175580e-05" ixy="0" ixz="0" iyy="1.1175580e-05" iyz="0" izz="2.0712558e-05"/>
       </inertial>
       <collision>
-        <origin rpy="-1.57 0 0" xyz="0.0 0.144 0.023"/>
         <geometry>
           <cylinder radius="0.033" length="0.018"/>
@@ -70,26 +71,17 @@
       </collision>
       <visual >
-        <origin rpy="0 0 0" xyz="0.0 0.144 0.023"/>
+        <origin rpy="1.57 0 0" xyz="0 0 0"/>
         <geometry>
-          <mesh filename="$(find custom_robots)/model/turtlebot3/meshes/tire.dae" scale="0.001 0.001 0.001"/>
+          <mesh filename="file://$(find custom_robots)/models/turtlebot3/meshes/tire.dae" scale="0.001 0.001 0.001"/>
         </geometry>
-        <gazebo>
-          <material>
-            <ambient>1 1 1 1</ambient>
-            <diffuse>1 1 1 1</diffuse>
-            <specular>0.2 0.2 0.2 1</specular>
-            <emissive>0 0 0 1</emissive>
-          </material>
-        </gazebo>
+        <material name="black"/>
       </visual>
     </link>
     <link name="wheel_right_link">
       <inertial>
-        <origin rpy="-1.57 0 0" xyz="0.0 -0.144 0.023"/>
         <mass value="0.1"/>
         <inertia ixx="1.1175580e-05" ixy="0" ixz="0" iyy="1.1175580e-05" iyz="0" izz="2.0712558e-05"/>
       </inertial>
       <collision>
-        <origin rpy="-1.57 0 0" xyz="0.0 -0.144 0.023"/>
         <geometry>
           <cylinder radius="0.033" length="0.018"/>
@@ -121,16 +113,9 @@
       </collision>
       <visual >
-        <origin rpy="0 0 0" xyz="0.0 -0.144 0.023"/>
+        <origin rpy="1.57 0 0" xyz="0 0 0"/>
         <geometry>
-          <mesh filename="$(find custom_robots)/model/turtlebot3/meshes/tire.dae" scale="0.001 0.001 0.001"/>
+          <mesh filename="file://$(find custom_robots)/models/turtlebot3/meshes/tire.dae" scale="0.001 0.001 0.001"/>
         </geometry>
-        <gazebo>
-          <material>
-            <ambient>1 1 1 1</ambient>
-            <diffuse>1 1 1 1</diffuse>
-            <specular>0.2 0.2 0.2 1</specular>
-            <emissive>0 0 0 1</emissive>
-          </material>
-        </gazebo>
+        <material name="black"/>
       </visual>
     </link>

File: CustomRobots/turtlebot3/models/turtlebot3/turtlebot3_gz.urdf.xacro (robot description, xacro)
@@ -93,4 +93,5 @@
           <mesh filename="file://$(find custom_robots)/models/turtlebot3/meshes/lds.dae" scale="0.001 0.001 0.001"/>
         </geometry>
+        <material name="dark"/>
       </visual>
     </link>
