Commit message: turtlebot burger RI

File: CustomRobots/turtlebot3/models/turtlebot3/turtlebot3_gz.urdf.xacro (robot description, xacro)
@@ -153,5 +153,5 @@
     </gazebo>
   </xacro:macro>
-  <xacro:macro name="velocity" params="namespace">
+  <xacro:macro name="velocity" params="namespace wheel_separation:=0.287">
     <gazebo>
       <plugin filename="gz-sim-diff-drive-system" name="gz::sim::systems::DiffDrive">
@@ -160,5 +160,5 @@
         <right_joint>wheel_right_joint</right_joint>
         <!-- kinematics -->
-        <wheel_separation>0.287</wheel_separation>
+        <wheel_separation>${wheel_separation}</wheel_separation>
         <wheel_radius>0.033</wheel_radius>
         <!-- limits -->
@@ -183,5 +183,5 @@
     </gazebo>
   </xacro:macro>
-  <xacro:macro name="noise_odom" params="namespace a1 a2 a3 a4">
+  <xacro:macro name="noise_odom" params="namespace a1 a2 a3 a4 wheel_separation:=0.287">
     <gazebo>
       <plugin filename="libNoisyOdometryPlugin.so" name="custom_plugins::NoisyOdometryPlugin">
@@ -193,5 +193,5 @@
         <right_joint>wheel_right_joint</right_joint>
         <wheel_radius>0.033</wheel_radius>
-        <wheel_separation>0.287</wheel_separation>
+        <wheel_separation>${wheel_separation}</wheel_separation>
         <alpha1>${a1}</alpha1>
         <alpha2>${a2}</alpha2>
