Commit message: reduce odometry noise in turtlebot 3 model

File: CustomRobots/turtlebot3/models/turtlebot3/turtlebot3.urdf.xacro (robot description, xacro)
@@ -6,8 +6,8 @@
   <xacro:property name="noise_level" value="$(arg noise_level)"/>
   <xacro:if value="${noise_level == 'low'}">
-    <xacro:property name="a1" value="0.1" />
-    <xacro:property name="a2" value="0.1" />
-    <xacro:property name="a3" value="0.05" />
-    <xacro:property name="a4" value="0.05" />
+    <xacro:property name="a1" value="0.01" />
+    <xacro:property name="a2" value="0.01" />
+    <xacro:property name="a3" value="0.005" />
+    <xacro:property name="a4" value="0.005" />
   </xacro:if>
   <xacro:if value="${noise_level == 'med'}">

Commit message: Make odometry noise step-rate independent and rescale levels

File: CustomRobots/turtlebot3/models/turtlebot3/turtlebot3.urdf.xacro (robot description, xacro)
@@ -5,21 +5,22 @@
   <xacro:arg name="noise_level" default="none"/>
   <xacro:property name="noise_level" value="$(arg noise_level)"/>
+  <!-- Odometry noise per difficulty (drift std ~ alpha*sqrt(distance)). -->
   <xacro:if value="${noise_level == 'low'}">
     <xacro:property name="a1" value="0.01" />
     <xacro:property name="a2" value="0.01" />
-    <xacro:property name="a3" value="0.005" />
-    <xacro:property name="a4" value="0.005" />
+    <xacro:property name="a3" value="0.01" />
+    <xacro:property name="a4" value="0.01" />
   </xacro:if>
   <xacro:if value="${noise_level == 'med'}">
-    <xacro:property name="a1" value="0.5" />
-    <xacro:property name="a2" value="0.5" />
+    <xacro:property name="a1" value="0.05" />
+    <xacro:property name="a2" value="0.05" />
+    <xacro:property name="a3" value="0.05" />
+    <xacro:property name="a4" value="0.05" />
+  </xacro:if>
+  <xacro:if value="${noise_level == 'high'}">
+    <xacro:property name="a1" value="0.25" />
+    <xacro:property name="a2" value="0.25" />
     <xacro:property name="a3" value="0.25" />
     <xacro:property name="a4" value="0.25" />
-  </xacro:if>
-  <xacro:if value="${noise_level == 'high'}">
-    <xacro:property name="a1" value="1.5" />
-    <xacro:property name="a2" value="1.5" />
-    <xacro:property name="a3" value="0.8" />
-    <xacro:property name="a4" value="0.8" />
   </xacro:if>
   <xacro:include filename="$(find custom_robots)/models/turtlebot3/turtlebot3_gz.urdf.xacro"/>
