Commit message: Update turtlebot3

File: CustomRobots/turtlebot3/models/turtlebot3/turtlebot3.urdf.xacro (robot description, xacro)
@@ -4,5 +4,7 @@
   <xacro:arg name="camera" default="true"/>
   <xacro:arg name="noise_level" default="none"/>
+  <xacro:arg name="namespace" default="vacuum_cleaner"/>
   <xacro:property name="noise_level" value="$(arg noise_level)"/>
+  <xacro:property name="namespace" value="$(arg namespace)"/>
   <!-- Odometry noise per difficulty (drift std ~ alpha*sqrt(distance)). -->
   <xacro:if value="${noise_level == 'low'}">
@@ -26,10 +28,10 @@
   <xacro:include filename="$(find custom_robots)/models/turtlebot3/turtlebot3_gz.urdf.xacro"/>
   <xacro:include filename="$(find custom_robots)/models/turtlebot3/turtlebot3_common.urdf.xacro"/>
-  <xacro:turtlebot3/>
+  <xacro:turtlebot3 namespace="${namespace}"/>
   <xacro:if value="$(arg camera)">
-    <xacro:camera xyz="0.069 -0.047 0.107" rpy="0 0 0" name="camera_rgb" parent="camera_link" topic="turtlebot3/camera"/>
+    <xacro:camera xyz="0.069 -0.047 0.107" rpy="0 0 0" name="camera" parent="camera_link" namespace="${namespace}"/>
   </xacro:if>
   <xacro:unless value="${noise_level == 'none'}">
-    <xacro:noise_odom topic="/turtlebot3/odom_noisy" a1="${a1}" a2="${a2}" a3="${a3}" a4="${a4}"/>
+    <xacro:noise_odom a1="${a1}" a2="${a2}" a3="${a3}" a4="${a4}" namespace="${namespace}"/>
   </xacro:unless>
 </robot>

File: CustomRobots/turtlebot3/models/turtlebot3/turtlebot3_common.urdf.xacro (robot description, xacro)
@@ -2,5 +2,5 @@
 <robot xmlns:xacro="http://ros.org/wiki/xacro">
   <xacro:include filename="$(find custom_robots)/models/turtlebot3/turtlebot3_gz.urdf.xacro"/>
-  <xacro:macro name="turtlebot3">
+  <xacro:macro name="turtlebot3" params="namespace">
     <!-- Init colour -->
     <material name="black">
@@ -134,8 +134,8 @@
       </inertial>
     </link>
-    <xacro:imu parent="imu_link" topic="turtlebot3/imu" xyz="-0.032 0 0.068" rpy="0 0 0"/>
-    <xacro:laser xyz="-0.064 0 0.121" rpy="0 0 0" name="lidar" parent="base_link" topic="turtlebot3/laser/scan"/>
-    <xacro:velocity topic="turtlebot3/cmd_vel"/>
-    <xacro:odom topic="/turtlebot3/odom" freq="50"/>
+    <xacro:imu parent="imu_link" xyz="-0.032 0 0.068" rpy="0 0 0" namespace="${namespace}"/>
+    <xacro:laser xyz="-0.064 0 0.121" rpy="0 0 0" name="laser" parent="base_link" namespace="${namespace}"/>
+    <xacro:velocity namespace="${namespace}"/>
+    <xacro:odom namespace="${namespace}" freq="50"/>
   </xacro:macro>
 </robot>

File: CustomRobots/turtlebot3/models/turtlebot3/turtlebot3_gz.urdf.xacro (robot description, xacro)
@@ -1,5 +1,5 @@
 <?xml version="1.0"?>
 <robot xmlns:xacro="http://ros.org/wiki/xacro">
-  <xacro:macro name="camera" params="xyz rpy name parent topic">
+  <xacro:macro name="camera" params="xyz rpy name parent namespace">
     <link name="${name}_link">
       <inertial>
@@ -18,8 +18,8 @@
         <visualize>true</visualize>
         <update_rate>30</update_rate>
-        <topic>/${topic}/image_raw</topic>
+        <topic>/${namespace}/${name}/image_raw</topic>
         <gz_frame_id>${name}_link</gz_frame_id>
         <camera name="${name}">
-          <camera_info_topic>/${topic}/camera_info</camera_info_topic>
+          <camera_info_topic>/${namespace}/${name}/camera_info</camera_info_topic>
           <horizontal_fov>1.02974</horizontal_fov>
           <image>
@@ -41,5 +41,5 @@
     </gazebo>
   </xacro:macro>
-  <xacro:macro name="laser" params="xyz rpy name parent topic">
+  <xacro:macro name="laser" params="xyz rpy name parent namespace">
     <link name="${name}_link">
       <inertial>
@@ -71,5 +71,5 @@
         <visualize>1</visualize>
         <update_rate>5</update_rate>
-        <topic>${topic}</topic>
+        <topic>/${namespace}/${name}/scan</topic>
         <gz_frame_id>${name}_link</gz_frame_id>
         <lidar>
@@ -91,5 +91,5 @@
     </gazebo>
   </xacro:macro>
-  <xacro:macro name="imu" params="parent topic xyz rpy">
+  <xacro:macro name="imu" params="parent namespace xyz rpy">
     <gazebo>
       <plugin filename="gz-sim-imu-system" name="gz::sim::systems::Imu">
@@ -107,5 +107,5 @@
         <always_on>1</always_on>
         <update_rate>200</update_rate>
-        <topic>${topic}</topic>
+        <topic>/${namespace}/imu</topic>
         <imu>
           <angular_velocity>
@@ -153,5 +153,5 @@
     </gazebo>
   </xacro:macro>
-  <xacro:macro name="velocity" params="topic">
+  <xacro:macro name="velocity" params="namespace">
     <gazebo>
       <plugin filename="gz-sim-diff-drive-system" name="gz::sim::systems::DiffDrive">
@@ -164,5 +164,5 @@
         <!-- limits -->
         <max_linear_acceleration>1.0</max_linear_acceleration>
-        <topic>${topic}</topic>
+        <topic>/${namespace}/cmd_vel</topic>
         <frame_id>odom</frame_id>
         <!-- <tf_topic>/tf</tf_topic> -->
@@ -172,5 +172,5 @@
     </gazebo>
   </xacro:macro>
-  <xacro:macro name="odom" params="topic freq">
+  <xacro:macro name="odom" params="namespace freq">
     <gazebo>
       <plugin filename="gz-sim-odometry-publisher-system" name="gz::sim::systems::OdometryPublisher">
@@ -178,13 +178,13 @@
         <robot_base_frame>base_footprint</robot_base_frame>
         <odom_publish_frequency>${freq}</odom_publish_frequency>
-        <odom_topic>${topic}</odom_topic>
+        <odom_topic>/${namespace}/odom</odom_topic>
         <dimensions>3</dimensions>
       </plugin>
     </gazebo>
   </xacro:macro>
-  <xacro:macro name="noise_odom" params="topic a1 a2 a3 a4">
+  <xacro:macro name="noise_odom" params="namespace a1 a2 a3 a4">
     <gazebo>
       <plugin filename="libNoisyOdometryPlugin.so" name="custom_plugins::NoisyOdometryPlugin">
-        <ros_topic>${topic}</ros_topic>
+        <ros_topic>/${namespace}/odom_noisy</ros_topic>
         <frame_id>odom</frame_id>
         <child_frame_id>base</child_frame_id>

Commit message: Fix dupe link

File: CustomRobots/turtlebot3/models/turtlebot3/turtlebot3.urdf.xacro (robot description, xacro)
@@ -30,5 +30,5 @@
   <xacro:turtlebot3 namespace="${namespace}"/>
   <xacro:if value="$(arg camera)">
-    <xacro:camera xyz="0.069 -0.047 0.107" rpy="0 0 0" name="camera" parent="camera_link" namespace="${namespace}"/>
+    <xacro:camera xyz="0.069 -0.047 0.107" rpy="0 0 0" name="camera" parent="camera_base_link" namespace="${namespace}"/>
   </xacro:if>
   <xacro:unless value="${noise_level == 'none'}">

File: CustomRobots/turtlebot3/models/turtlebot3/turtlebot3_common.urdf.xacro (robot description, xacro)
@@ -70,5 +70,5 @@
       </visual>
     </link>
-    <link name="camera_link"/>
+    <link name="camera_base_link"/>
     <joint name="base_to_base_link" type="fixed">
       <parent link="base_footprint"/>
@@ -79,5 +79,5 @@
     <joint name="camera_joint" type="fixed">
       <parent link="base_link"/>
-      <child link="camera_link"/>
+      <child link="camera_base_link"/>
       <origin xyz="0.064 -0.065 0.094" rpy="0 0 0"/>
       <axis xyz="0 0 1"/>

Commit message: turtlebot burger update

File: CustomRobots/turtlebot3/models/turtlebot3/turtlebot3.urdf.xacro (robot description, xacro)
@@ -31,5 +31,5 @@
   <xacro:turtlebot3 namespace="${namespace}"/>
   <xacro:if value="$(arg camera)">
-    <xacro:camera xyz="0.069 -0.047 0.107" rpy="0 0 0" name="camera" parent="camera_base_link" namespace="${namespace}"/>
+    <xacro:camera xyz="0.005 0.018 0.013" rpy="0 0 0" name="camera" parent="camera_base_link" namespace="${namespace}"/>
   </xacro:if>
   <!-- Beacon on top so a drone above can pick it out by color, only for follow_turtlebot -->

File: CustomRobots/turtlebot3/models/turtlebot3/turtlebot3_burger_common.urdf.xacro (robot description, xacro)
@@ -2,12 +2,13 @@
 <robot xmlns:xacro="http://ros.org/wiki/xacro">
   <xacro:include filename="$(find custom_robots)/models/turtlebot3/turtlebot3_gz.urdf.xacro"/>
-  <xacro:property name="burger_meshes" value="file://$(find custom_robots)/models/turtlebot3/meshes/burger"/>
+  <xacro:property name="tb3_meshes" value="file://$(find custom_robots)/models/turtlebot3/meshes"/>
   <!-- Geometry and inertia from ROBOTIS turtlebot3_description -->
   <xacro:macro name="turtlebot3_burger" params="namespace">
-    <material name="dark">
+    <!-- Greys used by the ROBOTIS Gazebo models -->
+    <material name="body_grey">
       <color rgba="0.3 0.3 0.3 1.0"/>
     </material>
-    <material name="light_black">
-      <color rgba="0.4 0.4 0.4 1.0"/>
+    <material name="parts_grey">
+      <color rgba="0.2 0.2 0.2 1.0"/>
     </material>
     <link name="base_footprint"/>
@@ -21,7 +22,7 @@
         <origin xyz="-0.032 0 0" rpy="0 0 0"/>
         <geometry>
-          <mesh filename="${burger_meshes}/burger_base.stl" scale="0.001 0.001 0.001"/>
+          <mesh filename="${tb3_meshes}/bases/burger_base.stl" scale="0.001 0.001 0.001"/>
         </geometry>
-        <material name="light_black"/>
+        <material name="body_grey"/>
       </visual>
       <collision>
@@ -68,7 +69,7 @@
       <visual>
         <geometry>
-          <mesh filename="${burger_meshes}/lds.stl" scale="0.001 0.001 0.001"/>
+          <mesh filename="${tb3_meshes}/sensors/lds.stl" scale="0.001 0.001 0.001"/>
         </geometry>
-        <material name="dark"/>
+        <material name="parts_grey"/>
       </visual>
       <collision>
@@ -129,7 +130,7 @@
         <origin xyz="0 0 0" rpy="1.57 0 0"/>
         <geometry>
-          <mesh filename="${burger_meshes}/${side}_tire.stl" scale="0.001 0.001 0.001"/>
+          <mesh filename="${tb3_meshes}/wheels/${side}_tire.stl" scale="0.001 0.001 0.001"/>
         </geometry>
-        <material name="dark"/>
+        <material name="parts_grey"/>
       </visual>
       <collision>

File: CustomRobots/turtlebot3/models/turtlebot3/turtlebot3_common.urdf.xacro (robot description, xacro)
@@ -7,9 +7,10 @@
       <color rgba="0.0 0.0 0.0 1.0"/>
     </material>
-    <material name="dark">
+    <!-- Greys used by the ROBOTIS Gazebo models -->
+    <material name="body_grey">
       <color rgba="0.3 0.3 0.3 1.0"/>
     </material>
-    <material name="light_black">
-      <color rgba="0.4 0.4 0.4 1.0"/>
+    <material name="parts_grey">
+      <color rgba="0.2 0.2 0.2 1.0"/>
     </material>
     <material name="white">
@@ -31,7 +32,7 @@
         <origin rpy="0 0 0" xyz="-0.064  0 0"/>
         <geometry>
-          <mesh filename="file://$(find custom_robots)/models/turtlebot3/meshes/waffle_base.dae" scale="0.001 0.001 0.001"/>
+          <mesh filename="file://$(find custom_robots)/models/turtlebot3/meshes/bases/waffle_base.stl" scale="0.001 0.001 0.001"/>
         </geometry>
-        <material name="light_black"/>
+        <material name="body_grey"/>
       </visual>
     </link>
@@ -46,9 +47,10 @@
         </geometry>
       </collision>
-      <visual >
+      <visual>
+        <origin xyz="0 0 0" rpy="1.57 0 0"/>
         <geometry>
-          <cylinder radius="0.033" length="0.018"/>
+          <mesh filename="file://$(find custom_robots)/models/turtlebot3/meshes/wheels/left_tire.stl" scale="0.001 0.001 0.001"/>
         </geometry>
-        <material name="black"/>
+        <material name="parts_grey"/>
       </visual>
     </link>
@@ -63,12 +65,20 @@
         </geometry>
       </collision>
-      <visual >
+      <visual>
+        <origin xyz="0 0 0" rpy="1.57 0 0"/>
         <geometry>
-          <cylinder radius="0.033" length="0.018"/>
+          <mesh filename="file://$(find custom_robots)/models/turtlebot3/meshes/wheels/right_tire.stl" scale="0.001 0.001 0.001"/>
         </geometry>
-        <material name="black"/>
+        <material name="parts_grey"/>
       </visual>
     </link>
-    <link name="camera_base_link"/>
+    <link name="camera_base_link">
+      <visual>
+        <origin xyz="0 0 0" rpy="1.57 0 1.57"/>
+        <geometry>
+          <mesh filename="file://$(find custom_robots)/models/turtlebot3/meshes/sensors/r200.dae"/>
+        </geometry>
+      </visual>
+    </link>
     <joint name="base_to_base_link" type="fixed">
       <parent link="base_footprint"/>

File: CustomRobots/turtlebot3/models/turtlebot3/turtlebot3_gz.urdf.xacro (robot description, xacro)
@@ -56,7 +56,7 @@
       <visual>
         <geometry>
-          <mesh filename="file://$(find custom_robots)/models/turtlebot3/meshes/lds.dae" scale="0.001 0.001 0.001"/>
+          <mesh filename="file://$(find custom_robots)/models/turtlebot3/meshes/sensors/lds.stl" scale="0.001 0.001 0.001"/>
         </geometry>
-        <material name="dark"/>
+        <material name="parts_grey"/>
       </visual>
     </link>
