Commit message: turtlebot burger colors + reset turtlebot waffle

File: CustomRobots/turtlebot3/models/turtlebot3/turtlebot3.urdf.xacro (robot description, xacro)
@@ -31,5 +31,5 @@
   <xacro:turtlebot3 namespace="${namespace}"/>
   <xacro:if value="$(arg camera)">
-    <xacro:camera xyz="0.005 0.018 0.013" rpy="0 0 0" name="camera" parent="camera_base_link" namespace="${namespace}"/>
+    <xacro:camera xyz="0.069 -0.047 0.107" rpy="0 0 0" name="camera" parent="camera_base_link" namespace="${namespace}"/>
   </xacro:if>
   <!-- Beacon on top so a drone above can pick it out by color, only for follow_turtlebot -->

File: CustomRobots/turtlebot3/models/turtlebot3/turtlebot3_burger.urdf.xacro (robot description, xacro)
@@ -7,23 +7,18 @@
   <xacro:property name="noise_level" value="$(arg noise_level)"/>
   <xacro:property name="namespace" value="$(arg namespace)"/>
+  <xacro:include filename="$(find custom_robots)/models/turtlebot3/turtlebot3_burger_common.urdf.xacro"/>
+  <xacro:turtlebot3_burger namespace="${namespace}"/>
+  <xacro:if value="$(arg camera)">
+    <xacro:burger_camera namespace="${namespace}"/>
+  </xacro:if>
   <!-- Odometry noise per difficulty (drift std ~ alpha*sqrt(distance)). -->
   <xacro:if value="${noise_level == 'low'}">
-    <xacro:property name="alpha" value="0.01"/>
+    <xacro:burger_noise_odom namespace="${namespace}" alpha="0.01"/>
   </xacro:if>
   <xacro:if value="${noise_level == 'med'}">
-    <xacro:property name="alpha" value="0.05"/>
+    <xacro:burger_noise_odom namespace="${namespace}" alpha="0.05"/>
   </xacro:if>
   <xacro:if value="${noise_level == 'high'}">
-    <xacro:property name="alpha" value="0.25"/>
+    <xacro:burger_noise_odom namespace="${namespace}" alpha="0.25"/>
   </xacro:if>
-  <xacro:include filename="$(find custom_robots)/models/turtlebot3/turtlebot3_gz.urdf.xacro"/>
-  <xacro:include filename="$(find custom_robots)/models/turtlebot3/turtlebot3_burger_common.urdf.xacro"/>
-  <xacro:turtlebot3_burger namespace="${namespace}"/>
-  <!-- Raspberry Pi camera at the turtlebot3_burger_cam mount -->
-  <xacro:if value="$(arg camera)">
-    <xacro:camera xyz="0.043 0 0.119" rpy="0 0 0" name="camera" parent="base_link" namespace="${namespace}"/>
-  </xacro:if>
-  <xacro:unless value="${noise_level == 'none'}">
-    <xacro:noise_odom a1="${alpha}" a2="${alpha}" a3="${alpha}" a4="${alpha}" namespace="${namespace}" wheel_separation="0.160"/>
-  </xacro:unless>
 </robot>

File: CustomRobots/turtlebot3/models/turtlebot3/turtlebot3_burger_common.urdf.xacro (robot description, xacro)
@@ -1,14 +1,41 @@
 <?xml version="1.0" ?>
 <robot xmlns:xacro="http://ros.org/wiki/xacro">
-  <xacro:include filename="$(find custom_robots)/models/turtlebot3/turtlebot3_gz.urdf.xacro"/>
-  <xacro:property name="tb3_meshes" value="file://$(find custom_robots)/models/turtlebot3/meshes"/>
+  <xacro:include filename="$(find custom_robots)/models/turtlebot3/turtlebot3_burger_gz.urdf.xacro"/>
+  <xacro:property name="burger_meshes" value="file://$(find custom_robots)/models/turtlebot3/meshes/burger"/>
+  <!-- The ROBOTIS meshes are split by material so each part gets the color of the real robot -->
+  <xacro:macro name="burger_part" params="mesh material xyz:='0 0 0' rpy:='0 0 0'">
+    <visual>
+      <origin xyz="${xyz}" rpy="${rpy}"/>
+      <geometry>
+        <mesh filename="${burger_meshes}/${mesh}.stl" scale="0.001 0.001 0.001"/>
+      </geometry>
+      <material name="${material}"/>
+    </visual>
+  </xacro:macro>
   <!-- Geometry and inertia from ROBOTIS turtlebot3_description -->
   <xacro:macro name="turtlebot3_burger" params="namespace">
-    <!-- Greys used by the ROBOTIS Gazebo models -->
-    <material name="body_grey">
-      <color rgba="0.3 0.3 0.3 1.0"/>
+    <material name="burger_plate">
+      <color rgba="0.05 0.05 0.05 1.0"/>
     </material>
-    <material name="parts_grey">
-      <color rgba="0.2 0.2 0.2 1.0"/>
+    <material name="burger_plastic">
+      <color rgba="0.12 0.12 0.12 1.0"/>
+    </material>
+    <material name="burger_dynamixel">
+      <color rgba="0.02 0.02 0.02 1.0"/>
+    </material>
+    <material name="burger_metal">
+      <color rgba="0.62 0.62 0.65 1.0"/>
+    </material>
+    <material name="burger_rpi">
+      <color rgba="0.05 0.40 0.15 1.0"/>
+    </material>
+    <material name="burger_opencr">
+      <color rgba="0.08 0.08 0.10 1.0"/>
+    </material>
+    <material name="burger_rubber">
+      <color rgba="0.03 0.03 0.03 1.0"/>
+    </material>
+    <material name="burger_rim">
+      <color rgba="0.20 0.20 0.20 1.0"/>
     </material>
     <link name="base_footprint"/>
@@ -19,11 +46,10 @@
     </joint>
     <link name="base_link">
-      <visual>
-        <origin xyz="-0.032 0 0" rpy="0 0 0"/>
-        <geometry>
-          <mesh filename="${tb3_meshes}/bases/burger_base.stl" scale="0.001 0.001 0.001"/>
-        </geometry>
-        <material name="body_grey"/>
-      </visual>
+      <xacro:burger_part mesh="burger_base_plates" material="burger_plate" xyz="-0.032 0 0"/>
+      <xacro:burger_part mesh="burger_base_plastic" material="burger_plastic" xyz="-0.032 0 0"/>
+      <xacro:burger_part mesh="burger_base_motors" material="burger_dynamixel" xyz="-0.032 0 0"/>
+      <xacro:burger_part mesh="burger_base_metal" material="burger_metal" xyz="-0.032 0 0"/>
+      <xacro:burger_part mesh="burger_base_rpi" material="burger_rpi" xyz="-0.032 0 0"/>
+      <xacro:burger_part mesh="burger_base_opencr" material="burger_opencr" xyz="-0.032 0 0"/>
       <collision>
         <origin xyz="-0.032 0 0.070" rpy="0 0 0"/>
@@ -61,4 +87,10 @@
       <mu2>0.0</mu2>
     </gazebo>
+    <joint name="imu_joint" type="fixed">
+      <parent link="base_link"/>
+      <child link="imu_link"/>
+      <origin xyz="-0.032 0 0.068" rpy="0 0 0"/>
+    </joint>
+    <link name="imu_link"/>
     <joint name="scan_joint" type="fixed">
       <parent link="base_link"/>
@@ -67,10 +99,6 @@
     </joint>
     <link name="base_scan">
-      <visual>
-        <geometry>
-          <mesh filename="${tb3_meshes}/sensors/lds.stl" scale="0.001 0.001 0.001"/>
-        </geometry>
-        <material name="parts_grey"/>
-      </visual>
+      <xacro:burger_part mesh="lds_body" material="burger_plastic"/>
+      <xacro:burger_part mesh="lds_metal" material="burger_metal"/>
       <collision>
         <origin xyz="0.015 0 -0.0065" rpy="0 0 0"/>
@@ -84,37 +112,7 @@
       </inertial>
     </link>
-    <!-- LDS-01 as simulated by ROBOTIS -->
-    <gazebo reference="base_scan">
-      <sensor name="laser" type="gpu_lidar">
-        <always_on>1</always_on>
-        <visualize>1</visualize>
-        <update_rate>5</update_rate>
-        <topic>/${namespace}/laser/scan</topic>
-        <gz_frame_id>base_scan</gz_frame_id>
-        <lidar>
-          <scan>
-            <horizontal>
-              <samples>360</samples>
-              <resolution>1</resolution>
-              <min_angle>0</min_angle>
-              <max_angle>6.28</max_angle>
-            </horizontal>
-          </scan>
-          <range>
-            <min>0.12</min>
-            <max>3.5</max>
-            <resolution>0.015</resolution>
-          </range>
-          <noise>
-            <type>gaussian</type>
-            <mean>0.0</mean>
-            <stddev>0.01</stddev>
-          </noise>
-        </lidar>
-      </sensor>
-    </gazebo>
-    <xacro:imu parent="base_link" xyz="-0.032 0 0.068" rpy="0 0 0" namespace="${namespace}"/>
-    <xacro:velocity namespace="${namespace}" wheel_separation="0.160"/>
-    <xacro:odom namespace="${namespace}" freq="50"/>
+    <xacro:burger_lds namespace="${namespace}"/>
+    <xacro:burger_imu namespace="${namespace}"/>
+    <xacro:burger_drive namespace="${namespace}"/>
   </xacro:macro>
   <xacro:macro name="burger_wheel" params="side y">
@@ -127,11 +125,6 @@
     </joint>
     <link name="wheel_${side}_link">
-      <visual>
-        <origin xyz="0 0 0" rpy="1.57 0 0"/>
-        <geometry>
-          <mesh filename="${tb3_meshes}/wheels/${side}_tire.stl" scale="0.001 0.001 0.001"/>
-        </geometry>
-        <material name="parts_grey"/>
-      </visual>
+      <xacro:burger_part mesh="${side}_tire_rubber" material="burger_rubber" rpy="1.57 0 0"/>
+      <xacro:burger_part mesh="${side}_tire_rim" material="burger_rim" rpy="1.57 0 0"/>
       <collision>
         <geometry>

File: CustomRobots/turtlebot3/models/turtlebot3/turtlebot3_common.urdf.xacro (robot description, xacro)
@@ -7,10 +7,9 @@
       <color rgba="0.0 0.0 0.0 1.0"/>
     </material>
-    <!-- Greys used by the ROBOTIS Gazebo models -->
-    <material name="body_grey">
+    <material name="dark">
       <color rgba="0.3 0.3 0.3 1.0"/>
     </material>
-    <material name="parts_grey">
-      <color rgba="0.2 0.2 0.2 1.0"/>
+    <material name="light_black">
+      <color rgba="0.4 0.4 0.4 1.0"/>
     </material>
     <material name="white">
@@ -32,7 +31,7 @@
         <origin rpy="0 0 0" xyz="-0.064  0 0"/>
         <geometry>
-          <mesh filename="file://$(find custom_robots)/models/turtlebot3/meshes/bases/waffle_base.stl" scale="0.001 0.001 0.001"/>
+          <mesh filename="file://$(find custom_robots)/models/turtlebot3/meshes/waffle_base.dae" scale="0.001 0.001 0.001"/>
         </geometry>
-        <material name="body_grey"/>
+        <material name="light_black"/>
       </visual>
     </link>
@@ -47,10 +46,9 @@
         </geometry>
       </collision>
-      <visual>
-        <origin xyz="0 0 0" rpy="1.57 0 0"/>
+      <visual >
         <geometry>
-          <mesh filename="file://$(find custom_robots)/models/turtlebot3/meshes/wheels/left_tire.stl" scale="0.001 0.001 0.001"/>
+          <cylinder radius="0.033" length="0.018"/>
         </geometry>
-        <material name="parts_grey"/>
+        <material name="black"/>
       </visual>
     </link>
@@ -65,20 +63,12 @@
         </geometry>
       </collision>
-      <visual>
-        <origin xyz="0 0 0" rpy="1.57 0 0"/>
+      <visual >
         <geometry>
-          <mesh filename="file://$(find custom_robots)/models/turtlebot3/meshes/wheels/right_tire.stl" scale="0.001 0.001 0.001"/>
+          <cylinder radius="0.033" length="0.018"/>
         </geometry>
-        <material name="parts_grey"/>
+        <material name="black"/>
       </visual>
     </link>
-    <link name="camera_base_link">
-      <visual>
-        <origin xyz="0 0 0" rpy="1.57 0 1.57"/>
-        <geometry>
-          <mesh filename="file://$(find custom_robots)/models/turtlebot3/meshes/sensors/r200.dae"/>
-        </geometry>
-      </visual>
-    </link>
+    <link name="camera_base_link"/>
     <joint name="base_to_base_link" type="fixed">
       <parent link="base_footprint"/>

File: CustomRobots/turtlebot3/models/turtlebot3/turtlebot3_gz.urdf.xacro (robot description, xacro)
@@ -56,7 +56,7 @@
       <visual>
         <geometry>
-          <mesh filename="file://$(find custom_robots)/models/turtlebot3/meshes/sensors/lds.stl" scale="0.001 0.001 0.001"/>
+          <mesh filename="file://$(find custom_robots)/models/turtlebot3/meshes/lds.dae" scale="0.001 0.001 0.001"/>
         </geometry>
-        <material name="parts_grey"/>
+        <material name="dark"/>
       </visual>
     </link>
@@ -153,5 +153,5 @@
     </gazebo>
   </xacro:macro>
-  <xacro:macro name="velocity" params="namespace wheel_separation:=0.287">
+  <xacro:macro name="velocity" params="namespace">
     <gazebo>
       <plugin filename="gz-sim-diff-drive-system" name="gz::sim::systems::DiffDrive">
@@ -160,5 +160,5 @@
         <right_joint>wheel_right_joint</right_joint>
         <!-- kinematics -->
-        <wheel_separation>${wheel_separation}</wheel_separation>
+        <wheel_separation>0.287</wheel_separation>
         <wheel_radius>0.033</wheel_radius>
         <!-- limits -->
@@ -183,5 +183,5 @@
     </gazebo>
   </xacro:macro>
-  <xacro:macro name="noise_odom" params="namespace a1 a2 a3 a4 wheel_separation:=0.287">
+  <xacro:macro name="noise_odom" params="namespace a1 a2 a3 a4">
     <gazebo>
       <plugin filename="libNoisyOdometryPlugin.so" name="custom_plugins::NoisyOdometryPlugin">
@@ -193,5 +193,5 @@
         <right_joint>wheel_right_joint</right_joint>
         <wheel_radius>0.033</wheel_radius>
-        <wheel_separation>${wheel_separation}</wheel_separation>
+        <wheel_separation>0.287</wheel_separation>
         <alpha1>${a1}</alpha1>
         <alpha2>${a2}</alpha2>
