Commit message: Add final ackermann robot

File: CustomRobots/logistic_ackermann_robot/models/logistic_ackermann_robot/logistic_ackermann_robot.urdf.xacro (robot description, xacro)
@@ -1,7 +1,7 @@
 <?xml version="1.0" ?>
-<robot name="logistic_holonomic_robot"
+<robot name="logistic ackermann robot"
   xmlns:xacro="http://ros.org/wiki/xacro">
-  <xacro:include filename="$(find custom_robots)/models/logistic_holonomic_robot/logistic_holonomic_robot_gz.urdf.xacro"/>
-  <xacro:include filename="$(find custom_robots)/models/logistic_holonomic_robot/logistic_holonomic_robot_common.urdf.xacro"/>
-  <xacro:logistic_holonomic_robot/>
+  <xacro:include filename="$(find custom_robots)/models/logistic_ackermann_robot/logistic_ackermann_robot_gz.urdf.xacro"/>
+  <xacro:include filename="$(find custom_robots)/models/logistic_ackermann_robot/logistic_ackermann_robot_common.urdf.xacro"/>
+  <xacro:logistic_ackermann_robot/>
 </robot>

File: CustomRobots/logistic_ackermann_robot/models/logistic_ackermann_robot/logistic_ackermann_robot_common.urdf.xacro (robot description, xacro)
@@ -1,272 +1,225 @@
 <?xml version="1.0" ?>
 <robot xmlns:xacro="http://ros.org/wiki/xacro">
-  <xacro:include filename="$(find custom_robots)/models/logistic_holonomic_robot/logistic_holonomic_robot_gz.urdf.xacro"/>
-  <xacro:macro name="logistic_holonomic_robot">
-    <link name="base_footprint" />
-    <link name="base">
-      <inertial>
-        <mass value="1.5"/>
-        <inertia ixx="0.001" ixy="0" ixz="0" iyy="0.001" iyz="0" izz="0.001"/>
-      </inertial>
-      <collision>
-        <origin rpy="0 0 0" xyz="0 0 0.07"/>
-        <geometry>
-          <box size="0.532 0.532 0.188"/>
-        </geometry>
-      </collision>
-      <visual>
-        <geometry>
-          <mesh filename="$(find custom_robots)/models/logistic_holonomic_robot/meshes/waffle_pi_base.dae" scale="0.002 0.002 0.002"/>
-        </geometry>
-      </visual>
-    </link>
-    <joint name="base_to_base_footprint" type="fixed">
-      <origin rpy="0 0 0" xyz="0 0 0.048"/>
-      <parent link="base_footprint"/>
-      <child link="base"/>
-    </joint>
-    <joint name="left_wheel_joint" type="continuous">
-      <origin rpy="-1.57 0 0" xyz="0.05 0.288 0.046"/>
-      <parent link="base"/>
-      <child link="left_wheel_link"/>
+  <xacro:include filename="$(find custom_robots)/models/logistic_ackermann_robot/logistic_ackermann_robot_gz.urdf.xacro"/>
+  <xacro:macro name="logistic_ackermann_robot">
+    <link name="base_link" />
+    <link name="chassis_link">
+      <inertial>
+        <origin rpy="0 0 0" xyz="0.07307 -1e-06 0.65096"/>
+        <mass value="1580"/>
+        <inertia ixx="442.769" ixy="0" ixz="62.5206" iyy="1997.86" iyz="0" izz="2238.05"/>
+      </inertial>
+      <collision>
+        <origin rpy="0 0 -1.5707963" xyz="0 0 0"/>
+        <geometry>
+          <mesh filename="$(find custom_robots)/models/logistic_ackermann_robot/meshes/chassis.dae" scale="0.5 0.5 0.5"/>
+        </geometry>
+        <gz>
+          <surface>
+            <friction>
+              <ode>
+                <mu>0.2</mu>
+                <mu2>0.2</mu2>
+              </ode>
+            </friction>
+          </surface>
+        </gz>
+      </collision>
+      <visual>
+        <origin rpy="0 0 -1.5707963" xyz="0 0 0"/>
+        <geometry>
+          <mesh filename="$(find custom_robots)/models/logistic_ackermann_robot/meshes/chassis.dae" scale="0.5 0.5 0.5"/>
+        </geometry>
+      </visual>
+    </link>
+    <joint name="chassis_link_joint" type="fixed">
+      <parent link="base_link"/>
+      <child link="chassis_link"/>
+    </joint>
+    <joint name="bl_axle" type="continuous">
+      <origin rpy="0 0 0" xyz="-0.244 0.18 0"/>
+      <parent link="chassis_link"/>
+      <child link="back_left_wheel_link"/>
+      <axis xyz="0 1 0"/>
+      <limit effort="1000" velocity="100"/>
+      <dynamics friction="12.0316061502"/>
+    </joint>
+    <link name="back_left_wheel_link">
+      <inertial>
+        <origin rpy="0 0 0" xyz="0 0.0377  0"/>
+        <mass value="24.5"/>
+        <inertia ixx="1.04961" ixy="0" ixz="0" iyy="1.84514" iyz="0" izz="1.04961"/>
+      </inertial>
+      <collision>
+        <origin rpy="1.57 0 0" xyz="0 0 0"/>
+        <geometry>
+          <cylinder radius="0.072" length="0.06"/>
+        </geometry>
+        <gz>
+          <surface>
+            <friction>
+              <ode>
+                <mu>1e+6</mu>
+                <mu2>1e+6</mu2>
+              </ode>
+            </friction>
+          </surface>
+        </gz>
+      </collision>
+      <visual>
+        <origin rpy="0 0 -1.57" xyz="0 0 0"/>
+        <geometry>
+          <mesh filename="$(find custom_robots)/models/logistic_ackermann_robot/meshes/wheel.dae" scale="0.5 0.5 0.5"/>
+        </geometry>
+      </visual>
+    </link>
+    <joint name="br_axle" type="continuous">
+      <origin rpy="0 0 0" xyz="-0.244 -0.18 0"/>
+      <parent link="chassis_link"/>
+      <child link="back_right_wheel_link"/>
+      <axis xyz="0 1 0"/>
+      <limit effort="1000" velocity="100"/>
+      <dynamics friction="12.0316061502"/>
+    </joint>
+    <link name="back_right_wheel_link">
+      <inertial>
+        <origin rpy="0 0 0" xyz="0 0.0377  0"/>
+        <mass value="24.5"/>
+        <inertia ixx="1.04961" ixy="0" ixz="0" iyy="1.84514" iyz="0" izz="1.04961"/>
+      </inertial>
+      <collision>
+        <origin rpy="1.57 0 0" xyz="0 0 0"/>
+        <geometry>
+          <cylinder radius="0.072" length="0.06"/>
+        </geometry>
+        <gz>
+          <surface>
+            <friction>
+              <ode>
+                <mu>1e+6</mu>
+                <mu2>1e+6</mu2>
+              </ode>
+            </friction>
+          </surface>
+        </gz>
+      </collision>
+      <visual>
+        <origin rpy="0 0 -1.57" xyz="0 0 0"/>
+        <geometry>
+          <mesh filename="$(find custom_robots)/models/logistic_ackermann_robot/meshes/wheel.dae" scale="0.5 0.5 0.5"/>
+        </geometry>
+      </visual>
+    </link>
+    <joint name="l_steer" type="revolute">
+      <origin rpy="0 0 0" xyz="0.244 0.236 0"/>
+      <parent link="chassis_link"/>
+      <child link="l_steer_1"/>
       <axis xyz="0 0 1"/>
-      <limit effort="1000" velocity="100"/>
-    </joint>
-    <link name="left_wheel_link">
-      <inertial>
-        <mass value="0.1"/>
-        <inertia ixx="0.001" ixy="0" ixz="0" iyy="0.001" iyz="0" izz="0.001"/>
-      </inertial>
-      <collision>
-        <geometry>
-          <cylinder radius="0.1" length="0.02"/>
-        </geometry>
-        <gz>
-          <surface>
-            <friction>
-              <ode>
-                <mu>10.0</mu>
-                <mu2>10.0</mu2>
-                <fdir1>0 0 0</fdir1>
-                <slip1>0.0</slip1>
-                <slip2>0.0</slip2>
-              </ode>
-            </friction>
-            <contact>
-              <ode>
-                <soft_cfm>0.001</soft_cfm>
-                <soft_erp>0.5</soft_erp>
-                <kp>1e+5</kp>
-                <kd>1</kd>
-                <max_vel>0.01</max_vel>
-                <min_depth>0.001</min_depth>
-              </ode>
-            </contact>
-          </surface>
-        </gz>
-      </collision>
-      <visual>
-        <origin rpy="1.57 0 0" xyz="0 0 0"/>
-        <geometry>
-          <mesh filename="$(find custom_robots)/models/logistic_holonomic_robot/meshes/left_tire.dae" scale="0.003 0.003 0.003"/>
-        </geometry>
-      </visual>
-    </link>
-    <joint name="right_wheel_joint" type="continuous">
-      <origin rpy="-1.57 0 0" xyz="0.05 -0.288 0.046"/>
-      <parent link="base"/>
-      <child link="right_wheel_link"/>
+      <limit lower="-0.95" upper="0.95" effort="1e6" velocity="10"/>
+      <dynamics friction="18.0474092253" damping="0.01"/>
+    </joint>
+    <link name="l_steer_1">
+      <origin rpy="0 -0 0" xyz="0 0 0"/>
+      <inertial>
+        <origin rpy="0 0 0" xyz="0 -0.003381 0.02162"/>
+        <mass value="1"/>
+        <inertia ixx="1" ixy="0" ixz="0" iyy="1" iyz="0" izz="1"/>
+      </inertial>
+    </link>
+    <joint name="front_left_wheel_joint" type="continuous">
+      <parent link="l_steer_1"/>
+      <child link="front_left_wheel_link"/>
+      <axis xyz="0 1 0"/>
+      <limit effort="1000" velocity="100"/>
+      <dynamics friction="12.0316061502"/>
+    </joint>
+    <link name="front_left_wheel_link">
+      <inertial>
+        <origin rpy="0 0 0" xyz="0 0.0377  0"/>
+        <mass value="24.5"/>
+        <inertia ixx="1.04961" ixy="0" ixz="0" iyy="1.84514" iyz="0" izz="1.04961"/>
+      </inertial>
+      <collision>
+        <origin rpy="1.57 0 0" xyz="0 0 0"/>
+        <geometry>
+          <cylinder radius="0.072" length="0.06"/>
+        </geometry>
+        <gz>
+          <surface>
+            <friction>
+              <ode>
+                <mu>1e+6</mu>
+                <mu2>1e+6</mu2>
+              </ode>
+            </friction>
+          </surface>
+        </gz>
+      </collision>
+      <visual>
+        <origin rpy="0 0 -1.57" xyz="0 0 0"/>
+        <geometry>
+          <mesh filename="$(find custom_robots)/models/logistic_ackermann_robot/meshes/wheel.dae" scale="0.5 0.5 0.5"/>
+        </geometry>
+      </visual>
+    </link>
+    <joint name="r_steer" type="revolute">
+      <origin rpy="0 0 0" xyz="0.244 -0.236 0"/>
+      <parent link="chassis_link"/>
+      <child link="r_steer_1"/>
       <axis xyz="0 0 1"/>
-      <limit effort="1000" velocity="100"/>
-    </joint>
-    <link name="right_wheel_link">
-      <inertial>
-        <mass value="0.1"/>
-        <inertia ixx="0.001" ixy="0" ixz="0" iyy="0.001" iyz="0" izz="0.001"/>
-      </inertial>
-      <collision>
-        <geometry>
-          <cylinder radius="0.1" length="0.02"/>
-        </geometry>
-        <gz>
-          <surface>
-            <friction>
-              <ode>
-                <mu>10.0</mu>
-                <mu2>10.0</mu2>
-                <fdir1>0 0 0</fdir1>
-                <slip1>0.0</slip1>
-                <slip2>0.0</slip2>
-              </ode>
-            </friction>
-            <contact>
-              <ode>
-                <soft_cfm>0.001</soft_cfm>
-                <soft_erp>0.5</soft_erp>
-                <kp>1e+5</kp>
-                <kd>1</kd>
-                <max_vel>0.01</max_vel>
-                <min_depth>0.001</min_depth>
-              </ode>
-            </contact>
-          </surface>
-        </gz>
-      </collision>
-      <visual>
-        <origin rpy="1.57 0 0" xyz="0 0 0"/>
-        <geometry>
-          <mesh filename="$(find custom_robots)/models/logistic_holonomic_robot/meshes/right_tire.dae" scale="0.003 0.003 0.003"/>
-        </geometry>
-      </visual>
-    </link>
-    <link name="back_right_caster_roll_link">
-      <inertial>
-        <mass value="0.0001"/>
+      <limit lower="-0.95" upper="0.95" effort="1e6" velocity="10"/>
+      <dynamics friction="18.0474092253" damping="0.01"/>
+    </joint>
+    <link name="r_steer_1">
+      <origin rpy="0 -0 0" xyz="0 0 0"/>
+      <inertial>
+        <origin rpy="0 0 0" xyz="0 -0.003381 0.02162"/>
+        <mass value="1"/>
         <inertia ixx="1" ixy="0" ixz="0" iyy="1" iyz="0" izz="1"/>
       </inertial>
     </link>
-    <link name="back_right_caster_pitch_link">
-      <inertial>
-        <mass value="0.0001"/>
-        <inertia ixx="1" ixy="0" ixz="0" iyy="1" iyz="0" izz="1"/>
-      </inertial>
-    </link>
-    <joint name="back_right_caster_joint_roll" type="continuous">
-      <origin rpy="0 0 0" xyz="-0.23 -0.13 -0.0175"/>
-      <parent link="base"/>
-      <child link="back_right_caster_roll_link"/>
-      <axis xyz="1 0 0"/>
-      <limit effort="1000" velocity="100"/>
-    </joint>
-    <joint name="back_right_caster_joint_pitch" type="continuous">
-      <origin rpy="0 0 0" xyz="0 0 0"/>
-      <parent link="back_right_caster_roll_link"/>
-      <child link="back_right_caster_pitch_link"/>
-      <axis xyz="0 1 0"/>
-      <limit effort="1000" velocity="100"/>
-    </joint>
-    <joint name="back_right_caster_joint_yaw" type="continuous">
-      <origin rpy="0 0 0" xyz="0 0 0"/>
-      <parent link="back_right_caster_pitch_link"/>
-      <child link="back_right_caster_link"/>
+    <joint name="front_right_wheel_joint" type="continuous">
+      <parent link="r_steer_1"/>
+      <child link="front_right_wheel_link"/>
+      <axis xyz="0 1 0"/>
+      <limit effort="1000" velocity="100"/>
+      <dynamics friction="12.0316061502"/>
+    </joint>
+    <link name="front_right_wheel_link">
+      <inertial>
+        <origin rpy="0 0 0" xyz="0 0.0377  0"/>
+        <mass value="24.5"/>
+        <inertia ixx="1.04961" ixy="0" ixz="0" iyy="1.84514" iyz="0" izz="1.04961"/>
+      </inertial>
+      <collision>
+        <origin rpy="1.57 0 0" xyz="0 0 0"/>
+        <geometry>
+          <cylinder radius="0.072" length="0.06"/>
+        </geometry>
+        <gz>
+          <surface>
+            <friction>
+              <ode>
+                <mu>1e+6</mu>
+                <mu2>1e+6</mu2>
+              </ode>
+            </friction>
+          </surface>
+        </gz>
+      </collision>
+      <visual>
+        <origin rpy="0 0 -1.57" xyz="0 0 0"/>
+        <geometry>
+          <mesh filename="$(find custom_robots)/models/logistic_ackermann_robot/meshes/wheel.dae" scale="0.5 0.5 0.5"/>
+        </geometry>
+      </visual>
+    </link>
+    <joint name="lift_joint" type="prismatic">
+      <origin rpy="0 0 0" xyz="0 0.0 0.165"/>
+      <parent link="base_link"/>
+      <child link="lift_link"/>
       <axis xyz="0 0 1"/>
-      <limit effort="1000" velocity="100"/>
-    </joint>
-    <link name="back_right_caster_link">
-      <inertial>
-        <mass value="0.8"/>
-        <inertia ixx="0.00001" ixy="0" ixz="0" iyy="0.00001" iyz="0" izz="0.00001"/>
-      </inertial>
-      <collision>
-        <geometry>
-          <sphere radius="0.025"/>
-        </geometry>
-        <gz>
-          <surface>
-            <contact>
-              <ode>
-                <soft_cfm>0</soft_cfm>
-                <soft_erp>0.2</soft_erp>
-                <kp>1e+5</kp>
-                <kd>1</kd>
-                <max_vel>0.01</max_vel>
-                <min_depth>0.001</min_depth>
-              </ode>
-            </contact>
-          </surface>
-        </gz>
-      </collision>
-      <visual>
-        <geometry>
-          <sphere radius="0.025"/>
-        </geometry>
-      </visual>
-    </link>
-    <link name="back_left_caster_roll_link">
-      <inertial>
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
File: CustomRobots/logistic_ackermann_robot/models/logistic_ackermann_robot/logistic_ackermann_robot_gz.urdf.xacro (robot description, xacro)
@@ -3,10 +3,18 @@
   <xacro:macro name="velocity" params="topic">
     <gazebo>
-      <plugin filename="gz-sim-diff-drive-system" name="gz::sim::systems::DiffDrive">
-        <left_joint>left_wheel_joint</left_joint>
-        <right_joint>right_wheel_joint</right_joint>
-        <wheel_separation>0.576</wheel_separation>
-        <wheel_radius>0.1</wheel_radius>
+      <plugin filename="gz-sim-ackermann-steering-system" name="gz::sim::systems::AckermannSteering">
+        <left_joint>bl_axle</left_joint>
+        <right_joint>br_axle</right_joint>
+        <left_steering_joint>l_steer</left_steering_joint>
+        <right_steering_joint>r_steer</right_steering_joint>
+        <kingpin_width>0.472</kingpin_width>
+        <steering_limit>0.64</steering_limit>
+        <wheel_base>0.488</wheel_base>
+        <wheel_separation>0.36</wheel_separation>
+        <wheel_radius>0.072</wheel_radius>
         <topic>${topic}</topic>
+        <!-- <odom_topic>/model/amazon_robot/odometry_noisy</odom_topic>
+        <tf_topic>/model/amazon_robot/tf_noisy</tf_topic> -->
+        <odom_publish_frequency>50</odom_publish_frequency>
       </plugin>
     </gazebo>
@@ -16,5 +24,5 @@
       <plugin filename="gz-sim-odometry-publisher-system" name="gz::sim::systems::OdometryPublisher">
         <odom_frame>odom</odom_frame>
-        <robot_base_frame>base_footprint</robot_base_frame>
+        <robot_base_frame>base_link</robot_base_frame>
         <odom_publish_frequency>${freq}</odom_publish_frequency>
         <odom_topic>${topic}</odom_topic>
@@ -33,6 +41,7 @@
         <i_gain>0.0</i_gain>
         <d_gain>0.1</d_gain>
-        <cmd_max>20</cmd_max>
-        <cmd_min>-20</cmd_min>
+        <cmd_max>100</cmd_max>
+        <cmd_min>-100</cmd_min>
+        <disable_braking>0</disable_braking>
       </plugin>
       <plugin filename="gz-sim-joint-state-publisher-system" name="gz::sim::systems::JointStatePublisher">
