Commit message: Add logistic ackermann robot

File: CustomRobots/logistic_ackermann_robot/models/logistic_ackermann_robot/logistic_ackermann_robot.urdf.xacro (robot description, xacro)
@@ -2,6 +2,8 @@
 <robot name="logistic ackermann robot"
   xmlns:xacro="http://ros.org/wiki/xacro">
+  <xacro:arg name="namespace" default="f1"/>
+  <xacro:property name="namespace" value="$(arg namespace)"/>
   <xacro:include filename="$(find custom_robots)/models/logistic_ackermann_robot/logistic_ackermann_robot_gz.urdf.xacro"/>
   <xacro:include filename="$(find custom_robots)/models/logistic_ackermann_robot/logistic_ackermann_robot_common.urdf.xacro"/>
-  <xacro:logistic_ackermann_robot/>
+  <xacro:logistic_ackermann_robot namespace="${namespace}"/>
 </robot>

File: CustomRobots/logistic_ackermann_robot/models/logistic_ackermann_robot/logistic_ackermann_robot_common.urdf.xacro (robot description, xacro)
@@ -2,5 +2,5 @@
 <robot xmlns:xacro="http://ros.org/wiki/xacro">
   <xacro:include filename="$(find custom_robots)/models/logistic_ackermann_robot/logistic_ackermann_robot_gz.urdf.xacro"/>
-  <xacro:macro name="logistic_ackermann_robot">
+  <xacro:macro name="logistic_ackermann_robot" params="namespace">
     <link name="base_link" />
     <link name="chassis_link">
@@ -277,7 +277,7 @@
       </visual>
     </link>
-    <xacro:velocity topic="/cmd_vel"/>
-    <xacro:odom topic="/model/amazon_robot/odometry" freq="50"/>
-    <xacro:joints topic="/robot/joint_state" vel_topic="/platform/cmd_vel"/>
+    <xacro:velocity namespace="${namespace}"/>
+    <xacro:odom namespace="${namespace}" freq="50"/>
+    <xacro:joints topic="joint_state" vel_topic="platform/cmd_vel" namespace="${namespace}"/>
   </xacro:macro>
 </robot>

File: CustomRobots/logistic_ackermann_robot/models/logistic_ackermann_robot/logistic_ackermann_robot_gz.urdf.xacro (robot description, xacro)
@@ -1,5 +1,5 @@
 <?xml version="1.0"?>
 <robot xmlns:xacro="http://ros.org/wiki/xacro">
-  <xacro:macro name="velocity" params="topic">
+  <xacro:macro name="velocity" params="namespace">
     <gazebo>
       <plugin filename="gz-sim-ackermann-steering-system" name="gz::sim::systems::AckermannSteering">
@@ -13,5 +13,5 @@
         <wheel_separation>0.36</wheel_separation>
         <wheel_radius>0.072</wheel_radius>
-        <topic>${topic}</topic>
+        <topic>/${namespace}/cmd_vel</topic>
         <!-- <odom_topic>/model/amazon_robot/odometry_noisy</odom_topic>
         <tf_topic>/model/amazon_robot/tf_noisy</tf_topic> -->
@@ -20,5 +20,5 @@
     </gazebo>
   </xacro:macro>
-  <xacro:macro name="odom" params="topic freq">
+  <xacro:macro name="odom" params="namespace freq">
     <gazebo>
       <plugin filename="gz-sim-odometry-publisher-system" name="gz::sim::systems::OdometryPublisher">
@@ -26,14 +26,14 @@
         <robot_base_frame>base_link</robot_base_frame>
         <odom_publish_frequency>${freq}</odom_publish_frequency>
-        <odom_topic>${topic}</odom_topic>
+        <odom_topic>/${namespace}/odom</odom_topic>
         <dimensions>3</dimensions>
       </plugin>
     </gazebo>
   </xacro:macro>
-  <xacro:macro name="joints" params="vel_topic topic">
+  <xacro:macro name="joints" params="vel_topic topic namespace">
     <gazebo>
       <plugin filename="gz-sim-joint-controller-system" name="gz::sim::systems::JointController">
         <joint_name>lift_joint</joint_name>
-        <topic>${vel_topic}</topic>
+        <topic>/${namespace}/${vel_topic}</topic>
         <initial_position>0.0</initial_position>
         <use_force_commands>true</use_force_commands>
@@ -46,5 +46,5 @@
       </plugin>
       <plugin filename="gz-sim-joint-state-publisher-system" name="gz::sim::systems::JointStatePublisher">
-        <topic>${topic}</topic>
+        <topic>/${namespace}/${topic}</topic>
         <joint_name>lift_joint</joint_name>
       </plugin>
