Commit message: Update rover_4wd

File: CustomRobots/rover_4wd/model/rover_4wd.urdf.xacro (robot description, xacro)
@@ -1,2 +1,3 @@
+<?xml version="1.0" ?>
 <robot xmlns:xacro="http://www.ros.org/wiki/xacro" name="rover_4wd">
   <!-- ================== Robot Parameters ================== -->
@@ -8,9 +9,20 @@
   <xacro:property name="wheel_mass" value="1.25" />
   <xacro:property name="chassis_mass" value="4.53592" />
-  <!-- ================== Accessories (Lidar, IMU, Payload) ================== -->
   <xacro:property name="payload_z_offset" value="0.096" />
-  <xacro:include filename="$(find custom_robots)/urdf/accessories/rover_dev_payload.urdf" />
-  <xacro:include filename="$(find custom_robots)/urdf/accessories/rplidar_s2.urdf" />
-  <xacro:include filename="$(find custom_robots)/urdf/accessories/imu.urdf" />
+  <xacro:arg name="noise_level" default="none"/>
+  <xacro:property name="noise_level" value="$(arg noise_level)"/>
+  <xacro:if value="${noise_level == 'low'}">
+    <xacro:property name="a1" value="0.0005" />
+    <xacro:property name="a2" value="0.0005" />
+    <xacro:property name="a3" value="0.0002" />
+    <xacro:property name="a4" value="0.0002" />
+  </xacro:if>
+  <xacro:if value="${noise_level == 'high'}">
+    <xacro:property name="a1" value="0.005" />
+    <xacro:property name="a2" value="0.005" />
+    <xacro:property name="a3" value="0.003" />
+    <xacro:property name="a4" value="0.003" />
+  </xacro:if>
+  <xacro:include filename="$(find custom_robots)/model/rover_4wd/rover_4wd_gz.urdf.xacro"/>
   <!-- ================== Links ================== -->
   <link name="base_link" />
@@ -19,5 +31,5 @@
       <origin xyz="0 0 0" rpy="1.57 -0 1.57" />
       <geometry>
-        <mesh filename="file://$(find custom_robots)/meshes/flipper_chassis.dae"/>
+        <mesh filename="file://$(find custom_robots)/model/rover_4wd/meshes/flipper_chassis.dae"/>
       </geometry>
     </visual>
@@ -25,5 +37,5 @@
       <origin xyz="0 ${track_y_offset} 0" rpy="1.57 3.1415 0" />
       <geometry>
-        <mesh filename="file://$(find custom_robots)/meshes/flipper_track.dae"/>
+        <mesh filename="file://$(find custom_robots)/model/rover_4wd/meshes/flipper_track.dae"/>
       </geometry>
     </visual>
@@ -31,5 +43,5 @@
       <origin xyz="0 ${track_y_offset} 0" rpy="1.57 3.1415 0" />
       <geometry>
-        <mesh filename="file://$(find custom_robots)/meshes/flipper_track.dae"/>
+        <mesh filename="file://$(find custom_robots)/model/rover_4wd/meshes/flipper_track.dae"/>
       </geometry>
     </collision>
@@ -37,5 +49,5 @@
       <origin xyz="0 ${-track_y_offset} 0" rpy="1.57 3.1415 0" />
       <geometry>
-        <mesh filename="file://$(find custom_robots)/meshes/flipper_track.dae"/>
+        <mesh filename="file://$(find custom_robots)/model/rover_4wd/meshes/flipper_track.dae"/>
       </geometry>
     </visual>
@@ -43,5 +55,5 @@
       <origin xyz="0 ${-track_y_offset} 0" rpy="1.57 3.1415 0" />
       <geometry>
-        <mesh filename="file://$(find custom_robots)/meshes/flipper_track.dae"/>
+        <mesh filename="file://$(find custom_robots)/model/rover_4wd/meshes/flipper_track.dae"/>
       </geometry>
     </collision>
@@ -49,5 +61,5 @@
       <origin xyz="0 0 0" rpy="1.57 -0 1.57" />
       <geometry>
-        <mesh filename="file://$(find custom_robots)/meshes/flipper_chassis.dae"/>
+        <mesh filename="file://$(find custom_robots)/model/rover_4wd/meshes/flipper_chassis.dae"/>
       </geometry>
     </collision>
@@ -69,5 +81,5 @@
       <origin xyz="0 0 0" rpy="-1.57 0 0" />
       <geometry>
-        <mesh filename="file://$(find custom_robots)/meshes/pro_tire.dae"/>
+        <mesh filename="file://$(find custom_robots)/model/rover_4wd/meshes/pro_tire.dae"/>
       </geometry>
     </visual>
@@ -75,5 +87,5 @@
       <origin xyz="0 0 0" rpy="-1.57 0 0" />
       <geometry>
-        <mesh filename="file://$(find custom_robots)/meshes/pro_tire.dae"/>
+        <mesh filename="file://$(find custom_robots)/model/rover_4wd/meshes/pro_tire.dae"/>
       </geometry>
     </collision>
@@ -95,5 +107,5 @@
       <origin xyz="0 0 0" rpy="1.57 0 0" />
       <geometry>
-        <mesh filename="file://$(find custom_robots)/meshes/pro_tire.dae"/>
+        <mesh filename="file://$(find custom_robots)/model/rover_4wd/meshes/pro_tire.dae"/>
       </geometry>
     </visual>
@@ -101,5 +113,5 @@
       <origin xyz="0 0 0" rpy="1.57 0 0" />
       <geometry>
-        <mesh filename="file://$(find custom_robots)/meshes/pro_tire.dae"/>
+        <mesh filename="file://$(find custom_robots)/model/rover_4wd/meshes/pro_tire.dae"/>
       </geometry>
     </collision>
@@ -121,5 +133,5 @@
       <origin xyz="0 0 0" rpy="1.57 0 3.1415" />
       <geometry>
-        <mesh filename="file://$(find custom_robots)/meshes/pro_tire.dae"/>
+        <mesh filename="file://$(find custom_robots)/model/rover_4wd/meshes/pro_tire.dae"/>
       </geometry>
     </visual>
@@ -127,5 +139,5 @@
       <origin xyz="0 0 0" rpy="1.57 0 3.1415" />
       <geometry>
-        <mesh filename="file://$(find custom_robots)/meshes/pro_tire.dae"/>
+        <mesh filename="file://$(find custom_robots)/model/rover_4wd/meshes/pro_tire.dae"/>
       </geometry>
     </collision>
@@ -147,5 +159,5 @@
       <origin xyz="0 0 0" rpy="-1.57 0 3.1415" />
       <geometry>
-        <mesh filename="file://$(find custom_robots)/meshes/pro_tire.dae"/>
+        <mesh filename="file://$(find custom_robots)/model/rover_4wd/meshes/pro_tire.dae"/>
       </geometry>
     </visual>
@@ -153,5 +165,5 @@
       <origin xyz="0 0 0" rpy="-1.57 0 3.1415" />
       <geometry>
-        <mesh filename="file://$(find custom_robots)/meshes/pro_tire.dae"/>
+        <mesh filename="file://$(find custom_robots)/model/rover_4wd/meshes/pro_tire.dae"/>
       </geometry>
     </collision>
@@ -168,46 +180,38 @@
     <origin xyz="${-wheel_x_offset} ${wheel_y_offset} 0"/>
   </joint>
+  <!-- ================== Payload ================== -->
+  <link name="payload_link">
+    <visual>
+      <origin xyz="0 0.0115 0" rpy="1.57 -0 1.57" />
+      <geometry>
+        <mesh filename="file://$(find custom_robots)/model/rover_4wd/meshes/rover_payload.dae"/>
+      </geometry>
+    </visual>
+    <collision>
+      <origin xyz="0 0.0115 0" rpy="1.57 -0 1.57" />
+      <geometry>
+        <mesh filename="file://$(find custom_robots)/model/rover_4wd/meshes/rover_payload.dae"/>
+      </geometry>
+    </collision>
+    <inertial>
+      <origin xyz="-0.01 0 0" rpy="0 0 0"/>
+      <mass value="2.95" />
+      <inertia ixx="0.018398" ixy="0.0" ixz="0.0" iyy="0.04064" iyz="0.0" izz="0.05396" />
+    </inertial>
+  </link>
+  <joint name="payload_to_chassis" type="fixed">
+    <parent link="chassis_link"/>
+    <child link="payload_link"/>
+    <origin xyz="0 0 ${payload_z_offset}"/>
+  </joint>
   <!-- ================== Gazebo Plugins ================== -->
-  <gazebo>
-    <plugin name="gz::sim::systems::DiffDrive" filename="gz-sim-diff-drive-system">
-        <num_wheel_pairs>2</num_wheel_pairs>
-        <!-- Wheel Information -->
-        <left_joint>rl_wheel_to_chassis</left_joint>
-        <left_joint>fl_wheel_to_chassis</left_joint>
-        <right_joint>rr_wheel_to_chassis</right_joint>
-        <right_joint>fr_wheel_to_chassis</right_joint>
-        <wheel_separation>0.24</wheel_separation>
-        <wheel_radius>0.122</wheel_radius>
-        <!-- Limits -->
-        <max_linear_acceleration>0.5</max_linear_acceleration>
-        <min_linear_acceleration>-0.5</min_linear_acceleration>
-        <max_angular_acceleration>0.8</max_angular_acceleration>
-        <min_angular_acceleration>-0.8</min_angular_acceleration>
-        <!-- Output -->
-        <frame_id>odom</frame_id>
-        <child_frame_id>base_link</child_frame_id>
-        <!-- Topics -->
-        <topic>/cmd_vel</topic>
-        <odom_topic>/odometry/wheels</odom_topic>
-        <tf_topic>/tf_gazebo</tf_topic>
-    </plugin>
-    <!-- Publicador de joint_states -->
-    <plugin name="gz::sim::systems::JointStatePublisher" filename="gz-sim-joint-state-publisher-system">
-      <topic>/joint_states</topic>
-    </plugin>
-    <!-- Publicador adicional de odometría -->
-    <plugin name="gz::sim::systems::OdometryPublisher" filename="gz-sim-odometry-publisher-system">
-      <odom_frame>odom</odom_frame>
-      <robot_base_frame>base_link</robot_base_frame>
-      <odom_topic>/odom</odom_topic>
-      <dimensions>3</dimensions>
-    </plugin>
-  </gazebo>
-  <!-- Publicador pose de gazebo-->
-  <plugin filename="gz-sim-pose-publisher-system" name="gz::sim::systems::PosePublisher">
-    <publish_model_pose>true</publish_model_pose>
-    <publish_nested_model>true</publish_nested_model>
-    <publish_nested_model_pose>true</publish_nested_model_pose>
-    <use_pose_vector_msg>true</use_pose_vector_msg>
-  </plugin>
+  <xacro:lidar xyz="0.174 0 0.10" rpy="0 0 0" name="lidar" parent="payload_link" topic="scan"/>
+  <xacro:imu xyz="0 0 0" rpy="0 0 0" parent="payload_link" topic="imu/data"/>
+  <xacro:velocity topic="/cmd_vel"/>
+  <xacro:joints topic="/joint_states"/>
+  <xacro:odom topic="/odom"/>
+  <xacro:unless value="${noise_level == 'none'}">
+    <xacro:noise_odom topic="/odom" vel_topic="/cmd_vel" a1="${a1}" a2="${a2}" a3="${a3}" a4="${a4}"/>
+  </xacro:unless>
+  <xacro:pose/>
 </robot>

Commit message: Update noise plugin

File: CustomRobots/rover_4wd/model/rover_4wd.urdf.xacro (robot description, xacro)
@@ -13,14 +13,14 @@
   <xacro:property name="noise_level" value="$(arg noise_level)"/>
   <xacro:if value="${noise_level == 'low'}">
-    <xacro:property name="a1" value="0.0005" />
-    <xacro:property name="a2" value="0.0005" />
-    <xacro:property name="a3" value="0.0002" />
-    <xacro:property name="a4" value="0.0002" />
+    <xacro:property name="a1" value="0.1" />
+    <xacro:property name="a2" value="0.1" />
+    <xacro:property name="a3" value="0.05" />
+    <xacro:property name="a4" value="0.05" />
   </xacro:if>
   <xacro:if value="${noise_level == 'high'}">
-    <xacro:property name="a1" value="0.005" />
-    <xacro:property name="a2" value="0.005" />
-    <xacro:property name="a3" value="0.003" />
-    <xacro:property name="a4" value="0.003" />
+    <xacro:property name="a1" value="1.5" />
+    <xacro:property name="a2" value="1.5" />
+    <xacro:property name="a3" value="0.8" />
+    <xacro:property name="a4" value="0.8" />
   </xacro:if>
   <xacro:include filename="$(find custom_robots)/model/rover_4wd/rover_4wd_gz.urdf.xacro"/>
@@ -212,5 +212,5 @@
   <xacro:odom topic="/odom"/>
   <xacro:unless value="${noise_level == 'none'}">
-    <xacro:noise_odom topic="/odom" vel_topic="/cmd_vel" a1="${a1}" a2="${a2}" a3="${a3}" a4="${a4}"/>
+    <xacro:noise_odom topic="/odom_noisy" a1="${a1}" a2="${a2}" a3="${a3}" a4="${a4}"/>
   </xacro:unless>
   <xacro:pose/>

File: CustomRobots/rover_4wd/model/rover_4wd_gz.urdf.xacro (robot description, xacro)
@@ -134,7 +134,11 @@
       <plugin filename="libNoisyOdometryPlugin.so" name="custom_plugins::NoisyOdometryPlugin">
         <ros_topic>${topic}</ros_topic>
-        <gz_cmd_vel_topic>${vel_topic}</gz_cmd_vel_topic>
         <frame_id>odom</frame_id>
         <child_frame_id>base_link</child_frame_id>
+        <!-- must match the DiffDrive plugin values above — one joint per side -->
+        <left_joint>fl_wheel_to_chassis</left_joint>
+        <right_joint>fr_wheel_to_chassis</right_joint>
+        <wheel_separation>0.24</wheel_separation>
+        <wheel_radius>0.122</wheel_radius>
         <alpha1>${a1}</alpha1>
         <alpha2>${a2}</alpha2>

File: CustomRobots/turtlebot3/models/turtlebot3/turtlebot3.urdf.xacro (robot description, xacro)
@@ -6,20 +6,20 @@
   <xacro:property name="noise_level" value="$(arg noise_level)"/>
   <xacro:if value="${noise_level == 'low'}">
-    <xacro:property name="a1" value="0.0005" />
-    <xacro:property name="a2" value="0.0005" />
-    <xacro:property name="a3" value="0.0002" />
-    <xacro:property name="a4" value="0.0002" />
+    <xacro:property name="a1" value="0.1" />
+    <xacro:property name="a2" value="0.1" />
+    <xacro:property name="a3" value="0.05" />
+    <xacro:property name="a4" value="0.05" />
   </xacro:if>
   <xacro:if value="${noise_level == 'med'}">
-    <xacro:property name="a1" value="0.002" />
-    <xacro:property name="a2" value="0.002" />
-    <xacro:property name="a3" value="0.001" />
-    <xacro:property name="a4" value="0.001" />
+    <xacro:property name="a1" value="0.5" />
+    <xacro:property name="a2" value="0.5" />
+    <xacro:property name="a3" value="0.25" />
+    <xacro:property name="a4" value="0.25" />
   </xacro:if>
   <xacro:if value="${noise_level == 'high'}">
-    <xacro:property name="a1" value="0.005" />
-    <xacro:property name="a2" value="0.005" />
-    <xacro:property name="a3" value="0.003" />
-    <xacro:property name="a4" value="0.003" />
+    <xacro:property name="a1" value="1.5" />
+    <xacro:property name="a2" value="1.5" />
+    <xacro:property name="a3" value="0.8" />
+    <xacro:property name="a4" value="0.8" />
   </xacro:if>
   <xacro:include filename="$(find custom_robots)/models/turtlebot3/turtlebot3_gz.urdf.xacro"/>
@@ -31,5 +31,5 @@
   </xacro:if>
   <xacro:unless value="${noise_level == 'none'}">
-    <xacro:noise_odom topic="/turtlebot3/odom_noisy" vel_topic="/turtlebot3/cmd_vel" a1="${a1}" a2="${a2}" a3="${a3}" a4="${a4}"/>
+    <xacro:noise_odom topic="/turtlebot3/odom_noisy" a1="${a1}" a2="${a2}" a3="${a3}" a4="${a4}"/>
   </xacro:unless>
 </robot>

File: CustomRobots/turtlebot3/models/turtlebot3/turtlebot3_gz.urdf.xacro (robot description, xacro)
@@ -218,15 +218,19 @@
     </gazebo>
   </xacro:macro>
-  <xacro:macro name="noise_odom" params="vel_topic topic">
+  <xacro:macro name="noise_odom" params="vel_topic topic a1 a2 a3 a4">
     <gazebo>
       <plugin filename="libNoisyOdometryPlugin.so" name="custom_plugins::NoisyOdometryPlugin">
         <ros_topic>${topic}</ros_topic>
-        <gz_cmd_vel_topic>${vel_topic}</gz_cmd_vel_topic>
         <frame_id>odom</frame_id>
         <child_frame_id>base</child_frame_id>
-        <alpha1>0.01</alpha1>
-        <alpha2>0.01</alpha2>
-        <alpha3>0.005</alpha3>
-        <alpha4>0.005</alpha4>
+        <!-- must match the DiffDrive plugin values above -->
+        <left_joint>wheel_left_joint</left_joint>
+        <right_joint>wheel_right_joint</right_joint>
+        <wheel_radius>0.033</wheel_radius>
+        <wheel_separation>0.287</wheel_separation>
+        <alpha1>${a1}</alpha1>
+        <alpha2>${a2}</alpha2>
+        <alpha3>${a3}</alpha3>
+        <alpha4>${a4}</alpha4>
       </plugin>
     </gazebo>
