Commit message: Simplify movement

File: CustomRobots/dingo/model/dingo/dingo.urdf.xacro (robot description, xacro)
@@ -4,4 +4,5 @@
   <xacro:arg name="gazebo_controllers" default="$(find custom_robots)/model/dingo/omni_4wd.yaml"/>
   <xacro:property name="PI" value="${math.pi}" />
+  <xacro:include filename="$(find custom_robots)/model/dingo/attachments/top_plate.urdf.xacro"/>
   <!-- D0150 Platform Macro -->
   <xacro:macro name="do150" params="control:='omni_4wd' front_wheels:='mecanum' rear_wheels:='mecanum'">
@@ -43,11 +44,9 @@
     <xacro:do100_drivetrain_wheels front_wheels="${front_wheels}" rear_wheels="${rear_wheels}"/>
     <!-- Add drivetrain -->
-    <xacro:include filename="$(find custom_robots)/model/dingo/drivetrain.urdf.xacro"/>
-    <!-- Hardware  -->
-    <xacro:property name="hardware_plugin" value="gz_ros2_control/GazeboSimSystem"/>
-    <xacro:unless value="${control == 'omni_4wd' or control == 'diff_4wd'}">
-      <xacro:error message="Invalid drivetrain control ${control}"/>
-    </xacro:unless>
-    <xacro:generic_drivetrain name="do150" control="${control}" front_wheels="${front_wheels}" rear_wheels="${rear_wheels}" hardware_plugin="${hardware_plugin}" />
+    <gazebo>
+      <plugin filename="gz-sim-velocity-control-system" name="gz::sim::systems::VelocityControl">
+        <topic>/cmd_vel</topic>
+      </plugin>
+    </gazebo>
     <!-- Internal IMU -->
     <link name="imu_0_link">
@@ -130,4 +129,5 @@
   <!-- Joint State Publisher -->
   <xacro:do150/>
+  <xacro:top_plate name="top_plate" parent_link="default_mount" height="1"/>
   <plugin filename="gz-sim-joint-state-publisher-system" name="gz::sim::systems::JointStatePublisher" />
 </robot>

Commit message: Update dingo sensors

File: CustomRobots/dingo/model/dingo/dingo.urdf.xacro (robot description, xacro)
@@ -5,4 +5,5 @@
   <xacro:property name="PI" value="${math.pi}" />
   <xacro:include filename="$(find custom_robots)/model/dingo/attachments/top_plate.urdf.xacro"/>
+  <xacro:include filename="$(find custom_robots)/models/dingo/dingo_gz.urdf.xacro"/>
   <!-- D0150 Platform Macro -->
   <xacro:macro name="do150" params="control:='omni_4wd' front_wheels:='mecanum' rear_wheels:='mecanum'">
@@ -43,31 +44,4 @@
     <xacro:include filename="$(find custom_robots)/model/dingo/wheels.urdf.xacro"/>
     <xacro:do100_drivetrain_wheels front_wheels="${front_wheels}" rear_wheels="${rear_wheels}"/>
-    <!-- Add drivetrain -->
-    <gazebo>
-      <plugin filename="gz-sim-velocity-control-system" name="gz::sim::systems::VelocityControl">
-        <topic>/cmd_vel</topic>
-      </plugin>
-    </gazebo>
-    <!-- Internal IMU -->
-    <link name="imu_0_link">
-      <inertial>
-        <mass value="0.001"/>
-        <origin xyz="0 0 0" rpy="0 0 0"/>
-        <inertia ixx="${dummy_inertia}" ixy="0.0" ixz="0.0" iyy="${dummy_inertia}" iyz="0.0" izz="${dummy_inertia}"/>
-      </inertial>
-    </link>
-    <joint name="imu_joint" type="fixed">
-      <parent link="chassis_link" />
-      <child link="imu_0_link" />
-    </joint>
-    <gazebo reference="imu_0_link">
-      <sensor type="imu" name="imu_0">
-        <always_on>true</always_on>
-        <update_rate>50</update_rate>
-        <visualize>true</visualize>
-        <gz_frame_id>imu_0_link</gz_frame_id>
-        <topic>$(arg namespace)/sensors/imu_0/data_raw</topic>
-      </sensor>
-    </gazebo>
     <!-- Mounting Hard Points -->
     <link name="default_mount"/>
@@ -129,7 +103,11 @@
   <!-- Joint State Publisher -->
   <xacro:do150/>
-  <xacro:top_plate name="top_plate" parent_link="default_mount" height="0.1">
+  <xacro:top_plate name="top_plate" parent_link="default_mount" height="0.15">
     <origin xyz="0 0 0"/>
   </xacro:top_plate>
+  <xacro:laser xyz="0 0 0.121" rpy="0 0 0" name="lidar" parent="chassis_link" topic="turtlebot3/laser/scan"/>
+  <xacro:imu parent="chassis_link" topic="turtlebot3/imu" xyz="0 0 0" rpy="0 0 0"/>
+  <xacro:odom topic="/turtlebot3/odom" freq="50"/>
+  <xacro:velocity topic="turtlebot3/cmd_vel"/>
   <plugin filename="gz-sim-joint-state-publisher-system" name="gz::sim::systems::JointStatePublisher" />
 </robot>

Commit message: Finished dingo base

File: CustomRobots/dingo/model/dingo/dingo.urdf.xacro (robot description, xacro)
@@ -5,5 +5,5 @@
   <xacro:property name="PI" value="${math.pi}" />
   <xacro:include filename="$(find custom_robots)/model/dingo/attachments/top_plate.urdf.xacro"/>
-  <xacro:include filename="$(find custom_robots)/models/dingo/dingo_gz.urdf.xacro"/>
+  <xacro:include filename="$(find custom_robots)/model/dingo/dingo_gz.urdf.xacro"/>
   <!-- D0150 Platform Macro -->
   <xacro:macro name="do150" params="control:='omni_4wd' front_wheels:='mecanum' rear_wheels:='mecanum'">
@@ -103,8 +103,8 @@
   <!-- Joint State Publisher -->
   <xacro:do150/>
-  <xacro:top_plate name="top_plate" parent_link="default_mount" height="0.15">
+  <xacro:top_plate name="top_plate" parent_link="default_mount" height="0.1">
     <origin xyz="0 0 0"/>
   </xacro:top_plate>
-  <xacro:laser xyz="0 0 0.121" rpy="0 0 0" name="lidar" parent="chassis_link" topic="turtlebot3/laser/scan"/>
+  <xacro:laser xyz="0 0 0.1" rpy="0 0 0" name="lidar" parent="chassis_link" topic="turtlebot3/laser/scan"/>
   <xacro:imu parent="chassis_link" topic="turtlebot3/imu" xyz="0 0 0" rpy="0 0 0"/>
   <xacro:odom topic="/turtlebot3/odom" freq="50"/>

File: CustomRobots/dingo/model/dingo/dingo_gz.urdf.xacro (robot description, xacro)
@@ -10,5 +10,5 @@
       <visual>
         <geometry>
-          <mesh filename="file://$(find custom_robots)/models/f1/meshes/hokuyo.dae"/>
+          <mesh filename="file://$(find custom_robots)/models/f1/meshes/hokuyo.dae" scale="10 10 10"/>
         </geometry>
         <material name="dark"/>

Commit message: Remove outdated resource and add dingo noise

File: CustomRobots/dingo/model/dingo/dingo.urdf.xacro (robot description, xacro)
@@ -3,5 +3,25 @@
   <xacro:arg name="namespace" default="" />
   <xacro:arg name="gazebo_controllers" default="$(find custom_robots)/model/dingo/omni_4wd.yaml"/>
+  <xacro:arg name="noise_level" default="none"/>
   <xacro:property name="PI" value="${math.pi}" />
+  <xacro:property name="noise_level" value="$(arg noise_level)"/>
+  <xacro:if value="${noise_level == 'low'}">
+    <xacro:property name="a1" value="0.1" />
+    <xacro:property name="a2" value="0.1" />
+    <xacro:property name="a3" value="0.05" />
+    <xacro:property name="a4" value="0.05" />
+  </xacro:if>
+  <xacro:if value="${noise_level == 'med'}">
+    <xacro:property name="a1" value="0.5" />
+    <xacro:property name="a2" value="0.5" />
+    <xacro:property name="a3" value="0.25" />
+    <xacro:property name="a4" value="0.25" />
+  </xacro:if>
+  <xacro:if value="${noise_level == 'high'}">
+    <xacro:property name="a1" value="1.5" />
+    <xacro:property name="a2" value="1.5" />
+    <xacro:property name="a3" value="0.8" />
+    <xacro:property name="a4" value="0.8" />
+  </xacro:if>
   <xacro:include filename="$(find custom_robots)/model/dingo/attachments/top_plate.urdf.xacro"/>
   <xacro:include filename="$(find custom_robots)/model/dingo/dingo_gz.urdf.xacro"/>
@@ -111,3 +131,6 @@
   <xacro:velocity topic="/cmd_vel"/>
   <plugin filename="gz-sim-joint-state-publisher-system" name="gz::sim::systems::JointStatePublisher" />
+  <xacro:unless value="${noise_level == 'none'}">
+    <xacro:noise_odom topic="/odom_noisy" a1="${a1}" a2="${a2}" a3="${a3}" a4="${a4}"/>
+  </xacro:unless>
 </robot>
