Commit message: odometry node, source Position for Dingo Robot

File: CustomRobots/dingo/model/dingo/dingo.urdf.xacro (robot description, xacro)
@@ -6,21 +6,23 @@
   <xacro:property name="PI" value="${math.pi}" />
   <xacro:property name="noise_level" value="$(arg noise_level)"/>
+  <!-- Odometry noise per difficulty — kept identical to the turtlebot3 levels
+       (drift std ~ alpha*sqrt(distance)). -->
   <xacro:if value="${noise_level == 'low'}">
-    <xacro:property name="a1" value="0.1" />
-    <xacro:property name="a2" value="0.1" />
+    <xacro:property name="a1" value="0.01" />
+    <xacro:property name="a2" value="0.01" />
+    <xacro:property name="a3" value="0.01" />
+    <xacro:property name="a4" value="0.01" />
+  </xacro:if>
+  <xacro:if value="${noise_level == 'med'}">
+    <xacro:property name="a1" value="0.05" />
+    <xacro:property name="a2" value="0.05" />
     <xacro:property name="a3" value="0.05" />
     <xacro:property name="a4" value="0.05" />
   </xacro:if>
-  <xacro:if value="${noise_level == 'med'}">
-    <xacro:property name="a1" value="0.5" />
-    <xacro:property name="a2" value="0.5" />
+  <xacro:if value="${noise_level == 'high'}">
+    <xacro:property name="a1" value="0.25" />
+    <xacro:property name="a2" value="0.25" />
     <xacro:property name="a3" value="0.25" />
     <xacro:property name="a4" value="0.25" />
-  </xacro:if>
-  <xacro:if value="${noise_level == 'high'}">
-    <xacro:property name="a1" value="1.5" />
-    <xacro:property name="a2" value="1.5" />
-    <xacro:property name="a3" value="0.8" />
-    <xacro:property name="a4" value="0.8" />
   </xacro:if>
   <xacro:include filename="$(find custom_robots)/model/dingo/attachments/top_plate.urdf.xacro"/>

File: CustomRobots/dingo/model/dingo/dingo_gz.urdf.xacro (robot description, xacro)
@@ -91,9 +91,10 @@
         <frame_id>odom</frame_id>
         <child_frame_id>chassis_link</child_frame_id>
-        <!-- must match the DiffDrive plugin values above -->
-        <left_joint>front_left_wheel_joint</left_joint>
-        <right_joint>front_right_wheel_joint</right_joint>
-        <wheel_radius>0.050</wheel_radius>
-        <wheel_separation>0.3708</wheel_separation>
+        <!-- Dingo is an omnidirectional (mecanum) platform driven kinematically by
+             the VelocityControl plugin, so wheel-encoder diff-drive reconstruction
+             does not apply. Derive the estimate from the model pose delta and track
+             lateral motion. -->
+        <odom_source>pose</odom_source>
+        <holonomic>true</holonomic>
         <alpha1>${a1}</alpha1>
         <alpha2>${a2}</alpha2>

Commit message: modify noise levels in dingo odometry

File: CustomRobots/dingo/model/dingo/dingo.urdf.xacro (robot description, xacro)
@@ -6,7 +6,14 @@
   <xacro:property name="PI" value="${math.pi}" />
   <xacro:property name="noise_level" value="$(arg noise_level)"/>
-  <!-- Odometry noise per difficulty — kept identical to the turtlebot3 levels
-       (drift std ~ alpha*sqrt(distance)). -->
+  <!-- Odometry noise per difficulty (drift std ~ alpha*sqrt(distance)).
+       Tuned lower than the turtlebot3 levels: the dingo estimate drifts faster,
+       so the whole scale is shifted down one notch (0.005 / 0.01 / 0.05). -->
   <xacro:if value="${noise_level == 'low'}">
+    <xacro:property name="a1" value="0.005" />
+    <xacro:property name="a2" value="0.005" />
+    <xacro:property name="a3" value="0.005" />
+    <xacro:property name="a4" value="0.005" />
+  </xacro:if>
+  <xacro:if value="${noise_level == 'med'}">
     <xacro:property name="a1" value="0.01" />
     <xacro:property name="a2" value="0.01" />
@@ -14,15 +21,9 @@
     <xacro:property name="a4" value="0.01" />
   </xacro:if>
-  <xacro:if value="${noise_level == 'med'}">
+  <xacro:if value="${noise_level == 'high'}">
     <xacro:property name="a1" value="0.05" />
     <xacro:property name="a2" value="0.05" />
     <xacro:property name="a3" value="0.05" />
     <xacro:property name="a4" value="0.05" />
-  </xacro:if>
-  <xacro:if value="${noise_level == 'high'}">
-    <xacro:property name="a1" value="0.25" />
-    <xacro:property name="a2" value="0.25" />
-    <xacro:property name="a3" value="0.25" />
-    <xacro:property name="a4" value="0.25" />
   </xacro:if>
   <xacro:include filename="$(find custom_robots)/model/dingo/attachments/top_plate.urdf.xacro"/>

Commit message: Add changes from 766

File: CustomRobots/dingo/model/dingo/dingo.urdf.xacro (robot description, xacro)
@@ -6,21 +6,24 @@
   <xacro:property name="PI" value="${math.pi}" />
   <xacro:property name="noise_level" value="$(arg noise_level)"/>
+  <!-- Odometry noise per difficulty (drift std ~ alpha*sqrt(distance)).
+       Tuned lower than the turtlebot3 levels: the dingo estimate drifts faster,
+       so the whole scale is shifted down one notch (0.005 / 0.01 / 0.05). -->
   <xacro:if value="${noise_level == 'low'}">
-    <xacro:property name="a1" value="0.1" />
-    <xacro:property name="a2" value="0.1" />
+    <xacro:property name="a1" value="0.005" />
+    <xacro:property name="a2" value="0.005" />
+    <xacro:property name="a3" value="0.005" />
+    <xacro:property name="a4" value="0.005" />
+  </xacro:if>
+  <xacro:if value="${noise_level == 'med'}">
+    <xacro:property name="a1" value="0.01" />
+    <xacro:property name="a2" value="0.01" />
+    <xacro:property name="a3" value="0.01" />
+    <xacro:property name="a4" value="0.01" />
+  </xacro:if>
+  <xacro:if value="${noise_level == 'high'}">
+    <xacro:property name="a1" value="0.05" />
+    <xacro:property name="a2" value="0.05" />
     <xacro:property name="a3" value="0.05" />
     <xacro:property name="a4" value="0.05" />
-  </xacro:if>
-  <xacro:if value="${noise_level == 'med'}">
-    <xacro:property name="a1" value="0.5" />
-    <xacro:property name="a2" value="0.5" />
-    <xacro:property name="a3" value="0.25" />
-    <xacro:property name="a4" value="0.25" />
-  </xacro:if>
-  <xacro:if value="${noise_level == 'high'}">
-    <xacro:property name="a1" value="1.5" />
-    <xacro:property name="a2" value="1.5" />
-    <xacro:property name="a3" value="0.8" />
-    <xacro:property name="a4" value="0.8" />
   </xacro:if>
   <xacro:include filename="$(find custom_robots)/model/dingo/attachments/top_plate.urdf.xacro"/>
@@ -132,5 +135,7 @@
   <plugin filename="gz-sim-joint-state-publisher-system" name="gz::sim::systems::JointStatePublisher" />
   <xacro:unless value="${noise_level == 'none'}">
-    <xacro:noise_odom topic="/odom_noisy" a1="${a1}" a2="${a2}" a3="${a3}" a4="${a4}"/>
+    <!-- ROS topic name matches the laser_mapping exercise interface. The plugin
+         publishes to ROS directly (not through the gz bridge). -->
+    <xacro:noise_odom topic="/turtlebot3/odom_noisy" a1="${a1}" a2="${a2}" a3="${a3}" a4="${a4}"/>
   </xacro:unless>
 </robot>

Commit message: Add namespace

File: CustomRobots/dingo/model/dingo/dingo.urdf.xacro (robot description, xacro)
@@ -6,4 +6,5 @@
   <xacro:property name="PI" value="${math.pi}" />
   <xacro:property name="noise_level" value="$(arg noise_level)"/>
+  <xacro:property name="namespace" value="$(arg namespace)"/>
   <!-- Odometry noise per difficulty (drift std ~ alpha*sqrt(distance)).
        Tuned lower than the turtlebot3 levels: the dingo estimate drifts faster,
@@ -137,5 +138,5 @@
     <!-- ROS topic name matches the laser_mapping exercise interface. The plugin
          publishes to ROS directly (not through the gz bridge). -->
-    <xacro:noise_odom topic="/turtlebot3/odom_noisy" a1="${a1}" a2="${a2}" a3="${a3}" a4="${a4}"/>
+    <xacro:noise_odom topic="/${namespace}/odom_noisy" a1="${a1}" a2="${a2}" a3="${a3}" a4="${a4}"/>
   </xacro:unless>
 </robot>
