Commit message: Fix meshes

File: CustomRobots/ur5/models/ur5/ur_generated.urdf (robot description, URDF)
Before this commit: robot ur5, 14 links, 13 joints
Links:
- link base_link_inertia: geometry collision mesh filename=package://ros2srrc_ur5_gazebo/meshes/ur5/collision/base.stl; visual mesh filename=package://ros2srrc_ur5_gazebo/meshes/ur5/visual/base.dae
- link forearm_link: geometry collision mesh filename=package://ros2srrc_ur5_gazebo/meshes/ur5/collision/forearm.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; visual mesh filename=package://ros2srrc_ur5_gazebo/meshes/ur5/visual/forearm.dae
- link shoulder_link: geometry collision mesh filename=package://ros2srrc_ur5_gazebo/meshes/ur5/collision/shoulder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; visual mesh filename=package://ros2srrc_ur5_gazebo/meshes/ur5/visual/shoulder.dae
- link upper_arm_link: geometry collision mesh filename=package://ros2srrc_ur5_gazebo/meshes/ur5/collision/upperarm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; visual mesh filename=package://ros2srrc_ur5_gazebo/meshes/ur5/visual/upperarm.dae
- link wrist_1_link: geometry collision mesh filename=package://ros2srrc_ur5_gazebo/meshes/ur5/collision/wrist1.s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; visual mesh filename=package://ros2srrc_ur5_gazebo/meshes/ur5/visual/wrist1.dae
- link wrist_2_link: geometry collision mesh filename=package://ros2srrc_ur5_gazebo/meshes/ur5/collision/wrist2.s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; visual mesh filename=package://ros2srrc_ur5_gazebo/meshes/ur5/visual/wrist2.dae
- link wrist_3_link: geometry collision mesh filename=package://ros2srrc_ur5_gazebo/meshes/ur5/collision/wrist3.s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; visual mesh filename=package://ros2srrc_ur5_gazebo/meshes/ur5/visual/wrist3.dae

Commit message: Test visual changes

File: CustomRobots/ur5/models/ur5/ur_generated.urdf (robot description, URDF)
Before this commit: robot ur5, 14 links, 13 joints
Links:
- link base_link_inertia: geometry collision mesh filename=package://ros2srrc_robots/ur5/meshes/collision/base.stl; visual mesh filename=package://ros2srrc_robots/ur5/meshes/visual/base.dae
- link forearm_link: geometry collision mesh filename=package://ros2srrc_robots/ur5/meshes/collision/forearm.stl; visual mesh filename=package://ros2srrc_robots/ur5/meshes/visual/forearm.dae
- link shoulder_link: geometry collision mesh filename=package://ros2srrc_robots/ur5/meshes/collision/shoulder.stl; visual mesh filename=package://ros2srrc_robots/ur5/meshes/visual/shoulder.dae
- link upper_arm_link: geometry collision mesh filename=package://ros2srrc_robots/ur5/meshes/collision/upperarm.stl; visual mesh filename=package://ros2srrc_robots/ur5/meshes/visual/upperarm.dae
- link wrist_1_link: geometry collision mesh filename=package://ros2srrc_robots/ur5/meshes/collision/wrist1.stl; visual mesh filename=package://ros2srrc_robots/ur5/meshes/visual/wrist1.dae
- link wrist_2_link: geometry collision mesh filename=package://ros2srrc_robots/ur5/meshes/collision/wrist2.stl; visual mesh filename=package://ros2srrc_robots/ur5/meshes/visual/wrist2.dae
- link wrist_3_link: geometry collision mesh filename=package://ros2srrc_robots/ur5/meshes/collision/wrist3.stl; visual mesh filename=package://ros2srrc_robots/ur5/meshes/visual/wrist3.dae
