Commit message: Change robot spawn position

File: Industrial/ros2_SimRealRobotControl_gz/packages/ur3/ros2srrc_ur3_gazebo/urdf/ur3_robotiq_2f85.urdf.xacro (robot description, xacro)
@@ -90,5 +90,5 @@
       <origin xyz="0 0 0" rpy=" 0 0 0"/>
       <geometry>
-        <box size = "0.2 0.2 1.0"/>
+        <box size = "0.2 0.2 0.8"/>
       </geometry>
     </collision>

Commit message: Add Ur3 launchers

File: Industrial/ros2_SimRealRobotControl_gz/packages/ur3/ros2srrc_ur3_gazebo/urdf/ur3_robotiq_2f85.urdf.xacro (robot description, xacro)
@@ -40,4 +40,6 @@
   <xacro:arg name="EE_name" default="none"/>
   <xacro:property name="EE_name" value="$(arg EE_name)"/>
+  <xacro:arg name="camera" default="false"/>
+  <xacro:property name="camera" value="$(arg camera)"/>
   <!-- UR3 Control ARGUMENTS -->
   <xacro:arg name="script_filename" default="none"/>
@@ -47,4 +49,10 @@
   <xacro:arg name="output_recipe_filename" default="none"/>
   <xacro:property name="output_recipe_filename" value="$(arg output_recipe_filename)"/>
+  <!-- Include cams -->
+  <xacro:include filename="$(find ros2srrc_ur5_gazebo)/urdf/common_properties.xacro"/>
+  <xacro:include filename="$(find ros2srrc_ur5_gazebo)/urdf/cam_on_hand_params.xacro"/>
+  <xacro:include filename="$(find ros2srrc_ur5_gazebo)/urdf/cam_on_hand.xacro"/>
+  <xacro:include filename="$(find ros2srrc_ur5_gazebo)/urdf/cam_on_base_params.xacro"/>
+  <xacro:include filename="$(find ros2srrc_ur5_gazebo)/urdf/cam_on_base.xacro"/>
   <!-- Include XACRO-MACRO file of the UR3: -->
   <xacro:include filename="$(find ros2srrc_robots)/ur3/urdf/ur3_macro.urdf.xacro"/>
@@ -64,4 +72,8 @@
     parent_link="tool0"
   />
+  <xacro:if value="${camera}">
+    <xacro:cam_on_hand/>
+    <xacro:cam_on_base/>
+  </xacro:if>
   <!-- Load ROS 2 Gazebo Plugin -->
   <xacro:unless value="${bringup}">
@@ -96,5 +108,5 @@
       <origin xyz="0 0 0" rpy=" 0 0 0"/>
       <geometry>
-        <box size = "0.2 0.2 1.0"/>
+        <box size = "0.2 0.2 0.8"/>
       </geometry>
     </visual>

Commit message: Fix xacro and add sausage spawn

File: Industrial/ros2_SimRealRobotControl_gz/packages/ur3/ros2srrc_ur3_gazebo/urdf/ur3_robotiq_2f85.urdf.xacro (robot description, xacro)
@@ -51,7 +51,12 @@
   <!-- Include cams -->
   <xacro:include filename="$(find ros2srrc_ur5_gazebo)/urdf/common_properties.xacro"/>
+  <!-- HAND CAMERA -->
   <xacro:include filename="$(find ros2srrc_ur5_gazebo)/urdf/cam_on_hand_params_gz.xacro"/>
+  <xacro:property name="parent_hand" value="tool0"/>
   <xacro:include filename="$(find ros2srrc_ur5_gazebo)/urdf/cam_on_hand_gz.xacro"/>
+  <!-- BASE CAMERA -->
   <xacro:include filename="$(find ros2srrc_ur5_gazebo)/urdf/cam_on_base_params_gz.xacro"/>
+  <xacro:property name="parent_base" value="base_link"/>
+  <xacro:property name="cam_base_pz" value="0.5"/>
   <xacro:include filename="$(find ros2srrc_ur5_gazebo)/urdf/cam_on_base_gz.xacro"/>
   <!-- Include XACRO-MACRO file of the UR3: -->
@@ -72,8 +77,4 @@
     parent_link="tool0"
   />
-  <xacro:if value="${camera}">
-    <xacro:cam_on_hand/>
-    <xacro:cam_on_base/>
-  </xacro:if>
   <!-- Load ROS 2 Gazebo Plugin -->
   <xacro:unless value="${bringup}">

Commit message: Fix xacro and robot spawn

File: Industrial/ros2_SimRealRobotControl_gz/packages/ur3/ros2srrc_ur3_gazebo/urdf/ur3_robotiq_2f85.urdf.xacro (robot description, xacro)
@@ -103,5 +103,5 @@
       <origin xyz="0 0 0" rpy=" 0 0 0"/>
       <geometry>
-        <box size = "0.2 0.2 0.8"/>
+        <box size = "0.2 0.2 1.0"/>
       </geometry>
     </collision>
@@ -109,5 +109,5 @@
       <origin xyz="0 0 0" rpy=" 0 0 0"/>
       <geometry>
-        <box size = "0.2 0.2 0.8"/>
+        <box size = "0.2 0.2 1.0"/>
       </geometry>
     </visual>

Commit message: Try to fix gripper controller

File: Industrial/ros2_SimRealRobotControl_gz/packages/ur3/ros2srrc_ur3_gazebo/urdf/ur3_robotiq_2f85.urdf.xacro (robot description, xacro)
@@ -62,19 +62,44 @@
   <!-- Include XACRO-MACRO file of the UR3: -->
   <xacro:include filename="$(find ros2srrc_robots)/ur3/urdf/ur3_macro.urdf.xacro"/>
+  <xacro:include filename="$(find robotiq_description)/urdf/robotiq_85_gripper.urdf.xacro"/>
+  <xacro:include filename="$(find robotiq_description)/urdf/robotiq_85_gripper.ros2_control.xacro"/>
   <xacro:ur3
     bringup="${bringup}"
     robot_ip="${robot_ip}"
-    EE="${EE}"
-    EE_name="${EE_name}"
+    EE="false"
+    EE_name="none"
     script_filename="${script_filename}"
     input_recipe_filename="${input_recipe_filename}"
     output_recipe_filename="${output_recipe_filename}"
   />
-  <!-- Include XACRO-MACRO file of the Robotiq 2f-85: -->
-  <xacro:include filename="$(find ros2srrc_endeffectors)/robotiq_2f85/urdf/robotiq_2f85_macro.urdf.xacro"/>
-  <xacro:robotiq_2f85
-    bringup="${bringup}"
-    parent_link="tool0"
-  />
+  <!-- Coupler -->
+  <link name="robotiq_coupler">
+    <visual>
+      <geometry>
+        <mesh filename="package://robotiq_description/meshes/robotiq_85_coupler.stl"/>
+      </geometry>
+    </visual>
+    <collision>
+      <geometry>
+        <cylinder radius="0.04" length="0.015"/>
+      </geometry>
+    </collision>
+  </link>
+  <joint name="robotiq_coupler_joint" type="fixed">
+    <origin xyz="0 0 0.004" rpy="0 0 ${-pi/2.0}" />
+    <parent link="tool0"/>
+    <child link="robotiq_coupler"/>
+  </joint>
+  <xacro:robotiq_85_gripper
+      prefix=""
+      parent="robotiq_coupler">
+      <origin xyz="0 0 0.004"
+              rpy="0 ${-pi/2} ${pi}"/>
+  </xacro:robotiq_85_gripper>
+  <xacro:robotiq_85_ros2_control
+    name="robotiq"
+    prefix=""
+    sim_gz="true"
+    use_fake_hardware="false"/>
   <!-- Load ROS 2 Gazebo Plugin -->
   <xacro:unless value="${bringup}">
@@ -84,7 +109,4 @@
         <parameters>
           $(find ros2srrc_robots)/ur3/config/controller.yaml
-        </parameters>
-        <parameters>
-          $(find ros2srrc_endeffectors)/${EE_name}/config/controller.yaml
         </parameters>
       </plugin>

Commit message: Restart gripper controller

File: Industrial/ros2_SimRealRobotControl_gz/packages/ur3/ros2srrc_ur3_gazebo/urdf/ur3_robotiq_2f85.urdf.xacro (robot description, xacro)
@@ -62,44 +62,19 @@
   <!-- Include XACRO-MACRO file of the UR3: -->
   <xacro:include filename="$(find ros2srrc_robots)/ur3/urdf/ur3_macro.urdf.xacro"/>
-  <xacro:include filename="$(find robotiq_description)/urdf/robotiq_85_gripper.urdf.xacro"/>
-  <xacro:include filename="$(find robotiq_description)/urdf/robotiq_85_gripper.ros2_control.xacro"/>
   <xacro:ur3
     bringup="${bringup}"
     robot_ip="${robot_ip}"
-    EE="false"
-    EE_name="none"
+    EE="${EE}"
+    EE_name="${EE_name}"
     script_filename="${script_filename}"
     input_recipe_filename="${input_recipe_filename}"
     output_recipe_filename="${output_recipe_filename}"
   />
-  <!-- Coupler -->
-  <link name="robotiq_coupler">
-    <visual>
-      <geometry>
-        <mesh filename="package://robotiq_description/meshes/robotiq_85_coupler.stl"/>
-      </geometry>
-    </visual>
-    <collision>
-      <geometry>
-        <cylinder radius="0.04" length="0.015"/>
-      </geometry>
-    </collision>
-  </link>
-  <joint name="robotiq_coupler_joint" type="fixed">
-    <origin xyz="0 0 0.004" rpy="0 0 ${-pi/2.0}" />
-    <parent link="tool0"/>
-    <child link="robotiq_coupler"/>
-  </joint>
-  <xacro:robotiq_85_gripper
-      prefix=""
-      parent="robotiq_coupler">
-      <origin xyz="0 0 0.004"
-              rpy="0 ${-pi/2} ${pi}"/>
-  </xacro:robotiq_85_gripper>
-  <xacro:robotiq_85_ros2_control
-    name="robotiq"
-    prefix=""
-    sim_gz="true"
-    use_fake_hardware="false"/>
+  <!-- Include XACRO-MACRO file of the Robotiq 2f-85: -->
+  <xacro:include filename="$(find ros2srrc_endeffectors)/robotiq_2f85/urdf/robotiq_2f85_macro.urdf.xacro"/>
+  <xacro:robotiq_2f85
+    bringup="${bringup}"
+    parent_link="tool0"
+  />
   <!-- Load ROS 2 Gazebo Plugin -->
   <xacro:unless value="${bringup}">
@@ -109,4 +84,7 @@
         <parameters>
           $(find ros2srrc_robots)/ur3/config/controller.yaml
+        </parameters>
+        <parameters>
+          $(find ros2srrc_endeffectors)/${EE_name}/config/controller.yaml
         </parameters>
       </plugin>

Commit message: try another method for gripper controller

File: Industrial/ros2_SimRealRobotControl_gz/packages/ur3/ros2srrc_ur3_gazebo/urdf/ur3_robotiq_2f85.urdf.xacro (robot description, xacro)
@@ -72,9 +72,34 @@
   />
   <!-- Include XACRO-MACRO file of the Robotiq 2f-85: -->
-  <xacro:include filename="$(find ros2srrc_endeffectors)/robotiq_2f85/urdf/robotiq_2f85_macro.urdf.xacro"/>
-  <xacro:robotiq_2f85
-    bringup="${bringup}"
-    parent_link="tool0"
-  />
+  <xacro:include filename="$(find robotiq_description)/urdf/robotiq_85_gripper.urdf.xacro"/>
+  <xacro:include filename="$(find robotiq_description)/urdf/robotiq_85_gripper.ros2_control.xacro"/>
+  <link name="robotiq_coupler">
+    <visual>
+      <geometry>
+        <mesh filename="package://robotiq_description/meshes/robotiq_85_coupler.stl"/>
+      </geometry>
+    </visual>
+    <collision>
+      <geometry>
+        <cylinder radius="0.04" length="0.015"/>
+      </geometry>
+    </collision>
+  </link>
+  <joint name="robotiq_coupler_joint" type="fixed">
+    <origin xyz="0 0 0.004" rpy="0 0 ${-pi/2.0}"/>
+    <parent link="tool0"/>
+    <child link="robotiq_coupler"/>
+  </joint>
+  <xacro:robotiq_85_gripper
+    prefix=""
+    parent="robotiq_coupler">
+    <origin xyz="0 0 0.004"
+            rpy="0 ${-pi/2} ${pi}"/>
+  </xacro:robotiq_85_gripper>
+  <xacro:robotiq_85_ros2_control
+    name="robotiq"
+    prefix=""
+    sim_gz="true"
+  use_fake_hardware="false"/>
   <!-- Load ROS 2 Gazebo Plugin -->
   <xacro:unless value="${bringup}">

Commit message: try another method for gripper controller

File: Industrial/ros2_SimRealRobotControl_gz/packages/ur3/ros2srrc_ur3_gazebo/urdf/ur3_robotiq_2f85.urdf.xacro (robot description, xacro)
@@ -72,10 +72,10 @@
   />
   <!-- Include XACRO-MACRO file of the Robotiq 2f-85: -->
-  <xacro:include filename="$(find robotiq_description)/urdf/robotiq_85_gripper.urdf.xacro"/>
-  <xacro:include filename="$(find robotiq_description)/urdf/robotiq_85_gripper.ros2_control.xacro"/>
+  <xacro:include filename="$(find robotiq_description)/urdf/robotiq_85_gripper.urdf.xacro" />
+  <!-- Coupler -->
   <link name="robotiq_coupler">
     <visual>
       <geometry>
-        <mesh filename="package://robotiq_description/meshes/robotiq_85_coupler.stl"/>
+        <mesh filename="file://$(find ros2srrc_endeffectors)/robotiq_2f85/meshes/robotiq_85_coupler.stl" />
       </geometry>
     </visual>
@@ -87,19 +87,11 @@
   </link>
   <joint name="robotiq_coupler_joint" type="fixed">
-    <origin xyz="0 0 0.004" rpy="0 0 ${-pi/2.0}"/>
+    <origin xyz="0 0 0.004" rpy="0 0 ${-pi/2.0}" />
     <parent link="tool0"/>
     <child link="robotiq_coupler"/>
   </joint>
-  <xacro:robotiq_85_gripper
-    prefix=""
-    parent="robotiq_coupler">
-    <origin xyz="0 0 0.004"
-            rpy="0 ${-pi/2} ${pi}"/>
+  <xacro:robotiq_85_gripper prefix="" parent="robotiq_coupler">
+    <origin xyz="0 0 0.004" rpy="0 ${-pi/2} ${pi}"/>
   </xacro:robotiq_85_gripper>
-  <xacro:robotiq_85_ros2_control
-    name="robotiq"
-    prefix=""
-    sim_gz="true"
-  use_fake_hardware="false"/>
   <!-- Load ROS 2 Gazebo Plugin -->
   <xacro:unless value="${bringup}">

Commit message: Restart

File: Industrial/ros2_SimRealRobotControl_gz/packages/ur3/ros2srrc_ur3_gazebo/urdf/ur3_robotiq_2f85.urdf.xacro (robot description, xacro)
@@ -72,26 +72,9 @@
   />
   <!-- Include XACRO-MACRO file of the Robotiq 2f-85: -->
-  <xacro:include filename="$(find robotiq_description)/urdf/robotiq_85_gripper.urdf.xacro" />
-  <!-- Coupler -->
-  <link name="robotiq_coupler">
-    <visual>
-      <geometry>
-        <mesh filename="file://$(find ros2srrc_endeffectors)/robotiq_2f85/meshes/robotiq_85_coupler.stl" />
-      </geometry>
-    </visual>
-    <collision>
-      <geometry>
-        <cylinder radius="0.04" length="0.015"/>
-      </geometry>
-    </collision>
-  </link>
-  <joint name="robotiq_coupler_joint" type="fixed">
-    <origin xyz="0 0 0.004" rpy="0 0 ${-pi/2.0}" />
-    <parent link="tool0"/>
-    <child link="robotiq_coupler"/>
-  </joint>
-  <xacro:robotiq_85_gripper prefix="" parent="robotiq_coupler">
-    <origin xyz="0 0 0.004" rpy="0 ${-pi/2} ${pi}"/>
-  </xacro:robotiq_85_gripper>
+  <xacro:include filename="$(find ros2srrc_endeffectors)/robotiq_2f85/urdf/robotiq_2f85_macro.urdf.xacro"/>
+  <xacro:robotiq_2f85
+    bringup="${bringup}"
+    parent_link="tool0"
+  />
   <!-- Load ROS 2 Gazebo Plugin -->
   <xacro:unless value="${bringup}">

Commit message: Delete robot stand in ur3 urdf

File: Industrial/ros2_SimRealRobotControl_gz/packages/ur3/ros2srrc_ur3_gazebo/urdf/ur3_robotiq_2f85.urdf.xacro (robot description, xacro)
@@ -93,35 +93,9 @@
   <!-- World: LINK -->
   <link name="world"/>
-  <!-- Robot Stand: LINK -->
-  <link name='robot_stand'>
-    <inertial>
-      <origin xyz="0 0 0" rpy="0 0 0"/>
-      <mass value="100"/>
-      <inertia ixx="0.01"  ixy="0"  ixz="0" iyy="0.01" iyz="0" izz="0.01" />
-    </inertial>
-    <collision name='collision'>
-      <origin xyz="0 0 0" rpy=" 0 0 0"/>
-      <geometry>
-        <box size = "0.2 0.2 1.0"/>
-      </geometry>
-    </collision>
-    <visual name='chassis_visual'>
-      <origin xyz="0 0 0" rpy=" 0 0 0"/>
-      <geometry>
-        <box size = "0.2 0.2 1.0"/>
-      </geometry>
-    </visual>
-  </link>
-  <!-- Robot Stand: FIXED JOINT -->
+  <!-- World -> Robot -->
   <joint name="world_joint" type="fixed">
-    <parent link= "world" />
-    <child link = "robot_stand" />
-    <origin xyz="0.0 0.0 0.5" rpy="0.0 0.0 0.0" />
-  </joint>
-  <!-- Robot Stand: Robot+Stand JOINT -->
-  <joint name="stand_joint" type="fixed">
-    <parent link= "robot_stand" />
-    <child link = "base_link" />
-    <origin xyz="0.0 0.0 0.505" rpy="0.0 0.0 0.0" />
+    <parent link="world"/>
+    <child link="base_link"/>
+    <origin xyz="0.0 0.0 1.005" rpy="0 0 0"/>
   </joint>
   <!-- ros2srrc_HMI CAMERA -->

Commit message: fix robot spawn position

File: Industrial/ros2_SimRealRobotControl_gz/packages/ur3/ros2srrc_ur3_gazebo/urdf/ur3_robotiq_2f85.urdf.xacro (robot description, xacro)
@@ -91,12 +91,4 @@
     </gazebo>
   </xacro:unless>
-  <!-- World: LINK -->
-  <link name="world"/>
-  <!-- World -> Robot -->
-  <joint name="world_joint" type="fixed">
-    <parent link="world"/>
-    <child link="base_link"/>
-    <origin xyz="0.0 0.0 1.005" rpy="0 0 0"/>
-  </joint>
   <!-- ros2srrc_HMI CAMERA -->
   <xacro:if value="${hmi}">

Commit message: Try to fiz planification

File: Industrial/ros2_SimRealRobotControl_gz/packages/ur3/ros2srrc_ur3_gazebo/urdf/ur3_robotiq_2f85.urdf.xacro (robot description, xacro)
@@ -91,4 +91,40 @@
     </gazebo>
   </xacro:unless>
+  <!-- World: LINK -->
+  <link name="world"/>
+  <!-- Robot Stand: LINK -->
+  <link name='robot_stand'>
+    <inertial>
+      <origin xyz="0 0 0" rpy="0 0 0"/>
+      <mass value="100"/>
+      <inertia ixx="0.01" ixy="0" ixz="0"
+               iyy="0.01" iyz="0"
+               izz="0.01" />
+    </inertial>
+    <collision name='collision'>
+      <origin xyz="0 0 0" rpy="0 0 0"/>
+      <geometry>
+        <box size="0.2 0.2 1.0"/>
+      </geometry>
+    </collision>
+    <visual name='chassis_visual'>
+      <origin xyz="0 0 0" rpy="0 0 0"/>
+      <geometry>
+        <box size="0.2 0.2 1.0"/>
+      </geometry>
+    </visual>
+  </link>
+  <!-- World -> Stand -->
+  <joint name="world_joint" type="fixed">
+    <parent link="world"/>
+    <child link="robot_stand"/>
+    <origin xyz="0.0 0.0 0.5" rpy="0 0 0"/>
+  </joint>
+  <!-- Stand -> Robot -->
+  <joint name="stand_joint" type="fixed">
+    <parent link="robot_stand"/>
+    <child link="base_link"/>
+    <origin xyz="0.0 0.0 0.505" rpy="0 0 0"/>
+  </joint>
   <!-- ros2srrc_HMI CAMERA -->
   <xacro:if value="${hmi}">

Commit message: Try to fix planification

File: Industrial/ros2_SimRealRobotControl_gz/packages/ur3/ros2srrc_ur3_gazebo/urdf/ur3_robotiq_2f85.urdf.xacro (robot description, xacro)
@@ -91,40 +91,4 @@
     </gazebo>
   </xacro:unless>
-  <!-- World: LINK -->
-  <link name="world"/>
-  <!-- Robot Stand: LINK -->
-  <link name='robot_stand'>
-    <inertial>
-      <origin xyz="0 0 0" rpy="0 0 0"/>
-      <mass value="100"/>
-      <inertia ixx="0.01" ixy="0" ixz="0"
-               iyy="0.01" iyz="0"
-               izz="0.01" />
-    </inertial>
-    <collision name='collision'>
-      <origin xyz="0 0 0" rpy="0 0 0"/>
-      <geometry>
-        <box size="0.2 0.2 1.0"/>
-      </geometry>
-    </collision>
-    <visual name='chassis_visual'>
-      <origin xyz="0 0 0" rpy="0 0 0"/>
-      <geometry>
-        <box size="0.2 0.2 1.0"/>
-      </geometry>
-    </visual>
-  </link>
-  <!-- World -> Stand -->
-  <joint name="world_joint" type="fixed">
-    <parent link="world"/>
-    <child link="robot_stand"/>
-    <origin xyz="0.0 0.0 0.5" rpy="0 0 0"/>
-  </joint>
-  <!-- Stand -> Robot -->
-  <joint name="stand_joint" type="fixed">
-    <parent link="robot_stand"/>
-    <child link="base_link"/>
-    <origin xyz="0.0 0.0 0.505" rpy="0 0 0"/>
-  </joint>
   <!-- ros2srrc_HMI CAMERA -->
   <xacro:if value="${hmi}">

Commit message: Add robot stand to xacro

File: Industrial/ros2_SimRealRobotControl_gz/packages/ur3/ros2srrc_ur3_gazebo/urdf/ur3_robotiq_2f85.urdf.xacro (robot description, xacro)
@@ -91,4 +91,38 @@
     </gazebo>
   </xacro:unless>
+  <!-- World: LINK -->
+  <link name="world"/>
+  <!-- Robot Stand: LINK -->
+  <link name='robot_stand'>
+    <inertial>
+      <origin xyz="0 0 0" rpy="0 0 0"/>
+      <mass value="100"/>
+      <inertia ixx="0.01"  ixy="0"  ixz="0" iyy="0.01" iyz="0" izz="0.01" />
+    </inertial>
+    <collision name='collision'>
+      <origin xyz="0 0 0" rpy=" 0 0 0"/>
+      <geometry>
+        <box size = "0.2 0.2 1.0"/>
+      </geometry>
+    </collision>
+    <visual name='chassis_visual'>
+      <origin xyz="0 0 0" rpy=" 0 0 0"/>
+      <geometry>
+        <box size = "0.2 0.2 1.0"/>
+      </geometry>
+    </visual>
+  </link>
+  <!-- Robot Stand: FIXED JOINT -->
+  <joint name="world_joint" type="fixed">
+    <parent link= "world" />
+    <child link = "robot_stand" />
+    <origin xyz="0.0 0.0 0.5" rpy="0.0 0.0 0.0" />
+  </joint>
+  <!-- Robot Stand: Robot+Stand JOINT -->
+  <joint name="stand_joint" type="fixed">
+    <parent link= "robot_stand" />
+    <child link = "base_link" />
+    <origin xyz="0.0 0.0 0.505" rpy="0.0 0.0 0.0" />
+  </joint>
   <!-- ros2srrc_HMI CAMERA -->
   <xacro:if value="${hmi}">

Commit message: add if camera to ur3 xacro

File: Industrial/ros2_SimRealRobotControl_gz/packages/ur3/ros2srrc_ur3_gazebo/urdf/ur3_robotiq_2f85.urdf.xacro (robot description, xacro)
@@ -50,14 +50,16 @@
   <xacro:property name="output_recipe_filename" value="$(arg output_recipe_filename)"/>
   <!-- Include cams -->
-  <xacro:include filename="$(find ros2srrc_ur5_gazebo)/urdf/common_properties.xacro"/>
-  <!-- HAND CAMERA -->
-  <xacro:include filename="$(find ros2srrc_ur5_gazebo)/urdf/cam_on_hand_params_gz.xacro"/>
-  <xacro:property name="parent_hand" value="tool0"/>
-  <xacro:include filename="$(find ros2srrc_ur5_gazebo)/urdf/cam_on_hand_gz.xacro"/>
-  <!-- BASE CAMERA -->
-  <xacro:include filename="$(find ros2srrc_ur5_gazebo)/urdf/cam_on_base_params_gz.xacro"/>
-  <xacro:property name="parent_base" value="base_link"/>
-  <xacro:property name="cam_base_pz" value="0.5"/>
-  <xacro:include filename="$(find ros2srrc_ur5_gazebo)/urdf/cam_on_base_gz.xacro"/>
+  <xacro:if value="${camera}">
+    <xacro:include filename="$(find ros2srrc_ur5_gazebo)/urdf/common_properties.xacro"/>
+    <!-- HAND CAMERA -->
+    <xacro:include filename="$(find ros2srrc_ur5_gazebo)/urdf/cam_on_hand_params_gz.xacro"/>
+    <xacro:property name="parent_hand" value="tool0"/>
+    <xacro:include filename="$(find ros2srrc_ur5_gazebo)/urdf/cam_on_hand_gz.xacro"/>
+    <!-- BASE CAMERA -->
+    <xacro:include filename="$(find ros2srrc_ur5_gazebo)/urdf/cam_on_base_params_gz.xacro"/>
+    <xacro:property name="parent_base" value="base_link"/>
+    <xacro:property name="cam_base_pz" value="0.5"/>
+    <xacro:include filename="$(find ros2srrc_ur5_gazebo)/urdf/cam_on_base_gz.xacro"/>
+  </xacro:if>
   <!-- Include XACRO-MACRO file of the UR3: -->
   <xacro:include filename="$(find ros2srrc_robots)/ur3/urdf/ur3_macro.urdf.xacro"/>

Commit message: Try to fix transformation

File: Industrial/ros2_SimRealRobotControl_gz/packages/ur3/ros2srrc_ur3_gazebo/urdf/ur3_robotiq_2f85.urdf.xacro (robot description, xacro)
@@ -119,5 +119,5 @@
     <parent link= "world" />
     <child link = "robot_stand" />
-    <origin xyz="0.0 0.0 0.5" rpy="0.0 0.0 0.0" />
+    <origin xyz="0.0 0.0 0.0" rpy="0.0 0.0 0.0" />
   </joint>
   <!-- Robot Stand: Robot+Stand JOINT -->
@@ -125,5 +125,5 @@
     <parent link= "robot_stand" />
     <child link = "base_link" />
-    <origin xyz="0.0 0.0 0.505" rpy="0.0 0.0 0.0" />
+    <origin xyz="0.0 0.0 0.0" rpy="0.0 0.0 0.0" />
   </joint>
   <!-- ros2srrc_HMI CAMERA -->

Commit message: Add debug to robpose

File: Industrial/ros2_SimRealRobotControl_gz/packages/ur3/ros2srrc_ur3_gazebo/urdf/ur3_robotiq_2f85.urdf.xacro (robot description, xacro)
@@ -119,5 +119,5 @@
     <parent link= "world" />
     <child link = "robot_stand" />
-    <origin xyz="0.0 0.0 0.0" rpy="0.0 0.0 0.0" />
+    <origin xyz="0.0 0.0 0.5" rpy="0.0 0.0 0.0" />
   </joint>
   <!-- Robot Stand: Robot+Stand JOINT -->
@@ -125,5 +125,5 @@
     <parent link= "robot_stand" />
     <child link = "base_link" />
-    <origin xyz="0.0 0.0 0.0" rpy="0.0 0.0 0.0" />
+    <origin xyz="0.0 0.0 0.505" rpy="0.0 0.0 0.0" />
   </joint>
   <!-- ros2srrc_HMI CAMERA -->
