Commit message: Delete robot stand from xacro

File: Industrial/ros2_SimRealRobotControl_gz/packages/ur3/ros2srrc_ur3_gazebo/urdf/ur3_robotiq_2f85.urdf.xacro (robot description, xacro)
@@ -93,38 +93,4 @@
     </gazebo>
   </xacro:unless>
-  <!-- World: LINK -->
-  <link name="world"/>
-  <!-- Robot Stand: LINK -->
-  <link name='robot_stand'>
-    <inertial>
-      <origin xyz="0 0 0" rpy="0 0 0"/>
-      <mass value="100"/>
-      <inertia ixx="0.01"  ixy="0"  ixz="0" iyy="0.01" iyz="0" izz="0.01" />
-    </inertial>
-    <collision name='collision'>
-      <origin xyz="0 0 0" rpy=" 0 0 0"/>
-      <geometry>
-        <box size = "0.2 0.2 1.0"/>
-      </geometry>
-    </collision>
-    <visual name='chassis_visual'>
-      <origin xyz="0 0 0" rpy=" 0 0 0"/>
-      <geometry>
-        <box size = "0.2 0.2 1.0"/>
-      </geometry>
-    </visual>
-  </link>
-  <!-- Robot Stand: FIXED JOINT -->
-  <joint name="world_joint" type="fixed">
-    <parent link= "world" />
-    <child link = "robot_stand" />
-    <origin xyz="0.0 0.0 0.5" rpy="0.0 0.0 0.0" />
-  </joint>
-  <!-- Robot Stand: Robot+Stand JOINT -->
-  <joint name="stand_joint" type="fixed">
-    <parent link= "robot_stand" />
-    <child link = "base_link" />
-    <origin xyz="0.0 0.0 0.505" rpy="0.0 0.0 0.0" />
-  </joint>
   <!-- ros2srrc_HMI CAMERA -->
   <xacro:if value="${hmi}">
@@ -139,3 +105,10 @@
     />
   </xacro:if>
+  <!-- Fijar el robot al mundo -->
+  <link name="world"/>
+  <joint name="world_joint" type="fixed">
+    <parent link="world"/>
+    <child link="base_link"/>
+    <origin xyz="0 0 0" rpy="0 0 0"/>
+  </joint>
 </robot>
