Commit message: Test new drone launcher

File: CustomRobots/quadrotor/models/quadrotor/quadrotor.urdf.xacro (robot description, xacro)
@@ -3,10 +3,11 @@
   xmlns:xacro="http://ros.org/wiki/xacro">
   <xacro:arg name="camera" default="true"/>
+  <xacro:arg name="namespace" default="dron0"/>
   <xacro:include filename="$(find custom_robots)/models/quadrotor/quadrotor_gz.urdf.xacro"/>
   <xacro:include filename="$(find custom_robots)/models/quadrotor/quadrotor_common.urdf.xacro"/>
-  <xacro:quadrotor/>
+  <xacro:quadrotor namespace="${namespace}"/>
   <xacro:if value="$(arg camera)">
-    <xacro:camera xyz="0 0 0" rpy="0 -1.57 0" mass="0.035" name="frontal_cam" parent="base_link" namespace="drone0"/>
-    <xacro:camera xyz="0 0 0" rpy="0 -1.57 0" mass="0.035" name="ventral_cam" parent="base_link" namespace="drone0"/>
+    <xacro:camera xyz="0 0 0" rpy="0 -1.57 0" mass="0.035" name="frontal_cam" parent="base_link" namespace="${namespace}"/>
+    <xacro:camera xyz="0 0 0" rpy="0 -1.57 0" mass="0.035" name="ventral_cam" parent="base_link" namespace="${namespace}"/>
   </xacro:if>
 </robot>

File: CustomRobots/quadrotor/models/quadrotor/quadrotor_common.urdf.xacro (robot description, xacro)
@@ -2,5 +2,5 @@
 <robot xmlns:xacro="http://ros.org/wiki/xacro">
   <xacro:include filename="$(find custom_robots)/models/quadrotor/quadrotor_gz.urdf.xacro"/>
-  <xacro:macro name="quadrotor">
+  <xacro:macro name="quadrotor" params="namespace">
     <gazebo>
       <include merge="true">
@@ -9,8 +9,8 @@
     </gazebo>
     <xacro:imu/>
-    <xacro:velocity namespace="drone0"/>
+    <xacro:velocity namespace="${namespace}"/>
     <xacro:tf freq="100"/>
-    <xacro:odom topic="/drone0/odom" freq="100"/>
-    <xacro:motors namespace="drone0"/>
+    <xacro:odom topic="/${namespace}/odom" freq="100"/>
+    <xacro:motors namespace="${namespace}"/>
   </xacro:macro>
 </robot>

File: CustomRobots/quadrotor/models/quadrotor/quadrotor_gz.urdf.xacro (robot description, xacro)
@@ -149,6 +149,6 @@
       </plugin>
     </gazebo>
-    <xacro:if value="${rotor}">
-      <xacro:motor rotor="${rotor-1}" />
+    <xacro:if value="${rotor - 1}">
+      <xacro:motor rotor="${rotor-1}" namespace="${namespace}"/>
     </xacro:if>
   </xacro:macro>

Commit message: Fix arg

File: CustomRobots/quadrotor/models/quadrotor/quadrotor.urdf.xacro (robot description, xacro)
@@ -4,4 +4,5 @@
   <xacro:arg name="camera" default="true"/>
   <xacro:arg name="namespace" default="drone0"/>
+  <xacro:property name="namespace" value="$(arg namespace)"/>
   <xacro:include filename="$(find custom_robots)/models/quadrotor/quadrotor_gz.urdf.xacro"/>
   <xacro:include filename="$(find custom_robots)/models/quadrotor/quadrotor_common.urdf.xacro"/>

Commit message: Test adding namespace

File: CustomRobots/quadrotor/models/quadrotor/quadrotor.urdf.xacro (robot description, xacro)
@@ -9,6 +9,6 @@
   <xacro:quadrotor namespace="${namespace}"/>
   <xacro:if value="$(arg camera)">
-    <xacro:camera xyz="0 0 0" rpy="0 -1.57 0" mass="0.035" name="frontal_cam" parent="base_link" namespace="${namespace}"/>
-    <xacro:camera xyz="0 0 0" rpy="0 -1.57 0" mass="0.035" name="ventral_cam" parent="base_link" namespace="${namespace}"/>
+    <xacro:camera xyz="0 0 0" rpy="0 -1.57 0" mass="0.035" name="frontal_cam" parent="${namespace}/base_link" namespace="${namespace}"/>
+    <xacro:camera xyz="0 0 0" rpy="0 -1.57 0" mass="0.035" name="ventral_cam" parent="${namespace}/base_link" namespace="${namespace}"/>
   </xacro:if>
 </robot>

File: CustomRobots/quadrotor/models/quadrotor/quadrotor_common.urdf.xacro (robot description, xacro)
@@ -8,6 +8,6 @@
     <color rgba="0 0 1 1.0"/>
   </material>
-  <xacro:macro name="rotor" params="rotor parent xyz color">
-    <link name='rotor_${rotor}'>
+  <xacro:macro name="rotor" params="rotor parent xyz color namespace">
+    <link name='${namespace}/rotor_${rotor}'>
       <inertial>
         <mass value="0.005"/>
@@ -28,8 +28,8 @@
       <velocity_decay/>
     </link>
-    <joint name='rotor_${rotor}_joint' type="revolute">
+    <joint name='${namespace}/rotor_${rotor}_joint' type="revolute">
       <origin rpy="0 0 0" xyz="${xyz}"/>
-      <parent link="${parent}"/>
-      <child link="rotor_${rotor}"/>
+      <parent link="${namespace}/${parent}"/>
+      <child link="${namespace}/rotor_${rotor}"/>
       <axis xyz="0 0 1" expressed_in="__model__"/>
       <limit lower="-1e+16" upper="1e+16" effort="1000" velocity="100"/>
@@ -38,7 +38,7 @@
   </xacro:macro>
   <xacro:macro name="quadrotor" params="namespace">
-    <link name="base"></link>
+    <link name="${namespace}/base"></link>
     <!-- This is from quadrotor_base from as2 -->
-    <link name="base_link">
+    <link name="${namespace}/base_link">
       <enable_wind>true</enable_wind>
       <inertial>
@@ -51,5 +51,5 @@
         </geometry>
       </collision>
-      <visual name='base_link_inertia_visual'>
+      <visual>
         <geometry>
           <mesh filename="$(find as2_gazebo_assets)/models/quadrotor_base/meshes/quadrotor.dae"/>
@@ -75,14 +75,14 @@
       </visual>
     </link>
-    <joint name="base_to_base_link" type="fixed">
-      <parent link="base"/>
-      <child link="base_link"/>
+    <joint name="${namespace}_base_to_base_link" type="fixed">
+      <parent link="${namespace}/base"/>
+      <child link="${namespace}/base_link"/>
       <origin xyz="0 0 0" rpy="0 0 0"/>
     </joint>
-    <xacro:rotor rotor="0" parent="base_link" xyz="0.13 -0.22 0.023" color="Blue"/>
-    <xacro:rotor rotor="1" parent="base_link" xyz="-0.13 0.2 0.023" color="Red"/>
-    <xacro:rotor rotor="2" parent="base_link" xyz="0.13 0.22 0.023" color="Blue"/>
-    <xacro:rotor rotor="3" parent="base_link" xyz="-0.13 -0.2 0.023" color="Red"/>
-    <xacro:imu mass="0.005" parent="base_link"/>
+    <xacro:rotor rotor="0" parent="base_link" xyz="0.13 -0.22 0.023" color="Blue" namespace="${namespace}"/>
+    <xacro:rotor rotor="1" parent="base_link" xyz="-0.13 0.2 0.023" color="Red" namespace="${namespace}"/>
+    <xacro:rotor rotor="2" parent="base_link" xyz="0.13 0.22 0.023" color="Blue" namespace="${namespace}"/>
+    <xacro:rotor rotor="3" parent="base_link" xyz="-0.13 -0.2 0.023" color="Red" namespace="${namespace}"/>
+    <xacro:imu mass="0.005" parent="${namespace}/base_link"/>
     <xacro:velocity namespace="${namespace}"/>
     <xacro:tf freq="100"/>

File: CustomRobots/quadrotor/models/quadrotor/quadrotor_gz.urdf.xacro (robot description, xacro)
@@ -99,7 +99,7 @@
     <gazebo>
       <plugin filename="gz-sim-odometry-publisher-system" name="gz::sim::systems::OdometryPublisher">
-        <!-- <odom_frame>odom</odom_frame>
+        <odom_frame>odom</odom_frame>
         <robot_base_frame>base</robot_base_frame>
-        <odom_topic>${topic}</odom_topic> -->
+        <odom_topic>${topic}</odom_topic>
         <odom_publish_frequency>${freq}</odom_publish_frequency>
         <dimensions>3</dimensions>
@@ -220,6 +220,6 @@
       <plugin filename="gz-sim-multicopter-motor-model-system" name="gz::sim::systems::MulticopterMotorModel">
         <robotNamespace>model/${namespace}</robotNamespace>
-        <jointName>rotor_${rotor-1}_joint</jointName>
-        <linkName>rotor_${rotor-1}</linkName>
+        <jointName>${namespace}/rotor_${rotor-1}_joint</jointName>
+        <linkName>${namespace}/rotor_${rotor-1}</linkName>
         <xacro:if value="${rotor-1 == 1 or rotor-1 == 0}">
           <turningDirection>ccw</turningDirection>

Commit message: Test with more namespaces

File: CustomRobots/quadrotor/models/quadrotor/quadrotor.urdf.xacro (robot description, xacro)
@@ -9,6 +9,6 @@
   <xacro:quadrotor namespace="${namespace}"/>
   <xacro:if value="$(arg camera)">
-    <xacro:camera xyz="0 0 0" rpy="0 -1.57 0" mass="0.035" name="frontal_cam" parent="${namespace}/base_link" namespace="${namespace}"/>
-    <xacro:camera xyz="0 0 0" rpy="0 -1.57 0" mass="0.035" name="ventral_cam" parent="${namespace}/base_link" namespace="${namespace}"/>
+    <xacro:camera xyz="0 0 0" rpy="0 -1.57 0" mass="0.035" name="frontal_cam" parent="base_link" namespace="${namespace}"/>
+    <xacro:camera xyz="0 0 0" rpy="0 -1.57 0" mass="0.035" name="ventral_cam" parent="base_link" namespace="${namespace}"/>
   </xacro:if>
 </robot>

File: CustomRobots/quadrotor/models/quadrotor/quadrotor_common.urdf.xacro (robot description, xacro)
@@ -75,5 +75,5 @@
       </visual>
     </link>
-    <joint name="${namespace}_base_to_base_link" type="fixed">
+    <joint name="${namespace}/base_to_base_link" type="fixed">
       <parent link="${namespace}/base"/>
       <child link="${namespace}/base_link"/>
@@ -85,7 +85,7 @@
     <xacro:rotor rotor="3" parent="base_link" xyz="-0.13 -0.2 0.023" color="Red" namespace="${namespace}"/>
     <xacro:imu mass="0.005" parent="${namespace}/base_link"/>
-    <xacro:velocity namespace="${namespace}"/>
     <xacro:tf freq="100"/>
     <xacro:odom topic="/${namespace}/odom" freq="100"/>
+    <xacro:velocity namespace="${namespace}"/>
     <xacro:motors namespace="${namespace}"/>
   </xacro:macro>

File: CustomRobots/quadrotor/models/quadrotor/quadrotor_gz.urdf.xacro (robot description, xacro)
@@ -2,5 +2,5 @@
 <robot xmlns:xacro="http://ros.org/wiki/xacro">
   <xacro:macro name="camera" params="xyz rpy name parent mass namespace">
-    <link name="${name}_link">
+    <link name="${namespace}/${name}_link">
       <inertial>
         <origin rpy="${rpy}" xyz="${xyz}"/>
@@ -9,10 +9,10 @@
       </inertial>
     </link>
-    <joint name="${name}_to_${parent}" type="fixed">
-      <parent link="${parent}"/>
-      <child link="${name}_link"/>
+    <joint name="${namespace}/${name}_to_${parent}" type="fixed">
+      <parent link="${namespace}/${parent}"/>
+      <child link="${namespace}/${name}_link"/>
       <origin xyz="${xyz}" rpy="${rpy}"/>
     </joint>
-    <gazebo reference="${name}_link">
+    <gazebo reference="${namespace}/${name}_link">
       <sensor name="${name}" type="camera">
         <always_on>true</always_on>
@@ -49,5 +49,5 @@
         <motorControlPubTopic>command/motor_speed</motorControlPubTopic>
         <enableSubTopic>velocity_controller/enable</enableSubTopic>
-        <comLinkName>base_link</comLinkName>
+        <comLinkName>${namespace}/base_link</comLinkName>
         <velocityGain>2.7 2.7 2.7</velocityGain>
         <attitudeGain>2 3 0.15</attitudeGain>
@@ -107,10 +107,10 @@
     </gazebo>
   </xacro:macro>
-  <xacro:macro name="imu" params="parent mass">
+  <xacro:macro name="imu" params="parent mass namespace">
     <gazebo>
       <plugin filename="gz-sim-imu-system" name="gz::sim::systems::Imu">
       </plugin>
     </gazebo>
-    <link name="imu_link">
+    <link name="${namespace}/imu_link">
       <inertial>
         <mass value="${mass}"/>
@@ -118,9 +118,9 @@
       </inertial>
     </link>
-    <joint name="imu_joint" type="fixed">
-      <parent link="${parent}"/>
-      <child link="imu_link"/>
+    <joint name="${namespace}/imu_joint" type="fixed">
+      <parent link="${namespace}/${parent}"/>
+      <child link="${namespace}/imu_link"/>
     </joint>
-    <gazebo reference="imu_link">
+    <gazebo reference="${namespace}/imu_link">
       <sensor name='imu' type='imu'>
         <always_on>1</always_on>
@@ -234,5 +234,5 @@
         <momentConstant>0.016</momentConstant>
         <commandSubTopic>command/motor_speed</commandSubTopic>
-        <motorNumber>${rotor-1}</motorNumber>
+        <actuator_number>${rotor-1}</actuator_number>
         <rotorDragCoefficient>8.06428e-05</rotorDragCoefficient>
         <rollingMomentCoefficient>1e-06</rollingMomentCoefficient>
