Commit message: drone gripper update (visual for the gripper in xacro), make the gripper plugin aware of the sim reset

File: CustomRobots/quadrotor/models/quadrotor/quadrotor.urdf.xacro (robot description, xacro)
@@ -3,4 +3,5 @@
   xmlns:xacro="http://ros.org/wiki/xacro">
   <xacro:arg name="camera" default="true"/>
+  <xacro:arg name="gripper" default="false"/>
   <xacro:arg name="namespace" default="drone0"/>
   <xacro:property name="namespace" value="$(arg namespace)"/>
@@ -12,3 +13,25 @@
     <xacro:camera xyz="0 0 0" rpy="0 1.57 0" mass="0.035" name="ventral_cam" parent="base_link" namespace="${namespace}"/>
   </xacro:if>
+  <!-- Electromagnet plate: flat disc under the drone (package_delivery). -->
+  <xacro:if value="$(arg gripper)">
+    <link name="magnet">
+      <inertial>
+        <mass value="0.01"/>
+        <inertia ixx="1e-5" ixy="0" ixz="0" iyy="1e-5" iyz="0" izz="1e-5"/>
+      </inertial>
+      <visual>
+        <geometry>
+          <cylinder length="0.02" radius="0.06"/>
+        </geometry>
+        <material name="MagnetBlack">
+          <color rgba="0.05 0.05 0.05 1.0"/>
+        </material>
+      </visual>
+    </link>
+    <joint name="magnet_joint" type="fixed">
+      <origin rpy="0 0 0" xyz="0 0 -0.07"/>
+      <parent link="base_link"/>
+      <child link="magnet"/>
+    </joint>
+  </xacro:if>
 </robot>

Commit message: avoid ventral camera oclusion with magnet

File: CustomRobots/quadrotor/models/quadrotor/quadrotor.urdf.xacro (robot description, xacro)
@@ -8,4 +8,22 @@
   <xacro:include filename="$(find custom_robots)/models/quadrotor/quadrotor_gz.urdf.xacro"/>
   <xacro:include filename="$(find custom_robots)/models/quadrotor/quadrotor_common.urdf.xacro"/>
+  <material name="MagnetBlack">
+    <color rgba="0.05 0.05 0.05 1.0"/>
+  </material>
+  <!-- One box segment of the magnet ring. The ring leaves an open center
+       so it does not block the downward-facing ventral camera. -->
+  <xacro:macro name="magnet_ring_seg" params="i n radius">
+    <xacro:if value="${i &lt; n}">
+      <xacro:property name="ang" value="${2*pi*i/n}"/>
+      <visual name="magnet_seg_${i}">
+        <origin xyz="${radius*cos(ang)} ${radius*sin(ang)} 0" rpy="0 0 ${ang + pi/2}"/>
+        <geometry>
+          <box size="${2*radius*sin(pi/n)} 0.02 0.02"/>
+        </geometry>
+        <material name="MagnetBlack"/>
+      </visual>
+      <xacro:magnet_ring_seg i="${i+1}" n="${n}" radius="${radius}"/>
+    </xacro:if>
+  </xacro:macro>
   <xacro:quadrotor namespace="${namespace}"/>
   <xacro:if value="$(arg camera)">
@@ -13,22 +31,16 @@
     <xacro:camera xyz="0 0 0" rpy="0 1.57 0" mass="0.035" name="ventral_cam" parent="base_link" namespace="${namespace}"/>
   </xacro:if>
-  <!-- Electromagnet plate: flat disc under the drone (package_delivery). -->
+  <!-- Electromagnet: flat ring hugging the drone belly, with an open center
+       so the downward ventral camera is not blocked (package_delivery). -->
   <xacro:if value="$(arg gripper)">
     <link name="magnet">
       <inertial>
-        <mass value="0.01"/>
-        <inertia ixx="1e-5" ixy="0" ixz="0" iyy="1e-5" iyz="0" izz="1e-5"/>
+        <mass value="0.02"/>
+        <inertia ixx="2e-5" ixy="0" ixz="0" iyy="2e-5" iyz="0" izz="4e-5"/>
       </inertial>
-      <visual>
-        <geometry>
-          <cylinder length="0.02" radius="0.06"/>
-        </geometry>
-        <material name="MagnetBlack">
-          <color rgba="0.05 0.05 0.05 1.0"/>
-        </material>
-      </visual>
+      <xacro:magnet_ring_seg i="0" n="12" radius="0.06"/>
     </link>
     <joint name="magnet_joint" type="fixed">
-      <origin rpy="0 0 0" xyz="0 0 -0.07"/>
+      <origin rpy="0 0 0" xyz="0 0 -0.05"/>
       <parent link="base_link"/>
       <child link="magnet"/>

Commit message: Move wrong urdf definitions

File: CustomRobots/quadrotor/models/quadrotor/quadrotor.urdf.xacro (robot description, xacro)
@@ -6,44 +6,11 @@
   <xacro:arg name="namespace" default="drone0"/>
   <xacro:property name="namespace" value="$(arg namespace)"/>
+  <xacro:property name="gripper" value="$(arg gripper)"/>
   <xacro:include filename="$(find custom_robots)/models/quadrotor/quadrotor_gz.urdf.xacro"/>
   <xacro:include filename="$(find custom_robots)/models/quadrotor/quadrotor_common.urdf.xacro"/>
-  <material name="MagnetBlack">
-    <color rgba="0.05 0.05 0.05 1.0"/>
-  </material>
-  <!-- One box segment of the magnet ring. The ring leaves an open center
-       so it does not block the downward-facing ventral camera. -->
-  <xacro:macro name="magnet_ring_seg" params="i n radius">
-    <xacro:if value="${i &lt; n}">
-      <xacro:property name="ang" value="${2*pi*i/n}"/>
-      <visual name="magnet_seg_${i}">
-        <origin xyz="${radius*cos(ang)} ${radius*sin(ang)} 0" rpy="0 0 ${ang + pi/2}"/>
-        <geometry>
-          <box size="${2*radius*sin(pi/n)} 0.02 0.02"/>
-        </geometry>
-        <material name="MagnetBlack"/>
-      </visual>
-      <xacro:magnet_ring_seg i="${i+1}" n="${n}" radius="${radius}"/>
-    </xacro:if>
-  </xacro:macro>
-  <xacro:quadrotor namespace="${namespace}"/>
+  <xacro:quadrotor namespace="${namespace}" gripper="${gripper}"/>
   <xacro:if value="$(arg camera)">
     <xacro:camera xyz="0 0 0" rpy="0 0 0" mass="0.035" name="frontal_cam" parent="base_link" namespace="${namespace}"/>
     <xacro:camera xyz="0 0 0" rpy="0 1.57 0" mass="0.035" name="ventral_cam" parent="base_link" namespace="${namespace}"/>
   </xacro:if>
-  <!-- Electromagnet: flat ring hugging the drone belly, with an open center
-       so the downward ventral camera is not blocked (package_delivery). -->
-  <xacro:if value="$(arg gripper)">
-    <link name="magnet">
-      <inertial>
-        <mass value="0.02"/>
-        <inertia ixx="2e-5" ixy="0" ixz="0" iyy="2e-5" iyz="0" izz="4e-5"/>
-      </inertial>
-      <xacro:magnet_ring_seg i="0" n="12" radius="0.06"/>
-    </link>
-    <joint name="magnet_joint" type="fixed">
-      <origin rpy="0 0 0" xyz="0 0 -0.05"/>
-      <parent link="base_link"/>
-      <child link="magnet"/>
-    </joint>
-  </xacro:if>
 </robot>

Commit message: fix quadrator xacro

File: CustomRobots/quadrotor/models/quadrotor/quadrotor.urdf.xacro (robot description, xacro)
@@ -14,23 +14,8 @@
     <xacro:camera xyz="0 0 0" rpy="0 1.57 0" mass="0.035" name="ventral_cam" parent="base_link" namespace="${namespace}"/>
   </xacro:if>
-<<<<<<< HEAD
-  <!-- Electromagnet: flat ring hugging the drone belly, with an open center
-       so the downward ventral camera is not blocked (package_delivery). -->
+  <!-- Magnetic gripper model plugin. The magnet visual is added by the
+       quadrotor macro (quadrotor_common); this adds the grabbing behavior.
+       The exercise publishes the graspable list on the graspable topic. -->
   <xacro:if value="$(arg gripper)">
-    <link name="magnet">
-      <inertial>
-        <mass value="0.02"/>
-        <inertia ixx="2e-5" ixy="0" ixz="0" iyy="2e-5" iyz="0" izz="4e-5"/>
-      </inertial>
-      <xacro:magnet_ring_seg i="0" n="12" radius="0.06"/>
-    </link>
-    <joint name="magnet_joint" type="fixed">
-      <origin rpy="0 0 0" xyz="0 0 -0.05"/>
-      <parent link="base_link"/>
-      <child link="magnet"/>
-    </joint>
-    <!-- Magnetic gripper: model plugin, so it belongs to this drone (works
-         with renames / several drones). The exercise publishes the graspable
-         list on the graspable topic. -->
     <gazebo>
       <plugin filename="libdrone_gripper.so" name="drone_gripper::DroneGripper">
@@ -43,5 +28,3 @@
     </gazebo>
   </xacro:if>
-=======
->>>>>>> upstream/drone-amazon-delivery
 </robot>

Commit message: electromagnet plugin in macro

File: CustomRobots/quadrotor/models/quadrotor/quadrotor.urdf.xacro (robot description, xacro)
@@ -14,17 +14,3 @@
     <xacro:camera xyz="0 0 0" rpy="0 1.57 0" mass="0.035" name="ventral_cam" parent="base_link" namespace="${namespace}"/>
   </xacro:if>
-  <!-- Magnetic gripper model plugin. The magnet visual is added by the
-       quadrotor macro (quadrotor_common); this adds the grabbing behavior.
-       The exercise publishes the graspable list on the graspable topic. -->
-  <xacro:if value="$(arg gripper)">
-    <gazebo>
-      <plugin filename="libdrone_gripper.so" name="drone_gripper::DroneGripper">
-        <gripper_link>base_link</gripper_link>
-        <attach_distance>0.15</attach_distance>
-        <magnet_topic>/${namespace}/gripper/magnet</magnet_topic>
-        <state_topic>/${namespace}/gripper/attached</state_topic>
-        <graspable_topic>/${namespace}/gripper/graspable</graspable_topic>
-      </plugin>
-    </gazebo>
-  </xacro:if>
 </robot>

File: CustomRobots/quadrotor/models/quadrotor/quadrotor_common.urdf.xacro (robot description, xacro)
@@ -113,4 +113,5 @@
         <child link="magnet"/>
       </joint>
+      <xacro:magnetic_gripper namespace="${namespace}"/>
     </xacro:if>
     <xacro:tf freq="100"/>

File: CustomRobots/quadrotor/models/quadrotor/quadrotor_gz.urdf.xacro (robot description, xacro)
@@ -42,4 +42,17 @@
     </gazebo>
   </xacro:macro>
+  <!-- Magnetic gripper: model plugin driven by ROS2 topics. The magnet visual
+       is added separately; this provides the grabbing behavior. -->
+  <xacro:macro name="magnetic_gripper" params="namespace">
+    <gazebo>
+      <plugin filename="libdrone_gripper.so" name="drone_gripper::DroneGripper">
+        <gripper_link>base_link</gripper_link>
+        <attach_distance>0.15</attach_distance>
+        <magnet_topic>/${namespace}/gripper/magnet</magnet_topic>
+        <state_topic>/${namespace}/gripper/attached</state_topic>
+        <graspable_topic>/${namespace}/gripper/graspable</graspable_topic>
+      </plugin>
+    </gazebo>
+  </xacro:macro>
   <xacro:macro name="velocity" params="namespace">
     <gazebo>

Commit message: Check used values in ros bridge

File: CustomRobots/quadrotor/models/quadrotor/quadrotor.urdf.xacro (robot description, xacro)
@@ -3,5 +3,5 @@
   xmlns:xacro="http://ros.org/wiki/xacro">
   <xacro:arg name="camera" default="true"/>
-  <xacro:arg name="namespace" default="drone0"/>
+  <xacro:arg name="namespace" default="drone"/>
   <xacro:property name="namespace" value="$(arg namespace)"/>
   <xacro:include filename="$(find custom_robots)/models/quadrotor/quadrotor_gz.urdf.xacro"/>

File: CustomRobots/quadrotor/models/quadrotor/quadrotor_common.urdf.xacro (robot description, xacro)
@@ -8,5 +8,5 @@
     <color rgba="0 0 1 1.0"/>
   </material>
-  <xacro:macro name="rotor" params="rotor parent xyz color namespace">
+  <xacro:macro name="rotor" params="rotor parent xyz color">
     <link name='rotor_${rotor}'>
       <inertial>
@@ -76,11 +76,11 @@
       </visual>
     </link>
-    <xacro:rotor rotor="0" parent="base_link" xyz="0.13 -0.22 0.023" color="Blue" namespace="${namespace}"/>
-    <xacro:rotor rotor="1" parent="base_link" xyz="-0.13 0.2 0.023" color="Red" namespace="${namespace}"/>
-    <xacro:rotor rotor="2" parent="base_link" xyz="0.13 0.22 0.023" color="Blue" namespace="${namespace}"/>
-    <xacro:rotor rotor="3" parent="base_link" xyz="-0.13 -0.2 0.023" color="Red" namespace="${namespace}"/>
+    <xacro:rotor rotor="0" parent="base_link" xyz="0.13 -0.22 0.023" color="Blue"/>
+    <xacro:rotor rotor="1" parent="base_link" xyz="-0.13 0.2 0.023" color="Red"/>
+    <xacro:rotor rotor="2" parent="base_link" xyz="0.13 0.22 0.023" color="Blue"/>
+    <xacro:rotor rotor="3" parent="base_link" xyz="-0.13 -0.2 0.023" color="Red"/>
     <xacro:tf freq="100"/>
     <xacro:imu mass="0.005" parent="base_link" namespace="${namespace}"/>
-    <xacro:odom topic="odom" freq="100" namespace="${namespace}"/>
+    <xacro:odom freq="100" namespace="${namespace}"/>
     <xacro:motors namespace="${namespace}"/>
     <xacro:velocity namespace="${namespace}"/>

File: CustomRobots/quadrotor/models/quadrotor/quadrotor_gz.urdf.xacro (robot description, xacro)
@@ -96,10 +96,10 @@
     </gazebo>
   </xacro:macro>
-  <xacro:macro name="odom" params="topic freq namespace">
+  <xacro:macro name="odom" params="freq namespace">
     <gazebo>
       <plugin filename="gz-sim-odometry-publisher-system" name="gz::sim::systems::OdometryPublisher">
         <!-- <odom_frame>odom</odom_frame>
         <robot_base_frame>base_link</robot_base_frame>
-        <odom_topic>${topic}</odom_topic> -->
+        <odom_topic>/${namespace}/odom</odom_topic> -->
         <odom_publish_frequency>${freq}</odom_publish_frequency>
         <dimensions>3</dimensions>

Commit message: Rebase

File: CustomRobots/quadrotor/models/quadrotor/quadrotor.urdf.xacro (robot description, xacro)
@@ -5,4 +5,5 @@
   <xacro:arg name="gripper" default="false"/>
   <xacro:arg name="namespace" default="drone"/>
+  <xacro:arg name="gripper" default="false"/>
   <xacro:property name="namespace" value="$(arg namespace)"/>
   <xacro:property name="gripper" value="$(arg gripper)"/>
@@ -14,3 +15,25 @@
     <xacro:camera xyz="0 0 0" rpy="0 1.57 0" mass="0.035" name="ventral_cam" parent="base_link" namespace="${namespace}"/>
   </xacro:if>
+  <!-- Electromagnet plate: flat disc under the drone (package_delivery). -->
+  <xacro:if value="$(arg gripper)">
+    <link name="magnet">
+      <inertial>
+        <mass value="0.01"/>
+        <inertia ixx="1e-5" ixy="0" ixz="0" iyy="1e-5" iyz="0" izz="1e-5"/>
+      </inertial>
+      <visual>
+        <geometry>
+          <cylinder length="0.02" radius="0.06"/>
+        </geometry>
+        <material name="MagnetBlack">
+          <color rgba="0.05 0.05 0.05 1.0"/>
+        </material>
+      </visual>
+    </link>
+    <joint name="magnet_joint" type="fixed">
+      <origin rpy="0 0 0" xyz="0 0 -0.07"/>
+      <parent link="base_link"/>
+      <child link="magnet"/>
+    </joint>
+  </xacro:if>
 </robot>

Commit message: Fix quadrotor

File: CustomRobots/quadrotor/models/quadrotor/quadrotor.urdf.xacro (robot description, xacro)
@@ -15,37 +15,3 @@
     <xacro:camera xyz="0 0 0" rpy="0 1.57 0" mass="0.035" name="ventral_cam" parent="base_link" namespace="${namespace}"/>
   </xacro:if>
-  <!-- Electromagnet plate: flat disc under the drone (package_delivery). -->
-  <xacro:if value="$(arg gripper)">
-    <link name="magnet">
-      <inertial>
-        <mass value="0.01"/>
-        <inertia ixx="1e-5" ixy="0" ixz="0" iyy="1e-5" iyz="0" izz="1e-5"/>
-      </inertial>
-      <visual>
-        <geometry>
-          <cylinder length="0.02" radius="0.06"/>
-        </geometry>
-        <material name="MagnetBlack">
-          <color rgba="0.05 0.05 0.05 1.0"/>
-        </material>
-      </visual>
-    </link>
-    <joint name="magnet_joint" type="fixed">
-      <origin rpy="0 0 0" xyz="0 0 -0.07"/>
-      <parent link="base_link"/>
-      <child link="magnet"/>
-    </joint>
-    <!-- Magnetic gripper: model plugin, so it belongs to this drone (works
-         with renames / several drones). The exercise publishes the graspable
-         list on the graspable topic. -->
-    <gazebo>
-      <plugin filename="libdrone_gripper.so" name="drone_gripper::DroneGripper">
-        <gripper_link>base_link</gripper_link>
-        <attach_distance>0.15</attach_distance>
-        <magnet_topic>/${namespace}/gripper/magnet</magnet_topic>
-        <state_topic>/${namespace}/gripper/attached</state_topic>
-        <graspable_topic>/${namespace}/gripper/graspable</graspable_topic>
-      </plugin>
-    </gazebo>
-  </xacro:if>
 </robot>

Commit message: solving color issue

File: CustomRobots/quadrotor/models/quadrotor/quadrotor.urdf.xacro (robot description, xacro)
@@ -5,7 +5,9 @@
   <xacro:arg name="namespace" default="drone"/>
   <xacro:property name="namespace" value="$(arg namespace)"/>
+  <xacro:arg name="color" default="Blue"/>
+  <xacro:property name="color" value="$(arg color)"/>
   <xacro:include filename="$(find custom_robots)/models/quadrotor/quadrotor_gz.urdf.xacro"/>
   <xacro:include filename="$(find custom_robots)/models/quadrotor/quadrotor_common.urdf.xacro"/>
-  <xacro:quadrotor namespace="${namespace}"/>
+  <xacro:quadrotor namespace="${namespace}" color="${color}"/>
   <xacro:if value="$(arg camera)">
     <xacro:camera xyz="0 0 0" rpy="0 0 0" mass="0.035" name="frontal_cam" parent="base_link" namespace="${namespace}"/>

File: CustomRobots/quadrotor/models/quadrotor/quadrotor_common.urdf.xacro (robot description, xacro)
@@ -7,4 +7,16 @@
   <material name="Blue">
     <color rgba="0 0 1 1.0"/>
+  </material>
+  <material name="Green">
+    <color rgba="0 0.8 0 1.0"/>
+  </material>
+  <material name="Yellow">
+    <color rgba="1 0.9 0 1.0"/>
+  </material>
+  <material name="Orange">
+    <color rgba="1 0.5 0 1.0"/>
+  </material>
+  <material name="White">
+    <color rgba="1 1 1 1.0"/>
   </material>
   <xacro:macro name="rotor" params="rotor parent xyz color">
@@ -37,5 +49,5 @@
     </joint>
   </xacro:macro>
-  <xacro:macro name="quadrotor" params="namespace">
+  <xacro:macro name="quadrotor" params="namespace color:='Blue'">
     <!-- This is from quadrotor_base from as2 -->
     <link name="base_link">
@@ -56,4 +68,5 @@
           <mesh filename="$(find as2_gazebo_assets)/models/quadrotor_base/meshes/quadrotor.dae"/>
         </geometry>
+        <material name="${color}"/>
       </visual>
       <visual name='marker_visual_1'>

Commit message: changed default color to blue

File: CustomRobots/quadrotor/models/quadrotor/quadrotor.urdf.xacro (robot description, xacro)
@@ -5,5 +5,5 @@
   <xacro:arg name="namespace" default="drone"/>
   <xacro:property name="namespace" value="$(arg namespace)"/>
-  <xacro:arg name="color" default="Blue"/>
+  <xacro:arg name="color" default="Orange"/>
   <xacro:property name="color" value="$(arg color)"/>
   <xacro:include filename="$(find custom_robots)/models/quadrotor/quadrotor_gz.urdf.xacro"/>

File: CustomRobots/quadrotor/models/quadrotor/quadrotor_common.urdf.xacro (robot description, xacro)
@@ -49,6 +49,5 @@
     </joint>
   </xacro:macro>
-  <xacro:macro name="quadrotor" params="namespace color:='Blue'">
-    <!-- This is from quadrotor_base from as2 -->
+  <xacro:macro name="quadrotor" params="namespace color:='Orange'">
     <link name="base_link">
       <gazebo>

Commit message: changed color and tested things locally also

File: CustomRobots/quadrotor/models/quadrotor/quadrotor.urdf.xacro (robot description, xacro)
@@ -5,5 +5,5 @@
   <xacro:arg name="namespace" default="drone"/>
   <xacro:property name="namespace" value="$(arg namespace)"/>
-  <xacro:arg name="color" default="Orange"/>
+  <xacro:arg name="color" default=""/>
   <xacro:property name="color" value="$(arg color)"/>
   <xacro:include filename="$(find custom_robots)/models/quadrotor/quadrotor_gz.urdf.xacro"/>

File: CustomRobots/quadrotor/models/quadrotor/quadrotor_common.urdf.xacro (robot description, xacro)
@@ -19,4 +19,7 @@
   <material name="White">
     <color rgba="1 1 1 1.0"/>
+  </material>
+  <material name="Magenta">
+    <color rgba="1 0 1 1.0"/>
   </material>
   <xacro:macro name="rotor" params="rotor parent xyz color">
@@ -49,5 +52,6 @@
     </joint>
   </xacro:macro>
-  <xacro:macro name="quadrotor" params="namespace color:='Orange'">
+  <xacro:macro name="quadrotor" params="namespace color:=''">
+    <!-- This is from quadrotor_base from as2 -->
     <link name="base_link">
       <gazebo>
@@ -67,5 +71,7 @@
           <mesh filename="$(find as2_gazebo_assets)/models/quadrotor_base/meshes/quadrotor.dae"/>
         </geometry>
-        <material name="${color}"/>
+        <xacro:if value="${color != ''}">
+          <material name="${color}"/>
+        </xacro:if>
       </visual>
       <visual name='marker_visual_1'>
