Commit message: TEst updated model

File: CustomRobots/quadrotor/models/quadrotor/quadrotor_common.urdf.xacro (robot description, xacro)
@@ -2,11 +2,84 @@
 <robot xmlns:xacro="http://ros.org/wiki/xacro">
   <xacro:include filename="$(find custom_robots)/models/quadrotor/quadrotor_gz.urdf.xacro"/>
+  <xacro:macro name="rotor" params="rotor parent xyz color">
+    <link name='rotor_${rotor}'>
+      <!-- <pose>0.13 -0.22 0.023 0 -0 0</pose> -->
+      <inertial>
+        <mass value="0.005"/>
+        <inertia ixx="9.75e-07" ixy="0" ixz="0" iyy="4.17041e-05" iyz="0" izz="4.26041e-05"/>
+      </inertial>
+      <collision name='rotor_${rotor}_collision'>
+        <geometry>
+          <cylinder length="0.005" radius="0.1"/>
+        </geometry>
+      </collision>
+      <visual name='rotor_${rotor}_visual'>
+        <geometry>
+          <mesh filename="$(find as2_gazebo_assets)/quadrotor_base/meshes/propeller_ccw.dae" scale="0.1 0.1 0.1"/>
+        </geometry>
+        <gazebo>
+          <material>
+            <diffuse>0 0 1 1</diffuse>
+            <script>
+              <name>Gazebo/${color}</name>
+            </script>
+          </material>
+        </gazebo>
+      </visual>
+      <gravity>1</gravity>
+      <velocity_decay/>
+    </link>
+    <joint name='rotor_${rotor}_joint' type="revolute">
+      <origin rpy="0 0 0" xyz="${xyz}"/>
+      <parent link="${parent}"/>
+      <child link="rotor_${rotor}"/>
+      <axis xyz="0 0 1" expressed_in="__model__"/>
+      <limit lower="-1e+16" upper="1e+16"/>
+      <dynamics spring_reference="0" spring_stiffness="0"/>
+    </joint>
+  </xacro:macro>
   <xacro:macro name="quadrotor" params="namespace">
-    <gazebo>
-      <include merge="true">
-        <uri>model://quadrotor_base</uri>
-      </include>
-    </gazebo>
-    <xacro:imu/>
+    <!-- This is from quadrotor_base from as2 -->
+    <!-- <pose>0 0 0.053302 0 0 0</pose> -->
+    <link name="base_link">
+      <enable_wind>true</enable_wind>
+      <inertial>
+        <mass value="1.5"/>
+        <inertia ixx="0.025" ixy="0" ixz="0" iyy="0.009" iyz="0" izz="0.033"/>
+      </inertial>
+      <collision>
+        <geometry>
+          <box size="0.47 0.47 0.11"/>
+        </geometry>
+      </collision>
+      <visual name='base_link_inertia_visual'>
+        <geometry>
+          <mesh filename="$(find as2_gazebo_assets)/quadrotor_base/meshes/quadrotor.dae"/>
+        </geometry>
+      </visual>
+      <visual name='marker_visual_1'>
+        <origin rpy="0 0 0" xyz="-0.07 0 0.065"/>
+        <geometry>
+          <mesh filename="$(find as2_gazebo_assets)/quadrotor_base/meshes/led.dae"/>
+        </geometry>
+      </visual>
+      <visual name='marker_visual_2'>
+        <origin rpy="-1.0472 -0 0.2" xyz="-0.08 0.037 0.04"/>
+        <geometry>
+          <mesh filename="$(find as2_gazebo_assets)/quadrotor_base/meshes/led.dae"/>
+        </geometry>
+      </visual>
+      <visual name='marker_visual_3'>
+        <origin rpy="1.0472 -0 -0.1" xyz="-0.08 -0.035 0.04"/>
+        <geometry>
+          <mesh filename="$(find as2_gazebo_assets)/quadrotor_base/meshes/led.dae"/>
+        </geometry>
+      </visual>
+    </link>
+    <xacro:rotor rotor="0" parent="base_link" xyz="0.13 -0.22 0.023" color="Blue"/>
+    <xacro:rotor rotor="1" parent="base_link" xyz="-0.13 0.2 0.023" color="Red"/>
+    <xacro:rotor rotor="2" parent="base_link" xyz="0.13 0.22 0.023" color="Blue"/>
+    <xacro:rotor rotor="3" parent="base_link" xyz="-0.13 -0.2 0.023" color="Red"/>
+    <xacro:imu mass="0.005" parent="base_link"/>
     <xacro:velocity namespace="${namespace}"/>
     <xacro:tf freq="100"/>

File: CustomRobots/quadrotor/models/quadrotor/quadrotor_gz.urdf.xacro (robot description, xacro)
@@ -107,8 +107,96 @@
     </gazebo>
   </xacro:macro>
-  <xacro:macro name="imu">
+  <xacro:macro name="imu" params="parent mass">
     <gazebo>
       <plugin filename="gz-sim-imu-system" name="gz::sim::systems::Imu">
       </plugin>
+    </gazebo>
+    <link name="imu_link">
+      <inertial>
+        <mass value="${mass}"/>
+        <inertia ixx="8.33e-06" ixy="0" ixz="0" iyy="8.33e-06" iyz="0" izz="8.33e-06"/>
+      </inertial>
+    </link>
+    <joint name="imu_joint" type="fixed">
+      <parent link="${parent}"/>
+      <child link="imu_link"/>
+    </joint>
+    <gazebo reference="imu_link">
+      <sensor name='imu' type='imu'>
+        <always_on>1</always_on>
+        <update_rate>250</update_rate>
+        <imu>
+          <angular_velocity>
+            <x>
+              <noise type='gaussian'>
+                <mean>0</mean>
+                <stddev>0.009</stddev>
+                <bias_mean>0.00075</bias_mean>
+                <bias_stddev>0.005</bias_stddev>
+                <dynamic_bias_stddev>0.00002</dynamic_bias_stddev>
+                <dynamic_bias_correlation_time>400.0</dynamic_bias_correlation_time>
+                <precision>0.00025</precision>
+              </noise>
+            </x>
+            <y>
+              <noise type='gaussian'>
+                <mean>0</mean>
+                <stddev>0.009</stddev>
+                <bias_mean>0.00075</bias_mean>
+                <bias_stddev>0.005</bias_stddev>
+                <dynamic_bias_stddev>0.00002</dynamic_bias_stddev>
+                <dynamic_bias_correlation_time>400.0</dynamic_bias_correlation_time>
+                <precision>0.00025</precision>
+              </noise>
+            </y>
+            <z>
+              <noise type='gaussian'>
+                <mean>0</mean>
+                <stddev>0.009</stddev>
+                <bias_mean>0.00075</bias_mean>
+                <bias_stddev>0.005</bias_stddev>
+                <dynamic_bias_stddev>0.00002</dynamic_bias_stddev>
+                <dynamic_bias_correlation_time>400.0</dynamic_bias_correlation_time>
+                <precision>0.00025</precision>
+              </noise>
+            </z>
+          </angular_velocity>
+          <linear_acceleration>
+            <x>
+              <noise type='gaussian'>
+                <mean>0</mean>
+                <stddev>0.021</stddev>
+                <bias_mean>0.05</bias_mean>
+                <bias_stddev>0.0075</bias_stddev>
+                <dynamic_bias_stddev>0.000375</dynamic_bias_stddev>
+                <dynamic_bias_correlation_time>175.0</dynamic_bias_correlation_time>
+                <precision>0.005</precision>
+              </noise>
+            </x>
+            <y>
+              <noise type='gaussian'>
+                <mean>0</mean>
+                <stddev>0.021</stddev>
+                <bias_mean>0.05</bias_mean>
+                <bias_stddev>0.0075</bias_stddev>
+                <dynamic_bias_stddev>0.000375</dynamic_bias_stddev>
+                <dynamic_bias_correlation_time>175.0</dynamic_bias_correlation_time>
+                <precision>0.005</precision>
+              </noise>
+            </y>
+            <z>
+              <noise type='gaussian'>
+                <mean>0</mean>
+                <stddev>0.021</stddev>
+                <bias_mean>0.05</bias_mean>
+                <bias_stddev>0.0075</bias_stddev>
+                <dynamic_bias_stddev>0.000375</dynamic_bias_stddev>
+                <dynamic_bias_correlation_time>175.0</dynamic_bias_correlation_time>
+                <precision>0.005</precision>
+              </noise>
+            </z>
+          </linear_acceleration>
+        </imu>
+      </sensor>
     </gazebo>
   </xacro:macro>

Commit message: Update launcher

File: CustomRobots/quadrotor/models/quadrotor/quadrotor_common.urdf.xacro (robot description, xacro)
@@ -4,5 +4,4 @@
   <xacro:macro name="rotor" params="rotor parent xyz color">
     <link name='rotor_${rotor}'>
-      <!-- <pose>0.13 -0.22 0.023 0 -0 0</pose> -->
       <inertial>
         <mass value="0.005"/>
@@ -35,6 +34,6 @@
       <child link="rotor_${rotor}"/>
       <axis xyz="0 0 1" expressed_in="__model__"/>
-      <limit lower="-1e+16" upper="1e+16"/>
-      <dynamics spring_reference="0" spring_stiffness="0"/>
+      <limit lower="-1e+16" upper="1e+16" effort="1000" velocity="100"/>
+      <dynamics spring_reference="0" spring_stiffness="0" friction="0" damping="0"/>
     </joint>
   </xacro:macro>

Commit message: Update meshes

File: CustomRobots/quadrotor/models/quadrotor/quadrotor_common.urdf.xacro (robot description, xacro)
@@ -15,5 +15,5 @@
       <visual name='rotor_${rotor}_visual'>
         <geometry>
-          <mesh filename="$(find as2_gazebo_assets)/quadrotor_base/meshes/propeller_ccw.dae" scale="0.1 0.1 0.1"/>
+          <mesh filename="$(find as2_gazebo_assets)/models/quadrotor_base/meshes/propeller_ccw.dae" scale="0.1 0.1 0.1"/>
         </geometry>
         <gazebo>
@@ -39,6 +39,6 @@
   </xacro:macro>
   <xacro:macro name="quadrotor" params="namespace">
+    <link name="base"></link>
     <!-- This is from quadrotor_base from as2 -->
-    <!-- <pose>0 0 0.053302 0 0 0</pose> -->
     <link name="base_link">
       <enable_wind>true</enable_wind>
@@ -54,5 +54,5 @@
       <visual name='base_link_inertia_visual'>
         <geometry>
-          <mesh filename="$(find as2_gazebo_assets)/quadrotor_base/meshes/quadrotor.dae"/>
+          <mesh filename="$(find as2_gazebo_assets)/models/quadrotor_base/meshes/quadrotor.dae"/>
         </geometry>
       </visual>
@@ -60,5 +60,5 @@
         <origin rpy="0 0 0" xyz="-0.07 0 0.065"/>
         <geometry>
-          <mesh filename="$(find as2_gazebo_assets)/quadrotor_base/meshes/led.dae"/>
+          <mesh filename="$(find as2_gazebo_assets)/models/quadrotor_base/meshes/led.dae"/>
         </geometry>
       </visual>
@@ -66,5 +66,5 @@
         <origin rpy="-1.0472 -0 0.2" xyz="-0.08 0.037 0.04"/>
         <geometry>
-          <mesh filename="$(find as2_gazebo_assets)/quadrotor_base/meshes/led.dae"/>
+          <mesh filename="$(find as2_gazebo_assets)/models/quadrotor_base/meshes/led.dae"/>
         </geometry>
       </visual>
@@ -72,8 +72,13 @@
         <origin rpy="1.0472 -0 -0.1" xyz="-0.08 -0.035 0.04"/>
         <geometry>
-          <mesh filename="$(find as2_gazebo_assets)/quadrotor_base/meshes/led.dae"/>
+          <mesh filename="$(find as2_gazebo_assets)/models/quadrotor_base/meshes/led.dae"/>
         </geometry>
       </visual>
     </link>
+    <joint name="base_to_base_link" type="fixed">
+      <parent link="base"/>
+      <child link="base_link"/>
+      <origin xyz="0 0 0.053302" rpy="0 0 0"/>
+    </joint>
     <xacro:rotor rotor="0" parent="base_link" xyz="0.13 -0.22 0.023" color="Blue"/>
     <xacro:rotor rotor="1" parent="base_link" xyz="-0.13 0.2 0.023" color="Red"/>

Commit message: TEst again

File: CustomRobots/quadrotor/models/quadrotor/quadrotor_common.urdf.xacro (robot description, xacro)
@@ -79,5 +79,5 @@
       <parent link="base"/>
       <child link="base_link"/>
-      <origin xyz="0 0 0.053302" rpy="0 0 0"/>
+      <origin xyz="0 0 0" rpy="0 0 0"/>
     </joint>
     <xacro:rotor rotor="0" parent="base_link" xyz="0.13 -0.22 0.023" color="Blue"/>

Commit message: Test again

File: CustomRobots/quadrotor/models/quadrotor/quadrotor_common.urdf.xacro (robot description, xacro)
@@ -2,4 +2,10 @@
 <robot xmlns:xacro="http://ros.org/wiki/xacro">
   <xacro:include filename="$(find custom_robots)/models/quadrotor/quadrotor_gz.urdf.xacro"/>
+  <material name="Red">
+    <color rgba="1 0 0 1.0"/>
+  </material>
+  <material name="Blue">
+    <color rgba="0 0 1 1.0"/>
+  </material>
   <xacro:macro name="rotor" params="rotor parent xyz color">
     <link name='rotor_${rotor}'>
@@ -17,10 +23,5 @@
           <mesh filename="$(find as2_gazebo_assets)/models/quadrotor_base/meshes/propeller_ccw.dae" scale="0.1 0.1 0.1"/>
         </geometry>
-        <gazebo>
-          <material>
-            <diffuse>${color} 1</diffuse>
-            <specular>0 0 0 1</specular>
-          </material>
-        </gazebo>
+        <material name="${color}"/>
       </visual>
       <gravity>1</gravity>
@@ -79,8 +80,8 @@
       <origin xyz="0 0 0" rpy="0 0 0"/>
     </joint>
-    <xacro:rotor rotor="0" parent="base_link" xyz="0.13 -0.22 0.023" color="0 0 1"/>
-    <xacro:rotor rotor="1" parent="base_link" xyz="-0.13 0.2 0.023" color="1 0 0"/>
-    <xacro:rotor rotor="2" parent="base_link" xyz="0.13 0.22 0.023" color="0 0 1"/>
-    <xacro:rotor rotor="3" parent="base_link" xyz="-0.13 -0.2 0.023" color="1 0 0"/>
+    <xacro:rotor rotor="0" parent="base_link" xyz="0.13 -0.22 0.023" color="Blue"/>
+    <xacro:rotor rotor="1" parent="base_link" xyz="-0.13 0.2 0.023" color="Red"/>
+    <xacro:rotor rotor="2" parent="base_link" xyz="0.13 0.22 0.023" color="Blue"/>
+    <xacro:rotor rotor="3" parent="base_link" xyz="-0.13 -0.2 0.023" color="Red"/>
     <xacro:imu mass="0.005" parent="base_link"/>
     <xacro:velocity namespace="${namespace}"/>

Commit message: Test again

File: CustomRobots/quadrotor/models/quadrotor/quadrotor_common.urdf.xacro (robot description, xacro)
@@ -14,10 +14,10 @@
         <inertia ixx="9.75e-07" ixy="0" ixz="0" iyy="4.17041e-05" iyz="0" izz="4.26041e-05"/>
       </inertial>
-      <collision name='rotor_${rotor}_collision'>
+      <collision>
         <geometry>
           <cylinder length="0.005" radius="0.1"/>
         </geometry>
       </collision>
-      <visual name='rotor_${rotor}_visual'>
+      <visual>
         <geometry>
           <mesh filename="$(find as2_gazebo_assets)/models/quadrotor_base/meshes/propeller_ccw.dae" scale="0.1 0.1 0.1"/>
@@ -84,8 +84,8 @@
     <xacro:rotor rotor="2" parent="base_link" xyz="0.13 0.22 0.023" color="Blue" namespace="${namespace}"/>
     <xacro:rotor rotor="3" parent="base_link" xyz="-0.13 -0.2 0.023" color="Red" namespace="${namespace}"/>
+    <xacro:velocity namespace="${namespace}"/>
     <xacro:imu mass="0.005" parent="${namespace}/base_link"/>
     <xacro:tf freq="100"/>
     <xacro:odom topic="/${namespace}/odom" freq="100"/>
-    <xacro:velocity namespace="${namespace}"/>
     <xacro:motors namespace="${namespace}"/>
   </xacro:macro>

Commit message: More tests

File: CustomRobots/quadrotor/models/quadrotor/quadrotor_common.urdf.xacro (robot description, xacro)
@@ -87,5 +87,5 @@
     <xacro:imu mass="0.005" parent="base_link" namespace="${namespace}"/>
     <xacro:tf freq="100"/>
-    <xacro:odom topic="/${namespace}/odom" freq="100"/>
+    <xacro:odom topic="odom" freq="100" namespace="${namespace}"/>
     <xacro:motors namespace="${namespace}"/>
   </xacro:macro>

File: CustomRobots/quadrotor/models/quadrotor/quadrotor_gz.urdf.xacro (robot description, xacro)
@@ -69,5 +69,5 @@
         <rotorConfiguration>
           <rotor>
-            <jointName>rotor_0_joint</jointName>
+            <jointName>${namespace}/rotor_0_joint</jointName>
             <forceConstant>8.54858e-06</forceConstant>
             <momentConstant>0.016</momentConstant>
@@ -75,5 +75,5 @@
           </rotor>
           <rotor>
-            <jointName>rotor_1_joint</jointName>
+            <jointName>${namespace}/rotor_1_joint</jointName>
             <forceConstant>8.54858e-06</forceConstant>
             <momentConstant>0.016</momentConstant>
@@ -81,5 +81,5 @@
           </rotor>
           <rotor>
-            <jointName>rotor_2_joint</jointName>
+            <jointName>${namespace}/rotor_2_joint</jointName>
             <forceConstant>8.54858e-06</forceConstant>
             <momentConstant>0.016</momentConstant>
@@ -87,5 +87,5 @@
           </rotor>
           <rotor>
-            <jointName>rotor_3_joint</jointName>
+            <jointName>${namespace}/rotor_3_joint</jointName>
             <forceConstant>8.54858e-06</forceConstant>
             <momentConstant>0.016</momentConstant>
@@ -96,10 +96,10 @@
     </gazebo>
   </xacro:macro>
-  <xacro:macro name="odom" params="topic freq">
+  <xacro:macro name="odom" params="topic freq namespace">
     <gazebo>
       <plugin filename="gz-sim-odometry-publisher-system" name="gz::sim::systems::OdometryPublisher">
-        <odom_frame>odom</odom_frame>
-        <robot_base_frame>base</robot_base_frame>
-        <odom_topic>${topic}</odom_topic>
+        <odom_frame>${namespace}/odom</odom_frame>
+        <robot_base_frame>${namespace}/base_link</robot_base_frame>
+        <odom_topic>${namespace}/${topic}</odom_topic>
         <odom_publish_frequency>${freq}</odom_publish_frequency>
         <dimensions>3</dimensions>

Commit message: Test joint

File: CustomRobots/quadrotor/models/quadrotor/quadrotor_common.urdf.xacro (robot description, xacro)
@@ -41,5 +41,7 @@
     <!-- This is from quadrotor_base from as2 -->
     <link name="${namespace}/base_link">
-      <enable_wind>true</enable_wind>
+      <gazebo>
+        <enable_wind>true</enable_wind>
+      </gazebo>
       <inertial>
         <mass value="1.5"/>
@@ -80,11 +82,38 @@
       <origin xyz="0 0 0" rpy="0 0 0"/>
     </joint>
-    <xacro:rotor rotor="0" parent="base_link" xyz="0.13 -0.22 0.023" color="Blue" namespace="${namespace}"/>
+    <!-- <xacro:rotor rotor="0" parent="base_link" xyz="0.13 -0.22 0.023" color="Blue" namespace="${namespace}"/> -->
     <xacro:rotor rotor="1" parent="base_link" xyz="-0.13 0.2 0.023" color="Red" namespace="${namespace}"/>
     <xacro:rotor rotor="2" parent="base_link" xyz="0.13 0.22 0.023" color="Blue" namespace="${namespace}"/>
     <xacro:rotor rotor="3" parent="base_link" xyz="-0.13 -0.2 0.023" color="Red" namespace="${namespace}"/>
+    <link name='${namespace}/rotor_0'>
+      <inertial>
+        <mass value="0.005"/>
+        <inertia ixx="9.75e-07" ixy="0" ixz="0" iyy="4.17041e-05" iyz="0" izz="4.26041e-05"/>
+      </inertial>
+      <collision>
+        <geometry>
+          <cylinder length="0.005" radius="0.1"/>
+        </geometry>
+      </collision>
+      <visual>
+        <geometry>
+          <mesh filename="$(find as2_gazebo_assets)/models/quadrotor_base/meshes/propeller_ccw.dae" scale="0.1 0.1 0.1"/>
+        </geometry>
+        <material name="Blue"/>
+      </visual>
+      <gravity>1</gravity>
+      <velocity_decay/>
+    </link>
+    <joint name='${namespace}/rotor_0_joint' type="revolute">
+      <origin rpy="0 0 0" xyz="${xyz}"/>
+      <parent link="${namespace}/${parent}"/>
+      <child link="${namespace}/rotor_0"/>
+      <axis xyz="0 0 1" expressed_in="__model__"/>
+      <limit lower="-1e+16" upper="1e+16" effort="1000" velocity="100"/>
+      <dynamics spring_reference="0" spring_stiffness="0" friction="0" damping="0"/>
+    </joint>
+    <xacro:tf freq="100"/>
     <xacro:velocity namespace="${namespace}"/>
     <xacro:imu mass="0.005" parent="base_link" namespace="${namespace}"/>
-    <xacro:tf freq="100"/>
     <xacro:odom topic="odom" freq="100" namespace="${namespace}"/>
     <xacro:motors namespace="${namespace}"/>

Commit message: Fix test

File: CustomRobots/quadrotor/models/quadrotor/quadrotor_common.urdf.xacro (robot description, xacro)
@@ -106,6 +106,6 @@
     </link>
     <joint name='${namespace}/rotor_0_joint' type="revolute">
-      <origin rpy="0 0 0" xyz="${xyz}"/>
-      <parent link="${namespace}/${parent}"/>
+      <origin rpy="0 0 0" xyz="0.13 -0.22 0.023"/>
+      <parent link="${namespace}/base_link"/>
       <child link="${namespace}/rotor_0"/>
       <axis xyz="0 0 1" expressed_in="__model__"/>

Commit message: And again

File: CustomRobots/quadrotor/models/quadrotor/quadrotor_common.urdf.xacro (robot description, xacro)
@@ -82,40 +82,13 @@
       <origin xyz="0 0 0" rpy="0 0 0"/>
     </joint>
-    <!-- <xacro:rotor rotor="0" parent="base_link" xyz="0.13 -0.22 0.023" color="Blue" namespace="${namespace}"/> -->
+    <xacro:rotor rotor="0" parent="base_link" xyz="0.13 -0.22 0.023" color="Blue" namespace="${namespace}"/>
     <xacro:rotor rotor="1" parent="base_link" xyz="-0.13 0.2 0.023" color="Red" namespace="${namespace}"/>
     <xacro:rotor rotor="2" parent="base_link" xyz="0.13 0.22 0.023" color="Blue" namespace="${namespace}"/>
     <xacro:rotor rotor="3" parent="base_link" xyz="-0.13 -0.2 0.023" color="Red" namespace="${namespace}"/>
-    <link name='${namespace}/rotor_0'>
-      <inertial>
-        <mass value="0.005"/>
-        <inertia ixx="9.75e-07" ixy="0" ixz="0" iyy="4.17041e-05" iyz="0" izz="4.26041e-05"/>
-      </inertial>
-      <collision>
-        <geometry>
-          <cylinder length="0.005" radius="0.1"/>
-        </geometry>
-      </collision>
-      <visual>
-        <geometry>
-          <mesh filename="$(find as2_gazebo_assets)/models/quadrotor_base/meshes/propeller_ccw.dae" scale="0.1 0.1 0.1"/>
-        </geometry>
-        <material name="Blue"/>
-      </visual>
-      <gravity>1</gravity>
-      <velocity_decay/>
-    </link>
-    <joint name='${namespace}/rotor_0_joint' type="revolute">
-      <origin rpy="0 0 0" xyz="0.13 -0.22 0.023"/>
-      <parent link="${namespace}/base_link"/>
-      <child link="${namespace}/rotor_0"/>
-      <axis xyz="0 0 1" expressed_in="__model__"/>
-      <limit lower="-1e+16" upper="1e+16" effort="1000" velocity="100"/>
-      <dynamics spring_reference="0" spring_stiffness="0" friction="0" damping="0"/>
-    </joint>
     <xacro:tf freq="100"/>
-    <xacro:velocity namespace="${namespace}"/>
     <xacro:imu mass="0.005" parent="base_link" namespace="${namespace}"/>
     <xacro:odom topic="odom" freq="100" namespace="${namespace}"/>
     <xacro:motors namespace="${namespace}"/>
+    <xacro:velocity namespace="${namespace}"/>
   </xacro:macro>
 </robot>
