Commit message: Remove namespace

File: CustomRobots/quadrotor/models/quadrotor/quadrotor_common.urdf.xacro (robot description, xacro)
@@ -9,5 +9,5 @@
   </material>
   <xacro:macro name="rotor" params="rotor parent xyz color namespace">
-    <link name='${namespace}/rotor_${rotor}'>
+    <link name='rotor_${rotor}'>
       <inertial>
         <mass value="0.005"/>
@@ -28,8 +28,8 @@
       <velocity_decay/>
     </link>
-    <joint name='${namespace}/rotor_${rotor}_joint' type="revolute">
+    <joint name='rotor_${rotor}_joint' type="revolute">
       <origin rpy="0 0 0" xyz="${xyz}"/>
-      <parent link="${namespace}/${parent}"/>
-      <child link="${namespace}/rotor_${rotor}"/>
+      <parent link="${parent}"/>
+      <child link="rotor_${rotor}"/>
       <axis xyz="0 0 1" expressed_in="__model__"/>
       <limit lower="-1e+16" upper="1e+16" effort="1000" velocity="100"/>
@@ -38,7 +38,7 @@
   </xacro:macro>
   <xacro:macro name="quadrotor" params="namespace">
-    <link name="${namespace}/base"></link>
+    <link name="base"></link>
     <!-- This is from quadrotor_base from as2 -->
-    <link name="${namespace}/base_link">
+    <link name="base_link">
       <gazebo>
         <enable_wind>true</enable_wind>
@@ -77,7 +77,7 @@
       </visual>
     </link>
-    <joint name="${namespace}/base_to_base_link" type="fixed">
-      <parent link="${namespace}/base"/>
-      <child link="${namespace}/base_link"/>
+    <joint name="base_to_base_link" type="fixed">
+      <parent link="base"/>
+      <child link="base_link"/>
       <origin xyz="0 0 0" rpy="0 0 0"/>
     </joint>

File: CustomRobots/quadrotor/models/quadrotor/quadrotor_gz.urdf.xacro (robot description, xacro)
@@ -2,5 +2,5 @@
 <robot xmlns:xacro="http://ros.org/wiki/xacro">
   <xacro:macro name="camera" params="xyz rpy name parent mass namespace">
-    <link name="${namespace}/${name}_link">
+    <link name="${name}_link">
       <inertial>
         <origin rpy="${rpy}" xyz="${xyz}"/>
@@ -9,10 +9,10 @@
       </inertial>
     </link>
-    <joint name="${namespace}/${name}_to_${parent}" type="fixed">
-      <parent link="${namespace}/${parent}"/>
-      <child link="${namespace}/${name}_link"/>
+    <joint name="${name}_to_${parent}" type="fixed">
+      <parent link="${parent}"/>
+      <child link="${name}_link"/>
       <origin xyz="${xyz}" rpy="${rpy}"/>
     </joint>
-    <gazebo reference="${namespace}/${name}_link">
+    <gazebo reference="${name}_link">
       <sensor name="${name}" type="camera">
         <always_on>true</always_on>
@@ -49,5 +49,5 @@
         <motorControlPubTopic>command/motor_speed</motorControlPubTopic>
         <enableSubTopic>velocity_controller/enable</enableSubTopic>
-        <comLinkName>${namespace}/base_link</comLinkName>
+        <comLinkName>base_link</comLinkName>
         <velocityGain>2.7 2.7 2.7</velocityGain>
         <attitudeGain>2 3 0.15</attitudeGain>
@@ -69,5 +69,5 @@
         <rotorConfiguration>
           <rotor>
-            <jointName>${namespace}/rotor_0_joint</jointName>
+            <jointName>rotor_0_joint</jointName>
             <forceConstant>8.54858e-06</forceConstant>
             <momentConstant>0.016</momentConstant>
@@ -75,5 +75,5 @@
           </rotor>
           <rotor>
-            <jointName>${namespace}/rotor_1_joint</jointName>
+            <jointName>rotor_1_joint</jointName>
             <forceConstant>8.54858e-06</forceConstant>
             <momentConstant>0.016</momentConstant>
@@ -81,5 +81,5 @@
           </rotor>
           <rotor>
-            <jointName>${namespace}/rotor_2_joint</jointName>
+            <jointName>rotor_2_joint</jointName>
             <forceConstant>8.54858e-06</forceConstant>
             <momentConstant>0.016</momentConstant>
@@ -87,5 +87,5 @@
           </rotor>
           <rotor>
-            <jointName>${namespace}/rotor_3_joint</jointName>
+            <jointName>rotor_3_joint</jointName>
             <forceConstant>8.54858e-06</forceConstant>
             <momentConstant>0.016</momentConstant>
@@ -99,7 +99,7 @@
     <gazebo>
       <plugin filename="gz-sim-odometry-publisher-system" name="gz::sim::systems::OdometryPublisher">
-        <odom_frame>${namespace}/odom</odom_frame>
-        <robot_base_frame>${namespace}/base_link</robot_base_frame>
-        <odom_topic>${namespace}/${topic}</odom_topic>
+        <!-- <odom_frame>odom</odom_frame>
+        <robot_base_frame>base_link</robot_base_frame>
+        <odom_topic>${topic}</odom_topic> -->
         <odom_publish_frequency>${freq}</odom_publish_frequency>
         <dimensions>3</dimensions>
@@ -112,5 +112,5 @@
       </plugin>
     </gazebo>
-    <link name="${namespace}/imu_link">
+    <link name="imu_link">
       <inertial>
         <mass value="${mass}"/>
@@ -118,9 +118,9 @@
       </inertial>
     </link>
-    <joint name="${namespace}/imu_joint" type="fixed">
-      <parent link="${namespace}/${parent}"/>
-      <child link="${namespace}/imu_link"/>
+    <joint name="imu_joint" type="fixed">
+      <parent link="${parent}"/>
+      <child link="imu_link"/>
     </joint>
-    <gazebo reference="${namespace}/imu_link">
+    <gazebo reference="imu_link">
       <sensor name='imu' type='imu'>
         <always_on>1</always_on>
@@ -220,6 +220,6 @@
       <plugin filename="gz-sim-multicopter-motor-model-system" name="gz::sim::systems::MulticopterMotorModel">
         <robotNamespace>model/${namespace}</robotNamespace>
-        <jointName>${namespace}/rotor_${rotor-1}_joint</jointName>
-        <linkName>${namespace}/rotor_${rotor-1}</linkName>
+        <jointName>rotor_${rotor-1}_joint</jointName>
+        <linkName>rotor_${rotor-1}</linkName>
         <xacro:if value="${rotor-1 == 1 or rotor-1 == 0}">
           <turningDirection>ccw</turningDirection>

Commit message: Working demo

File: CustomRobots/quadrotor/models/quadrotor/quadrotor_common.urdf.xacro (robot description, xacro)
@@ -38,5 +38,4 @@
   </xacro:macro>
   <xacro:macro name="quadrotor" params="namespace">
-    <link name="base"></link>
     <!-- This is from quadrotor_base from as2 -->
     <link name="base_link">
@@ -77,9 +76,4 @@
       </visual>
     </link>
-    <joint name="base_to_base_link" type="fixed">
-      <parent link="base"/>
-      <child link="base_link"/>
-      <origin xyz="0 0 0" rpy="0 0 0"/>
-    </joint>
     <xacro:rotor rotor="0" parent="base_link" xyz="0.13 -0.22 0.023" color="Blue" namespace="${namespace}"/>
     <xacro:rotor rotor="1" parent="base_link" xyz="-0.13 0.2 0.023" color="Red" namespace="${namespace}"/>
