Commit message: Fix relative imports

File: CustomRobots/quadrotor/models/quadrotor/quadrotor_common.urdf.xacro (robot description, xacro)
@@ -1,13 +1,13 @@
-<?xml version="1.0" ?>
+<?xml version="1.0"?>
 <robot xmlns:xacro="http://ros.org/wiki/xacro">
-  <xacro:include filename="$(find custom_robots)/models/quadrotor/quadrotor_gz.urdf.xacro"/>
+  <xacro:include filename="$(find custom_robots)/models/quadrotor/quadrotor_gz.urdf.xacro" />
   <material name="Red">
-    <color rgba="1 0 0 1.0"/>
+    <color rgba="1 0 0 1.0" />
   </material>
   <material name="Blue">
-    <color rgba="0 0 1 1.0"/>
+    <color rgba="0 0 1 1.0" />
   </material>
   <material name="MagnetBlack">
-    <color rgba="0.05 0.05 0.05 1.0"/>
+    <color rgba="0.05 0.05 0.05 1.0" />
   </material>
   <!-- One box segment of the magnet ring. The ring leaves an open center
@@ -15,54 +15,55 @@
   <xacro:macro name="magnet_ring_seg" params="i n radius">
     <xacro:if value="${i &lt; n}">
-      <xacro:property name="ang" value="${2*pi*i/n}"/>
+      <xacro:property name="ang" value="${2*pi*i/n}" />
       <visual name="magnet_seg_${i}">
-        <origin xyz="${radius*cos(ang)} ${radius*sin(ang)} 0" rpy="0 0 ${ang + pi/2}"/>
+        <origin xyz="${radius*cos(ang)} ${radius*sin(ang)} 0" rpy="0 0 ${ang + pi/2}" />
         <geometry>
-          <box size="${2*radius*sin(pi/n)} 0.02 0.02"/>
+          <box size="${2*radius*sin(pi/n)} 0.02 0.02" />
         </geometry>
-        <material name="MagnetBlack"/>
+        <material name="MagnetBlack" />
       </visual>
-      <xacro:magnet_ring_seg i="${i+1}" n="${n}" radius="${radius}"/>
+      <xacro:magnet_ring_seg i="${i+1}" n="${n}" radius="${radius}" />
     </xacro:if>
   </xacro:macro>
   <material name="Green">
-    <color rgba="0 0.8 0 1.0"/>
+    <color rgba="0 0.8 0 1.0" />
   </material>
   <material name="Yellow">
-    <color rgba="1 0.9 0 1.0"/>
+    <color rgba="1 0.9 0 1.0" />
   </material>
   <material name="White">
-    <color rgba="1 1 1 1.0"/>
+    <color rgba="1 1 1 1.0" />
   </material>
   <material name="Magenta">
-    <color rgba="1 0 1 1.0"/>
+    <color rgba="1 0 1 1.0" />
   </material>
   <xacro:macro name="rotor" params="rotor parent xyz color">
     <link name='rotor_${rotor}'>
       <inertial>
-        <mass value="0.005"/>
-        <inertia ixx="9.75e-07" ixy="0" ixz="0" iyy="4.17041e-05" iyz="0" izz="4.26041e-05"/>
+        <mass value="0.005" />
+        <inertia ixx="9.75e-07" ixy="0" ixz="0" iyy="4.17041e-05" iyz="0" izz="4.26041e-05" />
       </inertial>
       <collision>
         <geometry>
-          <cylinder length="0.005" radius="0.1"/>
+          <cylinder length="0.005" radius="0.1" />
         </geometry>
       </collision>
       <visual>
         <geometry>
-          <mesh filename="$(find as2_gazebo_assets)/models/quadrotor_base/meshes/propeller_ccw.dae" scale="0.1 0.1 0.1"/>
+          <mesh filename="$(find custom_robots)/models/quadrotor/meshes/propeller_ccw.dae"
+            scale="0.1 0.1 0.1" />
         </geometry>
-        <material name="${color}"/>
+        <material name="${color}" />
       </visual>
       <gravity>1</gravity>
-      <velocity_decay/>
+      <velocity_decay />
     </link>
     <joint name='rotor_${rotor}_joint' type="revolute">
-      <origin rpy="0 0 0" xyz="${xyz}"/>
-      <parent link="${parent}"/>
-      <child link="rotor_${rotor}"/>
-      <axis xyz="0 0 1" expressed_in="__model__"/>
-      <limit lower="-1e+16" upper="1e+16" effort="1000" velocity="100"/>
-      <dynamics spring_reference="0" spring_stiffness="0" friction="0" damping="0"/>
+      <origin rpy="0 0 0" xyz="${xyz}" />
+      <parent link="${parent}" />
+      <child link="rotor_${rotor}" />
+      <axis xyz="0 0 1" expressed_in="__model__" />
+      <limit lower="-1e+16" upper="1e+16" effort="1000" velocity="100" />
+      <dynamics spring_reference="0" spring_stiffness="0" friction="0" damping="0" />
     </joint>
   </xacro:macro>
@@ -74,43 +75,43 @@
       </gazebo>
       <inertial>
-        <mass value="1.5"/>
-        <inertia ixx="0.025" ixy="0" ixz="0" iyy="0.009" iyz="0" izz="0.033"/>
+        <mass value="1.5" />
+        <inertia ixx="0.025" ixy="0" ixz="0" iyy="0.009" iyz="0" izz="0.033" />
       </inertial>
       <collision>
         <geometry>
-          <box size="0.47 0.47 0.11"/>
+          <box size="0.47 0.47 0.11" />
         </geometry>
       </collision>
       <visual>
         <geometry>
-          <mesh filename="$(find as2_gazebo_assets)/models/quadrotor_base/meshes/quadrotor.dae"/>
+          <mesh filename="$(find custom_robots)/models/quadrotor/meshes/quadrotor.dae" />
         </geometry>
         <xacro:if value="${color != ''}">
-          <material name="${color}"/>
+          <material name="${color}" />
         </xacro:if>
       </visual>
       <visual name='marker_visual_1'>
-        <origin rpy="0 0 0" xyz="-0.07 0 0.065"/>
+        <origin rpy="0 0 0" xyz="-0.07 0 0.065" />
         <geometry>
-          <mesh filename="$(find as2_gazebo_assets)/models/quadrotor_base/meshes/led.dae"/>
+          <mesh filename="$(find custom_robots)/models/quadrotor/meshes/led.dae" />
         </geometry>
       </visual>
       <visual name='marker_visual_2'>
-        <origin rpy="-1.0472 -0 0.2" xyz="-0.08 0.037 0.04"/>
+        <origin rpy="-1.0472 -0 0.2" xyz="-0.08 0.037 0.04" />
         <geometry>
-          <mesh filename="$(find as2_gazebo_assets)/models/quadrotor_base/meshes/led.dae"/>
+          <mesh filename="$(find custom_robots)/models/quadrotor/meshes/led.dae" />
         </geometry>
       </visual>
       <visual name='marker_visual_3'>
-        <origin rpy="1.0472 -0 -0.1" xyz="-0.08 -0.035 0.04"/>
+        <origin rpy="1.0472 -0 -0.1" xyz="-0.08 -0.035 0.04" />
         <geometry>
-          <mesh filename="$(find as2_gazebo_assets)/models/quadrotor_base/meshes/led.dae"/>
+          <mesh filename="$(find custom_robots)/models/quadrotor/meshes/led.dae" />
         </geometry>
       </visual>
     </link>
-    <xacro:rotor rotor="0" parent="base_link" xyz="0.13 -0.22 0.023" color="Blue"/>
-    <xacro:rotor rotor="1" parent="base_link" xyz="-0.13 0.2 0.023" color="Red"/>
-    <xacro:rotor rotor="2" parent="base_link" xyz="0.13 0.22 0.023" color="Blue"/>
-    <xacro:rotor rotor="3" parent="base_link" xyz="-0.13 -0.2 0.023" color="Red"/>
+    <xacro:rotor rotor="0" parent="base_link" xyz="0.13 -0.22 0.023" color="Blue" />
+    <xacro:rotor rotor="1" parent="base_link" xyz="-0.13 0.2 0.023" color="Red" />
+    <xacro:rotor rotor="2" parent="base_link" xyz="0.13 0.22 0.023" color="Blue" />
+    <xacro:rotor rotor="3" parent="base_link" xyz="-0.13 -0.2 0.023" color="Red" />
     <!-- Electromagnet: flat ring hugging the drone belly, with an open center
         so the downward ventral camera is not blocked (package_delivery). -->
@@ -118,21 +119,21 @@
       <link name="magnet">
         <inertial>
-          <mass value="0.02"/>
-          <inertia ixx="2e-5" ixy="0" ixz="0" iyy="2e-5" iyz="0" izz="4e-5"/>
+          <mass value="0.02" />
+          <inertia ixx="2e-5" ixy="0" ixz="0" iyy="2e-5" iyz="0" izz="4e-5" />
         </inertial>
-        <xacro:magnet_ring_seg i="0" n="12" radius="0.06"/>
+        <xacro:magnet_ring_seg i="0" n="12" radius="0.06" />
       </link>
       <joint name="magnet_joint" type="fixed">
-        <origin rpy="0 0 0" xyz="0 0 -0.05"/>
-        <parent link="base_link"/>
-        <child link="magnet"/>
+        <origin rpy="0 0 0" xyz="0 0 -0.05" />
+        <parent link="base_link" />
+        <child link="magnet" />
       </joint>
-      <xacro:magnetic_gripper namespace="${namespace}"/>
+      <xacro:magnetic_gripper namespace="${namespace}" />
     </xacro:if>
-    <xacro:tf freq="100" namespace="${namespace}"/>
-    <xacro:imu mass="0.005" parent="base_link" namespace="${namespace}"/>
-    <xacro:odom freq="100" namespace="${namespace}"/>
-    <xacro:motors namespace="${namespace}"/>
-    <xacro:velocity namespace="${namespace}"/>
+    <xacro:tf freq="100" namespace="${namespace}" />
+    <xacro:imu mass="0.005" parent="base_link" namespace="${namespace}" />
+    <xacro:odom freq="100" namespace="${namespace}" />
+    <xacro:motors namespace="${namespace}" />
+    <xacro:velocity namespace="${namespace}" />
   </xacro:macro>
 </robot>
