Commit message: Revert change

File: CustomRobots/quadrotor/models/quadrotor/quadrotor_gz.urdf.xacro (robot description, xacro)
@@ -201,5 +201,5 @@
     </gazebo>
   </xacro:macro>
-  <xacro:macro name="tf" params="freq namespace">
+  <xacro:macro name="tf" params="freq">
     <gazebo>
       <plugin filename="gz-sim-pose-publisher-system" name="gz::sim::systems::PosePublisher">
@@ -213,5 +213,4 @@
         <static_publisher>true</static_publisher>
         <static_update_frequency>${freq}</static_update_frequency>
-        <topic>/${namespace}/tf</topic>
       </plugin>
     </gazebo>

Commit message: Test defining all values

File: CustomRobots/quadrotor/models/quadrotor/quadrotor_gz.urdf.xacro (robot description, xacro)
@@ -99,7 +99,7 @@
     <gazebo>
       <plugin filename="gz-sim-odometry-publisher-system" name="gz::sim::systems::OdometryPublisher">
-        <!-- <odom_frame>odom</odom_frame>
+        <odom_frame>odom</odom_frame>
         <robot_base_frame>base_link</robot_base_frame>
-        <odom_topic>/model/${namespace}/odometry</odom_topic> -->
+        <odom_topic>/model/${namespace}/odometry</odom_topic>
         <odom_publish_frequency>${freq}</odom_publish_frequency>
         <dimensions>3</dimensions>
@@ -124,4 +124,5 @@
     <gazebo reference="imu_link">
       <sensor name='imu' type='imu'>
+        <topic>/model/${namespace}/imu</topic>
         <always_on>1</always_on>
         <update_rate>250</update_rate>
@@ -201,5 +202,5 @@
     </gazebo>
   </xacro:macro>
-  <xacro:macro name="tf" params="freq">
+  <xacro:macro name="tf" params="freq namespace">
     <gazebo>
       <plugin filename="gz-sim-pose-publisher-system" name="gz::sim::systems::PosePublisher">
@@ -213,4 +214,5 @@
         <static_publisher>true</static_publisher>
         <static_update_frequency>${freq}</static_update_frequency>
+        <topic>/model/${namespace}/pose</topic>
       </plugin>
     </gazebo>
