Commit message: Change ur.urdf,xacro

File: CustomRobots/robot_arms/models/ur3/ur.urdf.xacro (robot description, xacro)
@@ -5,13 +5,12 @@
   <!-- import main macro -->
   <xacro:include filename="$(find custom_robots)/models/ur3/ur_macro.xacro"/>
-  <!-- possible 'ur_type' values: ur3, ur3e, ur5, ur5e, ur10, ur10e, ur16e -->
-  <!-- the default value should raise an error in case this was called without defining the type -->
+  <!-- robot type -->
   <xacro:arg name="ur_type" default="ur3"/>
   <!-- parameters -->
   <xacro:arg name="prefix" default="" />
-  <xacro:arg name="joint_limit_params" default="$(find custom_robots)/config/$(arg ur_type)/joint_limits.yaml"/>
-  <xacro:arg name="kinematics_params" default="$(find custom_robots)/config/$(arg ur_type)/default_kinematics.yaml"/>
-  <xacro:arg name="physical_params" default="$(find custom_robots)/config/$(arg ur_type)/physical_parameters.yaml"/>
-  <xacro:arg name="visual_params" default="$(find custom_robots)/config/$(arg ur_type)/visual_parameters.yaml"/>
+  <xacro:arg name="joint_limit_params" default=""/>
+  <xacro:arg name="kinematics_params" default=""/>
+  <xacro:arg name="physical_params" default=""/>
+  <xacro:arg name="visual_params" default=""/>
   <xacro:arg name="transmission_hw_interface" default=""/>
   <xacro:arg name="safety_limits" default="false"/>
@@ -19,53 +18,67 @@
   <xacro:arg name="safety_k_position" default="20"/>
   <!-- ros2_control related parameters -->
-  <xacro:arg name="headless_mode" default="false" />
-  <xacro:arg name="robot_ip" default="0.0.0.0" />
+  <xacro:arg name="headless_mode" default="false"/>
+  <xacro:arg name="robot_ip" default="0.0.0.0"/>
   <xacro:arg name="script_filename" default=""/>
   <xacro:arg name="output_recipe_filename" default=""/>
   <xacro:arg name="input_recipe_filename" default=""/>
-  <!--   tool communication related parameters-->
-  <xacro:arg name="use_tool_communication" default="false" />
-  <xacro:arg name="tool_voltage" default="24" />
-  <xacro:arg name="tool_parity" default="0" />
-  <xacro:arg name="tool_baud_rate" default="115200" />
-  <xacro:arg name="tool_stop_bits" default="1" />
-  <xacro:arg name="tool_rx_idle_chars" default="1.5" />
-  <xacro:arg name="tool_tx_idle_chars" default="3.5" />
-  <xacro:arg name="tool_device_name" default="/tmp/ttyUR" />
-  <xacro:arg name="tool_tcp_port" default="54321" />
+  <!-- tool communication related parameters -->
+  <xacro:arg name="use_tool_communication" default="false"/>
+  <xacro:arg name="tool_voltage" default="24"/>
+  <xacro:arg name="tool_parity" default="0"/>
+  <xacro:arg name="tool_baud_rate" default="115200"/>
+  <xacro:arg name="tool_stop_bits" default="1"/>
+  <xacro:arg name="tool_rx_idle_chars" default="1.5"/>
+  <xacro:arg name="tool_tx_idle_chars" default="3.5"/>
+  <xacro:arg name="tool_device_name" default="/tmp/ttyUR"/>
+  <xacro:arg name="tool_tcp_port" default="54321"/>
   <!-- Simulation parameters -->
-  <xacro:arg name="use_fake_hardware" default="false" />
-  <xacro:arg name="fake_sensor_commands" default="false" />
-  <xacro:arg name="sim_gazebo" default="false" />
-  <xacro:arg name="sim_gz" default="false" />
-  <xacro:arg name="simulation_controllers" default="" />
-  <!-- initial position for simulations (Fake Hardware, Gazebo) -->
-  <xacro:arg name="initial_positions_file" default="$(find custom_robots)/config/initial_positions.yaml"/>
-  <!-- convert to property to use substitution in function -->
-  <xacro:property name="initial_positions_file" default="$(arg initial_positions_file)"/>
-  <!-- create link fixed to the "world" -->
-  <link name="world" />
+  <xacro:arg name="use_fake_hardware" default="false"/>
+  <xacro:arg name="fake_sensor_commands" default="false"/>
+  <xacro:arg name="sim_gazebo" default="false"/>
+  <xacro:arg name="sim_gz" default="true"/>
+  <xacro:arg name="simulation_controllers" default=""/>
+  <!-- initial position for simulations -->
+  <xacro:arg name="initial_positions_file"
+             default="$(find custom_robots)/config/initial_positions.yaml"/>
+  <!-- convert to property -->
+  <xacro:property name="initial_positions_file"
+                  default="$(arg initial_positions_file)"/>
+  <!-- create link fixed to world -->
+  <link name="world"/>
   <!-- arm -->
-  <xacro:ur_robot name="$(arg name)" prefix="$(arg prefix)" parent="world" joint_limits_parameters_file="$(arg joint_limit_params)" kinematics_parameters_file="$(arg kinematics_params)" physical_parameters_file="$(arg physical_params)" visual_parameters_file="$(arg visual_params)" transmission_hw_interface="$(arg transmission_hw_interface)" safety_limits="$(arg safety_limits)" safety_pos_margin="$(arg safety_pos_margin)" safety_k_position="$(arg safety_k_position)" use_fake_hardware="$(arg use_fake_hardware)" fake_sensor_commands="$(arg fake_sensor_commands)" sim_gazebo="$(arg sim_gazebo)" sim_gz="$(arg sim_gz)" headless_mode="$(arg headless_mode)" initial_positions="${load_yaml(initial_positions_file)}" use_tool_communication="$(arg use_tool_communication)" tool_voltage="$(arg tool_voltage)" tool_parity="$(arg tool_parity)" tool_baud_rate="$(arg tool_baud_rate)" tool_stop_bits="$(arg tool_stop_bits)" tool_rx_idle_chars="$(arg tool_rx_idle_chars)" tool_tx_idle_chars="$(arg tool_tx_idle_chars)" tool_device_name="$(arg tool_device_name)" tool_tcp_port="$(arg tool_tcp_port)" robot_ip="$(arg robot_ip)" script_filename="$(arg script_filename)" output_recipe_filename="$(arg output_recipe_filename)" input_recipe_filename="$(arg input_recipe_filename)">
-    <origin xyz="0 0 0" rpy="0 0 0" />
+  <xacro:ur_robot
+      name="$(arg name)"
+      prefix="$(arg prefix)"
+      parent="world"
+      robot_ip="$(arg robot_ip)"
+      script_filename="$(arg script_filename)"
+      output_recipe_filename="$(arg output_recipe_filename)"
+      input_recipe_filename="$(arg input_recipe_filename)">
+    <origin xyz="0 0 0" rpy="0 0 0"/>
   </xacro:ur_robot>
+  <!-- Gazebo Classic -->
   <xacro:if value="$(arg sim_gazebo)">
-    <!-- Gazebo plugins -->
-    <!-- update the plugin  -->
     <gazebo reference="world">
     </gazebo>
     <gazebo>
-      <plugin filename="libgazebo_ros2_control.so" name="gazebo_ros2_control">
-        <parameters>$(arg simulation_controllers)</parameters>
+      <plugin filename="libgazebo_ros2_control.so"
+              name="gazebo_ros2_control">
+        <parameters>
+          $(arg simulation_controllers)
+        </parameters>
       </plugin>
     </gazebo>
   </xacro:if>
+  <!-- Gazebo Harmonic -->
   <xacro:if value="$(arg sim_gz)">
-    <!-- Gazebo Sim (Harmonic) plugins -->
     <gazebo reference="world">
     </gazebo>
     <gazebo>
-      <plugin filename="gz_ros2_control-system" name="gz_ros2_control::GazeboSimROS2ControlPlugin">
-        <parameters>$(arg simulation_controllers)</parameters>
+      <plugin filename="gz_ros2_control-system"
+              name="gz_ros2_control::GazeboSimROS2ControlPlugin">
+        <parameters>
+          $(arg simulation_controllers)
+        </parameters>
       </plugin>
     </gazebo>
