Commit message: Change joint friction in macro

File: CustomRobots/robot_arms/models/ur3/ur.urdf.xacro (robot description, xacro)
@@ -10,11 +10,11 @@
   <xacro:arg name="prefix" default="" />
   <xacro:arg name="joint_limit_params"
-            default="$(find custom_robots)/config/ur3/joint_limits.yaml"/>
+            default="$(find custom_robots)/config/$(arg ur_type)/joint_limits.yaml"/>
   <xacro:arg name="kinematics_params"
-            default="$(find custom_robots)/config/ur3/default_kinematics.yaml"/>
+            default="$(find custom_robots)/config/$(arg ur_type)/default_kinematics.yaml"/>
   <xacro:arg name="physical_params"
-            default="$(find custom_robots)/config/ur3/physical_parameters.yaml"/>
+            default="$(find custom_robots)/config/$(arg ur_type)/physical_parameters.yaml"/>
   <xacro:arg name="visual_params"
-            default="$(find custom_robots)/config/ur3/visual_parameters.yaml"/>
+            default="$(find custom_robots)/config/$(arg ur_type)/visual_parameters.yaml"/>
   <xacro:arg name="transmission_hw_interface" default=""/>
   <xacro:arg name="safety_limits" default="false"/>
@@ -41,5 +41,5 @@
   <xacro:arg name="fake_sensor_commands" default="false"/>
   <xacro:arg name="sim_gazebo" default="false"/>
-  <xacro:arg name="sim_gz" default="true"/>
+  <xacro:arg name="sim_gz" default="false"/>
   <xacro:arg name="simulation_controllers" default=""/>
   <!-- initial position for simulations -->

File: CustomRobots/robot_arms/models/ur3/ur3.urdf.xacro (robot description, xacro)
@@ -56,3 +56,15 @@
   <!-- ros2_control GRIPPER -->
   <xacro:robotiq_85_ros2_control name="robotiq" prefix="" sim_gz="true" use_fake_hardware="false"/>
+  <!-- ros2_control UR3 -->
+  <xacro:ur_ros2_control
+      name="ur"
+      prefix=""
+      sim_gz="true"
+      use_fake_hardware="false"
+      script_filename=""
+      output_recipe_filename=""
+      input_recipe_filename=""
+      tf_prefix=""
+      hash_kinematics=""
+      robot_ip="0.0.0.0"/>
 </robot>

File: CustomRobots/robot_arms/models/ur3/ur_macro.xacro (robot description, xacro)
@@ -227,5 +227,12 @@
       <limit lower="${shoulder_pan_lower_limit}" upper="${shoulder_pan_upper_limit}"
         effort="${shoulder_pan_effort_limit}" velocity="${shoulder_pan_velocity_limit}"/>
-      <dynamics damping="1.0" friction="100.0"/>
+      <xacro:if value="${safety_limits}">
+        <safety_controller
+            soft_lower_limit="${shoulder_pan_lower_limit + safety_pos_margin}"
+            soft_upper_limit="${shoulder_pan_upper_limit - safety_pos_margin}"
+            k_position="${safety_k_position}"
+            k_velocity="0.0"/>
+      </xacro:if>
+      <dynamics damping="1.0" friction="0"/>
     </joint>
     <joint name="${prefix}shoulder_lift_joint" type="revolute">
@@ -236,5 +243,12 @@
       <limit lower="${shoulder_lift_lower_limit}" upper="${shoulder_lift_upper_limit}"
         effort="${shoulder_lift_effort_limit}" velocity="${shoulder_lift_velocity_limit}"/>
-      <dynamics damping="1.0" friction="100.0"/>
+      <xacro:if value="${safety_limits}">
+        <safety_controller
+            soft_lower_limit="${shoulder_lift_lower_limit + safety_pos_margin}"
+            soft_upper_limit="${shoulder_lift_upper_limit - safety_pos_margin}"
+            k_position="${safety_k_position}"
+            k_velocity="0.0"/>
+      </xacro:if>
+      <dynamics damping="1.0" friction="0"/>
     </joint>
     <joint name="${prefix}elbow_joint" type="revolute">
@@ -245,5 +259,12 @@
       <limit lower="${elbow_joint_lower_limit}" upper="${elbow_joint_upper_limit}"
         effort="${elbow_joint_effort_limit}" velocity="${elbow_joint_velocity_limit}"/>
-      <dynamics damping="1.0" friction="100.0"/>
+      <xacro:if value="${safety_limits}">
+        <safety_controller
+            soft_lower_limit="${elbow_joint_lower_limit + safety_pos_margin}"
+            soft_upper_limit="${elbow_joint_upper_limit - safety_pos_margin}"
+            k_position="${safety_k_position}"
+            k_velocity="0.0"/>
+      </xacro:if>
+      <dynamics damping="1.0" friction="0"/>
     </joint>
     <joint name="${prefix}wrist_1_joint" type="revolute">
@@ -254,5 +275,12 @@
       <limit lower="${wrist_1_lower_limit}" upper="${wrist_1_upper_limit}"
         effort="${wrist_1_effort_limit}" velocity="${wrist_1_velocity_limit}"/>
-      <dynamics damping="1.0" friction="10.0"/>
+      <xacro:if value="${safety_limits}">
+        <safety_controller
+            soft_lower_limit="${wrist_1_lower_limit + safety_pos_margin}"
+            soft_upper_limit="${wrist_1_upper_limit - safety_pos_margin}"
+            k_position="${safety_k_position}"
+            k_velocity="0.0"/>
+      </xacro:if>
+      <dynamics damping="1.0" friction="0"/>
     </joint>
     <joint name="${prefix}wrist_2_joint" type="revolute">
@@ -263,5 +291,12 @@
       <limit lower="${wrist_2_lower_limit}" upper="${wrist_2_upper_limit}"
              effort="${wrist_2_effort_limit}" velocity="${wrist_2_velocity_limit}"/>
-      <dynamics damping="1.0" friction="10.0"/>
+      <xacro:if value="${safety_limits}">
+        <safety_controller
+            soft_lower_limit="${wrist_2_lower_limit + safety_pos_margin}"
+            soft_upper_limit="${wrist_2_upper_limit - safety_pos_margin}"
+            k_position="${safety_k_position}"
+            k_velocity="0.0"/>
+      </xacro:if>
+      <dynamics damping="1.0" friction="0"/>
     </joint>
     <joint name="${prefix}wrist_3_joint" type="revolute">
@@ -272,4 +307,11 @@
       <limit lower="${wrist_3_lower_limit}" upper="${wrist_3_upper_limit}"
              effort="${wrist_3_effort_limit}" velocity="${wrist_3_velocity_limit}"/>
+      <xacro:if value="${safety_limits}">
+        <safety_controller
+            soft_lower_limit="${wrist_3_lower_limit + safety_pos_margin}"
+            soft_upper_limit="${wrist_3_upper_limit - safety_pos_margin}"
+            k_position="${safety_k_position}"
+            k_velocity="0.0"/>
+      </xacro:if>
       <dynamics damping="1.0" friction="1.0"/>
     </joint>
