Commit message: Change ur3.urdf.xacro

File: CustomRobots/robot_arms/models/ur3/ur3.urdf.xacro (robot description, xacro)
@@ -1,5 +1,4 @@
-<?xml version="1.0"?>
-<robot name="ur3"
-  xmlns:xacro="http://www.ros.org/wiki/xacro">
+<?xml version="1.0" ?>
+<robot name="ur3" xmlns:xacro="http://ros.org/wiki/xacro">
   <xacro:arg name="name" default="ur"/>
   <xacro:arg name="ur_type" default="ur3"/>
@@ -11,20 +10,35 @@
   <xacro:arg name="simulation_controllers" default=""/>
   <xacro:arg name="camera" default="false"/>
-  <xacro:include filename="$(find custom_robots)/models/ur3/ur.urdf.xacro" />
-  <xacro:include filename="$(find robotiq_description)/urdf/robotiq_85_gripper.urdf.xacro" />
-  <xacro:include filename="$(find robotiq_description)/urdf/robotiq_85_gripper.ros2_control.xacro" />
-  <xacro:include filename="$(find custom_robots)/models/ur3/ur.ros2_control.xacro" />
+  <xacro:arg name="robot_ip" default="0.0.0.0"/>
+  <xacro:arg name="script_filename" default=""/>
+  <xacro:arg name="input_recipe_filename" default=""/>
+  <xacro:arg name="output_recipe_filename" default=""/>
+  <!-- Include cams -->
   <xacro:if value="$(arg camera)">
     <xacro:include filename="$(find ros2srrc_ur5_gazebo)/urdf/common_properties.xacro"/>
+    <!-- HAND CAMERA -->
     <xacro:include filename="$(find ros2srrc_ur5_gazebo)/urdf/cam_on_hand_params_gz.xacro"/>
+    <xacro:property name="parent_hand" value="tool0"/>
     <xacro:include filename="$(find ros2srrc_ur5_gazebo)/urdf/cam_on_hand_gz.xacro"/>
+    <!-- BASE CAMERA -->
     <xacro:include filename="$(find ros2srrc_ur5_gazebo)/urdf/cam_on_base_params_gz.xacro"/>
+    <xacro:property name="parent_base" value="base_link"/>
+    <xacro:property name="cam_base_pz" value="0.5"/>
     <xacro:include filename="$(find ros2srrc_ur5_gazebo)/urdf/cam_on_base_gz.xacro"/>
   </xacro:if>
+  <xacro:include filename="$(find custom_robots)/models/ur3/ur.urdf.xacro"/>
+  <xacro:include filename="$(find custom_robots)/models/ur3/ur.ros2_control.xacro"/>
+  <xacro:include filename="$(find robotiq_description)/urdf/robotiq_85_gripper.urdf.xacro"/>
+  <xacro:include filename="$(find robotiq_description)/urdf/robotiq_85_gripper.ros2_control.xacro"/>
+  <!-- UR3 -->
+  <xacro:ur_robot
+    name="ur3"
+    tf_prefix=""
+  />
   <!-- Coupler -->
   <link name="robotiq_coupler">
     <visual>
       <geometry>
-        <mesh filename="package://robotiq_description/meshes/robotiq_85_coupler.stl" />
+        <mesh filename="package://robotiq_description/meshes/robotiq_85_coupler.stl"/>
       </geometry>
     </visual>
@@ -36,15 +50,32 @@
   </link>
   <joint name="robotiq_coupler_joint" type="fixed">
-    <origin xyz="0 0 0.004" rpy="0 0 ${-pi/2.0}" />
+    <origin xyz="0 0 0.004" rpy="0 0 ${-pi/2.0}"/>
     <parent link="tool0"/>
     <child link="robotiq_coupler"/>
   </joint>
   <!-- Gripper -->
-  <xacro:robotiq_85_gripper prefix="" parent="robotiq_coupler">
-    <origin xyz="0 0 0.004" rpy="0 ${-pi/2} ${pi}"/>
+  <xacro:robotiq_85_gripper
+    prefix=""
+    parent="robotiq_coupler">
+    <origin xyz="0 0 0.004"
+            rpy="0 ${-pi/2} ${pi}"/>
   </xacro:robotiq_85_gripper>
   <!-- ros2_control GRIPPER -->
-  <xacro:robotiq_85_ros2_control name="robotiq" prefix="" sim_gz="true" use_fake_hardware="false"/>
+  <xacro:robotiq_85_ros2_control
+    name="robotiq"
+    prefix=""
+    sim_gz="true"
+    use_fake_hardware="false"/>
   <!-- ros2_control UR3 -->
-  <xacro:ur_ros2_control name="ur" prefix="" sim_gz="true" use_fake_hardware="false" script_filename="" output_recipe_filename="" input_recipe_filename="" tf_prefix="" hash_kinematics="" robot_ip="0.0.0.0" />
+  <xacro:ur_ros2_control
+    name="ur3"
+    prefix=""
+    sim_gz="true"
+    use_fake_hardware="false"
+    script_filename="$(arg script_filename)"
+    output_recipe_filename="$(arg output_recipe_filename)"
+    input_recipe_filename="$(arg input_recipe_filename)"
+    tf_prefix=""
+    hash_kinematics=""
+    robot_ip="$(arg robot_ip)"/>
 </robot>

Commit message: add gripper control to xacro

File: CustomRobots/robot_arms/models/ur3/ur3.urdf.xacro (robot description, xacro)
@@ -33,4 +33,5 @@
   <xacro:include filename="$(find robotiq_description)/urdf/robotiq_85_gripper.ros2_control.xacro"/>
   <xacro:include filename="$(find ros2srrc_endeffectors)/robotiq_2f85/urdf/robotiq_2f85_macro.urdf.xacro"/>
+  <xacro:include filename="$(find ros2srrc_endeffectors)/robotiq_2f85/urdf/robotiq_2f85_ros2_control.xacro"/>
   <xacro:robotiq_2f85
     bringup="false"
@@ -48,3 +49,7 @@
     hash_kinematics=""
     robot_ip="$(arg robot_ip)"/>
+  <xacro:robotiq_2f85_ros2_control
+    name="robotiq"
+    sim_gz="true"
+    use_fake_hardware="false"/>
 </robot>

File: Industrial/ros2_SimRealRobotControl_gz/ros2srrc_endeffectors/robotiq_2f85/urdf/robotiq_2f85_ros2control.xacro (robot description, xacro)
@@ -1,50 +1,63 @@
 <?xml version="1.0"?>
 <robot xmlns:xacro="http://www.ros.org/wiki/xacro">
-  <!-- ros2_control configuration for Robotiq 85 Gripper -->
-  <xacro:macro name="EE_ros2control" params="" >
-    <!-- Main actuated joint -->
-    <joint name="robotiq_85_left_knuckle_joint">
-      <command_interface name="position">
-        <param name="min">0.0</param>
-        <param name="max">0.80285</param>
-      </command_interface>
-      <state_interface name="position">
-        <param name="initial_value">0.0</param>
-      </state_interface>
-      <state_interface name="velocity"/>
-      <state_interface name="effort"/>
-    </joint>
-    <!-- Mimic joints - need to be included for proper state publishing -->
-    <joint name="robotiq_85_right_knuckle_joint">
-      <param name="mimic">robotiq_85_left_knuckle_joint</param>
-      <param name="multiplier">1.0</param>
-      <state_interface name="position"/>
-      <state_interface name="velocity"/>
-      <state_interface name="effort"/>
-    </joint>
-    <joint name="robotiq_85_left_inner_knuckle_joint">
-      <param name="mimic">robotiq_85_left_knuckle_joint</param>
-      <param name="multiplier">1.0</param>
-      <state_interface name="position"/>
-      <state_interface name="velocity"/>
-    </joint>
-    <joint name="robotiq_85_right_inner_knuckle_joint">
-      <param name="mimic">robotiq_85_left_knuckle_joint</param>
-      <param name="multiplier">1.0</param>
-      <state_interface name="position"/>
-      <state_interface name="velocity"/>
-    </joint>
-    <joint name="robotiq_85_left_finger_tip_joint">
-      <param name="mimic">robotiq_85_left_knuckle_joint</param>
-      <param name="multiplier">-1.0</param>
-      <state_interface name="position"/>
-      <state_interface name="velocity"/>
-    </joint>
-    <joint name="robotiq_85_right_finger_tip_joint">
-      <param name="mimic">robotiq_85_left_knuckle_joint</param>
-      <param name="multiplier">-1.0</param>
-      <state_interface name="position"/>
-      <state_interface name="velocity"/>
-    </joint>
+  <xacro:macro name="robotiq_2f85_ros2_control"
+               params="
+               name:=robotiq
+               sim_gz:=true
+               use_fake_hardware:=false">
+    <ros2_control name="${name}_gripper" type="system">
+      <hardware>
+        <xacro:if value="${sim_gz}">
+          <plugin>gz_ros2_control/GazeboSimSystem</plugin>
+        </xacro:if>
+        <xacro:if value="${use_fake_hardware}">
+          <plugin>mock_components/GenericSystem</plugin>
+        </xacro:if>
+      </hardware>
+      <!-- actuated joint -->
+      <joint name="robotiq_85_left_knuckle_joint">
+        <command_interface name="position">
+          <param name="min">0.0</param>
+          <param name="max">0.80285</param>
+        </command_interface>
+        <state_interface name="position">
+          <param name="initial_value">0.0</param>
+        </state_interface>
+        <state_interface name="velocity"/>
+        <state_interface name="effort"/>
+      </joint>
+      <!-- mimic joints -->
+      <joint name="robotiq_85_right_knuckle_joint">
+        <param name="mimic">robotiq_85_left_knuckle_joint</param>
+        <param name="multiplier">1.0</param>
+        <state_interface name="position"/>
+        <state_interface name="velocity"/>
+        <state_interface name="effort"/>
+      </joint>
+      <joint name="robotiq_85_left_inner_knuckle_joint">
+        <param name="mimic">robotiq_85_left_knuckle_joint</param>
+        <param name="multiplier">1.0</param>
+        <state_interface name="position"/>
+        <state_interface name="velocity"/>
+      </joint>
+      <joint name="robotiq_85_right_inner_knuckle_joint">
+        <param name="mimic">robotiq_85_left_knuckle_joint</param>
+        <param name="multiplier">1.0</param>
+        <state_interface name="position"/>
+        <state_interface name="velocity"/>
+      </joint>
+      <joint name="robotiq_85_left_finger_tip_joint">
+        <param name="mimic">robotiq_85_left_knuckle_joint</param>
+        <param name="multiplier">-1.0</param>
+        <state_interface name="position"/>
+        <state_interface name="velocity"/>
+      </joint>
+      <joint name="robotiq_85_right_finger_tip_joint">
+        <param name="mimic">robotiq_85_left_knuckle_joint</param>
+        <param name="multiplier">-1.0</param>
+        <state_interface name="position"/>
+        <state_interface name="velocity"/>
+      </joint>
+    </ros2_control>
   </xacro:macro>
-  </robot>
+</robot>

Commit message: Fix macro and ros2control for gripper

File: CustomRobots/robot_arms/models/ur3/ur3.urdf.xacro (robot description, xacro)
@@ -34,5 +34,6 @@
   <xacro:robotiq_2f85
     bringup="false"
-    parent_link="tool0"/>
+    parent_link="tool0"
+    prefix=""/>
   <!-- ros2_control UR3 -->
   <xacro:ur_ros2_control
@@ -49,4 +50,5 @@
   <xacro:robotiq_2f85_ros2_control
     name="robotiq"
+    prefix=""
     sim_gz="true"
     use_fake_hardware="false"/>

File: Industrial/ros2_SimRealRobotControl_gz/ros2srrc_endeffectors/robotiq_2f85/urdf/robotiq_2f85_macro.urdf.xacro (robot description, xacro)
@@ -30,5 +30,9 @@
 <robot xmlns:xacro="http://ros.org/wiki/xacro">
   <!-- XACRO-MACRO of Robotiq 2f-85: -->
-  <xacro:macro name="robotiq_2f85" params="bringup parent_link">
+  <xacro:macro name="robotiq_2f85"
+                params="
+                bringup
+                parent_link
+                prefix:=">
     <xacro:unless value="${bringup}">
       <!-- Robotiq 2f-85 TRANSMISSION: -->
@@ -67,5 +71,5 @@
     </gazebo>
     <!-- Robotiq: base_link -->
-    <link name="robotiq_85_base_link">
+    <link name="${prefix}robotiq_85_base_link">
       <visual>
         <geometry>
@@ -86,11 +90,11 @@
       </inertial>
     </link>
-    <joint name="robotiq_85_base_joint" type="fixed">
+    <joint name="${prefix}robotiq_85_base_joint" type="fixed">
       <origin xyz="0 0 0.004" rpy="0 ${-pi/2} ${pi}"/>
       <parent link="robotiq_coupler"/>
-      <child link="robotiq_85_base_link"/>
+      <child link="${prefix}robotiq_85_base_link"/>
     </joint>
     <!-- Robotiq: left_knuckle -->
-    <link name="robotiq_85_left_knuckle_link">
+    <link name="${prefix}robotiq_85_left_knuckle_link">
       <visual>
         <geometry>
@@ -111,15 +115,15 @@
       </inertial>
     </link>
-    <joint name="robotiq_85_left_knuckle_joint" type="revolute">
-      <parent link="robotiq_85_base_link"/>
-      <child link="robotiq_85_left_knuckle_link"/>
+    <joint name="${prefix}robotiq_85_left_knuckle_joint" type="revolute">
+      <parent link="${prefix}robotiq_85_base_link"/>
+      <child link="${prefix}robotiq_85_left_knuckle_link"/>
       <axis xyz="0 0 1"/>
       <origin rpy="${pi} 0.0 0.0" xyz="0.05490451627 0.03060114443 0.0"/>
-      <limit lower="-0.05" upper="0.80285" velocity="0.5" effort="1000"/>
+      <limit lower="0.0" upper="0.80285" velocity="0.5" effort="1000"/>
       <dynamics damping="1.0" friction="1.0"/>
     </joint>
     <!-- Robotiq: right_knuckle -->
     <!-- Robotiq: right_knuckle -->
-    <link name="robotiq_85_right_knuckle_link">
+    <link name="${prefix}robotiq_85_right_knuckle_link">
       <visual>
         <geometry>
@@ -140,15 +144,15 @@
       </inertial>
     </link>
-    <joint name="robotiq_85_right_knuckle_joint" type="revolute">
-      <parent link="robotiq_85_base_link"/>
-      <child link="robotiq_85_right_knuckle_link"/>
+    <joint name="${prefix}robotiq_85_right_knuckle_joint" type="revolute">
+      <parent link="${prefix}robotiq_85_base_link"/>
+      <child link="${prefix}robotiq_85_right_knuckle_link"/>
       <axis xyz="0 0 1"/>
       <origin rpy="0 0 0" xyz="0.05490451627 -0.03060114443 0.0"/>
-      <limit lower="-0.05" upper="0.80285" velocity="0.5" effort="1000"/>
-      <dynamics damping="1.0" friction="1.0"/>
-      <mimic joint="robotiq_85_left_knuckle_joint" multiplier="1.0"/>
+      <limit lower="0.0" upper="0.80285" velocity="0.5" effort="1000"/>
+      <dynamics damping="1.0" friction="1.0"/>
+      <mimic joint="${prefix}robotiq_85_left_knuckle_joint" multiplier="1.0"/>
     </joint>
     <!-- Robotiq: left_finger -->
-    <link name="robotiq_85_left_finger_link">
+    <link name="${prefix}robotiq_85_left_finger_link">
       <visual>
         <geometry>
@@ -169,12 +173,12 @@
       </inertial>
     </link>
-    <joint name="robotiq_85_left_finger_joint" type="fixed">
-      <parent link="robotiq_85_left_knuckle_link"/>
-      <child link="robotiq_85_left_finger_link"/>
+    <joint name="${prefix}robotiq_85_left_finger_joint" type="fixed">
+      <parent link="${prefix}robotiq_85_left_knuckle_link"/>
+      <child link="${prefix}robotiq_85_left_finger_link"/>
       <origin xyz="-0.00408552455 -0.03148604435 0.0" rpy="0 0 0" />
       <dynamics damping="1.0" friction="1.0"/>
     </joint>
     <!-- Robotiq: right_finger -->
-    <link name="robotiq_85_right_finger_link">
+    <link name="${prefix}robotiq_85_right_finger_link">
       <visual>
         <geometry>
@@ -195,12 +199,12 @@
       </inertial>
     </link>
-    <joint name="robotiq_85_right_finger_joint" type="fixed">
-      <parent link="robotiq_85_right_knuckle_link"/>
-      <child link="robotiq_85_right_finger_link"/>
+    <joint name="${prefix}robotiq_85_right_finger_joint" type="fixed">
+      <parent link="${prefix}robotiq_85_right_knuckle_link"/>
+      <child link="${prefix}robotiq_85_right_finger_link"/>
       <origin xyz="-0.00408552455 -0.03148604435 0.0" rpy="0 0 0" />
       <dynamics damping="1.0" friction="1.0"/>
     </joint>
     <!-- Robotiq: left_inner_knuckle -->
-    <link name="robotiq_85_left_inner_knuckle_link">
+    <link name="${prefix}robotiq_85_left_inner_knuckle_link">
       <visual>
         <geometry>
@@ -221,15 +225,15 @@
       </inertial>
     </link>
-    <joint name="robotiq_85_left_inner_knuckle_joint" type="continuous">
-      <parent link="robotiq_85_base_link"/>
-      <child link="robotiq_85_left_inner_knuckle_link"/>
+    <joint name="${prefix}robotiq_85_left_inner_knuckle_joint" type="continuous">
+      <parent link="${prefix}robotiq_85_base_link"/>
+      <child link="${prefix}robotiq_85_left_inner_knuckle_link"/>
       <axis xyz="0 0 1"/>
       <origin xyz="0.06142 0.0127 0" rpy="${pi} 0.0 0.0" />
       <limit lower="-0.05" upper="0.80285" velocity="0.5" effort="1000"/>
       <dynamics damping="1.0" friction="1.0"/>
-      <mimic joint="robotiq_85_left_knuckle_joint" multiplier="1.0"/>
+      <mimic joint="${prefix}robotiq_85_left_knuckle_joint" multiplier="1.0"/>
     </joint>
     <!-- Robotiq: right_inner_knuckle -->
-    <link name="robotiq_85_right_inner_knuckle_link">
+    <link name="${prefix}robotiq_85_right_inner_knuckle_link">
       <visual>
         <geometry>
@@ -250,15 +254,15 @@
       </inertial>
     </link>
-    <joint name="robotiq_85_right_inner_knuckle_joint" type="continuous">
-      <parent link="robotiq_85_base_link"/>
-      <child link="robotiq_85_right_inner_knuckle_link"/>
+    <joint name="${prefix}robotiq_85_right_inner_knuckle_joint" type="continuous">
+      <parent link="${prefix}robotiq_85_base_link"/>
+      <child link="${prefix}robotiq_85_right_inner_knuckle_link"/>
       <axis xyz="0 0 1"/>
       <origin xyz="0.06142 -0.0127 0" rpy="0 0 0"/>
       <limit lower="-0.05" upper="0.80285" velocity="0.5" effort="1000"/>
       <dynamics damping="1.0" friction="1.0"/>
-      <mimic joint="robotiq_85_left_knuckle_joint" multiplier="1.0"/>
+      <mimic joint="${prefix}robotiq_85_left_knuckle_joint" multiplier="1.0"/>
     </joint>
     <!-- Robotiq: left_finger_tip -->
-    <link name="robotiq_85_left_finger_tip_link">
+    <link name="${prefix}robotiq_85_left_finger_tip_link">
       <visual>
         <geometry>
@@ -281,15 +285,15 @@
       </inertial>
     </link>
-    <joint name="robotiq_85_left_finger_tip_joint" type="continuous">
-      <parent link="robotiq_85_left_inner_knuckle_link"/>
-      <child link="robotiq_85_left_finger_tip_link"/>
+    <joint name="${prefix}robotiq_85_left_finger_tip_joint" type="continuous">
+      <parent link="${prefix}robotiq_85_left_inner_knuckle_link"/>
+      <child link="${prefix}robotiq_85_left_finger_tip_link"/>
       <axis xyz="0 0 1"/>
       <origin xyz="0.04303959807 -0.03759940821 0.0" rpy="0.0 0.0 0.0"/>
       <limit lower="-0.80285" upper="0.05" velocity="0.5" effort="1000"/>
       <dynamics damping="1.0" friction="1.0"/>
-      <mimic joint="robotiq_85_left_knuckle_joint" multiplier="-1.0"/>
+      <mimic joint="${prefix}robotiq_85_left_knuckle_joint" multiplier="-1.0"/>
     </joint>
     <!-- Robotiq: right_finger_tip -->
-    <link name="robotiq_85_right_finger_tip_link">
+    <link name="${prefix}robotiq_85_right_finger_tip_link">
       <visual>
         <geometry>
@@ -312,12 +316,12 @@
       </inertial>
     </link>
-    <joint name="robotiq_85_right_finger_tip_joint" type="continuous">
-      <parent link="robotiq_85_right_inner_knuckle_link"/>
-      <child link="robotiq_85_right_finger_tip_link"/>
+    <joint name="${prefix}robotiq_85_right_finger_tip_joint" type="continuous">
+      <parent link="${prefix}robotiq_85_right_inner_knuckle_link"/>
+      <child link="${prefix}robotiq_85_right_finger_tip_link"/>
       <axis xyz="0 0 1"/>
       <origin rpy="0.0 0.0 0.0" xyz="0.04303959807 -0.03759940821  0.0"/>
       <limit lower="-0.80285" upper="0.05" velocity="0.5" effort="1000"/>
       <dynamics damping="1.0" friction="1.0"/>
-      <mimic joint="robotiq_85_left_knuckle_joint" multiplier="-1.0"/>
+      <mimic joint="${prefix}robotiq_85_left_knuckle_joint" multiplier="-1.0"/>
     </joint>
     <!-- SMALL CUBE FOR GRIPPER PLUGIN -->
@@ -341,5 +345,5 @@
     </link>
     <joint name="EE_robotiq_2f85_joint" type="fixed" >
-      <parent link="robotiq_85_base_link" />
+      <parent link="${prefix}robotiq_85_base_link" />
       <child link="EE_robotiq_2f85" />
       <origin xyz="0.128 0.0 0.0" rpy="0 0 0"/>

File: Industrial/ros2_SimRealRobotControl_gz/ros2srrc_endeffectors/robotiq_2f85/urdf/robotiq_2f85_ros2control.xacro (robot description, xacro)
@@ -2,8 +2,9 @@
 <robot xmlns:xacro="http://www.ros.org/wiki/xacro">
   <xacro:macro name="robotiq_2f85_ros2_control"
-               params="
-               name:=robotiq
-               sim_gz:=true
-               use_fake_hardware:=false">
+                params="
+                name
+                prefix
+                sim_gz:=true
+                use_fake_hardware:=false">
     <ros2_control name="${name}_gripper" type="system">
       <hardware>
@@ -16,5 +17,5 @@
       </hardware>
       <!-- actuated joint -->
-      <joint name="robotiq_85_left_knuckle_joint">
+      <joint name="${prefix}robotiq_85_left_knuckle_joint">
         <command_interface name="position">
           <param name="min">0.0</param>
@@ -28,32 +29,52 @@
       </joint>
       <!-- mimic joints -->
-      <joint name="robotiq_85_right_knuckle_joint">
-        <param name="mimic">robotiq_85_left_knuckle_joint</param>
+      <joint name="${prefix}robotiq_85_right_knuckle_joint">
+        <param name="mimic">${prefix}robotiq_85_left_knuckle_joint</param>
         <param name="multiplier">1.0</param>
+        <command_interface name="position">
+            <param name="min">0.0</param>
+            <param name="max">0.80285</param>
+        </command_interface>
         <state_interface name="position"/>
         <state_interface name="velocity"/>
         <state_interface name="effort"/>
       </joint>
-      <joint name="robotiq_85_left_inner_knuckle_joint">
-        <param name="mimic">robotiq_85_left_knuckle_joint</param>
+      <joint name="${prefix}robotiq_85_left_inner_knuckle_joint">
+        <param name="mimic">${prefix}robotiq_85_left_knuckle_joint</param>
         <param name="multiplier">1.0</param>
+        <command_interface name="position">
+            <param name="min">0.0</param>
+            <param name="max">0.80285</param>
+        </command_interface>
         <state_interface name="position"/>
         <state_interface name="velocity"/>
       </joint>
-      <joint name="robotiq_85_right_inner_knuckle_joint">
-        <param name="mimic">robotiq_85_left_knuckle_joint</param>
+      <joint name="${prefix}robotiq_85_right_inner_knuckle_joint">
+        <param name="mimic">${prefix}robotiq_85_left_knuckle_joint</param>
         <param name="multiplier">1.0</param>
+        <command_interface name="position">
+            <param name="min">0.0</param>
+            <param name="max">0.80285</param>
+        </command_interface>
         <state_interface name="position"/>
         <state_interface name="velocity"/>
       </joint>
-      <joint name="robotiq_85_left_finger_tip_joint">
-        <param name="mimic">robotiq_85_left_knuckle_joint</param>
+      <joint name="${prefix}robotiq_85_left_finger_tip_joint">
+        <param name="mimic">${prefix}robotiq_85_left_knuckle_joint</param>
         <param name="multiplier">-1.0</param>
+        <command_interface name="position">
+            <param name="min">-0.80285</param>
+            <param name="max">0.0</param>
+        </command_interface>
         <state_interface name="position"/>
         <state_interface name="velocity"/>
       </joint>
-      <joint name="robotiq_85_right_finger_tip_joint">
-        <param name="mimic">robotiq_85_left_knuckle_joint</param>
+      <joint name="${prefix}robotiq_85_right_finger_tip_joint">
+        <param name="mimic">${prefix}robotiq_85_left_knuckle_joint</param>
         <param name="multiplier">-1.0</param>
+        <command_interface name="position">
+            <param name="min">-0.80285</param>
+            <param name="max">0.0</param>
+        </command_interface>
         <state_interface name="position"/>
         <state_interface name="velocity"/>
