Commit message: Fix xacro for use new gripper macro

File: CustomRobots/robot_arms/models/ur3/ur3.urdf.xacro (robot description, xacro)
@@ -32,8 +32,28 @@
   <xacro:include filename="$(find ros2srrc_endeffectors)/robotiq_2f85/urdf/robotiq_2f85_macro.urdf.xacro"/>
   <xacro:include filename="$(find ros2srrc_endeffectors)/robotiq_2f85/urdf/robotiq_2f85_ros2control.xacro"/>
-  <xacro:robotiq_2f85
-    bringup="false"
-    parent_link="tool0"
-    prefix=""/>
+  <!-- Coupler -->
+  <link name="robotiq_coupler">
+    <visual>
+      <geometry>
+        <mesh filename="package://robotiq_description/meshes/robotiq_85_coupler.stl" />
+      </geometry>
+    </visual>
+    <collision>
+      <geometry>
+        <cylinder radius="0.04" length="0.015"/>
+      </geometry>
+    </collision>
+  </link>
+  <joint name="robotiq_coupler_joint" type="fixed">
+    <origin xyz="0 0 0.004" rpy="0 0 ${-pi/2.0}" />
+    <parent link="tool0"/>
+    <child link="robotiq_coupler"/>
+  </joint>
+  <!-- Gripper -->
+  <xacro:robotiq_85_gripper prefix="" parent="robotiq_coupler">
+    <origin xyz="0 0 0.004" rpy="0 ${-pi/2} ${pi}"/>
+  </xacro:robotiq_85_gripper>
+  <!-- ros2_control GRIPPER -->
+  <xacro:robotiq_85_ros2_control name="robotiq" prefix="" sim_gz="true" use_fake_hardware="false"/>
   <!-- ros2_control UR3 -->
   <xacro:ur_ros2_control
@@ -48,8 +68,3 @@
     hash_kinematics=""
     robot_ip="$(arg robot_ip)"/>
-  <xacro:robotiq_2f85_ros2_control
-    name="robotiq"
-    prefix=""
-    sim_gz="true"
-    use_fake_hardware="false"/>
 </robot>

Commit message: add sausage spawn and move base camera

File: CustomRobots/robot_arms/models/ur3/ur3.urdf.xacro (robot description, xacro)
@@ -24,5 +24,12 @@
     <xacro:include filename="$(find ros2srrc_ur5_gazebo)/urdf/cam_on_base_params_gz.xacro"/>
     <xacro:property name="parent_base" value="base_link"/>
-    <xacro:property name="cam_base_pz" value="0.5"/>
+    <!-- Posición -->
+    <xacro:property name="cam_base_px" value="0.8"/>
+    <xacro:property name="cam_base_py" value="-0.2"/>
+    <xacro:property name="cam_base_pz" value="1.2"/>
+    <!-- Orientación -->
+    <xacro:property name="cam_base_or" value="1.57"/>
+    <xacro:property name="cam_base_op" value="0.2"/>
+    <xacro:property name="cam_base_oy" value="3.14"/>
     <xacro:include filename="$(find ros2srrc_ur5_gazebo)/urdf/cam_on_base_gz.xacro"/>
   </xacro:if>

Commit message: Change camera base pose

File: CustomRobots/robot_arms/models/ur3/ur3.urdf.xacro (robot description, xacro)
@@ -25,11 +25,11 @@
     <xacro:property name="parent_base" value="base_link"/>
     <!-- Posición -->
-    <xacro:property name="cam_base_px" value="0.8"/>
-    <xacro:property name="cam_base_py" value="-0.2"/>
-    <xacro:property name="cam_base_pz" value="1.2"/>
+    <xacro:property name="cam_base_px" value="0.5"/>
+    <xacro:property name="cam_base_py" value="0.0"/>
+    <xacro:property name="cam_base_pz" value="0.9"/>
     <!-- Orientación -->
-    <xacro:property name="cam_base_or" value="1.57"/>
-    <xacro:property name="cam_base_op" value="0.2"/>
-    <xacro:property name="cam_base_oy" value="3.14"/>
+    <xacro:property name="cam_base_or" value="0.0"/>
+    <xacro:property name="cam_base_op" value="1.57"/>
+    <xacro:property name="cam_base_oy" value="0.0"/>
     <xacro:include filename="$(find ros2srrc_ur5_gazebo)/urdf/cam_on_base_gz.xacro"/>
   </xacro:if>
