Commit message: Move down base camera

File: CustomRobots/robot_arms/models/ur3/ur3.urdf.xacro (robot description, xacro)
@@ -27,5 +27,5 @@
     <xacro:property name="cam_base_px" value="0.5"/>
     <xacro:property name="cam_base_py" value="0.0"/>
-    <xacro:property name="cam_base_pz" value="0.9"/>
+    <xacro:property name="cam_base_pz" value="0.5"/>
     <!-- Orientación -->
     <xacro:property name="cam_base_or" value="0.0"/>

Commit message: Add cameras, delete real robot node, delete debug from moveit nodes and add sausage spawner

File: CustomRobots/robot_arms/models/ur3/ur3.urdf.xacro (robot description, xacro)
@@ -24,5 +24,12 @@
     <xacro:include filename="$(find ros2srrc_ur5_gazebo)/urdf/cam_on_base_params_gz.xacro"/>
     <xacro:property name="parent_base" value="base_link"/>
+    <!-- Posición -->
+    <xacro:property name="cam_base_px" value="0.5"/>
+    <xacro:property name="cam_base_py" value="0.0"/>
     <xacro:property name="cam_base_pz" value="0.5"/>
+    <!-- Orientación -->
+    <xacro:property name="cam_base_or" value="0.0"/>
+    <xacro:property name="cam_base_op" value="1.57"/>
+    <xacro:property name="cam_base_oy" value="0.0"/>
     <xacro:include filename="$(find ros2srrc_ur5_gazebo)/urdf/cam_on_base_gz.xacro"/>
   </xacro:if>

Commit message: Change camera position and robot position

File: CustomRobots/robot_arms/models/ur3/ur3.urdf.xacro (robot description, xacro)
@@ -26,5 +26,5 @@
     <!-- Posición -->
     <xacro:property name="cam_base_px" value="0.5"/>
-    <xacro:property name="cam_base_py" value="0.0"/>
+    <xacro:property name="cam_base_py" value="-0.2"/>
     <xacro:property name="cam_base_pz" value="0.5"/>
     <!-- Orientación -->

Commit message: Change camera pose

File: CustomRobots/robot_arms/models/ur3/ur3.urdf.xacro (robot description, xacro)
@@ -26,5 +26,5 @@
     <!-- Posición -->
     <xacro:property name="cam_base_px" value="0.5"/>
-    <xacro:property name="cam_base_py" value="-0.2"/>
+    <xacro:property name="cam_base_py" value="0.15"/>
     <xacro:property name="cam_base_pz" value="0.5"/>
     <!-- Orientación -->

Commit message: Change camera pose

File: CustomRobots/robot_arms/models/ur3/ur3.urdf.xacro (robot description, xacro)
@@ -26,5 +26,5 @@
     <!-- Posición -->
     <xacro:property name="cam_base_px" value="0.5"/>
-    <xacro:property name="cam_base_py" value="0.15"/>
+    <xacro:property name="cam_base_py" value="0.8"/>
     <xacro:property name="cam_base_pz" value="0.5"/>
     <!-- Orientación -->

Commit message: Change sausage scene

File: CustomRobots/robot_arms/models/ur3/ur3.urdf.xacro (robot description, xacro)
@@ -25,7 +25,7 @@
     <xacro:property name="parent_base" value="base_link"/>
     <!-- Posición -->
-    <xacro:property name="cam_base_px" value="0.0"/>
+    <xacro:property name="cam_base_px" value="-0.4"/>
     <xacro:property name="cam_base_py" value="1.2"/>
-    <xacro:property name="cam_base_pz" value="0.5"/>
+    <xacro:property name="cam_base_pz" value="0.1"/>
     <!-- Orientación -->
     <xacro:property name="cam_base_or" value="0.0"/>

Commit message: Change sausage scene

File: CustomRobots/robot_arms/models/ur3/ur3.urdf.xacro (robot description, xacro)
@@ -26,6 +26,6 @@
     <!-- Posición -->
     <xacro:property name="cam_base_px" value="-0.4"/>
-    <xacro:property name="cam_base_py" value="1.2"/>
-    <xacro:property name="cam_base_pz" value="0.1"/>
+    <xacro:property name="cam_base_py" value="0.95"/>
+    <xacro:property name="cam_base_pz" value="0.0"/>
     <!-- Orientación -->
     <xacro:property name="cam_base_or" value="0.0"/>

Commit message: change sausage scene

File: CustomRobots/robot_arms/models/ur3/ur3.urdf.xacro (robot description, xacro)
@@ -25,7 +25,7 @@
     <xacro:property name="parent_base" value="base_link"/>
     <!-- Posición -->
-    <xacro:property name="cam_base_px" value="-0.4"/>
-    <xacro:property name="cam_base_py" value="0.95"/>
-    <xacro:property name="cam_base_pz" value="0.0"/>
+    <xacro:property name="cam_base_px" value="-0.45"/>
+    <xacro:property name="cam_base_py" value="1.2"/>
+    <xacro:property name="cam_base_pz" value="-0.4"/>
     <!-- Orientación -->
     <xacro:property name="cam_base_or" value="0.0"/>

Commit message: Change sausage scene

File: CustomRobots/robot_arms/models/ur3/ur3.urdf.xacro (robot description, xacro)
@@ -25,7 +25,7 @@
     <xacro:property name="parent_base" value="base_link"/>
     <!-- Posición -->
-    <xacro:property name="cam_base_px" value="-0.45"/>
-    <xacro:property name="cam_base_py" value="1.2"/>
-    <xacro:property name="cam_base_pz" value="-0.4"/>
+    <xacro:property name="cam_base_px" value="-0.4"/>
+    <xacro:property name="cam_base_py" value="0.75"/>
+    <xacro:property name="cam_base_pz" value="0.5"/>
     <!-- Orientación -->
     <xacro:property name="cam_base_or" value="0.0"/>
