Commit message: Change base cam pose

File: CustomRobots/robot_arms/models/ur3/ur3_servo.urdf.xacro (robot description, xacro)
@@ -25,5 +25,5 @@
     <xacro:property name="parent_base" value="base_link"/>
     <!-- Posición -->
-    <xacro:property name="cam_base_px" value="-0.3"/>
+    <xacro:property name="cam_base_px" value="1.3"/>
     <xacro:property name="cam_base_py" value="1.2"/>
     <xacro:property name="cam_base_pz" value="0.0"/>

Commit message: Change base cam pose

File: CustomRobots/robot_arms/models/ur3/ur3_servo.urdf.xacro (robot description, xacro)
@@ -25,7 +25,7 @@
     <xacro:property name="parent_base" value="base_link"/>
     <!-- Posición -->
-    <xacro:property name="cam_base_px" value="1.3"/>
+    <xacro:property name="cam_base_px" value="0.0"/>
     <xacro:property name="cam_base_py" value="1.2"/>
-    <xacro:property name="cam_base_pz" value="0.0"/>
+    <xacro:property name="cam_base_pz" value="0.5"/>
     <!-- Orientación -->
     <xacro:property name="cam_base_or" value="0.0"/>

Commit message: Change base cam pose

File: CustomRobots/robot_arms/models/ur3/ur3_servo.urdf.xacro (robot description, xacro)
@@ -25,5 +25,5 @@
     <xacro:property name="parent_base" value="base_link"/>
     <!-- Posición -->
-    <xacro:property name="cam_base_px" value="0.0"/>
+    <xacro:property name="cam_base_px" value="1.0"/>
     <xacro:property name="cam_base_py" value="1.2"/>
     <xacro:property name="cam_base_pz" value="0.5"/>

Commit message: Change base cam pose

File: CustomRobots/robot_arms/models/ur3/ur3_servo.urdf.xacro (robot description, xacro)
@@ -25,7 +25,7 @@
     <xacro:property name="parent_base" value="base_link"/>
     <!-- Posición -->
-    <xacro:property name="cam_base_px" value="1.0"/>
+    <xacro:property name="cam_base_px" value="0.8"/>
     <xacro:property name="cam_base_py" value="1.2"/>
-    <xacro:property name="cam_base_pz" value="0.5"/>
+    <xacro:property name="cam_base_pz" value="0.0"/>
     <!-- Orientación -->
     <xacro:property name="cam_base_or" value="0.0"/>

Commit message: Change base cam pose

File: CustomRobots/robot_arms/models/ur3/ur3_servo.urdf.xacro (robot description, xacro)
@@ -26,6 +26,6 @@
     <!-- Posición -->
     <xacro:property name="cam_base_px" value="0.8"/>
-    <xacro:property name="cam_base_py" value="1.2"/>
-    <xacro:property name="cam_base_pz" value="0.0"/>
+    <xacro:property name="cam_base_py" value="0.4"/>
+    <xacro:property name="cam_base_pz" value="0.5"/>
     <!-- Orientación -->
     <xacro:property name="cam_base_or" value="0.0"/>

Commit message: Change base cam angle

File: CustomRobots/robot_arms/models/ur3/ur3_servo.urdf.xacro (robot description, xacro)
@@ -30,5 +30,5 @@
     <!-- Orientación -->
     <xacro:property name="cam_base_or" value="0.0"/>
-    <xacro:property name="cam_base_op" value="1.57"/>
+    <xacro:property name="cam_base_op" value="0.0"/>
     <xacro:property name="cam_base_oy" value="0.0"/>
     <xacro:include filename="$(find ros2srrc_ur5_gazebo)/urdf/cam_on_base_gz.xacro"/>

Commit message: Change base cam angle

File: CustomRobots/robot_arms/models/ur3/ur3_servo.urdf.xacro (robot description, xacro)
@@ -29,6 +29,6 @@
     <xacro:property name="cam_base_pz" value="0.5"/>
     <!-- Orientación -->
-    <xacro:property name="cam_base_or" value="0.0"/>
-    <xacro:property name="cam_base_op" value="0.0"/>
+    <xacro:property name="cam_base_or" value="1.57"/>
+    <xacro:property name="cam_base_op" value="1.57"/>
     <xacro:property name="cam_base_oy" value="0.0"/>
     <xacro:include filename="$(find ros2srrc_ur5_gazebo)/urdf/cam_on_base_gz.xacro"/>
