Commit message: Change stack

File: CustomRobots/robot_arms/models/ur3/inc/ur_common.xacro (robot description, xacro)
@@ -168,4 +168,16 @@
     <xacro:property name="forearm_radius" value="${sec_inertia_parameters['forearm_radius']}" scope="parent"/>
     <xacro:property name="wrist_radius" value="${sec_inertia_parameters['wrist_radius']}" scope="parent"/>
+    <xacro:property
+        name="wrist_1_visual_offset"
+        value="${sec_mesh_files['wrist_1']['visual_offset']}"
+        scope="parent"/>
+    <xacro:property
+        name="wrist_2_visual_offset"
+        value="${sec_mesh_files['wrist_2']['visual_offset']}"
+        scope="parent"/>
+    <xacro:property
+        name="wrist_3_visual_offset"
+        value="${sec_mesh_files['wrist_3']['visual_offset']}"
+        scope="parent"/>
     <!--KINEMATICS HASH-->
     <xacro:property name="kinematics_hash" value="${sec_kinematics['hash']}" scope="parent"/>

File: CustomRobots/robot_arms/models/ur3/ur.ros2_control.xacro (robot description, xacro)
@@ -57,10 +57,10 @@
       <joint name="${prefix}shoulder_pan_joint">
         <command_interface name="position">
-          <param name="min">{-2*pi}</param>
-          <param name="max">{2*pi}</param>
-        </command_interface>
-        <command_interface name="velocity">
-          <param name="min">-3.15</param>
-          <param name="max">3.15</param>
+            <param name="min">{-2*pi}</param>
+            <param name="max">{2*pi}</param>
+        </command_interface>
+        <command_interface name="velocity">
+            <param name="min">-3.15</param>
+            <param name="max">3.15</param>
         </command_interface>
         <state_interface name="position">
@@ -73,10 +73,10 @@
       <joint name="${prefix}shoulder_lift_joint">
         <command_interface name="position">
-          <param name="min">{-2*pi}</param>
-          <param name="max">{2*pi}</param>
-        </command_interface>
-        <command_interface name="velocity">
-          <param name="min">-3.15</param>
-          <param name="max">3.15</param>
+            <param name="min">{-2*pi}</param>
+            <param name="max">{2*pi}</param>
+        </command_interface>
+        <command_interface name="velocity">
+            <param name="min">-3.15</param>
+            <param name="max">3.15</param>
         </command_interface>
         <state_interface name="position">
@@ -89,10 +89,10 @@
       <joint name="${prefix}elbow_joint">
         <command_interface name="position">
-          <param name="min">{-pi}</param>
-          <param name="max">{pi}</param>
-        </command_interface>
-        <command_interface name="velocity">
-          <param name="min">-3.15</param>
-          <param name="max">3.15</param>
+            <param name="min">{-pi}</param>
+            <param name="max">{pi}</param>
+        </command_interface>
+        <command_interface name="velocity">
+            <param name="min">-3.15</param>
+            <param name="max">3.15</param>
         </command_interface>
         <state_interface name="position">
@@ -105,10 +105,10 @@
       <joint name="${prefix}wrist_1_joint">
         <command_interface name="position">
-          <param name="min">{-2*pi}</param>
-          <param name="max">{2*pi}</param>
-        </command_interface>
-        <command_interface name="velocity">
-          <param name="min">-3.2</param>
-          <param name="max">3.2</param>
+            <param name="min">{-2*pi}</param>
+            <param name="max">{2*pi}</param>
+        </command_interface>
+        <command_interface name="velocity">
+            <param name="min">-3.2</param>
+            <param name="max">3.2</param>
         </command_interface>
         <state_interface name="position">
@@ -121,10 +121,10 @@
       <joint name="${prefix}wrist_2_joint">
         <command_interface name="position">
-          <param name="min">{-2*pi}</param>
-          <param name="max">{2*pi}</param>
-        </command_interface>
-        <command_interface name="velocity">
-          <param name="min">-3.2</param>
-          <param name="max">3.2</param>
+            <param name="min">{-2*pi}</param>
+            <param name="max">{2*pi}</param>
+        </command_interface>
+        <command_interface name="velocity">
+            <param name="min">-3.2</param>
+            <param name="max">3.2</param>
         </command_interface>
         <state_interface name="position">
@@ -137,10 +137,10 @@
       <joint name="${prefix}wrist_3_joint">
         <command_interface name="position">
-          <param name="min">{-2*pi}</param>
-          <param name="max">{2*pi}</param>
-        </command_interface>
-        <command_interface name="velocity">
-          <param name="min">-3.2</param>
-          <param name="max">3.2</param>
+            <param name="min">{-2*pi}</param>
+            <param name="max">{2*pi}</param>
+        </command_interface>
+        <command_interface name="velocity">
+            <param name="min">-3.2</param>
+            <param name="max">3.2</param>
         </command_interface>
         <state_interface name="position">

File: CustomRobots/robot_arms/models/ur3/ur.urdf.xacro (robot description, xacro)
@@ -9,8 +9,12 @@
   <!-- parameters -->
   <xacro:arg name="prefix" default="" />
-  <xacro:arg name="joint_limit_params" default=""/>
-  <xacro:arg name="kinematics_params" default=""/>
-  <xacro:arg name="physical_params" default=""/>
-  <xacro:arg name="visual_params" default=""/>
+  <xacro:arg name="joint_limit_params"
+            default="$(find custom_robots)/config/ur3/joint_limits.yaml"/>
+  <xacro:arg name="kinematics_params"
+            default="$(find custom_robots)/config/ur3/default_kinematics.yaml"/>
+  <xacro:arg name="physical_params"
+            default="$(find custom_robots)/config/ur3/physical_parameters.yaml"/>
+  <xacro:arg name="visual_params"
+            default="$(find custom_robots)/config/ur3/visual_parameters.yaml"/>
   <xacro:arg name="transmission_hw_interface" default=""/>
   <xacro:arg name="safety_limits" default="false"/>
@@ -52,9 +56,32 @@
       prefix="$(arg prefix)"
       parent="world"
+      joint_limits_parameters_file="$(arg joint_limit_params)"
+      kinematics_parameters_file="$(arg kinematics_params)"
+      physical_parameters_file="$(arg physical_params)"
+      visual_parameters_file="$(arg visual_params)"
+      transmission_hw_interface="$(arg transmission_hw_interface)"
+      safety_limits="$(arg safety_limits)"
+      safety_pos_margin="$(arg safety_pos_margin)"
+      safety_k_position="$(arg safety_k_position)"
+      use_fake_hardware="$(arg use_fake_hardware)"
+      fake_sensor_commands="$(arg fake_sensor_commands)"
+      sim_gazebo="$(arg sim_gazebo)"
+      sim_gz="$(arg sim_gz)"
+      headless_mode="$(arg headless_mode)"
+      initial_positions="${load_yaml(initial_positions_file)}"
+      use_tool_communication="$(arg use_tool_communication)"
+      tool_voltage="$(arg tool_voltage)"
+      tool_parity="$(arg tool_parity)"
+      tool_baud_rate="$(arg tool_baud_rate)"
+      tool_stop_bits="$(arg tool_stop_bits)"
+      tool_rx_idle_chars="$(arg tool_rx_idle_chars)"
+      tool_tx_idle_chars="$(arg tool_tx_idle_chars)"
+      tool_device_name="$(arg tool_device_name)"
+      tool_tcp_port="$(arg tool_tcp_port)"
       robot_ip="$(arg robot_ip)"
       script_filename="$(arg script_filename)"
       output_recipe_filename="$(arg output_recipe_filename)"
       input_recipe_filename="$(arg input_recipe_filename)">
-    <origin xyz="0 0 0" rpy="0 0 0"/>
+      <origin xyz="0 0 0" rpy="0 0 0"/>
   </xacro:ur_robot>
   <!-- Gazebo Classic -->

File: CustomRobots/robot_arms/models/ur3/ur3.urdf.xacro (robot description, xacro)
@@ -29,45 +29,14 @@
   <xacro:include filename="$(find custom_robots)/models/ur3/ur.urdf.xacro"/>
   <xacro:include filename="$(find custom_robots)/models/ur3/ur.ros2_control.xacro"/>
+  <!-- Include XACRO-MACRO file of the Robotiq 2f-85: -->
   <xacro:include filename="$(find robotiq_description)/urdf/robotiq_85_gripper.urdf.xacro"/>
   <xacro:include filename="$(find robotiq_description)/urdf/robotiq_85_gripper.ros2_control.xacro"/>
-  <!-- UR3 -->
-  <xacro:ur_robot
-    name="ur3"
-    tf_prefix=""
-  />
-  <!-- Coupler -->
-  <link name="robotiq_coupler">
-    <visual>
-      <geometry>
-        <mesh filename="package://robotiq_description/meshes/robotiq_85_coupler.stl"/>
-      </geometry>
-    </visual>
-    <collision>
-      <geometry>
-        <cylinder radius="0.04" length="0.015"/>
-      </geometry>
-    </collision>
-  </link>
-  <joint name="robotiq_coupler_joint" type="fixed">
-    <origin xyz="0 0 0.004" rpy="0 0 ${-pi/2.0}"/>
-    <parent link="tool0"/>
-    <child link="robotiq_coupler"/>
-  </joint>
-  <!-- Gripper -->
-  <xacro:robotiq_85_gripper
-    prefix=""
-    parent="robotiq_coupler">
-    <origin xyz="0 0 0.004"
-            rpy="0 ${-pi/2} ${pi}"/>
-  </xacro:robotiq_85_gripper>
-  <!-- ros2_control GRIPPER -->
-  <xacro:robotiq_85_ros2_control
-    name="robotiq"
-    prefix=""
-    sim_gz="true"
-    use_fake_hardware="false"/>
+  <xacro:include filename="$(find ros2srrc_endeffectors)/robotiq_2f85/urdf/robotiq_2f85_macro.urdf.xacro"/>
+  <xacro:robotiq_2f85
+    bringup="false"
+    parent_link="tool0"/>
   <!-- ros2_control UR3 -->
   <xacro:ur_ros2_control
-    name="ur3"
+    name="ur"
     prefix=""
     sim_gz="true"
