Commit message: Change stack

File: CustomRobots/robot_arms/models/ur3/ur_macro.xacro (robot description, xacro)
@@ -1,6 +1,8 @@
 <?xml version="1.0"?>
-<robot xmlns:xacro="http://wiki.ros.org/xacro">
-  <xacro:include filename="$(find custom_robots)/models/ur3/inc/ur_transmissions.xacro" />
-  <xacro:include filename="$(find custom_robots)/models/ur3/inc/ur_common.xacro" />
+<robot xmlns:xacro="http://ros.org/wiki/xacro">
+  <!-- Include UR3 ROBOT SPECIFICATIONS: -->
+  <xacro:include filename="$(find custom_robots)/models/ur3/inc/ur_transmissions.xacro"/>
+  <xacro:include filename="$(find custom_robots)/models/ur3/inc/ur_common.xacro"/>
+  <!-- XACRO-MACRO of UR3: -->
   <xacro:macro name="ur_robot" params="
     name
@@ -11,15 +13,75 @@
     kinematics_parameters_file
     physical_parameters_file
-    visual_parameters_file transmission_hw_interface:=hardware_interface/PositionJointInterface safety_limits:=false safety_pos_margin:=0.15 safety_k_position:=20 use_fake_hardware:=false fake_sensor_commands:=false sim_gazebo:=false sim_gz:=false headless_mode:=false initial_positions:=${dict(shoulder_pan_joint=0.0,shoulder_lift_joint=-1.57,elbow_joint=0.0,wrist_1_joint=-1.57,wrist_2_joint=0.0,wrist_3_joint=0.0)} use_tool_communication:=false tool_voltage:=24 tool_parity:=0 tool_baud_rate:=115200 tool_stop_bits:=1 tool_rx_idle_chars:=1.5 tool_tx_idle_chars:=3.5 tool_device_name:=/tmp/ttyUR tool_tcp_port:=54321 robot_ip:=0.0.0.0 script_filename:=to_be_filled_by_ur_robot_driver output_recipe_filename:=to_be_filled_by_ur_robot_driver input_recipe_filename:=to_be_filled_by_ur_robot_driver reverse_port:=50001 script_sender_port:=50002">
-    <!-- Load configuration data from the provided .yaml files -->
-    <xacro:read_model_data joint_limits_parameters_file="${joint_limits_parameters_file}" kinematics_parameters_file="${kinematics_parameters_file}" physical_parameters_file="${physical_parameters_file}" visual_parameters_file="${visual_parameters_file}" force_abs_paths="${sim_gazebo or sim_gz}"/>
+    visual_parameters_file
+    transmission_hw_interface:=hardware_interface/PositionJointInterface
+    safety_limits:=false
+    safety_pos_margin:=0.15
+    safety_k_position:=20
+    use_fake_hardware:=false
+    fake_sensor_commands:=false
+    sim_gazebo:=false
+    sim_gz:=false
+    headless_mode:=false
+    initial_positions:=${dict(
+        shoulder_pan_joint=0.0,
+        shoulder_lift_joint=-1.57,
+        elbow_joint=0.0,
+        wrist_1_joint=-1.57,
+        wrist_2_joint=0.0,
+        wrist_3_joint=0.0)}
+    use_tool_communication:=false
+    tool_voltage:=24
+    tool_parity:=0
+    tool_baud_rate:=115200
+    tool_stop_bits:=1
+    tool_rx_idle_chars:=1.5
+    tool_tx_idle_chars:=3.5
+    tool_device_name:=/tmp/ttyUR
+    tool_tcp_port:=54321
+    robot_ip:=0.0.0.0
+    script_filename:=to_be_filled_by_ur_robot_driver
+    output_recipe_filename:=to_be_filled_by_ur_robot_driver
+    input_recipe_filename:=to_be_filled_by_ur_robot_driver
+    reverse_port:=50001
+    script_sender_port:=50002">
+    <!-- LOAD UR3-Common: -->
+    <xacro:read_model_data
+        joint_limits_parameters_file="${joint_limits_parameters_file}"
+        kinematics_parameters_file="${kinematics_parameters_file}"
+        physical_parameters_file="${physical_parameters_file}"
+        visual_parameters_file="${visual_parameters_file}"
+        force_abs_paths="${sim_gazebo or sim_gz}"/>
     <!-- ros2 control include -->
     <xacro:include filename="$(find custom_robots)/models/ur3/ur.ros2_control.xacro" />
     <!-- ros2 control instance -->
-    <xacro:ur_ros2_control name="${name}" prefix="${prefix}" use_fake_hardware="${use_fake_hardware}" initial_positions="${initial_positions}" fake_sensor_commands="${fake_sensor_commands}" headless_mode="${headless_mode}" sim_gazebo="${sim_gazebo}" sim_gz="${sim_gz}" script_filename="${script_filename}" output_recipe_filename="${output_recipe_filename}" input_recipe_filename="${input_recipe_filename}" tf_prefix="" hash_kinematics="${kinematics_hash}" robot_ip="${robot_ip}" use_tool_communication="${use_tool_communication}" tool_voltage="${tool_voltage}" tool_parity="${tool_parity}" tool_baud_rate="${tool_baud_rate}" tool_stop_bits="${tool_stop_bits}" tool_rx_idle_chars="${tool_rx_idle_chars}" tool_tx_idle_chars="${tool_tx_idle_chars}" tool_device_name="${tool_device_name}" tool_tcp_port="${tool_tcp_port}" reverse_port="${reverse_port}" script_sender_port="${script_sender_port}" />
-    <!-- Add URDF transmission elements (for ros_control) -->
-    <!--<xacro:ur_arm_transmission prefix="${prefix}" hw_interface="${transmission_hw_interface}" />-->
-    <!-- Placeholder for ros2_control transmission which don't yet exist -->
-    <!-- links -  main serial chain -->
+    <xacro:ur_ros2_control
+    name="${name}"
+    prefix="${prefix}"
+    use_fake_hardware="${use_fake_hardware}"
+    initial_positions="${initial_positions}"
+    fake_sensor_commands="${fake_sensor_commands}"
+    headless_mode="${headless_mode}"
+    sim_gazebo="${sim_gazebo}"
+    sim_gz="${sim_gz}"
+    script_filename="${script_filename}"
+    output_recipe_filename="${output_recipe_filename}"
+    input_recipe_filename="${input_recipe_filename}"
+    tf_prefix=""
+    hash_kinematics="${kinematics_hash}"
+    robot_ip="${robot_ip}"
+    use_tool_communication="${use_tool_communication}"
+    tool_voltage="${tool_voltage}"
+    tool_parity="${tool_parity}"
+    tool_baud_rate="${tool_baud_rate}"
+    tool_stop_bits="${tool_stop_bits}"
+    tool_rx_idle_chars="${tool_rx_idle_chars}"
+    tool_tx_idle_chars="${tool_tx_idle_chars}"
+    tool_device_name="${tool_device_name}"
+    tool_tcp_port="${tool_tcp_port}"
+    reverse_port="${reverse_port}"
+    script_sender_port="${script_sender_port}"
+    />
+    <!-- ***** UR3 ROBOT .urdf SERIAL CHAIN ***** -->
+    <!-- Links: -->
     <link name="${prefix}base_link"/>
     <link name="${prefix}base_link_inertia">
@@ -27,11 +89,11 @@
         <origin xyz="0 0 0" rpy="0 0 ${pi}"/>
         <geometry>
-          <xacro:get_mesh name="base" type="visual"/>
-        </geometry>
-      </visual>
-      <collision>
-        <origin xyz="0 0 0" rpy="0 0 0" />
-        <geometry>
-          <cylinder radius="${base_inertia_radius}" length="${base_inertia_length}"/>
+          <mesh filename="file://$(find ros2srrc_robots)/ur3/meshes/visual/base.dae"/>
+        </geometry>
+      </visual>
+      <collision>
+        <origin xyz="0 0 0" rpy="0 0 ${pi}"/>
+        <geometry>
+          <mesh filename="file://$(find ros2srrc_robots)/ur3/meshes/collision/base.stl"/>
         </geometry>
       </collision>
@@ -44,11 +106,11 @@
         <origin xyz="0 0 0" rpy="0 0 ${pi}"/>
         <geometry>
-          <xacro:get_mesh name="shoulder" type="visual"/>
-        </geometry>
-      </visual>
-      <collision>
-        <origin xyz="0 0 0" rpy="0 0 0" />
-        <geometry>
-          <cylinder radius="${shoulder_inertia_radius}" length="${shoulder_inertia_length}"/>
+          <mesh filename="file://$(find ros2srrc_robots)/ur3/meshes/visual/shoulder.dae"/>
+        </geometry>
+      </visual>
+      <collision>
+        <origin xyz="0 0 0" rpy="0 0 ${pi}"/>
+        <geometry>
+          <mesh filename="file://$(find ros2srrc_robots)/ur3/meshes/collision/shoulder.stl"/>
         </geometry>
       </collision>
@@ -61,11 +123,11 @@
         <origin xyz="0 0 ${shoulder_offset}" rpy="${pi/2} 0 ${-pi/2}"/>
         <geometry>
-          <xacro:get_mesh name="upper_arm" type="visual"/>
-        </geometry>
-      </visual>
-      <collision>
-        <origin xyz="${-0.5 * upperarm_inertia_length} 0.0 ${upper_arm_inertia_offset}" rpy="0 ${pi/2} 0" />
-        <geometry>
-          <cylinder radius="${upperarm_inertia_radius}" length="${upperarm_inertia_length}"/>
+          <mesh filename="file://$(find ros2srrc_robots)/ur3/meshes/visual/upperarm.dae"/>
+        </geometry>
+      </visual>
+      <collision>
+        <origin xyz="0 0 ${shoulder_offset}" rpy="${pi/2} 0 ${-pi/2}"/>
+        <geometry>
+          <mesh filename="file://$(find ros2srrc_robots)/ur3/meshes/collision/upperarm.stl"/>
         </geometry>
       </collision>
@@ -78,78 +140,74 @@
         <origin xyz="0 0 ${elbow_offset}" rpy="${pi/2} 0 ${-pi/2}"/>
         <geometry>
-          <xacro:get_mesh name="forearm" type="visual"/>
-        </geometry>
-      </visual>
-      <collision>
+          <mesh filename="file://$(find ros2srrc_robots)/ur3/meshes/visual/forearm.dae"/>
+        </geometry>
+      </visual>
+      <collision>
+        <origin xyz="0 0 ${elbow_offset}" rpy="${pi/2} 0 ${-pi/2}"/>
+        <geometry>
+          <mesh filename="file://$(find ros2srrc_robots)/ur3/meshes/collision/forearm.stl"/>
+        </geometry>
+      </collision>
+      <xacro:cylinder_inertial radius="${forearm_inertia_radius}" length="${forearm_inertia_length}"  mass="${forearm_mass}">
         <origin xyz="${-0.5 * forearm_inertia_length} 0.0 ${elbow_offset}" rpy="0 ${pi/2} 0" />
-        <geometry>
-          <cylinder radius="${forearm_inertia_radius}" length="${forearm_inertia_length}"/>
-        </geometry>
-      </collision>
-      <xacro:cylinder_inertial radius="${forearm_inertia_radius}" length="${forearm_inertia_length}" mass="${forearm_mass}">
-        <origin xyz="${-0.5 * forearm_inertia_length} 0.0 ${elbow_offset}" rpy="0 ${pi/2} 0" />
       </xacro:cylinder_inertial>
     </link>
     <link name="${prefix}wrist_1_link">
-      <xacro:get_visual_params name="wrist_1" type="visual_offset"/>
-      <visual>
-        <origin xyz="0 0 ${visual_params}" rpy="${pi/2} 0 0"/>
-        <geometry>
-          <xacro:get_mesh name="wrist_1" type="visual"/>
-        </geometry>
-      </visual>
-      <collision>
+      <visual>
+        <origin xyz="0 0 ${wrist_1_visual_offset}" rpy="${pi/2} 0 0"/>
+        <geometry>
+          <mesh filename="file://$(find ros2srrc_robots)/ur3/meshes/visual/wrist1.dae"/>
+        </geometry>
+      </visual>
+      <collision>
+        <origin xyz="0 0 ${wrist_1_visual_offset}" rpy="${pi/2} 0 0"/>
+        <geometry>
+          <mesh filename="file://$(find ros2srrc_robots)/ur3/meshes/collision/wrist1.stl"/>
+        </geometry>
+      </collision>
+      <xacro:cylinder_inertial radius="${wrist_1_inertia_radius}" length="${wrist_1_inertia_length}"  mass="${wrist_1_mass}">
         <origin xyz="0 0 0" rpy="0 0 0" />
-        <geometry>
-          <cylinder radius="${wrist_1_inertia_radius}" length="${wrist_1_inertia_length}"/>
-        </geometry>
-      </collision>
-      <xacro:cylinder_inertial radius="${wrist_1_inertia_radius}" length="${wrist_1_inertia_length}" mass="${wrist_1_mass}">
+      </xacro:cylinder_inertial>
+    </link>
+    <link name="${prefix}wrist_2_link">
+      <visual>
+        <origin xyz="0 0 ${wrist_2_visual_offset}" rpy="0 0 0"/>
+        <geometry>
+          <mesh filename="file://$(find ros2srrc_robots)/ur3/meshes/visual/wrist2.dae"/>
+        </geometry>
+      </visual>
+      <collision>
+        <origin xyz="0 0 ${wrist_2_visual_offset}" rpy="0 0 0"/>
+        <geometry>
+          <mesh filename="file://$(find ros2srrc_robots)/ur3/meshes/collision/wrist2.stl"/>
+        </geometry>
+      </collision>
+      <xacro:cylinder_inertial radius="${wrist_2_inertia_radius}" length="${wrist_2_inertia_length}"  mass="${wrist_2_mass}">
         <origin xyz="0 0 0" rpy="0 0 0" />
       </xacro:cylinder_inertial>
     </link>
-    <link name="${prefix}wrist_2_link">
-      <xacro:get_visual_params name="wrist_2" type="visual_offset"/>
-      <visual>
-        <origin xyz="0 0 ${visual_params}" rpy="0 0 0"/>
-        <geometry>
-          <xacro:get_mesh name="wrist_2" type="visual"/>
-        </geometry>
-      </visual>
-      <collision>
-        <origin xyz="0 0 0" rpy="0 0 0" />
-        <geometry>
-          <cylinder radius="${wrist_2_inertia_radius}" length="${wrist_2_inertia_length}"/>
-        </geometry>
-      </collision>
-      <xacro:cylinder_inertial radius="${wrist_2_inertia_radius}" length="${wrist_2_inertia_length}" mass="${wrist_2_mass}">
-        <origin xyz="0 0 0" rpy="0 0 0" />
-      </xacro:cylinder_inertial>
-    </link>
     <link name="${prefix}wrist_3_link">
-      <xacro:get_visual_params name="wrist_3" type="visual_offset"/>
-      <visual>
-        <origin xyz="0 0 ${visual_params}" rpy="${pi/2} 0 0"/>
-        <geometry>
-          <xacro:get_mesh name="wrist_3" type="visual"/>
-        </geometry>
-      </visual>
-      <collision>
+      <visual>
+        <origin xyz="0 0 ${wrist_3_visual_offset}" rpy="${pi/2} 0 0"/>
+        <geometry>
+          <mesh filename="file://$(find ros2srrc_robots)/ur3/meshes/visual/wrist3.dae"/>
+        </geometry>
+      </visual>
+      <collision>
+        <origin xyz="0 0 ${wrist_3_visual_offset}" rpy="${pi/2} 0 0"/>
+        <geometry>
+          <mesh filename="file://$(find ros2srrc_robots)/ur3/meshes/collision/wrist3.stl"/>
+        </geometry>
+      </collision>
+      <xacro:cylinder_inertial radius="${wrist_3_inertia_radius}" length="${wrist_3_inertia_length}"  mass="${wrist_3_mass}">
         <origin xyz="0.0 0.0 ${-0.5 * wrist_3_inertia_length}" rpy="0 0 0" />
-        <geometry>
-          <cylinder radius="${wrist_3_inertia_radius}" length="${wrist_3_inertia_length}"/>
-        </geometry>
-      </collision>
-      <xacro:cylinder_inertial radius="${wrist_3_inertia_radius}" length="${wrist_3_inertia_length}" mass="${wrist_3_mass}">
-        <origin xyz="0.0 0.0 ${-0.5 * wrist_3_inertia_length}" rpy="0 0 0" />
-      </xacro:cylinder_inertial>
-    </link>
-    <!-- base_joint fixes base_link to the environment -->
+      </xacro:cylinder_inertial>
+    </link>
+    <!-- Joints: -->
     <joint name="${prefix}base_joint" type="fixed">
-      <xacro:insert_block name="origin" />
-      <parent link="${parent}" />
-      <child link="${prefix}base_link" />
-    </joint>
-    <!-- joints - main serial chain -->
+        <xacro:insert_block name="origin" />
+        <parent link="${parent}" />
+        <child link="${prefix}base_link" />
+    </joint>
     <joint name="${prefix}base_link-base_link_inertia" type="fixed">
       <parent link="${prefix}base_link" />
@@ -167,9 +225,7 @@
       <origin xyz="${shoulder_x} ${shoulder_y} ${shoulder_z}" rpy="${shoulder_roll} ${shoulder_pitch} ${shoulder_yaw}" />
       <axis xyz="0 0 1" />
-      <limit lower="${shoulder_pan_lower_limit}" upper="${shoulder_pan_upper_limit}" effort="${shoulder_pan_effort_limit}" velocity="${shoulder_pan_velocity_limit}"/>
-      <xacro:if value="${safety_limits}">
-        <safety_controller soft_lower_limit="${shoulder_pan_lower_limit + safety_pos_margin}" soft_upper_limit="${shoulder_pan_upper_limit - safety_pos_margin}" k_position="${safety_k_position}" k_velocity="0.0"/>
-      </xacro:if>
-      <dynamics damping="0" friction="0"/>
+      <limit lower="${shoulder_pan_lower_limit}" upper="${shoulder_pan_upper_limit}"
+        effort="${shoulder_pan_effort_limit}" velocity="${shoulder_pan_velocity_limit}"/>
+      <dynamics damping="1.0" friction="100.0"/>
     </joint>
     <joint name="${prefix}shoulder_lift_joint" type="revolute">
@@ -178,9 +234,7 @@
       <origin xyz="${upper_arm_x} ${upper_arm_y} ${upper_arm_z}" rpy="${upper_arm_roll} ${upper_arm_pitch} ${upper_arm_yaw}" />
       <axis xyz="0 0 1" />
-      <limit lower="${shoulder_lift_lower_limit}" upper="${shoulder_lift_upper_limit}" effort="${shoulder_lift_effort_limit}" velocity="${shoulder_lift_velocity_limit}"/>
-      <xacro:if value="${safety_limits}">
-        <safety_controller soft_lower_limit="${shoulder_lift_lower_limit + safety_pos_margin}" soft_upper_limit="${shoulder_lift_upper_limit - safety_pos_margin}" k_position="${safety_k_position}" k_velocity="0.0"/>
-      </xacro:if>
-      <dynamics damping="0" friction="0"/>
+      <limit lower="${shoulder_lift_lower_limit}" upper="${shoulder_lift_upper_limit}"
+        effort="${shoulder_lift_effort_limit}" velocity="${shoulder_lift_velocity_limit}"/>
+      <dynamics damping="1.0" friction="100.0"/>
     </joint>
     <joint name="${prefix}elbow_joint" type="revolute">
@@ -189,9 +243,7 @@
       <origin xyz="${forearm_x} ${forearm_y} ${forearm_z}" rpy="${forearm_roll} ${forearm_pitch} ${forearm_yaw}" />
       <axis xyz="0 0 1" />
-      <limit lower="${elbow_joint_lower_limit}" upper="${elbow_joint_upper_limit}" effort="${elbow_joint_effort_limit}" velocity="${elbow_joint_velocity_limit}"/>
-      <xacro:if value="${safety_limits}">
-        <safety_controller soft_lower_limit="${elbow_joint_lower_limit + safety_pos_margin}" soft_upper_limit="${elbow_joint_upper_limit - safety_pos_margin}" k_position="${safety_k_position}" k_velocity="0.0"/>
-      </xacro:if>
-      <dynamics damping="0" friction="0"/>
+      <limit lower="${elbow_joint_lower_limit}" upper="${elbow_joint_upper_limit}"
+        effort="${elbow_joint_effort_limit}" velocity="${elbow_joint_velocity_limit}"/>
+      <dynamics damping="1.0" friction="100.0"/>
     </joint>
     <joint name="${prefix}wrist_1_joint" type="revolute">
@@ -200,9 +252,7 @@
       <origin xyz="${wrist_1_x} ${wrist_1_y} ${wrist_1_z}" rpy="${wrist_1_roll} ${wrist_1_pitch} ${wrist_1_yaw}" />
       <axis xyz="0 0 1" />
-      <limit lower="${wrist_1_lower_limit}" upper="${wrist_1_upper_limit}" effort="${wrist_1_effort_limit}" velocity="${wrist_1_velocity_limit}"/>
-      <xacro:if value="${safety_limits}">
-        <safety_controller soft_lower_limit="${wrist_1_lower_limit + safety_pos_margin}" soft_upper_limit="${wrist_1_upper_limit - safety_pos_margin}" k_position="${safety_k_position}" k_velocity="0.0"/>
-      </xacro:if>
-      <dynamics damping="0" friction="0"/>
+      <limit lower="${wrist_1_lower_limit}" upper="${wrist_1_upper_limit}"
+        effort="${wrist_1_effort_limit}" velocity="${wrist_1_velocity_limit}"/>
+      <dynamics damping="1.0" friction="10.0"/>
     </joint>
     <joint name="${prefix}wrist_2_joint" type="revolute">
@@ -211,9 +261,7 @@
       <origin xyz="${wrist_2_x} ${wrist_2_y} ${wrist_2_z}" rpy="${wrist_2_roll} ${wrist_2_pitch} ${wrist_2_yaw}" />
       <axis xyz="0 0 1" />
-      <limit lower="${wrist_2_lower_limit}" upper="${wrist_2_upper_limit}" effort="${wrist_2_effort_limit}" velocity="${wrist_2_velocity_limit}"/>
-      <xacro:if value="${safety_limits}">
-        <safety_controller soft_lower_limit="${wrist_2_lower_limit + safety_pos_margin}" soft_upper_limit="${wrist_2_upper_limit - safety_pos_margin}" k_position="${safety_k_position}" k_velocity="0.0"/>
-      </xacro:if>
-      <dynamics damping="0" friction="0"/>
+      <limit lower="${wrist_2_lower_limit}" upper="${wrist_2_upper_limit}"
+             effort="${wrist_2_effort_limit}" velocity="${wrist_2_velocity_limit}"/>
+      <dynamics damping="1.0" friction="10.0"/>
     </joint>
     <joint name="${prefix}wrist_3_joint" type="revolute">
@@ -222,15 +270,13 @@
       <origin xyz="${wrist_3_x} ${wrist_3_y} ${wrist_3_z}" rpy="${wrist_3_roll} ${wrist_3_pitch} ${wrist_3_yaw}" />
       <axis xyz="0 0 1" />
-      <limit lower="${wrist_3_lower_limit}" upper="${wrist_3_upper_limit}" effort="${wrist_3_effort_limit}" velocity="${wrist_3_velocity_limit}"/>
-      <xacro:if value="${safety_limits}">
-        <safety_controller soft_lower_limit="${wrist_3_lower_limit + safety_pos_margin}" soft_upper_limit="${wrist_3_upper_limit - safety_pos_margin}" k_position="${safety_k_position}" k_velocity="0.0"/>
-      </xacro:if>
-      <dynamics damping="0" friction="0"/>
+      <limit lower="${wrist_3_lower_limit}" upper="${wrist_3_upper_limit}"
+             effort="${wrist_3_effort_limit}" velocity="${wrist_3_velocity_limit}"/>
+      <dynamics damping="1.0" friction="1.0"/>
     </joint>
     <link name="${prefix}ft_frame"/>
     <joint name="${prefix}wrist_3_link-ft_frame" type="fixed">
-      <parent link="${prefix}wrist_3_link"/>
-      <child link="${prefix}ft_frame"/>
-      <origin xyz="0 0 0" rpy="${pi} 0 0"/>
+        <parent link="${prefix}wrist_3_link"/>
+        <child link="${prefix}ft_frame"/>
+        <origin xyz="0 0 0" rpy="${pi} 0 0"/>
     </joint>
     <!-- ROS-Industrial 'base' frame - base_link to UR 'Base' Coordinates transform -->
@@ -263,7 +309,7 @@
     <link name="${prefix}ee_link" />
     <joint name="manipulator_dummy_joint" type="fixed">
-      <origin xyz="0 0 0.16" rpy="0 0 0" />
-      <parent link="${prefix}tool0"/>
-      <child link="${prefix}ee_link"/>
+        <origin xyz="0 0 0.16" rpy="0 0 0" />
+        <parent link="${prefix}tool0"/>
+        <child link="${prefix}ee_link"/>
     </joint>
   </xacro:macro>
