Commit message: Fix xacro

File: Industrial/ros2_SimRealRobotControl_gz/ros2srrc_endeffectors/robotiq_2f85/urdf/robotiq_2f85_macro.urdf.xacro (robot description, xacro)
@@ -145,6 +145,5 @@
       <axis xyz="0 0 1"/>
       <origin rpy="0 0 0" xyz="0.05490451627 -0.03060114443 0.0"/>
-      <limit lower="-0.05" upper="0.80285" velocity="0.5" effort="1000"/>
-      <dynamics damping="1.0" friction="1.0"/>
+      <mimic joint="robotiq_85_left_knuckle_joint" multiplier="1"/>
     </joint>
     <!-- Robotiq: left_finger -->
@@ -225,5 +224,5 @@
       <axis xyz="0 0 1"/>
       <origin xyz="0.06142 0.0127 0" rpy="${pi} 0.0 0.0" />
-      <limit lower="-0.05" upper="0.80285" velocity="0.5" effort="1000"/>
+      <mimic joint="robotiq_85_left_knuckle_joint" multiplier="1"/>
       <dynamics damping="1.0" friction="1.0"/>
     </joint>
@@ -253,5 +252,5 @@
       <axis xyz="0 0 1"/>
       <origin xyz="0.06142 -0.0127 0" rpy="0 0 0"/>
-      <limit lower="-0.05" upper="0.80285" velocity="0.5" effort="1000"/>
+      <mimic joint="robotiq_85_left_knuckle_joint" multiplier="1"/>
       <dynamics damping="1.0" friction="1.0"/>
     </joint>
@@ -283,5 +282,5 @@
       <axis xyz="0 0 1"/>
       <origin xyz="0.04303959807 -0.03759940821 0.0" rpy="0.0 0.0 0.0"/>
-      <limit lower="-0.80285" upper="0.05" velocity="0.5" effort="1000"/>
+      <mimic joint="robotiq_85_left_knuckle_joint" multiplier="-1"/>
       <dynamics damping="1.0" friction="1.0"/>
     </joint>
@@ -313,5 +312,5 @@
       <axis xyz="0 0 1"/>
       <origin rpy="0.0 0.0 0.0" xyz="0.04303959807 -0.03759940821  0.0"/>
-      <limit lower="-0.80285" upper="0.05" velocity="0.5" effort="1000"/>
+      <mimic joint="robotiq_85_left_knuckle_joint" multiplier="-1"/>
       <dynamics damping="1.0" friction="1.0"/>
     </joint>

Commit message: Try to fix gripper controller

File: Industrial/ros2_SimRealRobotControl_gz/ros2srrc_endeffectors/robotiq_2f85/urdf/robotiq_2f85_macro.urdf.xacro (robot description, xacro)
@@ -147,4 +147,5 @@
       <limit lower="-0.05" upper="0.80285" velocity="0.5" effort="1000"/>
       <dynamics damping="1.0" friction="1.0"/>
+      <mimic joint="robotiq_85_left_knuckle_joint" multiplier="1.0"/>
     </joint>
     <!-- Robotiq: left_finger -->
@@ -227,4 +228,5 @@
       <limit lower="-0.05" upper="0.80285" velocity="0.5" effort="1000"/>
       <dynamics damping="1.0" friction="1.0"/>
+      <mimic joint="robotiq_85_left_knuckle_joint" multiplier="1.0"/>
     </joint>
     <!-- Robotiq: right_inner_knuckle -->
@@ -255,4 +257,5 @@
       <limit lower="-0.05" upper="0.80285" velocity="0.5" effort="1000"/>
       <dynamics damping="1.0" friction="1.0"/>
+      <mimic joint="robotiq_85_left_knuckle_joint" multiplier="1.0"/>
     </joint>
     <!-- Robotiq: left_finger_tip -->
@@ -285,4 +288,5 @@
       <limit lower="-0.80285" upper="0.05" velocity="0.5" effort="1000"/>
       <dynamics damping="1.0" friction="1.0"/>
+      <mimic joint="robotiq_85_left_knuckle_joint" multiplier="-1.0"/>
     </joint>
     <!-- Robotiq: right_finger_tip -->
@@ -315,4 +319,5 @@
       <limit lower="-0.80285" upper="0.05" velocity="0.5" effort="1000"/>
       <dynamics damping="1.0" friction="1.0"/>
+      <mimic joint="robotiq_85_left_knuckle_joint" multiplier="-1.0"/>
     </joint>
     <!-- SMALL CUBE FOR GRIPPER PLUGIN -->

File: Industrial/ros2_SimRealRobotControl_gz/ros2srrc_endeffectors/robotiq_2f85/urdf/robotiq_2f85_ros2control.xacro (robot description, xacro)
@@ -1,41 +1,11 @@
 <?xml version="1.0"?>
-<!--
-# ===================================== COPYRIGHT ===================================== #
-#                                                                                       #
-#  IFRA (Intelligent Flexible Robotics and Assembly) Group, CRANFIELD UNIVERSITY        #
-#  Created on behalf of the IFRA Group at Cranfield University, United Kingdom          #
-#  E-mail: IFRA@cranfield.ac.uk                                                         #
-#                                                                                       #
-#  Licensed under the Apache-2.0 License.                                               #
-#  You may not use this file except in compliance with the License.                     #
-#  You may obtain a copy of the License at: http://www.apache.org/licenses/LICENSE-2.0  #
-#                                                                                       #
-#  Unless required by applicable law or agreed to in writing, software distributed      #
-#  under the License is distributed on an "as-is" basis, without warranties or          #
-#  conditions of any kind, either express or implied. See the License for the specific  #
-#  language governing permissions and limitations under the License.                    #
-#                                                                                       #
-#  IFRA Group - Cranfield University                                                    #
-#  AUTHORS: Mikel Bueno Viso - Mikel.Bueno-Viso@cranfield.ac.uk                         #
-#           Dr. Seemal Asif  - s.asif@cranfield.ac.uk                                   #
-#           Prof. Phil Webb  - p.f.webb@cranfield.ac.uk                                 #
-#                                                                                       #
-#  Date: April, 2023.                                                                   #
-#                                                                                       #
-# ===================================== COPYRIGHT ===================================== #
-# ======= CITE OUR WORK ======= #
-# You can cite our work with the following statement:
-# IFRA-Cranfield (2023) ROS 2 Sim-to-Real Robot Control. URL: https://github.com/IFRA-Cranfield/ros2_SimRealRobotControl.
--->
 <robot xmlns:xacro="http://www.ros.org/wiki/xacro">
+  <!-- ros2_control configuration for Robotiq 85 Gripper -->
   <xacro:macro name="EE_ros2control" params="" >
+    <!-- Main actuated joint -->
     <joint name="robotiq_85_left_knuckle_joint">
       <command_interface name="position">
-        <param name="min">-0.05</param>
+        <param name="min">0.0</param>
         <param name="max">0.80285</param>
-      </command_interface>
-      <command_interface name="velocity">
-        <param name="min">0.5</param>
-        <param name="max">0.5</param>
       </command_interface>
       <state_interface name="position">
@@ -45,79 +15,36 @@
       <state_interface name="effort"/>
     </joint>
+    <!-- Mimic joints - need to be included for proper state publishing -->
     <joint name="robotiq_85_right_knuckle_joint">
-      <command_interface name="position">
-        <param name="min">-0.05</param>
-        <param name="max">0.80285</param>
-      </command_interface>
-      <command_interface name="velocity">
-        <param name="min">0.5</param>
-        <param name="max">0.5</param>
-      </command_interface>
-      <state_interface name="position">
-        <param name="initial_value">0.0</param>
-      </state_interface>
+      <param name="mimic">robotiq_85_left_knuckle_joint</param>
+      <param name="multiplier">1.0</param>
+      <state_interface name="position"/>
       <state_interface name="velocity"/>
       <state_interface name="effort"/>
     </joint>
     <joint name="robotiq_85_left_inner_knuckle_joint">
-      <command_interface name="position">
-        <param name="min">-0.05</param>
-        <param name="max">0.80285</param>
-      </command_interface>
-      <command_interface name="velocity">
-        <param name="min">0.5</param>
-        <param name="max">0.5</param>
-      </command_interface>
-      <state_interface name="position">
-        <param name="initial_value">0.0</param>
-      </state_interface>
+      <param name="mimic">robotiq_85_left_knuckle_joint</param>
+      <param name="multiplier">1.0</param>
+      <state_interface name="position"/>
       <state_interface name="velocity"/>
-      <state_interface name="effort"/>
     </joint>
     <joint name="robotiq_85_right_inner_knuckle_joint">
-      <command_interface name="position">
-        <param name="min">-0.05</param>
-        <param name="max">0.80285</param>
-      </command_interface>
-      <command_interface name="velocity">
-        <param name="min">0.5</param>
-        <param name="max">0.5</param>
-      </command_interface>
-      <state_interface name="position">
-        <param name="initial_value">0.0</param>
-      </state_interface>
+      <param name="mimic">robotiq_85_left_knuckle_joint</param>
+      <param name="multiplier">1.0</param>
+      <state_interface name="position"/>
       <state_interface name="velocity"/>
-      <state_interface name="effort"/>
     </joint>
     <joint name="robotiq_85_left_finger_tip_joint">
-      <command_interface name="position">
-        <param name="min">-0.80285</param>
-        <param name="max">0.05</param>
-      </command_interface>
-      <command_interface name="velocity">
-        <param name="min">0.5</param>
-        <param name="max">0.5</param>
-      </command_interface>
-      <state_interface name="position">
-        <param name="initial_value">0.0</param>
-      </state_interface>
+      <param name="mimic">robotiq_85_left_knuckle_joint</param>
+      <param name="multiplier">-1.0</param>
+      <state_interface name="position"/>
       <state_interface name="velocity"/>
-      <state_interface name="effort"/>
     </joint>
     <joint name="robotiq_85_right_finger_tip_joint">
-      <command_interface name="position">
-        <param name="min">-0.80285</param>
-        <param name="max">0.05</param>
-      </command_interface>
-      <command_interface name="velocity">
-        <param name="min">0.5</param>
-        <param name="max">0.5</param>
-      </command_interface>
-      <state_interface name="position">
-        <param name="initial_value">0.0</param>
-      </state_interface>
+      <param name="mimic">robotiq_85_left_knuckle_joint</param>
+      <param name="multiplier">-1.0</param>
+      <state_interface name="position"/>
       <state_interface name="velocity"/>
-      <state_interface name="effort"/>
     </joint>
   </xacro:macro>
-</robot>
+  </robot>
