Commit message: Change xacro and ros2control for gripper

File: Industrial/ros2_SimRealRobotControl_gz/ros2srrc_endeffectors/robotiq_2f85/urdf/robotiq_2f85_macro.urdf.xacro (robot description, xacro)
@@ -1,74 +1,11 @@
 <?xml version="1.0"?>
-<!--
-# ===================================== COPYRIGHT ===================================== #
-#                                                                                       #
-#  IFRA (Intelligent Flexible Robotics and Assembly) Group, CRANFIELD UNIVERSITY        #
-#  Created on behalf of the IFRA Group at Cranfield University, United Kingdom          #
-#  E-mail: IFRA@cranfield.ac.uk                                                         #
-#                                                                                       #
-#  Licensed under the Apache-2.0 License.                                               #
-#  You may not use this file except in compliance with the License.                     #
-#  You may obtain a copy of the License at: http://www.apache.org/licenses/LICENSE-2.0  #
-#                                                                                       #
-#  Unless required by applicable law or agreed to in writing, software distributed      #
-#  under the License is distributed on an "as-is" basis, without warranties or          #
-#  conditions of any kind, either express or implied. See the License for the specific  #
-#  language governing permissions and limitations under the License.                    #
-#                                                                                       #
-#  IFRA Group - Cranfield University                                                    #
-#  AUTHORS: Mikel Bueno Viso - Mikel.Bueno-Viso@cranfield.ac.uk                         #
-#           Dr. Seemal Asif  - s.asif@cranfield.ac.uk                                   #
-#           Prof. Phil Webb  - p.f.webb@cranfield.ac.uk                                 #
-#                                                                                       #
-#  Date: April, 2023.                                                                   #
-#                                                                                       #
-# ===================================== COPYRIGHT ===================================== #
-# ======= CITE OUR WORK ======= #
-# You can cite our work with the following statement:
-# IFRA-Cranfield (2023) ROS 2 Sim-to-Real Robot Control. URL: https://github.com/IFRA-Cranfield/ros2_SimRealRobotControl.
--->
-<robot xmlns:xacro="http://ros.org/wiki/xacro">
-  <!-- XACRO-MACRO of Robotiq 2f-85: -->
-  <xacro:macro name="robotiq_2f85"
-                params="
-                bringup
-                parent_link
-                prefix:=">
-    <xacro:unless value="${bringup}">
-      <!-- Robotiq 2f-85 TRANSMISSION: -->
-      <xacro:include filename="$(find ros2srrc_endeffectors)/robotiq_2f85/urdf/robotiq_2f85_transmission.xacro" />
-      <xacro:robotiq_2f85_transmission />
-    </xacro:unless>
-    <!-- ***** Robotiq 2f-85 GRIPPER .urdf SERIAL CHAIN ***** -->
-    <!-- Robotiq: coupler -->
-    <link name="robotiq_coupler">
-      <visual>
-        <geometry>
-          <mesh filename="file://$(find ros2srrc_endeffectors)/robotiq_2f85/meshes/robotiq_85_coupler.stl" />
-        </geometry>
-      </visual>
-      <collision>
-        <geometry>
-          <mesh filename="file://$(find ros2srrc_endeffectors)/robotiq_2f85/meshes/robotiq_85_coupler.stl" />
-        </geometry>
-      </collision>
-      <inertial>
-        <origin xyz="2.073e-05   1.45286e-03  -1.1049e-03" rpy="0 0 0" />
-        <mass value="0.168" />
-        <inertia ixx="6.69695624e-05" ixy="5.21511788e-09" ixz="-2.74383009e-08"
-                iyy="7.85088161e-05" iyz="5.41105193e-07" izz="1.41819717e-04"/>
-      </inertial>
-    </link>
-    <joint name="robotiq_coupler_joint" type="fixed">
-      <origin xyz="0 0 0.004" rpy="0 0 ${-pi/2.0}" />
-      <parent link="${parent_link}"/>
-      <child link="robotiq_coupler"/>
-    </joint>
-    <gazebo reference="robotiq_coupler">
-      <mu1>0.9</mu1>
-      <mu2>0.9</mu2>
-      <material>Gazebo/Black</material>
-    </gazebo>
-    <!-- Robotiq: base_link -->
+<robot name="robotiq_85_gripper" xmlns:xacro="http://www.ros.org/wiki/xacro">
+  <xacro:include filename="$(find robotiq_description)/urdf/robotiq_85_gripper.transmission.xacro" />
+  <xacro:macro name="robotiq_85_gripper" params="prefix parent *origin">
+    <joint name="${prefix}robotiq_85_base_joint" type="fixed">
+      <parent link="${parent}"/>
+      <child link="${prefix}robotiq_85_base_link"/>
+      <xacro:insert_block name="origin"/>
+    </joint>
     <link name="${prefix}robotiq_85_base_link">
       <visual>
@@ -79,5 +16,5 @@
       <collision>
         <geometry>
-          <mesh filename="file://$(find ros2srrc_endeffectors)/robotiq_2f85/meshes/collision/robotiq_85_base_link.stl"/>
+          <cylinder radius="0.04" length="0.1"/>
         </geometry>
       </collision>
@@ -86,31 +23,6 @@
         <origin xyz="0.0 0.0 0.0" />
         <inertia ixx = "0.000380" ixy = "0.000000" ixz = "0.000000"
-            iyx = "0.000000" iyy = "0.001110" iyz = "0.000000"
-            izx = "0.000000" izy = "0.000000" izz = "0.001171" />
-      </inertial>
-    </link>
-    <joint name="${prefix}robotiq_85_base_joint" type="fixed">
-      <origin xyz="0 0 0.004" rpy="0 ${-pi/2} ${pi}"/>
-      <parent link="robotiq_coupler"/>
-      <child link="${prefix}robotiq_85_base_link"/>
-    </joint>
-    <!-- Robotiq: left_knuckle -->
-    <link name="${prefix}robotiq_85_left_knuckle_link">
-      <visual>
-        <geometry>
-          <mesh filename="file://$(find ros2srrc_endeffectors)/robotiq_2f85/meshes/visual/robotiq_85_knuckle_link.dae"/>
-        </geometry>
-      </visual>
-      <collision>
-        <geometry>
-          <mesh filename="file://$(find ros2srrc_endeffectors)/robotiq_2f85/meshes/collision/robotiq_85_knuckle_link.stl"/>
-        </geometry>
-      </collision>
-      <inertial>
-        <origin xyz="0 0 0" rpy="0 0 0"/>
-        <mass value="0.05"/>
-        <inertia ixx="5.4167e-06" ixy="0" ixz="0"
-                iyy="1.6667e-05" iyz="0"
-                izz="1.8750e-05"/>
+             iyx = "0.000000" iyy = "0.001110" iyz = "0.000000"
+             izx = "0.000000" izy = "0.000000" izz = "0.001171" />
       </inertial>
     </link>
@@ -121,8 +33,32 @@
       <origin rpy="${pi} 0.0 0.0" xyz="0.05490451627 0.03060114443 0.0"/>
       <limit lower="0.0" upper="0.80285" velocity="0.5" effort="1000"/>
-      <dynamics damping="1.0" friction="1.0"/>
-    </joint>
-    <!-- Robotiq: right_knuckle -->
-    <!-- Robotiq: right_knuckle -->
+    </joint>
+    <joint name="${prefix}robotiq_85_right_knuckle_joint" type="continuous">
+      <parent link="${prefix}robotiq_85_base_link"/>
+      <child link="${prefix}robotiq_85_right_knuckle_link"/>
+      <axis xyz="0 0 1"/>
+      <origin rpy="0.0 0.0 0.0" xyz="0.05490451627 -0.03060114443 0.0"/>
+      <limit lower="-3.14" upper="3.14" velocity="100.0" effort="1000"/>
+      <mimic joint="${prefix}robotiq_85_left_knuckle_joint" multiplier="1.0"/>
+    </joint>
+    <link name="${prefix}robotiq_85_left_knuckle_link">
+      <visual>
+        <geometry>
+          <mesh filename="file://$(find ros2srrc_endeffectors)/robotiq_2f85/meshes/visual/robotiq_85_knuckle_link.dae"/>
+        </geometry>
+      </visual>
+      <collision>
+        <geometry>
+          <box size="0.03 0.03 0.03"/>
+        </geometry>
+      </collision>
+      <inertial>
+        <mass value="0.018491" />
+        <origin xyz="0.0 0.0 0.0" />
+        <inertia ixx = "0.000009" ixy = "-0.000001" ixz = "0.000000"
+             iyx = "-0.000001" iyy = "0.000001" iyz = "0.000000"
+             izx = "0.000000" izy = "0.000000" izz = "0.000010" />
+      </inertial>
+    </link>
     <link name="${prefix}robotiq_85_right_knuckle_link">
       <visual>
@@ -133,42 +69,13 @@
       <collision>
         <geometry>
-          <mesh filename="file://$(find ros2srrc_endeffectors)/robotiq_2f85/meshes/collision/robotiq_85_knuckle_link.stl"/>
-        </geometry>
-      </collision>
-      <inertial>
-        <origin xyz="0 0 0" rpy="0 0 0"/>
-        <mass value="0.05"/>
-        <inertia ixx="5.4167e-06" ixy="0" ixz="0"
-                iyy="1.6667e-05" iyz="0"
-                izz="1.8750e-05"/>
-      </inertial>
-    </link>
-    <joint name="${prefix}robotiq_85_right_knuckle_joint" type="revolute">
-      <parent link="${prefix}robotiq_85_base_link"/>
-      <child link="${prefix}robotiq_85_right_knuckle_link"/>
-      <axis xyz="0 0 1"/>
-      <origin rpy="0 0 0" xyz="0.05490451627 -0.03060114443 0.0"/>
-      <limit lower="0.0" upper="0.80285" velocity="0.5" effort="1000"/>
-      <dynamics damping="1.0" friction="1.0"/>
-      <mimic joint="${prefix}robotiq_85_left_knuckle_joint" multiplier="1.0"/>
-    </joint>
-    <!-- Robotiq: left_finger -->
-    <link name="${prefix}robotiq_85_left_finger_link">
-      <visual>
-        <geometry>
-          <mesh filename="file://$(find ros2srrc_endeffectors)/robotiq_2f85/meshes/visual/robotiq_85_finger_link.dae"/>
-        </geometry>
-      </visual>
-      <collision>
-        <geometry>
-          <mesh filename="file://$(find ros2srrc_endeffectors)/robotiq_2f85/meshes/collision/robotiq_85_finger_link.stl"/>
-        </geometry>
-      </collision>
-      <inertial>
-        <mass value="0.027309" />
-        <origin xyz="0.0 0.0 0.0" />
-        <inertia ixx = "0.000003" ixy = "-0.000002" ixz = "0.000000"
-            iyx = "-0.000002" iyy = "0.000021" iyz = "0.000000"
-            izx = "0.000000" izy = "0.000000" izz = "0.000020" />
+          <box size="0.03 0.03 0.03"/>
+        </geometry>
+      </collision>
+      <inertial>
+        <mass value="0.018491" />
+        <origin xyz="0.0 0.0 0.0" />
+        <inertia ixx = "0.000009" ixy = "-0.000001" ixz = "0.000000"
+             iyx = "-0.000001" iyy = "0.000001" iyz = "0.000000"
+             izx = "0.000000" izy = "0.000000" izz = "0.000010" />
       </inertial>
     </link>
@@ -177,33 +84,64 @@
       <child link="${prefix}robotiq_85_left_finger_link"/>
       <origin xyz="-0.00408552455 -0.03148604435 0.0" rpy="0 0 0" />
-      <dynamics damping="1.0" friction="1.0"/>
-    </joint>
-    <!-- Robotiq: right_finger -->
-    <link name="${prefix}robotiq_85_right_finger_link">
-      <visual>
-        <geometry>
-          <mesh filename="file://$(find ros2srrc_endeffectors)/robotiq_2f85/meshes/visual/robotiq_85_finger_link.dae"/>
-        </geometry>
-      </visual>
-      <collision>
-        <geometry>
-          <mesh filename="file://$(find ros2srrc_endeffectors)/robotiq_2f85/meshes/collision/robotiq_85_finger_link.stl"/>
-        </geometry>
-      </collision>
-      <inertial>
-        <mass value="0.027309" />
-        <origin xyz="0.0 0.0 0.0" />
-        <inertia ixx = "0.000003" ixy = "-0.000002" ixz = "0.000000"
-            iyx = "-0.000002" iyy = "0.000021" iyz = "0.000000"
-            izx = "0.000000" izy = "0.000000" izz = "0.000020" />
-      </inertial>
-    </link>
+    </joint>
     <joint name="${prefix}robotiq_85_right_finger_joint" type="fixed">
       <parent link="${prefix}robotiq_85_right_knuckle_link"/>
       <child link="${prefix}robotiq_85_right_finger_link"/>
       <origin xyz="-0.00408552455 -0.03148604435 0.0" rpy="0 0 0" />
-      <dynamics damping="1.0" friction="1.0"/>
-    </joint>
-    <!-- Robotiq: left_inner_knuckle -->
+    </joint>
+    <link name="${prefix}robotiq_85_left_finger_link">
+      <visual>
+        <geometry>
+          <mesh filename="file://$(find ros2srrc_endeffectors)/robotiq_2f85/meshes/visual/robotiq_85_finger_link.dae"/>
+        </geometry>
+      </visual>
+      <collision>
+        <geometry>
+          <box size="0.03 0.03 0.03"/>
+        </geometry>
+      </collision>
+      <inertial>
+        <mass value="0.027309" />
+        <origin xyz="0.0 0.0 0.0" />
+        <inertia ixx = "0.000003" ixy = "-0.000002" ixz = "0.000000"
+             iyx = "-0.000002" iyy = "0.000021" iyz = "0.000000"
+             izx = "0.000000" izy = "0.000000" izz = "0.000020" />
+      </inertial>
+    </link>
+    <link name="${prefix}robotiq_85_right_finger_link">
+      <visual>
+        <geometry>
+          <mesh filename="file://$(find ros2srrc_endeffectors)/robotiq_2f85/meshes/visual/robotiq_85_finger_link.dae"/>
+        </geometry>
+      </visual>
+      <collision>
+        <geometry>
+          <box size="0.03 0.03 0.03"/>
+        </geometry>
+      </collision>
+      <inertial>
+        <mass value="0.027309" />
+        <origin xyz="0.0 0.0 0.0" />
+        <inertia ixx = "0.000003" ixy = "-0.000002" ixz = "0.000000"
+             iyx = "-0.000002" iyy = "0.000021" iyz = "0.000000"
+             izx = "0.000000" izy = "0.000000" izz = "0.000020" />
+      </inertial>
+    </link>
+    <joint name="${prefix}robotiq_85_left_inner_knuckle_joint" type="continuous">
+      <parent link="${prefix}robotiq_85_base_link"/>
+      <child link="${prefix}robotiq_85_left_inner_knuckle_link"/>
+      <axis xyz="0 0 1"/>
+      <origin xyz="0.06142 0.0127 0" rpy="${pi} 0.0 0.0" />
+      <limit lower="-3.14" upper="3.14" velocity="100.0" effort="0.1"/>
+      <mimic joint="${prefix}robotiq_85_left_knuckle_joint" offset="0"/>
+    </joint>
+    <joint name="${prefix}robotiq_85_right_inner_knuckle_joint" type="continuous">
+      <parent link="${prefix}robotiq_85_base_link"/>
+      <child link="${prefix}robotiq_85_right_inner_knuckle_link"/>
+      <axis xyz="0 0 1"/>
+      <origin xyz="0.06142 -0.0127 0" rpy="0 0 0"/>
+      <limit lower="-3.14" upper="3.14" velocity="100.0" effort="0.1"/>
+      <mimic joint="${prefix}robotiq_85_left_knuckle_joint" offset="0"/>
+    </joint>
     <link name="${prefix}robotiq_85_left_inner_knuckle_link">
       <visual>
@@ -214,5 +152,5 @@
       <collision>
         <geometry>
-          <mesh filename="file://$(find ros2srrc_endeffectors)/robotiq_2f85/meshes/collision/robotiq_85_inner_knuckle_link.stl"/>
+          <box size="0.03 0.03 0.03"/>
         </geometry>
       </collision>
@@ -221,18 +159,8 @@
         <origin xyz="0.0 0.0 0.0" />
         <inertia ixx = "0.000039" ixy = "0.000000" ixz = "0.000000"
-            iyx = "0.000000" iyy = "0.000005" iyz = "0.000000"
-            izx = "0.000000" izy = "0.000000" izz = "0.000035" />
-      </inertial>
-    </link>
-    <joint name="${prefix}robotiq_85_left_inner_knuckle_joint" type="continuous">
-      <parent link="${prefix}robotiq_85_base_link"/>
-      <child link="${prefix}robotiq_85_left_inner_knuckle_link"/>
-      <axis xyz="0 0 1"/>
-      <origin xyz="0.06142 0.0127 0" rpy="${pi} 0.0 0.0" />
-      <limit lower="-0.05" upper="0.80285" velocity="0.5" effort="1000"/>
-      <dynamics damping="1.0" friction="1.0"/>
-      <mimic joint="${prefix}robotiq_85_left_knuckle_joint" multiplier="1.0"/>
-    </joint>
-    <!-- Robotiq: right_inner_knuckle -->
+             iyx = "0.000000" iyy = "0.000005" iyz = "0.000000"
+             izx = "0.000000" izy = "0.000000" izz = "0.000035" />
+      </inertial>
+    </link>
     <link name="${prefix}robotiq_85_right_inner_knuckle_link">
       <visual>
@@ -243,5 +171,5 @@
       <collision>
         <geometry>
-          <mesh filename="file://$(find ros2srrc_endeffectors)/robotiq_2f85/meshes/collision/robotiq_85_inner_knuckle_link.stl"/>
+          <box size="0.03 0.03 0.03"/>
         </geometry>
       </collision>
@@ -250,37 +178,6 @@
         <origin xyz="0.0 0.0 0.0" />
         <inertia ixx = "0.000039" ixy = "0.000000" ixz = "0.000000"
-            iyx = "0.000000" iyy = "0.000005" iyz = "0.000000"
-            izx = "0.000000" izy = "0.000000" izz = "0.000035" />
-      </inertial>
-    </link>
-    <joint name="${prefix}robotiq_85_right_inner_knuckle_joint" type="continuous">
-      <parent link="${prefix}robotiq_85_base_link"/>
-      <child link="${prefix}robotiq_85_right_inner_knuckle_link"/>
-      <axis xyz="0 0 1"/>
-      <origin xyz="0.06142 -0.0127 0" rpy="0 0 0"/>
-      <limit lower="-0.05" upper="0.80285" velocity="0.5" effort="1000"/>
-      <dynamics damping="1.0" friction="1.0"/>
-      <mimic joint="${prefix}robotiq_85_left_knuckle_joint" multiplier="1.0"/>
-    </joint>
-    <!-- Robotiq: left_finger_tip -->
-    <link name="${prefix}robotiq_85_left_finger_tip_link">
-      <visual>
-        <geometry>
-          <mesh filename="file://$(find ros2srrc_endeffectors)/robotiq_2f85/meshes/visual/robotiq_85_finger_tip_link.dae"/>
-        </geometry>
-      </visual>
-      <collision>
-        <geometry>
-          <!-- DMM: se sustituye por una caja muy pequeña para evitar que las piezas salgan disparadas -->
-          <box size= "0.005 0.005 0.005" />
-          <!--<mesh filename="file://$(find ros2srrc_endeffectors)/robotiq_2f85/meshes/collision/robotiq_85_finger_tip_link.stl"/>-->
-        </geometry>
-      </collision>
-      <inertial>
-        <mass value="0.019555" />
-        <origin xyz="0.0 0.0 0.0" />
-        <inertia ixx = "0.000002" ixy = "0.000000" ixz = "0.000000"
-            iyx = "0.000000" iyy = "0.000005" iyz = "0.000000"
-            izx = "0.000000" izy = "0.000000" izz = "0.000006" />
+             iyx = "0.000000" iyy = "0.000005" iyz = "0.000000"
+             izx = "0.000000" izy = "0.000000" izz = "0.000035" />
       </inertial>
     </link>
@@ -290,30 +187,7 @@
       <axis xyz="0 0 1"/>
       <origin xyz="0.04303959807 -0.03759940821 0.0" rpy="0.0 0.0 0.0"/>
-      <limit lower="-0.80285" upper="0.05" velocity="0.5" effort="1000"/>
-      <dynamics damping="1.0" friction="1.0"/>
-      <mimic joint="${prefix}robotiq_85_left_knuckle_joint" multiplier="-1.0"/>
-    </joint>
-    <!-- Robotiq: right_finger_tip -->
-    <link name="${prefix}robotiq_85_right_finger_tip_link">
-      <visual>
-        <geometry>
-          <mesh filename="file://$(find ros2srrc_endeffectors)/robotiq_2f85/meshes/visual/robotiq_85_finger_tip_link.dae"/>
-        </geometry>
-      </visual>
-      <collision>
-        <geometry>
-          <!-- DMM: se sustituye por una caja muy pequeña para evitar que las piezas salgan disparadas -->
-          <box size= "0.005 0.005 0.005" />
-          <!--<mesh filename="file://$(find ros2srrc_endeffectors)/robotiq_2f85/meshes/collision/robotiq_85_finger_tip_link.stl"/>-->
-        </geometry>
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
File: Industrial/ros2_SimRealRobotControl_gz/ros2srrc_endeffectors/robotiq_2f85/urdf/robotiq_2f85_ros2control.xacro (robot description, xacro)
@@ -1,10 +1,10 @@
 <?xml version="1.0"?>
 <robot xmlns:xacro="http://www.ros.org/wiki/xacro">
-  <xacro:macro name="robotiq_2f85_ros2_control"
-                params="
-                name
-                prefix
-                sim_gz:=true
-                use_fake_hardware:=false">
+  <!-- ros2_control configuration for Robotiq 85 Gripper -->
+  <xacro:macro name="robotiq_85_ros2_control" params="
+    name
+    prefix
+    sim_gz:=false
+    use_fake_hardware:=false">
     <ros2_control name="${name}_gripper" type="system">
       <hardware>
@@ -14,7 +14,9 @@
         <xacro:if value="${use_fake_hardware}">
           <plugin>mock_components/GenericSystem</plugin>
+          <param name="fake_sensor_commands">false</param>
+          <param name="state_following_offset">0.0</param>
         </xacro:if>
       </hardware>
-      <!-- actuated joint -->
+      <!-- Main actuated joint -->
       <joint name="${prefix}robotiq_85_left_knuckle_joint">
         <command_interface name="position">
@@ -28,11 +30,11 @@
         <state_interface name="effort"/>
       </joint>
-      <!-- mimic joints -->
+      <!-- Mimic joints - need to be included for proper state publishing -->
       <joint name="${prefix}robotiq_85_right_knuckle_joint">
         <param name="mimic">${prefix}robotiq_85_left_knuckle_joint</param>
         <param name="multiplier">1.0</param>
         <command_interface name="position">
-            <param name="min">0.0</param>
-            <param name="max">0.80285</param>
+          <param name="min">0.0</param>
+          <param name="max">0.80285</param>
         </command_interface>
         <state_interface name="position"/>
@@ -44,6 +46,6 @@
         <param name="multiplier">1.0</param>
         <command_interface name="position">
-            <param name="min">0.0</param>
-            <param name="max">0.80285</param>
+          <param name="min">0.0</param>
+          <param name="max">0.80285</param>
         </command_interface>
         <state_interface name="position"/>
@@ -54,6 +56,6 @@
         <param name="multiplier">1.0</param>
         <command_interface name="position">
-            <param name="min">0.0</param>
-            <param name="max">0.80285</param>
+          <param name="min">0.0</param>
+          <param name="max">0.80285</param>
         </command_interface>
         <state_interface name="position"/>
@@ -64,6 +66,6 @@
         <param name="multiplier">-1.0</param>
         <command_interface name="position">
-            <param name="min">-0.80285</param>
-            <param name="max">0.0</param>
+          <param name="min">-0.80285</param>
+          <param name="max">0.0</param>
         </command_interface>
         <state_interface name="position"/>
@@ -74,6 +76,6 @@
         <param name="multiplier">-1.0</param>
         <command_interface name="position">
-            <param name="min">-0.80285</param>
-            <param name="max">0.0</param>
+          <param name="min">-0.80285</param>
+          <param name="max">0.0</param>
         </command_interface>
         <state_interface name="position"/>
@@ -82,3 +84,3 @@
     </ros2_control>
   </xacro:macro>
-</robot>
+  </robot>
