Commit message: feat(palletizing): add moveit rviz config, fix kinematics limits, update spawner and urdf

File: CustomRobots/robot_arms/models/ur10/ur10_suction.urdf.xacro (robot description, xacro)
@@ -24,6 +24,8 @@
     </inertial>
     <collision name="collision">
+      <!-- Dartsim cannot parse .dae meshes for collision geometry. Using a primitive box. -->
+      <origin xyz="0.03 0.0 0.05" rpy="0 0 0"/>
       <geometry>
-        <mesh filename="file://$(find ros2srrc_endeffectors)/ls_vgr/meshes/ls_vgr.dae"/>
+        <box size="0.1 0.1 0.1"/>
       </geometry>
     </collision>
@@ -75,5 +77,5 @@
       <update_rate>100</update_rate>
       <contact>
-        <collision>collision</collision>
+        <collision>ls_vgr_link_fixed_joint_lump__collision_collision</collision>
       </contact>
     </sensor>
