Commit message: Update rover_4wd

File: CustomRobots/rover_4wd/model/rover_4wd/rover_4wd.urdf.xacro (robot description, xacro)
@@ -11,5 +11,7 @@
   <xacro:property name="payload_z_offset" value="0.096" />
   <xacro:arg name="noise_level" default="none"/>
+  <xacro:arg name="namespace" default="rover_4wd"/>
   <xacro:property name="noise_level" value="$(arg noise_level)"/>
+  <xacro:property name="namespace" value="$(arg namespace)"/>
   <xacro:if value="${noise_level == 'low'}">
     <xacro:property name="a1" value="0.1" />
@@ -206,12 +208,12 @@
   </joint>
   <!-- ================== Gazebo Plugins ================== -->
-  <xacro:lidar xyz="0.174 0 0.10" rpy="0 0 0" name="lidar" parent="payload_link" topic="scan"/>
-  <xacro:imu xyz="0 0 0" rpy="0 0 0" parent="payload_link" topic="imu/data"/>
-  <xacro:velocity topic="/cmd_vel"/>
-  <xacro:joints topic="/joint_states"/>
-  <xacro:odom topic="/odom"/>
+  <xacro:lidar xyz="0.174 0 0.10" rpy="0 0 0" name="lidar" parent="payload_link" namespace="${namespace}"/>
+  <xacro:imu xyz="0 0 0" rpy="0 0 0" parent="payload_link" namespace="${namespace}"/>
+  <xacro:velocity namespace="${namespace}"/>
+  <xacro:joints namespace="${namespace}"/>
+  <xacro:odom namespace="${namespace}"/>
+  <xacro:pose namespace="${namespace}"/>
   <xacro:unless value="${noise_level == 'none'}">
-    <xacro:noise_odom topic="/odom_noisy" a1="${a1}" a2="${a2}" a3="${a3}" a4="${a4}"/>
+    <xacro:noise_odom namespace="${namespace}" a1="${a1}" a2="${a2}" a3="${a3}" a4="${a4}"/>
   </xacro:unless>
-  <xacro:pose/>
 </robot>

File: CustomRobots/rover_4wd/model/rover_4wd/rover_4wd_gz.urdf.xacro (robot description, xacro)
@@ -1,5 +1,5 @@
 <?xml version="1.0"?>
 <robot xmlns:xacro="http://ros.org/wiki/xacro">
-  <xacro:macro name="lidar" params="xyz rpy name parent topic">
+  <xacro:macro name="lidar" params="xyz rpy name parent namespace">
     <link name="${name}_link">
       <visual>
@@ -26,5 +26,5 @@
         <visualize>1</visualize>
         <update_rate>10</update_rate>
-        <topic>${topic}</topic>
+        <topic>/${namespace}/laser/scan</topic>
         <gz_frame_id>base_link</gz_frame_id>
         <lidar>
@@ -57,5 +57,5 @@
     </gazebo>
   </xacro:macro>
-  <xacro:macro name="imu" params="xyz rpy parent topic">
+  <xacro:macro name="imu" params="xyz rpy parent namespace">
     <link name="imu_link"/>
     <joint name="imu_to_payload" type="fixed">
@@ -69,5 +69,5 @@
         <update_rate>50</update_rate>
         <visualize>true</visualize>
-        <topic>${topic}</topic>
+        <topic>/${namespace}/imu</topic>
         <enable_metrics>true</enable_metrics>
         <frame_id>imu_link</frame_id>
@@ -78,5 +78,5 @@
     </gazebo>
   </xacro:macro>
-  <xacro:macro name="velocity" params="topic">
+  <xacro:macro name="velocity" params="namespace">
     <gazebo>
       <plugin name="gz::sim::systems::DiffDrive" filename="gz-sim-diff-drive-system">
@@ -98,18 +98,18 @@
         <child_frame_id>base_link</child_frame_id>
         <!-- Topics -->
-        <topic>${topic}</topic>
-        <odom_topic>/odometry/wheels</odom_topic>
-        <tf_topic>/tf_gazebo</tf_topic>
+        <topic>/${namespace}/cmd_vel</topic>
+        <odom_topic>/${namespace}/odometry/wheels</odom_topic>
+        <tf_topic>/${namespace}/tf</tf_topic>
       </plugin>
     </gazebo>
   </xacro:macro>
-  <xacro:macro name="joints" params="topic">
+  <xacro:macro name="joints" params="namespace">
     <gazebo>
       <plugin name="gz::sim::systems::JointStatePublisher" filename="gz-sim-joint-state-publisher-system">
-        <topic>${topic}</topic>
+        <topic>/${namespace}/joint_states</topic>
       </plugin>
     </gazebo>
   </xacro:macro>
-  <xacro:macro name="pose">
+  <xacro:macro name="pose" params="namespace">
     <gazebo>
       <plugin filename="gz-sim-pose-publisher-system" name="gz::sim::systems::PosePublisher">
@@ -118,21 +118,22 @@
         <publish_nested_model_pose>true</publish_nested_model_pose>
         <use_pose_vector_msg>true</use_pose_vector_msg>
+        <topic>/model/${namespace}/pose</topic>
       </plugin>
     </gazebo>
   </xacro:macro>
-  <xacro:macro name="odom" params="topic">
+  <xacro:macro name="odom" params="namespace">
     <gazebo>
       <plugin filename="gz-sim-odometry-publisher-system" name="gz::sim::systems::OdometryPublisher">
         <odom_frame>odom</odom_frame>
         <robot_base_frame>base_link</robot_base_frame>
-        <odom_topic>${topic}</odom_topic>
+        <odom_topic>/${namespace}/odom</odom_topic>
         <dimensions>3</dimensions>
       </plugin>
     </gazebo>
   </xacro:macro>
-  <xacro:macro name="noise_odom" params="vel_topic topic a1 a2 a3 a4">
+  <xacro:macro name="noise_odom" params="namespace a1 a2 a3 a4">
     <gazebo>
       <plugin filename="libNoisyOdometryPlugin.so" name="custom_plugins::NoisyOdometryPlugin">
-        <ros_topic>${topic}</ros_topic>
+        <ros_topic>/${namespace}/odom_noisy</ros_topic>
         <frame_id>odom</frame_id>
         <child_frame_id>base_link</child_frame_id>
