Commit message: fix end effector joint

File: CustomRobots/robot_arms/models/dobot_magician/dobot_magician_macro.xacro (robot description, xacro)
@@ -58,4 +58,11 @@
     </joint>
   </xacro:macro>
+  <!-- dartsim doesn't reliably enforce a plain URDF/SDF <mimic> constraint,
+       the gz_mimic_joint plugin drives these joints for real instead, one
+       plugin instance per pair, added in dobot_magician below. That plugin
+       just copies the parent joint's raw value, so these joints use a
+       flipped axis to get the same physical motion a -1 multiplier would
+       have given on the original axis, and the <mimic> tag below (still
+       needed for MoveIt's own planning-time state) uses +1 to match. -->
   <xacro:macro name="dobot_joint_mimic" params="joint_name type parent child axis_xyz origin_xyz origin_rpy lower_limit upper_limit ref_joint">
     <joint name="${joint_name}" type="${type}">
@@ -65,8 +72,6 @@
       <limit effort="2000" velocity="1" lower="${lower_limit}" upper="${upper_limit}"/>
       <origin xyz="${origin_xyz}" rpy="${origin_rpy}"/>
-      <!-- Damping here matters more than on the driven joints, it's what
-           settles the parallelogram constraint instead of oscillating -->
       <dynamics damping="1.0" friction="0"/>
-      <mimic joint="${ref_joint}" multiplier="-1" offset="0"/>
+      <mimic joint="${ref_joint}" multiplier="1" offset="0"/>
     </joint>
   </xacro:macro>
@@ -104,12 +109,12 @@
     <xacro:dobot_joint_mimic joint_name="${prefix}joint_mimic_1" type="revolute"
       parent="${prefix}link_3" child="${prefix}link_virtual"
-      axis_xyz="0 1 0" origin_xyz="${link_3_length} 0 0" origin_rpy="0 0 0"
-      lower_limit="0" upper_limit="${2*pi}" ref_joint="${prefix}joint_2"/>
+      axis_xyz="0 -1 0" origin_xyz="${link_3_length} 0 0" origin_rpy="0 0 0"
+      lower_limit="${-5.0/180.0*pi}" upper_limit="${90.0/180.0*pi}" ref_joint="${prefix}joint_2"/>
     <xacro:dobot_armlink link_name="${prefix}link_4" visual_mesh="magicianLink4" collision_mesh="link4_collision"
       base_origin_xyz="${parallelogram_origin_xyz}" base_origin_rpy="0 0 0" mass="0.1" box_x="0.03" box_y="0.03" box_z="0.06"/>
     <xacro:dobot_joint_mimic joint_name="${prefix}joint_mimic_2" type="revolute"
       parent="${prefix}link_virtual" child="${prefix}link_4"
-      axis_xyz="0 1 0" origin_xyz="0 0 0" origin_rpy="0 0 0"
-      lower_limit="0" upper_limit="${2*pi}" ref_joint="${prefix}joint_3"/>
+      axis_xyz="0 -1 0" origin_xyz="0 0 0" origin_rpy="0 0 0"
+      lower_limit="${-15.0/180.0*pi}" upper_limit="${70.0/180.0*pi}" ref_joint="${prefix}joint_3"/>
     <!-- Real actuated wrist rotation, last of the 4 DOF -->
     <xacro:property name="gripper_core_origin_xyz"
@@ -132,6 +137,22 @@
     <xacro:dobot_joint_mimic joint_name="${prefix}joint_prismatic_r" type="prismatic"
       parent="${prefix}link_gripper_core" child="${prefix}link_gripper_jaw_right"
-      axis_xyz="0 1 0" origin_xyz="0 0 0" origin_rpy="0 0 0"
-      lower_limit="-0.0135" upper_limit="0" ref_joint="${prefix}joint_prismatic_l"/>
+      axis_xyz="0 -1 0" origin_xyz="0 0 0" origin_rpy="0 0 0"
+      lower_limit="0" upper_limit="0.0135" ref_joint="${prefix}joint_prismatic_l"/>
+    <!-- Actively drives the 3 mimic joints above, dartsim doesn't honor
+         their <mimic> tag by itself -->
+    <gazebo>
+      <plugin filename="libgz_mimic_joint.so" name="gz_mimic_joint::MimicJoint">
+        <parent_joint>${prefix}joint_2</parent_joint>
+        <mimic_joint>${prefix}joint_mimic_1</mimic_joint>
+      </plugin>
+      <plugin filename="libgz_mimic_joint.so" name="gz_mimic_joint::MimicJoint">
+        <parent_joint>${prefix}joint_3</parent_joint>
+        <mimic_joint>${prefix}joint_mimic_2</mimic_joint>
+      </plugin>
+      <plugin filename="libgz_mimic_joint.so" name="gz_mimic_joint::MimicJoint">
+        <parent_joint>${prefix}joint_prismatic_l</parent_joint>
+        <mimic_joint>${prefix}joint_prismatic_r</mimic_joint>
+      </plugin>
+    </gazebo>
   </xacro:macro>
 </robot>

Commit message: finger collision

File: CustomRobots/robot_arms/models/dobot_magician/dobot_magician_macro.xacro (robot description, xacro)
@@ -35,4 +35,24 @@
         <geometry>
           <mesh filename="package://custom_robots/models/dobot_magician/meshes/collision/${collision_mesh}.stl"/>
+        </geometry>
+      </collision>
+      <xacro:box_inertial mass="${mass}" x="${box_x}" y="${box_y}" z="${box_z}"/>
+    </link>
+  </xacro:macro>
+  <!-- Same as dobot_armlink, but a box collision instead of a mesh one.
+       dartsim can't build a contact sensor's shape from a mesh, only the
+       jaws need this since only one of them carries the sensor. -->
+  <xacro:macro name="dobot_armlink_box_collision" params="link_name visual_mesh base_origin_xyz base_origin_rpy mass box_x box_y box_z collision_origin_xyz collision_size">
+    <link name="${link_name}">
+      <visual>
+        <origin xyz="${base_origin_xyz}" rpy="${base_origin_rpy}"/>
+        <geometry>
+          <mesh filename="package://custom_robots/models/dobot_magician/meshes/visual/${visual_mesh}.dae"/>
+        </geometry>
+      </visual>
+      <collision>
+        <origin xyz="${collision_origin_xyz}" rpy="${base_origin_rpy}"/>
+        <geometry>
+          <box size="${collision_size}"/>
         </geometry>
       </collision>
@@ -118,6 +138,10 @@
       lower_limit="${-15.0/180.0*pi}" upper_limit="${70.0/180.0*pi}" ref_joint="${prefix}joint_3"/>
     <!-- Real actuated wrist rotation, last of the 4 DOF -->
+    <xacro:property name="gripper_core_origin_x"
+      value="${-1*(link_2_length*sin(joint_2_offset)+link_3_length*cos(joint_2_offset+joint_3_offset)+link_4_length) + 0.23517+0.0019}"/>
+    <xacro:property name="gripper_core_origin_z"
+      value="${link_2_length-1*(link_2_length*cos(joint_2_offset)+link_3_length*sin(joint_2_offset+joint_3_offset)) + 0.0497517 - 0.003 - 0.016}"/>
     <xacro:property name="gripper_core_origin_xyz"
-      value="${-1*(link_2_length*sin(joint_2_offset)+link_3_length*cos(joint_2_offset+joint_3_offset)+link_4_length) + 0.23517+0.0019} 0 ${link_2_length-1*(link_2_length*cos(joint_2_offset)+link_3_length*sin(joint_2_offset+joint_3_offset)) + 0.0497517 - 0.003 - 0.016}"/>
+      value="${gripper_core_origin_x} 0 ${gripper_core_origin_z}"/>
     <xacro:dobot_armlink link_name="${prefix}link_gripper_core" visual_mesh="gripper_core" collision_mesh="gripper_core"
       base_origin_xyz="${gripper_core_origin_xyz}" base_origin_rpy="0 0 0" mass="0.1" box_x="0.05" box_y="0.05" box_z="0.05"/>
@@ -129,13 +153,17 @@
          Both meshes sit at the same origin at rest, with zero travel that's
          already fully closed, so the joints run negative (limit 0 at rest,
-         closed) to open, matching HAL's 0 percent is open convention. -->
-    <xacro:dobot_armlink link_name="${prefix}link_gripper_jaw_left" visual_mesh="jaw_left" collision_mesh="jaw_left"
-      base_origin_xyz="${gripper_core_origin_xyz}" base_origin_rpy="0 0 0" mass="0.02" box_x="0.02" box_y="0.01" box_z="0.05"/>
+         closed) to open, matching HAL's 0 percent is open convention.
+         Collision is a plain box instead of the finger mesh, dartsim can't
+         build the contact sensor's shape from a mesh. -->
+    <xacro:dobot_armlink_box_collision link_name="${prefix}link_gripper_jaw_left" visual_mesh="jaw_left"
+      base_origin_xyz="${gripper_core_origin_xyz}" base_origin_rpy="0 0 0" mass="0.02" box_x="0.02" box_y="0.01" box_z="0.05"
+      collision_origin_xyz="${gripper_core_origin_x - 0.01535} 0 ${gripper_core_origin_z - 0.049}" collision_size="0.045 0.032 0.056"/>
     <xacro:dobot_joint joint_name="${prefix}joint_prismatic_l" type="prismatic"
       parent="${prefix}link_gripper_core" child="${prefix}link_gripper_jaw_left"
       axis_xyz="0 -1 0" origin_xyz="0 0 0" origin_rpy="0 0 0"
       lower_limit="-0.018" upper_limit="0"/>
-    <xacro:dobot_armlink link_name="${prefix}link_gripper_jaw_right" visual_mesh="jaw_right" collision_mesh="jaw_right"
-      base_origin_xyz="${gripper_core_origin_xyz}" base_origin_rpy="0 0 0" mass="0.02" box_x="0.02" box_y="0.01" box_z="0.05"/>
+    <xacro:dobot_armlink_box_collision link_name="${prefix}link_gripper_jaw_right" visual_mesh="jaw_right"
+      base_origin_xyz="${gripper_core_origin_xyz}" base_origin_rpy="0 0 0" mass="0.02" box_x="0.02" box_y="0.01" box_z="0.05"
+      collision_origin_xyz="${gripper_core_origin_x - 0.01535} 0 ${gripper_core_origin_z - 0.049}" collision_size="0.045 0.032 0.056"/>
     <xacro:dobot_joint_mimic joint_name="${prefix}joint_prismatic_r" type="prismatic"
       parent="${prefix}link_gripper_core" child="${prefix}link_gripper_jaw_right"

Commit message: delete ik solver + code style

File: CustomRobots/robot_arms/models/dobot_magician/dobot_magician_macro.xacro (robot description, xacro)
@@ -78,11 +78,9 @@
     </joint>
   </xacro:macro>
-  <!-- dartsim doesn't reliably enforce a plain URDF/SDF <mimic> constraint,
-       the gz_mimic_joint plugin drives these joints for real instead, one
-       plugin instance per pair, added in dobot_magician below. That plugin
-       just copies the parent joint's raw value, so these joints use a
-       flipped axis to get the same physical motion a -1 multiplier would
-       have given on the original axis, and the <mimic> tag below (still
-       needed for MoveIt's own planning-time state) uses +1 to match. -->
+  <!-- dartsim doesn't apply a plain mimic constraint reliably, the
+       gz_mimic_joint plugin below drives these joints for real. It only
+       copies the parent's raw value, so the axis here is flipped to
+       match what a negative multiplier would have done, and the mimic
+       tag stays just for MoveIt's own state tracking. -->
   <xacro:macro name="dobot_joint_mimic" params="joint_name type parent child axis_xyz origin_xyz origin_rpy lower_limit upper_limit ref_joint">
     <joint name="${joint_name}" type="${type}">
@@ -151,9 +149,7 @@
       lower_limit="${-150.0/180.0*pi}" upper_limit="${150.0/180.0*pi}"/>
     <!-- Gripper jaws, joint_prismatic_l drives, joint_prismatic_r mimics it.
-         Both meshes sit at the same origin at rest, with zero travel that's
-         already fully closed, so the joints run negative (limit 0 at rest,
-         closed) to open, matching HAL's 0 percent is open convention.
-         Collision is a plain box instead of the finger mesh, dartsim can't
-         build the contact sensor's shape from a mesh. -->
+         Both start at rest already closed, so the range runs negative to
+         open, matching HAL's 0 percent is open convention. Collision is a
+         box instead of the mesh, needed for the contact sensor below. -->
     <xacro:dobot_armlink_box_collision link_name="${prefix}link_gripper_jaw_left" visual_mesh="jaw_left"
       base_origin_xyz="${gripper_core_origin_xyz}" base_origin_rpy="0 0 0" mass="0.02" box_x="0.02" box_y="0.01" box_z="0.05"
