Commit message: fix dobot

File: CustomRobots/robot_arms/models/dobot_magician/dobot_magician.ros2_control.xacro (robot description, xacro)
@@ -86,10 +86,11 @@
         <state_interface name="effort"/>
       </joint>
-      <joint name="${prefix}joint_prismatic_r">
-        <param name="mimic">${prefix}joint_prismatic_l</param>
-        <param name="multiplier">-1.0</param>
-        <state_interface name="position"/>
-        <state_interface name="velocity"/>
-      </joint>
+      <!-- joint_prismatic_r stays out of ros2_control entirely. Crashed in
+           gz_ros2_control every time regardless of what interfaces it had,
+           the two revolute mimics above never crashed either way, so this
+           looks like a gz_ros2_control bug specific to prismatic mimics.
+           It still tracks joint_prismatic_l physically, gz-sim enforces the
+           URDF-level mimic tag on its own, ros2_control doesn't need to
+           know about it for that to work. -->
     </ros2_control>
   </xacro:macro>

Commit message: dobbot controllers and xacro to fix prismatic joint

File: CustomRobots/robot_arms/models/dobot_magician/dobot_magician.ros2_control.xacro (robot description, xacro)
@@ -61,23 +61,18 @@
         <state_interface name="effort"/>
       </joint>
-      <!-- Mimic joints only get a state_interface, gz_ros2_control expects that,
-           a command_interface here crashed it (worse for the prismatic one). -->
+      <!-- Mimic joints only get a state_interface. The mimic relationship
+           itself is declared once, on the joint in the URDF above, gz_ros2_control's
+           own gripper_mimic_joint_example does not repeat "mimic"/"multiplier"
+           params here, only bare state_interfaces. -->
       <joint name="${prefix}joint_mimic_1">
-        <param name="mimic">${prefix}joint_2</param>
-        <param name="multiplier">-1.0</param>
         <state_interface name="position"/>
         <state_interface name="velocity"/>
       </joint>
       <joint name="${prefix}joint_mimic_2">
-        <param name="mimic">${prefix}joint_3</param>
-        <param name="multiplier">-1.0</param>
         <state_interface name="position"/>
         <state_interface name="velocity"/>
       </joint>
     </ros2_control>
-    <!-- Gripper in its own hardware component. Mixing joint_prismatic_l with
-         the arm's revolute joints in one component crashed gz_ros2_control
-         right after the last joint every time, splitting it off is the same
-         pattern UR3/Robotiq already use in this repo. -->
+    <!-- Gripper in its own hardware component, same split UR3/UR5+Robotiq use. -->
     <ros2_control name="${name}_gripper" type="system">
       <hardware>
@@ -102,7 +97,8 @@
         <state_interface name="effort"/>
       </joint>
-      <!-- joint_prismatic_r stays out of ros2_control entirely, still tracks
-           joint_prismatic_l physically through the URDF-level mimic tag,
-           gz-sim enforces that on its own. -->
+      <joint name="${prefix}joint_prismatic_r">
+        <state_interface name="position"/>
+        <state_interface name="velocity"/>
+      </joint>
     </ros2_control>
   </xacro:macro>

Commit message: dobbot gripper controller

File: CustomRobots/robot_arms/models/dobot_magician/dobot_magician.ros2_control.xacro (robot description, xacro)
@@ -89,8 +89,10 @@
         <state_interface name="effort"/>
       </joint>
-      <joint name="${prefix}joint_prismatic_r">
-        <state_interface name="position"/>
-        <state_interface name="velocity"/>
-      </joint>
+      <!-- joint_prismatic_r stays out of ros2_control entirely, even a bare
+           state_interface-only declaration crashes gz_ros2_control right on
+           this joint, every single time, regardless of block layout or what
+           else changed around it. It still tracks joint_prismatic_l physically
+           through the URDF-level mimic tag, gz-sim enforces that on its own,
+           ros2_control does not need to know about it for that to work. -->
     </ros2_control>
   </xacro:macro>

Commit message: dobbot arm without gripper

File: CustomRobots/robot_arms/models/dobot_magician/dobot_magician.ros2_control.xacro (robot description, xacro)
@@ -73,27 +73,9 @@
         <state_interface name="velocity"/>
       </joint>
-      <!-- Gripper, same hardware component as the arm. The official gz_ros2_control
-           gripper_mimic_joint_example keeps its driving + mimic joint in one
-           ros2_control block too, splitting arm/gripper into two separate
-           hardware components crashed transitioning from the first to the
-           second every time, even with the mimic params already fixed. -->
-      <joint name="${prefix}joint_prismatic_l">
-        <command_interface name="position">
-          <param name="min">0.0</param>
-          <param name="max">0.0135</param>
-        </command_interface>
-        <state_interface name="position">
-          <param name="initial_value">0.0</param>
-        </state_interface>
-        <state_interface name="velocity"/>
-        <state_interface name="effort"/>
-      </joint>
-      <!-- joint_prismatic_r stays out of ros2_control entirely, even a bare
-           state_interface-only declaration crashes gz_ros2_control right on
-           this joint, every single time, regardless of block layout or what
-           else changed around it. It still tracks joint_prismatic_l physically
-           through the URDF-level mimic tag, gz-sim enforces that on its own,
-           ros2_control does not need to know about it for that to work. -->
     </ros2_control>
+    <!-- Gripper ros2_control temporarily removed, isolating whether the arm
+         alone loads cleanly in the real RADI before touching the gripper again.
+         The physical gripper links/joints are still in the URDF, just
+         uncontrolled, gripper_controller is not spawned for this test. -->
   </xacro:macro>
 </robot>

Commit message: dobbot meshes in stl format + fix controllers

File: CustomRobots/robot_arms/models/dobot_magician/dobot_magician.ros2_control.xacro (robot description, xacro)
@@ -73,9 +73,20 @@
         <state_interface name="velocity"/>
       </joint>
+      <joint name="${prefix}joint_prismatic_l">
+        <command_interface name="position">
+          <param name="min">0.0</param>
+          <param name="max">0.0135</param>
+        </command_interface>
+        <state_interface name="position">
+          <param name="initial_value">0.0</param>
+        </state_interface>
+        <state_interface name="velocity"/>
+        <state_interface name="effort"/>
+      </joint>
+      <joint name="${prefix}joint_prismatic_r">
+        <state_interface name="position"/>
+        <state_interface name="velocity"/>
+      </joint>
     </ros2_control>
-    <!-- Gripper ros2_control temporarily removed, isolating whether the arm
-         alone loads cleanly in the real RADI before touching the gripper again.
-         The physical gripper links/joints are still in the URDF, just
-         uncontrolled, gripper_controller is not spawned for this test. -->
   </xacro:macro>
 </robot>

File: CustomRobots/robot_arms/models/dobot_magician/dobot_magician_macro.xacro (robot description, xacro)
@@ -36,5 +36,5 @@
         <origin xyz="${base_origin_xyz}" rpy="${base_origin_rpy}"/>
         <geometry>
-          <mesh filename="package://custom_robots/models/dobot_magician/meshes/collision/${collision_mesh}.dae"/>
+          <mesh filename="package://custom_robots/models/dobot_magician/meshes/collision/${collision_mesh}.stl"/>
         </geometry>
       </collision>
@@ -44,14 +44,8 @@
   <xacro:macro name="dobot_mimiclink" params="link_name">
     <link name="${link_name}">
-      <visual>
-        <geometry>
-          <box size="0 0 0"/>
-        </geometry>
-      </visual>
-      <collision>
-        <geometry>
-          <box size="0 0 0"/>
-        </geometry>
-      </collision>
+      <!-- No collision here on purpose, a zero-size box asserts inside DART
+           when spawned while physics is already stepping. This link is a
+           bookkeeping placeholder for the parallelogram, it never needs to
+           collide with anything. -->
       <xacro:box_inertial mass="0.001" x="0.01" y="0.01" z="0.01"/>
     </link>

Commit message: avoid end-efector swing, and joint limmit array + code style

File: CustomRobots/robot_arms/models/dobot_magician/dobot_magician.ros2_control.xacro (robot description, xacro)
@@ -61,8 +61,6 @@
         <state_interface name="effort"/>
       </joint>
-      <!-- Mimic joints only get a state_interface. The mimic relationship
-           itself is declared once, on the joint in the URDF above, gz_ros2_control's
-           own gripper_mimic_joint_example does not repeat "mimic"/"multiplier"
-           params here, only bare state_interfaces. -->
+      <!-- Mimic joints only get a state_interface here. That relationship
+           is already declared once on the joint in the URDF above. -->
       <joint name="${prefix}joint_mimic_1">
         <state_interface name="position"/>

File: CustomRobots/robot_arms/models/dobot_magician/dobot_magician_macro.xacro (robot description, xacro)
@@ -1,10 +1,8 @@
 <?xml version="1.0"?>
 <robot xmlns:xacro="http://www.ros.org/wiki/xacro">
-  <!-- Real dimensions and joint layout ported from
-       https://github.com/jkaniuka/magician_ros2 (dobot_description), see NOTICE.
-       The arm closes its real parallelogram linkage with two mimic joints
-       (joint_mimic_1 follows joint_2, joint_mimic_2 follows joint_3) instead
-       of a closed kinematic loop, this keeps the end effector level without
-       needing the physical parallel bars in the model. -->
+  <!-- Dimensions and joint layout ported from
+       https://github.com/jkaniuka/magician_ros2, see NOTICE.
+       joint_mimic_1 and joint_mimic_2 close the real parallelogram
+       linkage without needing a closed kinematic loop. -->
   <xacro:property name="link_base_length" value="0.131305"/>
   <xacro:property name="link_2_length" value="0.135"/>
@@ -45,7 +43,6 @@
     <link name="${link_name}">
       <!-- No collision here on purpose, a zero-size box asserts inside DART
-           when spawned while physics is already stepping. This link is a
-           bookkeeping placeholder for the parallelogram, it never needs to
-           collide with anything. -->
+           once physics is stepping. This link just tracks the parallelogram
+           and never needs to collide with anything. -->
       <xacro:box_inertial mass="0.001" x="0.01" y="0.01" z="0.01"/>
     </link>
@@ -58,5 +55,5 @@
       <limit effort="2000" velocity="1" lower="${lower_limit}" upper="${upper_limit}"/>
       <origin xyz="${origin_xyz}" rpy="${origin_rpy}"/>
-      <dynamics damping="0.0" friction="0.0"/>
+      <dynamics damping="1.0" friction="0"/>
     </joint>
   </xacro:macro>
@@ -68,5 +65,7 @@
       <limit effort="2000" velocity="1" lower="${lower_limit}" upper="${upper_limit}"/>
       <origin xyz="${origin_xyz}" rpy="${origin_rpy}"/>
-      <dynamics damping="0.0" friction="0.0"/>
+      <!-- Damping here matters more than on the driven joints, it's what
+           settles the parallelogram constraint instead of oscillating -->
+      <dynamics damping="1.0" friction="0"/>
       <mimic joint="${ref_joint}" multiplier="-1" offset="0"/>
     </joint>

Commit message: autoatach dobot

File: CustomRobots/robot_arms/models/dobot_magician/dobot_magician.ros2_control.xacro (robot description, xacro)
@@ -73,9 +73,9 @@
       <joint name="${prefix}joint_prismatic_l">
         <command_interface name="position">
-          <param name="min">-0.0135</param>
+          <param name="min">-0.018</param>
           <param name="max">0.0</param>
         </command_interface>
         <state_interface name="position">
-          <param name="initial_value">-0.0135</param>
+          <param name="initial_value">-0.018</param>
         </state_interface>
         <state_interface name="velocity"/>

File: CustomRobots/robot_arms/models/dobot_magician/dobot_magician_macro.xacro (robot description, xacro)
@@ -135,5 +135,5 @@
       parent="${prefix}link_gripper_core" child="${prefix}link_gripper_jaw_left"
       axis_xyz="0 -1 0" origin_xyz="0 0 0" origin_rpy="0 0 0"
-      lower_limit="-0.0135" upper_limit="0"/>
+      lower_limit="-0.018" upper_limit="0"/>
     <xacro:dobot_armlink link_name="${prefix}link_gripper_jaw_right" visual_mesh="jaw_right" collision_mesh="jaw_right"
       base_origin_xyz="${gripper_core_origin_xyz}" base_origin_rpy="0 0 0" mass="0.02" box_x="0.02" box_y="0.01" box_z="0.05"/>
@@ -141,5 +141,16 @@
       parent="${prefix}link_gripper_core" child="${prefix}link_gripper_jaw_right"
       axis_xyz="0 1 0" origin_xyz="0 0 0" origin_rpy="0 0 0"
-      lower_limit="-0.0135" upper_limit="0" ref_joint="${prefix}joint_prismatic_l"/>
+      lower_limit="-0.018" upper_limit="0" ref_joint="${prefix}joint_prismatic_l"/>
+    <!-- Contact sensor for gz_link_attacher, on the jaw itself since
+         that's what actually touches a grasped object, not the core -->
+    <gazebo reference="${prefix}link_gripper_jaw_left">
+      <sensor name="suction_contact" type="contact">
+        <always_on>true</always_on>
+        <update_rate>100</update_rate>
+        <contact>
+          <collision>${prefix}link_gripper_jaw_left_collision</collision>
+        </contact>
+      </sensor>
+    </gazebo>
     <!-- Actively drives the 3 mimic joints above, dartsim doesn't honor
          their <mimic> tag by itself -->

Commit message: docker magician suction pick and place

File: CustomRobots/robot_arms/models/dobot_magician/dobot_magician.ros2_control.xacro (robot description, xacro)
@@ -5,5 +5,6 @@
     prefix:=''
     sim_gz:=false
-    use_fake_hardware:=false">
+    use_fake_hardware:=false
+    end_effector:='gripper'">
     <ros2_control name="${name}" type="system">
       <hardware>
@@ -71,4 +72,5 @@
         <state_interface name="velocity"/>
       </joint>
+      <xacro:if value="${end_effector == 'gripper'}">
       <joint name="${prefix}joint_prismatic_l">
         <command_interface name="position">
@@ -86,4 +88,5 @@
         <state_interface name="velocity"/>
       </joint>
+      </xacro:if>
     </ros2_control>
   </xacro:macro>

File: CustomRobots/robot_arms/models/dobot_magician/dobot_magician.urdf.xacro (robot description, xacro)
@@ -7,14 +7,16 @@
   <xacro:arg name="sim_gz" default="true"/>
   <xacro:arg name="simulation_controllers" default=""/>
+  <xacro:arg name="end_effector" default="gripper"/>
   <xacro:include filename="$(find custom_robots)/models/dobot_magician/dobot_magician_macro.xacro"/>
   <xacro:include filename="$(find custom_robots)/models/dobot_magician/dobot_magician.ros2_control.xacro"/>
   <!-- fixed base, anchor it to the world so it doesn't fall under gravity -->
   <link name="world"/>
-  <xacro:dobot_magician parent="world" prefix="$(arg prefix)"/>
+  <xacro:dobot_magician parent="world" prefix="$(arg prefix)" end_effector="$(arg end_effector)"/>
   <xacro:dobot_magician_ros2_control
     name="$(arg name)"
     prefix="$(arg prefix)"
     sim_gz="$(arg sim_gz)"
-    use_fake_hardware="$(arg use_fake_hardware)"/>
+    use_fake_hardware="$(arg use_fake_hardware)"
+    end_effector="$(arg end_effector)"/>
   <xacro:if value="$(arg sim_gz)">
     <gazebo>

File: CustomRobots/robot_arms/models/dobot_magician/dobot_magician_macro.xacro (robot description, xacro)
@@ -94,5 +94,5 @@
     </joint>
   </xacro:macro>
-  <xacro:macro name="dobot_magician" params="parent prefix:=''">
+  <xacro:macro name="dobot_magician" params="parent prefix:='' end_effector:='gripper'">
     <xacro:dobot_armlink link_name="${prefix}base_link" visual_mesh="magicianBase" collision_mesh="magicianBase"
       base_origin_xyz="0 0 0" base_origin_rpy="0 0 0" mass="1.5" box_x="0.15" box_y="0.15" box_z="0.13"/>
@@ -142,4 +142,5 @@
     <xacro:property name="gripper_core_origin_xyz"
       value="${gripper_core_origin_x} 0 ${gripper_core_origin_z}"/>
+    <xacro:if value="${end_effector == 'gripper'}">
     <xacro:dobot_armlink link_name="${prefix}link_gripper_core" visual_mesh="gripper_core" collision_mesh="gripper_core"
       base_origin_xyz="${gripper_core_origin_xyz}" base_origin_rpy="0 0 0" mass="0.1" box_x="0.05" box_y="0.05" box_z="0.05"/>
@@ -177,6 +178,35 @@
       </sensor>
     </gazebo>
-    <!-- Actively drives the 3 mimic joints above, dartsim doesn't honor
-         their <mimic> tag by itself -->
+    <gazebo>
+      <plugin filename="libgz_mimic_joint.so" name="gz_mimic_joint::MimicJoint">
+        <parent_joint>${prefix}joint_prismatic_l</parent_joint>
+        <mimic_joint>${prefix}joint_prismatic_r</mimic_joint>
+      </plugin>
+    </gazebo>
+    </xacro:if>
+    <!-- Suction cup, the real one is a pneumatic on/off tool with no
+         actuated joint. Grasping is done by gz_link_attacher in suction
+         mode through the contact sensor at the tip of the cup. -->
+    <xacro:if value="${end_effector == 'suction_cup'}">
+    <xacro:property name="suction_cup_origin_z" value="${gripper_core_origin_z + 0.016}"/>
+    <xacro:dobot_armlink_box_collision link_name="${prefix}link_suction_cup" visual_mesh="suction_cup"
+      base_origin_xyz="${gripper_core_origin_x} 0 ${suction_cup_origin_z}" base_origin_rpy="0 0 0" mass="0.05" box_x="0.03" box_y="0.03" box_z="0.06"
+      collision_origin_xyz="${gripper_core_origin_x} 0 ${suction_cup_origin_z - 0.053}" collision_size="0.02 0.02 0.012"/>
+    <xacro:dobot_joint joint_name="${prefix}joint_4" type="revolute"
+      parent="${prefix}link_4" child="${prefix}link_suction_cup"
+      axis_xyz="0 0 1" origin_xyz="0.06 0 0" origin_rpy="0 0 0"
+      lower_limit="${-150.0/180.0*pi}" upper_limit="${150.0/180.0*pi}"/>
+    <gazebo reference="${prefix}link_suction_cup">
+      <sensor name="suction_contact" type="contact">
+        <always_on>true</always_on>
+        <update_rate>100</update_rate>
+        <contact>
+          <collision>${prefix}link_suction_cup_collision</collision>
+        </contact>
+      </sensor>
+    </gazebo>
+    </xacro:if>
+    <!-- Actively drives the parallelogram mimic joints above, dartsim
+         doesn't honor their <mimic> tag by itself -->
     <gazebo>
       <plugin filename="libgz_mimic_joint.so" name="gz_mimic_joint::MimicJoint">
@@ -188,8 +218,4 @@
         <mimic_joint>${prefix}joint_mimic_2</mimic_joint>
       </plugin>
-      <plugin filename="libgz_mimic_joint.so" name="gz_mimic_joint::MimicJoint">
-        <parent_joint>${prefix}joint_prismatic_l</parent_joint>
-        <mimic_joint>${prefix}joint_prismatic_r</mimic_joint>
-      </plugin>
     </gazebo>
   </xacro:macro>
