Commit message: xlerobot arm configuration

File: CustomRobots/xlerobot/models/xlerobot/xlerobot.urdf.xacro (robot description, xacro)
@@ -3,5 +3,7 @@
   <xacro:arg name="namespace" default=""/>
   <xacro:property name="namespace" value="$(arg namespace)"/>
+  <xacro:arg name="simulation_controllers" default=""/>
+  <xacro:property name="simulation_controllers" value="$(arg simulation_controllers)"/>
   <xacro:include filename="$(find custom_robots)/models/xlerobot/xlerobot_common.urdf.xacro"/>
-  <xacro:xlerobot namespace="${namespace}"/>
+  <xacro:xlerobot namespace="${namespace}" simulation_controllers="${simulation_controllers}"/>
 </robot>

File: CustomRobots/xlerobot/models/xlerobot/xlerobot_common.urdf.xacro (robot description, xacro)
@@ -2,5 +2,5 @@
 <robot xmlns:xacro="http://ros.org/wiki/xacro">
   <xacro:include filename="$(find custom_robots)/models/xlerobot/xlerobot_gz.urdf.xacro"/>
-  <xacro:macro name="xlerobot" params="namespace">
+  <xacro:macro name="xlerobot" params="namespace simulation_controllers">
     <!-- base_footprint sits on the ground, chassis is the real link the source model was
          built around, offset up so the wheels below it touch the floor -->
@@ -970,8 +970,11 @@
       <origin xyz="0 0 0" rpy="0 0 0" />
     </joint>
-<joint name="Rotation_L" type="fixed">
+<joint name="Rotation_L" type="revolute">
       <parent link="Base" />
       <child link="Rotation_Pitch" />
       <origin xyz="0 -0.0452 0.0165" rpy="1.5708 0 0" />
+      <axis xyz="0 -1 0" />
+      <limit lower="-2.16" upper="2.16" effort="3.35" velocity="2.0" />
+      <dynamics damping="0.3" friction="0.1" />
     </joint>
 <joint name="fixed_Rotation_Pitch_geom_1" type="fixed">
@@ -980,8 +983,11 @@
       <origin xyz="0 0 0" rpy="0 0 0" />
     </joint>
-<joint name="Pitch_L" type="fixed">
+<joint name="Pitch_L" type="revolute">
       <parent link="Rotation_Pitch" />
       <child link="Upper_Arm" />
       <origin xyz="0 0.1025 0.0306" rpy="1.5708 0 0" />
+      <axis xyz="-1 0 0" />
+      <limit lower="-0.22" upper="3.37" effort="3.35" velocity="2.0" />
+      <dynamics damping="0.3" friction="0.1" />
     </joint>
 <joint name="fixed_Upper_Arm_geom_1" type="fixed">
@@ -990,8 +996,11 @@
       <origin xyz="0 0 0" rpy="0 0 0" />
     </joint>
-<joint name="Elbow_L" type="fixed">
+<joint name="Elbow_L" type="revolute">
       <parent link="Upper_Arm" />
       <child link="Lower_Arm" />
       <origin xyz="0 0.11257 0.028" rpy="-1.5708 0 0" />
+      <axis xyz="1 0 0" />
+      <limit lower="-0.22" upper="3.14" effort="3.35" velocity="2.0" />
+      <dynamics damping="0.3" friction="0.1" />
     </joint>
 <joint name="fixed_Lower_Arm_geom_1" type="fixed">
@@ -1000,8 +1009,11 @@
       <origin xyz="0 0 0" rpy="0 0 0" />
     </joint>
-<joint name="Wrist_Pitch_L" type="fixed">
+<joint name="Wrist_Pitch_L" type="revolute">
       <parent link="Lower_Arm" />
       <child link="Wrist_Pitch_Roll" />
       <origin xyz="0 0.0052 0.1349" rpy="-1.5708 0 0" />
+      <axis xyz="1 0 0" />
+      <limit lower="-1.6580628" upper="1.6580627" effort="3.35" velocity="2.0" />
+      <dynamics damping="0.3" friction="0.1" />
     </joint>
 <joint name="fixed_Wrist_Pitch_Roll_geom_1" type="fixed">
@@ -1010,8 +1022,11 @@
       <origin xyz="0 0 0" rpy="0 0 0" />
     </joint>
-<joint name="Wrist_Roll_L" type="fixed">
+<joint name="Wrist_Roll_L" type="revolute">
       <parent link="Wrist_Pitch_Roll" />
       <child link="Fixed_Jaw" />
       <origin xyz="0 -0.0601 0" rpy="0 1.5707927 0" />
+      <axis xyz="0 -1 0" />
+      <limit lower="-2.7438473" upper="2.8412063" effort="3.35" velocity="2.0" />
+      <dynamics damping="0.3" friction="0.1" />
     </joint>
 <joint name="fixed_Fixed_Jaw_geom_1" type="fixed">
@@ -1020,8 +1035,11 @@
       <origin xyz="0 0 0" rpy="0 0 0" />
     </joint>
-<joint name="Jaw_L" type="fixed">
+<joint name="Jaw_L" type="revolute">
       <parent link="Fixed_Jaw" />
       <child link="Moving_Jaw" />
       <origin xyz="-0.0202 -0.0244 0" rpy="3.1415854 -0.0000014 2.9531853" />
+      <axis xyz="0 0 1" />
+      <limit lower="-0.374533" upper="1.7453292" effort="10" velocity="2.0" />
+      <dynamics damping="0.3" friction="0.1" />
     </joint>
 <joint name="fixed_Right_Arm_Camera" type="fixed">
@@ -1045,8 +1063,11 @@
       <origin xyz="0 0 0" rpy="0 0 0" />
     </joint>
-<joint name="Rotation_R" type="fixed">
+<joint name="Rotation_R" type="revolute">
       <parent link="Base_2" />
       <child link="Rotation_Pitch_2" />
       <origin xyz="0 -0.0452 0.0165" rpy="1.5708 0 0" />
+      <axis xyz="0 -1 0" />
+      <limit lower="-2.16" upper="2.16" effort="3.35" velocity="2.0" />
+      <dynamics damping="0.3" friction="0.1" />
     </joint>
 <joint name="fixed_Rotation_Pitch_2_geom_1" type="fixed">
@@ -1055,8 +1076,11 @@
       <origin xyz="0 0 0" rpy="0 0 0" />
     </joint>
-<joint name="Pitch_R" type="fixed">
+<joint name="Pitch_R" type="revolute">
       <parent link="Rotation_Pitch_2" />
       <child link="Upper_Arm_2" />
       <origin xyz="0 0.1025 0.0306" rpy="1.5708 0 0" />
+      <axis xyz="-1 0 0" />
+      <limit lower="-0.22" upper="3.37" effort="3.35" velocity="2.0" />
+      <dynamics damping="0.3" friction="0.1" />
     </joint>
 <joint name="fixed_Upper_Arm_2_geom_1" type="fixed">
@@ -1065,8 +1089,11 @@
       <origin xyz="0 0 0" rpy="0 0 0" />
     </joint>
-<joint name="Elbow_R" type="fixed">
+<joint name="Elbow_R" type="revolute">
       <parent link="Upper_Arm_2" />
       <child link="Lower_Arm_2" />
       <origin xyz="0 0.11257 0.028" rpy="-1.5708 0 0" />
+      <axis xyz="1 0 0" />
+      <limit lower="-0.22" upper="3.14" effort="3.35" velocity="2.0" />
+      <dynamics damping="0.3" friction="0.1" />
     </joint>
 <joint name="fixed_Lower_Arm_2_geom_1" type="fixed">
@@ -1075,8 +1102,11 @@
       <origin xyz="0 0 0" rpy="0 0 0" />
     </joint>
-<joint name="Wrist_Pitch_R" type="fixed">
+<joint name="Wrist_Pitch_R" type="revolute">
       <parent link="Lower_Arm_2" />
       <child link="Wrist_Pitch_Roll_2" />
       <origin xyz="0 0.0052 0.1349" rpy="-1.5708 0 0" />
+      <axis xyz="1 0 0" />
+      <limit lower="-1.6580628" upper="1.6580627" effort="3.35" velocity="2.0" />
+      <dynamics damping="0.3" friction="0.1" />
     </joint>
 <joint name="fixed_Wrist_Pitch_Roll_2_geom_1" type="fixed">
@@ -1085,8 +1115,11 @@
       <origin xyz="0 0 0" rpy="0 0 0" />
     </joint>
-<joint name="Wrist_Roll_R" type="fixed">
+<joint name="Wrist_Roll_R" type="revolute">
       <parent link="Wrist_Pitch_Roll_2" />
       <child link="Fixed_Jaw_2" />
       <origin xyz="0 -0.0601 0" rpy="0 1.5707927 0" />
+      <axis xyz="0 -1 0" />
+      <limit lower="-2.7438473" upper="2.8412063" effort="3.35" velocity="2.0" />
+      <dynamics damping="0.3" friction="0.1" />
     </joint>
 <joint name="fixed_Fixed_Jaw_2_geom_1" type="fixed">
@@ -1095,8 +1128,11 @@
       <origin xyz="0 0 0" rpy="0 0 0" />
     </joint>
-<joint name="Jaw_R" type="fixed">
+<joint name="Jaw_R" type="revolute">
       <parent link="Fixed_Jaw_2" />
       <child link="Moving_Jaw_2" />
       <origin xyz="-0.0202 -0.0244 0" rpy="3.1415854 -0.0000014 2.9531853" />
+      <axis xyz="0 0 1" />
+      <limit lower="-0.374533" upper="1.7453292" effort="10" velocity="2.0" />
+      <dynamics damping="0.3" friction="0.1" />
     </joint>
 <joint name="fixed_Left_Arm_Camera" type="fixed">
@@ -1120,8 +1156,11 @@
       <origin xyz="0 0 0" rpy="0 0 0" />
     </joint>
-<joint name="head_pan_joint" type="fixed">
+<joint name="head_pan_joint" type="revolute">
       <parent link="top_base_link" />
       <child link="head_pan_link" />
       <origin xyz="-0.103 0 0.323" rpy="0 0 0" />
+      <axis xyz="0 0 1" />
+      <limit lower="-3.2" upper="3.2" effort="1.0" velocity="1.5" />
+      <dynamics damping="0.1" friction="0.02" />
     </joint>
 <joint name="fixed_head_pan_link_geom_1" type="fixed">
@@ -1130,8 +1169,11 @@
       <origin xyz="0 0 0" rpy="0 0 0" />
     </joint>
-<joint name="head_tilt_joint" type="fixed">
+<joint name="head_tilt_joint" type="revolute">
       <parent link="head_pan_link" />
       <child link="head_tilt_link" />
       <origin xyz="0.001 0.002 0.09815" rpy="0 0 3.1415927" />
+      <axis xyz="0 1 0" />
+      <limit lower="-0.76" upper="1.45" effort="1.0" velocity="1.5" />
+      <dynamics damping="0.1" friction="0.02" />
     </joint>
 <joint name="fixed_head_tilt_link_geom_1" type="fixed">
@@ -1173,4 +1215,5 @@
     <axis xyz="-0.5000 -0.8660 0" />
   </joint>
+    <xacro:arm_ros2_control simulation_controllers="${simulation_controllers}"/>
     <xacro:wheel_slip wheel_link="wheel_1_link" fdir1="1 0 0"/>
     <xacro:wheel_slip wheel_link="wheel_2_link" fdir1="-0.5 0.866 0"/>
@@ -1179,4 +1222,7 @@
     <xacro:odom namespace="${namespace}"/>
     <plugin filename="gz-sim-joint-state-publisher-system" name="gz::sim::systems::JointStatePublisher" />
+    <xacro:rgbd_camera link="head_camera_link" name="head_camera" namespace="${namespace}"/>
+    <xacro:wrist_camera link="Right_Arm_Camera" name="right_arm_camera" namespace="${namespace}"/>
+    <xacro:wrist_camera link="Left_Arm_Camera" name="left_arm_camera" namespace="${namespace}"/>
   </xacro:macro>
 </robot>

File: CustomRobots/xlerobot/models/xlerobot/xlerobot_gz.urdf.xacro (robot description, xacro)
@@ -46,3 +46,112 @@
     </gazebo>
   </xacro:macro>
+  <!-- head RGBD camera, one sensor gives color image, depth image and a point cloud together -->
+  <xacro:macro name="rgbd_camera" params="link name namespace">
+    <gazebo reference="${link}">
+      <sensor name="${name}" type="rgbd_camera">
+        <always_on>true</always_on>
+        <visualize>false</visualize>
+        <update_rate>15</update_rate>
+        <topic>/${namespace}/${name}</topic>
+        <camera name="${name}">
+          <camera_info_topic>/${namespace}/${name}/camera_info</camera_info_topic>
+          <horizontal_fov>1.047</horizontal_fov>
+          <image>
+            <width>640</width>
+            <height>480</height>
+            <format>R8G8B8</format>
+          </image>
+          <clip>
+            <near>0.05</near>
+            <far>8.0</far>
+          </clip>
+        </camera>
+      </sensor>
+    </gazebo>
+  </xacro:macro>
+  <!-- One arm side worth of ros2_control joint interfaces, called once per suffix (L/R) -->
+  <xacro:macro name="arm_joint_interfaces" params="suffix">
+    <joint name="Rotation_${suffix}">
+      <command_interface name="position"><param name="min">-2.16</param><param name="max">2.16</param></command_interface>
+      <state_interface name="position"/>
+      <state_interface name="velocity"/>
+    </joint>
+    <joint name="Pitch_${suffix}">
+      <command_interface name="position"><param name="min">-0.22</param><param name="max">3.37</param></command_interface>
+      <state_interface name="position"/>
+      <state_interface name="velocity"/>
+    </joint>
+    <joint name="Elbow_${suffix}">
+      <command_interface name="position"><param name="min">-0.22</param><param name="max">3.14</param></command_interface>
+      <state_interface name="position"/>
+      <state_interface name="velocity"/>
+    </joint>
+    <joint name="Wrist_Pitch_${suffix}">
+      <command_interface name="position"><param name="min">-1.6580628</param><param name="max">1.6580627</param></command_interface>
+      <state_interface name="position"/>
+      <state_interface name="velocity"/>
+    </joint>
+    <joint name="Wrist_Roll_${suffix}">
+      <command_interface name="position"><param name="min">-2.7438473</param><param name="max">2.8412063</param></command_interface>
+      <state_interface name="position"/>
+      <state_interface name="velocity"/>
+    </joint>
+    <joint name="Jaw_${suffix}">
+      <command_interface name="position"><param name="min">-0.374533</param><param name="max">1.7453292</param></command_interface>
+      <state_interface name="position"/>
+      <state_interface name="velocity"/>
+    </joint>
+  </xacro:macro>
+  <!-- Single ros2_control block for both arms, both grippers and the head, on purpose.
+       Splitting this into several separate ros2_control tags made gz_ros2_control crash
+       while loading the second one when the same thing was tried on the Dobot arm, so
+       every actuated joint that is not a wheel lives in this one block -->
+  <xacro:macro name="arm_ros2_control" params="simulation_controllers">
+    <ros2_control name="xlerobot_arms" type="system">
+      <hardware>
+        <plugin>gz_ros2_control/GazeboSimSystem</plugin>
+      </hardware>
+      <xacro:arm_joint_interfaces suffix="L"/>
+      <xacro:arm_joint_interfaces suffix="R"/>
+      <joint name="head_pan_joint">
+        <command_interface name="position"><param name="min">-3.2</param><param name="max">3.2</param></command_interface>
+        <state_interface name="position"/>
+        <state_interface name="velocity"/>
+      </joint>
+      <joint name="head_tilt_joint">
+        <command_interface name="position"><param name="min">-0.76</param><param name="max">1.45</param></command_interface>
+        <state_interface name="position"/>
+        <state_interface name="velocity"/>
+      </joint>
+    </ros2_control>
+    <gazebo>
+      <plugin filename="gz_ros2_control-system" name="gz_ros2_control::GazeboSimROS2ControlPlugin">
+        <parameters>${simulation_controllers}</parameters>
+      </plugin>
+    </gazebo>
+  </xacro:macro>
+  <!-- plain RGB wrist camera -->
+  <xacro:macro name="wrist_camera" params="link name namespace">
+    <gazebo reference="${link}">
+      <sensor name="${name}" type="camera">
+        <always_on>true</always_on>
+        <visualize>false</visualize>
+        <update_rate>15</update_rate>
+        <topic>/${namespace}/${name}/image_raw</topic>
+        <camera name="${name}">
+          <camera_info_topic>/${namespace}/${name}/camera_info</camera_info_topic>
+          <horizontal_fov>1.5</horizontal_fov>
+          <image>
+            <width>640</width>
+            <height>480</height>
+            <format>R8G8B8</format>
+          </image>
+          <clip>
+            <near>0.02</near>
+            <far>5.0</far>
+          </clip>
+        </camera>
+      </sensor>
+    </gazebo>
+  </xacro:macro>
 </robot>
