Commit message: xlerobot update

File: CustomRobots/xlerobot/models/xlerobot/xlerobot_common.urdf.xacro (robot description, xacro)
@@ -1215,5 +1215,5 @@
     <axis xyz="-0.5000 -0.8660 0" />
   </joint>
-    <xacro:arm_ros2_control simulation_controllers="${simulation_controllers}"/>
+    <xacro:arm_ros2_control simulation_controllers="${simulation_controllers}" namespace="${namespace}"/>
     <xacro:wheel_slip wheel_link="wheel_1_link" fdir1="1 0 0"/>
     <xacro:wheel_slip wheel_link="wheel_2_link" fdir1="-0.5 0.866 0"/>

File: CustomRobots/xlerobot/models/xlerobot/xlerobot_gz.urdf.xacro (robot description, xacro)
@@ -107,5 +107,5 @@
        while loading the second one when the same thing was tried on the Dobot arm, so
        every actuated joint that is not a wheel lives in this one block -->
-  <xacro:macro name="arm_ros2_control" params="simulation_controllers">
+  <xacro:macro name="arm_ros2_control" params="simulation_controllers namespace">
     <ros2_control name="xlerobot_arms" type="system">
       <hardware>
@@ -127,4 +127,10 @@
     <gazebo>
       <plugin filename="gz_ros2_control-system" name="gz_ros2_control::GazeboSimROS2ControlPlugin">
+        <!-- robot_state_publisher runs under this same namespace, without this the
+             plugin looks for a bare, unnamespaced robot_state_publisher node and just
+             hangs forever waiting for a service that is never going to answer -->
+        <ros>
+          <namespace>${namespace}</namespace>
+        </ros>
         <parameters>${simulation_controllers}</parameters>
       </plugin>

Commit message: xlerobot in a separate exercise + arm controllers

File: CustomRobots/xlerobot/models/xlerobot/xlerobot_common.urdf.xacro (robot description, xacro)
@@ -1232,4 +1232,6 @@
     <xacro:wrist_camera link="Right_Arm_Camera" name="right_arm_camera" namespace="${namespace}"/>
     <xacro:wrist_camera link="Left_Arm_Camera" name="left_arm_camera" namespace="${namespace}"/>
+    <xacro:suction_contact link="Moving_Jaw"/>
+    <xacro:suction_contact link="Moving_Jaw_2"/>
   </xacro:macro>
 </robot>

File: CustomRobots/xlerobot/models/xlerobot/xlerobot_gz.urdf.xacro (robot description, xacro)
@@ -137,4 +137,22 @@
     </gazebo>
   </xacro:macro>
+  <!-- Contact sensor on a gripper jaw, feeds gz_link_attacher's "suction mode"
+       code path. gz_link_attacher only knows Robotiq's 2-finger link names by
+       default, this repurposes its generic gripper_link_name option (it was
+       already there for real suction grippers) so a plain parallel jaw like
+       ours gets the same auto-attach behaviour without touching that C++ -->
+  <xacro:macro name="suction_contact" params="link">
+    <gazebo reference="${link}">
+      <sensor name="suction_contact" type="contact">
+        <always_on>true</always_on>
+        <update_rate>30</update_rate>
+        <contact>
+          <collision>${link}_collision</collision>
+          <collision>${link}_collision_1</collision>
+          <collision>${link}_collision_2</collision>
+        </contact>
+      </sensor>
+    </gazebo>
+  </xacro:macro>
   <!-- plain RGB wrist camera -->
   <xacro:macro name="wrist_camera" params="link name namespace">

Commit message: xlebot controllers

File: CustomRobots/xlerobot/models/xlerobot/xlerobot_common.urdf.xacro (robot description, xacro)
@@ -1221,12 +1221,10 @@
     <xacro:velocity namespace="${namespace}"/>
     <xacro:odom namespace="${namespace}"/>
-    <!-- wheels only, the arm/head joints already get their joint_states from
-         ros2_control's own joint_state_broadcaster, publishing both would
-         mean two sources fighting over the same topic -->
-    <plugin filename="gz-sim-joint-state-publisher-system" name="gz::sim::systems::JointStatePublisher">
-      <joint_name>wheel_1_joint</joint_name>
-      <joint_name>wheel_2_joint</joint_name>
-      <joint_name>wheel_3_joint</joint_name>
-    </plugin>
+    <!-- no separate gz-sim-joint-state-publisher-system for the wheels here
+         on purpose, they are folded into the same ros2_control
+         joint_state_broadcaster as the arms instead (see arm_ros2_control in
+         xlerobot_gz.urdf.xacro), a second publisher on a different topic is
+         exactly what left MoveGroupInterface waiting forever for a "complete"
+         robot state that never included the wheels -->
     <xacro:rgbd_camera link="head_camera_link" name="head_camera" namespace="${namespace}"/>
     <xacro:wrist_camera link="Right_Arm_Camera" name="right_arm_camera" namespace="${namespace}"/>

File: CustomRobots/xlerobot/models/xlerobot/xlerobot_gz.urdf.xacro (robot description, xacro)
@@ -124,4 +124,26 @@
         <state_interface name="velocity"/>
       </joint>
+      <!-- state only, on purpose, the wheels stay driven kinematically by
+           VelocityControl not by ros2_control, but MoveGroupInterface (used
+           by robmove/robpose/move_group) waits for a JointState covering
+           every joint in the URDF before it considers the robot state
+           "complete", wheels included, even though no SRDF group ever plans
+           for them. Without this it hangs forever repeating "The complete
+           state of the robot is not yet known, missing wheel_1_joint...".
+           Folding them into the same joint_state_broadcaster that already
+           covers the arms is what actually gets them onto
+           /<namespace>/joint_states, the one topic MoveIt listens to -->
+      <joint name="wheel_1_joint">
+        <state_interface name="position"/>
+        <state_interface name="velocity"/>
+      </joint>
+      <joint name="wheel_2_joint">
+        <state_interface name="position"/>
+        <state_interface name="velocity"/>
+      </joint>
+      <joint name="wheel_3_joint">
+        <state_interface name="position"/>
+        <state_interface name="velocity"/>
+      </joint>
     </ros2_control>
     <gazebo>

Commit message: xlerobot arm controll fix

File: CustomRobots/xlerobot/models/xlerobot/xlerobot_common.urdf.xacro (robot description, xacro)
@@ -1172,5 +1172,9 @@
       <parent link="head_pan_link" />
       <child link="head_tilt_link" />
-      <origin xyz="0.001 0.002 0.09815" rpy="0 0 3.1415927" />
+      <!-- the 180 degree yaw this used to carry made the head camera face
+           straight backward at pan 0, chassis and head_pan_link share the
+           same forward direction all the way up (every joint above this one
+           is rpy 0 0 0), nothing upstream compensates for that flip -->
+      <origin xyz="0.001 0.002 0.09815" rpy="0 0 0" />
       <axis xyz="0 1 0" />
       <limit lower="-0.76" upper="1.45" effort="1.0" velocity="1.5" />

Commit message: xlerobot TCP and tray tfs, RGBD camera support, update world

File: CustomRobots/xlerobot/models/xlerobot/xlerobot_common.urdf.xacro (robot description, xacro)
@@ -1043,4 +1043,13 @@
       <dynamics damping="0.3" friction="0.1" />
     </joint>
+<!-- TCP: fingertip contact point with the gripper mechanically closed
+     (Jaw_L at its lower limit), measured as the midpoint of the closest
+     Fixed_Jaw/Moving_Jaw mesh vertices at that configuration -->
+<link name="TCP_L" />
+<joint name="TCP_L_joint" type="fixed">
+      <parent link="Fixed_Jaw" />
+      <child link="TCP_L" />
+      <origin xyz="0.00713 -0.10003 -0.00360" rpy="0 0 0" />
+    </joint>
 <joint name="fixed_Right_Arm_Camera" type="fixed">
       <parent link="Fixed_Jaw" />
@@ -1136,4 +1145,12 @@
       <dynamics damping="0.3" friction="0.1" />
     </joint>
+<!-- TCP: same measured fingertip contact point as TCP_L, Fixed_Jaw_2 uses
+     the identical Fixed_Jaw/Moving_Jaw mesh pair mounted symmetrically -->
+<link name="TCP_R" />
+<joint name="TCP_R_joint" type="fixed">
+      <parent link="Fixed_Jaw_2" />
+      <child link="TCP_R" />
+      <origin xyz="0.00713 -0.10003 -0.00360" rpy="0 0 0" />
+    </joint>
 <joint name="fixed_Left_Arm_Camera" type="fixed">
       <parent link="Fixed_Jaw_2" />
@@ -1155,4 +1172,21 @@
       <child link="top_base_link_geom_1" />
       <origin xyz="0 0 0" rpy="0 0 0" />
+    </joint>
+<!-- Tray drop/pick anchor points, one per arm, positioned by hand in RViz
+     against the real basket mesh (see /tmp calibration session). This is the
+     floor contact point of each arm's slot, not the object's rest center:
+     whoever teleports an object here on drop must add half that object's
+     height in z so it does not clip through the floor -->
+<link name="tray_anchor_L" />
+<joint name="tray_anchor_L_joint" type="fixed">
+      <parent link="top_base_link" />
+      <child link="tray_anchor_L" />
+      <origin xyz="0.061 0.085 0.002" rpy="0 0 0" />
+    </joint>
+<link name="tray_anchor_R" />
+<joint name="tray_anchor_R_joint" type="fixed">
+      <parent link="top_base_link" />
+      <child link="tray_anchor_R" />
+      <origin xyz="0.061 -0.085 0.002" rpy="0 0 0" />
     </joint>
 <joint name="head_pan_joint" type="revolute">

Commit message: xlerobot world, collisions

File: CustomRobots/xlerobot/models/xlerobot/xlerobot_common.urdf.xacro (robot description, xacro)
@@ -1228,10 +1228,15 @@
       <parent link="head_camera_link" />
       <child link="head_camera_rgb_frame" />
-      <origin xyz="0 0 0" rpy="0 -1.5707911 -1.5707963" />
+      <!-- roll/pitch were swapped: this used to point optical +Z (forward)
+           along the robot's own +Y (left) instead of +X (ahead), confirmed
+           by computing the actual forward axis from the live TF transform.
+           Correct optical-frame convention is roll=-90, pitch=0, yaw=-90 -->
+      <origin xyz="0 0 0" rpy="-1.5707911 0 -1.5707963" />
     </joint>
 <joint name="fixed_head_camera_depth_frame" type="fixed">
       <parent link="head_camera_link" />
       <child link="head_camera_depth_frame" />
-      <origin xyz="0 0 0" rpy="0 -1.5707911 -1.5707963" />
+      <!-- same roll/pitch fix as fixed_head_camera_rgb_frame above -->
+      <origin xyz="0 0 0" rpy="-1.5707911 0 -1.5707963" />
     </joint>
   <joint name="wheel_1_joint" type="continuous">

File: CustomRobots/xlerobot/models/xlerobot/xlerobot_gz.urdf.xacro (robot description, xacro)
@@ -28,4 +28,24 @@
     </gazebo>
   </xacro:macro>
+  <!-- Safety net, not a substitute for not colliding: caps how hard ODE is
+       allowed to shove interpenetrating bodies apart in a single step. A
+       real bump against the table (chassis is the only link here with
+       collision geometry near the tray, top_base_link/the basket mesh has
+       none) otherwise resolves as a single large correction impulse that
+       shows up as the whole kinematic chain (arms included) jumping/
+       jittering, since they all ride on the chassis. max_vel/min_depth are
+       the standard ODE knobs for this, does not change normal driving. -->
+  <gazebo reference="chassis">
+    <collision>
+      <surface>
+        <contact>
+          <ode>
+            <max_vel>0.2</max_vel>
+            <min_depth>0.001</min_depth>
+          </ode>
+        </contact>
+      </surface>
+    </collision>
+  </gazebo>
   <xacro:macro name="velocity" params="namespace">
     <gazebo>

Commit message: collision xlerobot

File: CustomRobots/xlerobot/models/xlerobot/xlerobot_common.urdf.xacro (robot description, xacro)
@@ -777,4 +777,19 @@
         </material>
       </visual>
+      <!-- Had no collision geometry at all before, so arms could pass
+           straight through the tray/mast both in Gazebo and in MoveIt's
+           planning (nothing to check against). Box approximation, not the
+           real mesh (a cheaper primitive is the norm for collision, and
+           the real mesh's own footprint here still is not fully pinned
+           down), sized generously from the measured basket cavity (tray
+           anchors sit at x~0.06, y~+-0.085) up to just below the head
+           mount (head_pan_joint origin z=0.323) so the whole body is
+           covered, not just the basket -->
+      <collision>
+        <origin xyz="0 0 0.135" rpy="0 0 0" />
+        <geometry>
+          <box size="0.40 0.40 0.37" />
+        </geometry>
+      </collision>
       <inertial>
         <origin xyz="0 0 0" rpy="0 0 0" />

Commit message: xlerobot collisions update

File: CustomRobots/xlerobot/models/xlerobot/xlerobot_common.urdf.xacro (robot description, xacro)
@@ -779,15 +779,49 @@
       <!-- Had no collision geometry at all before, so arms could pass
            straight through the tray/mast both in Gazebo and in MoveIt's
-           planning (nothing to check against). Box approximation, not the
-           real mesh (a cheaper primitive is the norm for collision, and
-           the real mesh's own footprint here still is not fully pinned
-           down), sized generously from the measured basket cavity (tray
-           anchors sit at x~0.06, y~+-0.085) up to just below the head
-           mount (head_pan_joint origin z=0.323) so the whole body is
-           covered, not just the basket -->
-      <collision>
-        <origin xyz="0 0 0.135" rpy="0 0 0" />
-        <geometry>
-          <box size="0.40 0.40 0.37" />
+           planning (nothing to check against). Modeled hollow on purpose:
+           floor + 4 thin walls around the basket cavity (tray_anchor_L/R
+           sit at x~0.06, y~+-0.085, z~0, comfortably inside), open top so
+           dropInLeftTray/RightTray and pickFromLeftTray/RightTray can
+           still lower an object in from above, a single solid box here
+           would physically block the tray from ever being used. Solid
+           mast above the rim, up to just below the head mount
+           (head_pan_joint origin z=0.323), narrower to roughly match the
+           pole. All dimensions are a reasoned approximation around the
+           measured anchor points, not the real mesh, worth a visual
+           check once this is live. -->
+      <collision name="tray_floor">
+        <origin xyz="0.06 0 -0.045" rpy="0 0 0" />
+        <geometry>
+          <box size="0.28 0.36 0.03" />
+        </geometry>
+      </collision>
+      <collision name="tray_wall_back">
+        <origin xyz="-0.065 0 0.045" rpy="0 0 0" />
+        <geometry>
+          <box size="0.03 0.36 0.15" />
+        </geometry>
+      </collision>
+      <collision name="tray_wall_front">
+        <origin xyz="0.185 0 0.045" rpy="0 0 0" />
+        <geometry>
+          <box size="0.03 0.36 0.15" />
+        </geometry>
+      </collision>
+      <collision name="tray_wall_left">
+        <origin xyz="0.06 -0.165 0.045" rpy="0 0 0" />
+        <geometry>
+          <box size="0.22 0.03 0.15" />
+        </geometry>
+      </collision>
+      <collision name="tray_wall_right">
+        <origin xyz="0.06 0.165 0.045" rpy="0 0 0" />
+        <geometry>
+          <box size="0.22 0.03 0.15" />
+        </geometry>
+      </collision>
+      <collision name="mast">
+        <origin xyz="0.06 0 0.22" rpy="0 0 0" />
+        <geometry>
+          <box size="0.16 0.16 0.20" />
         </geometry>
       </collision>

Commit message: xlerobot map and camera frames

File: CustomRobots/xlerobot/models/xlerobot/xlerobot_common.urdf.xacro (robot description, xacro)
@@ -777,51 +777,22 @@
         </material>
       </visual>
-      <!-- Had no collision geometry at all before, so arms could pass
-           straight through the tray/mast both in Gazebo and in MoveIt's
-           planning (nothing to check against). Modeled hollow on purpose:
-           floor + 4 thin walls around the basket cavity (tray_anchor_L/R
-           sit at x~0.06, y~+-0.085, z~0, comfortably inside), open top so
-           dropInLeftTray/RightTray and pickFromLeftTray/RightTray can
-           still lower an object in from above, a single solid box here
-           would physically block the tray from ever being used. Solid
-           mast above the rim, up to just below the head mount
-           (head_pan_joint origin z=0.323), narrower to roughly match the
-           pole. All dimensions are a reasoned approximation around the
-           measured anchor points, not the real mesh, worth a visual
-           check once this is live. -->
-      <collision name="tray_floor">
-        <origin xyz="0.06 0 -0.045" rpy="0 0 0" />
-        <geometry>
-          <box size="0.28 0.36 0.03" />
-        </geometry>
-      </collision>
-      <collision name="tray_wall_back">
-        <origin xyz="-0.065 0 0.045" rpy="0 0 0" />
-        <geometry>
-          <box size="0.03 0.36 0.15" />
-        </geometry>
-      </collision>
-      <collision name="tray_wall_front">
-        <origin xyz="0.185 0 0.045" rpy="0 0 0" />
-        <geometry>
-          <box size="0.03 0.36 0.15" />
-        </geometry>
-      </collision>
-      <collision name="tray_wall_left">
-        <origin xyz="0.06 -0.165 0.045" rpy="0 0 0" />
-        <geometry>
-          <box size="0.22 0.03 0.15" />
-        </geometry>
-      </collision>
-      <collision name="tray_wall_right">
-        <origin xyz="0.06 0.165 0.045" rpy="0 0 0" />
-        <geometry>
-          <box size="0.22 0.03 0.15" />
-        </geometry>
-      </collision>
+      <!-- The basket itself is the chassis link (raskogbody.stl) and its
+           collision boxes already model the tray floor (top at z=0.68 in
+           base_footprint) and rim walls, tray_anchor_L/R sit inside that
+           cavity. top_base_link only carries the thin mast, which had no
+           collision at all so arms could pass through it. -->
+      <!-- Was centered at x=0.06 (that is the basket cavity's x, not the
+           mast's), 0.16m wide, which caused the left arm's own ready pose
+           to self-collide with it (checked against the actual joint
+           chain, the forearm passes right through z=0.16-0.28 there), so
+           every single planning request failed regardless of target.
+           Recentered on the real mast footprint from the topbase1.stl
+           cross-section (x=-0.131..-0.079, y=-0.022..0.022) and narrowed
+           to match, the arm's ready-pose links sit at y~-0.15, comfortably
+           clear of this now -->
       <collision name="mast">
-        <origin xyz="0.06 0 0.22" rpy="0 0 0" />
-        <geometry>
-          <box size="0.16 0.16 0.20" />
+        <origin xyz="-0.105 0 0.22" rpy="0 0 0" />
+        <geometry>
+          <box size="0.06 0.05 0.20" />
         </geometry>
       </collision>

Commit message: camera frecuency

File: CustomRobots/xlerobot/models/xlerobot/xlerobot_common.urdf.xacro (robot description, xacro)
@@ -1202,5 +1202,5 @@
       <parent link="top_base_link" />
       <child link="tray_anchor_L" />
-      <origin xyz="0.061 0.085 0.002" rpy="0 0 0" />
+      <origin xyz="0.061 -0.085 0.002" rpy="0 0 0" />
     </joint>
 <link name="tray_anchor_R" />
@@ -1208,5 +1208,5 @@
       <parent link="top_base_link" />
       <child link="tray_anchor_R" />
-      <origin xyz="0.061 -0.085 0.002" rpy="0 0 0" />
+      <origin xyz="0.061 0.085 0.002" rpy="0 0 0" />
     </joint>
 <joint name="head_pan_joint" type="revolute">

Commit message: tcp position

File: CustomRobots/xlerobot/models/xlerobot/xlerobot_common.urdf.xacro (robot description, xacro)
@@ -1063,12 +1063,18 @@
       <dynamics damping="0.3" friction="0.1" />
     </joint>
-<!-- TCP: fingertip contact point with the gripper mechanically closed
-     (Jaw_L at its lower limit), measured as the midpoint of the closest
-     Fixed_Jaw/Moving_Jaw mesh vertices at that configuration -->
+<!-- TCP: centre of the pocket a 50mm cube sits in between the two jaws,
+     in the Fixed_Jaw frame. The gripper is asymmetric, a fixed finger and a
+     moving one, so the point that matters is not where the pads touch when
+     fully closed (that put the TCP on the fixed finger's face, which then
+     shoved the cube out of the way). Measured from the meshes: the fixed
+     pad's most protruding point over the last 5cm of the fingers is at
+     x=0.0079, the cube's face rests there so its centre is 25mm further
+     towards the moving jaw (x=-0.0171), and y=-0.080 centres it on the 5cm
+     of pad, 2cm back from the fingertips -->
 <link name="TCP_L" />
 <joint name="TCP_L_joint" type="fixed">
       <parent link="Fixed_Jaw" />
       <child link="TCP_L" />
-      <origin xyz="0.00713 -0.10003 -0.00360" rpy="0 0 0" />
+      <origin xyz="-0.0171 -0.0800 0.0" rpy="0 0 0" />
     </joint>
 <joint name="fixed_Right_Arm_Camera" type="fixed">
@@ -1165,11 +1171,11 @@
       <dynamics damping="0.3" friction="0.1" />
     </joint>
-<!-- TCP: same measured fingertip contact point as TCP_L, Fixed_Jaw_2 uses
-     the identical Fixed_Jaw/Moving_Jaw mesh pair mounted symmetrically -->
+<!-- TCP: same pocket centre as TCP_L, Fixed_Jaw_2 uses the identical
+     Fixed_Jaw/Moving_Jaw mesh pair -->
 <link name="TCP_R" />
 <joint name="TCP_R_joint" type="fixed">
       <parent link="Fixed_Jaw_2" />
       <child link="TCP_R" />
-      <origin xyz="0.00713 -0.10003 -0.00360" rpy="0 0 0" />
+      <origin xyz="-0.0171 -0.0800 0.0" rpy="0 0 0" />
     </joint>
 <joint name="fixed_Left_Arm_Camera" type="fixed">

Commit message: tcp pos

File: CustomRobots/xlerobot/models/xlerobot/xlerobot_common.urdf.xacro (robot description, xacro)
@@ -1054,5 +1054,5 @@
       <parent link="Fixed_Jaw" />
       <child link="TCP_L" />
-      <origin xyz="-0.0171 -0.0800 0.0" rpy="0 0 0" />
+      <origin xyz="-0.0380 -0.0930 0.0" rpy="0 0 0" />
     </joint>
 <joint name="fixed_Right_Arm_Camera" type="fixed">
@@ -1154,5 +1154,5 @@
       <parent link="Fixed_Jaw_2" />
       <child link="TCP_R" />
-      <origin xyz="-0.0171 -0.0800 0.0" rpy="0 0 0" />
+      <origin xyz="-0.0380 -0.0930 0.0" rpy="0 0 0" />
     </joint>
 <joint name="fixed_Left_Arm_Camera" type="fixed">
