Commit message: xlerobot inertias

File: CustomRobots/xlerobot/models/xlerobot/xlerobot_common.urdf.xacro (robot description, xacro)
@@ -71,5 +71,5 @@
         <origin xyz="0 0 -0.38" rpy="0 0 0" />
         <mass value="10" />
-        <inertia ixx="0.001" ixy="0" ixz="0" iyy="0.001" iyz="0" izz="0.001" />
+        <inertia ixx="0.43" ixy="0" ixz="0" iyy="0.37" iyz="0" izz="0.21" />
       </inertial>
     </link>
@@ -87,5 +87,5 @@
         <origin xyz="0 0 0" rpy="0 0 0" />
         <mass value="0.001" />
-        <inertia ixx="0.1" ixy="0" ixz="0" iyy="0.1" iyz="0" izz="0.1" />
+        <inertia ixx="1e-6" ixy="0" ixz="0" iyy="1e-6" iyz="0" izz="1e-6" />
       </inertial>
     </link>
@@ -103,5 +103,5 @@
         <origin xyz="0 0 0" rpy="0 0 0" />
         <mass value="0.001" />
-        <inertia ixx="0.1" ixy="0" ixz="0" iyy="0.1" iyz="0" izz="0.1" />
+        <inertia ixx="1e-6" ixy="0" ixz="0" iyy="1e-6" iyz="0" izz="1e-6" />
       </inertial>
     </link>
@@ -147,5 +147,5 @@
         <origin xyz="0 0 0" rpy="0 0 0" />
         <mass value="0.001" />
-        <inertia ixx="0.1" ixy="0" ixz="0" iyy="0.1" iyz="0" izz="0.1" />
+        <inertia ixx="1e-6" ixy="0" ixz="0" iyy="1e-6" iyz="0" izz="1e-6" />
       </inertial>
     </link>
@@ -191,5 +191,5 @@
         <origin xyz="0 0 0" rpy="0 0 0" />
         <mass value="0.001" />
-        <inertia ixx="0.1" ixy="0" ixz="0" iyy="0.1" iyz="0" izz="0.1" />
+        <inertia ixx="1e-6" ixy="0" ixz="0" iyy="1e-6" iyz="0" izz="1e-6" />
       </inertial>
     </link>
@@ -235,5 +235,5 @@
         <origin xyz="0 0 0" rpy="0 0 0" />
         <mass value="0.001" />
-        <inertia ixx="0.1" ixy="0" ixz="0" iyy="0.1" iyz="0" izz="0.1" />
+        <inertia ixx="1e-6" ixy="0" ixz="0" iyy="1e-6" iyz="0" izz="1e-6" />
       </inertial>
     </link>
@@ -279,5 +279,5 @@
         <origin xyz="0 0 0" rpy="0 0 0" />
         <mass value="0.001" />
-        <inertia ixx="0.1" ixy="0" ixz="0" iyy="0.1" iyz="0" izz="0.1" />
+        <inertia ixx="1e-6" ixy="0" ixz="0" iyy="1e-6" iyz="0" izz="1e-6" />
       </inertial>
     </link>
@@ -323,5 +323,5 @@
         <origin xyz="0 0 0" rpy="0 0 0" />
         <mass value="0.001" />
-        <inertia ixx="0.1" ixy="0" ixz="0" iyy="0.1" iyz="0" izz="0.1" />
+        <inertia ixx="1e-6" ixy="0" ixz="0" iyy="1e-6" iyz="0" izz="1e-6" />
       </inertial>
     </link>
@@ -367,5 +367,5 @@
         <origin xyz="0 0 0" rpy="0 0 0" />
         <mass value="0.001" />
-        <inertia ixx="0.1" ixy="0" ixz="0" iyy="0.1" iyz="0" izz="0.1" />
+        <inertia ixx="1e-6" ixy="0" ixz="0" iyy="1e-6" iyz="0" izz="1e-6" />
       </inertial>
     </link>
@@ -433,5 +433,5 @@
         <origin xyz="0 0 0" rpy="0 0 0" />
         <mass value="0.001" />
-        <inertia ixx="0.1" ixy="0" ixz="0" iyy="0.1" iyz="0" izz="0.1" />
+        <inertia ixx="1e-6" ixy="0" ixz="0" iyy="1e-6" iyz="0" izz="1e-6" />
       </inertial>
     </link>
@@ -477,5 +477,5 @@
         <origin xyz="0 0 0" rpy="0 0 0" />
         <mass value="0.001" />
-        <inertia ixx="0.1" ixy="0" ixz="0" iyy="0.1" iyz="0" izz="0.1" />
+        <inertia ixx="1e-6" ixy="0" ixz="0" iyy="1e-6" iyz="0" izz="1e-6" />
       </inertial>
     </link>
@@ -521,5 +521,5 @@
         <origin xyz="0 0 0" rpy="0 0 0" />
         <mass value="0.001" />
-        <inertia ixx="0.1" ixy="0" ixz="0" iyy="0.1" iyz="0" izz="0.1" />
+        <inertia ixx="1e-6" ixy="0" ixz="0" iyy="1e-6" iyz="0" izz="1e-6" />
       </inertial>
     </link>
@@ -565,5 +565,5 @@
         <origin xyz="0 0 0" rpy="0 0 0" />
         <mass value="0.001" />
-        <inertia ixx="0.1" ixy="0" ixz="0" iyy="0.1" iyz="0" izz="0.1" />
+        <inertia ixx="1e-6" ixy="0" ixz="0" iyy="1e-6" iyz="0" izz="1e-6" />
       </inertial>
     </link>
@@ -609,5 +609,5 @@
         <origin xyz="0 0 0" rpy="0 0 0" />
         <mass value="0.001" />
-        <inertia ixx="0.1" ixy="0" ixz="0" iyy="0.1" iyz="0" izz="0.1" />
+        <inertia ixx="1e-6" ixy="0" ixz="0" iyy="1e-6" iyz="0" izz="1e-6" />
       </inertial>
     </link>
@@ -653,5 +653,5 @@
         <origin xyz="0 0 0" rpy="0 0 0" />
         <mass value="0.001" />
-        <inertia ixx="0.1" ixy="0" ixz="0" iyy="0.1" iyz="0" izz="0.1" />
+        <inertia ixx="1e-6" ixy="0" ixz="0" iyy="1e-6" iyz="0" izz="1e-6" />
       </inertial>
     </link>
@@ -697,5 +697,5 @@
         <origin xyz="0 0 0" rpy="0 0 0" />
         <mass value="0.001" />
-        <inertia ixx="0.1" ixy="0" ixz="0" iyy="0.1" iyz="0" izz="0.1" />
+        <inertia ixx="1e-6" ixy="0" ixz="0" iyy="1e-6" iyz="0" izz="1e-6" />
       </inertial>
     </link>
@@ -763,5 +763,5 @@
         <origin xyz="0 0 0" rpy="0 0 0" />
         <mass value="0.001" />
-        <inertia ixx="0.1" ixy="0" ixz="0" iyy="0.1" iyz="0" izz="0.1" />
+        <inertia ixx="1e-6" ixy="0" ixz="0" iyy="1e-6" iyz="0" izz="1e-6" />
       </inertial>
     </link>
@@ -802,5 +802,5 @@
         <origin xyz="0 0 0" rpy="0 0 0" />
         <mass value="0.001" />
-        <inertia ixx="0.1" ixy="0" ixz="0" iyy="0.1" iyz="0" izz="0.1" />
+        <inertia ixx="1e-6" ixy="0" ixz="0" iyy="1e-6" iyz="0" izz="1e-6" />
       </inertial>
     </link>
@@ -818,5 +818,5 @@
         <origin xyz="0 0 0" rpy="0 0 0" />
         <mass value="0.2556" />
-        <inertia ixx="0.0129" ixy="0" ixz="0" iyy="0.0095" iyz="0" izz="0.0184" />
+        <inertia ixx="0.0005" ixy="0" ixz="0" iyy="0.0005" iyz="0" izz="0.0005" />
       </inertial>
     </link>
@@ -834,5 +834,5 @@
         <origin xyz="0 0 0" rpy="0 0 0" />
         <mass value="0.001" />
-        <inertia ixx="0.1" ixy="0" ixz="0" iyy="0.1" iyz="0" izz="0.1" />
+        <inertia ixx="1e-6" ixy="0" ixz="0" iyy="1e-6" iyz="0" izz="1e-6" />
       </inertial>
     </link>
@@ -850,5 +850,5 @@
         <origin xyz="0 0 0" rpy="0 0 0" />
         <mass value="0.02087" />
-        <inertia ixx="0.0061" ixy="0" ixz="0" iyy="0.0014" iyz="0" izz="0.0061" />
+        <inertia ixx="0.00002" ixy="0" ixz="0" iyy="0.00002" iyz="0" izz="0.00002" />
       </inertial>
     </link>
@@ -866,5 +866,5 @@
         <origin xyz="0 0 0" rpy="0 0 0" />
         <mass value="0.001" />
-        <inertia ixx="0.1" ixy="0" ixz="0" iyy="0.1" iyz="0" izz="0.1" />
+        <inertia ixx="1e-6" ixy="0" ixz="0" iyy="1e-6" iyz="0" izz="1e-6" />
       </inertial>
     </link>
