Commit message: mmo500 wheel realistic movement + plan controller

File: CustomRobots/mmo500/models/mmo500/mmo500_common.urdf.xacro (robot description, xacro)
@@ -7,5 +7,5 @@
   <xacro:include filename="$(find robotiq_description)/urdf/robotiq_85_gripper.urdf.xacro"/>
   <xacro:include filename="$(find robotiq_description)/urdf/robotiq_85_gripper.ros2_control.xacro"/>
-  <!-- Wheels are fixed because the base is moved by VelocityControl -->
+  <!-- Passive wheels that roll on the floor while VelocityControl drives the base -->
   <xacro:macro name="omni_wheel" params="name xyz yaw">
     <link name="${name}_link">
@@ -25,8 +25,17 @@
       </collision>
     </link>
-    <joint name="${name}_joint" type="fixed">
+    <joint name="${name}_joint" type="continuous">
       <parent link="base_link"/>
       <child link="${name}_link"/>
       <origin xyz="${xyz}" rpy="0 0 ${yaw}"/>
+      <axis xyz="0 1 0"/>
+      <dynamics damping="0.01" friction="0.0"/>
+    </joint>
+    <xacro:rolling_wheel link="${name}_link"/>
+  </xacro:macro>
+  <xacro:macro name="wheel_state" params="name">
+    <joint name="${name}">
+      <state_interface name="position"/>
+      <state_interface name="velocity"/>
     </joint>
   </xacro:macro>
@@ -152,4 +161,14 @@
     <xacro:gpu_laser link="front_laser_link" name="front_laser" namespace="${namespace}"/>
     <xacro:gpu_laser link="back_laser_link" name="back_laser" namespace="${namespace}"/>
+    <!-- Wheels are state only because MoveIt waits for every joint of the URDF -->
+    <ros2_control name="mmo500_wheels" type="system">
+      <hardware>
+        <plugin>gz_ros2_control/GazeboSimSystem</plugin>
+      </hardware>
+      <xacro:wheel_state name="wheel_front_left_joint"/>
+      <xacro:wheel_state name="wheel_front_right_joint"/>
+      <xacro:wheel_state name="wheel_back_left_joint"/>
+      <xacro:wheel_state name="wheel_back_right_joint"/>
+    </ros2_control>
     <xacro:ros2_control_plugin namespace="${namespace}" simulation_controllers="${simulation_controllers}"/>
   </xacro:macro>

File: CustomRobots/mmo500/models/mmo500/mmo500_gz.urdf.xacro (robot description, xacro)
@@ -1,6 +1,6 @@
 <?xml version="1.0"?>
-<robot xmlns:xacro="http://ros.org/wiki/xacro">
-  <!-- Frictionless wheels so they only hold the base up while VelocityControl drives it -->
-  <xacro:macro name="frictionless" params="link">
+<robot xmlns:xacro="http://ros.org/wiki/xacro" xmlns:gz="http://gazebosim.org/schema">
+  <!-- Friction only across the wheel axis so the wheels roll and still slide sideways -->
+  <xacro:macro name="rolling_wheel" params="link">
     <gazebo reference="${link}">
       <collision>
@@ -9,5 +9,6 @@
             <ode>
               <mu>0.0</mu>
-              <mu2>0.0</mu2>
+              <mu2>1.0</mu2>
+              <fdir1 gz:expressed_in="${link}">0 1 0</fdir1>
             </ode>
           </friction>
@@ -16,8 +17,4 @@
     </gazebo>
   </xacro:macro>
-  <xacro:frictionless link="wheel_front_left_link"/>
-  <xacro:frictionless link="wheel_front_right_link"/>
-  <xacro:frictionless link="wheel_back_left_link"/>
-  <xacro:frictionless link="wheel_back_right_link"/>
   <xacro:macro name="velocity" params="namespace">
     <gazebo>
