Commit message: add myAGV + mechArm 270 robot, keep myCobot version as spare

File: CustomRobots/myagv_mecharm/models/myagv_mecharm/myagv_mecharm_common.urdf.xacro (robot description, xacro)
@@ -1,7 +1,5 @@
 <?xml version="1.0"?>
 <robot xmlns:xacro="http://ros.org/wiki/xacro">
-  <xacro:property name="mesh_dir" value="file://$(find custom_robots)/models/myagv_mycobot/meshes"/>
-  <!-- The myAGV and gripper meshes are shared with myagv_mecharm -->
-  <xacro:property name="shared_mesh_dir" value="file://$(find custom_robots)/models/myagv_mecharm/meshes"/>
+  <xacro:property name="mesh_dir" value="file://$(find custom_robots)/models/myagv_mecharm/meshes"/>
   <xacro:property name="wheel_radius" value="0.04"/>
   <xacro:property name="plate_top" value="0.1322"/>
@@ -12,10 +10,10 @@
   <!-- Arm folded over the base for driving and used as the SRDF home state -->
   <xacro:property name="home_j1" value="0.0"/>
-  <xacro:property name="home_j2" value="1.0"/>
-  <xacro:property name="home_j3" value="-2.3"/>
-  <xacro:property name="home_j4" value="-0.2"/>
-  <xacro:property name="home_j5" value="0.0"/>
+  <xacro:property name="home_j2" value="-0.1"/>
+  <xacro:property name="home_j3" value="0.2"/>
+  <xacro:property name="home_j4" value="0.0"/>
+  <xacro:property name="home_j5" value="1.5"/>
   <xacro:property name="home_j6" value="0.0"/>
-  <xacro:include filename="$(find custom_robots)/models/myagv_mycobot/myagv_mycobot_gz.urdf.xacro"/>
+  <xacro:include filename="$(find custom_robots)/models/myagv_mecharm/myagv_mecharm_gz.urdf.xacro"/>
   <material name="myagv_grey">
     <color rgba="0.25 0.25 0.27 1"/>
@@ -27,8 +25,8 @@
     <color rgba="0.08 0.08 0.08 1"/>
   </material>
-  <material name="mycobot_white">
+  <material name="arm_white">
     <color rgba="0.95 0.95 0.95 1"/>
   </material>
-  <material name="mycobot_grey">
+  <material name="arm_grey">
     <color rgba="0.6 0.6 0.6 1"/>
   </material>
@@ -68,5 +66,5 @@
       <visual>
         <geometry>
-          <mesh filename="${shared_mesh_dir}/myagv_${name}.stl"/>
+          <mesh filename="${mesh_dir}/myagv_${name}.stl"/>
         </geometry>
         <material name="myagv_wheel"/>
@@ -115,5 +113,5 @@
     </joint>
   </xacro:macro>
-  <xacro:macro name="myagv_mycobot" params="namespace simulation_controllers">
+  <xacro:macro name="myagv_mecharm" params="namespace simulation_controllers">
     <!-- myAGV 2023 base -->
     <link name="base_footprint"/>
@@ -126,5 +124,5 @@
       <visual>
         <geometry>
-          <mesh filename="${shared_mesh_dir}/myagv_body.stl"/>
+          <mesh filename="${mesh_dir}/myagv_body.stl"/>
         </geometry>
         <material name="myagv_grey"/>
@@ -132,5 +130,5 @@
       <visual>
         <geometry>
-          <mesh filename="${shared_mesh_dir}/myagv_top.stl"/>
+          <mesh filename="${mesh_dir}/myagv_top.stl"/>
         </geometry>
         <material name="myagv_plate"/>
@@ -167,5 +165,5 @@
       <origin xyz="0.13 0 0.131" rpy="0 0 0"/>
     </joint>
-    <!-- myCobot 280 Pi with the link and joint names of mycobot_description -->
+    <!-- mechArm 270 Pi with the link and joint names of mycobot_description -->
     <link name="g_base"/>
     <joint name="g_base_joint" type="fixed">
@@ -174,112 +172,112 @@
       <origin xyz="${arm_x} 0 ${plate_top}"/>
     </joint>
-    <xacro:mesh_link name="joint1" mesh="joint1_pi" material="mycobot_white"
-      vxyz="0 0 0" vrpy="0 0 0"
-      cxyz="-0.0013 0 0.0405" csize="0.0985 0.0926 0.0809"
-      mass="0.33" ixx="4.160e-04" iyy="4.466e-04" izz="5.027e-04"/>
-    <xacro:mesh_link name="joint2" mesh="joint2" material="mycobot_white"
-      vxyz="0 0 -0.06096" vrpy="0 0 -1.5708"
-      cxyz="0 -0.0063 -0.0206" csize="0.0480 0.0605 0.0871"
-      mass="0.12" ixx="1.124e-04" iyy="9.883e-05" izz="5.969e-05"/>
-    <xacro:mesh_link name="joint3" mesh="joint3" material="mycobot_white"
-      vxyz="0 0 0.03256" vrpy="0 -1.5708 0"
-      cxyz="-0.0540 0 0.0576" csize="0.1560 0.0480 0.0554"
-      mass="0.12" ixx="5.378e-05" iyy="2.741e-04" izz="2.664e-04"/>
-    <xacro:mesh_link name="joint4" mesh="joint4" material="mycobot_white"
-      vxyz="0 0 0.03056" vrpy="0 -1.5708 0"
-      cxyz="-0.0468 0 0.0065" csize="0.1368 0.0432 0.0578"
-      mass="0.10" ixx="4.339e-05" iyy="1.838e-04" izz="1.715e-04"/>
-    <xacro:mesh_link name="joint5" mesh="joint5" material="mycobot_white"
-      vxyz="0 -0.001 -0.0345" vrpy="0 -1.5708 1.5708"
-      cxyz="0.0001 -0.0095 -0.0081" csize="0.0386 0.0563 0.0528"
-      mass="0.08" ixx="3.974e-05" iyy="2.850e-05" izz="3.109e-05"/>
-    <xacro:mesh_link name="joint6" mesh="joint6" material="mycobot_white"
-      vxyz="0 0 -0.038" vrpy="0 0 0"
-      cxyz="0 0.0068 -0.0094" csize="0.0384 0.0567 0.0571"
-      mass="0.06" ixx="3.239e-05" iyy="2.369e-05" izz="2.345e-05"/>
-    <xacro:mesh_link name="joint6_flange" mesh="joint7" material="mycobot_grey"
-      vxyz="0 0 -0.012" vrpy="0 0 0"
-      cxyz="0 0 -0.0051" csize="0.0384 0.0384 0.0137"
-      mass="0.02" ixx="2.770e-06" iyy="2.770e-06" izz="4.915e-06"/>
-    <joint name="g_base_to_joint1" type="fixed">
+    <xacro:mesh_link name="base" mesh="mecharm_base" material="arm_white"
+      vxyz="0 0 0" vrpy="0 0 ${-pi}"
+      cxyz="-0.0050 0 0.0465" csize="0.1029 0.0929 0.0931"
+      mass="0.30" ixx="4.326e-04" iyy="4.816e-04" izz="4.808e-04"/>
+    <xacro:mesh_link name="link1" mesh="mecharm_link1" material="arm_white"
+      vxyz="0 0 -0.132" vrpy="0 0 0"
+      cxyz="-0.0005 0.0021 0.0160" csize="0.0900 0.0900 0.0911"
+      mass="0.15" ixx="2.050e-04" iyy="2.050e-04" izz="2.025e-04"/>
+    <xacro:mesh_link name="link2" mesh="mecharm_link2" material="arm_white"
+      vxyz="-0.005 0.21 0.002" vrpy="1.5708 ${-pi} 0"
+      cxyz="-0.0090 -0.0482 0.0018" csize="0.0679 0.1448 0.0920"
+      mass="0.15" ixx="3.680e-04" iyy="1.635e-04" izz="3.199e-04"/>
+    <xacro:mesh_link name="link3" mesh="mecharm_link3" material="arm_white"
+      vxyz="-0.09 0.306 0.005" vrpy="1.5708 ${pi} 0"
+      cxyz="0.0122 -0.0007 0.0015" csize="0.1100 0.0499 0.0728"
+      mass="0.12" ixx="7.794e-05" iyy="1.740e-04" izz="1.459e-04"/>
+    <xacro:mesh_link name="link4" mesh="mecharm_link4" material="arm_white"
+      vxyz="0.009 -0.311 -0.228" vrpy="0 1.5708 1.5708"
+      cxyz="-0.0021 -0.0009 -0.0150" csize="0.0640 0.0404 0.0718"
+      mass="0.10" ixx="5.659e-05" iyy="7.711e-05" izz="4.775e-05"/>
+    <xacro:mesh_link name="link5" mesh="mecharm_link5" material="arm_white"
+      vxyz="-0.292 -0.318 -0.007" vrpy="1.5708 0 ${pi}"
+      cxyz="0.0092 0 0.0010" csize="0.0844 0.0476 0.0480"
+      mass="0.08" ixx="3.046e-05" iyy="6.288e-05" izz="6.261e-05"/>
+    <xacro:mesh_link name="link6" mesh="mecharm_link6" material="arm_grey"
+      vxyz="-0.1645 0.0536 -0.211" vrpy="0 1.5708 0"
+      cxyz="-0.0010 0.0006 -0.0038" csize="0.0400 0.0400 0.0175"
+      mass="0.03" ixx="4.760e-06" iyy="4.756e-06" izz="7.989e-06"/>
+    <joint name="g_base_to_base" type="fixed">
       <parent link="g_base"/>
-      <child link="joint1"/>
+      <child link="base"/>
       <origin xyz="0 0 0" rpy="0 0 0"/>
     </joint>
+    <joint name="joint1_to_base" type="revolute">
+      <parent link="base"/>
+      <child link="link1"/>
+      <origin xyz="0 0 0.1" rpy="0 0 0"/>
+      <axis xyz="0 0 1"/>
+      <limit effort="${arm_effort}" lower="-2.7925" upper="2.7925" velocity="${arm_velocity}"/>
+    </joint>
     <joint name="joint2_to_joint1" type="revolute">
-      <parent link="joint1"/>
-      <child link="joint2"/>
-      <origin xyz="0 0 0.13956" rpy="0 0 0"/>
-      <axis xyz="0 0 1"/>
-      <limit effort="${arm_effort}" lower="-2.9321" upper="2.9321" velocity="${arm_velocity}"/>
+      <parent link="link1"/>
+      <child link="link2"/>
+      <origin xyz="0 0 0.038" rpy="-1.5708 0 0"/>
+      <axis xyz="0 0 1"/>
+      <limit effort="${arm_effort}" lower="-1.3089" upper="2.0943" velocity="${arm_velocity}"/>
     </joint>
     <joint name="joint3_to_joint2" type="revolute">
-      <parent link="joint2"/>
-      <child link="joint3"/>
-      <origin xyz="0 0 -0.001" rpy="0 1.5708 -1.5708"/>
-      <axis xyz="0 0 1"/>
-      <limit effort="${arm_effort}" lower="-2.4434" upper="2.4434" velocity="${arm_velocity}"/>
+      <parent link="link2"/>
+      <child link="link3"/>
+      <origin xyz="0 -0.1 0" rpy="0 0 0"/>
+      <axis xyz="0 0 1"/>
+      <limit effort="${arm_effort}" lower="-3.0543" upper="1.1344" velocity="${arm_velocity}"/>
     </joint>
     <joint name="joint4_to_joint3" type="revolute">
-      <parent link="joint3"/>
-      <child link="joint4"/>
-      <origin xyz="-0.1104 0 0" rpy="0 0 0"/>
-      <axis xyz="0 0 1"/>
-      <limit effort="${arm_effort}" lower="-2.6179" upper="2.6179" velocity="${arm_velocity}"/>
+      <parent link="link3"/>
+      <child link="link4"/>
+      <origin xyz="0.108 -0.005 -0.001" rpy="0 1.5708 0"/>
+      <axis xyz="0 0 1"/>
+      <limit effort="${arm_effort}" lower="-2.7052" upper="2.7052" velocity="${arm_velocity}"/>
     </joint>
     <joint name="joint5_to_joint4" type="revolute">
-      <parent link="joint4"/>
-      <child link="joint5"/>
-      <origin xyz="-0.096 0 0.06462" rpy="0 0 -1.5708"/>
-      <axis xyz="0 0 1"/>
-      <limit effort="${arm_effort}" lower="-2.6179" upper="2.6179" velocity="${arm_velocity}"/>
+      <parent link="link4"/>
+      <child link="link5"/>
+      <origin xyz="-0.001 0 0" rpy="0 -1.5708 0"/>
+      <axis xyz="0 0 1"/>
+      <limit effort="${arm_effort}" lower="-2.0071" upper="2.0071" velocity="${arm_velocity}"/>
     </joint>
     <joint name="joint6_to_joint5" type="revolute">
-      <parent link="joint5"/>
-      <child link="joint6"/>
-      <origin xyz="0 -0.07318 -0.001" rpy="1.5708 -1.5708 0"/>
-      <axis xyz="0 0 1"/>
-      <limit effort="${arm_effort}" lower="-2.7052" upper="2.7925" velocity="${arm_velocity}"/>
-    </joint>
-    <joint name="joint6output_to_joint6" type="revolute">
-      <parent link="joint6"/>
-      <child link="joint6_flange"/>
-      <origin xyz="0 0.0456 0" rpy="-1.5708 0 0"/>
-      <axis xyz="0 0 1"/>
-      <limit effort="${arm_effort}" lower="-3.14159" upper="3.14159" velocity="${arm_velocity}"/>
+      <parent link="link5"/>
+      <child link="link6"/>
+      <origin xyz="0.06 0 0" rpy="0 1.5708 0"/>
+      <axis xyz="0 0 1"/>
+      <limit effort="${arm_effort}" lower="-3.14" upper="3.14" velocity="${arm_velocity}"/>
     </joint>
     <!-- Adaptive gripper where one joint drives the whole linkage -->
-    <xacro:mesh_link name="gripper_base" mesh="gripper_base" material="gripper_black" dir="${shared_mesh_dir}"
+    <xacro:mesh_link name="gripper_base" mesh="gripper_base" material="gripper_black"
       vxyz="0 0 -0.012" vrpy="0 0 0"
       cxyz="0 -0.0012 0.0123" csize="0.0580 0.0622 0.0509"
       mass="0.06" ixx="3.232e-05" iyy="2.977e-05" izz="3.618e-05"/>
-    <xacro:mesh_link name="gripper_left1" mesh="gripper_left1" material="gripper_black" dir="${shared_mesh_dir}"
+    <xacro:mesh_link name="gripper_left1" mesh="gripper_left1" material="gripper_black"
       vxyz="0.039 -0.0133 -0.012" vrpy="0 0 0"
       cxyz="0.0065 0.0241 -0.0082" csize="0.0244 0.0582 0.0207"
       mass="0.01" ixx="3.178e-06" iyy="8.535e-07" izz="3.320e-06"/>
-    <xacro:mesh_link name="gripper_left2" mesh="gripper_left2" material="gripper_black" dir="${shared_mesh_dir}"
+    <xacro:mesh_link name="gripper_left2" mesh="gripper_left2" material="gripper_black"
       vxyz="0.005 -0.0195 -0.012" vrpy="0 0 0"
       cxyz="-0.0145 0.0075 -0.0082" csize="0.0359 0.0243 0.0200"
       mass="0.01" ixx="8.251e-07" iyy="1.409e-06" izz="1.567e-06"/>
-    <xacro:mesh_link name="gripper_left3" mesh="gripper_left3" material="gripper_black" dir="${shared_mesh_dir}"
+    <xacro:mesh_link name="gripper_left3" mesh="gripper_left3" material="gripper_black"
       vxyz="0.012 0.0025 -0.012" vrpy="0 0 0"
       cxyz="-0.0097 0.0025 -0.0007" csize="0.0450 0.0335 0.0050"
       mass="0.01" ixx="9.578e-07" iyy="1.711e-06" izz="2.627e-06"/>
-    <xacro:mesh_link name="gripper_right1" mesh="gripper_right1" material="gripper_black" dir="${shared_mesh_dir}"
+    <xacro:mesh_link name="gripper_right1" mesh="gripper_right1" material="gripper_black"
       vxyz="-0.039 -0.0133 -0.012" vrpy="0 0 0"
       cxyz="-0.0078 0.0245 -0.0082" csize="0.0244 0.0582 0.0207"
       mass="0.01" ixx="3.178e-06" iyy="8.535e-07" izz="3.320e-06"/>
-    <xacro:mesh_link name="gripper_right2" mesh="gripper_right2" material="gripper_black" dir="${shared_mesh_dir}"
+    <xacro:mesh_link name="gripper_right2" mesh="gripper_right2" material="gripper_black"
       vxyz="-0.005 -0.0195 -0.012" vrpy="0 0 0"
       cxyz="0.0134 0.0077 -0.0082" csize="0.0357 0.0247 0.0200"
       mass="0.01" ixx="8.407e-07" iyy="1.397e-06" izz="1.571e-06"/>
-    <xacro:mesh_link name="gripper_right3" mesh="gripper_right3" material="gripper_black" dir="${shared_mesh_dir}"
+    <xacro:mesh_link name="gripper_right3" mesh="gripper_right3" material="gripper_black"
       vxyz="-0.012 0.0025 -0.012" vrpy="0 0 0"
       cxyz="0.0085 0.0027 -0.0007" csize="0.0450 0.0339 0.0050"
       mass="0.01" ixx="9.801e-07" iyy="1.706e-06" izz="2.645e-06"/>
     <joint name="joint6output_to_gripper_base" type="fixed">
-      <parent link="joint6_flange"/>
+      <parent link="link6"/>
       <child link="gripper_base"/>
-      <origin xyz="0 0 0.034" rpy="1.579 0 0"/>
+      <origin xyz="0 0 0.038" rpy="1.579 0 0"/>
     </joint>
     <joint name="gripper_base_to_gripper_left3" type="revolute">
@@ -343,14 +341,14 @@
     <xacro:camera link="camera_link" namespace="${namespace}"/>
     <xacro:suction_contact link="gripper_left1"/>
-    <ros2_control name="mycobot" type="system">
+    <ros2_control name="mecharm" type="system">
       <hardware>
         <plugin>gz_ros2_control/GazeboSimSystem</plugin>
       </hardware>
-      <xacro:arm_joint_control name="joint2_to_joint1" lower="-2.9321" upper="2.9321" initial="${home_j1}"/>
-      <xacro:arm_joint_control name="joint3_to_joint2" lower="-2.4434" upper="2.4434" initial="${home_j2}"/>
-      <xacro:arm_joint_control name="joint4_to_joint3" lower="-2.6179" upper="2.6179" initial="${home_j3}"/>
-      <xacro:arm_joint_control name="joint5_to_joint4" lower="-2.6179" upper="2.6179" initial="${home_j4}"/>
-      <xacro:arm_joint_control name="joint6_to_joint5" lower="-2.7052" upper="2.7925" initial="${home_j5}"/>
-      <xacro:arm_joint_control name="joint6output_to_joint6" lower="-3.14159" upper="3.14159" initial="${home_j6}"/>
+      <xacro:arm_joint_control name="joint1_to_base" lower="-2.7925" upper="2.7925" initial="${home_j1}"/>
+      <xacro:arm_joint_control name="joint2_to_joint1" lower="-1.3089" upper="2.0943" initial="${home_j2}"/>
+      <xacro:arm_joint_control name="joint3_to_joint2" lower="-3.0543" upper="1.1344" initial="${home_j3}"/>
+      <xacro:arm_joint_control name="joint4_to_joint3" lower="-2.7052" upper="2.7052" initial="${home_j4}"/>
+      <xacro:arm_joint_control name="joint5_to_joint4" lower="-2.0071" upper="2.0071" initial="${home_j5}"/>
+      <xacro:arm_joint_control name="joint6_to_joint5" lower="-3.14" upper="3.14" initial="${home_j6}"/>
       <xacro:arm_joint_control name="gripper_base_to_gripper_left3" lower="-0.74" upper="0.15" initial="0.0"/>
       <xacro:mimic_joint_control name="gripper_base_to_gripper_left2" multiplier="1.0"/>
